File: av3/straingauge/straingaugerev0.brd (EAGLE design)
At the start: 160 x 100 mm, 36 parts, among them IC1 AD8655RM, U1 AD8290

Commit message: components placed but signals not routed
Parts:
- removed C12: 100nF, rcl:C0402
- removed C14: 10uF, rcl:C0805
- removed C15: 68nF, rcl:C0402
- removed U$1: LT3060, straingauge:TSOT-23-8
- removed U$2: AD7685, straingauge:MSOP-10
- removed U$6: ADR4525, straingauge:SOIC-8
- added C2: 100nF, rcl:C0402
- added TP11, TP12: TEST-POINT, straingauge:2MM-TEST-POINT
- added U2: AD7685, straingauge:MSOP-10
- added U5: LT3060, straingauge:TSOT-23-8
- added U6: ADR4525, straingauge:SOIC-8
- moved R3 250.7 mm to (48.5, 36.9)
- moved X3 223.9 mm to (14.0, 36.0)
- moved X1 219.6 mm to (37.0, 27.0), turned to 270 degrees
- moved X2 197.3 mm to (21.0, 5.00), turned to 180 degrees
- moved C10 113.5 mm to (17.9, 31.0), turned to 180 degrees
- moved C5 112.2 mm to (28.3, 24.7)
- moved C4 109.6 mm to (28.8, 27.0)
- moved C3 100.1 mm to (18.0, 29.0)
- moved C1 94.6 mm to (50.3, 18.7)
- moved C8 94.6 mm to (59.1, 23.8)
- moved C9 94.6 mm to (50.3, 13.6)
- moved R1 94.6 mm to (50.3, 8.52)
- moved R2 94.6 mm to (50.3, 3.44)
- moved C13 90.2 mm to (11.0, 27.0), turned to 180 degrees
- moved C11 81.8 mm to (11.0, 25.9)
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Connections:
- net N$1 renamed RSET
- net N$10 renamed V1
- net N$5 renamed CF1
- net N$6 renamed CF2
- net N$7 renamed VINP
- net N$8 renamed VINN
- net N$9 renamed V+
- removed net N$11: C9.2, IC1.2, IC1.6, TP1.1, U$2.3
- removed net N$12: C11.1, U$1.5
- removed net N$13: U$2.9, X1.2
- removed net N$14: U$2.6, X1.1
- removed net N$16: C13.2, U$1.6
- removed net N$17: U$2.4
- removed net N$2: U$2.8, X1.4
- removed net N$3: TP2.1, U$2.1, U$6.6
- removed net N$4: U$2.7, X1.3
- removed net VDD: U$2.2
- removed net VIN: U$6.2
- new net +3V3: C10.1, C13.1, C2.1, C3.1, R3.2, TP7.1, U1.2, U5.7, X3.4
- new net ADJ: C13.2, U5.6
- new net AGND: C1.2, C6.2, C7.2, IC1.4, R5.1, TP5.1, TP6.1, U1.10, U2.4, U6.4, X2.3
- new net CNV: U2.6, X1.1
- new net DGND: TP12.1, U2.5
- new net IN+: C9.2, IC1.2, IC1.6, TP1.1, U2.3
- new net NA: C11.2
- new net REF: TP2.1, U2.1, U6.6
- new net REFB: C11.1, U5.5
- new net SCK: U2.8, X1.4
- new net SDI: U2.9, X1.2
- new net SDO: U2.7, X1.3
- net 3V3: now also U2.10, U2.2, U6.2; no longer C10.1, C12.1, C13.1, C14.1, C3.1, R3.2, TP7.1, U$1.7, U$2.10, U1.2
- net ENBL: no longer X3.3
- net GND: now also C2.2, C5.2, U5.2, U5.3, U5.4, X3.1; no longer C1.2, C11.2, C12.2, C14.2, C15.2, C6.2, C7.2, IC1.4, R5.1, TP5.1, TP6.1, U$1.2, U$1.3, U$1.4, U$2.5, U$6.4, U1.10, X2.3
- net VCC: now also U5.1, U5.8, X3.3; no longer U$1.1, U$1.8, X3.1
- net VOUT: now also TP11.1; no longer C15.1
Routing:
- net AGND: track 0.00 -> 9.13 mm
- added copper zone on layer 1, net AGND
- added copper zone on layer 16, net AGND
- added copper zone on layer 1, net DGND
- added copper zone on layer 1, net GND
Other:
- board size 160 x 100 mm -> 42 x 41 mm
