File: av3/straingauge/straingaugerev0.sch (EAGLE design)
At the start: 36 parts, among them IC1 AD8655RM, U1 AD8290

Commit message: schematic is ready for a design review
Parts:
- removed C12: 100nF, rcl:C-EUC0402
- removed C14: 10uF, rcl:C-EUC0805
- removed C15: 68nF, rcl:C-EUC0402
- removed U$1: LT3060, straingauge:LT3060
- removed U$2: AD7685, straingauge:AD7685
- removed U$6: ADR4525, straingauge:ADR4525
- added C2: 100nF, rcl:C-EUC0402
- added TP11, TP12: TEST-POINT, straingauge:TEST-POINT
- added U2: AD7685, straingauge:AD7685
- added U5: LT3060, straingauge:LT3060
- added U6: ADR4525, straingauge:ADR4525
Connections:
- net N$1 renamed RSET
- net N$10 renamed V1
- net N$5 renamed CF1
- net N$6 renamed CF2
- net N$7 renamed VINP
- net N$8 renamed VINN
- net N$9 renamed V+
- removed net N$11: C9.2, IC1.IN-, IC1.OUT, TP1.1, U$2.IN+
- removed net N$12: C11.1, U$1.REFB
- removed net N$13: U$2.SDI, X1-2.1
- removed net N$14: U$2.CNV, X1-1.1
- removed net N$16: C13.2, U$1.ADJ
- removed net N$17: U$2.IN-
- removed net N$2: U$2.SCK, X1-4.1
- removed net N$3: TP2.1, U$2.REF, U$6.VOUT
- removed net N$4: U$2.SDO, X1-3.1
- new net +3V3: C10.1, C13.1, C2.1, C3.1, R3.2, TP7.1, U1.VCC, U5.OUT, X3-4.1
- new net ADJ: C13.2, U5.ADJ
- new net AGND: C1.2, C6.2, C7.2, IC1.-VS, R5.1, TP5.1, TP6.1, U1.GND, U2.IN-, U6.GND, X2-3.1
- new net CNV: U2.CNV, X1-1.1
- new net DGND: TP12.1, U2.GND
- new net IN+: C9.2, IC1.IN-, IC1.OUT, TP1.1, U2.IN+
- new net NA: C11.2
- new net REF: TP2.1, U2.REF, U6.VOUT
- new net REFB: C11.1, U5.REFB
- new net SCK: U2.SCK, X1-4.1
- new net SDI: U2.SDI, X1-2.1
- new net SDO: U2.SDO, X1-3.1
- net 3V3: now also U2.VDD, U2.VIO, U6.VIN; no longer C10.1, C12.1, C13.1, C14.1, C3.1, R3.2, TP7.1, U$1.OUT, U$2.VIO, U1.VCC
- net ENBL: no longer X3-3.1
- net GND: now also C2.2, C5.2, U5.GND, U5.GND@1, U5.GND@2, X3-1.1; no longer C1.2, C11.2, C12.2, C14.2, C15.2, C6.2, C7.2, IC1.-VS, R5.1, TP5.1, TP6.1, U$1.GND, U$1.GND@1, U$1.GND@2, U$2.GND, U$6.GND, U1.GND, X2-3.1
- net VCC: now also U5.!SHTDN, U5.IN, X3-3.1; no longer U$1.!SHTDN, U$1.IN, X3-1.1
- net VOUT: now also TP11.1; no longer C15.1
Other:
- note added: "ADC"
- note added: "Differential voltage"
- note added: "Power"
- note added: "SG Amplifier"
- note added: "Voltage Reference"
- note added: "from strain gauge"
- note added: "use different gnd syb"
- note removed: "Anti-aliasing filter"
- note removed: "Differential voltage from strain gauge."
- note removed: "Strain Gauge Bridge"
- note removed: "Use a "star" topology with the power to limit noise from the digital and the power circuitry."
- note removed: "is 68nF antialiasing filter necessary with the sallen key low pass filter?"
- note removed: "what power and data line connectors should be used"
- moved on the sheet: C1, C10, C11, C13, C3, C4, C5, C6, C7, C8, C9, IC1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
