File: av3/rf-power/rf-power.brd (EAGLE design)
At the start: 63.5 x 50.8 mm, 26 parts, among them J1 CON-2MM-4X1, J2 CON-2MM-5X1, Q3 PMV45EN, Q5 PMV45EN, U1 UEI15, U2 UEI15, U3 IC-CPC1302GS

Commit message: Changed "from ATV" connector to 0.1" euroterminal because I'm paranoid. Moved SPSs up to deal with euroterminals. ERCed and DRCed.
Parts:
- removed J2: CON-2MM-5X1, Tova:2MM-5X1
- added X3: 22-23-2051, con-molex:22-23-2051
- moved C3 13.7 mm to (22.1, 15.2), turned to 270 degrees
- moved C5 3.39 mm to (45.0, 31.8), turned to 180 degrees
- moved J1 2.03 mm to (50.3, 42.4)
- moved U3 1.27 mm to (7.87, 23.9)
- moved R2 1.27 mm to (4.06, 32.0)
- moved R8 1.27 mm to (9.14, 32.0)
- moved R6 1.02 mm to (14.2, 13.0), turned to 90 degrees
- moved C1 0.57 mm to (37.3, 11.2)
- moved C4 0.51 mm to (17.5, 33.0)
- moved U1 0.51 mm to (46.0, 23.9)
- moved U2 0.51 mm to (17.5, 23.9)
- moved X1 0.51 mm to (31.8, 6.35), turned to 180 degrees
- moved Q3 0.51 mm to (56.1, 30.2)
- moved Q5 0.51 mm to (27.7, 30.2)
- moved R1 0.51 mm to (39.6, 13.7)
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Connections:
- net 12V-ATV-OUT: now also X1.3, X3.3; no longer J2.3, X1.2
- net 12V-WIFI-OUT: now also X1.1; no longer X1.4
- net AUDIO: now also X3.2; no longer J2.2
- net GND: now also X1.2, X1.4, X3.1; no longer J2.1, X1.1, X1.3
- net VBATT: now also X3.5; no longer J2.5
- net VIDEO: now also X3.4; no longer J2.4
Routing:
- net VBATT: track 74.6 -> 81.0 mm, vias 2 -> 1
- net 12V-ATV-OUT: track 91.2 -> 94.5 mm
- net 12V-WIFI-OUT: track 11.7 -> 13.0 mm
- net ATV-CTRL: track 11.6 -> 10.3 mm
- net ISO-GND: track 29.5 -> 28.2 mm
- net VIDEO: track 18.2 -> 18.9 mm
Other:
- board text added: "12"
- board text added: "V"

Commit message: Added pulldown resistors on Nch mosfets to protect them from excessively high system voltage.
Parts:
- added R10, R9: 10k, rcl_custom:0805-C-NOSILK
Connections:
- net GND: now also R10.1, R9.1
- net N$6: now also R9.2
- net N$8: now also R10.2
Changed lines of the file:
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@@
 <attribute name="OC_FARNELL" value="1462952" x="36.068" y="41.402" size="1.778" layer="27" display="off"/>
 </element>
+<element name="R9" library="rcl_custom" package="0805-C-NOSILK" value="10k" x="1.524" y="-2.54"/>
+<element name="R10" library="rcl_custom" package="0805-C-NOSILK" value="10k" x="1.524" y="-7.366"/>
 </elements>
 <signals>
@@
 <contactref element="X1" pad="4"/>
 <contactref element="X1" pad="2"/>
+<contactref element="R9" pad="1"/>
+<contactref element="R10" pad="1"/>
+<wire x1="0.724" y1="-2.54" x2="0.724" y2="-7.366" width="0" layer="19" extent="1-1"/>
+<wire x1="10.414" y1="2.032" x2="0.724" y2="-2.54" width="0" layer="19" extent="1-1"/>
 </signal>
 <signal name="12V-WIFI-OUT">
@@
 <wire x1="56.896" y1="24.384" x2="56.896" y2="26.886" width="0.508" layer="16"/>
 <wire x1="56.896" y1="26.886" x2="56.934" y2="26.924" width="0.508" layer="16"/>
+<contactref element="R9" pad="2"/>
+<wire x1="2.324" y1="-2.54" x2="4.064" y2="19.4272" width="0" layer="19" extent="1-16"/>
 </signal>
 <signal name="N$8">
@@
 <wire x1="26.416" y1="22.606" x2="28.74" y2="24.93" width="0.508" layer="16"/>
 <wire x1="28.74" y1="26.924" x2="28.74" y2="24.93" width="0.508" layer="16"/>
+<contactref element="R10" pad="2"/>
+<wire x1="2.324" y1="-7.366" x2="9.144" y2="19.4272" width="0" layer="19" extent="1-16"/>
 </signal>
 <signal name="N$1">
