File: av3/rf-power/rf-power.sch (EAGLE design)
At the start: 22 parts, among them J1 CON-2MM-4X1, J2 CON-2MM-5X1, Q3 PMV45EN, Q5 PMV45EN, U1 UEI15, U2 UEI15, U3 IC-CPC1302GS, X1 22-23-2041, X2 22-23-2021, X4 22-23-2041

Commit message: Changed "from ATV" connector to 0.1" euroterminal because I'm paranoid. Moved SPSs up to deal with euroterminals. ERCed and DRCed.
Parts:
- removed J2: CON-2MM-5X1, Tova:CON-2MM-5X1
- added X3: 22-23-2051, con-molex:22-23-2051
Connections:
- net 12V-ATV-OUT: now also X1-3.S, X3-3.S; no longer J2.3, X1-2.S
- net 12V-WIFI-OUT: now also X1-1.S; no longer X1-4.S
- net AUDIO: now also X3-2.S; no longer J2.2
- net GND: now also X1-2.S, X1-4.S, X3-1.S; no longer J2.1, X1-1.S, X1-3.S
- net VBATT: now also X3-5.S; no longer J2.5
- net VIDEO: now also X3-4.S; no longer J2.4
Other:
- note added: "(SPARE)"
- moved on the sheet: X1-1, X1-2, X1-3, X1-4
Changed lines of the file:
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@@
 <setting verticaltext="up"/>
 </settings>
-<grid distance="0.05" unitdist="inch" unit="inch" style="lines" multiple="2" display="yes" altdistance="0.01" altunitdist="inch" altunit="inch"/>
+<grid distance="0.1" unitdist="inch" unit="inch" style="lines" multiple="1" display="yes" altdistance="0.01" altunitdist="inch" altunit="inch"/>
 <layers>
 <layer number="1" name="Top" color="4" fill="1" visible="no" active="no"/>
@@
 <part name="J1" library="2mmx4" deviceset="CON-2MM-4X1" device=""/>
 <part name="SUPPLY9" library="supply2" deviceset="GND" device=""/>
-<part name="J2" library="Tova" deviceset="CON-2MM-5X1" device=""/>
 <part name="C1" library="rcl_custom" deviceset="C-EU" device="1206-B" value="33uF"/>
 <part name="C3" library="rcl_custom" deviceset="C-EU" device="1206-B" value="33uF"/>
@@
 <part name="SUPPLY16" library="supply2" deviceset="GND" device=""/>
 <part name="SUPPLY17" library="supply2" deviceset="GND" device=""/>
+<part name="X3" library="con-molex" deviceset="22-23-2051" device=""/>
 </parts>
 <sheets>
@@
 <text x="132.08" y="176.53" size="1.778" layer="97">ATV PASS THROUGH</text>
 <text x="162.56" y="149.86" size="1.778" layer="97">TO TRANSMITTER</text>
-<text x="162.56" y="162.56" size="1.778" layer="97">FROM CAMERA/DVR/GFE/OVERLAY</text>
+<text x="167.64" y="162.56" size="1.778" layer="97">FROM CAMERA/DVR/GFE/OVERLAY</text>
+<text x="238.76" y="58.42" size="1.778" layer="97" rot="R90">(SPARE)</text>
 </plain>
 <instances>
 <instance part="SUPPLY1" gate="GND" x="218.44" y="58.42"/>
-<instance part="X1" gate="-1" x="223.52" y="63.5"/>
-<instance part="X1" gate="-2" x="223.52" y="68.58"/>
-<instance part="X1" gate="-3" x="223.52" y="119.38"/>
-<instance part="X1" gate="-4" x="223.52" y="124.46"/>
+<instance part="X1" gate="-1" x="223.52" y="124.46"/>
+<instance part="X1" gate="-2" x="223.52" y="119.38"/>
+<instance part="X1" gate="-3" x="223.52" y="68.58"/>
+<instance part="X1" gate="-4" x="223.52" y="63.5"/>
 <instance part="SUPPLY2" gate="GND" x="218.44" y="114.3"/>
 <instance part="X2" gate="-1" x="43.18" y="116.84" rot="R180"/>
@@
 <instance part="J1" gate="G$1" x="157.48" y="152.4"/>
 <instance part="SUPPLY9" gate="GND" x="152.4" y="142.24"/>
-<instance part="J2" gate="G$1" x="157.48" y="167.64"/>
 <instance part="C1" gate="CE" x="210.82" y="121.92"/>
 <instance part="C3" gate="CE" x="210.82" y="66.04"/>
@@
 <instance part="SUPPLY16" gate="GND" x="139.7" y="111.76"/>
 <instance part="SUPPLY17" gate="GND" x="139.7" y="55.88"/>
+<instance part="X3" gate="-1" x="157.48" y="170.18"/>
+<instance part="X3" gate="-2" x="157.48" y="167.64"/>
+<instance part="X3" gate="-3" x="157.48" y="165.1"/>
+<instance part="X3" gate="-4" x="157.48" y="162.56"/>
+<instance part="X3" gate="-5" x="157.48" y="160.02"/>
 </instances>
 <busses>
@@
 <net name="GND" class="0">
 <segment>
+<wire x1="218.44" y1="63.5" x2="218.44" y2="60.96" width="0.1524" layer="91"/>
+<pinref part="SUPPLY1" gate="GND" pin="GND"/>
+<pinref part="X1" gate="-4" pin="S"/>
 <wire x1="220.98" y1="63.5" x2="218.44" y2="63.5" width="0.1524" layer="91"/>
-<wire x1="218.44" y1="63.5" x2="218.44" y2="60.96" width="0.1524" layer="91"/>
-<pinref part="X1" gate="-1" pin="S"/>
-<pinref part="SUPPLY1" gate="GND" pin="GND"/>
-</segment>
-<segment>
+</segment>
+<segment>
+<wire x1="218.44" y1="119.38" x2="218.44" y2="116.84" width="0.1524" layer="91"/>
+<pinref part="SUPPLY2" gate="GND" pin="GND"/>
+<pinref part="X1" gate="-2" pin="S"/>
 <wire x1="220.98" y1="119.38" x2="218.44" y2="119.38" width="0.1524" layer="91"/>
-<wire x1="218.44" y1="119.38" x2="218.44" y2="116.84" width="0.1524" layer="91"/>
-<pinref part="X1" gate="-3" pin="S"/>
-<pinref part="SUPPLY2" gate="GND" pin="GND"/>
 </segment>
 <segment>
@@
 <wire x1="152.4" y1="154.94" x2="154.94" y2="154.94" width="0.1524" layer="91"/>
 <label x="149.86" y="154.94" size="1.778" layer="95" rot="MR0"/>
-<pinref part="J2" gate="G$1" pin="1"/>
 <label x="149.86" y="170.18" size="1.778" layer="95" rot="MR0"/>
 <wire x1="152.4" y1="170.18" x2="154.94" y2="170.18" width="0.1524" layer="91"/>
 <wire x1="152.4" y1="154.94" x2="152.4" y2="170.18" width="0.1524" layer="91"/>
 <junction x="152.4" y="154.94"/>
+<pinref part="X3" gate="-1" pin="S"/>
 </segment>
 <segment>
@@
 <segment>
 <pinref part="U1" gate="G$1" pin="VOUT"/>
-<pinref part="X1" gate="-4" pin="S"/>
 <wire x1="190.5" y1="124.46" x2="203.2" y2="124.46" width="0.1524" layer="91"/>
 <pinref part="R1" gate="R" pin="2"/>
@@
 <junction x="203.2" y="124.46"/>
 <pinref part="C1" gate="CE" pin="1"/>
-<wire x1="210.82" y1="124.46" x2="220.98" y2="124.46" width="0.1524" layer="91"/>
+<pinref part="X1" gate="-1" pin="S"/>
+<wire x1="220.98" y1="124.46" x2="210.82" y2="124.46" width="0.1524" layer="91"/>
 <junction x="210.82" y="124.46"/>
 </segment>
@@
 <segment>
 <pinref part="U2" gate="G$1" pin="VOUT"/>
-<pinref part="X1" gate="-2" pin="S"/>
 <wire x1="190.5" y1="68.58" x2="203.2" y2="68.58" width="0.1524" layer="91"/>
 <pinref part="R5" gate="R" pin="2"/>
@@
 <junction x="203.2" y="68.58"/>
 <pinref part="J1" gate="G$1" pin="3"/>
-<wire x1="210.82" y1="68.58" x2="220.98" y2="68.58" width="0.1524" layer="91"/>
 <wire x1="154.94" y1="149.86" x2="129.54" y2="149.86" width="0.1524" layer="91"/>
 <wire x1="129.54" y1="149.86" x2="129.54" y2="137.16" width="0.1524" layer="91"/>
@@
 <wire x1="243.84" y1="86.36" x2="203.2" y2="86.36" width="0.1524" layer="91"/>
 <wire x1="203.2" y1="86.36" x2="203.2" y2="68.58" width="0.1524" layer="91"/>
-<pinref part="J2" gate="G$1" pin="3"/>
 <wire x1="154.94" y1="165.1" x2="129.54" y2="165.1" width="0.1524" layer="91"/>
 <wire x1="129.54" y1="165.1" x2="129.54" y2="149.86" width="0.1524" layer="91"/>
@@
 <label x="149.86" y="165.1" size="1.778" layer="95" rot="MR0"/>
 <pinref part="C3" gate="CE" pin="1"/>
+<pinref part="X3" gate="-3" pin="S"/>
+<pinref part="X1" gate="-3" pin="S"/>
+<wire x1="220.98" y1="68.58" x2="210.82" y2="68.58" width="0.1524" layer="91"/>
 <junction x="210.82" y="68.58"/>
 </segment>
@@
 <wire x1="134.62" y1="55.88" x2="134.62" y2="66.04" width="0.1524" layer="91"/>
 <junction x="134.62" y="66.04"/>
-<pinref part="J2" gate="G$1" pin="5"/>
 <wire x1="154.94" y1="160.02" x2="66.04" y2="160.02" width="0.1524" layer="91"/>
 <wire x1="66.04" y1="160.02" x2="66.04" y2="121.92" width="0.1524" layer="91"/>
@@
 <pinref part="C5" gate="CE" pin="1"/>
 <junction x="139.7" y="66.04"/>
+<pinref part="X3" gate="-5" pin="S"/>
 </segment>
 </net>
@@
 <wire x1="154.94" y1="152.4" x2="127" y2="152.4" width="0.1524" layer="91"/>
 <wire x1="127" y1="152.4" x2="127" y2="167.64" width="0.1524" layer="91"/>
-<pinref part="J2" gate="G$1" pin="2"/>
 <wire x1="127" y1="167.64" x2="154.94" y2="167.64" width="0.1524" layer="91"/>
 <label x="149.86" y="152.4" size="1.778" layer="95" rot="MR0"/>
 <label x="149.86" y="167.64" size="1.778" layer="95" rot="MR0"/>
+<pinref part="X3" gate="-2" pin="S"/>
 </segment>
 </net>
 <net name="VIDEO" class="0">
 <segment>
-<pinref part="J2" gate="G$1" pin="4"/>
 <wire x1="154.94" y1="162.56" x2="124.46" y2="162.56" width="0.1524" layer="91"/>
 <wire x1="124.46" y1="162.56" x2="124.46" y2="147.32" width="0.1524" layer="91"/>
@@
 <label x="149.86" y="147.32" size="1.778" layer="95" rot="MR0"/>
 <label x="149.86" y="162.56" size="1.778" layer="95" rot="MR0"/>
-</segment>
-</net>
+<pinref part="X3" gate="-4" pin="S"/>
+</segment>
+</net>

Commit message: Added pulldown resistors on Nch mosfets to protect them from excessively high system voltage.
Parts:
- added R10, R9: 10k, rcl_custom:R-US_0805-C-NOSILK
Connections:
- net GND: now also R10.1, R9.1
- net N$6: now also R9.2
- net N$8: now also R10.2
Other:
- note added: "PMV45EN has a Vgs breakdown of 20 V"
- note added: "V/2 voltage divider protects Vgs"
Changed lines of the file:
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@@
 <setting verticaltext="up"/>
 </settings>
-<grid distance="0.1" unitdist="inch" unit="inch" style="lines" multiple="1" display="yes" altdistance="0.01" altunitdist="inch" altunit="inch"/>
+<grid distance="0.1" unitdist="inch" unit="inch" style="lines" multiple="1" display="no" altdistance="0.01" altunitdist="inch" altunit="inch"/>
 <layers>
 <layer number="1" name="Top" color="4" fill="1" visible="no" active="no"/>
@@
 <part name="SUPPLY17" library="supply2" deviceset="GND" device=""/>
 <part name="X3" library="con-molex" deviceset="22-23-2051" device=""/>
+<part name="R9" library="rcl_custom" deviceset="R-US_" device="0805-C-NOSILK" value="10k"/>
+<part name="R10" library="rcl_custom" deviceset="R-US_" device="0805-C-NOSILK" value="10k"/>
+<part name="SUPPLY18" library="supply2" deviceset="GND" device=""/>
+<part name="SUPPLY19" library="supply2" deviceset="GND" device=""/>
 </parts>
 <sheets>
@@
 <text x="167.64" y="162.56" size="1.778" layer="97">FROM CAMERA/DVR/GFE/OVERLAY</text>
 <text x="238.76" y="58.42" size="1.778" layer="97" rot="R90">(SPARE)</text>
+<text x="114.3" y="25.4" size="1.778" layer="97">PMV45EN has a Vgs breakdown of 20 V</text>
+<text x="114.3" y="22.86" size="1.778" layer="97">V/2 voltage divider protects Vgs</text>
 </plain>
 <instances>
@@
 <instance part="X3" gate="-4" x="157.48" y="162.56"/>
 <instance part="X3" gate="-5" x="157.48" y="160.02"/>
+<instance part="R9" gate="R" x="134.62" y="96.52" rot="R90"/>
+<instance part="R10" gate="R" x="134.62" y="40.64" rot="R90"/>
+<instance part="SUPPLY18" gate="GND" x="134.62" y="88.9"/>
+<instance part="SUPPLY19" gate="GND" x="134.62" y="33.02"/>
 </instances>
 <busses>
@@
 <pinref part="C5" gate="CE" pin="2"/>
 <pinref part="SUPPLY17" gate="GND" pin="GND"/>
+</segment>
+<segment>
+<pinref part="R9" gate="R" pin="1"/>
+<pinref part="SUPPLY18" gate="GND" pin="GND"/>
+</segment>
+<segment>
+<pinref part="R10" gate="R" pin="1"/>
+<pinref part="SUPPLY19" gate="GND" pin="GND"/>
 </segment>
 </net>
@@
 <junction x="134.62" y="101.6"/>
 <wire x1="129.54" y1="101.6" x2="134.62" y2="101.6" width="0.1524" layer="91"/>
+<pinref part="R9" gate="R" pin="2"/>
 </segment>
 </net>
@@
 <pinref part="U3" gate="G$1" pin="C2"/>
 <wire x1="129.54" y1="83.82" x2="121.92" y2="83.82" width="0.1524" layer="91"/>
-</segment>
-</net>
+<pinref part="R10" gate="R" pin="2"/>
+</segment>
+</net>
