File: av3/battery-board/battery-board.brd (EAGLE design)
At the start: 71.2 x 35.2 mm, 72 parts, among them J100 87758-0216, J101 87758-0216, Q100 SI4435DDY, Q101 SI4435DDY, Q102 SI4435DDY, Q103 SI1023X, Q104 SI1023X, U100 BQ3060PW, X1 22-23-2041, X2 22-23-2041

Commit message: Bob's changes to the battery board - fully routed! Hooray.
Parts:
- moved R102 52.0 mm to (21.6, 16.7), turned to 270 degrees
- moved C101 51.2 mm to (21.4, 12.8)
- moved R108 49.6 mm to (2.51, 20.1), turned to 270 degrees
- moved Q103 48.6 mm to (24.0, 15.7), turned to 90 degrees
- moved R107 45.3 mm to (1.32, 14.2), turned to 270 degrees
- moved R105 44.3 mm to (26.7, 17.2)
- moved C102 44.0 mm to (24.7, 13.0), turned to 90 degrees
- moved R116 42.7 mm to (27.1, 23.9), turned to 180 degrees
- moved R111 42.6 mm to (21.7, 23.6), turned to 270 degrees
- moved R109 42.3 mm to (26.2, 13.0), turned to 270 degrees
- moved Q104 40.3 mm to (24.0, 23.3), turned to 90 degrees
- moved C114 40.2 mm to (24.3, 20.5), turned to 90 degrees
- moved R110 39.2 mm to (23.1, 12.9), turned to 90 degrees
- moved R119 37.8 mm to (25.9, 20.4), turned to 270 degrees
- moved C105 37.1 mm to (21.7, 19.6), turned to 90 degrees
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Routing:
- net TRIANGLE_GND: track 15.9 -> 113.7 mm, vias 0 -> 3
- net N$29: track 12.4 -> 85.3 mm, vias 0 -> 1
- net N$30: track 12.9 -> 80.0 mm, vias 0 -> 1
- net B+: track 15.4 -> 71.2 mm, vias 0 -> 3
- net N$43: track 8.97 -> 60.7 mm, vias 0 -> 2
- net N$19: track 12.1 -> 60.3 mm, vias 1 -> 2
- net N$27: track 10.1 -> 50.5 mm
- net BAR_GND: track 15.7 -> 55.9 mm, vias 14 -> 4
- net N$10: track 10.5 -> 46.4 mm, vias 1 -> 4
- net N$11: track 9.66 -> 43.0 mm, vias 1 -> 4
- net N$12: track 11.3 -> 41.4 mm, vias 2 -> 4
- net N$36: track 1.92 -> 24.5 mm
- net N$22: track 0.00 -> 18.9 mm
- net N$25: track 0.00 -> 14.2 mm, vias 0 -> 1
- net N$4: track 33.1 -> 46.7 mm, vias 1 -> 3
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Other:
- board size 71.2 x 35.2 mm -> 71.2 x 35.3 mm
