File: av3/battery-board/battery-board.brd (EAGLE design)
At the start: 76.7 x 63.9 mm, 72 parts, among them J100 87758-0216, J101 87758-0216, Q100 SI4435DDY, Q101 SI4435DDY, Q102 SI4435DDY, Q103 SI1023X, Q104 SI1023X, U100 BQ3060PW, X1 22-23-2041, X2 22-23-2041

Commit message: Added blank battery board, used to laser cut out the back plate. Added latest "short" (4S1P) version of the battery sensor board. Added the battery breakout board, which adds a fuse to the battery. Added LPKF CAM job. Fixed bottom trestrict in mount.lbr
Parts:
- R100: device rcl_custom:0603-B-NOSILK -> rcl_custom:1206-B
- moved C101 78.6 mm to (48.6, -30.5), turned to 90 degrees
- moved R102 73.7 mm to (47.8, -28.2), turned to 0 degrees
- moved Q103 70.5 mm to (48.6, -26.2), turned to 180 degrees
- moved C102 66.6 mm to (47.8, -24.4), turned to 0 degrees
- moved R109 64.4 mm to (48.6, -22.9), turned to 180 degrees
- moved R105 61.6 mm to (48.6, -21.4), turned to 180 degrees
- moved R106 61.4 mm to (42.7, -12.2), turned to 90 degrees
- moved C108 58.9 mm to (66.1, 30.5), turned to 0 degrees
- moved D103 58.0 mm to (62.0, 38.5), turned to 90 degrees
- moved R113 57.8 mm to (66.1, 32.1), turned to 180 degrees
- moved D105 57.0 mm to (66.1, 33.7), turned to 180 degrees
- moved C110 56.7 mm to (63.0, 23.4), turned to 0 degrees
- moved TP106 56.5 mm to (62.7, 19.1), turned to 180 degrees
- moved TP108 56.5 mm to (60.5, 44.3), turned to 180 degrees
- moved TP100 56.5 mm to (42.7, -9.72), turned to 180 degrees
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Routing:
- net B+: track 110.1 -> 15.4 mm, vias 2 -> 0
- net N$32: track 80.9 -> 8.97 mm
- net N$39: track 52.9 -> 1.91 mm
- net TRIANGLE_GND: track 64.6 -> 15.9 mm, vias 2 -> 0
- net N$36: track 43.3 -> 1.92 mm
- net N$27: track 48.4 -> 10.1 mm, vias 0 -> 1
- net N$34: track 39.3 -> 3.72 mm
- net N$23: track 41.5 -> 5.98 mm, vias 2 -> 0
- net N$19: track 43.9 -> 12.1 mm, vias 0 -> 1
- net N$10: track 39.3 -> 10.5 mm, vias 0 -> 1
- net N$16: track 29.3 -> 4.86 mm, vias 2 -> 0
- net N$29: track 36.3 -> 12.4 mm
- net N$2: track 30.2 -> 6.41 mm, vias 2 -> 0
- net N$15: track 21.1 -> 0.00 mm
- net N$7: track 7.86 -> 23.6 mm
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- removed copper zone on layer 1, net N$4
- removed copper zone on layer 1, net N$7
- removed copper zone on layer 1, net N$8
Other:
- board size 76.7 x 63.9 mm -> 71.2 x 35.2 mm

Commit message: Small changes to layout, including routing final airwires, moved 2nd layer ground plane.
Parts:
- moved R102 52.0 mm to (21.6, 16.7), turned to 270 degrees
- moved C101 51.2 mm to (21.4, 12.8)
- moved R108 49.6 mm to (2.51, 20.1), turned to 270 degrees
- moved Q103 48.6 mm to (24.0, 15.7), turned to 90 degrees
- moved R107 45.3 mm to (1.32, 14.2), turned to 270 degrees
- moved R105 44.3 mm to (26.7, 17.2)
- moved C102 44.0 mm to (24.7, 13.0), turned to 90 degrees
- moved R116 42.7 mm to (27.1, 23.9), turned to 180 degrees
- moved R111 42.6 mm to (21.7, 23.6), turned to 270 degrees
- moved R109 42.3 mm to (26.2, 13.0), turned to 270 degrees
- moved Q104 40.3 mm to (24.0, 23.3), turned to 90 degrees
- moved C114 40.2 mm to (24.3, 20.5), turned to 90 degrees
- moved R110 39.2 mm to (23.1, 12.9), turned to 90 degrees
- moved R119 37.8 mm to (25.9, 20.4), turned to 270 degrees
- moved C105 37.1 mm to (21.7, 19.6), turned to 90 degrees
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Routing:
- net TRIANGLE_GND: track 15.9 -> 113.7 mm, vias 0 -> 3
- net N$29: track 12.4 -> 85.3 mm, vias 0 -> 1
- net N$30: track 12.9 -> 80.0 mm, vias 0 -> 1
- net B+: track 15.4 -> 71.2 mm, vias 0 -> 3
- net N$43: track 8.97 -> 60.7 mm, vias 0 -> 2
- net BAR_GND: track 15.7 -> 64.3 mm, vias 14 -> 6
- net N$19: track 12.1 -> 60.3 mm, vias 1 -> 2
- net N$27: track 10.1 -> 50.5 mm
- net N$10: track 10.5 -> 46.4 mm, vias 1 -> 4
- net N$11: track 9.66 -> 43.0 mm, vias 1 -> 4
- net N$12: track 11.3 -> 41.4 mm, vias 2 -> 4
- net N$36: track 1.92 -> 24.5 mm
- net N$22: track 0.00 -> 18.9 mm
- net N$25: track 0.00 -> 14.2 mm, vias 0 -> 1
- net N$4: track 33.1 -> 46.7 mm, vias 1 -> 3
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Other:
- board size 71.2 x 35.2 mm -> 71.2 x 35.3 mm

Commit message: Various changes to daughterboards, including updating libraries, etc. ISSUE: Connectors still flipped on "bottom" of boards.
Parts:
- removed X1, X2: 22-23-2041, con-molex:22-23-2041
- added J1: ROCKETNET-BATTERY-14, rocketnet-connector:ROCKETNET-CONNECTOR-M-14
- C101, C102, C105, C109, C111, C112, C113, C114, R101, R102, R103, R104, R106, R107, R108, R109, R111, R119, R120, R121: device rcl_custom:0603-B-NOSILK -> rcl_custom:0402-B-NOSILK
- R100: value 301 -> 301 1W
- R105, R110, R116, R122: value 100 -> 100 .25W
- moved C108 32.8 mm to (48.8, 33.3), turned to 90 degrees
- moved C107 29.9 mm to (53.1, 33.3), turned to 90 degrees
- moved C106 28.0 mm to (57.4, 33.3), turned to 90 degrees
- moved C105 26.9 mm to (47.8, 13.4), turned to 0 degrees
- moved C101 26.5 mm to (47.8, 10.6), turned to 0 degrees
- moved R118 26.1 mm to (56.6, 31.0)
- moved TP100 25.7 mm to (52.2, 23.1), turned to 0 degrees
- moved D105 25.5 mm to (47.2, 33.3)
- moved R115 25.2 mm to (52.3, 31.0)
- moved R113 25.2 mm to (48.0, 31.0)
- moved D103 24.5 mm to (55.8, 33.3)
- moved C114 24.1 mm to (47.8, 15.2), turned to 0 degrees
- moved D104 24.1 mm to (51.5, 33.3)
- moved C102 23.2 mm to (47.8, 12.4), turned to 0 degrees
- moved TP101 19.8 mm to (56.0, 14.3), turned to 0 degrees
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Connections:
- net N$41 renamed PRE-CHARGE
- removed net N$26: F100.2, X1.1, X1.2
- new net B+PACKOUT: F100.2, J1.B+@1, J1.B+@2, J1.B+@3, J1.B+@4
- net N$22: now also J1.SMDAT@7, J1.SMDAT@8; no longer X2.3
- net N$25: now also J1.SMCLK@3, J1.SMCLK@4; no longer X2.2
- net N$35: now also J1.!PRSNT@10, J1.!PRSNT@9; no longer X2.1
- net TRIANGLE_GND: now also J1.B-@11, J1.B-@12, J1.B-@13, J1.B-@14; no longer X1.3, X1.4, X2.4
Routing:
- net TRIANGLE_GND: track 113.7 -> 47.7 mm, vias 3 -> 1
- net BAR_GND: track 64.3 -> 26.2 mm, vias 6 -> 15
- net B+: track 71.2 -> 46.3 mm, vias 3 -> 1
- net N$4: track 46.7 -> 22.3 mm, vias 3 -> 0
- net N$25: track 14.2 -> 37.5 mm
- net N$22: track 18.9 -> 39.8 mm, vias 0 -> 1
- net N$35: track 8.83 -> 29.4 mm, vias 0 -> 1
- net N$24: track 7.83 -> 26.4 mm, vias 2 -> 0
- net N$17: track 6.48 -> 24.9 mm
- net N$19: track 60.3 -> 43.2 mm, vias 2 -> 0
- net N$33: track 11.7 -> 26.6 mm, vias 2 -> 0
- net N$36: track 24.5 -> 10.7 mm
- net N$40: track 1.37 -> 14.5 mm
- net N$30: track 80.0 -> 91.2 mm
- net N$45: track 15.0 -> 4.50 mm
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- added copper zone on layer 1, net B+PACKOUT
- added copper zone on layer 16, net BAR_GND
- added copper zone on layer 1, net PRE-CHARGE
- removed copper zone on layer 1, net N$26
Other:
- board text added: "2013/05/01"
- board text added: "PSAS Battery Board v1"
