File: av3/battery-board/battery-board.sch (EAGLE design)
At the start: 72 parts, among them J100 87758-0216, J101 87758-0216, Q100 SI4435DDY, Q101 SI4435DDY, Q102 SI4435DDY, Q103 SI1023X, Q104 SI1023X, U100 BQ3060PW, X1 22-23-2041, X2 22-23-2041

Commit message: Added blank battery board, used to laser cut out the back plate. Added latest "short" (4S1P) version of the battery sensor board. Added the battery breakout board, which adds a fuse to the battery. Added LPKF CAM job. Fixed bottom trestrict in mount.lbr
Parts:
- R100: device rcl_custom:R-US_0603-B-NOSILK -> rcl_custom:R-US_1206-B
Changed lines of the file:
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@@
 <part name="R104" library="rcl_custom" deviceset="R-US_" device="0603-B-NOSILK" value="1M"/>
 <part name="R101" library="rcl_custom" deviceset="R-US_" device="0603-B-NOSILK" value="1M"/>
-<part name="R100" library="rcl_custom" deviceset="R-US_" device="0603-B-NOSILK" value="301"/>
+<part name="R100" library="rcl_custom" deviceset="R-US_" device="1206-B" value="301"/>
 <part name="B103A" library="battery" deviceset="LIPO-8AHR" device=""/>
 <part name="B102A" library="battery" deviceset="LIPO-8AHR" device=""/>
@@
 <wire x1="83.82" y1="190.5" x2="83.82" y2="195.58" width="1.27" layer="91"/>
 <wire x1="83.82" y1="190.5" x2="101.6" y2="190.5" width="0.1524" layer="91"/>
-<wire x1="82.55" y1="180.34" x2="85.09" y2="180.34" width="1.27" layer="91"/>
+<wire x1="82.55" y1="180.34" x2="83.82" y2="180.34" width="1.27" layer="91"/>
+<wire x1="83.82" y1="180.34" x2="85.09" y2="180.34" width="1.27" layer="91"/>
 <wire x1="83.82" y1="180.34" x2="85.09" y2="180.34" width="1.27" layer="91"/>
 <wire x1="83.82" y1="180.34" x2="83.82" y2="190.5" width="1.27" layer="91"/>
@@
 <pinref part="C116" gate="CE" pin="1"/>
 <pinref part="R103" gate="R" pin="1"/>
+<junction x="83.82" y="180.34"/>
 </segment>
 </net>
@@
 <wire x1="101.6" y1="162.56" x2="101.6" y2="165.1" width="0.1524" layer="91"/>
 <wire x1="83.82" y1="154.94" x2="83.82" y2="165.1" width="1.27" layer="91"/>
-<wire x1="82.55" y1="172.72" x2="85.09" y2="172.72" width="1.27" layer="91"/>
+<wire x1="82.55" y1="172.72" x2="83.82" y2="172.72" width="1.27" layer="91"/>
+<wire x1="83.82" y1="172.72" x2="85.09" y2="172.72" width="1.27" layer="91"/>
 <wire x1="85.09" y1="172.72" x2="83.82" y2="172.72" width="1.27" layer="91"/>
 <wire x1="83.82" y1="165.1" x2="83.82" y2="172.72" width="1.27" layer="91"/>
@@
 <pinref part="B103A" gate="G$1" pin="B-@1"/>
 <pinref part="B103A" gate="G$1" pin="B-@2"/>
-</segment>
-</net>
+<junction x="83.82" y="172.72"/>
+</segment>
+</net>

Commit message: Small changes to layout, including routing final airwires, moved 2nd layer ground plane.
Other:
- moved on the sheet: B100A, B101A, B102A, B103A, C100, C106, C107, C108, C109, C110, C111, C112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

Commit message: Various changes to daughterboards, including updating libraries, etc. ISSUE: Connectors still flipped on "bottom" of boards.
Parts:
- removed X1, X2: 22-23-2041, con-molex:22-23-2041
- added J1: ROCKETNET-BATTERY-14, rocketnet-connector:ROCKETNET-BATTERY-14
- C101, C102, C105, C109, C111, C112, C113, C114: device rcl_custom:C-EU0603-B-NOSILK -> rcl_custom:C-EU0402-B-NOSILK
- R100: value 301 -> 301 1W
- R101, R102, R103, R104, R106, R107, R108, R109, R111, R119, R120, R121: device rcl_custom:R-US_0603-B-NOSILK -> rcl_custom:R-US_0402-B-NOSILK
- R105, R110, R116, R122: value 100 -> 100 .25W
Connections:
- net N$41 renamed PRE-CHARGE
- removed net N$26: F100.2, X1-1.S, X1-2.S
- new net B+PACKOUT: F100.2, J1.B+@1, J1.B+@2, J1.B+@3, J1.B+@4
- net N$22: now also J1.SMDAT@1, J1.SMDAT@2; no longer X2-3.S
- net N$25: now also J1.SMCLK@1, J1.SMCLK@2; no longer X2-2.S
- net N$35: now also J1.!PRSNT@1, J1.!PRSNT@2; no longer X2-1.S
- net TRIANGLE_GND: now also J1.B-@1, J1.B-@2, J1.B-@3, J1.B-@4; no longer X1-3.S, X1-4.S, X2-4.S
