File: av3/rocketnet-hub/eagle/node_conn.sch (EAGLE design)
At the start: 63 parts, among them J1 ROCKETBUS, J2 ROCKETBUS, J3 ROCKETBUS, J4 ROCKETBUS, J5 ROCKETBUS, J6 ROCKETBUS, J7 ROCKETBUS, J8 ROCKETBUS, X1 87758-0416, X2 87758-0416, X3 87758-0416, X4 87758-0416, X5 87758-0416, X6 87758-0416, X7 87758-0416, X8 87758-0416

Commit message: Updated TPS2420 components in node_conn and renamed INOM to IMON in TPS2420 library
Parts:
- added C1, C2, C3, C4, C5, C6, C7: (no value), rcl:C-EUC0402K
- added R11, R12, R13, R14, R15, R16, R17, R18, R19, R20, R21, R22, R23, R24: (no value), rcl:R-US_R0402
Connections:
- net NODE1_EN renamed NODE1_!EN
- net NODE1_FLT renamed NODE1_!FLT
- net NODE1_\P\G renamed NODE1_!PG
- net PD11 renamed NODE2_!FLT
- net PD16 renamed NODE2_!EN
- net PD17 renamed NODE3_!FLT
- net PD18 renamed NODE3_!EN
- net PD19 renamed NODE4_!FLT
- net PD20 renamed NODE4_!EN
- net PD21 renamed NODE5_!FLT
- net PD22 renamed NODE5_!EN
- net PD23 renamed NODE6_!FLT
- net PD24 renamed NODE7_!FLT
- net PD25 renamed NODE7_!EN
- net PD26 renamed NODE8_!FLT
- net PD27 renamed NODE8_!EN
- net PD28 renamed NODE6_!EN
- net VBAT renamed +18V
- removed net +UB: C13.1, C14.1, C15.1, C16.1, C17.1, C18.1, U$11.AD0, U$11.VDD, U$12.AD0, U$12.AD1, U$12.VDD, U$13.AD1, U$13.VDD
- removed net NODE1_INOM: R1.2, U$2.INOM
- removed net NODE2_LED: LED2.A, R2.1
- removed net NODE3_ILIM: U$11.W1, U$4.IMAX
- removed net NODE3_LED: LED3.A, R3.1
- removed net NODE4_LED: LED4.A, R4.1
- removed net NODE5_ILIM: U$13.W1, U$6.IMAX
- removed net NODE5_LED: LED5.A, R5.1
- removed net NODE6_LED: LED6.A, R6.1
- removed net NODE7_ILIM: U$12.W1, U$8.IMAX
- removed net NODE7_LED: LED7.A, R7.1
- removed net NODE8_LED: LED8.A, R8.1
- new net N$1: LED2.A, R3.1
- new net N$12: LED6.A, R13.1
- new net N$13: LED7.A, R15.1
- new net N$2: LED3.A, R5.1
- new net N$23: LED8.A, R17.1
- new net N$24: C1.1
- new net N$26: R21.2
- new net N$29: R22.2
- new net N$30: R23.2
- new net N$31: R24.2
- new net N$32: U$13.W1, U$6.IFLT
- new net N$33: C2.1, U$4.CT
- new net N$34: C3.1, U$6.CT
- new net N$35: C4.1, U$5.CT
- new net N$36: C5.1, U$7.CT
- new net N$37: C6.1, U$8.CT
- new net N$38: C7.1, U$9.CT
- new net N$4: LED4.A, R7.1
- new net N$40: U$11.W1, U$4.IFLT
- new net N$41: R19.2
- new net N$43: R20.2
- new net N$44: U$12.W1, U$8.IFLT
- new net N$48: R18.2, U$3.IMAX
- new net N$5: LED5.A, R11.1
- new net NODE1_IMON: R1.2, U$2.IMON
- new net NODE2_!PG: LED2.C, U$3.!PG
- new net NODE2_IMON: R2.2, U$3.IMON
- new net NODE2_LTCH: U$3.LTCH
- new net NODE2_RXM: J2.USB_L@1, J2.USB_L@2
- new net NODE2_RXP: J2.USB_H@1, J2.USB_H@2
- new net NODE2_TXM: J2.CAN_L@1, J2.CAN_L@2
- new net NODE2_TXP: J2.CAN_H@1, J2.CAN_H@2
- new net NODE3_!PG: LED3.C, U$4.!PG
- new net NODE3_IMON: R4.2, U$4.IMON
- new net NODE3_LTCH: U$4.LTCH
- new net NODE3_RXM: J3.USB_L@1, J3.USB_L@2
- new net NODE3_RXP: J3.USB_H@1, J3.USB_H@2
- new net NODE3_TXM: J3.CAN_L@1, J3.CAN_L@2
- new net NODE3_TXP: J3.CAN_H@1, J3.CAN_H@2
- new net NODE4_!PG: LED5.C, U$5.!PG
- new net NODE4_IMON: R8.2, U$5.IMON
- new net NODE4_LTCH: U$5.LTCH
- new net NODE4_RXM: J4.USB_L@1, J4.USB_L@2
- new net NODE4_RXP: J4.USB_H@1, J4.USB_H@2
- new net NODE4_TXM: J4.CAN_L@1, J4.CAN_L@2
- new net NODE4_TXP: J4.CAN_H@1, J4.CAN_H@2
- new net NODE5_!PG: LED4.C, U$6.!PG
- new net NODE5_IMON: R6.2, U$6.IMON
- new net NODE5_LTCH: U$6.LTCH
- new net NODE5_RXM: J5.USB_L@1, J5.USB_L@2
- new net NODE5_RXP: J5.USB_H@1, J5.USB_H@2
- new net NODE5_TXM: J5.CAN_L@1, J5.CAN_L@2
- new net NODE5_TXP: J5.CAN_H@1, J5.CAN_H@2
- new net NODE6_!PG: LED6.C, U$7.!PG
- new net NODE6_IMON: R12.2, U$7.IMON
- new net NODE6_LTCH: U$7.LTCH
- new net NODE6_RXM: J6.USB_L@1, J6.USB_L@2
- new net NODE6_RXP: J6.USB_H@1, J6.USB_H@2
- new net NODE6_TXM: J6.CAN_L@1, J6.CAN_L@2
- new net NODE6_TXP: J6.CAN_H@1, J6.CAN_H@2
- new net NODE7_!PG: LED7.C, U$8.!PG
- new net NODE7_IMON: R14.2, U$8.IMON
- new net NODE7_LTCH: U$8.LTCH
- new net NODE7_RXM: J7.USB_L@1, J7.USB_L@2
- new net NODE7_RXP: J7.USB_H@1, J7.USB_H@2
- new net NODE7_TXM: J7.CAN_L@1, J7.CAN_L@2
- new net NODE7_TXP: J7.CAN_H@1, J7.CAN_H@2
- new net NODE8_!PG: LED8.C, U$9.!PG
- new net NODE8_IMON: R16.2, U$9.IMON
- new net NODE8_LTCH: U$9.LTCH
- new net NODE8_RXM: J8.USB_L@1, J8.USB_L@2
- new net NODE8_RXP: J8.USB_H@1, J8.USB_H@2
- new net NODE8_TXM: J8.CAN_L@1, J8.CAN_L@2
- new net NODE8_TXP: J8.CAN_H@1, J8.CAN_H@2
- net +3V3: now also C13.1, C14.1, C15.1, C16.1, C17.1, C18.1, R11.2, R13.2, R15.2, R17.2, R3.2, R5.2, R7.2, U$11.AD0, U$11.VDD, U$12.AD0, U$12.AD1, U$12.VDD, U$13.AD1, U$13.VDD
- net GND: now also C1.2, C2.2, C3.2, C4.2, C5.2, C6.2, C7.2, R12.1, R14.1, R16.1, R18.1, R19.1, R2.1, R20.1, R21.1, R22.1, R23.1, R24.1, R4.1, R6.1, R8.1; no longer LED2.C, LED3.C, LED4.C, LED5.C, LED6.C, LED7.C, LED8.C
- net NODE2_ILIM: now also U$3.IFLT; no longer U$3.IMAX
- net NODE2_VOUT: no longer R2.2
- net NODE3_VOUT: no longer R3.2
- net NODE4_ILIM: now also U$5.IFLT; no longer U$5.IMAX
- net NODE4_VOUT: no longer R4.2
- net NODE5_VOUT: no longer R5.2
- net NODE6_ILIM: now also U$7.IFLT; no longer U$7.IMAX
- net NODE6_VOUT: no longer R6.2
- net NODE7_VOUT: no longer R7.2
- net NODE8_ILIM: now also U$9.IFLT; no longer U$9.IMAX
- net NODE8_VOUT: no longer R8.2
- net SCL: now also U$11.SCL, U$12.SCL, U$13.SCL
- net SDA: now also U$11.SDA, U$12.SDA, U$13.SDA
Other:
- moved on the sheet: C13, C14, C15, C16, C17, C18, C20, C21, C23, C24, C25, C26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

Commit message: updated mcu, eth, and connector schematics.
Parts:
- removed C12, C13, C14, C15: 0.1u, rcl:C-EUC0402
- removed C16, C17, C18, C19: 1u, rcl:C-EUC0603K
- removed U$10, U$11, U$12, U$13: AD5248MSOP-10, RNH_AD5248:AD5248MSOP-10
Connections:
- removed net NODE2_ILIM: U$10.W2, U$3.IFLT
- removed net NODE4_ILIM: U$11.W2, U$5.IFLT
- removed net NODE6_ILIM: U$13.W2, U$7.IFLT
- removed net SCL: U$10.SCL, U$11.SCL, U$12.SCL, U$13.SCL
- removed net SDA: U$10.SDA, U$11.SDA, U$12.SDA, U$13.SDA
- new net N$25: U$3.IFLT
- new net N$39: U$5.IFLT
- new net N$42: U$7.IFLT
- net +3V3: no longer C12.1, C13.1, C14.1, C15.1, C16.1, C17.1, C18.1, C19.1, U$10.VDD, U$11.AD0, U$11.VDD, U$12.AD0, U$12.AD1, U$12.VDD, U$13.AD1, U$13.VDD
- net GND: no longer C12.2, C13.2, C14.2, C15.2, C16.2, C17.2, C18.2, C19.2, U$10.AD0, U$10.AD1, U$10.B1, U$10.B2, U$10.GND, U$11.AD1, U$11.B1, U$11.B2, U$11.GND, U$12.B1, U$12.B2, U$12.GND, U$13.AD0, U$13.B1, U$13.B2, U$13.GND
- net N$32: no longer U$13.W1
- net N$40: no longer U$11.W1
- net N$44: no longer U$12.W1
- net NODE1_ILIM: no longer U$10.W1
- net NODE8_ILIM: no longer U$12.W2
