File: av3/rocketnet-hub/eagle/batterycharger_page.sch (EAGLE design)
At the start: 10 parts

Commit message: Added more datasheets; added two mosfet parts
Parts:
- removed D2: BAT54C, diode:BAT54C
- removed L1: (no value), rcl_custom:L-US0603-B
- added C10, C11, C12, C13, C14, C15, C16, C17, C18, C19, C20, C21, C22, C23, C24, C25, C26, C4, C5, C6, C7, C8, C9: (no value), rcl_custom:C-USC0603
- added D3: BAT54C, diode:BAT54C
- added JP1, JP2, JP3: (no value), pinhead:PINHD-1X3
- added JP4, JP5: (no value), pinhead:PINHD-1X2
- added L2: (no value), rcl_custom:L-US0603-B
- added R10, R11: 4.02k, rcl_custom:R-US_0603-B
- added R12: 66.5k, rcl_custom:R-US_0603-B
- added R13, R15, R16: 430k, rcl_custom:R-US_0603-B
- added R14: 10, rcl_custom:R-US_0603-B
- added R17, R18, R19, R20, R22, R23: (no value), rcl_custom:R-US_0603-B
- added R21, R24, R8: 12.1k, rcl_custom:R-US_0603-B
- added R4: 100k, rcl_custom:R-US_0603-B
- added R5: 316k, rcl_custom:R-US_0603-B
- added R9: 10k, rcl_custom:R-US_0603-B
- added U$2: BSS138W-7-F, RNH_BSS138W-7-F:BSS138W-7-F
- R1: value (none) -> 12.1k
Connections:
- removed net N$5: C3.2
- new net N$10: R8.2, R9.1, U$1.ACOK
- new net N$11: R11.1, U$1.CMSRC
- new net N$12: D3.CC, R14.2
- new net N$13: D3.A1, JP4.1
- new net N$14: R3.2, U$1.SRN
- new net N$15: C7.1, C8.1, D3.A2, JP5.1, R13.2
- new net N$16: R17.2, U$1.SRP
- new net N$17: C7.2, R15.2, R16.2
- new net N$18: C2.1, C9.1, L2.2, R17.1, R19.2
- new net N$19: C12.1, C25.1, C26.2, C3.1, C9.2, JP3.2, R19.1, R24.1, R3.1
- new net N$20: C10.1, D1.A, U$1.REGN
- new net N$21: R18.2, U$1.BTST
- new net N$22: C11.1, D1.C, R18.1
- new net N$23: C17.1, C18.1, R1.1, U$1.ACN
- new net N$24: C26.1, R2.1, R24.2
- new net N$25: C19.1, C20.1, C21.1, C23.1, C24.1, JP3.3, R1.2, R20.1
- new net N$26: C15.1, U$1.LODRV
- new net N$27: C13.1, C14.1, C17.2, R20.2, U$1.ACP
- new net N$29: C16.1, U$1.HIDRV
- new net N$32: R22.1, R23.2, U$2.G\
- new net N$33: C22.1, R11.2, R21.2, R23.1, U$2.S
- new net N$34: C22.2, C8.2, R10.2, R21.1, U$2.D
- new net N$6: C5.1, U$1.IOUT
- new net N$7: C6.1, R12.2, R13.1, U$1.ACDET
- new net N$9: R10.1, U$1.ACDRV
- new net SCL: JP1.3, U$1.SCL
- new net SDA: JP1.2, U$1.SDA
- net GND: now also C10.2, C12.2, C13.2, C14.2, C15.2, C18.2, C19.2, C20.2, C21.2, C23.2, C24.2, C25.2, C3.2, C4.2, C5.2, C6.2, JP1.1, JP3.1, JP5.2, R12.1, R15.1, R16.1, R22.2, R4.1, R8.1, U$1.GND
- net N$1: now also U$1.VCC; no longer R1.1
- net N$2: now also R2.2, U$1.BATDRV; no longer D2.CC, R1.2
- net N$3: now also C4.1, R4.2, R5.1, U$1.ILIM; no longer C2.1, D1.A
- net N$4: now also C11.2, C16.2, L2.1, U$1.PHASE; no longer C3.1, D1.C
Other:
- note added: "PSAS Rocketnet Hub Battery Charger Schematic"
- note added: "v1"
- moved on the sheet: C1, C2, C3, D1, R1, R2, R3

Commit message: Modified part symbols to look more like FETs
Parts:
- added U$3, U$4, U$5: FDS6680ASOIC-8, RNH_FDS6680A:FDS6680ASOIC-8
Connections:
- net N$19: now also U$5.S@1, U$5.S@3
- net N$24: now also U$5.G
- net N$33: now also U$3.S@1, U$3.S@2, U$3.S@3, U$4.S@1, U$4.S@2, U$4.S@3
- net N$34: now also U$3.G, U$4.G
Changed lines of the file:
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@@
 <?xml version="1.0" encoding="utf-8"?>
 <!DOCTYPE eagle SYSTEM "eagle.dtd">
-<eagle version="6.3">
+<eagle version="6.4">
 <drawing>
 <settings>
@@
 <part name="SUPPLY25" library="supply2" deviceset="GND" device=""/>
 <part name="C1" library="rcl_custom" deviceset="C-US" device="C0603"/>
+<part name="FRAME1" library="frames" deviceset="FRAME_B_L" device=""/>
 <part name="U$2" library="RNH_BSS138W-7-F" deviceset="BSS138W-7-F" device=""/>
-<part name="FRAME1" library="frames" deviceset="FRAME_B_L" device=""/>
+<part name="U$3" library="RNH_FDS6680A" deviceset="FDS6680A" device="SOIC-8"/>
+<part name="U$4" library="RNH_FDS6680A" deviceset="FDS6680A" device="SOIC-8"/>
+<part name="U$5" library="RNH_FDS6680A" deviceset="FDS6680A" device="SOIC-8"/>
 </parts>
 <sheets>
@@
 <instance part="SUPPLY25" gate="GND" x="129.54" y="27.94"/>
 <instance part="C1" gate="C" x="-15.24" y="33.02"/>
-<instance part="U$2" gate="G$1" x="-43.18" y="104.14" rot="R270"/>
 <instance part="FRAME1" gate="G$1" x="-205.74" y="-106.68"/>
 <instance part="FRAME1" gate="G$2" x="119.38" y="-106.68"/>
+<instance part="U$2" gate="G$1" x="-50.8" y="109.22"/>
+<instance part="U$3" gate="G$1" x="-81.28" y="76.2" rot="R90"/>
+<instance part="U$4" gate="G$1" x="-30.48" y="76.2" rot="MR90"/>
+<instance part="U$5" gate="G$1" x="109.22" y="71.12" rot="MR0"/>
 </instances>
 <busses>
@@
 <wire x1="-91.44" y1="81.28" x2="-86.36" y2="81.28" width="0.2032" layer="91"/>
 <junction x="-91.44" y="81.28"/>
+<wire x1="-86.36" y1="78.74" x2="-86.36" y2="81.28" width="0.2032" layer="91"/>
 </segment>
 </net>
@@
 <pinref part="C26" gate="C" pin="1"/>
 <wire x1="139.7" y1="66.04" x2="121.92" y2="66.04" width="0.2032" layer="91"/>
-<wire x1="121.92" y1="66.04" x2="111.76" y2="66.04" width="0.2032" layer="91"/>
+<wire x1="121.92" y1="66.04" x2="113.284" y2="66.04" width="0.2032" layer="91"/>
+<wire x1="113.284" y1="66.04" x2="111.76" y2="66.04" width="0.2032" layer="91"/>
 <wire x1="121.92" y1="53.34" x2="121.92" y2="66.04" width="0.2032" layer="91"/>
 <pinref part="R24" gate="R" pin="2"/>
@@
 <junction x="121.92" y="66.04"/>
 <junction x="139.7" y="66.04"/>
+<pinref part="U$5" gate="G$1" pin="G"/>
+<junction x="113.284" y="66.04"/>
 </segment>
 </net>
@@
 <junction x="106.68" y="38.1"/>
 <junction x="162.56" y="38.1"/>
-<wire x1="104.14" y1="38.1" x2="104.14" y2="53.34" width="0.2032" layer="91"/>
+<wire x1="104.14" y1="38.1" x2="104.14" y2="59.944" width="0.2032" layer="91"/>
 <pinref part="C25" gate="C" pin="1"/>
 <junction x="129.54" y="38.1"/>
 <pinref part="C26" gate="C" pin="2"/>
+<wire x1="104.14" y1="59.944" x2="104.14" y2="62.484" width="0.2032" layer="91"/>
+<wire x1="104.14" y1="62.484" x2="104.14" y2="64.262" width="0.2032" layer="91"/>
+<wire x1="104.14" y1="64.262" x2="104.14" y2="64.516" width="0.2032" layer="91"/>
 <wire x1="121.92" y1="45.72" x2="121.92" y2="38.1" width="0.2032" layer="91"/>
 <pinref part="R24" gate="R" pin="1"/>
@@
 <junction x="121.92" y="38.1"/>
 <junction x="104.14" y="38.1"/>
+<pinref part="U$5" gate="G$1" pin="S@1"/>
+<junction x="104.14" y="64.262"/>
+<junction x="104.14" y="62.484"/>
+<pinref part="U$5" gate="G$1" pin="S@3"/>
+<junction x="104.14" y="59.944"/>
 </segment>
 </net>
@@
 <wire x1="60.96" y1="81.28" x2="73.66" y2="81.28" width="0.2032" layer="91"/>
 <wire x1="73.66" y1="81.28" x2="83.82" y2="81.28" width="0.2032" layer="91"/>
-<wire x1="83.82" y1="81.28" x2="104.14" y2="81.28" width="0.2032" layer="91"/>
-<wire x1="104.14" y1="81.28" x2="170.18" y2="81.28" width="0.2032" layer="91"/>
+<wire x1="83.82" y1="81.28" x2="106.68" y2="81.28" width="0.2032" layer="91"/>
+<wire x1="106.68" y1="81.28" x2="170.18" y2="81.28" width="0.2032" layer="91"/>
 <wire x1="170.18" y1="81.28" x2="172.72" y2="81.28" width="0.2032" layer="91"/>
 <wire x1="170.18" y1="40.64" x2="170.18" y2="81.28" width="0.2032" layer="91"/>
@@
 <junction x="83.82" y="81.28"/>
 <junction x="170.18" y="81.28"/>
-<wire x1="104.14" y1="81.28" x2="104.14" y2="76.2" width="0.2032" layer="91"/>
 <wire x1="60.96" y1="81.28" x2="60.96" y2="68.58" width="0.2032" layer="91"/>
-<junction x="104.14" y="81.28"/>
 <junction x="60.96" y="81.28"/>
+<wire x1="106.68" y1="76.2" x2="106.68" y2="81.28" width="0.2032" layer="91"/>
+<junction x="106.68" y="81.28"/>
 </segment>
 </net>
@@
 <wire x1="-22.86" y1="81.28" x2="-20.32" y2="81.28" width="0.2032" layer="91"/>
 <junction x="-22.86" y="63.5"/>
+<wire x1="-25.4" y1="78.74" x2="-25.4" y2="81.28" width="0.2032" layer="91"/>
+<wire x1="-25.4" y1="81.28" x2="-22.86" y2="81.28" width="0.2032" layer="91"/>
 <junction x="-22.86" y="81.28"/>
-<wire x1="-22.86" y1="81.28" x2="-30.48" y2="81.28" width="0.2032" layer="91"/>
 </segment>
 </net>
@@
 <pinref part="R23" gate="R" pin="1"/>
 <wire x1="-48.26" y1="93.98" x2="-48.26" y2="81.28" width="0.2032" layer="91"/>
-<wire x1="-48.26" y1="93.98" x2="-48.26" y2="101.6" width="0.2032" layer="91"/>
-<wire x1="-63.5" y1="81.28" x2="-68.58" y2="81.28" width="0.2032" layer="91"/>
+<wire x1="-48.26" y1="93.98" x2="-48.26" y2="99.06" width="0.2032" layer="91"/>
 <junction x="-48.26" y="81.28"/>
 <junction x="-63.5" y="81.28"/>
-<wire x1="-48.26" y1="81.28" x2="-40.64" y2="81.28" width="0.2032" layer="91"/>
+<wire x1="-48.26" y1="81.28" x2="-41.656" y2="81.28" width="0.2032" layer="91"/>
 <pinref part="U$2" gate="G$1" pin="S"/>
+<junction x="-48.26" y="93.98"/>
+<wire x1="-63.5" y1="81.28" x2="-70.104" y2="81.28" width="0.2032" layer="91"/>
+<pinref part="U$3" gate="G$1" pin="S@1"/>
+<junction x="-74.422" y="81.28"/>
+<pinref part="U$3" gate="G$1" pin="S@2"/>
+<junction x="-72.39" y="81.28"/>
+<wire x1="-70.104" y1="81.28" x2="-72.39" y2="81.28" width="0.2032" layer="91"/>
+<wire x1="-72.39" y1="81.28" x2="-74.422" y2="81.28" width="0.2032" layer="91"/>
+<pinref part="U$3" gate="G$1" pin="S@3"/>
+<junction x="-70.104" y="81.28"/>
+<pinref part="U$4" gate="G$1" pin="S@3"/>
+<junction x="-41.656" y="81.28"/>
+<wire x1="-38.1" y1="81.28" x2="-39.116" y2="81.28" width="0.2032" layer="91"/>
+<pinref part="U$4" gate="G$1" pin="S@1"/>
+<wire x1="-39.116" y1="81.28" x2="-39.37" y2="81.28" width="0.2032" layer="91"/>
+<wire x1="-39.37" y1="81.28" x2="-41.656" y2="81.28" width="0.2032" layer="91"/>
+<wire x1="-37.338" y1="81.28" x2="-38.1" y2="81.28" width="0.2032" layer="91"/>
+<pinref part="U$4" gate="G$1" pin="S@2"/>
+<junction x="-39.37" y="81.28"/>
+<junction x="-37.338" y="81.28"/>
 </segment>
 </net>
@@
 <wire x1="-68.58" y1="93.98" x2="-63.5" y2="93.98" width="0.2032" layer="91"/>
 <wire x1="-63.5" y1="93.98" x2="-58.42" y2="93.98" width="0.2032" layer="91"/>
-<wire x1="-63.5" y1="93.98" x2="-63.5" y2="106.68" width="0.2032" layer="91"/>
+<wire x1="-63.5" y1="93.98" x2="-63.5" y2="104.14" width="0.2032" layer="91"/>
+<junction x="-63.5" y="93.98"/>
 <pinref part="U$2" gate="G$1" pin="G\"/>
-<wire x1="-63.5" y1="106.68" x2="-48.26" y2="106.68" width="0.2032" layer="91"/>
-<junction x="-63.5" y="93.98"/>
+<wire x1="-60.96" y1="104.14" x2="-63.5" y2="104.14" width="0.2032" layer="91"/>
 </segment>
 </net>
 <net name="N$34" class="0">
 <segment>
-<wire x1="-38.1" y1="119.38" x2="-99.06" y2="119.38" width="0.2032" layer="91"/>
 <wire x1="-99.06" y1="119.38" x2="-99.06" y2="68.58" width="0.2032" layer="91"/>
 <pinref part="C8" gate="C" pin="2"/>
 <wire x1="-91.44" y1="71.12" x2="-91.44" y2="68.58" width="0.2032" layer="91"/>
 <pinref part="R21" gate="R" pin="1"/>
-<wire x1="-91.44" y1="68.58" x2="-78.74" y2="68.58" width="0.2032" layer="91"/>
 <pinref part="C22" gate="C" pin="2"/>
-<wire x1="-78.74" y1="68.58" x2="-63.5" y2="68.58" width="0.2032" layer="91"/>
+<wire x1="-91.44" y1="68.58" x2="-76.2" y2="68.58" width="0.2032" layer="91"/>
+<wire x1="-76.2" y1="68.58" x2="-63.5" y2="68.58" width="0.2032" layer="91"/>
 <wire x1="-63.5" y1="68.58" x2="-58.42" y2="68.58" width="0.2032" layer="91"/>
 <pinref part="R10" gate="R" pin="2"/>
 <wire x1="-58.42" y1="68.58" x2="-55.88" y2="68.58" width="0.2032" layer="91"/>
 <wire x1="-58.42" y1="68.58" x2="-58.42" y2="12.7" width="0.2032" layer="91"/>
-<wire x1="-78.74" y1="68.58" x2="-78.74" y2="73.66" width="0.2032" layer="91"/>
-<wire x1="-35.56" y1="73.66" x2="-35.56" y2="68.58" width="0.2032" layer="91"/>
+<wire x1="-35.56" y1="73.66" x2="-35.56" y2="72.136" width="0.2032" layer="91"/>
+<wire x1="-35.56" y1="72.136" x2="-35.56" y2="68.58" width="0.2032" layer="91"/>
 <wire x1="-55.88" y1="68.58" x2="-35.56" y2="68.58" width="0.2032" layer="91"/>
 <junction x="-58.42" y="68.58"/>
 <junction x="-55.88" y="68.58"/>
 <junction x="-63.5" y="68.58"/>
-<junction x="-78.74" y="68.58"/>
 <wire x1="-99.06" y1="68.58" x2="-91.44" y2="68.58" width="0.2032" layer="91"/>
 <junction x="-91.44" y="68.58"/>
 <pinref part="U$2" gate="G$1" pin="D"/>
-<wire x1="-38.1" y1="104.14" x2="-38.1" y2="119.38" width="0.2032" layer="91"/>
-</segment>
-</net>
+<wire x1="-48.26" y1="116.84" x2="-48.26" y2="119.38" width="0.2032" layer="91"/>
+<wire x1="-48.26" y1="119.38" x2="-99.06" y2="119.38" width="0.2032" layer="91"/>
+<wire x1="-76.2" y1="68.58" x2="-76.2" y2="71.882" width="0.2032" layer="91"/>
+<pinref part="U$3" gate="G$1" pin="G"/>
+<pinref part="U$4" gate="G$1" pin="G"/>
+<junction x="-35.56" y="72.136"/>
+<junction x="-76.2" y="71.882"/>
+<wire x1="-76.2" y1="71.882" x2="-76.2" y2="72.136" width="0.2032" layer="91"/>
+</segment>
+</net>

Commit message: Included SiS412DN MOSFET in battery charger
Parts:
- added U$6, U$7: SIS412DNSOP-8, RNH_SIS412DN:SIS412DNSOP-8
Connections:
- net N$26: now also U$7.G
- net N$29: now also U$6.G
Other:
- note added: "Schematic is missing: - Chassis ground - Net names - TP1? - Test points - Component values"
Changed lines of the file:
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@@
 <part name="U$4" library="RNH_FDS6680A" deviceset="FDS6680A" device="SOIC-8"/>
 <part name="U$5" library="RNH_FDS6680A" deviceset="FDS6680A" device="SOIC-8"/>
+<part name="U$6" library="RNH_SIS412DN" deviceset="SIS412DN" device="SOP-8"/>
+<part name="U$7" library="RNH_SIS412DN" deviceset="SIS412DN" device="SOP-8"/>
 </parts>
 <sheets>
@@
 Battery Charger Schematic</text>
 <text x="211.836" y="-99.568" size="2.54" layer="97">v1</text>
+<text x="175.26" y="-60.96" size="1.778" layer="97">Schematic is missing:
+- Chassis ground
+- Net names
+- TP1?
+- Test points
+- Component values</text>
 </plain>
 <instances>
@@
 <instance part="U$4" gate="G$1" x="-30.48" y="76.2" rot="MR90"/>
 <instance part="U$5" gate="G$1" x="109.22" y="71.12" rot="MR0"/>
+<instance part="U$6" gate="G$1" x="54.61" y="62.23"/>
+<instance part="U$7" gate="G$1" x="57.15" y="29.21"/>
 </instances>
 <busses>
@@
 <wire x1="43.18" y1="10.16" x2="58.42" y2="10.16" width="0.2032" layer="91"/>
 <pinref part="SUPPLY1" gate="GND" pin="GND"/>
+<wire x1="60.96" y1="22.86" x2="60.96" y2="10.16" width="0.2032" layer="91"/>
+<wire x1="58.42" y1="10.16" x2="60.96" y2="10.16" width="0.2032" layer="91"/>
 </segment>
 <segment>
@@
 <junction x="2.54" y="81.28"/>
 <junction x="-7.62" y="81.28"/>
-<wire x1="22.86" y1="81.28" x2="60.96" y2="81.28" width="0.2032" layer="91"/>
-<wire x1="60.96" y1="81.28" x2="73.66" y2="81.28" width="0.2032" layer="91"/>
+<wire x1="22.86" y1="81.28" x2="58.42" y2="81.28" width="0.2032" layer="91"/>
+<wire x1="58.42" y1="81.28" x2="73.66" y2="81.28" width="0.2032" layer="91"/>
 <wire x1="73.66" y1="81.28" x2="83.82" y2="81.28" width="0.2032" layer="91"/>
 <wire x1="83.82" y1="81.28" x2="106.68" y2="81.28" width="0.2032" layer="91"/>
@@
 <junction x="83.82" y="81.28"/>
 <junction x="170.18" y="81.28"/>
-<wire x1="60.96" y1="81.28" x2="60.96" y2="68.58" width="0.2032" layer="91"/>
-<junction x="60.96" y="81.28"/>
 <wire x1="106.68" y1="76.2" x2="106.68" y2="81.28" width="0.2032" layer="91"/>
 <junction x="106.68" y="81.28"/>
+<wire x1="58.166" y1="68.834" x2="58.42" y2="68.834" width="0.2032" layer="91"/>
+<wire x1="58.42" y1="68.834" x2="58.42" y2="68.58" width="0.2032" layer="91"/>
+<wire x1="58.42" y1="68.834" x2="58.42" y2="81.28" width="0.2032" layer="91"/>
+<junction x="58.42" y="81.28"/>
 </segment>
 </net>
@@
 <pinref part="C15" gate="C" pin="1"/>
 <wire x1="43.18" y1="25.4" x2="43.18" y2="22.86" width="0.2032" layer="91"/>
-<wire x1="43.18" y1="25.4" x2="50.8" y2="25.4" width="0.2032" layer="91"/>
+<wire x1="43.18" y1="25.4" x2="48.26" y2="25.4" width="0.2032" layer="91"/>
+<pinref part="U$7" gate="G$1" pin="G"/>
+<wire x1="53.34" y1="25.4" x2="48.26" y2="25.4" width="0.2032" layer="91"/>
+<wire x1="50.8" y1="25.4" x2="53.34" y2="25.4" width="0.2032" layer="91"/>
+<junction x="43.18" y="25.4"/>
 </segment>
 </net>
@@
 <wire x1="43.18" y1="58.42" x2="50.8" y2="58.42" width="0.2032" layer="91"/>
 <junction x="43.18" y="58.42"/>
+<pinref part="U$6" gate="G$1" pin="G"/>
 </segment>
 </net>
@@
 </segment>
 </net>
-<net name="N$4" class="0">
-<segment>
-<pinref part="L2" gate="L" pin="1"/>
-<pinref part="C11" gate="C" pin="2"/>
-<wire x1="50.8" y1="38.1" x2="58.42" y2="38.1" width="0.2032" layer="91"/>
-<wire x1="58.42" y1="38.1" x2="58.42" y2="25.4" width="0.2032" layer="91"/>
-<junction x="58.42" y="38.1"/>
-<wire x1="58.42" y1="38.1" x2="60.96" y2="38.1" width="0.2032" layer="91"/>
-<wire x1="60.96" y1="38.1" x2="68.58" y2="38.1" width="0.2032" layer="91"/>
-<junction x="60.96" y="38.1"/>
-<wire x1="68.58" y1="38.1" x2="71.12" y2="38.1" width="0.2032" layer="91"/>
-<wire x1="60.96" y1="43.18" x2="60.96" y2="38.1" width="0.2032" layer="91"/>
-<wire x1="60.96" y1="43.18" x2="60.96" y2="58.42" width="0.2032" layer="91"/>
+<net name="N$5" class="0">
+<segment>
 <pinref part="C16" gate="C" pin="2"/>
 <wire x1="43.18" y1="45.72" x2="43.18" y2="43.18" width="0.2032" layer="91"/>
-<wire x1="43.18" y1="43.18" x2="60.96" y2="43.18" width="0.2032" layer="91"/>
-<junction x="43.18" y="43.18"/>
 <wire x1="-5.08" y1="43.18" x2="43.18" y2="43.18" width="0.2032" layer="91"/>
 <pinref part="U$1" gate="G$1" pin="PHASE"/>
 <wire x1="-5.08" y1="22.86" x2="-5.08" y2="43.18" width="0.2032" layer="91"/>
+<pinref part="L2" gate="L" pin="1"/>
+<wire x1="68.58" y1="38.1" x2="71.12" y2="38.1" width="0.2032" layer="91"/>
 <wire x1="68.58" y1="38.1" x2="68.58" y2="121.92" width="0.2032" layer="91"/>
+<pinref part="C11" gate="C" pin="2"/>
+<wire x1="50.8" y1="38.1" x2="58.42" y2="38.1" width="0.2032" layer="91"/>
+<wire x1="68.58" y1="38.1" x2="60.96" y2="38.1" width="0.2032" layer="91"/>
+<wire x1="60.96" y1="38.1" x2="58.42" y2="38.1" width="0.2032" layer="91"/>
+<wire x1="58.42" y1="55.88" x2="58.42" y2="43.18" width="0.2032" layer="91"/>
+<wire x1="58.42" y1="43.18" x2="58.42" y2="38.1" width="0.2032" layer="91"/>
+<wire x1="60.96" y1="35.56" x2="60.96" y2="38.1" width="0.2032" layer="91"/>
+<wire x1="43.18" y1="43.18" x2="58.42" y2="43.18" width="0.2032" layer="91"/>
+<junction x="58.42" y="43.18"/>
+<junction x="58.42" y="38.1"/>
 <junction x="68.58" y="38.1"/>
-</segment>
-</net>
+<junction x="60.96" y="38.1"/>
+</segment>
+</net>

Commit message: Added labels in Battery Charger Page and fixed pad size in SIS412DN library
Parts:
- added R6, R7: 10, rcl_custom:R-US_0603-B
Connections:
- net N$1 renamed VCC@1
- net N$10 renamed ACOK
- net N$11 renamed CMSRC
- net N$15 renamed VIN
- net N$19 renamed BAT@1
- net N$20 renamed REGN@1
- net N$24 renamed BATDRV
- net N$25 renamed SYS
- net N$3 renamed ILIM
- net N$6 renamed IOUT
- net N$7 renamed ACDET
- net N$9 renamed ACDRV
- new net 3V3: R6.1, R7.1
- new net 3V3@1: R5.2
- new net BAT: JP4.2
- new net REGN: R9.2
- new net VCC: R14.1
- net SCL: now also R6.2
- net SDA: now also R7.2
Other:
- moved on the sheet: R13, R8, R9

Commit message: changed US capacitor symbols to EU capacitor symbol
Parts:
- C1, C10, C11, C12, C13, C14, C15, C16, C17, C18, C19, C2, C20, C21, C22, C23, C24, C25, C26, C3, C4, C5, C6, C7, C8, C9: device rcl_custom:C-USC0603 -> rcl:C-EUC0402
Connections:
- removed net REGN@1: C10.1, D1.A, U$1.REGN
- net REGN: now also C10.1, D1.A, U$1.REGN

Commit message: Updated nets, removed headers on batterycharger, corrected BQ24725, BSS138W, SIS412 package outlines, added PG and FLT LED indicators and fixed nets on mcu_page
Parts:
- removed JP1, JP2, JP3: (no value), pinhead:PINHD-1X3
- removed JP4, JP5: (no value), pinhead:PINHD-1X2
- added R25: 0, rcl_custom:R-US_0402-B
- R14, R6, R7: device rcl_custom:R-US_0603-B -> rcl_custom:R-US_0402-B
Connections:
- removed net 3V3: R6.1, R7.1
- removed net 3V3@1: R5.2
- removed net BAT@1: C12.1, C25.1, C26.2, C3.1, C9.2, JP3.2, R19.1, R24.1, R3.1, U$5.S@1, U$5.S@3
- removed net N$13: D3.A1, JP4.1
- removed net VCC@1: C1.1, U$1.VCC
- removed net VIN: C7.1, C8.1, D3.A2, JP5.1, R13.2
- new net +3V3: R5.2, R6.1, R7.1
- new net N$1: D3.A1, R25.2
- new net SHORE_POWER: C7.1, C8.1, D3.A2, R13.2
- net BAT: now also C12.1, C25.1, C26.2, C3.1, C9.2, R19.1, R24.1, R25.1, R3.1, U$5.S@1, U$5.S@3; no longer JP4.2
- net GND: no longer C18.2, JP1.1, JP3.1, JP5.2
- net SCL: no longer JP1.3
- net SDA: no longer JP1.2
- net SYS: no longer JP3.3
- net VCC: now also C1.1, U$1.VCC
Other:
- note removed: "Schematic is missing: - Chassis ground - Net names - TP1? - Test points - Component values"
- moved on the sheet: U$2
