File: av3/rocketnet-hub/eagle/mcu_page.sch (EAGLE design)
At the start: 333 parts, among them J1 ROCKETBUS, J2 ROCKETBUS, J3 ROCKETBUS, J4 ROCKETBUS, J5 ROCKETBUS, J6 ROCKETBUS, J7 ROCKETBUS, J8 ROCKETBUS, Q1 25.000MHz, X1 87758-0416, X2 87758-0416, X3 87758-0416, X4 87758-0416, X5 87758-0416, X6 87758-0416, X7 87758-0416, X8 87758-0416

Commit message: Updated nets, removed headers on batterycharger, corrected BQ24725, BSS138W, SIS412 package outlines, added PG and FLT LED indicators and fixed nets on mcu_page
Parts:
- added LED47, LED50, LED51, LED52, LED53, LED54, LED55, LED56: (no value), led:LEDSML0603
- added R100, R101, R102, R103, R104, R105, R106, R107, R108, R109, R110, R111, R112, R113, R114, R115, R116, R117, R118, R119, R120, R121, R122, R123, R124, R125, R126, R127, R128, R129, R130, R99: (no value), rcl:R-US_R0402
Connections:
- new net N$173: LED47.A, R101.2, R99.1
- new net N$176: LED50.A, R112.1, R114.2
- new net N$177: LED51.A, R115.1, R117.2
- new net N$178: LED52.A, R116.1, R118.2
- new net N$179: LED53.A, R119.1, R121.2
- new net N$180: LED54.A, R120.1, R122.2
- new net N$181: LED55.A, R123.1, R125.2
- new net N$182: LED56.A, R124.1, R126.2
- new net NODE1_!FLT2: LED42.C, R61.1
- new net NODE1_!FLT3: LED43.C, R106.1
- new net NODE1_!FLT4: LED45.C, R110.1
- new net NODE1_!FLT5: LED50.C, R114.1
- new net NODE1_!FLT6: LED52.C, R118.1
- new net NODE1_!FLT7: LED54.C, R122.1
- new net NODE1_!FLT8: LED56.C, R126.1
- new net NODE1_!PG2: LED40.C, R59.1
- new net NODE1_!PG3: LED41.C, R65.1
- new net NODE1_!PG4: LED44.C, R109.1
- new net NODE1_!PG5: LED46.C, R113.1
- new net NODE1_!PG6: LED51.C, R117.1
- new net NODE1_!PG7: LED53.C, R121.1
- new net NODE1_!PG8: LED55.C, R125.1
- net +3V3: now also R107.2, R108.2, R111.2, R112.2, R115.2, R116.2, R119.2, R120.2, R123.2, R124.2, R99.2; no longer R59.2, R61.2, R65.2
- net GND: now also R102.1, R103.1, R104.1, R105.1, R127.1, R128.1, R129.1, R130.1
- net N$131: now also R100.2
- net N$133: now also R59.2
- net N$134: now also R65.2
- net N$135: now also R61.2
- net N$136: now also R106.2, R63.1; no longer R59.1
- net N$137: now also R107.1, R109.2; no longer R61.1
- net N$138: now also R108.1, R110.2; no longer R63.1
- net N$139: now also R111.1, R113.2; no longer R65.1
- net N$147: now also R104.2
- net N$154: now also R127.2
- net N$155: now also R129.2
- net N$157: now also R103.2
- net N$158: now also R105.2
- net N$159: now also R128.2
- net NODE1_!FLT: now also LED47.C, R101.1
- net NODE1_!PG: now also R100.1
- net NODE1_ILIM: now also R102.2
- net NODE2_!PG: no longer LED40.C
- net NODE3_!PG: no longer LED41.C
- net NODE4_!PG: no longer LED43.C
- net NODE5_!PG: no longer LED42.C
- net NODE6_!PG: no longer LED44.C
- net NODE7_!PG: no longer LED45.C
- net NODE8_!PG: no longer LED46.C
- net NODE8_ILIM: now also R130.2
Other:
- moved on the sheet: LED39, LED40, LED41, LED42, LED43, LED44, LED45, LED46, R50, R53, R55, R57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

Commit message: layout updates
Parts:
- removed C10, C11: 27p, rcl:C-EUC0402
- removed LED47, LED50, LED51, LED52, LED53, LED54, LED55, LED56: (no value), led:LEDSML0603
- removed Q1: 25.000MHz, crystal:CRYSTALSM49
- removed R100, R101, R102, R103, R104, R105, R106, R107, R108, R109, R110, R111, R112, R113, R114, R115, R116, R117, R118, R119, R120, R121, R122, R123, R124, R125, R126, R127, R128, R129, R130, R99: (no value), rcl:R-US_R0402
- added U$20: ASE, crystal:ASE
Connections:
- net N$23 renamed RX1_N
- net N$24 renamed RX2_N
- net N$25 renamed TX1_P
- net N$26 renamed TX2_P
- net N$29 renamed RX3_N
- net N$30 renamed TX3_P
- net N$31 renamed RX4_N
- net N$32 renamed TX4_P
- net NODE2_RXM renamed NODE2_RX_N
- net NODE2_RXP renamed NODE2_RX_P
- net NODE2_TXM renamed NODE2_TX_N
- net NODE3_RXM renamed NODE3_RX_N
- net NODE3_RXP renamed NODE3_RX_P
- net NODE3_TXM renamed NODE3_TX_N
- net NODE3_TXP renamed NODE3_TX_P
- net NODE4_RXM renamed NODE4_RX_N
- net NODE4_RXP renamed NODE4_RX_P
- net NODE4_TXM renamed NODE4_TX_N
- net NODE4_TXP renamed NODE4_TX_P
- net RXP1 renamed RX1_P
- net RXP2 renamed RX2_P
- net RXP3 renamed RX3_P
- net RXP4 renamed RX4_P
- net TXM1 renamed TX1_N
- net TXM2 renamed TX2_N
- net TXM3 renamed TX3_N
- net TXM4 renamed TX4_N
- removed net N$125: C90.2, U$6.GND@5
- removed net N$152: R71.2
- removed net N$153: R72.2
- removed net N$154: R127.2, U$7.IFLT
- removed net N$155: R129.2, U$9.IFLT
- removed net N$157: R103.2, U$4.IFLT
- removed net N$158: R105.2, U$6.IFLT
- removed net N$159: R128.2, U$8.IFLT
- removed net N$173: LED47.A, R101.2, R99.1
- removed net N$176: LED50.A, R112.1, R114.2
- removed net N$177: LED51.A, R115.1, R117.2
- removed net N$178: LED52.A, R116.1, R118.2
- removed net N$179: LED53.A, R119.1, R121.2
- removed net N$180: LED54.A, R120.1, R122.2
- removed net N$181: LED55.A, R123.1, R125.2
- removed net N$182: LED56.A, R124.1, R126.2
- removed net N$2 (its old number): C10.2, Q1.2, U$1.PH1
- removed net N$4 (its old number): C11.1
- removed net NODE1_!FLT2: LED42.C, R61.1
- removed net NODE1_!FLT3: LED43.C, R106.1
- removed net NODE1_!FLT4: LED45.C, R110.1
- removed net NODE1_!FLT5: LED50.C, R114.1
- removed net NODE1_!FLT6: LED52.C, R118.1
- removed net NODE1_!FLT7: LED54.C, R122.1
- removed net NODE1_!FLT8: LED56.C, R126.1
- removed net NODE1_!PG2: LED40.C, R59.1
- removed net NODE1_!PG3: LED41.C, R65.1
- removed net NODE1_!PG4: LED44.C, R109.1
- removed net NODE1_!PG5: LED46.C, R113.1
- removed net NODE1_!PG6: LED51.C, R117.1
- removed net NODE1_!PG7: LED53.C, R121.1
- removed net NODE1_!PG8: LED55.C, R125.1
- removed net NODE1_ILIM: R102.2, U$3.IFLT
- removed net NODE8_ILIM: R130.2, U$10.IFLT
- new net N$130: R67.2, U$5.IMAX
- new net NODE1_RX_N: C29.2
- new net NODE1_RX_P: C30.2
- new net NODE1_TX_P: C31.2, C32.2
- new net NODE2_TX_P: C36.2
- net +3V3: now also R59.2, R61.2, R65.2, U$20.TRI, U$20.VDD; no longer R107.2, R108.2, R111.2, R112.2, R115.2, R116.2, R119.2, R120.2, R123.2, R124.2, R99.2
- net GND: now also C90.2, U$20.GND, U$6.GND@5; no longer C10.1, R102.1, R103.1, R104.1, R105.1, R127.1, R128.1, R129.1, R130.1
- net N$1: now also U$20.OUT; no longer C11.2, Q1.1
- net N$131: no longer R100.2
- net N$133: no longer R59.2
- net N$134: no longer R65.2
- net N$135: no longer R61.2
- net N$136: now also R59.1; no longer R106.2, R63.1
- net N$137: now also R61.1; no longer R107.1, R109.2
- net N$138: now also R63.1; no longer R108.1, R110.2
- net N$139: now also R65.1; no longer R111.1, R113.2
- net N$147: now also R68.2, U$6.IMAX; no longer R104.2, U$5.IFLT
- net N$148: now also R69.2, U$7.IMAX; no longer R67.2
- net N$149: now also R70.2, U$8.IMAX; no longer R68.2
- net N$150: now also R71.2, U$9.IMAX; no longer R69.2
- net N$151: now also R72.2, U$10.IMAX; no longer R70.2
- net NODE1_!FLT: no longer LED47.C, R101.1
- net NODE1_!PG: no longer R100.1
- net NODE1_RXM: no longer C29.2
- net NODE1_RXP: no longer C30.2
- net NODE1_TXM: no longer C31.2
- net NODE1_TXP: no longer C32.2
- net NODE2_!PG: now also LED40.C
- net NODE2_TXP: no longer C36.2
- net NODE3_!PG: now also LED41.C
- net NODE4_!PG: now also LED43.C
- net NODE5_!PG: now also LED42.C
- net NODE6_!PG: now also LED44.C
- net NODE7_!PG: now also LED45.C
- net NODE8_!PG: now also LED46.C
Other:
- moved on the sheet: C90, LED39, LED40, LED41, LED42, LED43, LED44, LED45, LED46, R50, R53, R55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

Commit message: Rearranged the layout of switch circuit - work in progress
Connections:
- net N$141 renamed RATSNET
- removed net N$123: C88.2, U$4.GND@5
- removed net N$124: C87.2, U$5.GND@5
- net GND: now also C87.2, C88.2, U$4.GND@5, U$5.GND@5
Changed lines of the file:
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@@
 <wire x1="27.94" y1="111.76" x2="27.94" y2="114.3" width="0.1524" layer="91"/>
 <pinref part="GND45" gate="1" pin="GND"/>
-<wire x1="27.94" y1="114.3" x2="27.94" y2="119.38" width="0.1524" layer="91"/>
 <junction x="27.94" y="114.3"/>
+<wire x1="50.8" y1="121.92" x2="50.8" y2="119.38" width="0.1524" layer="91"/>
+<pinref part="U$5" gate="G$1" pin="GND@5"/>
+<wire x1="50.8" y1="119.38" x2="27.94" y2="119.38" width="0.1524" layer="91"/>
+<wire x1="27.94" y1="119.38" x2="27.94" y2="114.3" width="0.1524" layer="91"/>
+<pinref part="C87" gate="G$1" pin="2"/>
+<wire x1="27.94" y1="119.38" x2="27.94" y2="127" width="0.1524" layer="91"/>
+<junction x="27.94" y="119.38"/>
 </segment>
 <segment>
@@
 <pinref part="R72" gate="G$1" pin="1"/>
 <pinref part="GND62" gate="1" pin="GND"/>
+</segment>
+<segment>
+<wire x1="50.8" y1="233.68" x2="50.8" y2="231.14" width="0.1524" layer="91"/>
+<pinref part="C88" gate="G$1" pin="2"/>
+<wire x1="27.94" y1="236.22" x2="27.94" y2="231.14" width="0.1524" layer="91"/>
+<wire x1="27.94" y1="231.14" x2="50.8" y2="231.14" width="0.1524" layer="91"/>
+<pinref part="U$4" gate="G$1" pin="GND@5"/>
+<pinref part="GND44" gate="1" pin="GND"/>
+<wire x1="27.94" y1="226.06" x2="27.94" y2="231.14" width="0.1524" layer="91"/>
+<junction x="27.94" y="231.14"/>
 </segment>
 </net>
@@
 </segment>
 </net>
-<net name="N$123" class="0">
-<segment>
-<wire x1="50.8" y1="233.68" x2="50.8" y2="231.14" width="0.1524" layer="91"/>
-<pinref part="C88" gate="G$1" pin="2"/>
-<wire x1="27.94" y1="236.22" x2="27.94" y2="231.14" width="0.1524" layer="91"/>
-<wire x1="27.94" y1="231.14" x2="50.8" y2="231.14" width="0.1524" layer="91"/>
-<pinref part="U$4" gate="G$1" pin="GND@5"/>
-<wire x1="27.94" y1="223.52" x2="27.94" y2="231.14" width="0.1524" layer="91"/>
-<junction x="27.94" y="231.14"/>
-</segment>
-</net>
-<net name="N$124" class="0">
-<segment>
-<wire x1="50.8" y1="121.92" x2="50.8" y2="119.38" width="0.1524" layer="91"/>
-<pinref part="C87" gate="G$1" pin="2"/>
-<wire x1="27.94" y1="127" x2="27.94" y2="119.38" width="0.1524" layer="91"/>
-<wire x1="27.94" y1="119.38" x2="50.8" y2="119.38" width="0.1524" layer="91"/>
-<pinref part="U$5" gate="G$1" pin="GND@5"/>
-<junction x="27.94" y="119.38"/>
-</segment>
-</net>
 <net name="N$126" class="0">
 <segment>
@@
 </segment>
 </net>
-<net name="N$141" class="0">
+<net name="RATSNET" class="0">
 <segment>
 <pinref part="C97" gate="G$1" pin="1"/>

Commit message: added vias to center pad to package
Parts:
- added U$26, U$27: MAX4734ETC+, max4734:MAX4734ETC+
Connections:
- new net N$30: U$26.GND
- new net N$31: U$26.COM
- net NODE1_IMON: now also U$26.N0
- net NODE2_IMON: now also U$26.N2
- net NODE3_IMON: now also U$26.N3
- net NODE4_IMON: now also U$26.N4
Other:
- moved on the sheet: U$10, U$3, U$4, U$5, U$6, U$7, U$8, U$9
Changed lines of the file:
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@@
 <part name="+3V17" library="supply1" deviceset="+3V3" device=""/>
 <part name="+3V18" library="supply1" deviceset="+3V3" device=""/>
+<part name="U$26" library="max4734" deviceset="MAX4734ETC+" device=""/>
+<part name="U$27" library="max4734" deviceset="MAX4734ETC+" device=""/>
 </parts>
 <sheets>
@@
 <instance part="P+8" gate="1" x="30.48" y="-309.88"/>
 <instance part="P+9" gate="1" x="30.48" y="-426.72"/>
+<instance part="U$26" gate="G$1" x="-30.48" y="195.58"/>
+<instance part="U$27" gate="G$1" x="-10.16" y="-276.86"/>
 </instances>
 <busses>
@@
 <wire x1="66.04" y1="406.4" x2="66.04" y2="419.1" width="0.1524" layer="91"/>
 <wire x1="66.04" y1="419.1" x2="81.28" y2="419.1" width="0.1524" layer="91"/>
-<wire x1="66.04" y1="419.1" x2="43.18" y2="419.1" width="0.1524" layer="91"/>
 <junction x="66.04" y="419.1"/>
 <pinref part="R49" gate="G$1" pin="2"/>
 <label x="43.18" y="419.1" size="1.016" layer="95" rot="R180" xref="yes"/>
+<pinref part="U$26" gate="G$1" pin="N0"/>
+<wire x1="-43.18" y1="198.12" x2="-45.72" y2="198.12" width="0.1524" layer="91"/>
+<wire x1="-45.72" y1="198.12" x2="-45.72" y2="419.1" width="0.1524" layer="91"/>
+<wire x1="-45.72" y1="419.1" x2="66.04" y2="419.1" width="0.1524" layer="91"/>
 </segment>
 </net>
@@
 <net name="NODE2_IMON" class="0">
 <segment>
-<wire x1="43.18" y1="287.02" x2="66.04" y2="287.02" width="0.1524" layer="91"/>
 <pinref part="U$4" gate="G$1" pin="IMON"/>
 <wire x1="66.04" y1="287.02" x2="66.04" y2="274.32" width="0.1524" layer="91"/>
@@
 <junction x="66.04" y="287.02"/>
 <label x="43.18" y="287.02" size="1.016" layer="95" rot="R180" xref="yes"/>
+<pinref part="U$26" gate="G$1" pin="N2"/>
+<wire x1="-17.78" y1="198.12" x2="-12.7" y2="198.12" width="0.1524" layer="91"/>
+<wire x1="-12.7" y1="198.12" x2="-12.7" y2="287.02" width="0.1524" layer="91"/>
+<wire x1="-12.7" y1="287.02" x2="66.04" y2="287.02" width="0.1524" layer="91"/>
 </segment>
 </net>
@@
 <pinref part="U$5" gate="G$1" pin="IMON"/>
 <wire x1="66.04" y1="162.56" x2="66.04" y2="175.26" width="0.1524" layer="91"/>
-<wire x1="66.04" y1="175.26" x2="43.18" y2="175.26" width="0.1524" layer="91"/>
 <pinref part="R54" gate="G$1" pin="2"/>
 <wire x1="66.04" y1="175.26" x2="81.28" y2="175.26" width="0.1524" layer="91"/>
 <junction x="66.04" y="175.26"/>
 <label x="43.18" y="175.26" size="1.016" layer="95" rot="R180" xref="yes"/>
+<pinref part="U$26" gate="G$1" pin="N3"/>
+<wire x1="-43.18" y1="193.04" x2="-45.72" y2="193.04" width="0.1524" layer="91"/>
+<wire x1="-45.72" y1="193.04" x2="-45.72" y2="175.26" width="0.1524" layer="91"/>
+<wire x1="-45.72" y1="175.26" x2="66.04" y2="175.26" width="0.1524" layer="91"/>
 </segment>
 </net>
@@
 <pinref part="R58" gate="G$1" pin="2"/>
 <wire x1="81.28" y1="53.34" x2="66.04" y2="53.34" width="0.1524" layer="91"/>
-<wire x1="66.04" y1="53.34" x2="43.18" y2="53.34" width="0.1524" layer="91"/>
 <label x="43.18" y="53.34" size="1.016" layer="95" rot="R180" xref="yes"/>
 <junction x="66.04" y="53.34"/>
+<pinref part="U$26" gate="G$1" pin="N4"/>
+<wire x1="-17.78" y1="193.04" x2="-12.7" y2="193.04" width="0.1524" layer="91"/>
+<wire x1="-12.7" y1="193.04" x2="-12.7" y2="53.34" width="0.1524" layer="91"/>
+<wire x1="-12.7" y1="53.34" x2="66.04" y2="53.34" width="0.1524" layer="91"/>
 </segment>
 </net>
@@
 </segment>
 </net>
+<net name="N$30" class="0">
+<segment>
+<pinref part="U$26" gate="G$1" pin="GND"/>
+<wire x1="-43.18" y1="195.58" x2="-50.8" y2="195.58" width="0.1524" layer="91"/>
+<wire x1="-50.8" y1="195.58" x2="-50.8" y2="185.42" width="0.1524" layer="91"/>
+</segment>
+</net>
+<net name="N$31" class="0">
+<segment>
+<pinref part="U$26" gate="G$1" pin="COM"/>
+<wire x1="-17.78" y1="195.58" x2="-5.08" y2="195.58" width="0.1524" layer="91"/>
+</segment>
+</net>
