File: av3/rocketnet-hub/eagle/mcu_page.sch (EAGLE design)
At the start: 333 parts, among them J1 ROCKETBUS, J2 ROCKETBUS, J3 ROCKETBUS, J4 ROCKETBUS, J5 ROCKETBUS, J6 ROCKETBUS, J7 ROCKETBUS, J8 ROCKETBUS, X1 87758-0416, X2 87758-0416, X3 87758-0416, X4 87758-0416, X5 87758-0416, X6 87758-0416, X7 87758-0416, X8 87758-0416

Commit message: updated layout.
Parts:
- removed C105, C106, C107, C108, C109, C110, C111, C112, C113, C114, C115, C116, C117, C118, C119, C120, C121, C122, C123, C124, C125, C126, C127, C128, C129, C130: (no value), rcl:C-EUC0402
- removed D3: BAT54, diode:BAT54
- removed D4: BAT54C, diode:BAT54C
- removed JP1, JP2, JP3: (no value), pinhead:PINHD-1X3
- removed JP4, JP5: (no value), pinhead:PINHD-1X2
- removed L2: (no value), rcl_custom:L-US0603-B
- removed R75, R76, R88, R89, R90, R92, R94, R95: (no value), rcl_custom:R-US_0603-B
- removed R77: 100k, rcl_custom:R-US_0603-B
- removed R78: 316k, rcl_custom:R-US_0603-B
- removed R79, R91, R93, R96: 12.1k, rcl_custom:R-US_0603-B
- removed R80: 10k, rcl_custom:R-US_0603-B
- removed R81, R82: 4.02k, rcl_custom:R-US_0603-B
- removed R83: 66.5k, rcl_custom:R-US_0603-B
- removed R84, R86, R87: 430k, rcl_custom:R-US_0603-B
- removed R85, R97, R98: 10, rcl_custom:R-US_0603-B
- removed U$12: BQ24725QFN-20, RNH_BQ24725:BQ24725QFN-20
- removed U$13: BSS138W-7-F, RNH_BSS138W-7-F:BSS138W-7-F
- removed U$15, U$16, U$17: FDS6680ASOIC-8, RNH_FDS6680A:FDS6680ASOIC-8
- removed U$18, U$19: SIS412DNSOP-8, RNH_SIS412DN:SIS412DNSOP-8
- added C10: (no value), rcl:C-EUC0402K
Connections:
- net N$31 renamed NODE1_4_IMON
- net N$33 renamed RX5_N
- net N$34 renamed TX5_P
- net N$35 renamed RX6_N
- net N$36 renamed TX6_P
- net N$37 renamed RX7_N
- net N$38 renamed TX7_P
- net N$39 renamed RX8_N
- net N$40 renamed TX8_P
- net RXP5 renamed RX5_P
- net RXP6 renamed RX6_P
- net RXP7 renamed RX7_P
- net RXP8 renamed RX8_P
- net TXM5 renamed TX5_N
- net TXM6 renamed TX6_N
- net TXM7 renamed TX7_N
- net TXM8 renamed TX8_N
- removed net 3V3: R97.1, R98.1
- removed net 3V3@1: R78.2
- removed net ACDET: C108.1, R83.2, R84.1, U$12.ACDET
- removed net ACDRV: R81.1, U$12.ACDRV
- removed net BAT: JP4.2
- removed net BAT@1: C105.1, C112.2, C115.1, C128.1, C129.2, JP3.2, R76.1, R90.1, R96.1, U$17.S@1, U$17.S@3
- removed net BATDRV: C129.1, R75.1, R96.2, U$17.G
- removed net CMSRC: R82.1, U$12.CMSRC
- removed net ILIM: C106.1, R77.2, R78.1, U$12.ILIM
- removed net IOUT: C107.1, U$12.IOUT
- removed net N$118: D4.CC, R85.2
- removed net N$119: D4.A1, JP4.1
- removed net N$120: C109.2, R86.2, R87.2
- removed net N$121: R75.2, U$12.BATDRV
- removed net N$122: C89.2, U$3.GND@5
- removed net N$160: R76.2, U$12.SRN
- removed net N$161: R88.2, U$12.SRP
- removed net N$162: C111.1, C112.1, L2.2, R88.1, R90.2
- removed net N$163: R89.2, U$12.BTST
- removed net N$164: C114.1, D3.C, R89.1
- removed net N$165: C116.1, C117.1, C120.2, R92.2, U$12.ACP
- removed net N$166: C118.1, U$12.LODRV, U$19.G
- removed net N$167: C119.1, U$12.HIDRV, U$18.G
- removed net N$168: C120.1, C121.1, R91.1, U$12.ACN
- removed net N$169: C125.1, R82.2, R93.2, R95.1, U$13.S, U$15.S@1, U$15.S@2, U$15.S@3, U$16.S@1, U$16.S@2, U$16.S@3
- removed net N$170: R94.1, R95.2, U$13.G\
- removed net N$171: C110.2, C125.2, R81.2, R93.1, U$13.D, U$15.G, U$16.G
- removed net N$172: C114.2, C119.2, L2.1, U$12.PHASE
- removed net N$30: U$26.GND
- removed net REGN: C113.1, D3.A, R80.2, U$12.REGN
- removed net SYS: C122.1, C123.1, C124.1, C126.1, C127.1, JP3.3, R91.2, R92.1
- removed net VCC: R85.1
- removed net VCC@1: C130.1, U$12.VCC
- removed net VIN: C109.1, C110.1, D4.A2, JP5.1, R84.2
- new net IMON_A0: U$26.A0
- new net IMON_A1: U$26.A1
- new net NODE1_IMON_IN: R49.2, U$26.N0, U$3.IMON
- new net NODE2_IMON_IN: R52.2, U$26.N2, U$4.IMON
- new net NODE3_IMON_IN: R54.2, U$26.N3, U$5.IMON
- new net NODE4_IMON_IN: R58.2, U$26.N4, U$6.IMON
- net +3V3: now also C10.1, U$26.EN, U$26.V+
- net ACOK: no longer R79.2, R80.1, U$12.ACOK
- net GND: now also C10.2, C89.2, U$26.GND, U$3.GND@5; no longer C105.2, C106.2, C107.2, C108.2, C111.2, C113.2, C115.2, C116.2, C117.2, C118.2, C121.2, C122.2, C123.2, C124.2, C126.2, C127.2, C128.2, C130.2, JP1.1, JP3.1, JP5.2, R77.1, R79.1, R83.1, R86.1, R87.1, R94.2, U$12.GND
- net NODE1_IMON: no longer R49.2, U$26.N0, U$3.IMON
- net NODE2_IMON: no longer R52.2, U$26.N2, U$4.IMON
- net NODE3_IMON: no longer R54.2, U$26.N3, U$5.IMON
- net NODE4_IMON: no longer R58.2, U$26.N4, U$6.IMON
- net SCL: no longer JP1.3, R97.2, U$12.SCL
- net SDA: no longer JP1.2, R98.2, U$12.SDA
Other:
- note removed: "PSAS Rocketnet Hub Battery Charger Schematic"
- note removed: "Schematic is missing: - Chassis ground - Net names - TP1? - Test points - Component values"
- note removed: "v1"

Commit message: more routing and layout work
Parts:
- added C11: (no value), rcl:C-EUC0402K
- added R75, R76, R77, R78, R79, R80, R81, R82: (no value), rcl:R-US_R0402
Connections:
- removed net AUTOMDIX: U$1.PB2, U$14.AUTOMDIX
- removed net MODESEL0: U$1.PB5
- removed net MODESEL1: U$1.PB10, U$14.MODESEL[1]
- removed net MODESEL2: U$1.PB14, U$14.MODESEL[2]
- removed net MODESEL3: U$1.PB15, U$14.MODESEL[0], U$14.MODESEL[3]
- removed net N$126: C91.2, U$7.GND@5
- removed net N$127: C92.2, U$8.GND@5
- removed net N$128: C93.2, U$9.GND@5
- removed net N$129: C94.2, U$10.GND@5
- removed net NODE1_IMON: U$1.PA2
- removed net NODE1_RXM: J1.USB_L@1
- removed net NODE1_RXP: J1.USB_H@1
- removed net NODE1_TXM: J1.CAN_L@1
- removed net NODE1_TXP: J1.CAN_H@1, J1.CAN_H@2
- removed net NODE2_IMON: U$1.PA4
- removed net NODE3_IMON: U$1.PA5
- removed net NODE4_IMON: U$1.PA6
- new net NODE1_TX_N: C31.2, J1.CAN_L@1, J1.CAN_L@2, R76.2, R80.1
- new net NODE5_8_IMON: U$1.PC1, U$27.COM
- net +3V3: now also C11.1, R75.1, R76.1, R77.1, R78.1, U$27.EN, U$27.V+
- net GND: now also C11.2, C91.2, C92.2, C93.2, C94.2, J1.CHASSIS@1, J1.CHASSIS@2, J2.CHASSIS@1, J2.CHASSIS@2, J3.CHASSIS@1, J3.CHASSIS@2, J4.CHASSIS@1, J4.CHASSIS@2, J5.CHASSIS@1, J5.CHASSIS@2, J6.CHASSIS@1, J6.CHASSIS@2, J7.CHASSIS@1, J7.CHASSIS@2, J8.CHASSIS@1, J8.CHASSIS@2, R79.2, R80.2, R81.2, R82.2, U$10.GND@5, U$27.GND, U$7.GND@5, U$8.GND@5, U$9.GND@5
- net IMON_A0: now also U$1.PA4, U$27.A0
- net IMON_A1: now also U$1.PA5, U$27.A1
- net MIIS0: no longer U$14.MIIS[0]
- net MIIS1: no longer U$14.MIIS[1]
- net MTXD0: no longer U$14.MTXD[1]
- net MTXD1: now also U$14.MTXD[1]; no longer U$14.MTXD[2]
- net MTXD2: now also U$14.MTXD[2]
- net NODE1_4_IMON: now also U$1.PC0
- net NODE1_RX_N: now also J1.USB_L@1, J1.USB_L@2, R78.2, R82.1
- net NODE1_RX_P: now also J1.USB_H@1, J1.USB_H@2, R77.2, R81.1
- net NODE1_TX_P: now also J1.CAN_H@1, J1.CAN_H@2, R75.2, R79.1; no longer C31.2
- net NODE5_IMON: now also U$27.N0; no longer U$1.PC0
- net NODE6_IMON: now also U$27.N2; no longer U$1.PC1
- net NODE7_IMON: now also U$27.N3
- net NODE8_IMON: now also U$27.N4
Other:
- moved on the sheet: J1

Commit message: updated mcu page and symbol drawings
Parts:
- removed C102, C94: (no value), rcl:C-EUC0402K
- removed C35, C36, C39, C40, C43, C44, C47, C48, C51, C52, C53, C54, C55, C56, C59, C60: (no value), rcl:C-EUC0402
- removed E1, E2, E3, E4, E6: (no value), rcl_custom:L-BEAD-0603-B
- removed JTAG: BH20R, con-harting-ml:ML20R
- removed LED19, LED20, LED23, LED24, LED26, LED27, LED28, LED30, LED31, LED32, LED34, LED35, LED36: (no value), led:LEDCHIPLED_0603
- removed LED40, LED41, LED42, LED43, LED44, LED45, LED46: (no value), led:LEDSML0603
- removed R-T: Open, jumper:SJSJ_SMALLER
- removed RM4: NA(10k), OLIMEX_DISCRET:R_MATRIX_4E
- removed RM5: 10k, OLIMEX_DISCRET:R_MATRIX_4E
- removed SV1: (no value), con-lstb:MA06-1
- removed U$10: TPS2420QFN-16, RNH_TPS2420:TPS2420QFN-16
- removed U$20: ASE, crystal:ASE
- removed X8: 87758-0416, con-molex:87758-0416
- added C105: NP, rcl:C-EUC0402
- added C106, C107: (no value), rcl:C-EUC0402
- added D3: DIODE-0603, diode-0603:DIODE-0603
- added J9: DEBUG-CONNECTOR, ScottsLib:DEBUG-CONNECTOR
- added JP1: (no value), jumper:JP1Q
- added Q1: (no value), crystal:CRYSTALCTS406
- added R100, R101, R102, R103, R104, R105, R106, R115, R83, R84, R85, R86, R87, R88, R89, R90, R91, R92, R93, R94, R95, R96, R97, R98: (no value), rcl:R-US_R0402
- added R107, R110, R112: 220R, rcl:R-US_R0402
- added R108, R109, R111, R113, R114, R99: 10k, rcl:R-US_R0402
- added R116, R117, R118, R119, R120, R128: 10, rcl:R-US_R0402
- added R121, R122, R123, R124, R125, R126, R127: TBD, rcl:R-US_R0402
- added R129: 100R, rcl:R-US_R0402
- added TP1, TP10, TP11, TP12, TP13, TP14, TP15, TP16, TP17, TP18, TP19, TP2, TP20, TP21, TP22, TP23, TP24, TP25, TP26, TP27, TP28, TP29, TP3, TP30, TP31, TP32, TP33, TP34, TP35, TP37, TP38, TP39, TP4, TP40, TP41, TP42, TP5, TP6, TP7, TP8, TP9: TPTP06R, testpad:TPTP06R
- C7: value 0.1u -> NP
- LED10, LED12, LED15, LED18, LED2, LED4, LED7: value (none) -> RED; device led:LEDCHIPLED_0603 -> led:LEDSML0603
- LED11, LED14, LED16, LED3, LED6, LED8: value (none) -> GREEN; device led:LEDCHIPLED_0603 -> led:LEDSML0603
- LED39: value (none) -> GREEN
- R10, R2, R3, R4, R6, R7, R8: value 220 -> 10
- R11: value 1k -> 0R
- R14: value 220 -> 1k
- R15, R17: value 220 -> 2.2k
- R18, R21, R22, R25, R27, R29, R31, R35, R37, R40, R41: value 220 -> 10k
- R19, R23, R26, R30, R36, R39: value 220 -> 220R
- R33: value NA -> 220R; device rcl:R-EU_R0603_5MIL_DWS_NA -> rcl:R-US_R0402
- R34: value NA -> 10k; device rcl:R-EU_R0603_5MIL_DWS_NA -> rcl:R-US_R0402
- R49, R51, R52, R54, R56, R58, R60, R62, R66, R67, R68, R69, R70, R71: value (none) -> TBD
- R50, R53, R57, R63: value (none) -> 220R
- R55, R59, R61, R64, R65, R72: value (none) -> 10k
Connections:
- net N$15 renamed ETH_EN
- removed net +5V: U$2.IN
- removed net +5V_JTAG: JTAG.19, RM5G1.1
- removed net CTS: SV1.6, U$1.PD11
- removed net MIIS0: U$1.PA10
- removed net MIIS1: U$1.PA9
- removed net N$108: C16.2, C17.2, C19.2, C21.2, C22.2, C23.2, C24.2, C25.2, C26.2, C27.2, C28.2, C61.2, C62.2, C63.2, C64.2, C65.2, C66.2, C67.2, C68.2, C69.2, C70.2, C71.2, C78.2, C79.2, C80.2, E1.1, U$14.VDD_RCV, U$14.VDD_RCV1, U$14.VDD_RCV2, U$14.VDD_RCV3, U$14.VDD_RCV4, U$14.VDD_RCV5, U$14.VDD_RCV6, U$14.VDD_RCV7, U$14.VDD_RX, U$14.VDD_RX1, U$14.VDD_RX2, U$14.VDD_RX3, U$14.VDD_RX4, U$14.VDD_RX5, U$14.VDD_RX6, U$14.VDD_RX7, U$14.VDD_TX, U$14.VDD_TX1, U$14.VDD_TX2, U$14.VDD_TX3, U$14.VDD_TX4, U$14.VDD_TX5, U$14.VDD_TX6, U$14.VDD_TX7
- removed net N$112: E3.1
- removed net N$133: LED40.A, R53.1
- removed net N$134: LED41.A, R55.1
- removed net N$135: LED42.A, R57.1
- removed net N$136: LED43.A, R59.1
- removed net N$137: LED44.A, R61.1
- removed net N$138: LED45.A, R63.1
- removed net N$139: LED46.A, R65.1
- removed net N$146: C102.1, U$10.CT
- removed net N$151: R72.2, U$10.IMAX
- removed net NODE1_RX_N: C29.2, J1.USB_L@1, J1.USB_L@2, R78.2, R82.1
- removed net NODE1_RX_P: C30.2, J1.USB_H@1, J1.USB_H@2, R77.2, R81.1
- removed net NODE1_TX_N: C31.2, J1.CAN_L@1, J1.CAN_L@2, R76.2, R80.1
- removed net NODE1_TX_P: C32.2, J1.CAN_H@1, J1.CAN_H@2, R75.2, R79.1
- removed net NODE2_RX_N: C33.2, J2.USB_L@1, J2.USB_L@2
- removed net NODE2_RX_P: C34.2, J2.USB_H@1, J2.USB_H@2
- removed net NODE2_TXP: J2.CAN_H@1, J2.CAN_H@2
- removed net NODE2_TX_N: C35.2, J2.CAN_L@1, J2.CAN_L@2
- removed net NODE2_TX_P: C36.2
- removed net NODE3_RX_N: C37.2, J3.USB_L@1, J3.USB_L@2
- removed net NODE3_RX_P: C38.2, J3.USB_H@1, J3.USB_H@2
- removed net NODE3_TX_N: C39.2, J3.CAN_L@1, J3.CAN_L@2
- removed net NODE3_TX_P: C40.2, J3.CAN_H@1, J3.CAN_H@2
- removed net NODE4_RX_N: C41.2, J4.USB_L@1, J4.USB_L@2
- removed net NODE4_RX_P: C42.2, J4.USB_H@1, J4.USB_H@2
- removed net NODE4_TX_N: C43.2, J4.CAN_L@1, J4.CAN_L@2
- removed net NODE4_TX_P: C44.2, J4.CAN_H@1, J4.CAN_H@2
- removed net NODE5_RXM: C45.2, J5.USB_L@1, J5.USB_L@2
- removed net NODE5_RXP: C46.2, J5.USB_H@1, J5.USB_H@2
- removed net NODE5_TXM: C47.2, J5.CAN_L@1, J5.CAN_L@2
- removed net NODE6_RXM: C49.2, J6.USB_L@1, J6.USB_L@2
- removed net NODE6_RXP: C50.2, J6.USB_H@1, J6.USB_H@2
- removed net NODE6_TXM: C51.2, J6.CAN_L@1, J6.CAN_L@2
- removed net NODE7_RXM: C53.2, J7.USB_L@1, J7.USB_L@2
- removed net NODE7_RXP: C54.2, J7.USB_H@1, J7.USB_H@2
- removed net NODE7_TXM: C55.2, J7.CAN_L@1, J7.CAN_L@2
- removed net NODE7_TXP: C56.2, J7.CAN_H@1, J7.CAN_H@2
- removed net NODE8_!EN: U$1.PE7, U$10.!EN
- removed net NODE8_!FLT: U$1.PE15, U$10.!FLT
- removed net NODE8_!PG: LED46.C, U$1.PC13, U$10.!PG
- removed net NODE8_IMON: R64.2, U$10.IMON, U$27.N4
- removed net NODE8_LTCH: U$1.PD5, U$10.LTCH
- removed net NODE8_RSV1: J8.AUX_2@2, X8-1.S
- removed net NODE8_RSV2: J8.AUX_1@2, X8-2.S
- removed net NODE8_RSV3: J8.AUX_2@1, X8-3.S
- removed net NODE8_RSV4: J8.AUX_1@1, X8-4.S
- removed net NODE8_RXM: C57.2, J8.USB_L@1, J8.USB_L@2
- removed net NODE8_RXP: C58.2, J8.USB_H@1, J8.USB_H@2
- removed net NODE8_TXM: C59.2, J8.CAN_L@1, J8.CAN_L@2
- removed net NODE8_TXP: C60.2, J8.CAN_H@1, J8.CAN_H@2
- removed net NODE8_VOUT: J8.B+@1, J8.B+@2, U$10.OUT@10, U$10.OUT@11, U$10.OUT@12
- removed net RESET_N: C7.1, D1.CATHODE, R11.2, R12.2
- removed net RTS: SV1.2, U$1.PD12
- removed net VDD_IO: C13.2, C14.2, C15.2, C77.2, E3.2, T1.D, U$14.VDD-IO, U$14.VDD-IO1, U$14.VDD-IO2
- new net BAT_IMON: U$1.PA2
- new net BOOT0: J9.PORT2.10/!EINT0, R64.1, U$1.BOOT0
- new net DEBUG0: J9.DEBUG.13, TP40.TP
- new net DEBUG1: J9.DEBUG.14, TP41.TP
- new net DEBUG2: J9.DEBUG.15, TP42.TP
- new net ETH_RST_N: D3.CATHODE, U$1.PD4
- new net N$120: C42.1, J5.CAN_L@1, J5.CAN_L@2
- new net N$124: C46.1, J6.CAN_L@1, J6.CAN_L@2
- new net N$127: C49.1, J7.CAN_H@1, J7.CAN_H@2
- new net N$128: C50.1, J7.CAN_L@1, J7.CAN_L@2
- new net N$15: C107.2, Q1.2, U$1.PH0
- new net N$23: C29.2, J2.CAN_H@1, J2.CAN_H@2
- new net N$25: C30.2, J2.CAN_L@1, J2.CAN_L@2
- new net N$29: JP1.2, U$11.PGOOD
- new net N$30: JP1.1, LED22.C
- new net N$31: LED22.A, R128.1
- new net N$32: J9.3.3V, R129.1
- new net N$33: C58.1, J1.CAN_L@1, J1.CAN_L@2
- new net N$34: C57.1, J1.CAN_H@1, J1.CAN_H@2
- new net N$35: C33.2, J3.CAN_H@1, J3.CAN_H@2
- new net N$36: C34.2, J3.CAN_L@1, J3.CAN_L@2
- new net N$37: R72.1, U$1.PA10
- new net N$38: C31.1, J8.CAN_H@1, J8.CAN_H@2
- new net N$39: C37.2, J4.CAN_H@1, J4.CAN_H@2
- new net N$40: C38.2, J4.CAN_L@1, J4.CAN_L@2
- new net RESETOUT: J9.!RSTOUT, TP39.TP
- new net RTCK: J9.RTCK, TP38.TP
- new net VDDIO_IN: C13.2, C14.2, C15.2, C77.2, T1.D, U$14.VDD-IO, U$14.VDD-IO1, U$14.VDD-IO2
- new net VIN: J8.B+@1, J8.B+@2
- net +18V: no longer C94.1, U$10.IN@1, U$10.IN@2, U$10.IN@3, U$10.IN@4
- net +3V3: now also C1.1, C2.1, C3.1, C4.1, C5.1, C6.1, R107.2, R109.2, R110.2, R112.2, R114.2, R129.2, R15.1, R17.1, U$1.VDD1, U$1.VDD2, U$1.VDD3, U$1.VDD4, U$1.VDD5, U$1.VDD6, U$2.IN; no longer E4.1, JTAG.1, JTAG.2, R10.2, R14.2, R15.2, R17.2, R18.2, R2.2, R21.2, R25.2, R27.2, R3.2, R31.2, R34.2, R37.2, R4.2, R40.2, R55.2, R59.2, R6.2, R65.2, R7.2, R75.1, R76.1, R77.1, R78.1, R8.2, RM4G1.2, RM4G3.2, RM4G4.2, SV1.3, U$20.TRI, U$20.VDD
- net 25MHZ_REF_CLK: now also C105.1, C7.2, R11.1, R11.2
- net ACOK: now also U$1.PD0; no longer U$1.PA12
- net GND: now also C105.2, C106.1, C107.1, C77.1, C78.1, C79.1, C80.1, C81.1, J9.GRND, R10.2, R117.2, R118.2, R119.2, R120.2, R121.1, R122.1, R123.1, R124.1, R126.1, R127.1, R128.2, R14.1, R4.2, R6.2, R64.2, R7.2, R72.2, R8.2, R99.2; no longer C102.2, C7.2, C94.2, JTAG.10, JTAG.12, JTAG.14, JTAG.16, JTAG.18, JTAG.20, JTAG.4, JTAG.6, JTAG.8, R64.1, R72.1, R79.2, R80.2, R81.2, R82.2, RM4G2.1, RM5G1.2, RM5G2.2, RM5G3.2, SV1.1, U$10.GND@5, U$20.GND
- net IMON_A0: now also U$1.PD7; no longer U$1.PA4
- net IMON_A1: now also U$1.PD8; no longer U$1.PA5
- net JTAG_TCK: now also J9.TCK; no longer JTAG.9, RM4G2.2
- net JTAG_TDI: now also J9.TDI; no longer JTAG.5, RM4G1.1
- net JTAG_TDO: now also J9.TDO; no longer JTAG.13, R34.1
- net JTAG_TMS: now also J9.TMS; no longer JTAG.7, RM4G3.1
- net JTAG_TRST: now also J9.!TRST; no longer JTAG.3, R-T.1, RM4G4.1
- net MTXEN: now also R99.1
- net N$1: now also TP28.TP, U$2.FLG; no longer U$1.PH0, U$20.OUT
- net N$10: now also R6.1, U$14.MODESEL[2]; no longer LED3.A, R3.1
- net N$105: now also R14.2
- net N$107: now also D3.ANODE
- net N$109: now also R118.1, U$14.RLPBK; no longer C73.2, C74.2, C75.2, C76.2, C82.2, E2.1, U$14.VDD, U$14.VDD1, U$14.VDD2, U$14.VDD3
- net N$11: now also TP3.TP; no longer LED4.C
- net N$110: now also R119.1, U$14.SCANEN; no longer C72.2, C81.2, E6.1, U$14.VDD_PLL
- net N$111: now also R120.1, U$14.TESTEN; no longer C1.1, C2.1, C3.1, C4.1, C5.1, C6.1, E4.2, U$1.VDD1, U$1.VDD2, U$1.VDD3, U$1.VDD4, U$1.VDD5, U$1.VDD6
- net N$113: now also U$1.VREF+
- net N$131: now also R18.2
- net N$14: now also R7.1, U$14.MODESEL[1]; no longer LED4.A, R4.1
- net N$18: now also TP4.TP; no longer LED6.C
- net N$19: now also R8.1, U$14.MODESEL[0]; no longer LED6.A, R6.1
- net N$20: now also TP5.TP; no longer LED7.C
- net N$21: now also R10.1, U$14.CFGMODE; no longer LED7.A, R7.1
- net N$22: now also TP6.TP; no longer LED8.C
- net N$27: now also R2.1, U$14.MIIS[0]; no longer LED8.A, R8.1
- net N$44: now also TP7.TP; no longer LED10.C
- net N$45: now also LED3.A, R23.1, R25.2; no longer LED10.A, R10.1
- net N$46: now also TP8.TP; no longer LED11.C
- net N$47: now also R3.1, U$14.PRSV; no longer LED11.A, R14.1
- net N$48: now also TP9.TP; no longer LED12.C
- net N$49: now also LED2.A, R19.1, R21.2; no longer LED12.A, R15.1
- net N$5: now also C106.2, Q1.1, U$1.PH1; no longer JTAG.17, RM5G2.1
- net N$52: now also TP10.TP; no longer LED14.C
- net N$53: now also LED4.A, R26.1, R27.2; no longer LED14.A, R17.1
- net N$54: now also TP11.TP; no longer LED15.C
- net N$55: now also LED6.A, R30.1, R31.2; no longer LED15.A, R18.1
- net N$56: now also TP12.TP; no longer LED16.C
- net N$57: now also LED7.A, R33.1, R34.2; no longer LED16.A, R19.1
- net N$58: now also LED8.A, R36.1, R37.2; no longer U$1.PD15, U$2.FLG
- net N$60: now also TP13.TP; no longer LED18.C
- net N$61: now also LED10.A, R39.1, R40.2; no longer LED18.A, R21.1
- net N$62: now also TP14.TP; no longer LED19.C
- net N$63: now also LED11.A, R53.1, R55.2; no longer LED19.A, R22.1
- net N$64: now also TP15.TP; no longer LED20.C
- net N$65: now also LED12.A, R57.1, R59.2; no longer LED20.A, R23.1
- net N$66: now also U$1.PD12; no longer U$1.PD10
- net N$68: now also TP16.TP; no longer LED22.C
- net N$69: now also LED14.A, R63.1, R65.2; no longer LED22.A, R25.1
- net N$7: now also TP1.TP; no longer LED2.C
- net N$70: now also TP17.TP; no longer LED23.C
- net N$71: now also LED15.A, R107.1, R108.2; no longer LED23.A, R26.1
- net N$72: now also TP18.TP; no longer LED24.C
- net N$73: now also LED16.A, R110.1, R111.2; no longer LED24.A, R27.1
- net N$74: now also U$1.PD11; no longer U$1.PD7
- net N$76: now also TP19.TP; no longer LED26.C
- net N$77: now also LED18.A, R112.1, R113.2; no longer LED26.A, R29.1
- net N$78: now also TP20.TP; no longer LED27.C
- net N$79: now also C32.1, J8.CAN_L@1, J8.CAN_L@2; no longer LED27.A, R30.1
- net N$8: now also R4.1, U$14.MODESEL[3]; no longer LED2.A, R2.1
- net N$80: now also TP21.TP; no longer LED28.C
- net N$81: now also R117.1, U$14.BIST; no longer LED28.A, R31.1
- net N$84: now also TP22.TP; no longer LED30.C
- net N$85: now also R116.1, U$14.IO_SWM; no longer JTAG.11, R33.1, RM5G3.1
- net N$86: now also R121.2, U$9.IFLT; no longer LED30.A, R35.1
- net N$87: now also TP23.TP; no longer LED31.C
- net N$88: now also R122.2, U$8.IFLT; no longer LED31.A, R36.1
- net N$89: now also TP24.TP; no longer LED32.C
- net N$9: now also TP2.TP; no longer LED3.C
- net N$90: now also R123.2, U$7.IFLT; no longer LED32.A, R37.1
- net N$93: now also TP25.TP; no longer LED34.C
- net N$94: now also R124.2, U$6.IFLT; no longer LED34.A, R39.1
- net N$95: now also TP26.TP; no longer LED35.C
- net N$96: now also R126.2, U$4.IFLT; no longer LED35.A, R40.1
- net N$97: now also TP27.TP; no longer LED36.C
- net N$98: now also R127.2, U$3.IFLT; no longer LED36.A, R41.1
- net NODE1_!EN: now also R22.1
- net NODE1_!FLT: now also LED2.C, R21.1
- net NODE1_!PG: now also R18.1; no longer U$1.PC6
- net NODE1_IMON_IN: now also U$26.N1; no longer U$26.N0
- net NODE1_LTCH: no longer U$1.PC14
- net NODE2_!EN: now also R29.1
- net NODE2_!FLT: now also LED4.C, R27.1
- net NODE2_!PG: now also LED3.C, R25.1; no longer LED40.C, U$1.PC7
- net NODE2_LTCH: no longer U$1.PC15
- net NODE3_!EN: now also R35.1
- net NODE3_!FLT: now also LED7.C, R34.1
- net NODE3_!PG: now also LED6.C, R31.1; no longer LED41.C, U$1.PC8
- net NODE3_LTCH: no longer U$1.PD0
- net NODE4_!EN: now also R41.1
- net NODE4_!FLT: now also LED10.C, R40.1
- net NODE4_!PG: now also LED8.C, R37.1; no longer LED43.C, U$1.PD6
- net NODE4_LTCH: no longer U$1.PD1
- net NODE5_!EN: now also R61.1
- net NODE5_!FLT: now also LED12.C, R59.1
- net NODE5_!PG: now also LED11.C, R55.1; no longer LED42.C, U$1.PC10
- net NODE5_IMON: now also U$27.N1; no longer U$27.N0
- net NODE5_LTCH: no longer U$1.PD2
- net NODE5_TXP: now also C41.1; no longer C48.2
- net NODE6_!EN: now also R109.1
- net NODE6_!FLT: now also LED15.C, R108.1
- net NODE6_!PG: now also LED14.C, R65.1; no longer LED44.C, U$1.PC11
- net NODE6_LTCH: no longer U$1.PD3
- net NODE6_TXP: now also C45.1; no longer C52.2
- net NODE7_!EN: now also R114.1
- net NODE7_!FLT: now also LED18.C, R113.1
- net NODE7_!PG: now also LED16.C, R111.1; no longer LED45.C, U$1.PC12
- net NODE7_LTCH: no longer U$1.PD4
- net ROCKET_RDY: now also J8.AUX_1@1, J8.AUX_1@2, U$1.PD2; no longer U$1.PA11
- net RST_N: now also D1.CATHODE, J8.AUX_2@1, J8.AUX_2@2, J9.!RESET, R12.2, TP37.TP; no longer JTAG.15, R-T.2, R11.1, U$11.PGOOD
- net RX1_N: now also J1.USB_L@1, J1.USB_L@2, R78.2; no longer C29.1
- net RX1_P: now also J1.USB_H@1, J1.USB_H@2, R77.2; no longer C30.1
- net RX2_N: now also J2.USB_L@1, J2.USB_L@2, R82.2; no longer C33.1
- net RX2_P: now also J2.USB_H@1, J2.USB_H@2, R81.2; no longer C34.1
- net RX3_N: now also J3.USB_L@1, J3.USB_L@2, R86.2; no longer C37.1
- net RX3_P: now also J3.USB_H@1, J3.USB_H@2, R85.2; no longer C38.1
- net RX4_N: now also J4.USB_L@1, J4.USB_L@2, R90.2; no longer C41.1
- net RX4_P: now also J4.USB_H@1, J4.USB_H@2, R89.2; no longer C42.1
- net RX5_N: now also J5.USB_L@1, J5.USB_L@2, R94.2; no longer C45.1
- net RX5_P: now also J5.USB_H@1, J5.USB_H@2, R93.2; no longer C46.1
- net RX6_N: now also J6.USB_L@1, J6.USB_L@2, R106.2; no longer C49.1
- net RX6_P: now also J6.USB_H@1, J6.USB_H@2, R105.2; no longer C50.1
- net RX7_N: now also J7.USB_L@1, J7.USB_L@2, R98.2; no longer C53.1
- net RX7_P: now also J7.USB_H@1, J7.USB_H@2, R97.2; no longer C54.1
- net RX8_N: now also J8.USB_L@1, J8.USB_L@2, R115.2; no longer C57.1
- net RX8_P: now also J8.USB_H@1, J8.USB_H@2, R102.2; no longer C58.1
- net RXD: now also J9.PORT0.3/RXD0, U$1.PC11; no longer SV1.4, U$1.PD9
- net SCL: now also R17.2
- net SDA: now also R15.2
- net TX1_N: now also C58.2, R76.2; no longer C31.1
- net TX1_P: now also C57.2, R75.2; no longer C32.1
- net TX2_N: now also C30.1, R80.2; no longer C35.1
- net TX2_P: now also C29.1, R79.2; no longer C36.1
- net TX3_N: now also C34.1, R84.2; no longer C39.1
- net TX3_P: now also C33.1, R83.2; no longer C40.1
- net TX4_N: now also C38.1, R88.2; no longer C43.1
- net TX4_P: now also C37.1, R87.2; no longer C44.1
- net TX5_N: now also C42.2, R92.2; no longer C47.1
- net TX5_P: now also C41.2, R91.2; no longer C48.1
- net TX6_N: now also C46.2, R104.2; no longer C51.1
- net TX6_P: now also C45.2, R103.2; no longer C52.1
- net TX7_N: now also C50.2, R96.2; no longer C55.1
- net TX7_P: now also C49.2, R95.2; no longer C56.1
- net TX8_N: now also C32.2, R101.2; no longer C59.1
- net TX8_P: now also C31.2, R100.2; no longer C60.1
- net TXD: now also J9.PORT0.2/TXD0, U$1.PC10; no longer SV1.5, U$1.PD8
- net VDD: now also C16.2, C17.2, C18.2, C19.2, C20.2, C21.2, C22.2, C23.2, C24.2, C25.2, C26.2, C27.2, C28.2, C61.2, C62.2, C63.2, C64.2, C65.2, C66.2, C67.2, C68.2, C69.2, C7.1, C70.2, C71.2, C72.2, C73.2, C74.2, C75.2, C76.2, C78.2, C79.2, C80.2, C81.2, C82.2, R100.1, R101.1, R102.1, R103.1, R104.1, R105.1, R106.1, R115.1, R116.2, R2.2, R3.2, R75.1, R76.1, R77.1, R78.1, R79.1, R80.1, R81.1, R82.1, R83.1, R84.1, R85.1, R86.1, R87.1, R88.1, R89.1, R90.1, R91.1, R92.1, R93.1, R94.1, R95.1, R96.1, R97.1, R98.1, U$14.VDD, U$14.VDD1, U$14.VDD2, U$14.VDD3, U$14.VDD_PLL, U$14.VDD_RCV, U$14.VDD_RCV1, U$14.VDD_RCV2, U$14.VDD_RCV3, U$14.VDD_RCV4, U$14.VDD_RCV5, U$14.VDD_RCV6, U$14.VDD_RCV7, U$14.VDD_RX, U$14.VDD_RX1, U$14.VDD_RX2, U$14.VDD_RX3, U$14.VDD_RX4, U$14.VDD_RX5, U$14.VDD_RX6, U$14.VDD_RX7, U$14.VDD_TX, U$14.VDD_TX1, U$14.VDD_TX2, U$14.VDD_TX3, U$14.VDD_TX4, U$14.VDD_TX5, U$14.VDD_TX6, U$14.VDD_TX7; no longer E1.2, E2.2, E6.2
Other:
- note added: "2.1V Linear Supply"
- note added: "3.3V Switching Supply"
- note added: "Debug Header"
- note added: "Launch Tower Connection"
- note removed: "JTAG"
- note removed: "Reset"
- note removed: "UART"

Commit message: Added component selection guide for all ICs
Parts:
- removed C105, C7: NP, rcl:C-EUC0402
- added R130, R131: 10k, rcl:R-US_R0402
- added R132, R133: NP, rcl:R-US_R0402
- Q1: value (none) -> 25MHz
- renumbered U$1 to U1
Connections:
- net 25MHZ_REF_CLK: now also R132.2, R133.1; no longer C105.1, C7.2
- net ETH_EN: now also R130.1
- net GND: now also R130.2, R131.2, R133.2; no longer C105.2
- net NODE5_LTCH: now also TP33.TP
- net NODE6_LTCH: now also TP34.TP
- net NODE7_LTCH: now also TP35.TP
- net SYNC: now also R131.1
- net VDD: now also R132.1; no longer C7.1
Other:
- moved on the sheet: C100, C101, C11, C41, C42, C45, C46, C49, C50, C91, C92, C93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

Commit message: re-placed layout on mcu_page
Parts:
- added C35, C36, C39, C40, C43, C44, C47, C48, C51, C52, C53, C54, C55, C7: (no value), rcl:C-EUC0402
- R107, R110, R112, R19, R23, R26, R30, R33, R36, R39, R50, R53, R57, R63: value 220R -> 56
Connections:
- net NODE5_VOUT renamed NODE8_VOUT
- new net N$112: C7.1, J1.USB_H@1, J1.USB_H@2
- new net N$118: C35.1, J1.USB_L@1, J1.USB_L@2
- new net N$119: C55.1, J7.USB_L@1, J7.USB_L@2
- new net N$121: C54.1, J7.USB_H@1, J7.USB_H@2
- new net N$122: C53.1, J6.USB_L@1, J6.USB_L@2
- new net N$123: C52.1, J6.USB_H@1, J6.USB_H@2
- new net N$125: C51.1, J5.USB_L@1, J5.USB_L@2
- new net N$126: C48.1, J5.USB_H@1, J5.USB_H@2
- new net N$129: C44.2, J4.USB_H@1, J4.USB_H@2
- new net N$133: C47.2, J4.USB_L@1, J4.USB_L@2
- new net N$134: C40.2, J3.USB_H@1, J3.USB_H@2
- new net N$135: C43.2, J3.USB_L@1, J3.USB_L@2
- new net N$136: C36.2, J2.USB_H@1, J2.USB_H@2
- new net N$137: C39.2, J2.USB_L@1, J2.USB_L@2
- new net N$138: R11.1, R132.2, R133.1, U$14.X1
- new net N$139: R125.2, U$5.IFLT
- new net NODE8_!EN: R61.1, U$7.!EN
- new net NODE8_!FLT: LED12.C, R59.1, U$7.!FLT
- net +3V3: now also R108.2, R111.2, R113.2, R18.2, R21.2, R25.2, R27.2, R31.2, R34.2, R37.2, R40.2, R55.2, R59.2, R65.2
- net 25MHZ_REF_CLK: no longer R11.1, R132.2, R133.1, U$14.X1
- net GND: now also R125.1
- net N$131: no longer R18.2
- net N$45: no longer R25.2
- net N$49: no longer R21.2
- net N$53: no longer R27.2
- net N$55: no longer R31.2
- net N$57: no longer R34.2
- net N$58: no longer R37.2
- net N$61: no longer R40.2
- net N$63: no longer R55.2
- net N$65: no longer R59.2
- net N$69: no longer R65.2
- net N$71: no longer R108.2
- net N$73: no longer R111.2
- net N$77: no longer R113.2
- net NODE1_LTCH: now also TP29.TP
- net NODE2_LTCH: now also TP30.TP
- net NODE3_LTCH: now also TP31.TP
- net NODE4_LTCH: now also TP32.TP
- net NODE5_!EN: no longer R61.1, U$7.!EN
- net NODE5_!FLT: no longer LED12.C, R59.1, U$7.!FLT
- net RX1_N: now also C58.2, R76.2; no longer J1.USB_L@1, J1.USB_L@2, R78.2
- net RX1_P: now also C57.2, R75.2; no longer J1.USB_H@1, J1.USB_H@2, R77.2
- net RX2_N: now also C39.1; no longer J2.USB_L@1, J2.USB_L@2
- net RX2_P: now also C36.1; no longer J2.USB_H@1, J2.USB_H@2
- net RX3_N: now also C34.1, R84.2; no longer J3.USB_L@1, J3.USB_L@2, R86.2
- net RX3_P: now also C33.1, R83.2; no longer J3.USB_H@1, J3.USB_H@2, R85.2
- net RX4_N: now also C47.1; no longer J4.USB_L@1, J4.USB_L@2
- net RX4_P: now also C44.1; no longer J4.USB_H@1, J4.USB_H@2
- net RX5_N: no longer J5.USB_L@1, J5.USB_L@2, R94.2
- net RX5_P: no longer J5.USB_H@1, J5.USB_H@2, R93.2
- net RX6_N: now also C53.2; no longer J6.USB_L@1, J6.USB_L@2
- net RX6_P: now also C52.2; no longer J6.USB_H@1, J6.USB_H@2
- net RX7_N: now also C55.2; no longer J7.USB_L@1, J7.USB_L@2
- net RX7_P: now also C54.2; no longer J7.USB_H@1, J7.USB_H@2
- net RX8_N: now also C51.2, R94.2
- net RX8_P: now also C48.2, R93.2
- net TX1_N: now also C35.2, R78.2; no longer C58.2, R76.2
- net TX1_P: now also C7.2, R77.2; no longer C57.2, R75.2
- net TX3_N: now also C43.1, R86.2; no longer C34.1, R84.2
- net TX3_P: now also C40.1, R85.2; no longer C33.1, R83.2
- net TX5_N: no longer C42.2, R92.2
- net TX5_P: no longer C41.2, R91.2
- net TX8_N: now also C42.2, R92.2
- net TX8_P: now also C41.2, R91.2
Other:
- moved on the sheet: J2, J3, J4, J5, J6, J7, R125, TP31, TP32

Commit message: switched J5 and J8 nets on the mcu page
Parts:
- added C56, C59: (no value), rcl:C-EUC0402
Connections:
- new net N$108: C59.1, J8.USB_L@1, J8.USB_L@2
- new net N$141: C56.1, J8.USB_H@1, J8.USB_H@2
- net RX5_N: now also C59.2, R115.2
- net RX5_P: now also C56.2, R102.2
- net RX8_N: no longer J8.USB_L@1, J8.USB_L@2, R115.2
- net RX8_P: no longer J8.USB_H@1, J8.USB_H@2, R102.2
- net TX5_N: now also C32.2, R101.2
- net TX5_P: now also C31.2, R100.2
- net TX8_N: no longer C32.2, R101.2
- net TX8_P: no longer C31.2, R100.2
Other:
- moved on the sheet: C31, C32, J8, R100, R101, R102, R115

Commit message: moved ethernet switch and mcu/sps around
Connections:
- removed net NODE5_RSV1: J5.AUX_2@2, X5-1.S
- removed net NODE5_RSV2: J5.AUX_1@2, X5-2.S
- removed net NODE5_RSV3: J5.AUX_2@1, X5-3.S
- removed net NODE5_RSV4: J5.AUX_1@1, X5-4.S
- removed net NODE5_TXP: C41.1, J5.CAN_H@1, J5.CAN_H@2
- new net NODE8_RSV1: J8.AUX_2@2, X5-1.S
- new net NODE8_RSV2: J8.AUX_1@2, X5-2.S
- new net NODE8_RSV3: J8.AUX_2@1, X5-3.S
- new net NODE8_RSV4: J8.AUX_1@1, X5-4.S
- new net NODE8_TXP: C41.1, J8.CAN_H@1, J8.CAN_H@2
- net N$108: now also J5.USB_L@1, J5.USB_L@2; no longer J8.USB_L@1, J8.USB_L@2
- net N$120: now also J8.CAN_L@1, J8.CAN_L@2; no longer J5.CAN_L@1, J5.CAN_L@2
- net N$125: now also J8.USB_L@1, J8.USB_L@2; no longer J5.USB_L@1, J5.USB_L@2
- net N$126: now also J8.USB_H@1, J8.USB_H@2; no longer J5.USB_H@1, J5.USB_H@2
- net N$141: now also J5.USB_H@1, J5.USB_H@2; no longer J8.USB_H@1, J8.USB_H@2
- net N$38: now also J5.CAN_H@1, J5.CAN_H@2; no longer J8.CAN_H@1, J8.CAN_H@2
- net N$79: now also J5.CAN_L@1, J5.CAN_L@2; no longer J8.CAN_L@1, J8.CAN_L@2
- net NODE8_VOUT: now also J8.B+@1, J8.B+@2; no longer J5.B+@1, J5.B+@2
- net ROCKET_RDY: now also J5.AUX_1@1, J5.AUX_1@2; no longer J8.AUX_1@1, J8.AUX_1@2
- net RST_N: now also J5.AUX_2@1, J5.AUX_2@2; no longer J8.AUX_2@1, J8.AUX_2@2
- net VIN: now also J5.B+@1, J5.B+@2; no longer J8.B+@1, J8.B+@2

Commit message: added center mounting hole
Parts:
- removed R11: 0R, rcl:R-US_R0402
- removed R132, R133: NP, rcl:R-US_R0402
Connections:
- removed net N$138: R11.1, R132.2, R133.1, U$14.X1
- net 25MHZ_REF_CLK: now also U$14.X1; no longer R11.2
- net GND: no longer R133.2
- net VDD: no longer R132.1
Changed lines of the file:
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@@
 <part name="TP28" library="testpad" deviceset="TP" device="TP06R"/>
 <part name="GND7" library="supply1" deviceset="GND" device=""/>
-<part name="R11" library="rcl" deviceset="R-US_" device="R0402" value="0R"/>
-<part name="VDD14" library="supply1" deviceset="VDD" device=""/>
-<part name="GND10" library="supply1" deviceset="GND" device=""/>
 <part name="R15" library="rcl" deviceset="R-US_" device="R0402" value="2.2k"/>
 <part name="R17" library="rcl" deviceset="R-US_" device="R0402" value="2.2k"/>
@@
 <part name="R131" library="rcl" deviceset="R-US_" device="R0402" value="10k"/>
 <part name="GND57" library="supply1" deviceset="GND" device=""/>
-<part name="R132" library="rcl" deviceset="R-US_" device="R0402" value="NP"/>
-<part name="R133" library="rcl" deviceset="R-US_" device="R0402" value="NP"/>
 <part name="C7" library="rcl" deviceset="C-EU" device="C0402"/>
 <part name="C35" library="rcl" deviceset="C-EU" device="C0402"/>
@@
 <instance part="R14" gate="G$1" x="195.58" y="30.48" rot="R90"/>
 <instance part="GND7" gate="1" x="187.96" y="236.22"/>
-<instance part="R11" gate="G$1" x="20.32" y="149.86" rot="R180"/>
-<instance part="VDD14" gate="G$1" x="50.8" y="167.64"/>
-<instance part="GND10" gate="1" x="50.8" y="132.08"/>
 <instance part="D3" gate="G$1" x="15.24" y="180.34"/>
 <instance part="R116" gate="G$1" x="66.04" y="86.36" rot="R180"/>
@@
 <instance part="R120" gate="G$1" x="66.04" y="27.94" rot="R180"/>
 <instance part="FRAME4" gate="G$1" x="287.02" y="7.62"/>
-<instance part="R132" gate="G$1" x="50.8" y="157.48" rot="R270"/>
-<instance part="R133" gate="G$1" x="50.8" y="142.24" rot="R270"/>
 </instances>
 <busses>
@@
 <wire x1="187.96" y1="241.3" x2="187.96" y2="238.76" width="0.1524" layer="91"/>
 </segment>
-<segment>
-<pinref part="GND10" gate="1" pin="GND"/>
-<pinref part="R133" gate="G$1" pin="2"/>
-<wire x1="50.8" y1="134.62" x2="50.8" y2="137.16" width="0.1524" layer="91"/>
-</segment>
 </net>
 <net name="+3V3" class="1">
@@
 <net name="25MHZ_REF_CLK" class="0">
 <segment>
-<pinref part="R11" gate="G$1" pin="2"/>
-<wire x1="10.16" y1="149.86" x2="15.24" y2="149.86" width="0.1524" layer="91"/>
 <label x="10.16" y="149.86" size="1.016" layer="95" rot="R180" xref="yes"/>
+<pinref part="U$14" gate="G$1" pin="X1"/>
+<wire x1="10.16" y1="149.86" x2="78.74" y2="149.86" width="0.1524" layer="91"/>
 </segment>
 </net>
@@
 <wire x1="48.26" y1="223.52" x2="50.8" y2="223.52" width="0.1524" layer="91"/>
 </segment>
-<segment>
-<pinref part="VDD14" gate="G$1" pin="VDD"/>
-<wire x1="50.8" y1="162.56" x2="50.8" y2="165.1" width="0.1524" layer="91"/>
-<pinref part="R132" gate="G$1" pin="1"/>
-</segment>
 </net>
 <net name="ETH_EN" class="0">
@@
 </segment>
 </net>
-<net name="N$138" class="0">
-<segment>
-<pinref part="R11" gate="G$1" pin="1"/>
-<pinref part="U$14" gate="G$1" pin="X1"/>
-<wire x1="25.4" y1="149.86" x2="50.8" y2="149.86" width="0.1524" layer="91"/>
-<pinref part="R133" gate="G$1" pin="1"/>
-<wire x1="50.8" y1="149.86" x2="78.74" y2="149.86" width="0.1524" layer="91"/>
-<wire x1="50.8" y1="147.32" x2="50.8" y2="149.86" width="0.1524" layer="91"/>
-<junction x="50.8" y="149.86"/>
-<pinref part="R132" gate="G$1" pin="2"/>
-<wire x1="50.8" y1="149.86" x2="50.8" y2="152.4" width="0.1524" layer="91"/>
-</segment>
-</net>
