File: av3/rocketnet-hub/eagle/mcu_page.brd (EAGLE design)
At the start: 113 x 77 mm, 333 parts, among them J1 ROCKETBUS, J2 ROCKETBUS, J3 ROCKETBUS, J4 ROCKETBUS, J5 ROCKETBUS, J6 ROCKETBUS, J7 ROCKETBUS, J8 ROCKETBUS, Q1 25.000MHz, X1 87758-0416, X2 87758-0416, X3 87758-0416, X4 87758-0416, X5 87758-0416, X6 87758-0416, X7 87758-0416, X8 87758-0416

Commit message: incremental
Parts:
- moved C10 52.5 mm to (109.8, 34.7)
- moved C11 52.5 mm to (94.8, 34.9)
- moved C1 52.2 mm to (101.7, 48.4)
- moved C5 52.2 mm to (96.9, 58.2)
- moved C6 52.2 mm to (97.7, 47.7)
- moved C86 52.2 mm to (107.0, 48.9)
- moved C9 52.2 mm to (98.2, 58.2)
- moved LED37 52.2 mm to (112.2, 67.6)
- moved Q1 52.2 mm to (102.2, 37.5)
- moved R44 52.2 mm to (110.9, 63.1)
- moved SV1 52.2 mm to (100.8, 71.3)
- moved C2 52.2 mm to (105.6, 48.9)
- moved C3 52.2 mm to (108.3, 48.9)
- moved C4 52.2 mm to (107.6, 59.3)
- moved C8 52.2 mm to (107.6, 58.1)
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
Commit message: layout updates
Parts:
- removed C10, C11: 27p, rcl:C0402
- removed Q1: 25.000MHz, crystal:SM49
- added U$20: ASE, crystal:ASE
- added U$21, U$22, U$23, U$24, U$25: #4-BARE_MOUNTING_HOLE/.300, mount:#4/.300-BARE+STD_NUT_OR_STAR_WASHER
- moved R51 104.4 mm to (96.9, 72.6), turned to 90 degrees
- moved LED39 102.0 mm to (91.9, 78.5), turned to 270 degrees
- moved R74 100.9 mm to (104.1, 56.0), turned to 180 degrees
- moved U$11 100.4 mm to (106.6, 61.7), turned to 180 degrees
- moved C104 98.7 mm to (107.5, 67.5), turned to 0 degrees
- moved R73 94.4 mm to (99.6, 57.3), turned to 90 degrees
- moved C103 94.1 mm to (104.1, 67.5), turned to 0 degrees
- moved R52 94.0 mm to (79.9, 80.4), flipped to the bottom, turned to 90 degrees
- moved R65 84.7 mm to (100.6, 28.1)
- moved R66 82.9 mm to (71.0, 73.5), turned to 270 degrees
- moved R53 82.9 mm to (68.5, 78.5), flipped to the bottom, turned to 90 degrees
- moved LED40 81.7 mm to (68.5, 78.6), turned to 270 degrees
- moved R59 80.7 mm to (35.3, 87.7), flipped to the bottom, turned to 90 degrees
- moved R58 80.2 mm to (33.5, 87.7), flipped to the bottom, turned to 270 degrees
- moved R49 77.9 mm to (104.8, 80.3), flipped to the bottom, turned to 90 degrees
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Connections:
- net N$23 renamed RX1_N
- net N$24 renamed RX2_N
- net N$25 renamed TX1_P
- net N$26 renamed TX2_P
- net N$29 renamed RX3_N
- net N$30 renamed TX3_P
- net N$31 renamed RX4_N
- net N$32 renamed TX4_P
- net NODE2_RXM renamed NODE2_RX_N
- net NODE2_RXP renamed NODE2_RX_P
- net NODE2_TXM renamed NODE2_TX_N
- net NODE3_RXM renamed NODE3_RX_N
- net NODE3_RXP renamed NODE3_RX_P
- net NODE3_TXM renamed NODE3_TX_N
- net NODE3_TXP renamed NODE3_TX_P
- net NODE4_RXM renamed NODE4_RX_N
- net NODE4_RXP renamed NODE4_RX_P
- net NODE4_TXM renamed NODE4_TX_N
- net NODE4_TXP renamed NODE4_TX_P
- net RXP1 renamed RX1_P
- net RXP2 renamed RX2_P
- net RXP3 renamed RX3_P
- net RXP4 renamed RX4_P
- net TXM1 renamed TX1_N
- net TXM2 renamed TX2_N
- net TXM3 renamed TX3_N
- net TXM4 renamed TX4_N
- removed net N$125: C90.2, U$6.5
- removed net N$152: R71.2
- removed net N$153: R72.2
- removed net N$154: U$7.8
- removed net N$155: U$9.8
- removed net N$157: U$4.8
- removed net N$158: U$6.8
- removed net N$159: U$8.8
- removed net N$2 (its old number): C10.2, Q1.2, U$1.13
- removed net N$4 (its old number): C11.1
- removed net NODE1_ILIM: U$3.8
- removed net NODE8_ILIM: U$10.8
- new net N$130: R67.2, U$5.7
- new net NODE1_RX_N: C29.2
- new net NODE1_RX_P: C30.2
- new net NODE1_TX_P: C31.2, C32.2
- new net NODE2_TX_P: C36.2
- net +3V3: now also U$20.1, U$20.4
- net GND: now also C90.2, U$20.2, U$6.5; no longer C10.1
- net N$1: now also U$20.3; no longer C11.2, Q1.1
- net N$147: now also R68.2, U$6.7; no longer U$5.8
- net N$148: now also R69.2, U$7.7; no longer R67.2
- net N$149: now also R70.2, U$8.7; no longer R68.2
- net N$150: now also R71.2, U$9.7; no longer R69.2
- net N$151: now also R72.2, U$10.7; no longer R70.2
- net NODE1_RXM: no longer C29.2
- net NODE1_RXP: no longer C30.2
- net NODE1_TXM: no longer C31.2
- net NODE1_TXP: no longer C32.2
- net NODE2_TXP: no longer C36.2
Routing:
- net N$108: track 0.00 -> 111.3 mm, vias 0 -> 23
- net RX1_P: track 0.00 -> 48.8 mm
- net RX1_N: track 0.00 -> 48.0 mm
- net RX4_N: track 0.00 -> 40.6 mm
- net RX4_P: track 0.00 -> 39.9 mm
- net TX4_N: track 0.00 -> 37.2 mm
- net TX4_P: track 0.00 -> 36.5 mm
- net TX2_N: track 0.00 -> 31.2 mm
- net TX2_P: track 0.00 -> 31.1 mm
- net RX2_P: track 0.00 -> 30.1 mm
- net RX2_N: track 0.00 -> 29.2 mm
- net TX3_P: track 0.00 -> 19.3 mm
- net TX3_N: track 0.00 -> 19.1 mm
- net RX3_P: track 0.00 -> 13.5 mm, vias 0 -> 2
- net RX3_N: track 0.00 -> 13.3 mm, vias 0 -> 2
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- added copper zone on layer 15, net +18V
- added copper zone on layer 16, net +18V
- added copper zone on layer 16, net GND
- added copper zone on layer 2, net GND
- added copper zone on layer 16, net NODE4_VOUT
- added copper zone on layer 15, net TEMP
- added copper zone on layer 3, net TEMP
- added copper zone on layer 16, net VDD
Other:
- board size 113 x 77 mm -> 112.7 x 76.2 mm

Commit message: Rearranged the layout of switch circuit - work in progress
Parts:
- moved X5 23.0 mm to (17.6, 23.2)
- moved R50 21.3 mm to (112.8, 74.1), turned to 270 degrees
- moved R62 20.3 mm to (88.1, 17.6), flipped to the bottom
- moved R55 19.6 mm to (61.0, 87.5)
- moved R53 19.5 mm to (85.8, 87.5)
- moved R28 17.2 mm to (66.0, 79.0), turned to 180 degrees
- moved R60 16.9 mm to (64.5, 17.3), flipped to the bottom
- moved R32 16.8 mm to (41.4, 78.7), turned to 180 degrees
- moved R24 16.7 mm to (91.2, 78.7), turned to 180 degrees
- moved LED25 16.7 mm to (66.4, 78.9), turned to 270 degrees
- moved LED29 16.3 mm to (41.8, 78.6), turned to 270 degrees
- moved LED21 16.3 mm to (91.5, 78.7), turned to 270 degrees
- moved R29 16.3 mm to (66.1, 77.7), turned to 180 degrees
- moved R35 16.1 mm to (41.5, 77.5), turned to 180 degrees
- moved LED26 15.9 mm to (66.4, 77.9), turned to 270 degrees
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Connections:
- net N$141 renamed RATSNET
- removed net N$123: C88.2, U$4.5
- removed net N$124: C87.2, U$5.5
- net GND: now also C87.2, C88.2, U$4.5, U$5.5
Routing:
- net RX1_N: track 48.0 -> 54.3 mm
- net RX1_P: track 48.8 -> 54.9 mm
- net NODE3_IMON: track 0.00 -> 6.10 mm
- net NODE2_IMON: track 0.00 -> 6.00 mm
- net N$133: track 0.00 -> 5.76 mm, vias 0 -> 1
- net N$134: track 0.00 -> 5.76 mm, vias 0 -> 1
- net TX2_P: track 31.1 -> 36.7 mm
- net TX2_N: track 31.2 -> 36.8 mm
- net RX2_P: track 30.1 -> 35.6 mm
- net GND: track 3.38 -> 8.00 mm, vias 6 -> 16
- net TX3_N: track 19.1 -> 23.7 mm
- net RX3_P: track 13.5 -> 18.1 mm
- net RX3_N: track 13.3 -> 17.9 mm
- net TX3_P: track 19.3 -> 23.8 mm
- net N$4: track 0.00 -> 4.01 mm, vias 0 -> 1
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- added copper zone on layer 16, net NODE2_VOUT
- added copper zone on layer 16, net NODE3_VOUT

Commit message: Improved upon layout for bottom switches on layout
Parts:
- moved C98 2.06 mm to (34.3, 25.9), turned to 90 degrees
- moved C102 1.98 mm to (107.0, 25.9)
- moved R72 1.84 mm to (104.7, 27.6), turned to 0 degrees
- moved C94 1.63 mm to (101.7, 26.0), turned to 90 degrees
- moved C92 1.49 mm to (56.1, 25.8)
- moved C91 1.22 mm to (28.9, 25.9)
- moved C101 1.21 mm to (85.1, 26.0)
- moved C100 1.20 mm to (61.4, 25.8)
- moved C93 1.00 mm to (79.8, 26.0), turned to 90 degrees
- moved R69 1.00 mm to (32.0, 27.8), turned to 0 degrees
- moved R70 0.92 mm to (59.1, 27.6), turned to 0 degrees
- moved R62 0.61 mm to (87.5, 17.7)
- moved LED44 0.60 mm to (59.1, 22.2)
- moved U$8 0.60 mm to (59.4, 24.2)
- moved LED42 0.51 mm to (32.0, 22.3)
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
Commit message: Routed some capacitors/resistors on the current switch
Parts:
- moved R56 0.51 mm to (37.2, 17.6)
- turned LED42 to 180 degrees
Routing:
- net N$137: track 0.00 -> 7.57 mm, vias 0 -> 1
- net N$135: track 0.00 -> 7.24 mm, vias 0 -> 1
- net N$138: track 0.00 -> 6.86 mm, vias 0 -> 1
- net NODE5_IMON: track 0.00 -> 6.65 mm
- net GND: track 8.00 -> 14.1 mm
- net NODE7_IMON: track 0.00 -> 6.00 mm
- net N$148: track 0.00 -> 2.74 mm, vias 0 -> 1
- net N$149: track 0.00 -> 2.72 mm, vias 0 -> 1
- net N$150: track 0.00 -> 2.72 mm, vias 0 -> 1
- net N$151: track 0.00 -> 2.54 mm, vias 0 -> 1
- net NODE6_IMON: track 0.00 -> 0.64 mm

Commit message: added vias to center pad to package
Parts:
- added U$26, U$27: MAX4734ETC+, max4734:TQFN-12
- flipped C99 to the top
Connections:
- new net N$30: U$26.P$13, U$26.P$2
- new net N$31: U$26.P$8
- net GND: now also U$4.DAP, U$4.P$10, U$4.P$2, U$4.P$3, U$4.P$4, U$4.P$5, U$4.P$6, U$4.P$7, U$4.P$8, U$4.P$9, U$5.DAP, U$5.P$10, U$5.P$2, U$5.P$3, U$5.P$4, U$5.P$5, U$5.P$6, U$5.P$7, U$5.P$8, U$5.P$9, U$6.DAP, U$6.P$10, U$6.P$2, U$6.P$3, U$6.P$4, U$6.P$5, U$6.P$6, U$6.P$7, U$6.P$8, U$6.P$9
- net N$122: now also U$3.DAP, U$3.P$10, U$3.P$2, U$3.P$3, U$3.P$4, U$3.P$5, U$3.P$6, U$3.P$7, U$3.P$8, U$3.P$9
- net N$126: now also U$7.DAP, U$7.P$10, U$7.P$2, U$7.P$3, U$7.P$4, U$7.P$5, U$7.P$6, U$7.P$7, U$7.P$8, U$7.P$9
- net N$127: now also U$8.DAP, U$8.P$10, U$8.P$2, U$8.P$3, U$8.P$4, U$8.P$5, U$8.P$6, U$8.P$7, U$8.P$8, U$8.P$9
- net N$128: now also U$9.DAP, U$9.P$10, U$9.P$2, U$9.P$3, U$9.P$4, U$9.P$5, U$9.P$6, U$9.P$7, U$9.P$8, U$9.P$9
- net N$129: now also U$10.DAP, U$10.P$10, U$10.P$2, U$10.P$3, U$10.P$4, U$10.P$5, U$10.P$6, U$10.P$7, U$10.P$8, U$10.P$9
- net NODE1_IMON: now also U$26.P$1
- net NODE2_IMON: now also U$26.P$9
- net NODE3_IMON: now also U$26.P$3
- net NODE4_IMON: now also U$26.P$7
Routing:
- net NODE4_IMON: track 5.87 -> 45.9 mm, vias 0 -> 2
- net NODE3_IMON: track 6.10 -> 19.7 mm
- net N$143: track 0.74 -> 1.47 mm
- net GND: track 14.1 -> 14.4 mm, vias 16 -> 15

Commit message: updated layout.
Parts:
- removed C105, C106, C107, C108, C109, C110, C111, C112, C113, C114, C115, C116, C117, C118, C119, C120, C121, C122, C123, C124, C125, C126, C127, C128, C129, C130: (no value), rcl:C0402
- removed D3: BAT54, diode:SOT23
- removed D4: BAT54C, diode:SOT23
- removed JP1, JP2, JP3: (no value), pinhead:1X03
- removed JP4, JP5: (no value), pinhead:1X02
- removed L2, R75, R76, R88, R89, R90, R92, R94, R95: (no value), rcl_custom:0603-B
- removed R77: 100k, rcl_custom:0603-B
- removed R78: 316k, rcl_custom:0603-B
- removed R79, R91, R93, R96: 12.1k, rcl_custom:0603-B
- removed R80: 10k, rcl_custom:0603-B
- removed R81, R82: 4.02k, rcl_custom:0603-B
- removed R83: 66.5k, rcl_custom:0603-B
- removed R84, R86, R87: 430k, rcl_custom:0603-B
- removed R85, R97, R98: 10, rcl_custom:0603-B
- removed U$12: BQ24725QFN-20, RNH_BQ24725:S-PVQFN-N20
- removed U$13: BSS138W-7-F, RNH_BSS138W-7-F:SOT-23
- removed U$15, U$16, U$17: FDS6680ASOIC-8, RNH_FDS6680A:MS-012
- removed U$18, U$19: SIS412DNSOP-8, RNH_SIS412DN:1212-8
- added C10: (no value), rcl:C0402K
- moved RM5 139.8 mm to (5.45, 16.7), turned to 180 degrees
- moved R34 132.8 mm to (6.65, 21.5), turned to 180 degrees
- moved JTAG 109.7 mm to (11.2, 37.3), turned to 270 degrees
- moved RM4 92.5 mm to (5.77, 51.1), turned to 180 degrees
- moved R-T 86.2 mm to (5.46, 56.0), turned to 0 degrees
- moved R33 80.6 mm to (5.87, 60.0), turned to 180 degrees
- moved LED37 33.1 mm to (106.5, 29.5)
- moved R44 33.1 mm to (106.5, 28.7)
- moved R45 33.1 mm to (105.5, 30.4)
- moved R46 33.1 mm to (107.7, 30.4)
- moved LED1 30.1 mm to (106.4, 33.8)
- moved LED2 30.1 mm to (107.5, 33.8)
- moved LED3 30.1 mm to (106.3, 36.5)
- moved LED4 30.1 mm to (107.5, 36.5)
- moved R1 30.1 mm to (106.2, 33.9)
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Connections:
- net N$31 renamed NODE1_4_IMON
- net N$33 renamed RX5_N
- net N$34 renamed TX5_P
- net N$35 renamed RX6_N
- net N$36 renamed TX6_P
- net N$37 renamed RX7_N
- net N$38 renamed TX7_P
- net N$39 renamed RX8_N
- net N$40 renamed TX8_P
- net RXP5 renamed RX5_P
- net RXP6 renamed RX6_P
- net RXP7 renamed RX7_P
- net RXP8 renamed RX8_P
- net TXM5 renamed TX5_N
- net TXM6 renamed TX6_N
- net TXM7 renamed TX7_N
- net TXM8 renamed TX8_N
- removed net 3V3: R97.1, R98.1
- removed net 3V3@1: R78.2
- removed net ACDET: C108.1, R83.2, R84.1, U$12.6
- removed net ACDRV: R81.1, U$12.4
- removed net BAT: JP4.2
- removed net BAT@1: C105.1, C112.2, C115.1, C128.1, C129.2, JP3.2, R76.1, R90.1, R96.1, U$17.1, U$17.3
- removed net BATDRV: C129.1, R75.1, R96.2, U$17.4
- removed net CMSRC: R82.1, U$12.3
- removed net ILIM: C106.1, R77.2, R78.1, U$12.10
- removed net IOUT: C107.1, U$12.7
- removed net N$118: D4.3, R85.2
- removed net N$119: D4.1, JP4.1
- removed net N$120: C109.2, R86.2, R87.2
- removed net N$121: R75.2, U$12.11
- removed net N$122: C89.2, U$3.5, U$3.DAP, U$3.P$10, U$3.P$2, U$3.P$3, U$3.P$4, U$3.P$5, U$3.P$6, U$3.P$7, U$3.P$8, U$3.P$9
- removed net N$160: R76.2, U$12.12
- removed net N$161: R88.2, U$12.13
- removed net N$162: C111.1, C112.1, L2.2, R88.1, R90.2
- removed net N$163: R89.2, U$12.17
- removed net N$164: C114.1, D3.3, R89.1
- removed net N$165: C116.1, C117.1, C120.2, R92.2, U$12.2
- removed net N$166: C118.1, U$12.15, U$19.4
- removed net N$167: C119.1, U$12.18, U$18.4
- removed net N$168: C120.1, C121.1, R91.1, U$12.1
- removed net N$169: C125.1, R82.2, R93.2, R95.1, U$13.2, U$15.1, U$15.2, U$15.3, U$16.1, U$16.2, U$16.3
- removed net N$170: R94.1, R95.2, U$13.1
- removed net N$171: C110.2, C125.2, R81.2, R93.1, U$13.3, U$15.4, U$16.4
- removed net N$172: C114.2, C119.2, L2.1, U$12.19
- removed net N$30: U$26.P$13, U$26.P$2
- removed net REGN: C113.1, D3.1, R80.2, U$12.16
- removed net SYS: C122.1, C123.1, C124.1, C126.1, C127.1, JP3.3, R91.2, R92.1
- removed net VCC: R85.1
- removed net VCC@1: C130.1, U$12.20
- removed net VIN: C109.1, C110.1, D4.2, JP5.1, R84.2
- new net IMON_A0: U$26.P$12
- new net IMON_A1: U$26.P$10
- new net NODE1_IMON_IN: R49.2, U$26.P$1, U$3.13
- new net NODE2_IMON_IN: R52.2, U$26.P$9, U$4.13
- new net NODE3_IMON_IN: R54.2, U$26.P$3, U$5.13
- new net NODE4_IMON_IN: R58.2, U$26.P$7, U$6.13
- net +3V3: now also C10.1, U$26.P$4, U$26.P$6
- net ACOK: no longer R79.2, R80.1, U$12.5
- net GND: now also C10.2, C89.2, U$26.P$13, U$26.P$2, U$3.5, U$3.DAP, U$3.P$10, U$3.P$2, U$3.P$3, U$3.P$4, U$3.P$5, U$3.P$6, U$3.P$7, U$3.P$8, U$3.P$9; no longer C105.2, C106.2, C107.2, C108.2, C111.2, C113.2, C115.2, C116.2, C117.2, C118.2, C121.2, C122.2, C123.2, C124.2, C126.2, C127.2, C128.2, C130.2, JP1.1, JP3.1, JP5.2, R77.1, R79.1, R83.1, R86.1, R87.1, R94.2, U$12.14
- net NODE1_IMON: no longer R49.2, U$26.P$1, U$3.13
- net NODE2_IMON: no longer R52.2, U$26.P$9, U$4.13
- net NODE3_IMON: no longer R54.2, U$26.P$3, U$5.13
- net NODE4_IMON: no longer R58.2, U$26.P$7, U$6.13
- net SCL: no longer JP1.3, R97.2, U$12.9
- net SDA: no longer JP1.2, R98.2, U$12.8
Routing:
- net TX1_N: track 0.00 -> 56.3 mm
- net TX1_P: track 0.00 -> 56.2 mm
- net GND: track 14.4 -> 65.3 mm, vias 15 -> 26
- net RX8_N: track 0.00 -> 49.6 mm
- net RX8_P: track 0.00 -> 49.6 mm
- net TX8_N: track 0.00 -> 48.7 mm
- net TX8_P: track 0.00 -> 48.6 mm
- net NODE4_IMON: track 45.9 -> 0.00 mm, vias 2 -> 0
- net TX5_P: track 0.00 -> 40.8 mm, vias 0 -> 1
- net TX5_N: track 0.00 -> 40.2 mm, vias 0 -> 1
- net RX5_P: track 0.00 -> 37.9 mm
- net RX5_N: track 0.00 -> 37.4 mm
- net NODE4_RSV: track 9.76 -> 41.5 mm
- net RX7_N: track 0.00 -> 30.5 mm
- net RX7_P: track 0.00 -> 30.4 mm
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- added copper zone on layer 1, net +18V
- added copper zone on layer 1, net +3V3
- added copper zone on layer 16, net +3V3
- added copper zone on layer 1, net GND

Commit message: more routing and layout work
Parts:
- added C11: (no value), rcl:C0402K
- added R75, R76, R77, R78, R79, R80, R81, R82: (no value), rcl:R0402
- moved U$27 108.2 mm to (59.0, 15.4), flipped to the bottom, turned to 180 degrees
- moved R57 27.1 mm to (4.45, 13.5), turned to 90 degrees
- moved R56 26.7 mm to (6.45, 13.5), turned to 270 degrees
- moved R64 24.5 mm to (84.0, 4.40), turned to 90 degrees
- moved R65 23.9 mm to (82.7, 4.40), turned to 270 degrees
- moved R60 22.8 mm to (33.8, 3.75), turned to 90 degrees
- moved R61 22.7 mm to (32.0, 3.75)
- moved R63 22.2 mm to (57.4, 3.25)
- moved R62 22.0 mm to (58.9, 3.35)
- moved LED18 20.5 mm to (26.5, 25.7)
- moved LED19 20.5 mm to (29.0, 26.9)
- moved LED20 20.5 mm to (29.0, 25.8)
- moved R20 20.5 mm to (26.2, 26.9)
- moved R21 20.5 mm to (26.2, 25.7)
- moved R22 20.5 mm to (29.4, 27.0)
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Connections:
- removed net AUTOMDIX: U$1.37, U$14.87
- removed net CHASSIS: J1.CHASSIS@1, J1.CHASSIS@2, J2.CHASSIS@1, J2.CHASSIS@2, J3.CHASSIS@1, J3.CHASSIS@2, J4.CHASSIS@1, J4.CHASSIS@2, J5.CHASSIS@1, J5.CHASSIS@2, J6.CHASSIS@1, J6.CHASSIS@2, J7.CHASSIS@1, J7.CHASSIS@2, J8.CHASSIS@1, J8.CHASSIS@2
- removed net MODESEL0: U$1.91
- removed net MODESEL1: U$1.47, U$14.166
- removed net MODESEL2: U$1.53, U$14.165
- removed net MODESEL3: U$1.54, U$14.164, U$14.167
- removed net N$126: C91.2, U$7.5, U$7.DAP, U$7.P$10, U$7.P$2, U$7.P$3, U$7.P$4, U$7.P$5, U$7.P$6, U$7.P$7, U$7.P$8, U$7.P$9
- removed net N$127: C92.2, U$8.5, U$8.DAP, U$8.P$10, U$8.P$2, U$8.P$3, U$8.P$4, U$8.P$5, U$8.P$6, U$8.P$7, U$8.P$8, U$8.P$9
- removed net N$128: C93.2, U$9.5, U$9.DAP, U$9.P$10, U$9.P$2, U$9.P$3, U$9.P$4, U$9.P$5, U$9.P$6, U$9.P$7, U$9.P$8, U$9.P$9
- removed net N$129: C94.2, U$10.5, U$10.DAP, U$10.P$10, U$10.P$2, U$10.P$3, U$10.P$4, U$10.P$5, U$10.P$6, U$10.P$7, U$10.P$8, U$10.P$9
- removed net NODE1_IMON: U$1.25
- removed net NODE1_RXM: J1.USB_L@1
- removed net NODE1_RXP: J1.USB_H@1
- removed net NODE1_TXM: J1.CAN_L@1
- removed net NODE1_TXP: J1.CAN_H@1, J1.CAN_H@2
- removed net NODE2_IMON: U$1.29
- removed net NODE3_IMON: U$1.30
- removed net NODE4_IMON: U$1.31
- new net NODE1_TX_N: C31.2, J1.CAN_L@1, J1.CAN_L@2, R76.2, R80.1
- new net NODE5_8_IMON: U$1.16, U$27.P$8
- net +3V3: now also C11.1, R75.1, R76.1, R77.1, R78.1, U$27.P$4, U$27.P$6
- net GND: now also C11.2, C91.2, C92.2, C93.2, C94.2, J1.CHASSIS@1, J1.CHASSIS@2, J2.CHASSIS@1, J2.CHASSIS@2, J3.CHASSIS@1, J3.CHASSIS@2, J4.CHASSIS@1, J4.CHASSIS@2, J5.CHASSIS@1, J5.CHASSIS@2, J6.CHASSIS@1, J6.CHASSIS@2, J7.CHASSIS@1, J7.CHASSIS@2, J8.CHASSIS@1, J8.CHASSIS@2, R79.2, R80.2, R81.2, R82.2, U$10.5, U$10.DAP, U$10.P$10, U$10.P$2, U$10.P$3, U$10.P$4, U$10.P$5, U$10.P$6, U$10.P$7, U$10.P$8, U$10.P$9, U$27.P$13, U$27.P$2, U$7.5, U$7.DAP, U$7.P$10, U$7.P$2, U$7.P$3, U$7.P$4, U$7.P$5, U$7.P$6, U$7.P$7, U$7.P$8, U$7.P$9, U$8.5, U$8.DAP, U$8.P$10, U$8.P$2, U$8.P$3, U$8.P$4, U$8.P$5, U$8.P$6, U$8.P$7, U$8.P$8, U$8.P$9, U$9.5, U$9.DAP, U$9.P$10, U$9.P$2, U$9.P$3, U$9.P$4, U$9.P$5, U$9.P$6, U$9.P$7, U$9.P$8, U$9.P$9
- net IMON_A0: now also U$1.29, U$27.P$12
- net IMON_A1: now also U$1.30, U$27.P$10
- net MIIS0: no longer U$14.163
- net MIIS1: no longer U$14.162
- net MTXD0: no longer U$14.99
- net MTXD1: now also U$14.99; no longer U$14.98
- net MTXD2: now also U$14.98
- net NODE1_4_IMON: now also U$1.15
- net NODE1_RX_N: now also J1.USB_L@1, J1.USB_L@2, R78.2, R82.1
- net NODE1_RX_P: now also J1.USB_H@1, J1.USB_H@2, R77.2, R81.1
- net NODE1_TX_P: now also J1.CAN_H@1, J1.CAN_H@2, R75.2, R79.1; no longer C31.2
- net NODE5_IMON: now also U$27.P$1; no longer U$1.15
- net NODE6_IMON: now also U$27.P$9; no longer U$1.16
- net NODE7_IMON: now also U$27.P$3
- net NODE8_IMON: now also U$27.P$7
Routing:
- net IMON_A1: track 0.00 -> 100.5 mm, vias 0 -> 5
- net IMON_A0: track 0.00 -> 99.5 mm, vias 0 -> 5
- net NODE7_!EN: track 0.00 -> 66.4 mm, vias 0 -> 3
- net NODE7_!FLT: track 0.00 -> 64.9 mm, vias 0 -> 4
- net NODE5_8_IMON: track 0.00 -> 61.9 mm, vias 0 -> 3
- net MTXD2: track 0.00 -> 60.0 mm, vias 0 -> 4
- net MCOL: track 0.00 -> 52.7 mm, vias 0 -> 3
- net MTXC: track 0.00 -> 52.4 mm, vias 0 -> 3
- net MCRS: track 0.00 -> 50.7 mm, vias 0 -> 3
- net 25MHZ_REF_CLK: track 0.00 -> 50.6 mm, vias 0 -> 3
- net NODE7_!PG: track 0.00 -> 48.9 mm, vias 0 -> 3
- net NODE8_!EN: track 0.00 -> 47.2 mm, vias 0 -> 3
- net NODE8_IMON: track 0.00 -> 46.3 mm, vias 0 -> 4
- net NODE7_LTCH: track 0.00 -> 46.2 mm, vias 0 -> 3
- net MTXEN: track 0.00 -> 45.3 mm, vias 0 -> 3
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- added copper zone on layer 15, net +3V3
- added copper zone on layer 16, net NODE1_VOUT
- added copper zone on layer 16, net NODE5_VOUT
- added copper zone on layer 16, net NODE6_VOUT
- added copper zone on layer 16, net NODE7_VOUT
- added copper zone on layer 16, net NODE8_VOUT
- removed copper zone on layer 15, net TEMP
