File: av3/rocketnet-hub/eagle/batterycharger_page_isolated.sch (EAGLE design)
At the start: 61 parts

Commit message: updated schematic
Parts:
- removed C1, C10, C11, C12, C13, C14, C15, C16, C17, C18, C19, C2, C20, C21, C22, C23, C24, C25, C26, C3, C4, C5, C6, C7, C8, C9: (no value), rcl:C-EUC0402
- removed R14: 10, rcl_custom:R-US_0402-B
- removed R15, R16: 430k, rcl_custom:R-US_0402-B
- removed R19, R20: (no value), rcl_custom:R-US_0402-B
- added C101, C102, C103, C104, C105, C106, C107: (no value), rcl_custom:C-EU0603-B
- added C108, C109, C110, C111, C112, C113, C114, C115, C116, C117, C118, C119, C120, C121, C122, C123, C124, C125, C126: (no value), rcl_custom:C-EU0402-B
- added R101, R102: (no value), rcl_custom:R-US_0603-B
- added R106, R107: 430k, rcl_custom:R-US_0603-B
- added R116: 10, rcl_custom:R-US_0603-B
- R118, R119: value 10 -> 10k
- renumbered R1 to R103, R12 to R114, R13 to R115, R17 to R124, R18 to R105, R2 to R113, R21 to R110, R22 to R112, R24 to R111, R25 to RJP1, R3 to R104, R4 to R120, R5 to R122, R6 to R118, R7 to R119, R8 to R121, R9 to R117, U$2 to Q6, U$3 to Q1, U$4 to Q2, U$5 to Q3, U$6 to Q4, U$7 to Q5
Connections:
- net ACDET: now also C113.1; no longer C6.1
- net BAT: now also C106.1, C107.1, C112.2, C117.2, C119.1, R102.1; no longer C12.1, C25.1, C26.2, C3.1, C9.2, R19.1
- net BATDRV: now also C112.1; no longer C26.1
- net GND: now also C102.2, C103.2, C104.2, C105.2, C106.2, C107.2, C109.2, C110.2, C111.2, C113.2, C114.2, C116.2, C118.2, C119.2, C120.2, C122.2, C125.2, C126.2, R106.1, R107.1; no longer C1.2, C10.2, C12.2, C13.2, C14.2, C15.2, C18.2, C19.2, C2.2, C20.2, C21.2, C23.2, C24.2, C25.2, C3.2, C4.2, C5.2, C6.2, R15.1, R16.1
- net ILIM: now also C111.1; no longer C4.1
- net IOUT: now also C122.1; no longer C5.1
- net N$12: now also R116.2; no longer R14.2
- net N$17: now also C101.2, R106.2, R107.2; no longer C7.2, R15.2, R16.2
- net N$18: now also C117.1, C118.1, R102.2; no longer C2.1, C9.1, R19.2
- net N$22: now also C121.1; no longer C11.1
- net N$23: now also C115.1, C116.1; no longer C17.1, C18.1
- net N$26: now also C126.1; no longer C15.1
- net N$27: now also C114.1, C115.2, C125.1, R101.2; no longer C13.1, C14.1, C17.2, R20.2
- net N$29: now also C124.1; no longer C16.1
- net N$33: now also C108.1; no longer C22.1
- net N$34: now also C108.2, C123.2; no longer C22.2, C8.2
- net N$5: now also C121.2, C124.2; no longer C11.2, C16.2
- net REGN: now also C110.1; no longer C10.1
- net SHORE_POWER: now also C101.1, C123.1; no longer C7.1, C8.1
- net SYS: now also C102.1, C103.1, C104.1, C105.1, C109.1, R101.1; no longer C19.1, C20.1, C21.1, C23.1, C24.1, R20.1
- net VCC: now also C120.1, R116.1; no longer C1.1, R14.1

Commit message: updated battery charger isolated schematic with component size and names from eval board
Parts:
- removed C101, C102, C103, C104, C105, C106, C107: (no value), rcl_custom:C-EU0603-B
- removed C108, C109, C110, C111, C112, C113, C114, C115, C116, C117, C118, C119, C121, C122, C123, C124, C126: (no value), rcl_custom:C-EU0402-B
- removed R101, R102: (no value), rcl_custom:R-US_0603-B
- removed R103, R110, R111, R121: 12.1k, rcl_custom:R-US_0402-B
- removed R105, R112, R124: (no value), rcl_custom:R-US_0402-B
- removed R106, R107: 430k, rcl_custom:R-US_0603-B
- removed R114: 66.5k, rcl_custom:R-US_0402-B
- removed R115: 430k, rcl_custom:R-US_0402-B
- removed R116: 10, rcl_custom:R-US_0603-B
- removed R117, R118, R119: 10k, rcl_custom:R-US_0402-B
- removed R120: 100k, rcl_custom:R-US_0402-B
- removed R122: 316k, rcl_custom:R-US_0402-B
- added C1: (no value), rcl_custom:C-EUC1210
- added C10, C11, C12, C13, C14, C15, C16, C17, C18, C19, C21, C22, C23, C24, C26, C8, C9: (no value), rcl_custom:C-EUC0603
- added C2, C3, C4, C5, C6, C7: (no value), rcl_custom:C-EUC1206
- added R1, R2: (no value), rcl_custom:R-US_1206-B
- added R12, R24, R5: (no value), rcl_custom:R-US_0603-B
- added R14: 66.5k, rcl_custom:R-US_0603-B
- added R15: 430k, rcl_custom:R-US_0603-B
- added R16: 10, rcl_custom:R-US_1206-B
- added R17, R18, R19: 10k, rcl_custom:R-US_0603-B
- added R20: 100k, rcl_custom:R-US_0603-B
- added R21, R3: 12.1k, rcl_custom:R-US_0603-B
- added R22: 316k, rcl_custom:R-US_0603-B
- added R6, R7: 430k, rcl_custom:R-US_R1210
- added R8, R9: 4.02k, rcl_custom:R-US_0603-B
- R10, R11: value 4.02k -> 12.1k; device rcl_custom:R-US_0402-B -> rcl_custom:R-US_0603-B
- R23: device rcl_custom:R-US_0402-B -> rcl_custom:R-US_0603-B
- renumbered C120 to C20, C125 to C25, R104 to R4, R113 to R13
Connections:
- removed net SDA: R119.2, U$1.SDA
- new net R19: R19.2, U$1.SDA
- net +3V3: now also R18.1, R19.1, R22.2; no longer R118.1, R119.1, R122.2
- net ACDET: now also C13.1, R14.2, R15.1; no longer C113.1, R114.2, R115.1
- net ACDRV: now also R8.1; no longer R10.1
- net ACOK: now also R17.1, R21.2; no longer R117.1, R121.2
- net BAT: now also C12.2, C17.2, C19.1, C6.1, C7.1, R11.1, R2.1; no longer C106.1, C107.1, C112.2, C117.2, C119.1, R102.1, R111.1
- net BATDRV: now also C12.1, R11.2; no longer C112.1, R111.2
- net CMSRC: now also R9.1; no longer R11.1
- net GND: now also C10.2, C11.2, C13.2, C14.2, C16.2, C18.2, C19.2, C2.2, C22.2, C26.2, C3.2, C4.2, C5.2, C6.2, C7.2, C9.2, R12.2, R14.1, R20.1, R21.1, R6.1, R7.1; no longer C102.2, C103.2, C104.2, C105.2, C106.2, C107.2, C109.2, C110.2, C111.2, C113.2, C114.2, C116.2, C118.2, C119.2, C122.2, C126.2, R106.1, R107.1, R112.2, R114.1, R120.1, R121.1
- net ILIM: now also C11.1, R20.2, R22.1; no longer C111.1, R120.2, R122.1
- net IOUT: now also C22.1; no longer C122.1
- net N$12: now also R16.2; no longer R116.2
- net N$16: now also R24.2; no longer R124.2
- net N$17: now also C1.2, R6.2, R7.2; no longer C101.2, R106.2, R107.2
- net N$18: now also C17.1, C18.1, R2.2, R24.1; no longer C117.1, C118.1, R102.2, R124.1
- net N$21: now also R5.2; no longer R105.2
- net N$22: now also C21.1, R5.1; no longer C121.1, R105.1
- net N$23: now also C15.1, C16.1, R3.1; no longer C115.1, C116.1, R103.1
- net N$26: now also C26.1; no longer C126.1
- net N$27: now also C14.1, C15.2, R1.2; no longer C114.1, C115.2, R101.2
- net N$29: now also C24.1; no longer C124.1
- net N$32: now also R12.1; no longer R112.1
- net N$33: now also C8.1, R10.2, R9.2; no longer C108.1, R11.2, R110.2
- net N$34: now also C23.2, C8.2, R10.1, R8.2; no longer C108.2, C123.2, R10.2, R110.1
- net N$5: now also C21.2, C24.2; no longer C121.2, C124.2
- net REGN: now also C10.1, R17.2; no longer C110.1, R117.2
- net SCL: now also R18.2; no longer R118.2
- net SHORE_POWER: now also C1.1, C23.1, R15.2; no longer C101.1, C123.1, R115.2
- net SYS: now also C2.1, C3.1, C4.1, C5.1, C9.1, R1.1, R3.2; no longer C102.1, C103.1, C104.1, C105.1, C109.1, R101.1, R103.2
- net VCC: now also R16.1; no longer R116.1
Other:
- moved on the sheet: R10, R11

Commit message: swapped out battery charger schematic; modified symbols for BQ24725, BSS138W-7-F, FDS6680A, SiS412DN
Parts:
- removed C18, C19, C21, C22, C23, C24, C26: (no value), rcl_custom:C-EUC0603
- removed C20, C25: (no value), rcl_custom:C-EU0402-B
- removed Q1, Q2, Q3: FDS6680ASOIC-8, RNH_FDS6680A:FDS6680ASOIC-8
- removed Q4, Q5: SIS412DNSOP-8, RNH_SIS412DN:SIS412DNSOP-8
- removed Q6: BSS138W-7-F, RNH_BSS138W-7-F:BSS138W-7-F
- removed R19: 10k, rcl_custom:R-US_0603-B
- removed R20: 100k, rcl_custom:R-US_0603-B
- removed R21: 12.1k, rcl_custom:R-US_0603-B
- removed R22: 316k, rcl_custom:R-US_0603-B
- removed R23, R24: (no value), rcl_custom:R-US_0603-B
- removed RJP1: 0, rcl_custom:R-US_0402-B
- added U$2, U$3, U$5: FDS6680ASOIC-8, RNH_FDS6680A:FDS6680ASOIC-8
- added U$4: BSS138W-7-F, RNH_BSS138W-7-F:BSS138W-7-F
- added U$6, U$7: SIS412DNSOP-8, RNH_SIS412DN:SIS412DNSOP-8
- C1: value (none) -> 2.2uF
- C10, C12: value (none) -> 1uF; device rcl_custom:C-EUC0603 -> rcl_custom:C-EU0603-B
- C11: value (none) -> 0.01uF; device rcl_custom:C-EUC0603 -> rcl_custom:C-EU0603-B
- C13: value (none) -> 0.047uF; device rcl_custom:C-EUC0603 -> rcl_custom:C-EU0603-B
- C14, C15, C16, C17: value (none) -> 10uF; device rcl_custom:C-EUC0603 -> rcl_custom:C-EU1206-B
- C2, C4, C5, C6: value (none) -> 0.1uF; device rcl_custom:C-EUC1206 -> rcl_custom:C-EU0603-B
- C3: value (none) -> 2200pF; device rcl_custom:C-EUC1206 -> rcl_custom:C-EU0603-B
- C7: value (none) -> 100pF; device rcl_custom:C-EUC1206 -> rcl_custom:C-EUC0603
- C8, C9: value (none) -> 0.1uF; device rcl_custom:C-EUC0603 -> rcl_custom:C-EU0603-B
- D2: value BAT54C -> (none); device diode:BAT54C -> diode:ZENER-DIODEF126-12
- R1: value (none) -> 2
- R10, R11: value 12.1k -> 10k; device rcl_custom:R-US_0603-B -> rcl_custom:R-US_R0603
- R12: value (none) -> 10k; device rcl_custom:R-US_0603-B -> rcl_custom:R-US_R0603
- R13: value (none) -> 316k; device rcl_custom:R-US_0402-B -> rcl_custom:R-US_R0603
- R14: value 66.5k -> 7.5
- R15: value 430k -> 10
- R17: value 10k -> 4.02k
- R18: value 10k -> 10m; device rcl_custom:R-US_0603-B -> rcl_custom:R-US_1206-B
- R2: value (none) -> 1M; device rcl_custom:R-US_1206-B -> rcl_custom:R-US_0603-B
- R3: value 12.1k -> 3.01M
- R4: value (none) -> 10m; device rcl_custom:R-US_0402-B -> rcl_custom:R-US_1206-B
- R5: value (none) -> 4.02k
- R6: value 430k -> 4.02k; device rcl_custom:R-US_R1210 -> rcl_custom:R-US_0603-B
- R7: device rcl_custom:R-US_R1210 -> rcl_custom:R-US_0603-B
- R8: value 4.02k -> 66.5k; device rcl_custom:R-US_0603-B -> rcl_custom:R-US_1206-B
- R9: value 4.02k -> 100k; device rcl_custom:R-US_0603-B -> rcl_custom:R-US_R0603
Connections:
- removed net ACDET: C13.1, R14.2, R15.1, U$1.ACDET
- removed net ACDRV: R8.1, U$1.ACDRV
- removed net BATDRV: C12.1, Q3.G, R11.2, R13.1
- removed net CMSRC: R9.1, U$1.CMSRC
- removed net ILIM: C11.1, R20.2, R22.1, U$1.ILIM
- removed net N$23: C15.1, C16.1, R3.1, U$1.ACN
- removed net N$26: C26.1, Q5.G, U$1.LODRV
- removed net N$27: C14.1, C15.2, C25.1, Q2.D@5, R1.2, U$1.ACP
- removed net N$29: C24.1, Q4.G, U$1.HIDRV
- removed net N$32: Q6.G\, R12.1, R23.2
- removed net N$33: C8.1, Q1.S@1, Q1.S@2, Q1.S@3, Q2.S@1, Q2.S@2, Q2.S@3, Q6.S, R10.2, R23.1, R9.2
- removed net N$34: C23.2, C8.2, Q1.G, Q2.G, Q6.D, R10.1, R8.2
- removed net N$5: C21.2, C24.2, L1.1, Q4.S, Q5.D, U$1.PHASE
- removed net R19: R19.2, U$1.SDA
- removed net REGN: C10.1, D1.A, R17.2, U$1.REGN
- removed net SHORE_POWER: C1.1, C23.1, D2.A2, Q1.D@5, R15.2
- removed net SYS: C2.1, C3.1, C4.1, C5.1, C9.1, Q3.D@5, Q4.D, R1.1, R3.2
- removed net VCC: C20.1, R16.1, U$1.VCC
- new net N$10: R7.1, R8.2, U$1.ACDET
- new net N$11: R13.2, R9.2, U$1.ILIM
- new net N$15: C13.2, L1.1, U$1.PHASE, U$6.S, U$7.D
- new net N$19: C11.1, R17.2, U$5.G
- new net N$20: U$1.HIDRV, U$6.G
- new net N$25: U$1.LODRV, U$7.G
- new net N$3: C1.1, R1.1
- new net N$4: C2.1, R3.1, R5.2, U$2.S, U$3.D, U$4.S
- new net N$6: C5.1, C6.1, R4.1, U$1.ACP, U$3.S
- new net N$8: R5.1, U$1.CMSRC
- new net N$9: R6.1, U$1.ACDRV
- new net SDA: R11.1, U$1.SDA
- new net SYSTEM: C14.1, C15.1, C4.1, C6.2, R16.2, R4.2, U$1.ACN, U$5.D, U$6.D
- new net VIN: C3.1, D2.C, R1.2, R7.2, U$2.D
- net +3V3: now also R10.2, R11.2, R12.2, R13.1; no longer R18.1, R19.1, R22.2
- net ACOK: now also R12.1; no longer R17.1, R21.2
- net BAT: now also C11.2, C16.1, C17.1, C8.2, C9.1, R14.2, R18.2, U$5.S; no longer C12.2, C17.2, C19.1, C6.1, C7.1, Q3.S@1, Q3.S@2, Q3.S@3, R11.1, R2.1, R4.1, RJP1.1
- net GND: now also C1.2, C12.2, C15.2, C17.2, D2.A, R2.2, R8.1, R9.1, U$7.S; no longer C11.2, C13.2, C18.2, C19.2, C2.2, C20.2, C22.2, C25.2, C26.2, C3.2, C6.2, R12.2, R14.1, R20.1, R21.1, R6.1, R7.1
- net IOUT: now also C7.1; no longer C22.1
- net N$1: now also C2.2, C3.2, R6.2, U$2.G, U$3.G, U$4.D; no longer D2.A1, RJP1.2
- net N$12: now also R15.1, U$1.SRP; no longer D2.CC, R16.2
- net N$14: now also R14.1; no longer R4.2
- net N$16: now also C8.1, L1.2, R15.2, R18.1; no longer R24.2, U$1.SRP
- net N$17: now also C10.1, R16.1, U$1.VCC; no longer C1.2, R6.2, R7.2
- net N$18: now also R17.1, U$1.BATDRV; no longer C17.1, C18.1, L1.2, R2.2, R24.1
- net N$2: now also R2.1, R3.2, U$4.G\; no longer R13.2, U$1.BATDRV
- net N$21: now also C12.1, D1.A, U$1.REGN; no longer R5.2, U$1.BTST
- net N$22: now also C13.1, U$1.BTST; no longer C21.1, R5.1
- net SCL: now also R10.1; no longer R18.2
Other:
- moved on the sheet: C1, C10, C11, C12, C13, C14, C15, C16, C17, C2, C3, C4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

Commit message: added 4.7uH inductor library and SMAJ18CA TVS diode library; updated battery charger board with new parts
Parts:
- removed L1: (no value), rcl_custom:L-US0603-B
- added U$8: 4.7uH, RNH_IHLP-2525CZ-01:IHLP-2525CZ-01
- D2: value (none) -> SMAJ18CA; device diode:ZENER-DIODEF126-12 -> RNH_SMAJ18CA:SMAJ18CA
Connections:
- net N$15: now also U$8.P$2; no longer L1.1
- net N$16: now also U$8.P$1; no longer L1.2
Other:
- moved on the sheet: C1, C10, C11, C12, C13, C14, C15, C16, C17, C2, C3, C4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

Commit message: updated library names; fixed ERC; flipped S and D of Q3 transistor
Parts:
- removed U$2, U$3, U$5: FDS6680ASOIC-8, RNH_FDS6680A:FDS6680ASOIC-8
- removed U$4: BSS138W-7-F, RNH_BSS138W-7-F:BSS138W-7-F
- removed U$6, U$7: SIS412DNSOP-8, RNH_SIS412DN:SIS412DNSOP-8
- removed U$8: 4.7uH, RNH_IHLP-2525CZ-01:IHLP-2525CZ-01
- added Q1, Q6: SIS412DNSOP-8, RNH_SIS412DN:SIS412DNSOP-8
- added Q2, Q3, Q5: FDS6680ASOIC-8, RNH_FDS6680A:FDS6680ASOIC-8
- added Q4: BSS138W-7-F, RNH_BSS138W-7-F:BSS138W-7-F
- added U8: 4.7uH, RNH_IHLP-2525CZ-01:IHLP-2525CZ-01
- renumbered U$1 to U1
Connections:
- removed net N$4: C2.1, R3.1, R5.2, U$2.S, U$3.D, U$4.S
- new net N$5: C2.1, Q2.S, Q3.S, Q4.S, R3.1
- net BAT: now also Q5.S; no longer U$5.S
- net GND: now also Q1.S; no longer U$7.S
- net N$1: now also Q2.G, Q3.G, Q4.D, R5.2; no longer U$2.G, U$3.G, U$4.D
- net N$15: now also Q1.D, Q6.S, U8.P$2; no longer U$6.S, U$7.D, U$8.P$2
- net N$16: now also U8.P$1; no longer U$8.P$1
- net N$19: now also Q5.G; no longer U$5.G
- net N$2: now also Q4.G\; no longer U$4.G\
- net N$20: now also Q6.G; no longer U$6.G
- net N$25: now also Q1.G; no longer U$7.G
- net N$6: now also Q3.D; no longer U$3.S
- net SYSTEM: now also Q5.D, Q6.D; no longer U$5.D, U$6.D
- net VIN: now also Q2.D; no longer U$2.D
Other:
- moved on the sheet: C11

Commit message: battery charger current state
Parts:
- removed C13: 0.047uF, rcl_custom:C-EU0603-B
- removed R10, R11: 10k, rcl_custom:R-US_R0603
- removed R16: 10, rcl_custom:R-US_1206-B
- removed R17, R5, R6: 4.02k, rcl_custom:R-US_0603-B
- removed R3: 3.01M, rcl_custom:R-US_0603-B
- removed R7: 430k, rcl_custom:R-US_0603-B
- added C19: 0.1uF, rcl_custom:C-EU0402-B
- added C20, C25: 1uF, rcl_custom:C-EU0603-B
- added C22: 100pF, rcl_custom:C-EU0402-B
- added C23: 2200pF, rcl_custom:C-EU0402-B
- added C24: 0.047uF, rcl_custom:C-EU0402-B
- added R19, R21-17: 10k, rcl_custom:R-US_0402-B
- added R20: 100k, rcl_custom:R-US_0402-B
- added R22: 316k, rcl_custom:R-US_0402-B
- added R23: 3.01M, rcl_custom:R-US_0402-B
- added R24: 10, rcl_custom:R-US_0603-B
- added R67: 2, rcl_custom:R-US_1206-B
- C11: value 0.01uF -> 0.1uF; device rcl_custom:C-EU0603-B -> rcl_custom:C-EU0402-B
- C12: value 1uF -> 0.01uF; device rcl_custom:C-EU0603-B -> rcl_custom:C-EU0402-B
- C14, C15, C16, C17: value 10uF -> 0.1uF; device rcl_custom:C-EU1206-B -> rcl_custom:C-EU0402-B
- C2, C4, C5, C6: value 0.1uF -> 10uF; device rcl_custom:C-EU0603-B -> rcl_custom:C-EU1206-B
- C3: value 2200pF -> 10uF; device rcl_custom:C-EU0603-B -> rcl_custom:C-EU1206-B
- C7: value 100pF -> 10uF; device rcl_custom:C-EUC0603 -> rcl_custom:C-EU1206-B
- C8: device rcl_custom:C-EU0603-B -> rcl_custom:C-EU0402-B
- C9: value 0.1uF -> 1uF
- Q1: value SIS412DNSOP-8 -> FDS6680ASOIC-8; device RNH_SIS412DN:SIS412DNSOP-8 -> RNH_FDS6680A:FDS6680ASOIC-8
- Q4: value BSS138W-7-F -> SIS412DNSOP-8; device RNH_BSS138W-7-F:BSS138W-7-F -> RNH_SIS412DN:SIS412DNSOP-8
- Q5: value FDS6680ASOIC-8 -> SIS412DNSOP-8; device RNH_FDS6680A:FDS6680ASOIC-8 -> RNH_SIS412DN:SIS412DNSOP-8
- Q6: value SIS412DNSOP-8 -> BSS138W-7-F; device RNH_SIS412DN:SIS412DNSOP-8 -> RNH_BSS138W-7-F:BSS138W-7-F
- R1: value 2 -> 10m
- R12: value 10k -> 1M; device rcl_custom:R-US_R0603 -> rcl_custom:R-US_0402-B
- R13: value 316k -> 4.02k; device rcl_custom:R-US_R0603 -> rcl_custom:R-US_0402-B
- R14: value 7.5 -> 66.5k; device rcl_custom:R-US_0603-B -> rcl_custom:R-US_0402-B
- R15: value 10 -> 430k; device rcl_custom:R-US_0603-B -> rcl_custom:R-US_0402-B
- R18: value 10m -> 10k; device rcl_custom:R-US_1206-B -> rcl_custom:R-US_0402-B
- R2: value 1M -> 10m; device rcl_custom:R-US_0603-B -> rcl_custom:R-US_1206-B
- R4: value 10m -> 7.5; device rcl_custom:R-US_1206-B -> rcl_custom:R-US_0603-B
- R8: value 66.5k -> 4.02k; device rcl_custom:R-US_1206-B -> rcl_custom:R-US_0402-B
- R9: value 100k -> 4.02k; device rcl_custom:R-US_R0603 -> rcl_custom:R-US_0402-B
- renumbered U8 to L1
Connections:
- removed net N$17: C10.1, R16.1, U1.VCC
- net +3V3: now also R18.2, R19.2, R21-17.2, R22.1; no longer R10.2, R11.2, R12.2, R13.1
- net ACOK: now also R21-17.1; no longer R12.1
- net BAT: now also C12.2, C17.2, C19.1, C6.1, C7.1, Q3.S, R2.2, R4.2; no longer C11.2, C16.1, C17.1, C8.2, C9.1, Q5.S, R14.2, R18.2
- net GND: now also C11.2, C19.2, C2.2, C20.2, C22.2, C25.2, C3.2, C6.2, Q5.S, R12.2, R14.1, R20.1; no longer C12.2, C15.2, C17.2, Q1.S, R2.2, R8.1, R9.1
- net IOUT: now also C22.1; no longer C7.1
- net N$1: now also C23.2, C8.2, Q1.G, Q6.D, R8.2, R9.2; no longer C2.2, C3.2, Q3.G, Q4.D, R5.2, R6.2
- net N$10: now also R14.2, R15.1; no longer R7.1, R8.2
- net N$11: now also C11.1, R20.2, R22.2; no longer R13.2, R9.2
- net N$12: now also R24.1; no longer R15.1
- net N$14: now also R4.1; no longer R14.1
- net N$15: now also C24.2, Q4.S, Q5.D; no longer C13.2, Q1.D, Q6.S
- net N$16: now also C17.1, R2.1, R24.2; no longer C8.1, R15.2, R18.1
- net N$18: now also R13.1; no longer R17.1
- net N$19: now also C12.1, Q3.G, R13.2; no longer C11.1, Q5.G, R17.2
- net N$2: now also Q6.G\, R12.1, R23.2; no longer Q4.G\, R2.1, R3.2
- net N$20: now also Q4.G; no longer Q6.G
- net N$21: now also C10.1; no longer C12.1
- net N$22: now also C24.1; no longer C13.1
- net N$25: now also Q5.G; no longer Q1.G
- net N$3: now also R67.1; no longer R1.1
- net N$5: now also C8.1, Q1.S, Q6.S, R23.1; no longer C2.1, Q3.S, Q4.S, R3.1
- net N$6: now also C14.1, C15.1, C25.1, Q2.D, R1.1; no longer C5.1, C6.1, Q3.D, R4.1
- net N$8: now also R9.1; no longer R5.1
- net N$9: now also R8.1; no longer R6.1
- net SCL: now also R18.1; no longer R10.1
- net SDA: now also R19.1; no longer R11.1
- net SYSTEM: now also C15.2, C16.1, C2.1, C20.1, C3.1, C5.1, C9.1, Q3.D, Q4.D, R1.2, U1.VCC; no longer C14.1, C15.1, C6.2, Q5.D, Q6.D, R16.2, R4.2
- net VIN: now also C23.1, Q1.D, R15.2, R67.2; no longer C3.1, Q2.D, R1.2, R7.2
Other:
- moved on the sheet: C10, C11, C12, C14, C15, C16, C17, C2, C3, C4, C5, C6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

Commit message: removed optional components not installed
Parts:
- C11: value 0.1uF -> 0.01uF
- R1: value 10m -> 0.01
- renumbered C24 to C21
Changed lines of the file:
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@@
 <part name="C14" library="rcl_custom" deviceset="C-EU" device="0402-B" value="0.1uF"/>
 <part name="C15" library="rcl_custom" deviceset="C-EU" device="0402-B" value="0.1uF"/>
-<part name="R1" library="rcl_custom" deviceset="R-US_" device="1206-B" value="10m"/>
+<part name="R1" library="rcl_custom" deviceset="R-US_" device="1206-B" value="0.01"/>
 <part name="R9" library="rcl_custom" deviceset="R-US_" device="0402-B" value="4.02k"/>
 <part name="R8" library="rcl_custom" deviceset="R-US_" device="0402-B" value="4.02k"/>
@@
 <part name="GND9" library="supply1" deviceset="GND" device=""/>
 <part name="D1" library="diode" deviceset="BAT54" device=""/>
-<part name="C24" library="rcl_custom" deviceset="C-EU" device="0402-B" value="0.047uF"/>
+<part name="C21" library="rcl_custom" deviceset="C-EU" device="0402-B" value="0.047uF"/>
 <part name="Q4" library="RNH_SIS412DN" deviceset="SIS412DN" device="SOP-8"/>
 <part name="Q5" library="RNH_SIS412DN" deviceset="SIS412DN" device="SOP-8"/>
@@
 <part name="C25" library="rcl_custom" deviceset="C-EU" device="0603-B" value="1uF"/>
 <part name="GND17" library="supply1" deviceset="GND" device=""/>
-<part name="C11" library="rcl_custom" deviceset="C-EU" device="0402-B" value="0.1uF"/>
+<part name="C11" library="rcl_custom" deviceset="C-EU" device="0402-B" value="0.01uF"/>
 <part name="C2" library="rcl_custom" deviceset="C-EU" device="1206-B" value="10uF"/>
 <part name="C3" library="rcl_custom" deviceset="C-EU" device="1206-B" value="10uF"/>
@@
 <instance part="GND9" gate="1" x="35.56" y="17.78" rot="R90"/>
 <instance part="D1" gate="G$1" x="22.86" y="12.7" rot="R270"/>
-<instance part="C24" gate="CE" x="22.86" y="0"/>
+<instance part="C21" gate="CE" x="22.86" y="0"/>
 <instance part="Q4" gate="&gt;NAME" x="43.18" y="10.16"/>
 <instance part="Q5" gate="&gt;NAME" x="43.18" y="-10.16"/>
@@
 <wire x1="17.78" y1="7.62" x2="22.86" y2="7.62" width="0.1524" layer="91"/>
 <wire x1="22.86" y1="7.62" x2="22.86" y2="10.16" width="0.1524" layer="91"/>
-<pinref part="C24" gate="CE" pin="1"/>
+<pinref part="C21" gate="CE" pin="1"/>
 <wire x1="22.86" y1="7.62" x2="22.86" y2="2.54" width="0.1524" layer="91"/>
 <junction x="22.86" y="7.62"/>
@@
 <segment>
 <pinref part="U1" gate="G$1" pin="PHASE"/>
-<pinref part="C24" gate="CE" pin="2"/>
+<pinref part="C21" gate="CE" pin="2"/>
 <wire x1="17.78" y1="-5.08" x2="22.86" y2="-5.08" width="0.1524" layer="91"/>
 <pinref part="Q4" gate="&gt;NAME" pin="S"/>
