File: av3/rocketnet-hub/eagle/batterycharger_page_isolated.sch (EAGLE design)
At the start: 49 parts, among them Q1 FDS6680ASOIC-8, Q2 FDS6680ASOIC-8, Q3 FDS6680ASOIC-8, Q4 SIS412DNSOP-8, Q5 SIS412DNSOP-8, Q6 BSS138W-7-F, U1 BQ24725QFN-20

Commit message: seperated grounds, power and analog
Connections:
- net SYSTEM renamed +18V
