File: av3/rocketnet-hub/eagle/batterycharger_page_isolated.brd (EAGLE design)
At the start: 61 parts

Commit message: updated layout
Parts:
- removed C1, C10, C11, C12, C13, C14, C15, C16, C17, C18, C19, C2, C20, C21, C22, C23, C24, C25, C26, C3, C4, C5, C6, C7, C8, C9: (no value), rcl:C0402
- removed R1, R21, R8: 12.1k, rcl_custom:0402-B
- removed R12: 66.5k, rcl_custom:0402-B
- removed R13, R15, R16: 430k, rcl_custom:0402-B
- removed R14: 10, rcl_custom:0402-B
- removed R17, R18, R19, R2, R20, R22, R3: (no value), rcl_custom:0402-B
- removed R25: 0, rcl_custom:0402-B
- removed R4: 100k, rcl_custom:0402-B
- removed R5: 316k, rcl_custom:0402-B
- removed R9: 10k, rcl_custom:0402-B
- removed U$2: BSS138W-7-F, RNH_BSS138W-7-F:SOT323
- removed U$3, U$4, U$5: FDS6680ASOIC-8, RNH_FDS6680A:MS-012
- removed U$6, U$7: SIS412DNSOP-8, RNH_SIS412DN:1212-8
- added C101, C102, C103, C104, C105, C106, C107, R101, R102: (no value), rcl_custom:0603-B
- added C108, C109, C110, C111, C112, C113, C114, C115, C116, C117, C118, C119, C120, C121, C122, C123, C124, C125, C126, R104, R105, R112, R113, R124: (no value), rcl_custom:0402-B
- added Q1, Q2, Q3: FDS6680ASOIC-8, RNH_FDS6680A:MS-012
- added Q4, Q5: SIS412DNSOP-8, RNH_SIS412DN:1212-8
- added Q6: BSS138W-7-F, RNH_BSS138W-7-F:SOT323
- added R103, R110, R121: 12.1k, rcl_custom:0402-B
- added R106, R107: 430k, rcl_custom:0603-B
- added R114: 66.5k, rcl_custom:0402-B
- added R115: 430k, rcl_custom:0402-B
- added R116: 10, rcl_custom:0603-B
- added R117: 10k, rcl_custom:0402-B
- added R120: 100k, rcl_custom:0402-B
- added R122: 316k, rcl_custom:0402-B
- added RJP1: 0, rcl_custom:0402-B
- R118, R119: value 10 -> 10k
- moved R11 4.88 mm to (28.1, 41.6)
- moved R23 4.12 mm to (25.9, 46.1)
- moved R10 3.86 mm to (17.6, 41.8)
- moved L1 3.82 mm to (32.6, 22.5)
- moved U$1 3.71 mm to (23.3, 31.6)
- moved D1 1.69 mm to (24.2, 26.0), turned to 270 degrees
- moved D2 0.92 mm to (11.7, 31.1)
- renumbered R24 to R111, R6 to R118, R7 to R119
Connections:
- net +3V3: now also R122.2; no longer R5.2
- net ACDET: now also C113.1, R114.2, R115.1; no longer C6.1, R12.2, R13.1
- net ACOK: now also R117.1, R121.2; no longer R8.2, R9.1
- net BAT: now also C106.1, C107.1, C112.2, C117.2, C119.1, Q3.1, Q3.2, Q3.3, R102.1, R104.1, RJP1.1; no longer C12.1, C25.1, C26.2, C3.1, C9.2, R19.1, R25.1, R3.1, U$5.1, U$5.2, U$5.3
- net BATDRV: now also C112.1, Q3.4, R113.1; no longer C26.1, R2.1, U$5.4
- net GND: now also C102.2, C103.2, C104.2, C105.2, C106.2, C107.2, C109.2, C110.2, C111.2, C113.2, C114.2, C116.2, C118.2, C119.2, C120.2, C122.2, C125.2, C126.2, R106.1, R107.1, R112.2, R114.1, R120.1, R121.1; no longer C1.2, C10.2, C12.2, C13.2, C14.2, C15.2, C18.2, C19.2, C2.2, C20.2, C21.2, C23.2, C24.2, C25.2, C3.2, C4.2, C5.2, C6.2, R12.1, R15.1, R16.1, R22.2, R4.1, R8.1
- net ILIM: now also C111.1, R120.2, R122.1; no longer C4.1, R4.2, R5.1
- net IOUT: now also C122.1; no longer C5.1
- net N$1: now also RJP1.2; no longer R25.2
- net N$12: now also R116.2; no longer R14.2
- net N$14: now also R104.2; no longer R3.2
- net N$16: now also R124.2; no longer R17.2
- net N$17: now also C101.2, R106.2, R107.2; no longer C7.2, R15.2, R16.2
- net N$18: now also C117.1, C118.1, R102.2, R124.1; no longer C2.1, C9.1, R17.1, R19.2
- net N$2: now also R113.2; no longer R2.2
- net N$21: now also R105.2; no longer R18.2
- net N$22: now also C121.1, R105.1; no longer C11.1, R18.1
- net N$23: now also C115.1, C116.1, R103.1; no longer C17.1, C18.1, R1.1
- net N$26: now also C126.1, Q5.4; no longer C15.1, U$7.4
- net N$27: now also C114.1, C115.2, C125.1, Q2.5, Q2.6, Q2.7, Q2.8, R101.2; no longer C13.1, C14.1, C17.2, R20.2, U$4.5, U$4.6, U$4.7, U$4.8
- net N$29: now also C124.1, Q4.4; no longer C16.1, U$6.4
- net N$32: now also Q6.2, R112.1; no longer R22.1, U$2.2
- net N$33: now also C108.1, Q1.1, Q1.2, Q1.3, Q2.1, Q2.2, Q2.3, Q6.3, R110.2; no longer C22.1, R21.2, U$2.3, U$3.1, U$3.2, U$3.3, U$4.1, U$4.2, U$4.3
- net N$34: now also C108.2, C123.2, Q1.4, Q2.4, Q6.1, R110.1; no longer C22.2, C8.2, R21.1, U$2.1, U$3.4, U$4.4
- net N$5: now also C121.2, C124.2, Q4.1, Q4.2, Q4.3, Q5.5, Q5.6, Q5.7, Q5.8, Q5.9; no longer C11.2, C16.2, U$6.1, U$6.2, U$6.3, U$7.5, U$7.6, U$7.7, U$7.8, U$7.9
- net REGN: now also C110.1, R117.2; no longer C10.1, R9.2
- net SHORE_POWER: now also C101.1, C123.1, Q1.5, Q1.6, Q1.7, Q1.8, R115.2; no longer C7.1, C8.1, R13.2, U$3.5, U$3.6, U$3.7, U$3.8
- net SYS: now also C102.1, C103.1, C104.1, C105.1, C109.1, Q3.5, Q3.6, Q3.7, Q3.8, Q4.5, Q4.6, Q4.7, Q4.8, Q4.9, R101.1, R103.2; no longer C19.1, C20.1, C21.1, C23.1, C24.1, R1.2, R20.1, U$5.5, U$5.6, U$5.7, U$5.8, U$6.5, U$6.6, U$6.7, U$6.8, U$6.9
- net VCC: now also C120.1, R116.1; no longer C1.1, R14.1
Routing:
- net +3V3: track 18.0 -> 0.00 mm
- net SYS: track 16.5 -> 0.00 mm
- net SHORE_POWER: track 15.0 -> 0.00 mm
- net BAT: track 14.8 -> 0.00 mm, vias 1 -> 0
- net N$34: track 12.2 -> 0.00 mm, vias 1 -> 0
- net N$33: track 10.9 -> 0.00 mm, vias 1 -> 0
- net N$5: track 7.88 -> 0.00 mm
- net N$18: track 6.75 -> 0.00 mm
- net N$27: track 6.27 -> 0.00 mm
- net N$14: track 6.14 -> 0.00 mm
- net N$16: track 6.09 -> 0.00 mm
- net N$17: track 5.22 -> 0.00 mm
- net GND: track 4.75 -> 0.00 mm
- net N$12: track 3.61 -> 0.00 mm
- net N$29: track 3.28 -> 0.00 mm
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- removed copper zone on layer 1, net N$5
- removed copper zone on layer 1, net SYS

Commit message: updated board
Parts:
- moved C109 0.18 mm to (30.8, 37.2)
Routing:
- added copper zone on layer 1, net SYS

Commit message: battery charger current state
Parts:
- removed C101, C102, C103, C104, C105, C106, C107, R101, R102: (no value), rcl_custom:0603-B
- removed C108, C109, C110, C111, C112, C113, C114, C115, C116, C117, C118, C119, C120, C121, C122, C123, C124, C125, C126, R104, R105, R112, R113, R124: (no value), rcl_custom:0402-B
- removed R10, R11: 4.02k, rcl_custom:0402-B
- removed R103, R110, R111, R121: 12.1k, rcl_custom:0402-B
- removed R106, R107: 430k, rcl_custom:0603-B
- removed R114: 66.5k, rcl_custom:0402-B
- removed R115: 430k, rcl_custom:0402-B
- removed R116: 10, rcl_custom:0603-B
- removed R117, R118, R119: 10k, rcl_custom:0402-B
- removed R120: 100k, rcl_custom:0402-B
- removed R122: 316k, rcl_custom:0402-B
- removed RJP1: 0, rcl_custom:0402-B
- removed U$1: BQ24725QFN-20, RNH_BQ24725:S-PVQFN-N20
- added C1: 2.2uF, rcl_custom:C1210
- added C10, C20, C25, C9: 1uF, rcl_custom:0603-B
- added C11, C14, C15, C16, C17, C19, C8: 0.1uF, rcl_custom:0402-B
- added C12: 0.01uF, rcl_custom:0402-B
- added C2, C3, C4, C5, C6, C7: 10uF, rcl_custom:1206-B
- added C22: 100pF, rcl_custom:0402-B
- added C23: 2200pF, rcl_custom:0402-B
- added C24: 0.047uF, rcl_custom:0402-B
- added R1, R2: 10m, rcl_custom:1206-B
- added R12: 1M, rcl_custom:0402-B
- added R13, R8, R9: 4.02k, rcl_custom:0402-B
- added R14: 66.5k, rcl_custom:0402-B
- added R15: 430k, rcl_custom:0402-B
- added R18, R19, R21-17: 10k, rcl_custom:0402-B
- added R20: 100k, rcl_custom:0402-B
- added R22: 316k, rcl_custom:0402-B
- added R24: 10, rcl_custom:0603-B
- added R4: 7.5, rcl_custom:0603-B
- added R67: 2, rcl_custom:1206-B
- added U1: BQ24725QFN-20, RNH_BQ24725:S-PVQFN-N20
- D2: value BAT54C -> SMAJ18CA; device diode:SOT23 -> RNH_SMAJ18CA:D0-214AC
- L1: value (none) -> 4.7uH; device rcl_custom:0603-B -> RNH_IHLP-2525CZ-01:2525
- R23: value (none) -> 3.01M
- moved D1 75.0 mm to (-50.8, 25.4), flipped to the top, turned to 0 degrees
- moved R23 56.4 mm to (-30.5, 45.7), flipped to the top, turned to 0 degrees
- moved Q6 49.0 mm to (-24.1, 55.9), flipped to the top, turned to 0 degrees
- moved D2 47.2 mm to (-29.2, 54.6), flipped to the top, turned to 0 degrees
- moved L1 14.1 mm to (34.4, 36.4)
- moved Q3 13.6 mm to (22.9, 26.7)
- moved Q1 11.9 mm to (25.4, 55.9)
- moved Q2 11.6 mm to (32.3, 54.7)
- moved Q4 11.4 mm to (37.5, 43.6)
- moved Q5 11.3 mm to (32.6, 43.6)
Connections:
- removed net ACDET: C113.1, R114.2, R115.1, U$1.6
- removed net ACDRV: R10.1, U$1.4
- removed net BATDRV: C112.1, Q3.4, R111.2, R113.1
- removed net CMSRC: R11.1, U$1.3
- removed net ILIM: C111.1, R120.2, R122.1, U$1.10
- removed net N$17: C101.2, R106.2, R107.2
- removed net N$23: C115.1, C116.1, R103.1, U$1.1
- removed net N$26: C126.1, Q5.4, U$1.15
- removed net N$27: C114.1, C115.2, C125.1, Q2.5, Q2.6, Q2.7, Q2.8, R101.2, U$1.2
- removed net N$29: C124.1, Q4.4, U$1.18
- removed net N$32: Q6.2, R112.1, R23.2
- removed net N$33: C108.1, Q1.1, Q1.2, Q1.3, Q2.1, Q2.2, Q2.3, Q6.3, R11.2, R110.2, R23.1
- removed net N$34: C108.2, C123.2, Q1.4, Q2.4, Q6.1, R10.2, R110.1
- removed net REGN: C110.1, D1.1, R117.2, U$1.16
- removed net SHORE_POWER: C101.1, C123.1, D2.2, Q1.5, Q1.6, Q1.7, Q1.8, R115.2
- removed net SYS: C102.1, C103.1, C104.1, C105.1, C109.1, Q3.5, Q3.6, Q3.7, Q3.8, Q4.5, Q4.6, Q4.7, Q4.8, Q4.9, R101.1, R103.2
- removed net VCC: C120.1, R116.1, U$1.20
- new net N$10: R14.2, R15.1, U1.6
- new net N$11: C11.1, R20.2, R22.2, U1.10
- new net N$15: C24.2, L1.P$2, Q4.1, Q4.2, Q4.3, Q5.5, Q5.6, Q5.7, Q5.8, Q5.9, U1.19
- new net N$19: C12.1, Q3.4, R13.2
- new net N$20: Q4.4, U1.18
- new net N$25: Q5.4, U1.15
- new net N$3: C1.1, R67.1
- new net N$6: C14.1, C15.1, C25.1, Q2.5, Q2.6, Q2.7, Q2.8, R1.1, U1.2
- new net N$8: R9.1, U1.3
- new net N$9: R8.1, U1.4
- new net SYSTEM: C15.2, C16.1, C2.1, C20.1, C3.1, C4.1, C5.1, C9.1, Q3.5, Q3.6, Q3.7, Q3.8, Q4.5, Q4.6, Q4.7, Q4.8, Q4.9, R1.2, U1.1, U1.20
- new net VIN: C23.1, D2.P$2, Q1.5, Q1.6, Q1.7, Q1.8, R15.2, R67.2
- net +3V3: now also R18.2, R19.2, R21-17.2, R22.1; no longer R118.1, R119.1, R122.2
- net ACOK: now also R21-17.1, U1.5; no longer R117.1, R121.2, U$1.5
- net BAT: now also C12.2, C17.2, C19.1, C6.1, C7.1, R2.2, R4.2; no longer C106.1, C107.1, C112.2, C117.2, C119.1, R102.1, R104.1, R111.1, RJP1.1
- net GND: now also C1.2, C10.2, C11.2, C14.2, C16.2, C19.2, C2.2, C20.2, C22.2, C25.2, C3.2, C4.2, C5.2, C6.2, C7.2, C9.2, D2.P$1, Q5.1, Q5.2, Q5.3, R12.2, R14.1, R20.1, U1.14, U1.POWERPAD; no longer C102.2, C103.2, C104.2, C105.2, C106.2, C107.2, C109.2, C110.2, C111.2, C113.2, C114.2, C116.2, C118.2, C119.2, C120.2, C122.2, C125.2, C126.2, R106.1, R107.1, R112.2, R114.1, R120.1, R121.1, U$1.14, U$1.POWERPAD
- net IOUT: now also C22.1, U1.7; no longer C122.1, U$1.7
- net N$1: now also C23.2, C8.2, Q1.4, Q2.4, Q6.1, R8.2, R9.2; no longer D2.1, RJP1.2
- net N$12: now also R24.1, U1.13; no longer D2.3, R116.2
- net N$14: now also R4.1, U1.12; no longer R104.2, U$1.12
- net N$16: now also C17.1, L1.P$1, R2.1, R24.2; no longer R124.2, U$1.13
- net N$18: now also R13.1, U1.11; no longer C117.1, C118.1, L1.2, R102.2, R124.1
- net N$2: now also Q6.2, R12.1, R23.2; no longer R113.2, U$1.11
- net N$21: now also C10.1, D1.1, U1.16; no longer R105.2, U$1.17
- net N$22: now also C24.1, U1.17; no longer C121.1, R105.1
- net N$5: now also C8.1, Q1.1, Q1.2, Q1.3, Q2.1, Q2.2, Q2.3, Q6.3, R23.1; no longer C121.2, C124.2, L1.1, Q4.1, Q4.2, Q4.3, Q5.5, Q5.6, Q5.7, Q5.8, Q5.9, U$1.19
- net SCL: now also R18.1, U1.9; no longer R118.2, U$1.9
- net SDA: now also R19.1, U1.8; no longer R119.2, U$1.8
Routing:
- removed copper zone on layer 1, net SYS
Other:
- board outline added: 160 x 100 mm

Commit message: placement mostly complete
Parts:
- removed C24: 0.047uF, rcl_custom:0402-B
- added C21: 0.047uF, rcl_custom:0402-B
- C11: value 0.1uF -> 0.01uF
- R1: value 10m -> 0.01
- moved R12 146.2 mm to (88.6, 29.0)
- moved D1 138.3 mm to (85.1, 51.3)
- moved C22 127.4 mm to (76.5, 46.4)
- moved C20 125.7 mm to (84.8, 43.3)
- moved C8 123.3 mm to (87.1, 33.5), turned to 270 degrees
- moved R23 117.8 mm to (86.4, 31.0)
- moved Q6 112.8 mm to (85.3, 28.8), turned to 90 degrees
- moved R9 112.2 mm to (89.8, 37.6), turned to 270 degrees
- moved R21-17 110.1 mm to (76.7, 42.0)
- moved R22 104.6 mm to (80.3, 50.7)
- moved R8 104.4 mm to (76.8, 36.8), turned to 270 degrees
- moved C12 101.1 mm to (76.1, 59.4)
- moved C23 100.5 mm to (81.5, 30.4)
- moved D2 99.8 mm to (70.2, 46.5)
- moved R19 98.8 mm to (59.7, 47.1)
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Connections:
- net N$15: now also C21.2; no longer C24.2
- net N$22: now also C21.1; no longer C24.1

Commit message: placement mostly complete
Parts:
- moved R19 1.98 mm to (61.2, 48.4)
- moved R18 1.98 mm to (61.3, 52.7)
- moved D2 1.02 mm to (71.2, 46.4)
- moved C2 0.65 mm to (32.6, 50.9)
- moved C3 0.28 mm to (32.6, 48.3)
- moved C9 0.18 mm to (32.5, 46.2)

Commit message: most components on bottom of board
Parts:
- moved R12 76.6 mm to (12.3, 35.3), turned to 270 degrees
- moved Q6 73.8 mm to (12.2, 38.6), turned to 0 degrees
- moved R23 72.3 mm to (14.4, 37.6), turned to 270 degrees
- moved C8 70.3 mm to (16.9, 36.8), turned to 180 degrees
- moved R9 68.9 mm to (21.0, 34.2), turned to 180 degrees
- moved C23 68.9 mm to (13.7, 42.4), turned to 270 degrees
- moved C20 58.3 mm to (26.7, 39.1), turned to 270 degrees
- moved R8 57.6 mm to (20.2, 47.1), turned to 180 degrees
- moved C21 54.3 mm to (30.6, 39.6), turned to 90 degrees
- moved D1 51.9 mm to (34.7, 38.9), turned to 270 degrees
- moved R21-17 51.6 mm to (25.4, 47.2), turned to 270 degrees
- moved R22 46.8 mm to (34.0, 43.7), turned to 270 degrees
- moved C22 46.7 mm to (29.7, 47.5), turned to 270 degrees
- moved R20 45.3 mm to (35.8, 43.7), turned to 270 degrees
- moved C7 42.9 mm to (42.7, 58.4), flipped to the bottom, turned to 90 degrees
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Connections:
- net SYSTEM renamed +18V
