File: av3/rocketnet-hub/eagle/mcu_page_combined.brd (EAGLE design)
At the start: 112.7 x 76.3 mm, 393 parts, among them J1 ROCKETNET-CONNECTOR-16M, J10 ROCKETNET-UMBILICAL-12, J11 1.27MM_HDR_2X5, J12 1.27MM_HDR_2X12X1, J2 ROCKETNET-CONNECTOR-16M, J3 ROCKETNET-CONNECTOR-16M, J4 ROCKETNET-CONNECTOR-16M, J5 1.27MM_HDR_2X12X1, J6 ROCKETNET-CONNECTOR-16M, J7 ROCKETNET-CONNECTOR-16M, J8 ROCKETNET-CONNECTOR-16M, J9 ROCKETNET-BATTERY-14, Q1 25MHz, Q2 FDS6680ASOIC-8, Q3 FDS6680ASOIC-8, Q4 FDS6680ASOIC-8, Q5 SIS412DNSOP-8, Q6 BSS138W-7-F, Q7 SIS412DNSOP-8, U1 STM32F407V100-PIN_QFP, U2 BQ24725QFN-20

Commit message: compressed battery charger and placed some polys
Parts:
- moved R135 6.81 mm to (14.9, 37.0)
- moved C114 6.78 mm to (34.2, 23.8)
- moved C102 5.89 mm to (7.62, 29.6)
- moved C110 5.89 mm to (23.6, 24.5)
- moved C113 5.89 mm to (20.6, 32.9)
- moved C94 5.89 mm to (10.8, 35.2)
- moved D5 5.89 mm to (23.6, 19.3)
- moved Q6 5.89 mm to (6.10, 33.4)
- moved R132 5.89 mm to (6.22, 36.7)
- moved R133 5.89 mm to (8.26, 34.4)
- moved R136 5.89 mm to (14.1, 24.9)
- moved R139 5.89 mm to (29.7, 28.3)
- moved R142 5.89 mm to (27.9, 28.3)
- moved R21-17 5.89 mm to (19.3, 24.8)
- moved C116 5.89 mm to (24.5, 32.4)
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Routing:
- net N$169: track 0.00 -> 10.5 mm
- net GND: vias 22 -> 21
- added copper zone on layer 1, net N$165

Commit message: battery charger analog grounds properly named + more routing
Parts:
- moved C112 0.92 mm to (26.4, 23.3)
- moved C111 0.82 mm to (26.4, 25.3)
Connections:
- new net GNDA: C115.2, C117.2, C118.2, C119.2, C120.2, C123.2, C124.2, C125.2, C60.2
- net GND: no longer C115.2, C117.2, C118.2, C119.2, C120.2, C123.2, C124.2, C125.2, C60.2
Routing:
- net N$166: track 0.00 -> 11.0 mm
- net N$169: track 10.5 -> 0.00 mm
- added copper zone on layer 1, net BAT
- added copper zone on layer 1, net N$166
- added copper zone on layer 1, net N$167

Commit message: Renamed +18Vx fills to +18V for current switch
Routing:
- removed copper zone on layer 16, net +18V4
- removed copper zone on layer 16, net +18V6
- removed copper zone on layer 16, net +18V8

Commit message: Fixed some ERC issues; check Approved ERC for list of pending fixes
Connections:
- net BOOT1: now also R150.1
- net JTAG_TRST: now also R147.2
Changed lines of the file:
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@@
 <signal name="JTAG_TRST">
 <contactref element="U1" pad="90"/>
+<contactref element="R147" pad="2"/>
+<wire x1="2.15" y1="-28.4" x2="46.081828125" y2="42.85175625" width="0" layer="19" extent="1-1"/>
 </signal>
 <signal name="SCL">
@@
 <wire x1="31.703" y1="54.4426" x2="103.413" y2="53.4" width="0" layer="19" extent="1-1"/>
 </signal>
-<signal name="VDD">
+<signal name="VDD" class="1">
 <contactref element="U$2" pad="3"/>
 <contactref element="C84" pad="1"/>
@@
 </polygon>
 </signal>
-<signal name="VDDIO_IN">
+<signal name="VDDIO_IN" class="1">
 <contactref element="U$14" pad="148"/>
 <contactref element="C13" pad="2"/>
@@
 <wire x1="88.09" y1="8.77" x2="83.29" y2="22.7596" width="0" layer="19" extent="1-16"/>
 </signal>
-<signal name="NODE1_VOUT">
+<signal name="NODE1_VOUT" class="1">
 <contactref element="U$3" pad="12"/>
 <contactref element="U$3" pad="11"/>
@@
 <wire x1="88.095" y1="72.395" x2="88.095" y2="75.08" width="0" layer="19" extent="1-1"/>
 </signal>
-<signal name="NODE2_VOUT">
+<signal name="NODE2_VOUT" class="1">
 <contactref element="U$4" pad="12"/>
 <contactref element="U$4" pad="11"/>
@@
 <wire x1="65.095" y1="72.395" x2="65.095" y2="75.08" width="0" layer="19" extent="1-1"/>
 </signal>
-<signal name="NODE3_VOUT">
+<signal name="NODE3_VOUT" class="1">
 <contactref element="U$5" pad="12"/>
 <contactref element="U$5" pad="11"/>
@@
 <wire x1="91.905" y1="1" x2="91.905" y2="3.685" width="0" layer="19" extent="1-1"/>
 </signal>
-<signal name="NODE6_VOUT">
+<signal name="NODE6_VOUT" class="1">
 <contactref element="U$8" pad="12"/>
 <contactref element="U$8" pad="11"/>
@@
 <wire x1="45.905" y1="1" x2="45.905" y2="3.685" width="0" layer="19" extent="1-1"/>
 </signal>
-<signal name="NODE7_VOUT">
+<signal name="NODE7_VOUT" class="1">
 <contactref element="U$9" pad="12"/>
 <contactref element="U$9" pad="11"/>
@@
 <wire x1="68.905" y1="1" x2="68.905" y2="3.685" width="0" layer="19" extent="1-1"/>
 </signal>
-<signal name="NODE8_VOUT">
+<signal name="NODE8_VOUT" class="1">
 <polygon width="0.127" layer="16" thermals="no">
 <vertex x="83.6104" y="2.6742"/>
@@
 <contactref element="J10" pad="A1"/>
 <contactref element="J10" pad="A2"/>
+<contactref element="R148" pad="2"/>
+<contactref element="R147" pad="1"/>
 <contactref element="J11" pad="P$10"/>
 <contactref element="R148" pad="1"/>
-<contactref element="R148" pad="2"/>
-<contactref element="R147" pad="1"/>
 <wire x1="47.1424875" y1="32.28758125" x2="103.3148" y2="14.7464" width="0" layer="19" extent="1-16"/>
 <wire x1="46.2876" y1="31.4218" x2="47.1424875" y2="32.28758125" width="0" layer="19" extent="1-1"/>
@@
 <wire x1="23.3046" y1="25.3492" x2="21.41" y2="27.1352" width="0" layer="19" extent="1-1"/>
 </signal>
-<signal name="BAT">
+<signal name="BAT" class="1">
 <contactref element="R143" pad="2"/>
 <contactref element="C111" pad="2"/>
@@
 <contactref element="J12" pad="P$1"/>
 <contactref element="U1" pad="37"/>
+<contactref element="R150" pad="1"/>
 <wire x1="2.1" y1="-32.465" x2="57.353109375" y2="32.28758125" width="0" layer="19" extent="1-1"/>
+<wire x1="0.85" y1="-42.8" x2="2.1" y2="-32.465" width="0" layer="19" extent="1-1"/>
 </signal>
 <signal name="GNDA" class="1">

Commit message: Positioned TX/RX LEDs
Parts:
- moved R38 73.3 mm to (104.0, 60.0)
- moved LED33 73.3 mm to (104.0, 60.0)
- moved J9 61.3 mm to (7.50, 52.0), turned to 90 degrees
- moved R150 60.0 mm to (7.60, 16.9), flipped to the bottom, turned to 180 degrees
- moved J12 48.3 mm to (7.10, 14.9)
- moved R147 45.7 mm to (10.5, 16.4), flipped to the bottom, turned to 180 degrees
- moved R148 39.2 mm to (10.5, 14.6), flipped to the bottom, turned to 180 degrees
- moved R11 38.1 mm to (34.3, 43.6), turned to 180 degrees
- moved C60 34.4 mm to (35.5, 39.1), turned to 270 degrees
- moved R132 32.5 mm to (35.8, 23.3), turned to 270 degrees
- moved Q6 30.6 mm to (35.9, 26.6), turned to 0 degrees
- moved C120 30.4 mm to (8.35, 38.4), turned to 90 degrees
- moved C118 30.1 mm to (6.49, 26.1), turned to 270 degrees
- moved C114 29.1 mm to (7.81, 36.2), turned to 270 degrees
- moved R64 28.6 mm to (7.60, 21.5), turned to 180 degrees
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Routing:
- net N$27: track 6.60 -> 7.47 mm

Commit message: Fixed DRC clearance issues
Parts:
- moved TP40 13.2 mm to (30.6, 50.5)
- moved R43 5.41 mm to (102.5, 20.0)
- moved R148 4.00 mm to (10.7, 18.6)
- moved R147 3.61 mm to (10.7, 20.0)
- moved T1 2.24 mm to (105.0, 22.0)
- moved C75 1.89 mm to (104.5, 26.4)
- moved R117 1.60 mm to (104.5, 27.5)
- moved R14 1.50 mm to (95.0, 10.5)
- moved R13 1.35 mm to (71.5, 38.2)
- moved R89 1.27 mm to (71.5, 40.8)
- moved R90 1.25 mm to (71.5, 39.5)
- moved R42 1.12 mm to (107.5, 20.0)
- moved T2 1.12 mm to (105.0, 18.5)
- moved C78 1.10 mm to (79.0, 33.3)
- moved C12 1.02 mm to (105.0, 16.2)
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Routing:
- net GND: track 79.6 -> 78.3 mm
- net NODE7_!EN: track 3.46 -> 2.90 mm
- added copper zone on layer 16, net N$169
- added copper zone on layer 16, net N$170

Commit message: Replaced pull up resistors for ethernet switch
Parts:
- moved C74 24.1 mm to (79.0, 38.7), turned to 0 degrees
- moved C73 24.0 mm to (79.0, 40.9), turned to 0 degrees
- moved C82 12.6 mm to (90.4, 49.5), turned to 90 degrees
- moved R83 3.73 mm to (71.8, 49.2)
- moved R84 3.71 mm to (71.8, 48.1)
- moved R13 1.02 mm to (72.5, 38.4), flipped to the top, turned to 180 degrees
- moved R80 1.00 mm to (80.0, 58.0)
- moved R115 0.40 mm to (71.8, 35.6)
- moved R77 0.40 mm to (83.6, 54.0)
- moved R79 0.40 mm to (81.4, 58.0)
- moved R102 0.38 mm to (71.8, 36.7)
- moved R96 0.36 mm to (81.2, 18.5)
- moved R95 0.35 mm to (80.0, 18.5)
- moved R90 0.34 mm to (71.8, 39.7)
- moved TP28 0.34 mm to (94.5, 32.6)
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Routing:
- removed copper zone on layer 16, net N$169
- removed copper zone on layer 16, net N$170

Commit message: Fixed ground vias DRC errors
Parts:
- moved TP37 0.30 mm to (46.0, 31.4)
- moved TP27 0.19 mm to (102.0, 54.7)
- moved TP25 0.11 mm to (103.0, 54.7)
- moved TP26 0.10 mm to (102.5, 55.5)
Routing:
- net N$95: track 2.01 -> 0.00 mm
- net N$93: track 1.38 -> 0.00 mm
- net N$97: track 1.37 -> 0.00 mm
Changed lines of the file:
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@@
 <layers>
 <layer number="1" name="Top" color="4" fill="1" visible="yes" active="yes"/>
-<layer number="2" name="GND" color="1" fill="3" visible="no" active="yes"/>
+<layer number="2" name="GND" color="1" fill="3" visible="yes" active="yes"/>
 <layer number="3" name="Power" color="4" fill="3" visible="no" active="yes"/>
 <layer number="14" name="NS" color="1" fill="6" visible="yes" active="yes"/>
@@
 <attribute name="TP_SIGNAL_NAME" value="" x="107.8" y="49.35" size="1.778" layer="27" rot="R90" display="off"/>
 </element>
-<element name="TP25" library="testpad" package="TP06R" value="TPTP06R" x="103.063" y="54.7096" rot="R90">
-<attribute name="TP_SIGNAL_NAME" value="" x="103.063" y="54.7096" size="1.778" layer="27" rot="R90" display="off"/>
+<element name="TP25" library="testpad" package="TP06R" value="TPTP06R" x="102.95" y="54.7" rot="R90">
+<attribute name="TP_SIGNAL_NAME" value="" x="102.95" y="54.7" size="1.778" layer="27" rot="R90" display="off"/>
 </element>
-<element name="TP26" library="testpad" package="TP06R" value="TPTP06R" x="102.413" y="55.4096" rot="R90">
-<attribute name="TP_SIGNAL_NAME" value="" x="102.413" y="55.4096" size="1.778" layer="27" rot="R90" display="off"/>
+<element name="TP26" library="testpad" package="TP06R" value="TPTP06R" x="102.45" y="55.5" rot="R90">
+<attribute name="TP_SIGNAL_NAME" value="" x="102.45" y="55.5" size="1.778" layer="27" rot="R90" display="off"/>
 </element>
-<element name="TP27" library="testpad" package="TP06R" value="TPTP06R" x="101.763" y="54.7096" rot="R90">
-<attribute name="TP_SIGNAL_NAME" value="" x="101.763" y="54.7096" size="1.778" layer="27" rot="R90" display="off"/>
+<element name="TP27" library="testpad" package="TP06R" value="TPTP06R" x="101.95" y="54.7" rot="R90">
+<attribute name="TP_SIGNAL_NAME" value="" x="101.95" y="54.7" size="1.778" layer="27" rot="R90" display="off"/>
 </element>
 <element name="R2" library="rcl" package="R0402" value="10" x="106" y="56" rot="MR90"/>
@@
 </element>
 <element name="D3" library="diode-0603" package="0603-B-NOSILK-DIODE" value="DIODE-0603" x="104" y="14" rot="MR90"/>
-<element name="TP37" library="testpad" package="TP06R" value="TPTP06R" x="46.2876" y="31.4218">
-<attribute name="TP_SIGNAL_NAME" value="" x="46.0876" y="31.4218" size="1.778" layer="27" display="off"/>
+<element name="TP37" library="testpad" package="TP06R" value="TPTP06R" x="46" y="31.35">
+<attribute name="TP_SIGNAL_NAME" value="" x="45.8" y="31.35" size="1.778" layer="27" display="off"/>
 </element>
 <element name="JP1" library="jumper" package="JP1" value="" x="18.3" y="58" rot="R270"/>
@@
 <wire x1="52.04038125" y1="42.540378125" x2="53.923328125" y2="47.094396875" width="0" layer="19" extent="1-16"/>
 </signal>
-<signal name="GND" class="1" airwireshidden="yes">
+<signal name="GND" class="1">
 <contactref element="U1" pad="10"/>
 <contactref element="C1" pad="2"/>
@@
 <wire x1="27" y1="66.45" x2="27.295" y2="66.448" width="0.127" layer="1"/>
 <wire x1="27.295" y1="66.448" x2="27.85" y2="65.9" width="0.127" layer="1"/>
-<wire x1="32.2" y1="74.15" x2="32.2" y2="75.5142" width="0.127" layer="16"/>
-<wire x1="32.2" y1="75.5142" x2="32.1818" y2="75.5142" width="0.127" layer="16"/>
-<via x="32.1818" y="75.5142" extent="1-16" drill="0.2032" diameter="0.6096"/>
 <wire x1="32.1818" y1="75.5142" x2="32.1818" y2="75.7174" width="0.127" layer="2"/>
-<wire x1="32.1818" y1="75.7174" x2="32.2072" y2="75.7174" width="0.127" layer="2"/>
-<wire x1="55.2" y1="74.15" x2="55.2" y2="75.3872" width="0.127" layer="16"/>
-<wire x1="55.2" y1="75.3872" x2="55.1688" y2="75.3872" width="0.127" layer="16"/>
-<via x="55.1688" y="75.3872" extent="1-16" drill="0.2032" diameter="0.6096"/>
-<wire x1="55.1688" y1="75.3872" x2="55.1688" y2="75.4634" width="0.127" layer="2"/>
+<wire x1="32.1818" y1="75.7174" x2="32.2" y2="75.7174" width="0.127" layer="2"/>
 <wire x1="78.2" y1="74.15" x2="78.2" y2="75.343" width="0.127" layer="16"/>
 <wire x1="78.2" y1="75.343" x2="78.1812" y2="75.3618" width="0.127" layer="16"/>
@@
 <wire x1="78.1812" y1="75.3618" x2="78.1812" y2="75.438" width="0.127" layer="2"/>
 <wire x1="78.1812" y1="75.438" x2="78.2066" y2="75.4634" width="0.127" layer="2"/>
-<wire x1="101.4" y1="74.15" x2="101.4" y2="75.4126" width="0.127" layer="16"/>
-<wire x1="101.4" y1="75.4126" x2="101.3968" y2="75.4126" width="0.127" layer="16"/>
-<via x="101.3968" y="75.4126" extent="1-16" drill="0.2032" diameter="0.6096"/>
-<wire x1="101.3968" y1="75.4126" x2="101.3968" y2="75.5142" width="0.127" layer="2"/>
 <wire x1="32.2" y1="2.35" x2="32.2" y2="0.889" width="0.127" layer="16"/>
 <wire x1="32.2" y1="0.889" x2="32.2326" y2="0.889" width="0.127" layer="16"/>
@@
 <vertex x="81.9" y="30.2"/>
 </polygon>
-<wire x1="99.1" y1="64.8" x2="99.04" y2="63.99" width="0" layer="19" extent="16-16"/>
+<wire x1="32.2" y1="74.15" x2="32.2" y2="75.3" width="0.127" layer="16"/>
+<via x="32.2" y="75.3" extent="1-16" drill="0.2032" diameter="0.6096"/>
+<wire x1="32.2" y1="75.3" x2="32.2" y2="75.7174" width="0.127" layer="2"/>
+<wire x1="32.2" y1="75.7174" x2="32.2072" y2="75.7174" width="0.127" layer="2"/>
 <wire x1="79" y1="13.6" x2="79.65" y2="14" width="0" layer="19" extent="1-16"/>
 <wire x1="56" y1="13.6" x2="56.65" y2="14" width="0" layer="19" extent="1-16"/>
 <wire x1="33" y1="13.6" x2="33.65" y2="14" width="0" layer="19" extent="1-16"/>
+<wire x1="99.04" y1="63.99" x2="99.1" y2="64.8" width="0" layer="19" extent="16-16"/>
 <wire x1="76.04" y1="63.99" x2="76.1" y2="64.8" width="0" layer="19" extent="16-16"/>
 <wire x1="53.04" y1="63.99" x2="53.1" y2="64.8" width="0" layer="19" extent="16-16"/>
@@
 <wire x1="8.25" y1="21.5" x2="12.282" y2="32.1336" width="0" layer="19" extent="16-16"/>
 <wire x1="8.25" y1="16.9" x2="8.25" y2="21.5" width="0" layer="19" extent="16-16"/>
+<wire x1="55.2" y1="74.15" x2="55.2" y2="75.3" width="0.127" layer="16"/>
+<via x="55.2" y="75.3" extent="1-16" drill="0.2032" diameter="0.6096"/>
+<wire x1="55.2" y1="75.3" x2="55.2" y2="75.4" width="0.127" layer="2"/>
+<wire x1="55.2" y1="75.4" x2="62.555" y2="72.395" width="0" layer="19" extent="1-16"/>
+<wire x1="101.4" y1="74.15" x2="101.4" y2="75.3" width="0.127" layer="16"/>
+<via x="101.4" y="75.3" extent="1-16" drill="0.2032" diameter="0.6096"/>
+<wire x1="101.4" y1="75.3" x2="101.4" y2="75.4" width="0.127" layer="2"/>
+<wire x1="101.4" y1="75.4" x2="99.1" y2="67" width="0" layer="19" extent="1-16"/>
 </signal>
 <signal name="+3V3" class="1">
@@
 <contactref element="U$14" pad="159"/>
 <contactref element="TP25" pad="TP"/>
-<wire x1="102.95" y1="53.4" x2="102.903" y2="54.5496" width="0.127" layer="1"/>
-<wire x1="102.903" y1="54.5496" x2="103.063" y2="54.7096" width="0.127" layer="1"/>
+<wire x1="102.95" y1="54.7" x2="102.95" y2="53.4" width="0" layer="19" extent="1-1"/>
 </signal>
 <signal name="N$95">
 <contactref element="U$14" pad="160"/>
 <contactref element="TP26" pad="TP"/>
-<wire x1="102.45" y1="53.4" x2="102.413" y2="55.4096" width="0.127" layer="1"/>
+<wire x1="102.45" y1="55.5" x2="102.45" y2="53.4" width="0" layer="19" extent="1-1"/>
 </signal>
 <signal name="N$97">
 <contactref element="U$14" pad="161"/>
 <contactref element="TP27" pad="TP"/>
-<wire x1="101.763" y1="54.7096" x2="101.903" y2="54.5696" width="0.127" layer="1"/>
-<wire x1="101.903" y1="54.5696" x2="101.95" y2="53.4" width="0.127" layer="1"/>
+<wire x1="101.95" y1="54.7" x2="101.95" y2="53.4" width="0" layer="19" extent="1-1"/>
 </signal>
 <signal name="N$100">
@@
 <contactref element="R148" pad="1"/>
 <wire x1="46.8946875" y1="32.28758125" x2="102" y2="14.8" width="0" layer="19" extent="1-16"/>
-<wire x1="46.2876" y1="31.4218" x2="46.8946875" y2="32.28758125" width="0" layer="19" extent="1-1"/>
+<wire x1="46" y1="31.35" x2="46.8946875" y2="32.28758125" width="0" layer="19" extent="1-1"/>
 <wire x1="32.23" y1="51.905" x2="46.8946875" y2="32.28758125" width="0" layer="19" extent="1-1"/>
 <wire x1="32.35" y1="54" x2="32.23" y2="51.905" width="0" layer="19" extent="16-16"/>
-<wire x1="20.365" y1="4.955" x2="46.2876" y2="31.4218" width="0" layer="19" extent="1-1"/>
+<wire x1="20.365" y1="4.955" x2="46" y2="31.35" width="0" layer="19" extent="1-1"/>
 <wire x1="20.365" y1="3.685" x2="20.365" y2="4.955" width="0" layer="19" extent="1-1"/>
 <wire x1="11.35" y1="18.6" x2="20.365" y2="4.955" width="0" layer="19" extent="16-16"/>
