File: av3/rocketnet-hub/eagle/mcu_page_combined.brd (EAGLE design)
At the start: 112.7 x 76.3 mm, 447 parts, among them J1 ROCKETNET-CONNECTOR-16M, J10 1.27MM_HDR_1X4_TX_RX, J12 1.27MM_HDR_2X12X1, J13 1.27MM_HDR_2X12X1, J14 ROCKETNET-UMBILICAL-18, J15 1.27MM_HDR_1X4, J16 1.27MM_HDR_1X4, J17 1.27MM_HDR_1X4, J18 1.27MM_HDR_1X4, J19 1.27MM_HDR_1X4, J2 ROCKETNET-CONNECTOR-16M, J20 1.27MM_HDR_1X4, J21 1.27MM_HDR_1X4, J22 1.27MM_HDR_2X5, J3 ROCKETNET-CONNECTOR-16M, J4 ROCKETNET-CONNECTOR-16M, J5 1.27MM_HDR_2X12X1, J6 ROCKETNET-CONNECTOR-16M, J7 ROCKETNET-CONNECTOR-16M, J8 ROCKETNET-CONNECTOR-16M, J9 ROCKETNET-BATTERY-14, Q2 FDS6680ASOIC8, Q3 FDS6680ASOIC8, Q4 FDS6680ASOIC8, Q5 SIS412DNSOP-8, Q6 BSS138W-7-F, Q7 SIS412DNSOP-8, T1 BSS84, T10 ALT4532, T11 ALT4532, T12 ALT4532, T13 ALT4532, T14 ALT4532, T15 ALT4532, T16 ALT4532, T17 ALT4532, T18 ALT4532, T19 BSS84, T2 2N7000, T3 ALT4532, T4 ALT4532, T5 ALT4532, T6 ALT4532, T7 ALT4532, T8 ALT4532, T9 ALT4532, U1 STM32F407V100-PIN_QFP, U10 TPS2420QFN-16, U11 TPS2420QFN-16, U12 TPS2420QFN-16, U13 TPS2420QFN-16, U14 MAX4734ETC+, U15 MAX4734ETC+, U2 BQ24725QFN-20, U3 SN65220DBV, U4 KS8999, U5 LTM8023, U6 MIC37101-2.1YM, U7 TPS2420QFN-16, U8 TPS2420QFN-16, U9 TPS2420QFN-16

Commit message: Updated libraries for better readability; cleaned up and organized subcircuits; added/removed/modified various components
Parts:
- removed R111, R18, R25, R31, R37, R55, R65: 10k, rcl_custom:0402-B
- removed R140, R141: 10k, rcl_custom:0402-B-NOSILK
- added C46, C47: 1u, rcl_custom:0603-B-NOSILK
- added C52: 4.7u/TBD, rcl_custom:0402-B
- C100, C101, C95, C96, C97, C98, C99: value NP -> TBD
- C102: value 2200pF -> 2200pF/40V
- C105, C94: value 0.1uF -> 0.1uF/40V
- C113, C124: value 1uF -> 1uF/40V
- C117, C118, C123, C125: value 10uF -> 10uF/40V
- C39: value 100n -> 100n/40V
- C43: value 1u -> 1u/40V
- C60: value 2.2uF -> 2.2uF/40V
- C84: value 47u -> 4.7u
- J10: value 1.27MM_HDR_1X4_TX_RX -> UART Header
- J12: value 1.27MM_HDR_2X12X1 -> BOOT1 Jumper
- J13: value 1.27MM_HDR_2X12X1 -> PGOOD Jumper
- J22: value 1.27MM_HDR_2X5 -> Debug Header
- J5: value 1.27MM_HDR_2X12X1 -> BOOT0 Jumper
- L1: value 4.7uH -> 4.7uH/IHLP2525CZER4R7M01
- LED1, LED13, LED17, LED21, LED25, LED29, LED33, LED5, LED9: value (none) -> AMBER
- R128: value 10 -> 1k
- R134: value 0.01 -> PMR18EZPFU10L0/0.5 Watt
- R146: value 10m -> WSLP1206R0100FEA/1.0 Watt
- T2: value 2N7000 -> NDS335N
Connections:
- net VDD renamed +2V1
- removed net N$208: R148.2, R167.1, T19.2, U3.4, U3.6
- new net N$31: R148.2, R167.1, T19.1, U3.4, U3.6
- net +3V3: now also C46.1, C52.1, T19.2; no longer R111.2, R140.2, R141.2, R18.2, R25.2, R31.2, R37.2, R55.2, R65.2, T19.1
- net GND: now also C46.2, C47.2, C52.2
- net N$113: now also C47.1
- net NODE1_!PG: no longer R18.1
- net NODE2_!PG: no longer R25.1
- net NODE3_!PG: no longer R31.1
- net NODE4_!PG: no longer R37.1
- net NODE5_!PG: no longer R55.1
- net NODE6_!PG: no longer R65.1
- net NODE7_!PG: no longer R111.1
- net SCL: no longer R140.1
- net SDA: no longer R141.1
Routing:
- net N$161: track 15.4 -> 0.00 mm, vias 2 -> 0
- net BAT: track 10.4 -> 5.59 mm, vias 6 -> 5
- net N$37: track 1.27 -> 0.00 mm
- net N$159: track 6.68 -> 5.74 mm
- net +18V: track 20.0 -> 19.5 mm
- added copper zone on layer 1, net N$32
- removed copper zone on layer 1, net N$115

Commit message: Added shunt diode for Ethernet Enable circuitry; added DNI pull-up resistor pads for Mode Select pins on the KSZ8999
Parts:
- added D1: DIODE-0603, diode-0603:0603-B-NOSILK-DIODE
- added R18, R25, R31, R37: 0, rcl_custom:0402-B
- C52: value 4.7u/TBD -> 1u-4.7u
- C83: value .1u -> 0.1u
Connections:
- net +2V1: now also R18.2, R25.2, R31.2, R37.2
- net ETH_EN: now also D1.ANODE
- net GND: now also D1.CATHODE
- net N$10: now also R31.1, R7.1, U4.166; no longer R6.1, U4.165
- net N$14: now also R25.1, R6.1, U4.165; no longer R7.1, U4.166
- net N$19: now also R18.1, R4.1, U4.164; no longer R8.1, U4.167
- net N$8: now also R37.1, R8.1, U4.167; no longer R4.1, U4.164
Routing:
- net N$27: track 7.58 -> 0.00 mm, vias 1 -> 0
Changed lines of the file:
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@@
 <element name="D2" library="diode-0603" package="0603-B-NOSILK-DIODE" value="DIODE-0603" x="106" y="14" rot="MR90"/>
 <element name="R47" library="rcl_custom" package="0402-B" value="10k" x="108" y="14" rot="MR270"/>
-<element name="C83" library="rcl_custom" package="0402-B" value=".1u" x="100" y="14" rot="MR90"/>
+<element name="C83" library="rcl_custom" package="0402-B" value="0.1u" x="100" y="14" rot="MR90"/>
 <element name="C84" library="rcl_custom" package="1206-B" value="4.7u" x="100" y="36.3" rot="MR180"/>
 <element name="C85" library="rcl_custom" package="0402-B" value=".1u" x="100" y="34" rot="MR180"/>
@@
 <element name="C46" library="rcl_custom" package="0603-B-NOSILK" value="1u" x="-7" y="-39"/>
 <element name="C47" library="rcl_custom" package="0603-B-NOSILK" value="1u" x="-7" y="-44"/>
-<element name="C52" library="rcl_custom" package="0402-B" value="4.7u/TBD" x="-7" y="-49"/>
+<element name="C52" library="rcl_custom" package="0402-B" value="1u-4.7u" x="-7" y="-49"/>
+<element name="R18" library="rcl_custom" package="0402-B" value="0" x="-7" y="-54"/>
+<element name="R25" library="rcl_custom" package="0402-B" value="0" x="-3" y="-54"/>
+<element name="R31" library="rcl_custom" package="0402-B" value="0" x="-7" y="-59"/>
+<element name="R37" library="rcl_custom" package="0402-B" value="0" x="-3" y="-59"/>
+<element name="D1" library="diode-0603" package="0603-B-NOSILK-DIODE" value="DIODE-0603" x="-7" y="-64"/>
 </elements>
 <signals>
@@
 <contactref element="U5" pad="GND@19"/>
 <contactref element="U5" pad="GND@22"/>
+<contactref element="D1" pad="CATHODE"/>
 <wire x1="100.1" y1="67" x2="101.4" y2="73.98" width="0" layer="19" extent="16-16"/>
 <wire x1="99" y1="67" x2="100.1" y2="67" width="0" layer="19" extent="1-1"/>
@@
 <wire x1="-6.2" y1="-44" x2="-6.2" y2="-39" width="0" layer="19" extent="1-1"/>
 <wire x1="-6.52" y1="-49" x2="-6.2" y2="-44" width="0" layer="19" extent="1-1"/>
+<wire x1="-6.2" y1="-64" x2="-6.52" y2="-49" width="0" layer="19" extent="1-1"/>
 </signal>
 <signal name="+3V3" class="1">
@@
 <contactref element="U6" pad="1"/>
 <contactref element="R130" pad="1"/>
+<contactref element="D1" pad="ANODE"/>
 <wire x1="96.4" y1="28.795" x2="102.5" y2="20.48" width="0" layer="19" extent="16-16"/>
 <wire x1="94.58" y1="28.8" x2="96.4" y2="28.795" width="0" layer="19" extent="16-16"/>
 <wire x1="58.16596875" y1="42.85175625" x2="94.58" y2="28.8" width="0" layer="19" extent="1-16"/>
+<wire x1="-7.8" y1="-64" x2="58.16596875" y2="42.85175625" width="0" layer="19" extent="1-1"/>
 </signal>
 <signal name="N$16">
@@
 <wire x1="105.0254" y1="19.516" x2="105.9906" y2="20.984" width="0" layer="19" extent="16-16"/>
 </signal>
-<signal name="N$28">
-<contactref element="C12" pad="1"/>
-<contactref element="R43" pad="1"/>
-<contactref element="T2" pad="3"/>
-<wire x1="105.9906" y1="17.484" x2="105.48" y2="16.2" width="0" layer="19" extent="16-16"/>
-<wire x1="102.5" y1="19.52" x2="105.9906" y2="17.484" width="0" layer="19" extent="16-16"/>
-</signal>
 <signal name="N$50">
 <contactref element="U1" pad="60"/>
@@
 <wire x1="46.825" y1="65.5" x2="46.9" y2="67.075" width="0" layer="19" extent="1-1"/>
 </signal>
-<signal name="N$8">
-<contactref element="R4" pad="1"/>
-<contactref element="U4" pad="164"/>
-<wire x1="100.45" y1="53.4" x2="102.2" y2="56.52" width="0" layer="19" extent="1-16"/>
-</signal>
-<signal name="N$10">
-<contactref element="R6" pad="1"/>
-<contactref element="U4" pad="165"/>
-<wire x1="99.95" y1="53.4" x2="101.1" y2="56.52" width="0" layer="19" extent="1-16"/>
-</signal>
-<signal name="N$14">
-<contactref element="R7" pad="1"/>
-<contactref element="U4" pad="166"/>
-<wire x1="99.45" y1="53.4" x2="100" y2="56.52" width="0" layer="19" extent="1-16"/>
-</signal>
-<signal name="N$19">
-<contactref element="R8" pad="1"/>
-<contactref element="U4" pad="167"/>
-<wire x1="98.95" y1="53.4" x2="98.9" y2="56.52" width="0" layer="19" extent="1-16"/>
-</signal>
-<signal name="N$27">
-<contactref element="U4" pad="163"/>
-<contactref element="R2" pad="1"/>
-<wire x1="106" y1="55.52" x2="102.613" y2="52.2596" width="0.1778" layer="16"/>
-<wire x1="102.613" y1="52.2596" x2="100.913" y2="52.2596" width="0.1778" layer="16"/>
-<via x="100.913" y="52.2596" extent="1-16" drill="0.2032" diameter="0.508"/>
-<wire x1="100.913" y1="52.2596" x2="100.95" y2="53.4" width="0.1778" layer="1"/>
-<wire x1="100.913" y1="53.4196" x2="100.95" y2="53.4" width="0.1778" layer="1"/>
-</signal>
 <signal name="N$47">
 <contactref element="U4" pad="170"/>
@@
 <wire x1="94.663" y1="50.3" x2="93.363" y2="49.98" width="0.254" layer="16"/>
 <wire x1="94.663" y1="50.3" x2="95.483" y2="50.4796" width="0.254" layer="16"/>
-<contactref element="R2" pad="2"/>
 <contactref element="C57" pad="2"/>
 <contactref element="T6" pad="6"/>
@@
 <contactref element="T17" pad="6"/>
 <contactref element="T18" pad="6"/>
+<contactref element="R18" pad="2"/>
+<contactref element="R25" pad="2"/>
+<contactref element="R31" pad="2"/>
+<contactref element="R37" pad="2"/>
+<contactref element="R2" pad="2"/>
 <wire x1="106" y1="56.48" x2="107.1" y2="56.48" width="0" layer="19" extent="16-16"/>
 <wire x1="103.95" y1="53.4" x2="106" y2="56.48" width="0" layer="19" extent="1-16"/>
@@
 <wire x1="21.15" y1="11" x2="21.48" y2="13" width="0" layer="19" extent="1-16"/>
 <wire x1="14.65" y1="11" x2="21.15" y2="11" width="0" layer="19" extent="1-1"/>
+<wire x1="-2.52" y1="-54" x2="14.65" y2="11" width="0" layer="19" extent="1-1"/>
+<wire x1="-6.52" y1="-54" x2="-2.52" y2="-54" width="0" layer="19" extent="1-1"/>
+<wire x1="-6.52" y1="-59" x2="-6.52" y2="-54" width="0" layer="19" extent="1-1"/>
+<wire x1="-2.52" y1="-59" x2="-6.52" y2="-59" width="0" layer="19" extent="1-1"/>
 </signal>
 <signal name="N$115">
@@
 <wire x1="7.7608" y1="34.4314" x2="7.8094" y2="35.7098" width="0" layer="19" extent="1-16"/>
 </signal>
+<signal name="N$8">
+<contactref element="U4" pad="167"/>
+<contactref element="R8" pad="1"/>
+<contactref element="R37" pad="1"/>
+<wire x1="98.95" y1="53.4" x2="98.9" y2="56.52" width="0" layer="19" extent="1-16"/>
+<wire x1="-3.48" y1="-59" x2="98.95" y2="53.4" width="0" layer="19" extent="1-1"/>
+</signal>
+<signal name="N$10">
+<contactref element="U4" pad="166"/>
+<contactref element="R7" pad="1"/>
+<contactref element="R31" pad="1"/>
+<wire x1="99.45" y1="53.4" x2="100" y2="56.52" width="0" layer="19" extent="1-16"/>
+<wire x1="-7.48" y1="-59" x2="99.45" y2="53.4" width="0" layer="19" extent="1-1"/>
+</signal>
+<signal name="N$14">
+<contactref element="U4" pad="165"/>
+<contactref element="R6" pad="1"/>
+<contactref element="R25" pad="1"/>
+<wire x1="99.95" y1="53.4" x2="101.1" y2="56.52" width="0" layer="19" extent="1-16"/>
+<wire x1="-3.48" y1="-54" x2="99.95" y2="53.4" width="0" layer="19" extent="1-1"/>
+</signal>
+<signal name="N$19">
+<contactref element="R4" pad="1"/>
+<contactref element="U4" pad="164"/>
+<contactref element="R18" pad="1"/>
+<wire x1="100.45" y1="53.4" x2="102.2" y2="56.52" width="0" layer="19" extent="1-16"/>
+<wire x1="-7.48" y1="-54" x2="100.45" y2="53.4" width="0" layer="19" extent="1-1"/>
+</signal>
+<signal name="N$27">
+<contactref element="U4" pad="163"/>
+<contactref element="R2" pad="1"/>
+<wire x1="100.95" y1="53.4" x2="106" y2="55.52" width="0" layer="19" extent="1-16"/>
+</signal>
+<signal name="N$28">
+<contactref element="T2" pad="3"/>
+<contactref element="R43" pad="1"/>
+<contactref element="C12" pad="1"/>
+<wire x1="105.48" y1="16.2" x2="105.9906" y2="17.484" width="0" layer="19" extent="16-16"/>
+<wire x1="102.5" y1="19.52" x2="105.9906" y2="17.484" width="0" layer="19" extent="16-16"/>
+</signal>
 </signals>

Commit message: making sure brd and sch stay in sync
Parts:
- R1, R16, R20, R24, R28, R32, R38, R44, R45, R46, R5, R9: value 220 -> 750
- R107, R110, R112, R128, R19, R23, R26, R30, R33, R36, R39, R50, R53, R57, R63: value 1k -> 750
- R2: value 10 -> 0
- R48: value 1k -> 150

Commit message: Tidied schematics up; fixed PGOOD jumper
Parts:
- removed R72: 10k, rcl_custom:0402-B
- added R55: 22, rcl_custom:0402-B-NOSILK
- added TP39, TP40: TPTP06R, testpad:TP06R
- C52: value 1u-4.7u -> 4.7u
- E5: value FB -> TBD/FB; device rcl_custom:0603-B -> rcl_custom:0603-B-NOSILK
- J15, J16, J17, J18, J19, J20, J21: value 1.27MM_HDR_1X4 -> Auxiliary Header
- R134: value PMR18EZPFU10L0/0.5 Watt -> 10m/PMR18EZPFU10L0/0.5 Watt
- R146: value WSLP1206R0100FEA/1.0 Watt -> 10m/WSLP1206R0100FEA/1.0 Watt
- R18, R25, R31, R37: value 0 -> NP
- moved R130 147.1 mm to (-7.00, -78.0), flipped to the top
Connections:
- net NODE1_!PG renamed N$168
- net RXD renamed STM32_RX
- net TXD renamed STM32_TX
- removed net MTXER: U4.101
- new net N$208: TP39.TP, U4.101
- new net N$251: TP40.TP, U4.87
- net ETH_EN: now also D1.CATHODE; no longer D1.ANODE
- net GND: now also R4.1, R6.1, R7.1, R8.1; no longer D1.CATHODE, R4.2, R6.2, R7.2, R72.2, R8.2
- net N$10: now also R7.2; no longer R7.1
- net N$14: now also R6.2; no longer R6.1
- net N$167: now also C134.1, R55.1; no longer R72.1, U1.69
- net N$19: now also R4.2; no longer R4.1
- net N$28: now also D1.ANODE
- net N$29: now also J13.2, LED22.A; no longer J13.1, R128.2
- net N$30: now also J13.1, R128.2; no longer J13.2, LED22.A
- net N$5: now also R55.2; no longer C134.1
- net N$8: now also R8.2; no longer R8.1
Routing:
- net N$2: track 2.71 -> 0.00 mm, vias 1 -> 0
- net NODE1_IMON_IN: track 6.54 -> 5.59 mm
- net GND: track 29.4 -> 28.6 mm

Commit message: Cleaned up a couple current switch circuity
Connections:
- net NODE2_!PG renamed N$212
- net NODE3_!PG renamed N$217
- net NODE4_!PG renamed N$250
- net NODE4_LTCH renamed N$249
Routing:
- net GND: track 28.6 -> 23.9 mm
- net N$130: track 2.72 -> 0.00 mm, vias 1 -> 0
- net NODE2_IMON_IN: track 6.46 -> 5.53 mm
- net NODE3_IMON_IN: track 6.46 -> 5.55 mm
- net NODE4_IMON_IN: track 6.48 -> 5.63 mm

Commit message: Tidied up Node Connections page
Connections:
- net NODE6_!PG renamed N$252
- net NODE7_!PG renamed N$253
- removed net NODE5_IMON: R56.2, U13.13, U15.1
- new net NODE8_IMON: R56.2, U13.13, U15.7
Routing:
- net NODE5_IMON: track 6.51 -> 0.00 mm
- net NODE8_IMON: track 0.00 -> 5.52 mm
- net N$149: track 2.93 -> 0.00 mm, vias 1 -> 0
- net N$148: track 2.93 -> 0.00 mm, vias 1 -> 0

Commit message: Replaced passives with No-Silk outline; moved components on the board to approximate location
Parts:
- C1, C10, C100, C101, C106, C107, C11, C12, C126, C127, C128, C129, C13, C130, C132, C133, C14, C15, C16, C17, C18, C19, C2, C20, C21, C22, C23, C24, C25, C26, C27, C28, C29, C3, C30, C31, C32, C33, C34, C35, C36, C37, C38, C4, C40, C41, C42, C44, C45, C48, C49, C5, C50, C51, C53, C54, C55, C56, C57, C6, C61, C62, C63, C64, C65, C66, C67, C68, C69, C7, C70, C71, C72, C73, C74, C75, C76, C8, C83, C85, C86, C9, C95, C96, C97, C98, C99, R1, R10, R100, R101, R102, R103, R104, R105, R106, R107, R108, R109, R110, R112, R113, R114, R115, R116, R117, R118, R119, R12, R120, R121, R122, R123, R124, R125, R126, R127, R128, R13, R130, R131, R14, R147, R148, R149, R15, R150, R151, R152, R153, R154, R155, R156, R157, R158, R159, R16, R160, R161, R162, R163, R164, R165, R167, R17, R18, R19, R2, R20, R21, R22, R23, R24, R25, R26, R27, R28, R29, R3, R30, R31, R32, R33, R34, R35, R36, R37, R38, R39, R4, R41, R42, R43, R44, R45, R46, R47, R48, R49, R5, R50, R51, R52, R53, R54, R56, R57, R58, R59, R6, R60, R61, R62, R63, R64, R66, R67, R68, R69, R7, R70, R71, R73, R74, R75, R76, R77, R78, R79, R8, R80, R81, R82, R83, R84, R85, R86, R87, R88, R89, R9, R90, R91, R92, R93, R94, R95, R96, R97, R98, R99: device rcl_custom:0402-B -> rcl_custom:0402-B-NOSILK
- C103, C104, C52, C87, C88, C89, C90, C91, C92, C93: device rcl_custom:0402-B -> rcl_custom:0603-B-NOSILK
- C77, C78, C79, C80, C81, C82: device rcl_custom:0603-B-NOSILK -> rcl_custom:0603-A-NOSILK
- R168: device rcl:R0402 -> rcl_custom:0402-B-NOSILK
- moved R18 153.6 mm to (97.0, 59.0)
- moved R25 153.6 mm to (101.0, 59.0)
- moved R31 153.6 mm to (97.0, 54.0)
- moved R37 153.6 mm to (101.0, 54.0)
- moved TP40 149.2 mm to (95.0, 20.0)
- moved TP39 142.9 mm to (103.0, 21.0)
- moved R130 139.7 mm to (61.0, 44.0)
- moved D1 135.0 mm to (101.0, 17.0)
- moved R55 129.2 mm to (50.0, 33.0), flipped to the bottom, turned to 135 degrees
- moved C52 128.5 mm to (92.0, 33.0)
- moved C47 101.5 mm to (50.0, 40.0), flipped to the bottom, turned to 315 degrees
- moved C46 97.0 mm to (52.0, 38.0), flipped to the bottom, turned to 315 degrees
- moved R168 92.4 mm to (41.0, 49.0), flipped to the bottom, turned to 180 degrees
- moved TP38 91.4 mm to (38.0, 44.0)
- moved J22 83.5 mm to (40.0, 46.0)
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
Commit message: Added SPI interface for MCU <-> KSZ8999; approved POWER pin ERC warnings
Parts:
- added R65: 10K, rcl_custom:0402-B-NOSILK
Connections:
- new net SPI3_MISO: R65.2, U1.79
- new net SPI3_MOSI: U1.80, U4.92
- new net SPI3_SCK: U1.78, U4.93
- net GND: now also R65.1
- net SCL: no longer U4.93
- net SDA: no longer U4.92
- net STM32_RX: now also U1.69; no longer U1.79
- net STM32_TX: now also U1.68; no longer U1.78
