File: av3/rocketnet-hub/eagle/mcu_page_combined.sch (EAGLE design)
At the start: 386 parts, among them J1 ROCKETNET-CONNECTOR-16M, J2 ROCKETNET-CONNECTOR-16M, J3 ROCKETNET-CONNECTOR-16M, J4 ROCKETNET-CONNECTOR-16M, J5 ROCKETNET-CONNECTOR-16M, J6 ROCKETNET-CONNECTOR-16M, J7 ROCKETNET-CONNECTOR-16M, J8 ROCKETNET-CONNECTOR-16M, J9 DEBUG-CONNECTOR, Q1 25MHz, Q2 FDS6680ASOIC-8, Q3 FDS6680ASOIC-8, Q4 FDS6680ASOIC-8, Q5 SIS412DNSOP-8, Q6 BSS138W-7-F, Q7 SIS412DNSOP-8, U1 STM32F407V100-PIN_QFP, U2 BQ24725QFN-20

Commit message: Replaced Umbilical connector with 14-pin
Parts:
- removed J5: ROCKETNET-CONNECTOR-16M, rocketnet-connector:ROCKETNET-CONNECTOR-16M
- added J10: ROCKETNET-UMBILICAL-12, rocketnet-connector:ROCKETNET-UMBILICAL-12
Connections:
- net GND: no longer J5.B-@1, J5.B-@2
- net N$108: now also J10.RX-@1, J10.RX-@2; no longer J5.RX-@1, J5.RX-@2
- net N$141: now also J10.RX+@1, J10.RX+@2; no longer J5.RX+@1, J5.RX+@2
- net N$38: now also J10.TX+@1, J10.TX+@2; no longer J5.TX+@1, J5.TX+@2
- net N$79: now also J10.TX-@1, J10.TX-@2; no longer J5.TX-@1, J5.TX-@2
- net ROCKET_RDY: now also J10.RR@1, J10.RR@2; no longer J5.AUX1, J5.AUX2
- net RST_N: now also J10.AUX1, J10.AUX2; no longer J5.AUX3, J5.AUX4
- net VIN: no longer J5.B+@1, J5.B+@2
Changed lines of the file:
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@@
 <part name="GND39" library="supply1" deviceset="GND" device=""/>
 <part name="GND43" library="supply1" deviceset="GND" device=""/>
-<part name="GND50" library="supply1" deviceset="GND" device=""/>
 <part name="R100" library="rcl" deviceset="R-US_" device="R0402"/>
 <part name="R101" library="rcl" deviceset="R-US_" device="R0402"/>
@@
 <part name="C125" library="rcl_custom" deviceset="C-EU" device="1206-B" value="10uF"/>
 <part name="P+2" library="supply1" deviceset="+18V" device=""/>
-<part name="J5" library="rocketnet-connector" deviceset="ROCKETNET-CONNECTOR-16" device="M"/>
 <part name="J1" library="rocketnet-connector" deviceset="ROCKETNET-CONNECTOR-16" device="M"/>
 <part name="J2" library="rocketnet-connector" deviceset="ROCKETNET-CONNECTOR-16" device="M"/>
@@
 <part name="U$17" library="headers" deviceset="1.27MM_HDR_1X4" device=""/>
 <part name="U$18" library="headers" deviceset="1.27MM_HDR_1X4" device=""/>
+<part name="J10" library="rocketnet-connector" deviceset="ROCKETNET-UMBILICAL-12" device=""/>
 </parts>
 <sheets>
@@
 <instance part="TP42" gate="G$1" x="50.8" y="43.18" rot="R270"/>
 <instance part="R129" gate="G$1" x="25.4" y="86.36" rot="R90"/>
-<instance part="GND50" gate="1" x="162.56" y="27.94"/>
 <instance part="R100" gate="G$1" x="88.9" y="86.36" rot="R270"/>
 <instance part="R101" gate="G$1" x="96.52" y="86.36" rot="R270"/>
@@
 <instance part="C56" gate="G$1" x="139.7" y="63.5" rot="MR90"/>
 <instance part="C59" gate="G$1" x="149.86" y="58.42" rot="MR90"/>
-<instance part="J5" gate="G$1" x="170.18" y="63.5" rot="MR0"/>
+<instance part="J10" gate="G$1" x="170.18" y="63.5" rot="MR0"/>
 </instances>
 <busses>
@@
 <pinref part="GND81" gate="1" pin="GND"/>
 </segment>
-<segment>
-<wire x1="165.1" y1="45.72" x2="162.56" y2="45.72" width="0.1524" layer="91"/>
-<wire x1="162.56" y1="45.72" x2="162.56" y2="43.18" width="0.1524" layer="91"/>
-<wire x1="162.56" y1="43.18" x2="165.1" y2="43.18" width="0.1524" layer="91"/>
-<wire x1="162.56" y1="43.18" x2="162.56" y2="38.1" width="0.1524" layer="91"/>
-<junction x="162.56" y="43.18"/>
-<pinref part="GND50" gate="1" pin="GND"/>
-<wire x1="162.56" y1="38.1" x2="162.56" y2="35.56" width="0.1524" layer="91"/>
-<wire x1="162.56" y1="35.56" x2="162.56" y2="30.48" width="0.1524" layer="91"/>
-<wire x1="162.56" y1="38.1" x2="165.1" y2="38.1" width="0.1524" layer="91"/>
-<junction x="162.56" y="38.1"/>
-<wire x1="162.56" y1="35.56" x2="165.1" y2="35.56" width="0.1524" layer="91"/>
-<junction x="162.56" y="35.56"/>
-<pinref part="J5" gate="G$1" pin="B-@1"/>
-<pinref part="J5" gate="G$1" pin="B-@2"/>
-</segment>
 </net>
 <net name="+3V3" class="1">
@@
 <junction x="162.56" y="48.26"/>
 <label x="81.28" y="48.26" size="1.016" layer="95" rot="R180" xref="yes"/>
-<pinref part="J5" gate="G$1" pin="AUX3"/>
-<pinref part="J5" gate="G$1" pin="AUX4"/>
+<pinref part="J10" gate="G$1" pin="AUX1"/>
+<pinref part="J10" gate="G$1" pin="AUX2"/>
 </segment>
 </net>
@@
 <junction x="162.56" y="53.34"/>
 <label x="81.28" y="53.34" size="1.016" layer="95" rot="R180" xref="yes"/>
-<pinref part="J5" gate="G$1" pin="AUX1"/>
-<pinref part="J5" gate="G$1" pin="AUX2"/>
+<pinref part="J10" gate="G$1" pin="RR@1"/>
+<pinref part="J10" gate="G$1" pin="RR@2"/>
 </segment>
 </net>
@@
 <wire x1="162.56" y1="76.2" x2="162.56" y2="73.66" width="0.2032" layer="91"/>
 <wire x1="165.1" y1="76.2" x2="162.56" y2="76.2" width="0.2032" layer="91"/>
-<pinref part="J5" gate="G$1" pin="TX+@1"/>
-<pinref part="J5" gate="G$1" pin="TX+@2"/>
+<pinref part="J10" gate="G$1" pin="TX+@1"/>
+<pinref part="J10" gate="G$1" pin="TX+@2"/>
 </segment>
 </net>
@@
 <wire x1="162.56" y1="71.12" x2="162.56" y2="68.58" width="0.2032" layer="91"/>
 <wire x1="165.1" y1="71.12" x2="162.56" y2="71.12" width="0.2032" layer="91"/>
-<pinref part="J5" gate="G$1" pin="TX-@1"/>
-<pinref part="J5" gate="G$1" pin="TX-@2"/>
-</segment>
-</net>
-<net name="VIN" class="1">
-<segment>
-<wire x1="81.28" y1="78.74" x2="162.56" y2="78.74" width="0.1524" layer="91"/>
-<wire x1="162.56" y1="78.74" x2="165.1" y2="78.74" width="0.1524" layer="91"/>
-<wire x1="162.56" y1="78.74" x2="162.56" y2="81.28" width="0.1524" layer="91"/>
-<junction x="162.56" y="78.74"/>
-<wire x1="162.56" y1="81.28" x2="165.1" y2="81.28" width="0.1524" layer="91"/>
-<label x="81.28" y="78.74" size="1.016" layer="95" rot="R180" xref="yes"/>
-<pinref part="J5" gate="G$1" pin="B+@1"/>
-<pinref part="J5" gate="G$1" pin="B+@2"/>
+<pinref part="J10" gate="G$1" pin="TX-@1"/>
+<pinref part="J10" gate="G$1" pin="TX-@2"/>
 </segment>
 </net>
@@
 <wire x1="162.56" y1="58.42" x2="152.4" y2="58.42" width="0.2032" layer="91"/>
 <pinref part="C59" gate="G$1" pin="1"/>
-<pinref part="J5" gate="G$1" pin="RX-@1"/>
-<pinref part="J5" gate="G$1" pin="RX-@2"/>
+<pinref part="J10" gate="G$1" pin="RX-@1"/>
+<pinref part="J10" gate="G$1" pin="RX-@2"/>
 </segment>
 </net>
@@
 <wire x1="142.24" y1="63.5" x2="162.56" y2="63.5" width="0.1524" layer="91"/>
 <junction x="162.56" y="63.5"/>
-<pinref part="J5" gate="G$1" pin="RX+@1"/>
-<pinref part="J5" gate="G$1" pin="RX+@2"/>
+<pinref part="J10" gate="G$1" pin="RX+@1"/>
+<pinref part="J10" gate="G$1" pin="RX+@2"/>
 </segment>
 </net>

Commit message: Added library parts: 1.27 mm 2x1 and 2x5 header; swapped out umbilical and debug connectors; added battery connector; added 2x1 header for BOOT0 to Vdd jumper
Parts:
- removed TP38, TP39, TP41, TP42: TPTP06R, testpad:TPTP06R
- added J11: 1.27MM_HDR_2X5, headers:1.27MM_HDR_2X5
- added J5: 1.27MM_HDR_2X1, headers:1.27MM_HDR_2X1
- J9: value DEBUG-CONNECTOR -> ROCKETNET-BATTERY-14; device ScottsLib:DEBUG-CONNECTOR -> rocketnet-connector:ROCKETNET-BATTERY-14
Connections:
- removed net DEBUG0: J9.DEBUG.13, TP40.TP
- removed net DEBUG1: J9.DEBUG.14, TP41.TP
- removed net DEBUG2: J9.DEBUG.15, TP42.TP
- removed net RESETOUT: J9.!RSTOUT, TP39.TP
- removed net RTCK: J9.RTCK, TP38.TP
- new net N$168: J11.9, TP40.TP
- net +3V3: now also J5.2
- net BOOT0: now also J5.1; no longer J9.PORT2.10/!EINT0
- net GND: now also J11.3, J11.5; no longer J9.GRND
- net JTAG_TCK: now also J11.4; no longer J9.TCK
- net JTAG_TDI: now also J11.8; no longer J9.TDI
- net JTAG_TDO: now also J11.6; no longer J9.TDO
- net JTAG_TMS: now also J11.2; no longer J9.TMS
- net JTAG_TRST: no longer J9.!TRST
- net N$32: now also J11.1; no longer J9.3.3V
- net RST_N: now also J11.10; no longer J9.!RESET
- net RXD: no longer J9.PORT0.3/RXD0
- net TXD: no longer J9.PORT0.2/TXD0
Other:
- note added: "Battery Connector"
- moved on the sheet: R129, TP40

Commit message: Connected battery charger connector to respective signal lines/power nets
Connections:
- net BAT: now also J9.B+@1, J9.B+@2, J9.B+@3, J9.B+@4
- net GND: now also J9.!PRSNT@1, J9.!PRSNT@2, J9.B-@1, J9.B-@2, J9.B-@3, J9.B-@4
- net SCL: now also J9.SMCLK@1, J9.SMCLK@2
- net SDA: now also J9.SMDAT@1, J9.SMDAT@2
Other:
- moved on the sheet: J9
Changed lines of the file:
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@@
 <part name="J11" library="headers" deviceset="1.27MM_HDR_2X5" device=""/>
 <part name="J9" library="rocketnet-connector" deviceset="ROCKETNET-BATTERY-14" device=""/>
+<part name="GND50" library="supply1" deviceset="GND" device=""/>
 </parts>
 <sheets>
@@
 <text x="-5.08" y="106.68" size="5.08" layer="97">Debug Header</text>
 <text x="66.04" y="106.68" size="5.08" layer="97">Launch Tower Connection</text>
-<text x="-114.3" y="109.22" size="5.08" layer="97">Battery Connector</text>
+<text x="-101.6" y="106.68" size="5.08" layer="97">Battery Connector</text>
 </plain>
 <instances>
@@
 <instance part="J10" gate="G$1" x="170.18" y="63.5" rot="MR0"/>
 <instance part="J11" gate="J" x="25.4" y="60.96"/>
-<instance part="J9" gate="G$1" x="-114.3" y="71.12"/>
+<instance part="J9" gate="G$1" x="-73.66" y="71.12"/>
+<instance part="GND50" gate="1" x="-68.58" y="48.26"/>
 </instances>
 <busses>
@@
 <junction x="20.32" y="63.5"/>
 </segment>
+<segment>
+<pinref part="J9" gate="G$1" pin="!PRSNT@2"/>
+<pinref part="J9" gate="G$1" pin="B-@1"/>
+<wire x1="-68.58" y1="66.04" x2="-68.58" y2="63.5" width="0.1524" layer="91"/>
+<pinref part="J9" gate="G$1" pin="B-@2"/>
+<wire x1="-68.58" y1="60.96" x2="-68.58" y2="63.5" width="0.1524" layer="91"/>
+<junction x="-68.58" y="63.5"/>
+<pinref part="J9" gate="G$1" pin="B-@3"/>
+<wire x1="-68.58" y1="60.96" x2="-68.58" y2="58.42" width="0.1524" layer="91"/>
+<junction x="-68.58" y="60.96"/>
+<pinref part="J9" gate="G$1" pin="B-@4"/>
+<wire x1="-68.58" y1="58.42" x2="-68.58" y2="55.88" width="0.1524" layer="91"/>
+<junction x="-68.58" y="58.42"/>
+<wire x1="-68.58" y1="55.88" x2="-68.58" y2="50.8" width="0.1524" layer="91"/>
+<junction x="-68.58" y="55.88"/>
+<pinref part="GND50" gate="1" pin="GND"/>
+<pinref part="J9" gate="G$1" pin="!PRSNT@1"/>
+<wire x1="-68.58" y1="68.58" x2="-68.58" y2="66.04" width="0.1524" layer="91"/>
+<junction x="-68.58" y="66.04"/>
+</segment>
 </net>
 <net name="+3V3" class="1">
@@
 </segment>
 </net>
+<net name="SCL" class="0">
+<segment>
+<pinref part="J9" gate="G$1" pin="SMCLK@1"/>
+<pinref part="J9" gate="G$1" pin="SMCLK@2"/>
+<wire x1="-68.58" y1="78.74" x2="-68.58" y2="76.2" width="0.1524" layer="91"/>
+<wire x1="-68.58" y1="78.74" x2="-60.96" y2="78.74" width="0.1524" layer="91"/>
+<junction x="-68.58" y="78.74"/>
+<label x="-60.96" y="78.74" size="1.778" layer="95" xref="yes"/>
+</segment>
+</net>
+<net name="SDA" class="0">
+<segment>
+<pinref part="J9" gate="G$1" pin="SMDAT@1"/>
+<pinref part="J9" gate="G$1" pin="SMDAT@2"/>
+<wire x1="-68.58" y1="73.66" x2="-68.58" y2="71.12" width="0.1524" layer="91"/>
+<wire x1="-68.58" y1="73.66" x2="-60.96" y2="73.66" width="0.1524" layer="91"/>
+<junction x="-68.58" y="73.66"/>
+<label x="-60.96" y="73.66" size="1.778" layer="95" xref="yes"/>
+</segment>
+</net>
+<net name="BAT" class="0">
+<segment>
+<pinref part="J9" gate="G$1" pin="B+@4"/>
+<pinref part="J9" gate="G$1" pin="B+@3"/>
+<wire x1="-68.58" y1="81.28" x2="-68.58" y2="83.82" width="0.1524" layer="91"/>
+<pinref part="J9" gate="G$1" pin="B+@2"/>
+<wire x1="-68.58" y1="83.82" x2="-68.58" y2="86.36" width="0.1524" layer="91"/>
+<junction x="-68.58" y="83.82"/>
+<pinref part="J9" gate="G$1" pin="B+@1"/>
+<wire x1="-68.58" y1="86.36" x2="-68.58" y2="88.9" width="0.1524" layer="91"/>
+<junction x="-68.58" y="86.36"/>
+<wire x1="-68.58" y1="88.9" x2="-68.58" y2="91.44" width="0.1524" layer="91"/>
+<junction x="-68.58" y="88.9"/>
+<label x="-68.58" y="91.44" size="1.778" layer="95" rot="R90" xref="yes"/>
+</segment>
+</net>

Commit message: Added option on debug header to select RST_N and/or JTAG_TRST
Parts:
- added J12: 1.27MM_HDR_2X12X1, headers:1.27MM_HDR_2X12X1
- added R147, R148: 0, rcl:R-US_R0402
- added R150: 10k, rcl:R-US_R0402
- J5: value 1.27MM_HDR_2X1 -> 1.27MM_HDR_2X12X1; device headers:1.27MM_HDR_2X1 -> headers:1.27MM_HDR_2X12X1
Connections:
- new net BOOT1: J12.1, U1.PB2
- net +3V3: now also J12.2
- net GND: now also R150.2
- net RST_N: now also R147.1, R148.1, R148.2
Other:
- moved on the sheet: R15, R17
Changed lines of the file:
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@@
 <part name="U$18" library="headers" deviceset="1.27MM_HDR_1X4" device=""/>
 <part name="J10" library="rocketnet-connector" deviceset="ROCKETNET-UMBILICAL-12" device=""/>
-<part name="J5" library="headers" deviceset="1.27MM_HDR_2X1" device=""/>
+<part name="J5" library="headers" deviceset="1.27MM_HDR_2X1" device="2X1"/>
 <part name="+3V34" library="supply1" deviceset="+3V3" device=""/>
 <part name="J11" library="headers" deviceset="1.27MM_HDR_2X5" device=""/>
 <part name="J9" library="rocketnet-connector" deviceset="ROCKETNET-BATTERY-14" device=""/>
 <part name="GND50" library="supply1" deviceset="GND" device=""/>
+<part name="R148" library="rcl" deviceset="R-US_" device="R0402" value="0"/>
+<part name="R147" library="rcl" deviceset="R-US_" device="R0402" value="0"/>
+<part name="J12" library="headers" deviceset="1.27MM_HDR_2X1" device="2X1"/>
+<part name="+3V35" library="supply1" deviceset="+3V3" device=""/>
+<part name="R150" library="rcl" deviceset="R-US_" device="R0402" value="10k"/>
+<part name="GND98" library="supply1" deviceset="GND" device=""/>
 </parts>
 <sheets>
@@
 <instance part="C86" gate="G$1" x="99.06" y="314.96"/>
 <instance part="GND17" gate="1" x="99.06" y="297.18"/>
-<instance part="R15" gate="G$1" x="15.24" y="370.84" rot="R270"/>
-<instance part="R17" gate="G$1" x="7.62" y="370.84" rot="R270"/>
-<instance part="+3V6" gate="G$1" x="7.62" y="381"/>
-<instance part="+3V17" gate="G$1" x="15.24" y="381"/>
+<instance part="R15" gate="G$1" x="-5.08" y="370.84" rot="R270"/>
+<instance part="R17" gate="G$1" x="-12.7" y="370.84" rot="R270"/>
+<instance part="+3V6" gate="G$1" x="-12.7" y="381"/>
+<instance part="+3V17" gate="G$1" x="-5.08" y="381"/>
 <instance part="Q1" gate="G$1" x="63.5" y="462.28" rot="R270"/>
 <instance part="C106" gate="G$1" x="55.88" y="467.36" rot="R90"/>
@@
 <instance part="GND43" gate="1" x="20.32" y="332.74"/>
 <instance part="FRAME1" gate="G$1" x="182.88" y="289.56"/>
-<instance part="J5" gate="G$1" x="-7.62" y="444.5" rot="R180"/>
+<instance part="J5" gate="J" x="-7.62" y="444.5" rot="R180"/>
 <instance part="+3V34" gate="G$1" x="-5.08" y="452.12"/>
+<instance part="J12" gate="J" x="-22.86" y="424.18" rot="R180"/>
+<instance part="+3V35" gate="G$1" x="-20.32" y="431.8"/>
+<instance part="R150" gate="G$1" x="-2.54" y="414.02" rot="R270"/>
+<instance part="GND98" gate="1" x="-2.54" y="406.4"/>
 </instances>
 <busses>
@@
 <wire x1="20.32" y1="337.82" x2="20.32" y2="335.28" width="0.1524" layer="91"/>
 </segment>
+<segment>
+<pinref part="R150" gate="G$1" pin="2"/>
+<pinref part="GND98" gate="1" pin="GND"/>
+</segment>
 </net>
 <net name="+3V3" class="1">
@@
 <segment>
 <pinref part="R17" gate="G$1" pin="1"/>
-<wire x1="7.62" y1="375.92" x2="7.62" y2="378.46" width="0.1524" layer="91"/>
+<wire x1="-12.7" y1="375.92" x2="-12.7" y2="378.46" width="0.1524" layer="91"/>
 <pinref part="+3V6" gate="G$1" pin="+3V3"/>
 </segment>
 <segment>
 <pinref part="R15" gate="G$1" pin="1"/>
-<wire x1="15.24" y1="375.92" x2="15.24" y2="378.46" width="0.1524" layer="91"/>
+<wire x1="-5.08" y1="375.92" x2="-5.08" y2="378.46" width="0.1524" layer="91"/>
 <pinref part="+3V17" gate="G$1" pin="+3V3"/>
 </segment>
 <segment>
-<pinref part="J5" gate="G$1" pin="2"/>
+<pinref part="J5" gate="J" pin="2"/>
 <pinref part="+3V34" gate="G$1" pin="+3V3"/>
 <wire x1="-5.08" y1="441.96" x2="-5.08" y2="449.58" width="0.1524" layer="91"/>
 </segment>
+<segment>
+<pinref part="J12" gate="J" pin="2"/>
+<pinref part="+3V35" gate="G$1" pin="+3V3"/>
+<wire x1="-20.32" y1="421.64" x2="-20.32" y2="429.26" width="0.1524" layer="91"/>
+</segment>
 </net>
 <net name="JTAG_TMS" class="0">
@@
 <segment>
 <pinref part="U1" gate="G$1" pin="PB6"/>
-<wire x1="2.54" y1="363.22" x2="7.62" y2="363.22" width="0.1524" layer="91"/>
-<label x="2.54" y="363.22" size="1.016" layer="95" rot="R180" xref="yes"/>
+<wire x1="-17.78" y1="363.22" x2="-12.7" y2="363.22" width="0.1524" layer="91"/>
+<label x="-17.78" y="363.22" size="1.016" layer="95" rot="R180" xref="yes"/>
 <pinref part="R17" gate="G$1" pin="2"/>
-<wire x1="7.62" y1="363.22" x2="43.18" y2="363.22" width="0.1524" layer="91"/>
-<wire x1="7.62" y1="365.76" x2="7.62" y2="363.22" width="0.1524" layer="91"/>
-<junction x="7.62" y="363.22"/>
+<wire x1="-12.7" y1="363.22" x2="43.18" y2="363.22" width="0.1524" layer="91"/>
+<wire x1="-12.7" y1="365.76" x2="-12.7" y2="363.22" width="0.1524" layer="91"/>
+<junction x="-12.7" y="363.22"/>
 </segment>
 </net>
@@
 <segment>
 <pinref part="U1" gate="G$1" pin="PB7"/>
-<wire x1="2.54" y1="360.68" x2="15.24" y2="360.68" width="0.1524" layer="91"/>
-<label x="2.54" y="360.68" size="1.016" layer="95" rot="R180" xref="yes"/>
+<wire x1="-17.78" y1="360.68" x2="-5.08" y2="360.68" width="0.1524" layer="91"/>
+<label x="-17.78" y="360.68" size="1.016" layer="95" rot="R180" xref="yes"/>
 <pinref part="R15" gate="G$1" pin="2"/>
-<wire x1="15.24" y1="360.68" x2="43.18" y2="360.68" width="0.1524" layer="91"/>
-<wire x1="15.24" y1="365.76" x2="15.24" y2="360.68" width="0.1524" layer="91"/>
-<junction x="15.24" y="360.68"/>
+<wire x1="-5.08" y1="360.68" x2="43.18" y2="360.68" width="0.1524" layer="91"/>
+<wire x1="-5.08" y1="365.76" x2="-5.08" y2="360.68" width="0.1524" layer="91"/>
+<junction x="-5.08" y="360.68"/>
 </segment>
 </net>
@@
 <pinref part="R64" gate="G$1" pin="1"/>
 <junction x="27.94" y="439.42"/>
-<pinref part="J5" gate="G$1" pin="1"/>
+<pinref part="J5" gate="J" pin="1"/>
 <wire x1="27.94" y1="439.42" x2="15.24" y2="439.42" width="0.1524" layer="91"/>
 <wire x1="15.24" y1="439.42" x2="-5.08" y2="439.42" width="0.1524" layer="91"/>
@@
 </segment>
 </net>
+<net name="BOOT1" class="0">
+<segment>
+<pinref part="J12" gate="J" pin="1"/>
+<wire x1="0" y1="419.1" x2="-2.54" y2="419.1" width="0.1524" layer="91"/>
+<pinref part="U1" gate="G$1" pin="PB2"/>
+<wire x1="-2.54" y1="419.1" x2="-20.32" y2="419.1" width="0.1524" layer="91"/>
+<wire x1="43.18" y1="373.38" x2="10.16" y2="373.38" width="0.1524" layer="91"/>
+<wire x1="10.16" y1="373.38" x2="10.16" y2="419.1" width="0.1524" layer="91"/>
+<wire x1="10.16" y1="419.1" x2="0" y2="419.1" width="0.1524" layer="91"/>
+<label x="10.16" y="419.1" size="1.016" layer="95" xref="yes"/>
+</segment>
+</net>
 </nets>
 </sheet>
@@
 <instance part="J9" gate="G$1" x="-73.66" y="71.12"/>
 <instance part="GND50" gate="1" x="-68.58" y="48.26"/>
+<instance part="R148" gate="G$1" x="40.64" y="55.88"/>
+<instance part="R147" gate="G$1" x="40.64" y="48.26"/>
 </instances>
 <busses>
@@
 <net name="RST_N" class="0">
 <segment>
-<wire x1="27.94" y1="55.88" x2="40.64" y2="55.88" width="0.1524" layer="91"/>
-<label x="40.64" y="55.88" size="1.016" layer="95" rot="MR180" xref="yes"/>
+<wire x1="27.94" y1="55.88" x2="33.02" y2="55.88" width="0.1524" layer="91"/>
 <pinref part="J11" gate="J" pin="10"/>
+<pinref part="R148" gate="G$1" pin="1"/>
+<wire x1="33.02" y1="55.88" x2="35.56" y2="55.88" width="0.1524" layer="91"/>
+<wire x1="33.02" y1="55.88" x2="33.02" y2="48.26" width="0.1524" layer="91"/>
+<junction x="33.02" y="55.88"/>
+<pinref part="R147" gate="G$1" pin="1"/>
+<wire x1="33.02" y1="48.26" x2="35.56" y2="48.26" width="0.1524" layer="91"/>
 </segment>
 <segment>
@@
 <pinref part="J10" gate="G$1" pin="AUX2"/>
 </segment>
+<segment>
+<pinref part="R148" gate="G$1" pin="2"/>
+<wire x1="45.72" y1="55.88" x2="48.26" y2="55.88" width="0.1524" layer="91"/>
+<label x="48.26" y="55.88" size="1.016" layer="95" rot="MR180" xref="yes"/>
+</segment>
 </net>
 <net name="ROCKET_RDY" class="0">
@@
 </segment>
 </net>
+<net name="JTAG_TRST" class="0">
+<segment>
+<wire x1="48.26" y1="48.26" x2="45.72" y2="48.26" width="0.1524" layer="91"/>
+<label x="48.26" y="48.26" size="1.016" layer="95" xref="yes"/>
+</segment>
+</net>
