File: av3/rocketnet-hub/eagle/mcu_page_combined.sch (EAGLE design)
At the start: 388 parts, among them J1 ROCKETNET-CONNECTOR-16M, J10 ROCKETNET-UMBILICAL-12, J11 1.27MM_HDR_2X5, J12 1.27MM_HDR_2X12X1, J2 ROCKETNET-CONNECTOR-16M, J3 ROCKETNET-CONNECTOR-16M, J4 ROCKETNET-CONNECTOR-16M, J5 1.27MM_HDR_2X12X1, J6 ROCKETNET-CONNECTOR-16M, J7 ROCKETNET-CONNECTOR-16M, J8 ROCKETNET-CONNECTOR-16M, J9 ROCKETNET-BATTERY-14, Q1 25MHz, Q2 FDS6680ASOIC-8, Q3 FDS6680ASOIC-8, Q4 FDS6680ASOIC-8, Q5 SIS412DNSOP-8, Q6 BSS138W-7-F, Q7 SIS412DNSOP-8, U1 STM32F407V100-PIN_QFP, U2 BQ24725QFN-20

Commit message: battery charger analog grounds properly named + more routing
Connections:
- new net GNDA: C115.2, C117.2, C118.2, C119.2, C120.2, C123.2, C124.2, C125.2, C60.2
- net GND: no longer C115.2, C117.2, C118.2, C119.2, C120.2, C123.2, C124.2, C125.2, C60.2
Changed lines of the file:
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@@
 <part name="GND62" library="supply1" deviceset="GND" device=""/>
 <part name="GND82" library="supply1" deviceset="GND" device=""/>
-<part name="GND83" library="supply1" deviceset="GND" device=""/>
+<part name="NAME'" library="supply1" deviceset="GNDA" device=""/>
 <part name="GND84" library="supply1" deviceset="GND" device=""/>
 <part name="R139" library="rcl_custom" deviceset="R-US_" device="0402-B" value="100k"/>
@@
 <part name="C114" library="rcl_custom" deviceset="C-EU" device="0402-B" value="0.01uF"/>
 <part name="C115" library="rcl_custom" deviceset="C-EU" device="0603-B" value="1uF"/>
-<part name="GND88" library="supply1" deviceset="GND" device=""/>
+<part name="GND88" library="supply1" deviceset="GNDA" device=""/>
 <part name="D4" library="diode" deviceset="BAT54" device=""/>
 <part name="C116" library="rcl_custom" deviceset="C-EU" device="0402-B" value="0.047uF"/>
@@
 <part name="C117" library="rcl_custom" deviceset="C-EU" device="1206-B" value="10uF"/>
 <part name="C118" library="rcl_custom" deviceset="C-EU" device="1206-B" value="10uF"/>
-<part name="GND91" library="supply1" deviceset="GND" device=""/>
+<part name="GND91" library="supply1" deviceset="GNDA" device=""/>
 <part name="C119" library="rcl_custom" deviceset="C-EU" device="1206-B" value="10uF"/>
 <part name="C120" library="rcl_custom" deviceset="C-EU" device="1206-B" value="10uF"/>
-<part name="GND92" library="supply1" deviceset="GND" device=""/>
-<part name="GND93" library="supply1" deviceset="GND" device=""/>
+<part name="GND92" library="supply1" deviceset="GNDA" device=""/>
+<part name="GND93" library="supply1" deviceset="GNDA" device=""/>
 <part name="D5" library="RNH_SMAJ18CA" deviceset="SMAJ18CA" device=""/>
 <part name="GND94" library="supply1" deviceset="GND" device=""/>
@@
 <part name="C122" library="rcl_custom" deviceset="C-EU" device="0402-B" value="0.01uF"/>
 <part name="C123" library="rcl_custom" deviceset="C-EU" device="1206-B" value="10uF"/>
-<part name="GND96" library="supply1" deviceset="GND" device=""/>
+<part name="GND96" library="supply1" deviceset="GNDA" device=""/>
 <part name="C124" library="rcl_custom" deviceset="C-EU" device="0603-B" value="1uF"/>
 <part name="C125" library="rcl_custom" deviceset="C-EU" device="1206-B" value="10uF"/>
@@
 <instance part="GND62" gate="1" x="-38.1" y="27.94"/>
 <instance part="GND82" gate="1" x="-88.9" y="66.04"/>
-<instance part="GND83" gate="1" x="-111.76" y="35.56"/>
+<instance part="NAME'" gate="1" x="-111.76" y="33.02"/>
 <instance part="GND84" gate="1" x="-104.14" y="-2.54"/>
 <instance part="R139" gate="R" x="-27.94" y="2.54" rot="R90"/>
@@
 <instance part="C114" gate="CE" x="76.2" y="20.32"/>
 <instance part="C115" gate="CE" x="27.94" y="17.78" rot="R90"/>
-<instance part="GND88" gate="1" x="35.56" y="17.78" rot="R90"/>
+<instance part="GND88" gate="1" x="38.1" y="17.78" rot="R90"/>
 <instance part="D4" gate="G$1" x="22.86" y="12.7" rot="R270"/>
 <instance part="C116" gate="CE" x="22.86" y="0"/>
@@
 <instance part="Q7" gate="&gt;NAME" x="43.18" y="-10.16"/>
 <instance part="GND89" gate="1" x="48.26" y="-22.86"/>
-<instance part="GND90" gate="1" x="53.34" y="-43.18"/>
+<instance part="GND90" gate="1" x="53.34" y="-45.72"/>
 <instance part="R146" gate="R" x="86.36" y="-5.08"/>
 <instance part="C117" gate="CE" x="55.88" y="50.8"/>
@@
 </segment>
 <segment>
-<pinref part="C60" gate="CE" pin="2"/>
-<pinref part="GND83" gate="1" pin="GND"/>
-</segment>
-<segment>
 <pinref part="R138" gate="R" pin="1"/>
 <pinref part="GND84" gate="1" pin="GND"/>
@@
 </segment>
 <segment>
-<pinref part="C115" gate="CE" pin="2"/>
-<pinref part="GND88" gate="1" pin="GND"/>
-</segment>
-<segment>
 <pinref part="Q7" gate="&gt;NAME" pin="S"/>
 <pinref part="GND89" gate="1" pin="GND"/>
@@
 <pinref part="C112" gate="CE" pin="2"/>
 <pinref part="GND90" gate="1" pin="GND"/>
-</segment>
-<segment>
-<pinref part="C118" gate="CE" pin="2"/>
-<pinref part="GND91" gate="1" pin="GND"/>
-<wire x1="66.04" y1="40.64" x2="66.04" y2="43.18" width="0.1524" layer="91"/>
-<pinref part="C117" gate="CE" pin="2"/>
-<wire x1="66.04" y1="43.18" x2="66.04" y2="45.72" width="0.1524" layer="91"/>
-<wire x1="55.88" y1="45.72" x2="55.88" y2="43.18" width="0.1524" layer="91"/>
-<wire x1="55.88" y1="43.18" x2="66.04" y2="43.18" width="0.1524" layer="91"/>
-<junction x="66.04" y="43.18"/>
-</segment>
-<segment>
-<pinref part="C119" gate="CE" pin="2"/>
-<pinref part="GND92" gate="1" pin="GND"/>
-<wire x1="104.14" y1="-15.24" x2="104.14" y2="-12.7" width="0.1524" layer="91"/>
-</segment>
-<segment>
-<pinref part="C120" gate="CE" pin="2"/>
-<pinref part="GND93" gate="1" pin="GND"/>
-<wire x1="116.84" y1="-15.24" x2="116.84" y2="-12.7" width="0.1524" layer="91"/>
+<wire x1="53.34" y1="-43.18" x2="53.34" y2="-40.64" width="0.1524" layer="91"/>
 </segment>
 <segment>
@@
 <pinref part="GND95" gate="1" pin="GND"/>
 </segment>
-<segment>
-<pinref part="GND96" gate="1" pin="GND"/>
-<wire x1="2.54" y1="43.18" x2="2.54" y2="45.72" width="0.1524" layer="91"/>
-<pinref part="C123" gate="CE" pin="2"/>
-<wire x1="2.54" y1="45.72" x2="2.54" y2="48.26" width="0.1524" layer="91"/>
-<wire x1="-5.08" y1="48.26" x2="-5.08" y2="45.72" width="0.1524" layer="91"/>
-<wire x1="-5.08" y1="45.72" x2="2.54" y2="45.72" width="0.1524" layer="91"/>
-<junction x="2.54" y="45.72"/>
-<wire x1="10.16" y1="45.72" x2="2.54" y2="45.72" width="0.1524" layer="91"/>
-<pinref part="C124" gate="CE" pin="2"/>
-<wire x1="10.16" y1="48.26" x2="10.16" y2="45.72" width="0.1524" layer="91"/>
-<pinref part="C125" gate="CE" pin="2"/>
-</segment>
 </net>
 <net name="IOUT" class="0">
@@
 </segment>
 </net>
+<net name="GNDA" class="1">
+<segment>
+<pinref part="C60" gate="CE" pin="2"/>
+<pinref part="NAME'" gate="1" pin="GNDA"/>
+<wire x1="-111.76" y1="35.56" x2="-111.76" y2="38.1" width="0.1524" layer="91"/>
+</segment>
+<segment>
+<pinref part="GND96" gate="1" pin="GNDA"/>
+<wire x1="2.54" y1="43.18" x2="2.54" y2="45.72" width="0.1524" layer="91"/>
+<pinref part="C123" gate="CE" pin="2"/>
+<wire x1="2.54" y1="45.72" x2="2.54" y2="48.26" width="0.1524" layer="91"/>
+<wire x1="-5.08" y1="48.26" x2="-5.08" y2="45.72" width="0.1524" layer="91"/>
+<wire x1="-5.08" y1="45.72" x2="2.54" y2="45.72" width="0.1524" layer="91"/>
+<junction x="2.54" y="45.72"/>
+<wire x1="10.16" y1="45.72" x2="2.54" y2="45.72" width="0.1524" layer="91"/>
+<pinref part="C124" gate="CE" pin="2"/>
+<wire x1="10.16" y1="48.26" x2="10.16" y2="45.72" width="0.1524" layer="91"/>
+<pinref part="C125" gate="CE" pin="2"/>
+</segment>
+<segment>
+<pinref part="C119" gate="CE" pin="2"/>
+<pinref part="GND92" gate="1" pin="GNDA"/>
+<wire x1="104.14" y1="-15.24" x2="104.14" y2="-12.7" width="0.1524" layer="91"/>
+</segment>
+<segment>
+<pinref part="C120" gate="CE" pin="2"/>
+<pinref part="GND93" gate="1" pin="GNDA"/>
+<wire x1="116.84" y1="-15.24" x2="116.84" y2="-12.7" width="0.1524" layer="91"/>
+</segment>
+<segment>
+<pinref part="C115" gate="CE" pin="2"/>
+<pinref part="GND88" gate="1" pin="GNDA"/>
+<wire x1="35.56" y1="17.78" x2="33.02" y2="17.78" width="0.1524" layer="91"/>
+</segment>
+<segment>
+<pinref part="C118" gate="CE" pin="2"/>
+<pinref part="GND91" gate="1" pin="GNDA"/>
+<wire x1="66.04" y1="40.64" x2="66.04" y2="43.18" width="0.1524" layer="91"/>
+<pinref part="C117" gate="CE" pin="2"/>
+<wire x1="66.04" y1="43.18" x2="66.04" y2="45.72" width="0.1524" layer="91"/>
+<wire x1="55.88" y1="45.72" x2="55.88" y2="43.18" width="0.1524" layer="91"/>
+<wire x1="55.88" y1="43.18" x2="66.04" y2="43.18" width="0.1524" layer="91"/>
+<junction x="66.04" y="43.18"/>
+</segment>
+</net>

Commit message: Fixed some ERC issues; check Approved ERC for list of pending fixes
Connections:
- net BOOT1: now also R150.1
- net JTAG_TRST: now also R147.2
Changed lines of the file:
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@@
 <wire x1="10.16" y1="419.1" x2="0" y2="419.1" width="0.1524" layer="91"/>
 <label x="10.16" y="419.1" size="1.016" layer="95" xref="yes"/>
+<pinref part="R150" gate="G$1" pin="1"/>
+<junction x="-2.54" y="419.1"/>
 </segment>
 </net>
@@
 </segment>
 </net>
-<net name="NODE1_VOUT" class="0">
+<net name="NODE1_VOUT" class="1">
 <segment>
 <wire x1="78.74" y1="388.62" x2="81.28" y2="388.62" width="0.1524" layer="91"/>
@@
 </segment>
 </net>
-<net name="NODE2_VOUT" class="0">
+<net name="NODE2_VOUT" class="1">
 <segment>
 <wire x1="78.74" y1="256.54" x2="81.28" y2="256.54" width="0.1524" layer="91"/>
@@
 </segment>
 </net>
-<net name="NODE3_VOUT" class="0">
+<net name="NODE3_VOUT" class="1">
 <segment>
 <wire x1="78.74" y1="144.78" x2="81.28" y2="144.78" width="0.1524" layer="91"/>
@@
 </segment>
 </net>
-<net name="NODE8_VOUT" class="0">
+<net name="NODE8_VOUT" class="1">
 <segment>
 <wire x1="345.44" y1="386.08" x2="347.98" y2="386.08" width="0.1524" layer="91"/>
@@
 </segment>
 </net>
-<net name="NODE6_VOUT" class="0">
+<net name="NODE6_VOUT" class="1">
 <segment>
 <wire x1="345.44" y1="274.32" x2="347.98" y2="274.32" width="0.1524" layer="91"/>
@@
 </segment>
 </net>
-<net name="NODE7_VOUT" class="0">
+<net name="NODE7_VOUT" class="1">
 <segment>
 <wire x1="347.98" y1="157.48" x2="350.52" y2="157.48" width="0.1524" layer="91"/>
@@
 </segment>
 </net>
-<net name="VDD" class="0">
+<net name="VDD" class="1">
 <segment>
 <pinref part="R75" gate="G$1" pin="1"/>
@@
 </segment>
 </net>
-<net name="VDD" class="0">
+<net name="VDD" class="1">
 <segment>
 <pinref part="U$2" gate="G$1" pin="OUT"/>
@@
 </segment>
 </net>
-<net name="VDD" class="0">
+<net name="VDD" class="1">
 <segment>
 <pinref part="VDD2" gate="G$1" pin="VDD"/>
@@
 </segment>
 </net>
-<net name="VDDIO_IN" class="0">
+<net name="VDDIO_IN" class="1">
 <segment>
 <pinref part="U$14" gate="G$1" pin="VDD-IO2"/>
@@
 <net name="RST_N" class="0">
 <segment>
-<wire x1="27.94" y1="55.88" x2="33.02" y2="55.88" width="0.1524" layer="91"/>
-<pinref part="J11" gate="J" pin="10"/>
-<pinref part="R148" gate="G$1" pin="1"/>
-<wire x1="33.02" y1="55.88" x2="35.56" y2="55.88" width="0.1524" layer="91"/>
 <wire x1="33.02" y1="55.88" x2="33.02" y2="48.26" width="0.1524" layer="91"/>
-<junction x="33.02" y="55.88"/>
 <pinref part="R147" gate="G$1" pin="1"/>
 <wire x1="33.02" y1="48.26" x2="35.56" y2="48.26" width="0.1524" layer="91"/>
+<pinref part="J11" gate="J" pin="10"/>
+<wire x1="33.02" y1="55.88" x2="27.94" y2="55.88" width="0.1524" layer="91"/>
+<pinref part="R148" gate="G$1" pin="1"/>
+<wire x1="35.56" y1="55.88" x2="33.02" y2="55.88" width="0.1524" layer="91"/>
+<junction x="33.02" y="55.88"/>
 </segment>
 <segment>
@@
 </segment>
 </net>
-<net name="VDD" class="0">
+<net name="VDD" class="1">
 <segment>
 <pinref part="R100" gate="G$1" pin="1"/>
@@
 </segment>
 </net>
-<net name="BAT" class="0">
+<net name="BAT" class="1">
 <segment>
 <pinref part="J9" gate="G$1" pin="B+@4"/>
@@
 <net name="JTAG_TRST" class="0">
 <segment>
-<wire x1="48.26" y1="48.26" x2="45.72" y2="48.26" width="0.1524" layer="91"/>
 <label x="48.26" y="48.26" size="1.016" layer="95" xref="yes"/>
+<pinref part="R147" gate="G$1" pin="2"/>
+<wire x1="48.26" y1="48.26" x2="45.72" y2="48.26" width="0.1524" layer="91"/>
 </segment>
 </net>
@@
 </segment>
 </net>
-<net name="BAT" class="0">
+<net name="BAT" class="1">
 <segment>
 <pinref part="R143" gate="R" pin="2"/>
@@
 </sheet>
 </sheets>
+<errors>
+</errors>
 </schematic>
 </drawing>

Commit message: Replaced capacitive coupling with new ALT4532 magnetics
Parts:
- added C126, C127, C128, C129, C130, C131, C132: (no value), rcl:C-EUC0402
- added T10, T11, T12, T13, T14, T15, T16, T3, T4, T5, T6, T7, T8, T9: ALT4532, alt4532:ALT4532
Connections:
- net NODE6_RSV4 renamed N$119
- removed net N$119 (its old number): C55.1, J7.RX-@1, J7.RX-@2
- removed net N$124: C46.1, J6.TX-@1, J6.TX-@2
- removed net NODE6_TXP: C45.1, J6.TX+@1, J6.TX+@2
- removed net NODE8_TXP: C41.1, J8.TX+@1, J8.TX+@2
- new net N$169: J2.RX-@1, J2.RX-@2, T4.4
- new net N$170: C29.2, R79.1, R80.1
- new net N$171: C30.2, R81.1, R82.1
- new net N$172: C39.2, T4.3
- new net N$173: C126.2, T3.3
- new net N$174: C7.2
- new net N$175: C35.2
- new net N$176: C58.2, T6.3
- new net N$177: C127.2, T5.3
- new net N$178: J3.RX+@1, J3.RX+@2, T7.5
- new net N$179: C37.2
- new net N$180: C43.2, T7.3
- new net N$181: C128.2, T8.3
- new net N$182: C38.2
- new net N$184: C47.2, T9.3
- new net N$185: C129.2, T10.3
- new net N$186: J7.RX-@1, J7.RX-@2, T16.4
- new net N$187: J7.RX+@1, J7.RX+@2, T16.5
- new net N$188: J7.TX-@1, J7.TX-@2, T15.4
- new net N$189: J7.TX+@1, J7.TX+@2, T15.5
- new net N$191: C41.2
- new net N$192: C42.2
- new net N$193: C46.2, T12.3
- new net N$194: C48.2, T11.3
- new net N$195: C49.2
- new net N$196: C50.2
- new net N$197: C52.2, T14.3
- new net N$198: C53.2, T13.3
- new net N$199: C54.2
- new net N$200: C55.2
- new net N$201: C131.2, T16.3
- new net N$202: C132.2, T15.3
- net GND: now also C126.1, C127.1, C128.1, C129.1, C130.1, C131.1, C132.1, C29.1, C30.1, C33.1, C34.1, C35.1, C36.1, C37.1, C38.1, C39.1, C40.1, C41.1, C42.1, C43.1, C44.1, C45.1, C46.1, C47.1, C48.1, C49.1, C50.1, C51.1, C52.1, C53.1, C54.1, C55.1, C57.1, C58.1, C7.1
- net N$112: now also T6.5; no longer C7.1
- net N$118: now also T6.4; no longer C35.1
- net N$120: now also J8.RX-@2, T12.4; no longer C42.1, J8.TX-@1, J8.TX-@2
- net N$121: now also J8.RX+@1, J8.RX+@2, T12.5; no longer C54.1, J7.RX+@1, J7.RX+@2
- net N$122: now also J8.TX-@1, J8.TX-@2, T11.4; no longer C53.1, J6.RX-@1, J6.RX-@2
- net N$123: now also J8.TX+@1, J8.TX+@2, T11.5; no longer C52.1, J6.RX+@1, J6.RX+@2
- net N$125: now also J6.RX-@1, J6.RX-@2, T14.4; no longer C51.1, J8.RX-@1, J8.RX-@2
- net N$126: now also J6.RX+@1, J6.RX+@2, T14.5; no longer C48.1, J8.RX+@1, J8.RX+@2
- net N$127: now also J6.TX-@1, J6.TX-@2, T13.4; no longer C49.1, J7.TX+@1, J7.TX+@2
- net N$128: now also J6.TX+@1, J6.TX+@2, T13.5; no longer C50.1, J7.TX-@1, J7.TX-@2
- net N$129: now also T9.5; no longer C44.2
- net N$133: now also T9.4; no longer C47.2
- net N$134: now also J3.RX-@1, J3.RX-@2, T7.4; no longer C40.2, J3.RX+@1, J3.RX+@2
- net N$135: now also C34.2; no longer C43.2, J3.RX-@1, J3.RX-@2
- net N$136: now also J2.TX-@1, J2.TX-@2, T3.4; no longer C36.2, J2.RX+@1, J2.RX+@2
- net N$137: now also J2.RX+@1, J2.RX+@2, T4.5; no longer C39.2, J2.RX-@1, J2.RX-@2
- net N$23: now also T3.5; no longer C29.2
- net N$25: now also C33.2; no longer C30.2, J2.TX-@1, J2.TX-@2
- net N$33: now also T5.4; no longer C58.1
- net N$34: now also T5.5; no longer C57.1
- net N$35: now also T8.5; no longer C33.2
- net N$36: now also T8.4; no longer C34.2
- net N$39: now also T10.5; no longer C37.2
- net N$40: now also T10.4; no longer C38.2
- net RX1_N: now also R78.2, T6.2; no longer C58.2, R76.2
- net RX1_P: now also R77.2, T6.1; no longer C57.2, R75.2
- net RX2_N: now also T4.2; no longer C39.1
- net RX2_P: now also T4.1; no longer C36.1
- net RX3_N: now also R86.1, T7.2; no longer C34.1, R84.2
- net RX3_P: now also R85.1, T7.1; no longer C33.1, R83.2
- net RX4_N: now also T9.2; no longer C47.1
- net RX4_P: now also T9.1; no longer C44.1
- net RX6_N: now also T14.2; no longer C53.2
- net RX6_P: now also T14.1; no longer C52.2
- net RX7_N: now also T16.2; no longer C55.2
- net RX7_P: now also T16.1; no longer C54.2
- net RX8_N: now also T12.2; no longer C51.2
- net RX8_P: now also T12.1; no longer C48.2
- net TX1_N: now also R76.2, T5.2; no longer C35.2, R78.2
- net TX1_P: now also R75.2, T5.1; no longer C7.2, R77.2
- net TX2_N: now also T3.2; no longer C30.1
- net TX2_P: now also T3.1; no longer C29.1
- net TX3_N: now also R84.1, T8.2; no longer C43.1, R86.2
- net TX3_P: now also R83.1, T8.1; no longer C40.1, R85.2
- net TX4_N: now also T10.2; no longer C38.1
- net TX4_P: now also T10.1; no longer C37.1
- net TX6_N: now also T13.2; no longer C46.2
- net TX6_P: now also T13.1; no longer C45.2
- net TX7_N: now also T15.2; no longer C50.2
- net TX7_P: now also T15.1; no longer C49.2
- net TX8_N: now also T11.2; no longer C42.2
- net TX8_P: now also T11.1; no longer C41.2
- net VDD: now also C130.2, C36.2, C40.2, C44.2, C45.2, C51.2, C57.2, T10.6, T11.6, T12.6, T13.6, T14.6, T15.6, T16.6, T3.6, T4.6, T5.6, T6.6, T7.6, T8.6, T9.6; no longer R103.1, R104.1, R105.1, R106.1, R75.1, R76.1, R77.1, R78.1, R79.1, R80.1, R81.1, R82.1, R83.1, R84.1, R85.1, R86.1, R87.1, R88.1, R89.1, R90.1, R91.1, R92.1, R93.1, R94.1, R95.1, R96.1, R97.1, R98.1
Other:
- moved on the sheet: C101, C29, C30, C33, C34, C35, C36, C37, C38, C39, C40, C41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
