File: av3/rocketnet-hub/eagle/mcu_page_combined_routed.brd (EAGLE design)
At the start: 112.7 x 76.3 mm, 444 parts, among them J1 ROCKETNET-CONNECTOR-16M, J10 UART Header, J12 BOOT1 Jumper, J13 PGOOD Jumper, J14 ROCKETNET-UMBILICAL-18, J15 Auxiliary Header, J16 Auxiliary Header, J17 Auxiliary Header, J18 Auxiliary Header, J19 Auxiliary Header, J2 ROCKETNET-CONNECTOR-16M, J20 Auxiliary Header, J21 Auxiliary Header, J22 Debug Header, J3 ROCKETNET-CONNECTOR-16M, J4 ROCKETNET-CONNECTOR-16M, J5 BOOT0 Jumper, J6 ROCKETNET-CONNECTOR-16M, J7 ROCKETNET-CONNECTOR-16M, J8 ROCKETNET-CONNECTOR-16M, J9 ROCKETNET-BATTERY-14, Q2 FDS6680ASOIC8, Q3 FDS6680ASOIC8, Q4 FDS6680ASOIC8, Q5 SIS412DNSOP-8, Q6 BSS138W-7-F, Q7 SIS412DNSOP-8, T1 BSS84, T10 ALT4532, T11 ALT4532, T12 ALT4532, T13 ALT4532, T14 ALT4532, T15 ALT4532, T16 ALT4532, T17 ALT4532, T18 ALT4532, T19 BSS84, T2 NDS335N, T20 NDS335N, T3 ALT4532, T4 ALT4532, T5 ALT4532, T6 ALT4532, T7 ALT4532, T8 ALT4532, T9 ALT4532, U1 STM32F407V100-PIN_QFP, U10 TPS2420QFN-16, U11 TPS2420QFN-16, U12 TPS2420QFN-16, U13 TPS2420QFN-16, U14 MAX4734ETC+, U15 MAX4734ETC+, U2 BQ24725QFN-20, U3 SN65220DBV, U4 KS8999, U5 LTM8023, U6 MIC37101-2.1YM, U7 TPS2420QFN-16, U8 TPS2420QFN-16, U9 TPS2420QFN-16

Commit message: Started fixing autorouter nets
Parts:
- moved R116 1.14 mm to (106.0, 52.3)
- moved C10 1.08 mm to (58.7, 54.7)
- moved C29 0.13 mm to (82.5, 60.9), turned to 0 degrees
- moved R150 0.13 mm to (43.2, 25.0)
Routing:
- net +3V3: track 415.8 -> 404.9 mm
- net +2V2: track 10.2 -> 0.00 mm, vias 8 -> 0
- net +2V1: track 172.4 -> 167.4 mm, vias 49 -> 52
- net NODE1_LTCH: track 4.55 -> 0.00 mm, vias 1 -> 0
- net N$85: track 0.00 -> 4.26 mm, vias 0 -> 1
- net N$91: track 4.28 -> 8.14 mm
- net N$249: track 3.43 -> 0.00 mm, vias 1 -> 0
- net NODE3_LTCH: track 3.36 -> 0.00 mm, vias 1 -> 0
- net NODE2_LTCH: track 3.34 -> 0.00 mm, vias 1 -> 0
- net NODE7_LTCH: track 3.27 -> 0.00 mm, vias 1 -> 0
- net NODE6_LTCH: track 2.43 -> 0.00 mm, vias 1 -> 0
- net N$212: track 17.6 -> 20.0 mm
- net N$217: track 17.6 -> 19.9 mm
- net N$99: track 3.77 -> 6.06 mm
- net NODE5_LTCH: track 2.20 -> 0.00 mm, vias 1 -> 0
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
Commit message: routed and cleaned up new version of brd.
Routing:
- net +3V3: track 404.9 -> 259.8 mm, vias 60 -> 72
- net N$101: track 110.0 -> 106.0 mm
- net NODE1_LTCH: track 0.00 -> 3.58 mm, vias 0 -> 1
- net NODE3_LTCH: track 0.00 -> 2.91 mm, vias 0 -> 1
- net N$249: track 0.00 -> 2.86 mm, vias 0 -> 1
- net NODE2_LTCH: track 0.00 -> 2.84 mm, vias 0 -> 1
- net NODE1_!FLT: track 70.3 -> 71.7 mm
- net N$168: track 19.5 -> 20.5 mm
- net NODE4_!FLT: track 79.3 -> 78.5 mm

Commit message: Fixed missing airwires, added +3v3 fill on bottom board
Parts:
- moved TP34 1.69 mm to (35.8, 15.2)
- moved TP35 1.33 mm to (58.7, 15.2)
- moved TP33 1.09 mm to (81.7, 15.2)
- moved C69 0.51 mm to (99.2, 20.4)
Routing:
- net +3V3: track 259.8 -> 265.7 mm, vias 72 -> 86
- net NODE6_LTCH: track 0.00 -> 3.15 mm, vias 0 -> 1
- net NODE7_LTCH: track 0.00 -> 3.10 mm, vias 0 -> 1
- net NODE4_!FLT: track 78.5 -> 81.6 mm, vias 3 -> 4
- net NODE5_LTCH: track 0.00 -> 3.07 mm, vias 0 -> 1
- net GND: track 253.1 -> 255.0 mm, vias 115 -> 114
- net NODE3_!FLT: track 62.2 -> 63.7 mm
- net ETH_EN: track 77.6 -> 76.7 mm
- net NODE3_!EN: track 50.6 -> 51.4 mm
- net N$185: track 1.67 -> 2.33 mm
- net N$83: track 2.55 -> 3.16 mm
- net +2V1: track 167.4 -> 167.9 mm

Commit message: Added a 1x3 50mil header for I2C interface, added 10k pulldown on U15 pin N1, fixed +3v3 nets on bottom area of the board
Parts:
- added J11: I2C Header, headers:1.27MM_3X1
- added R18: 10k, rcl_custom:0402-B-NOSILK
- moved T1 0.25 mm to (104.9, 19.1)
Connections:
- new net N$32: R18.2, U15.1
- net GND: now also J11.3, R18.1
- net SCL: now also J11.1
- net SDA: now also J11.2
Routing:
- net +3V3: track 265.7 -> 144.4 mm, vias 86 -> 87
- net N$100: track 82.3 -> 81.4 mm, vias 3 -> 2
- net VDDIO_IN: track 43.5 -> 42.8 mm

Commit message: Fixed more routing
Parts:
- moved R44 17.5 mm to (42.6, 28.7)
- moved LED37 16.3 mm to (41.5, 29.6)
- moved R46 16.2 mm to (41.6, 30.7), turned to 180 degrees
- moved R45 15.4 mm to (40.7, 28.7), turned to 180 degrees
- moved J11 8.07 mm to (30.2, 42.7), turned to 180 degrees
- moved R168 4.09 mm to (34.2, 48.3), turned to 180 degrees
- moved J22 2.87 mm to (33.7, 43.8)
- moved TP38 2.84 mm to (33.7, 40.7)
- moved C2 1.94 mm to (41.2, 33.3), turned to 45 degrees
- moved R17 1.73 mm to (41.6, 43.8)
- moved J12 1.45 mm to (42.8, 26.2)
- moved J5 1.45 mm to (40.1, 26.2)
- moved R150 0.97 mm to (42.8, 24.2)
- moved R64 0.97 mm to (40.1, 24.2)
- moved R18 0.64 mm to (51.2, 20.8)
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Routing:
- net RST_N: track 18.8 -> 37.2 mm
- net NODE1_!EN: track 90.4 -> 77.7 mm
- net ROCKET_RDY_MCU: track 69.5 -> 57.5 mm
- net SCL: track 61.3 -> 49.8 mm, vias 4 -> 2
- net NODE3_!EN: track 51.4 -> 58.9 mm, vias 3 -> 2
- net N$74: track 31.7 -> 24.2 mm, vias 4 -> 3
- net N$91: track 8.14 -> 1.78 mm
- net N$66: track 40.8 -> 34.7 mm
- net N$99: track 6.06 -> 1.70 mm
- net N$206: track 5.47 -> 1.32 mm, vias 1 -> 0
- net JTAG_TMS: track 17.5 -> 21.5 mm
- net +3V3: track 144.4 -> 148.3 mm, vias 87 -> 88
- net GND: track 255.0 -> 258.8 mm, vias 114 -> 115
- net JTAG_TDI: track 14.0 -> 17.8 mm
- net SPI3_SCK: track 65.0 -> 68.6 mm, vias 4 -> 3
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
Commit message: Changed routed traces on GND layer to a different layer
Routing:
- net N$41: track 58.5 -> 61.2 mm
- net N$100: track 81.4 -> 79.1 mm
Changed lines of the file:
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@@
 <layers>
 <layer number="1" name="Top" color="4" fill="1" visible="yes" active="yes"/>
-<layer number="2" name="GND" color="1" fill="6" visible="no" active="yes"/>
+<layer number="2" name="GND" color="9" fill="1" visible="yes" active="yes"/>
 <layer number="3" name="Power" color="12" fill="1" visible="no" active="yes"/>
 <layer number="14" name="NS" color="11" fill="1" visible="yes" active="yes"/>
@@
 <wire x1="49.251" y1="29.572825" x2="48.430221875" y2="28.752046875" width="0.127" layer="1"/>
 <wire x1="106.045" y1="33.955" x2="105.329" y2="34.798" width="0.127" layer="16"/>
-<wire x1="105.329" y1="34.798" x2="105.283" y2="34.925" width="0.127" layer="16"/>
-<via x="105.283" y="34.925" extent="1-16" drill="0.2032" diameter="0.4572"/>
-<wire x1="105.283" y1="34.925" x2="105.208" y2="34.85" width="0.127" layer="1"/>
+<wire x1="105.329" y1="34.798" x2="105.283" y2="34.798" width="0.127" layer="16"/>
+<via x="105.283" y="34.798" extent="1-16" drill="0.2032" diameter="0.4572"/>
+<wire x1="105.283" y1="34.798" x2="105.208" y2="34.85" width="0.127" layer="1"/>
 <wire x1="105.208" y1="34.85" x2="106.5" y2="34.85" width="0.127" layer="1"/>
 </signal>
@@
 <contactref element="U4" pad="115"/>
 <contactref element="LED5" pad="C"/>
-<wire x1="104.14" y1="31.75" x2="96.266" y2="39.624" width="0.127" layer="2"/>
 <wire x1="62.103" y1="62.484" x2="61.341" y2="62.484" width="0.1778" layer="1"/>
 <wire x1="63.373" y1="61.722" x2="62.103" y2="62.484" width="0.1778" layer="14"/>
@@
 <wire x1="83.82" y1="50.419" x2="74.676" y2="50.419" width="0.1778" layer="14"/>
 <wire x1="94.615" y1="39.624" x2="83.82" y2="50.419" width="0.1778" layer="14"/>
-<wire x1="96.266" y1="39.624" x2="94.615" y2="39.624" width="0.1778" layer="14"/>
+<wire x1="100.965" y1="39.624" x2="94.615" y2="39.624" width="0.1778" layer="14"/>
 <wire x1="61.341" y1="62.484" x2="61.25" y2="62.5" width="0.1778" layer="1"/>
 <wire x1="105.537" y1="30.353" x2="106.426" y2="30.353" width="0.1778" layer="1"/>
@@
 <wire x1="106.426" y1="30.353" x2="106.5" y2="30.35" width="0.1778" layer="1"/>
 <via x="62.103" y="62.484" extent="1-16" drill="0.2032" diameter="0.4572"/>
-<via x="96.266" y="39.624" extent="1-16" drill="0.2032" diameter="0.4572"/>
+<via x="100.965" y="39.624" extent="1-16" drill="0.2032" diameter="0.4572"/>
 <via x="104.14" y="31.75" extent="1-16" drill="0.2032" diameter="0.4572"/>
+<wire x1="100.965" y1="39.624" x2="100.965" y2="34.925" width="0.1778" layer="15"/>
+<wire x1="100.965" y1="34.925" x2="104.14" y2="31.75" width="0.1778" layer="15"/>
 </signal>
 <signal name="N$43">
@@
 <contactref element="U4" pad="127"/>
 <contactref element="LED9" pad="C"/>
-<wire x1="101.473" y1="37.338" x2="99.822" y2="38.989" width="0.127" layer="2"/>
 <wire x1="39.243" y1="62.484" x2="38.354" y2="62.484" width="0.1778" layer="1"/>
 <wire x1="48.006" y1="62.484" x2="39.243" y2="62.484" width="0.1778" layer="14"/>
@@
 <wire x1="83.693" y1="50.038" x2="60.452" y2="50.038" width="0.1778" layer="14"/>
 <wire x1="94.742" y1="38.989" x2="83.693" y2="50.038" width="0.1778" layer="14"/>
-<wire x1="99.822" y1="38.989" x2="94.742" y2="38.989" width="0.1778" layer="14"/>
+<wire x1="99.06" y1="38.989" x2="94.742" y2="38.989" width="0.1778" layer="14"/>
 <wire x1="38.354" y1="62.484" x2="38.25" y2="62.5" width="0.1778" layer="1"/>
 <via x="39.243" y="62.484" extent="1-16" drill="0.2032" diameter="0.4572"/>
-<via x="99.822" y="38.989" extent="1-16" drill="0.2032" diameter="0.4572"/>
-<wire x1="99.822" y1="38.989" x2="99.949" y2="38.989" width="0.1778" layer="1"/>
-<wire x1="99.949" y1="38.989" x2="102.588" y2="36.35" width="0.1778" layer="1"/>
-<wire x1="102.588" y1="36.35" x2="106.5" y2="36.35" width="0.1778" layer="1"/>
+<via x="99.06" y="38.989" extent="1-16" drill="0.2032" diameter="0.4572"/>
+<wire x1="99.06" y1="38.989" x2="99.314" y2="38.735" width="0.1778" layer="1"/>
+<wire x1="99.314" y1="38.735" x2="101.572" y2="36.35" width="0.1778" layer="1"/>
+<wire x1="101.572" y1="36.35" x2="106.5" y2="36.35" width="0.1778" layer="1"/>
 </signal>
 <signal name="N$101">
@@
 <wire x1="96.012" y1="25.527" x2="68.199" y2="25.527" width="0.1778" layer="14"/>
 <wire x1="101.981" y1="31.496" x2="96.012" y2="25.527" width="0.1778" layer="14"/>
-<wire x1="101.981" y1="37.719" x2="101.981" y2="31.496" width="0.1778" layer="14"/>
-<wire x1="104.775" y1="40.513" x2="101.981" y2="37.719" width="0.1778" layer="1"/>
-<wire x1="104.775" y1="40.64" x2="104.775" y2="40.513" width="0.1778" layer="1"/>
-<wire x1="105.537" y1="41.402" x2="104.775" y2="40.64" width="0.1778" layer="1"/>
+<wire x1="101.981" y1="37.846" x2="101.981" y2="31.496" width="0.1778" layer="14"/>
+<wire x1="105.537" y1="41.402" x2="101.981" y2="37.846" width="0.1778" layer="1"/>
 <wire x1="106.426" y1="41.402" x2="105.537" y2="41.402" width="0.1778" layer="1"/>
 <wire x1="27.305" y1="8.382" x2="27.25" y2="8.5" width="0.1778" layer="1"/>
 <wire x1="106.426" y1="41.402" x2="106.5" y2="41.35" width="0.1778" layer="1"/>
 <via x="28.829" y="8.382" extent="1-16" drill="0.2032" diameter="0.4572"/>
-<via x="101.981" y="37.719" extent="1-16" drill="0.2032" diameter="0.4572"/>
+<via x="101.981" y="37.846" extent="1-16" drill="0.2032" diameter="0.4572"/>
 <wire x1="30.607" y1="6.604" x2="28.829" y2="8.382" width="0.1778" layer="14"/>
 </signal>
@@
 <wire x1="98.171" y1="20.955" x2="92.71" y2="20.955" width="0.1778" layer="14"/>
 <wire x1="103.378" y1="26.162" x2="98.171" y2="20.955" width="0.1778" layer="14"/>
-<wire x1="103.378" y1="34.417" x2="103.378" y2="26.162" width="0.1778" layer="14"/>
-<wire x1="106.045" y1="37.084" x2="103.378" y2="34.417" width="0.1778" layer="14"/>
-<wire x1="106.045" y1="42.037" x2="106.045" y2="37.084" width="0.1778" layer="14"/>
+<wire x1="103.378" y1="34.798" x2="103.378" y2="26.162" width="0.1778" layer="14"/>
+<wire x1="106.045" y1="37.465" x2="103.378" y2="34.798" width="0.1778" layer="14"/>
+<wire x1="106.045" y1="42.037" x2="106.045" y2="37.465" width="0.1778" layer="14"/>
 <wire x1="104.267" y1="43.815" x2="106.045" y2="42.037" width="0.1778" layer="14"/>
 <wire x1="105.791" y1="45.339" x2="104.267" y2="43.815" width="0.1778" layer="1"/>

Commit message: Updated pin 189 on KS8999
Connections:
- net GND: now also U4.189
Changed lines of the file:
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@@
 <wire x1="67.31" y1="47.879" x2="67.183" y2="48.006" width="0.1778" layer="16"/>
 <wire x1="67.183" y1="48.006" x2="66.294" y2="48.006" width="0.1778" layer="16"/>
+<contactref element="U4" pad="189"/>
 </signal>
 <signal name="+3V3" class="1">

Commit message: battery charger routing clean up
Parts:
- moved C94 1.66 mm to (31.3, 23.1)
- moved C113 0.66 mm to (20.8, 27.3), turned to 180 degrees
- moved R135 0.64 mm to (27.7, 23.0)
- moved R137 0.15 mm to (27.1, 37.4)
Routing:
- net NODE4_!EN: track 62.2 -> 48.1 mm
- net N$115: track 15.4 -> 8.09 mm
- net +3V3: track 148.3 -> 141.0 mm
- net VIN: track 9.54 -> 4.39 mm
- net N$146: track 31.7 -> 29.1 mm
- net SCL: track 49.8 -> 52.2 mm
- net GND: track 258.8 -> 256.9 mm
- net N$162: track 9.77 -> 7.97 mm
- net +18V: track 36.2 -> 34.9 mm
- net N$163: track 11.6 -> 12.8 mm
- net GNDA: track 1.12 -> 0.00 mm, vias 19 -> 20
- net N$153: track 30.8 -> 30.2 mm
- added copper zone on layer 16, net N$115
- added copper zone on layer 16, net N$138
- added copper zone on layer 1, net N$162
