File: av3/rocketnet-hub/eagle/mcu_page_combined_routed.brd (EAGLE design)
At the start: 112.7 x 76.3 mm, 446 parts, among them J1 ROCKETNET-CONNECTOR-16M, J10 UART Header, J11 I2C Header, J12 BOOT1 Jumper, J13 PGOOD Jumper, J14 ROCKETNET-UMBILICAL-18, J15 Auxiliary Header, J16 Auxiliary Header, J17 Auxiliary Header, J18 Auxiliary Header, J19 Auxiliary Header, J2 ROCKETNET-CONNECTOR-16M, J20 Auxiliary Header, J21 Auxiliary Header, J22 Debug Header, J3 ROCKETNET-CONNECTOR-16M, J4 ROCKETNET-CONNECTOR-16M, J5 BOOT0 Jumper, J6 ROCKETNET-CONNECTOR-16M, J7 ROCKETNET-CONNECTOR-16M, J8 ROCKETNET-CONNECTOR-16M, J9 ROCKETNET-BATTERY-14, Q2 FDS6680ASOIC8, Q3 FDS6680ASOIC8, Q4 FDS6680ASOIC8, Q5 SIS412DNSOP-8, Q6 BSS138W-7-F, Q7 SIS412DNSOP-8, T1 BSS84, T10 ALT4532, T11 ALT4532, T12 ALT4532, T13 ALT4532, T14 ALT4532, T15 ALT4532, T16 ALT4532, T17 ALT4532, T18 ALT4532, T19 BSS84, T2 NDS335N, T20 NDS335N, T3 ALT4532, T4 ALT4532, T5 ALT4532, T6 ALT4532, T7 ALT4532, T8 ALT4532, T9 ALT4532, U1 STM32F407V100-PIN_QFP, U10 TPS2420QFN-16, U11 TPS2420QFN-16, U12 TPS2420QFN-16, U13 TPS2420QFN-16, U14 MAX4734ETC+, U15 MAX4734ETC+, U2 BQ24725QFN-20, U3 SN65220DBV, U4 KS8999, U5 LTM8023, U6 MIC37101-2.1YM, U7 TPS2420QFN-16, U8 TPS2420QFN-16, U9 TPS2420QFN-16

Commit message: fixed rout
Routing:
- net TX8_P: track 12.0 -> 11.2 mm
- net TX7_P: track 22.6 -> 21.8 mm
- net RX5_P: track 73.9 -> 73.2 mm
- net RX6_N: track 40.9 -> 40.4 mm
- net RX6_P: track 41.6 -> 41.1 mm
- net RX7_P: track 24.6 -> 24.1 mm
- net TX6_P: track 45.4 -> 44.8 mm
- net TX7_N: track 22.3 -> 21.8 mm
- net RX5_N: track 72.9 -> 72.3 mm

Commit message: battery charger: routing and clean up, attached 18v on top
Parts:
- moved C60 5.52 mm to (11.5, 20.9), turned to 90 degrees
- moved C118 1.89 mm to (8.38, 25.7)
- moved C117 1.71 mm to (10.9, 25.7)
Routing:
- net +18V: track 34.9 -> 24.8 mm
- net GND: track 256.8 -> 255.3 mm
- net +3V3: track 141.0 -> 141.8 mm
- net N$166: track 9.86 -> 9.32 mm
- net N$146: track 29.1 -> 29.2 mm, vias 4 -> 3
- net N$153: vias 3 -> 2

Commit message: fixed routing
Parts:
- moved R38 71.0 mm to (38.8, 34.0), turned to 90 degrees
- moved LED33 69.6 mm to (40.6, 33.1), turned to 270 degrees
Routing:
- net N$106: track 4.09 -> 90.3 mm, vias 0 -> 4
- net +3V3: track 141.8 -> 146.1 mm, vias 88 -> 89
- net NODE2_IMON_IN: track 39.5 -> 43.3 mm
- net NODE4_IMON_IN: track 36.9 -> 40.5 mm
- net NODE4_!FLT: track 81.6 -> 83.7 mm
- net N$217: track 19.9 -> 18.4 mm
- net GND: track 255.3 -> 254.2 mm
- net +18V: vias 30 -> 89

Commit message: fixed all drc issues
Parts:
- moved TP34 0.28 mm to (35.9, 15.5)
- moved R64 0.28 mm to (40.1, 23.9)
- moved R150 0.28 mm to (42.8, 23.9)
Routing:
- net VDDIO_IN: track 42.8 -> 44.5 mm
- net NODE4_IMON_IN: track 40.5 -> 42.2 mm
- net +3V3: track 146.1 -> 146.7 mm
- net GND: track 254.2 -> 254.7 mm

Commit message: fixed thermal creation in poly's
Routing:
- net GND: track 254.7 -> 254.8 mm, vias 115 -> 116
- net +18V: vias 89 -> 87
Changed lines of the file:
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@@
 <setting verticaltext="up"/>
 </settings>
-<grid distance="5" unitdist="mil" unit="mil" style="lines" multiple="1" display="yes" altdistance="0.1" altunitdist="mil" altunit="mil"/>
+<grid distance="5" unitdist="mil" unit="mil" style="lines" multiple="1" display="yes" altdistance="1" altunitdist="mil" altunit="mil"/>
 <layers>
 <layer number="1" name="Top" color="4" fill="1" visible="yes" active="yes"/>
 <layer number="2" name="GND" color="9" fill="1" visible="no" active="yes"/>
 <layer number="3" name="Power" color="12" fill="1" visible="no" active="yes"/>
-<layer number="14" name="NS" color="11" fill="1" visible="yes" active="yes"/>
-<layer number="15" name="EW" color="6" fill="1" visible="yes" active="yes"/>
+<layer number="14" name="NS" color="11" fill="1" visible="no" active="yes"/>
+<layer number="15" name="EW" color="6" fill="1" visible="no" active="yes"/>
 <layer number="16" name="Bottom" color="1" fill="1" visible="yes" active="yes"/>
 <layer number="17" name="Pads" color="2" fill="1" visible="yes" active="yes"/>
@@
 <via x="11" y="50.8" extent="1-16" drill="0.2032" diameter="0.4572"/>
 <wire x1="11" y1="50.8" x2="11.1" y2="50.9" width="0.127" layer="2"/>
-<polygon width="0.127" layer="16">
-<vertex x="30.8" y="64.3"/>
-<vertex x="35.9" y="64.3"/>
-<vertex x="35.9" y="61.4"/>
-<vertex x="30.8" y="61.4"/>
-</polygon>
-<polygon width="0.127" layer="16">
-<vertex x="76.8" y="64.3"/>
-<vertex x="81.9" y="64.3"/>
-<vertex x="81.9" y="61.8"/>
-<vertex x="76.8" y="61.8"/>
-</polygon>
-<polygon width="0.127" layer="16">
-<vertex x="99.8" y="64.3"/>
-<vertex x="104.3" y="64.3"/>
-<vertex x="104.3" y="61.4"/>
-<vertex x="99.8" y="61.4"/>
-</polygon>
-<polygon width="0.127" layer="16">
-<vertex x="52.3" y="15.1"/>
-<vertex x="57.2" y="15.1"/>
-<vertex x="57.2" y="12.2"/>
-<vertex x="52.3" y="12.2"/>
-</polygon>
-<polygon width="0.127" layer="16">
-<vertex x="75.3" y="15.1"/>
-<vertex x="80.2" y="15.1"/>
-<vertex x="80.2" y="12.2"/>
-<vertex x="75.3" y="12.2"/>
-</polygon>
-<polygon width="0.127" layer="16">
-<vertex x="29.3" y="15.1"/>
-<vertex x="34.2" y="15.1"/>
-<vertex x="34.2" y="12.2"/>
-<vertex x="29.3" y="12.2"/>
-</polygon>
-<polygon width="0.127" layer="16">
-<vertex x="53.8" y="64.3"/>
-<vertex x="58.9" y="64.3"/>
-<vertex x="58.9" y="61.4"/>
-<vertex x="53.8" y="61.4"/>
+<polygon width="0.127" layer="16" thermals="no">
+<vertex x="30.8" y="63.051"/>
+<vertex x="30.8" y="65.151"/>
+<vertex x="31.2928" y="65.151"/>
+<vertex x="31.2928" y="64.389"/>
+<vertex x="34.036" y="64.389"/>
+<vertex x="34.122" y="64.3"/>
+<vertex x="34.122" y="63.051"/>
+</polygon>
+<polygon width="0.127" layer="16" thermals="no">
+<vertex x="76.8" y="63.07"/>
+<vertex x="76.8" y="65.151"/>
+<vertex x="77.343" y="65.151"/>
+<vertex x="77.343" y="64.389"/>
+<vertex x="80.137" y="64.389"/>
+<vertex x="80.122" y="63.07"/>
+</polygon>
+<polygon width="0.127" layer="16" thermals="no">
+<vertex x="99.8" y="62.797"/>
+<vertex x="99.8" y="65.024"/>
+<vertex x="100.33" y="65.024"/>
+<vertex x="100.33" y="64.389"/>
+<vertex x="103.284" y="64.389"/>
+<vertex x="103.284" y="62.797"/>
+</polygon>
+<polygon width="0.127" layer="16" thermals="no">
+<vertex x="53.824" y="13.703"/>
+<vertex x="57.2" y="13.703"/>
+<vertex x="57.2" y="11.734"/>
+<vertex x="57.15" y="11.684"/>
+<vertex x="56.7182" y="11.6586"/>
+<vertex x="56.7182" y="12.192"/>
+<vertex x="53.824" y="12.192"/>
+</polygon>
+<polygon width="0.127" layer="16" thermals="no">
+<vertex x="76.697" y="13.703"/>
+<vertex x="80.2" y="13.703"/>
+<vertex x="80.2" y="11.747"/>
+<vertex x="80.137" y="11.684"/>
+<vertex x="79.7052" y="11.684"/>
+<vertex x="79.7052" y="12.192"/>
+<vertex x="76.697" y="12.2"/>
+</polygon>
+<polygon width="0.127" layer="16" thermals="no">
+<vertex x="30.824" y="13.576"/>
+<vertex x="34.2" y="13.576"/>
+<vertex x="34.2" y="11.557"/>
+<vertex x="33.7058" y="11.557"/>
+<vertex x="33.7058" y="12.192"/>
+<vertex x="30.861" y="12.192"/>
+<vertex x="30.824" y="12.2"/>
+</polygon>
+<polygon width="0.127" layer="16" thermals="no">
+<vertex x="54.3052" y="65.141"/>
+<vertex x="54.3052" y="64.389"/>
+<vertex x="57.023" y="64.389"/>
+<vertex x="57.023" y="62.611"/>
+<vertex x="53.721" y="62.611"/>
+<vertex x="53.721" y="65.151"/>
 </polygon>
 <wire x1="47.879" y1="30.988" x2="48.006" y2="31.115" width="0.127" layer="2"/>
@@
 <wire x1="94.742" y1="49.657" x2="96.52" y2="49.657" width="0.1778" layer="16"/>
 <wire x1="96.52" y1="49.657" x2="96.5" y2="49.7" width="0.1778" layer="16"/>
-<wire x1="80.01" y1="11.811" x2="79.629" y2="12.192" width="0.1778" layer="16"/>
-<wire x1="79.629" y1="12.192" x2="79.6341" y2="12.215896875" width="0.1778" layer="16"/>
-<wire x1="80.01" y1="11.811" x2="79.9" y2="11.75" width="0.1778" layer="16"/>
 <wire x1="48.895" y1="33.147" x2="49.022" y2="33.274" width="0.1778" layer="16"/>
 <wire x1="96.139" y1="58.039" x2="96.139" y2="57.531" width="0.1778" layer="16"/>
@@
 <wire x1="76.962" y1="64.262" x2="76.975" y2="63.925" width="0.1778" layer="16"/>
 <wire x1="77.089" y1="64.77" x2="77.1" y2="64.8" width="0.1778" layer="16"/>
-<wire x1="57.023" y1="11.811" x2="56.642" y2="12.192" width="0.1778" layer="16"/>
-<wire x1="56.642" y1="12.192" x2="56.6341" y2="12.215896875" width="0.1778" layer="16"/>
 <wire x1="57.023" y1="11.811" x2="56.9" y2="11.75" width="0.1778" layer="16"/>
 <wire x1="30.988" y1="64.77" x2="30.988" y2="64.262" width="0.1778" layer="16"/>
@@
 <wire x1="20.5" y1="61.161" x2="21.336" y2="60.325" width="0.1778" layer="16"/>
 <via x="21.336" y="60.325" extent="1-16" drill="0.2032" diameter="0.4572"/>
-<wire x1="78.92" y1="61" x2="78.92" y2="62.537" width="0.1778" layer="16"/>
-<wire x1="78.92" y1="62.537" x2="78.994" y2="62.611" width="0.1778" layer="16"/>
 <wire x1="68.199" y1="42.418" x2="67.691" y2="42.418" width="0.1778" layer="16"/>
 <wire x1="67.691" y1="42.418" x2="66.929" y2="43.18" width="0.1778" layer="16"/>
@@
 </polygon>
 <wire x1="104.013" y1="26.162" x2="104.013" y2="25.908" width="0.1778" layer="16"/>
+<wire x1="78.92" y1="61" x2="78.92" y2="63.31" width="0.254" layer="16"/>
+<wire x1="78.92" y1="63.31" x2="79.4" y2="63.79" width="0.254" layer="16"/>
+<via x="77.343" y="15.1" extent="1-16" drill="0.2032" diameter="0.2032"/>
 </signal>
 <signal name="+3V3" class="1">
@@
 <contactref element="U11" pad="16"/>
 <contactref element="R109" pad="1"/>
-<wire x1="33.909" y1="8.128" x2="33.655" y2="7.874" width="0.1778" layer="16"/>
-<wire x1="33.655" y1="7.874" x2="32.893" y2="7.112" width="0.1778" layer="16"/>
-<wire x1="33.909" y1="8.636" x2="33.909" y2="8.128" width="0.1778" layer="16"/>
+<wire x1="34.036" y1="8.128" x2="33.782" y2="7.747" width="0.1778" layer="16"/>
+<wire x1="33.782" y1="7.747" x2="32.893" y2="7.112" width="0.1778" layer="16"/>
+<wire x1="34.036" y1="8.636" x2="34.036" y2="8.128" width="0.1778" layer="16"/>
 <wire x1="32.893" y1="7.112" x2="32.8" y2="7.08" width="0.1778" layer="16"/>
-<wire x1="33.909" y1="8.636" x2="34.025" y2="8.675" width="0.1778" layer="16"/>
+<wire x1="34.036" y1="8.636" x2="34.025" y2="8.675" width="0.1778" layer="16"/>
 <wire x1="40.64" y1="29.591" x2="40.64" y2="35.179" width="0.1778" layer="14"/>
 <wire x1="34.925" y1="23.876" x2="40.64" y2="29.591" width="0.1778" layer="14"/>
@@
 <wire x1="32.639" y1="8.89" x2="32.639" y2="13.335" width="0.1778" layer="14"/>
 <wire x1="33.782" y1="7.747" x2="32.639" y2="8.89" width="0.1778" layer="14"/>
-<wire x1="33.655" y1="7.874" x2="33.782" y2="7.747" width="0.1778" layer="16"/>
 <via x="40.64" y="35.179" extent="1-16" drill="0.2032" diameter="0.4572"/>
 <via x="33.782" y="7.747" extent="1-16" drill="0.2032" diameter="0.4572"/>
@@
 </polygon>
 <polygon width="0.127" layer="16" thermals="no">
-<vertex x="58.9" y="68.65"/>
+<vertex x="58.265" y="68.65"/>
 <vertex x="54.6" y="68.65"/>
 <vertex x="54.6" y="64.8"/>
-<vertex x="58.9" y="64.8"/>
+<vertex x="58.265" y="64.8"/>
 </polygon>
 <polygon width="0.127" layer="16" thermals="no">
-<vertex x="81.9" y="68.65"/>
+<vertex x="81.265" y="68.65"/>
 <vertex x="77.6" y="68.65"/>
 <vertex x="77.6" y="64.8"/>
-<vertex x="81.9" y="64.8"/>
+<vertex x="81.265" y="64.8"/>
 </polygon>
 <polygon width="0.127" layer="16" thermals="no">
@@
 <wire x1="29.337" y1="8.636" x2="29.337" y2="8.637253125" width="0.1778" layer="3"/>
 <via x="100.838" y="67.564" extent="1-16" drill="0.2032" diameter="0.4572"/>
-<via x="58.547" y="65.024" extent="1-16" drill="0.2032" diameter="0.4572"/>
-<via x="80.391" y="64.897" extent="1-16" drill="0.2032" diameter="0.4572"/>
 <wire x1="19.939" y1="27.2096" x2="19.9974" y2="27.268" width="0.2032" layer="16"/>
 <wire x1="19.939" y1="27.2096" x2="19.0816" y2="27.2096" width="0.2032" layer="16"/>
@@
 <via x="102.108" y="67.437" extent="1-16" drill="0.2032" diameter="0.4572"/>
 <via x="102.108" y="68.326" extent="1-16" drill="0.2032" diameter="0.4572"/>
-<wire x1="29.972" y1="8.255" x2="29.337" y2="8.636" width="0" layer="19" extent="1-3"/>
 </signal>
 <signal name="N$116">
@@
 <vertex x="103.505" y="12.192"/>
 <vertex x="99.314" y="12.192"/>
-<vertex x="99.314" y="8.255"/>
+<vertex x="99.441" y="8.255"/>
+<vertex x="78.994" y="8.255"/>
+<vertex x="78.994" y="7.493"/>
+<vertex x="74.422" y="7.493"/>
+<vertex x="74.422" y="8.255"/>
+<vertex x="56.007" y="8.255"/>
+<vertex x="56.007" y="7.493"/>
+<vertex x="51.816" y="7.493"/>
+<vertex x="51.816" y="8.255"/>
+<vertex x="33.02" y="8.255"/>
+<vertex x="32.893" y="7.62"/>
+<vertex x="29.083" y="7.62"/>
+<vertex x="29.083" y="8.255"/>
+<vertex x="10.125" y="8.255" curve="-90"/>
 </polygon>
 <polygon width="0.127" layer="3" isolate="0.254">

Commit message: finished layout, no airwires, no unapproved DRC errors, ready for silk
Parts:
- moved C13 2.52 mm to (106.1, 35.8)
- moved C11 2.10 mm to (52.7, 23.5), turned to 0 degrees
- moved LED33 1.09 mm to (39.6, 33.5)
Routing:
- net VDDIO_IN: track 44.5 -> 15.7 mm, vias 5 -> 10
- net NODE6_!FLT: track 47.5 -> 59.2 mm, vias 3 -> 4
- net NODE8_!FLT: track 20.1 -> 31.5 mm
- net NODE6_IMON: track 33.6 -> 42.9 mm
- net GND: track 254.8 -> 258.7 mm, vias 116 -> 117
- net +3V3: track 146.7 -> 143.3 mm, vias 89 -> 91
- net N$104: track 57.3 -> 60.0 mm
- net N$102: track 98.2 -> 100.8 mm, vias 2 -> 3
- net NODE7_IMON: track 33.5 -> 31.7 mm, vias 2 -> 3
- net N$103: track 68.8 -> 70.4 mm, vias 4 -> 5
- net N$106: track 90.3 -> 89.8 mm
- net N$107: track 28.3 -> 28.5 mm, vias 2 -> 3
- net +18V: vias 87 -> 94
- added copper zone on layer 15, net VDDIO_IN
- added copper zone on layer 16, net VDDIO_IN

Commit message: Fixed routes
Parts:
- moved T20 0.13 mm to (106.0, 60.6)
Routing:
- net NODE4_IMON_IN: track 42.2 -> 40.1 mm
- net N$14: track 4.81 -> 3.61 mm
- net NODE1_LTCH: track 3.58 -> 2.85 mm
- net +2V1: track 167.9 -> 168.5 mm
- net N$19: track 5.75 -> 5.76 mm, vias 2 -> 1

Commit message: Fixed more routes
Routing:
- net GND: track 258.7 -> 259.6 mm
- net N$12: track 3.95 -> 3.25 mm
Changed lines of the file:
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@@
 <layer number="49" name="Reference" color="7" fill="1" visible="no" active="yes"/>
 <layer number="50" name="dxf" color="7" fill="1" visible="no" active="no"/>
-<layer number="51" name="tDocu" color="7" fill="1" visible="no" active="yes"/>
-<layer number="52" name="bDocu" color="7" fill="1" visible="no" active="yes"/>
+<layer number="51" name="tDocu" color="7" fill="1" visible="yes" active="yes"/>
+<layer number="52" name="bDocu" color="7" fill="1" visible="yes" active="yes"/>
 <layer number="53" name="tGND_GNDA" color="7" fill="1" visible="no" active="no"/>
 <layer number="54" name="bGND_GNDA" color="7" fill="1" visible="no" active="no"/>
@@
 <attribute name="VALUE" x="59.064" y="34.604" size="0.0254" layer="27"/>
 </element>
-<element name="J11" library="headers" package="1.27MM_3X1" value="I2C Header" x="30.226" y="42.672" rot="R180"/>
-<element name="R18" library="rcl_custom" package="0402-B-NOSILK" value="10k" x="51.181" y="20.828" rot="MR180"/>
+<element name="J11" library="headers" package="1.27MM_3X1" value="I2C Header" x="30.226" y="42.672" smashed="yes" rot="R180">
+<attribute name="NAME" x="31.626" y="41.242" size="0.6096" layer="25" rot="R180"/>
+<attribute name="VALUE" x="31.626" y="45.972" size="0.6096" layer="27" rot="R180"/>
+</element>
+<element name="R18" library="rcl_custom" package="0402-B-NOSILK" value="10k" x="51.181" y="20.828" smashed="yes" rot="MR180">
+<attribute name="NAME" x="50.381" y="20.028" size="1" layer="26" ratio="10" rot="MR180"/>
+<attribute name="VALUE" x="50.381" y="22.678" size="1" layer="28" ratio="10" rot="MR180"/>
+</element>
 </elements>
 <signals>
@@
 <contactref element="U1" pad="49"/>
 <wire x1="57.658" y1="37.973" x2="57.023" y2="38.608" width="0.1778" layer="16"/>
-<wire x1="57.658" y1="37.719" x2="57.658" y2="37.973" width="0.1778" layer="1"/>
-<wire x1="57.531" y1="37.592" x2="57.658" y2="37.719" width="0.1778" layer="1"/>
-<wire x1="57.531" y1="37.084" x2="57.531" y2="37.592" width="0.1778" layer="1"/>
-<wire x1="57.658" y1="36.957" x2="57.531" y2="37.084" width="0.1778" layer="1"/>
-<wire x1="58.928" y1="36.957" x2="57.658" y2="36.957" width="0.1778" layer="1"/>
-<wire x1="59.309" y1="36.576" x2="58.928" y2="36.957" width="0.1778" layer="1"/>
 <wire x1="57.023" y1="38.608" x2="56.9764125" y2="38.6435875" width="0.1778" layer="16"/>
 <wire x1="59.309" y1="36.576" x2="59.34795" y2="36.530221875" width="0.1778" layer="1"/>
 <via x="57.658" y="37.973" extent="1-16" drill="0.2032" diameter="0.4572"/>
+<wire x1="59.309" y1="36.576" x2="57.912" y2="37.973" width="0.1778" layer="1"/>
+<wire x1="57.912" y1="37.973" x2="57.658" y2="37.973" width="0.1778" layer="1"/>
 </signal>
 <signal name="GND" class="1">
@@
 <wire x1="107.696" y1="40.894" x2="106.172" y2="39.37" width="0.127" layer="16"/>
 <via x="11.176" y="16.51" extent="1-16" drill="0.2032" diameter="0.4572"/>
-<via x="21.971" y="10.414" extent="1-16" drill="0.2032" diameter="0.4572"/>
 <via x="25.281" y="29.845" extent="1-16" drill="0.2032" diameter="0.4572"/>
 <via x="37.719" y="22.733" extent="1-16" drill="0.2032" diameter="0.4572"/>
@@
 <via x="23.56" y="28.74" extent="1-16" drill="0.2032" diameter="0.4572"/>
 <wire x1="20.1" y1="10.38" x2="21.937" y2="10.38" width="0.127" layer="16"/>
-<wire x1="21.937" y1="10.38" x2="21.971" y2="10.414" width="0.127" layer="16"/>
 <wire x1="92.71" y1="54.356" x2="92.71" y2="55.118" width="0.1778" layer="1"/>
 <wire x1="92.964" y1="54.102" x2="92.71" y2="54.356" width="0.1778" layer="1"/>
@@
 <wire x1="71.374" y1="38.354" x2="71.374" y2="37.719" width="0.254" layer="16"/>
 <wire x1="71.374" y1="37.719" x2="71.755" y2="37.338" width="0.254" layer="16"/>
-<wire x1="74.041" y1="44.168" x2="72.898" y2="44.168" width="0.254" layer="1"/>
 <wire x1="72.362" y1="44.168" x2="71.501" y2="43.307" width="0.254" layer="1"/>
 <wire x1="92.546" y1="57.48" x2="92.47" y2="57.404" width="0.254" layer="16"/>
@@
 <via x="104.14" y="59.563" extent="1-16" drill="0.2032" diameter="0.4572"/>
 <wire x1="104.14" y1="59.563" x2="104.013" y2="59.563" width="0.1778" layer="2"/>
+<via x="21.937" y="10.38" extent="1-16" drill="0.2032" diameter="0.4572"/>
+<wire x1="21.937" y1="10.38" x2="21.971" y2="10.38" width="0.127" layer="2"/>
+<wire x1="21.971" y1="10.38" x2="21.971" y2="10.414" width="0.127" layer="2"/>
+<wire x1="74.041" y1="44.168" x2="74.069" y2="44.196" width="0.1778" layer="1"/>
+<wire x1="74.069" y1="44.196" x2="74.676" y2="44.196" width="0.254" layer="1"/>
+<wire x1="74.676" y1="44.196" x2="75.022" y2="43.85" width="0.254" layer="1"/>
+<wire x1="75.022" y1="43.85" x2="75.9" y2="43.85" width="0.254" layer="1"/>
+<polygon width="0.1778" layer="1">
+<vertex x="72.517" y="44.45"/>
+<vertex x="74.549" y="44.45"/>
+<vertex x="74.549" y="43.942"/>
+<vertex x="72.517" y="43.942"/>
+</polygon>
 </signal>
 <signal name="+3V3" class="1">
