File: av3/rocketnet-hub/eagle/mcu_page_combined_routed.sch (EAGLE design)
At the start: 439 parts, among them J1 ROCKETNET-CONNECTOR-16M, J10 UART Header, J12 BOOT1 Jumper, J13 PGOOD Jumper, J14 ROCKETNET-UMBILICAL-18, J15 Auxiliary Header, J16 Auxiliary Header, J17 Auxiliary Header, J18 Auxiliary Header, J19 Auxiliary Header, J2 ROCKETNET-CONNECTOR-16M, J20 Auxiliary Header, J21 Auxiliary Header, J22 Debug Header, J3 ROCKETNET-CONNECTOR-16M, J4 ROCKETNET-CONNECTOR-16M, J5 BOOT0 Jumper, J6 ROCKETNET-CONNECTOR-16M, J7 ROCKETNET-CONNECTOR-16M, J8 ROCKETNET-CONNECTOR-16M, J9 ROCKETNET-BATTERY-14, Q2 FDS6680ASOIC8, Q3 FDS6680ASOIC8, Q4 FDS6680ASOIC8, Q5 SIS412DNSOP-8, Q6 BSS138W-7-F, Q7 SIS412DNSOP-8, T1 BSS84, T10 ALT4532, T11 ALT4532, T12 ALT4532, T13 ALT4532, T14 ALT4532, T15 ALT4532, T16 ALT4532, T17 ALT4532, T18 ALT4532, T19 BSS84, T2 NDS335N, T20 NDS335N, T3 ALT4532, T4 ALT4532, T5 ALT4532, T6 ALT4532, T7 ALT4532, T8 ALT4532, T9 ALT4532, U1 STM32F407V100-PIN_QFP, U10 TPS2420QFN-16, U11 TPS2420QFN-16, U12 TPS2420QFN-16, U13 TPS2420QFN-16, U14 MAX4734ETC+, U15 MAX4734ETC+, U2 BQ24725QFN-20, U3 SN65220DBV, U4 KS8999, U5 LTM8023, U6 MIC37101-2.1YM, U7 TPS2420QFN-16, U8 TPS2420QFN-16, U9 TPS2420QFN-16

Commit message: Added a 1x3 50mil header for I2C interface, added 10k pulldown on U15 pin N1, fixed +3v3 nets on bottom area of the board
Parts:
- added J11: I2C Header, headers:1.27MM_HDR_1X3
- added R18: 10k, rcl_custom:R-US_0402-B-NOSILK
Connections:
- new net N$32: R18.2, U15.N1
- net GND: now also J11.GND, R18.1
- net SCL: now also J11.SCL
- net SDA: now also J11.SDA
Other:
- moved on the sheet: J12, J5, R150, R64
Changed lines of the file:
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@@
 <part name="+3V42" library="supply1" deviceset="+3V3" device=""/>
 <part name="TP39" library="testpad" deviceset="TP" device="TP06R"/>
+<part name="J11" library="headers" deviceset="1.27MM_HDR_1X3" device="" value="I2C Header"/>
+<part name="GND8" library="supply1" deviceset="GND" device=""/>
+<part name="R18" library="rcl_custom" deviceset="R-US_" device="0402-B-NOSILK" value="10k"/>
+<part name="GND9" library="supply1" deviceset="GND" device=""/>
 </parts>
 <sheets>
@@
 <wire x1="327.66" y1="322.58" x2="327.66" y2="401.32" width="0.1524" layer="97" style="shortdash"/>
 <wire x1="327.66" y1="401.32" x2="220.98" y2="401.32" width="0.1524" layer="97" style="shortdash"/>
-<wire x1="-63.5" y1="378.46" x2="-63.5" y2="327.66" width="0.1524" layer="97" style="shortdash"/>
-<wire x1="-63.5" y1="327.66" x2="-7.62" y2="327.66" width="0.1524" layer="97" style="shortdash"/>
-<wire x1="-7.62" y1="327.66" x2="-7.62" y2="378.46" width="0.1524" layer="97" style="shortdash"/>
-<wire x1="-7.62" y1="378.46" x2="-63.5" y2="378.46" width="0.1524" layer="97" style="shortdash"/>
-<text x="-53.34" y="373.38" size="2.54" layer="97">Boot Configuration</text>
+<wire x1="-78.74" y1="378.46" x2="-78.74" y2="327.66" width="0.1524" layer="97" style="shortdash"/>
+<wire x1="-78.74" y1="327.66" x2="-22.86" y2="327.66" width="0.1524" layer="97" style="shortdash"/>
+<wire x1="-22.86" y1="327.66" x2="-22.86" y2="378.46" width="0.1524" layer="97" style="shortdash"/>
+<wire x1="-22.86" y1="378.46" x2="-78.74" y2="378.46" width="0.1524" layer="97" style="shortdash"/>
+<text x="-68.58" y="373.38" size="2.54" layer="97">Boot Configuration</text>
 <wire x1="220.98" y1="469.9" x2="220.98" y2="416.56" width="0.1524" layer="97" style="shortdash"/>
 <wire x1="220.98" y1="416.56" x2="287.02" y2="416.56" width="0.1524" layer="97" style="shortdash"/>
@@
 <instance part="TP37" gate="G$1" x="50.8" y="447.04"/>
 <instance part="GND80" gate="1" x="91.44" y="304.8"/>
-<instance part="R64" gate="R" x="-45.72" y="342.9" rot="R270"/>
-<instance part="GND1" gate="1" x="-45.72" y="332.74"/>
-<instance part="J5" gate="J" x="-48.26" y="358.14" rot="R180"/>
-<instance part="+3V34" gate="G$1" x="-45.72" y="365.76"/>
-<instance part="J12" gate="J" x="-20.32" y="358.14" rot="R180"/>
-<instance part="+3V35" gate="G$1" x="-17.78" y="365.76"/>
-<instance part="R150" gate="R" x="-17.78" y="342.9" rot="R270"/>
-<instance part="GND98" gate="1" x="-17.78" y="332.74"/>
+<instance part="R64" gate="R" x="-60.96" y="342.9" rot="R270"/>
+<instance part="GND1" gate="1" x="-60.96" y="332.74"/>
+<instance part="J5" gate="J" x="-63.5" y="358.14" rot="R180"/>
+<instance part="+3V34" gate="G$1" x="-60.96" y="365.76"/>
+<instance part="J12" gate="J" x="-35.56" y="358.14" rot="R180"/>
+<instance part="+3V35" gate="G$1" x="-33.02" y="365.76"/>
+<instance part="R150" gate="R" x="-33.02" y="342.9" rot="R270"/>
+<instance part="GND98" gate="1" x="-33.02" y="332.74"/>
 <instance part="C134" gate="C$1" x="83.82" y="464.82" rot="R270"/>
 <instance part="GND137" gate="1" x="88.9" y="459.74"/>
@@
 <instance part="+3V42" gate="G$1" x="233.68" y="388.62"/>
 <instance part="TP39" gate="G$1" x="17.78" y="355.6"/>
+<instance part="J11" gate="J" x="-12.7" y="358.14" rot="MR0"/>
+<instance part="GND8" gate="1" x="-5.08" y="350.52"/>
 </instances>
 <busses>
@@
 <pinref part="R64" gate="R" pin="2"/>
 <pinref part="GND1" gate="1" pin="GND"/>
-<wire x1="-45.72" y1="337.82" x2="-45.72" y2="335.28" width="0.1524" layer="91"/>
+<wire x1="-60.96" y1="337.82" x2="-60.96" y2="335.28" width="0.1524" layer="91"/>
 </segment>
 <segment>
 <pinref part="R150" gate="R" pin="2"/>
 <pinref part="GND98" gate="1" pin="GND"/>
-<wire x1="-17.78" y1="337.82" x2="-17.78" y2="335.28" width="0.1524" layer="91"/>
+<wire x1="-33.02" y1="337.82" x2="-33.02" y2="335.28" width="0.1524" layer="91"/>
 </segment>
 <segment>
@@
 <wire x1="17.78" y1="340.36" x2="17.78" y2="335.28" width="0.1524" layer="91"/>
 </segment>
+<segment>
+<pinref part="J11" gate="J" pin="GND"/>
+<wire x1="-5.08" y1="358.14" x2="-5.08" y2="353.06" width="0.1524" layer="91"/>
+<pinref part="GND8" gate="1" pin="GND"/>
+</segment>
 </net>
 <net name="+3V3" class="1">
@@
 <pinref part="J5" gate="J" pin="2"/>
 <pinref part="+3V34" gate="G$1" pin="+3V3"/>
-<wire x1="-45.72" y1="355.6" x2="-45.72" y2="363.22" width="0.1524" layer="91"/>
+<wire x1="-60.96" y1="355.6" x2="-60.96" y2="363.22" width="0.1524" layer="91"/>
 </segment>
 <segment>
 <pinref part="J12" gate="J" pin="2"/>
 <pinref part="+3V35" gate="G$1" pin="+3V3"/>
-<wire x1="-17.78" y1="355.6" x2="-17.78" y2="363.22" width="0.1524" layer="91"/>
+<wire x1="-33.02" y1="355.6" x2="-33.02" y2="363.22" width="0.1524" layer="91"/>
 </segment>
 <segment>
@@
 <segment>
 <pinref part="U1" gate="U1" pin="PB6"/>
-<wire x1="2.54" y1="363.22" x2="5.08" y2="363.22" width="0.1524" layer="91"/>
-<label x="2.54" y="363.22" size="1.016" layer="95" rot="R180" xref="yes"/>
+<label x="0" y="365.76" size="1.016" layer="95" rot="R180" xref="yes"/>
 <pinref part="R17" gate="R" pin="2"/>
 <wire x1="5.08" y1="363.22" x2="63.5" y2="363.22" width="0.1524" layer="91"/>
 <wire x1="5.08" y1="365.76" x2="5.08" y2="363.22" width="0.1524" layer="91"/>
 <junction x="5.08" y="363.22"/>
+<pinref part="J11" gate="J" pin="SCL"/>
+<wire x1="5.08" y1="363.22" x2="-5.08" y2="363.22" width="0.1524" layer="91"/>
 </segment>
 </net>
@@
 <segment>
 <pinref part="U1" gate="U1" pin="PB7"/>
-<wire x1="2.54" y1="360.68" x2="12.7" y2="360.68" width="0.1524" layer="91"/>
-<label x="2.54" y="360.68" size="1.016" layer="95" rot="R180" xref="yes"/>
+<label x="5.08" y="358.14" size="1.016" layer="95" rot="R180" xref="yes"/>
 <pinref part="R15" gate="R" pin="2"/>
 <wire x1="12.7" y1="360.68" x2="63.5" y2="360.68" width="0.1524" layer="91"/>
 <wire x1="12.7" y1="365.76" x2="12.7" y2="360.68" width="0.1524" layer="91"/>
 <junction x="12.7" y="360.68"/>
+<pinref part="J11" gate="J" pin="SDA"/>
+<wire x1="-5.08" y1="360.68" x2="12.7" y2="360.68" width="0.1524" layer="91"/>
 </segment>
 </net>
@@
 <pinref part="J5" gate="J" pin="1"/>
 <pinref part="R64" gate="R" pin="1"/>
-<wire x1="-45.72" y1="347.98" x2="-45.72" y2="353.06" width="0.1524" layer="91"/>
-<wire x1="-45.72" y1="347.98" x2="-38.1" y2="347.98" width="0.1524" layer="91"/>
-<wire x1="-38.1" y1="347.98" x2="-38.1" y2="439.42" width="0.1524" layer="91"/>
-<junction x="-45.72" y="347.98"/>
-<wire x1="-38.1" y1="439.42" x2="78.74" y2="439.42" width="0.1524" layer="91"/>
+<wire x1="-60.96" y1="347.98" x2="-60.96" y2="353.06" width="0.1524" layer="91"/>
+<wire x1="-60.96" y1="347.98" x2="-53.34" y2="347.98" width="0.1524" layer="91"/>
+<wire x1="-53.34" y1="347.98" x2="-53.34" y2="439.42" width="0.1524" layer="91"/>
+<junction x="-60.96" y="347.98"/>
+<wire x1="-53.34" y1="439.42" x2="78.74" y2="439.42" width="0.1524" layer="91"/>
 </segment>
 </net>
@@
 <pinref part="J12" gate="J" pin="1"/>
 <pinref part="R150" gate="R" pin="1"/>
-<wire x1="-17.78" y1="347.98" x2="-17.78" y2="353.06" width="0.1524" layer="91"/>
-<wire x1="-17.78" y1="347.98" x2="-10.16" y2="347.98" width="0.1524" layer="91"/>
-<wire x1="-10.16" y1="347.98" x2="-10.16" y2="386.08" width="0.1524" layer="91"/>
-<junction x="-17.78" y="347.98"/>
-<wire x1="-10.16" y1="386.08" x2="17.78" y2="386.08" width="0.1524" layer="91"/>
+<wire x1="-33.02" y1="347.98" x2="-33.02" y2="353.06" width="0.1524" layer="91"/>
+<wire x1="-33.02" y1="347.98" x2="-25.4" y2="347.98" width="0.1524" layer="91"/>
+<wire x1="-25.4" y1="347.98" x2="-25.4" y2="386.08" width="0.1524" layer="91"/>
+<junction x="-33.02" y="347.98"/>
+<wire x1="-25.4" y1="386.08" x2="17.78" y2="386.08" width="0.1524" layer="91"/>
 <wire x1="17.78" y1="386.08" x2="17.78" y2="373.38" width="0.1524" layer="91"/>
 <pinref part="U1" gate="U1" pin="PB2"/>
@@
 <instance part="NODE_CONNECTIONS" gate="G$1" x="223.52" y="-144.78"/>
 <instance part="NODE_CONNECTIONS" gate="G$2" x="675.64" y="-195.58"/>
+<instance part="R18" gate="R" x="302.26" y="170.18" rot="MR90"/>
+<instance part="GND9" gate="1" x="302.26" y="162.56"/>
 </instances>
 <busses>
@@
 <wire x1="411.48" y1="91.44" x2="411.48" y2="96.52" width="0.1524" layer="91"/>
 </segment>
+<segment>
+<pinref part="R18" gate="R" pin="1"/>
+<pinref part="GND9" gate="1" pin="GND"/>
+</segment>
 </net>
 <net name="NODE1_VOUT" class="1">
@@
 </segment>
 </net>
+<net name="N$32" class="0">
+<segment>
+<pinref part="U15" gate="U$1" pin="N1"/>
+<wire x1="287.02" y1="198.12" x2="302.26" y2="198.12" width="0.1524" layer="91"/>
+<pinref part="R18" gate="R" pin="2"/>
+<wire x1="302.26" y1="175.26" x2="302.26" y2="198.12" width="0.1524" layer="91"/>
+</segment>
+</net>

Commit message: Updated pin 189 on KS8999
Connections:
- net +2V1: now also U4.VDD_PLLTX; no longer U4.VDD_PLL
- net GND: now also U4.GND_RCV7
- net MRXD3: now also U4.MRXD[3]; no longer U4.MRXD[4]
Changed lines of the file:
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@@
 <pinref part="U4" gate="U" pin="GND-ISO3"/>
 <junction x="175.26" y="12.7"/>
+<pinref part="U4" gate="U" pin="GND_RCV7"/>
+<wire x1="177.8" y1="12.7" x2="180.34" y2="12.7" width="0.1524" layer="91"/>
 </segment>
 <segment>
@@
 <net name="MRXD3" class="0">
 <segment>
-<pinref part="U4" gate="U" pin="MRXD[4]"/>
+<pinref part="U4" gate="U" pin="MRXD[3]"/>
 <wire x1="76.2" y1="208.28" x2="78.74" y2="208.28" width="0.1524" layer="91"/>
 <label x="76.2" y="208.28" size="1.016" layer="95" rot="R180" xref="yes"/>
@@
 <junction x="165.1" y="243.84"/>
 <wire x1="165.1" y1="243.84" x2="165.1" y2="238.76" width="0.1524" layer="91"/>
-<pinref part="U4" gate="U" pin="VDD_PLL"/>
+<pinref part="U4" gate="U" pin="VDD_PLLTX"/>
 <pinref part="C72" gate="CE" pin="2"/>
 <pinref part="C81" gate="CE" pin="2"/>

Commit message: Cleaned up libraries and updated LDO 2V1 schematic; added silkscreen to FDS6680A
Connections:
- net GND: now also U6.GND; no longer U6.GND@5, U6.GND@6, U6.GND@7, U6.GND@8
Other:
- moved on the sheet: C52, C84, C85, TP28

Commit message: change C102 package from 0805 to 0402.
Parts:
- C102: device rcl_custom:C-EU0805-B-NOSILK -> rcl_custom:C-EU0402-B-NOSILK
Changed lines of the file:
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@@
 <grid distance="0.1" unitdist="inch" unit="inch" style="lines" multiple="1" display="no" altdistance="0.01" altunitdist="inch" altunit="inch"/>
 <layers>
-<layer number="1" name="Top" color="4" fill="1" visible="no" active="no"/>
-<layer number="2" name="Route2" color="1" fill="6" visible="no" active="no"/>
-<layer number="3" name="Route3" color="12" fill="1" visible="no" active="no"/>
-<layer number="14" name="Route14" color="13" fill="1" visible="no" active="no"/>
-<layer number="15" name="Route15" color="6" fill="1" visible="no" active="no"/>
-<layer number="16" name="Bottom" color="1" fill="1" visible="no" active="no"/>
-<layer number="17" name="Pads" color="2" fill="1" visible="no" active="no"/>
-<layer number="18" name="Vias" color="2" fill="1" visible="no" active="no"/>
-<layer number="19" name="Unrouted" color="6" fill="1" visible="no" active="no"/>
-<layer number="20" name="Dimension" color="15" fill="1" visible="no" active="no"/>
-<layer number="21" name="tPlace" color="7" fill="1" visible="no" active="no"/>
-<layer number="22" name="bPlace" color="7" fill="1" visible="no" active="no"/>
-<layer number="23" name="tOrigins" color="15" fill="1" visible="no" active="no"/>
-<layer number="24" name="bOrigins" color="15" fill="1" visible="no" active="no"/>
-<layer number="25" name="tNames" color="7" fill="1" visible="no" active="no"/>
-<layer number="26" name="bNames" color="7" fill="1" visible="no" active="no"/>
-<layer number="27" name="tValues" color="7" fill="1" visible="no" active="no"/>
-<layer number="28" name="bValues" color="7" fill="1" visible="no" active="no"/>
+<layer number="1" name="Top" color="4" fill="1" visible="yes" active="no"/>
+<layer number="2" name="Route2" color="9" fill="1" visible="yes" active="no"/>
+<layer number="3" name="Route3" color="12" fill="1" visible="yes" active="no"/>
+<layer number="14" name="Route14" color="11" fill="3" visible="yes" active="no"/>
+<layer number="15" name="Route15" color="6" fill="1" visible="yes" active="no"/>
+<layer number="16" name="Bottom" color="1" fill="1" visible="yes" active="no"/>
+<layer number="17" name="Pads" color="2" fill="1" visible="yes" active="no"/>
+<layer number="18" name="Vias" color="2" fill="1" visible="yes" active="no"/>
+<layer number="19" name="Unrouted" color="6" fill="1" visible="yes" active="no"/>
+<layer number="20" name="Dimension" color="15" fill="1" visible="yes" active="no"/>
+<layer number="21" name="tPlace" color="7" fill="1" visible="yes" active="no"/>
+<layer number="22" name="bPlace" color="7" fill="1" visible="yes" active="no"/>
+<layer number="23" name="tOrigins" color="15" fill="1" visible="yes" active="no"/>
+<layer number="24" name="bOrigins" color="15" fill="1" visible="yes" active="no"/>
+<layer number="25" name="tNames" color="7" fill="1" visible="yes" active="no"/>
+<layer number="26" name="bNames" color="7" fill="1" visible="yes" active="no"/>
+<layer number="27" name="tValues" color="7" fill="1" visible="yes" active="no"/>
+<layer number="28" name="bValues" color="7" fill="1" visible="yes" active="no"/>
 <layer number="29" name="tStop" color="7" fill="3" visible="no" active="no"/>
 <layer number="30" name="bStop" color="7" fill="6" visible="no" active="no"/>
@@
 <layer number="35" name="tGlue" color="7" fill="4" visible="no" active="no"/>
 <layer number="36" name="bGlue" color="7" fill="5" visible="no" active="no"/>
-<layer number="37" name="tTest" color="7" fill="1" visible="no" active="no"/>
-<layer number="38" name="bTest" color="7" fill="1" visible="no" active="no"/>
+<layer number="37" name="tTest" color="7" fill="1" visible="yes" active="no"/>
+<layer number="38" name="bTest" color="7" fill="1" visible="yes" active="no"/>
 <layer number="39" name="tKeepout" color="4" fill="11" visible="no" active="no"/>
 <layer number="40" name="bKeepout" color="1" fill="11" visible="no" active="no"/>
@@
 <layer number="44" name="Drills" color="7" fill="1" visible="no" active="no"/>
 <layer number="45" name="Holes" color="7" fill="1" visible="no" active="no"/>
-<layer number="46" name="Milling" color="3" fill="1" visible="no" active="no"/>
-<layer number="47" name="Measures" color="7" fill="1" visible="no" active="no"/>
-<layer number="48" name="Document" color="7" fill="1" visible="no" active="no"/>
-<layer number="49" name="Reference" color="7" fill="1" visible="no" active="no"/>
-<layer number="50" name="dxf" color="7" fill="1" visible="no" active="no"/>
-<layer number="51" name="tDocu" color="7" fill="1" visible="no" active="no"/>
-<layer number="52" name="bDocu" color="7" fill="1" visible="no" active="no"/>
-<layer number="53" name="tGND_GNDA" color="7" fill="1" visible="no" active="no"/>
-<layer number="54" name="bGND_GNDA" color="7" fill="1" visible="no" active="no"/>
-<layer number="56" name="wert" color="7" fill="1" visible="no" active="no"/>
+<layer number="46" name="Milling" color="3" fill="1" visible="yes" active="no"/>
+<layer number="47" name="Measures" color="7" fill="1" visible="yes" active="no"/>
+<layer number="48" name="Document" color="7" fill="1" visible="yes" active="no"/>
+<layer number="49" name="Reference" color="7" fill="1" visible="yes" active="no"/>
+<layer number="50" name="dxf" color="7" fill="1" visible="yes" active="no"/>
+<layer number="51" name="tDocu" color="7" fill="1" visible="yes" active="no"/>
+<layer number="52" name="bDocu" color="7" fill="1" visible="yes" active="no"/>
+<layer number="53" name="tGND_GNDA" color="7" fill="1" visible="yes" active="no"/>
+<layer number="54" name="bGND_GNDA" color="7" fill="1" visible="yes" active="no"/>
+<layer number="56" name="wert" color="7" fill="1" visible="yes" active="no"/>
 <layer number="91" name="Nets" color="2" fill="1" visible="yes" active="yes"/>
 <layer number="92" name="Busses" color="1" fill="1" visible="yes" active="yes"/>
@@
 <part name="Q3" library="RNH_FDS6680A" deviceset="FDS6680A" device="SOIC8"/>
 <part name="C94" library="rcl_custom" deviceset="C-EU" device="0402-B-NOSILK" value="0.1uF/40V"/>
-<part name="C102" library="rcl_custom" deviceset="C-EU" device="0805-B-NOSILK" value="2200pF/40V"/>
+<part name="C102" library="rcl_custom" deviceset="C-EU" device="0402-B-NOSILK" value="2200pF/40V"/>
 <part name="Q6" library="RNH_BSS138W-7-F" deviceset="BSS138W-7-F" device=""/>
 <part name="R132" library="rcl_custom" deviceset="R-US_" device="0402-B-NOSILK" value="1M"/>
