File: av3/rocketnet-hub/eagle/mcu_page_combined_routed.sch (EAGLE design)
At the start: 441 parts, among them J1 ROCKETNET-CONNECTOR-16M, J10 UART Header, J11 I2C Header, J12 BOOT1 Jumper, J13 PGOOD Jumper, J14 ROCKETNET-UMBILICAL-18, J15 Auxiliary Header, J16 Auxiliary Header, J17 Auxiliary Header, J18 Auxiliary Header, J19 Auxiliary Header, J2 ROCKETNET-CONNECTOR-16M, J20 Auxiliary Header, J21 Auxiliary Header, J22 Debug Header, J3 ROCKETNET-CONNECTOR-16M, J4 ROCKETNET-CONNECTOR-16M, J5 BOOT0 Jumper, J6 ROCKETNET-CONNECTOR-16M, J7 ROCKETNET-CONNECTOR-16M, J8 ROCKETNET-CONNECTOR-16M, J9 ROCKETNET-BATTERY-14, Q2 FDS6680ASOIC8, Q3 FDS6680ASOIC8, Q4 FDS6680ASOIC8, Q5 SIS412DNSOP-8, Q6 BSS138W-7-F, Q7 SIS412DNSOP-8, T1 BSS84, T10 ALT4532, T11 ALT4532, T12 ALT4532, T13 ALT4532, T14 ALT4532, T15 ALT4532, T16 ALT4532, T17 ALT4532, T18 ALT4532, T19 BSS84, T2 NDS335N, T20 NDS335N, T3 ALT4532, T4 ALT4532, T5 ALT4532, T6 ALT4532, T7 ALT4532, T8 ALT4532, T9 ALT4532, U1 STM32F407V100-PIN_QFP, U10 TPS2420QFN-16, U11 TPS2420QFN-16, U12 TPS2420QFN-16, U13 TPS2420QFN-16, U14 MAX4734ETC+, U15 MAX4734ETC+, U2 BQ24725QFN-20, U3 SN65220DBV, U4 KS8999, U5 LTM8023, U6 MIC37101-2.1YM, U7 TPS2420QFN-16, U8 TPS2420QFN-16, U9 TPS2420QFN-16

Commit message: R151 value changed from 1n to 51
Parts:
- R151: value 1n -> 51
Changed lines of the file:
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@@
 <grid distance="0.1" unitdist="inch" unit="inch" style="lines" multiple="1" display="no" altdistance="0.01" altunitdist="inch" altunit="inch"/>
 <layers>
-<layer number="1" name="Top" color="4" fill="1" visible="yes" active="no"/>
-<layer number="2" name="Route2" color="9" fill="1" visible="yes" active="no"/>
-<layer number="3" name="Route3" color="12" fill="1" visible="yes" active="no"/>
-<layer number="14" name="Route14" color="11" fill="3" visible="yes" active="no"/>
-<layer number="15" name="Route15" color="6" fill="1" visible="yes" active="no"/>
-<layer number="16" name="Bottom" color="1" fill="1" visible="yes" active="no"/>
-<layer number="17" name="Pads" color="2" fill="1" visible="yes" active="no"/>
-<layer number="18" name="Vias" color="2" fill="1" visible="yes" active="no"/>
-<layer number="19" name="Unrouted" color="6" fill="1" visible="yes" active="no"/>
-<layer number="20" name="Dimension" color="15" fill="1" visible="yes" active="no"/>
-<layer number="21" name="tPlace" color="7" fill="1" visible="yes" active="no"/>
-<layer number="22" name="bPlace" color="7" fill="1" visible="yes" active="no"/>
-<layer number="23" name="tOrigins" color="15" fill="1" visible="yes" active="no"/>
-<layer number="24" name="bOrigins" color="15" fill="1" visible="yes" active="no"/>
-<layer number="25" name="tNames" color="7" fill="1" visible="yes" active="no"/>
-<layer number="26" name="bNames" color="7" fill="1" visible="yes" active="no"/>
-<layer number="27" name="tValues" color="7" fill="1" visible="yes" active="no"/>
-<layer number="28" name="bValues" color="7" fill="1" visible="yes" active="no"/>
+<layer number="1" name="Top" color="4" fill="1" visible="no" active="no"/>
+<layer number="2" name="Route2" color="9" fill="1" visible="no" active="no"/>
+<layer number="3" name="Route3" color="12" fill="1" visible="no" active="no"/>
+<layer number="14" name="Route14" color="11" fill="3" visible="no" active="no"/>
+<layer number="15" name="Route15" color="6" fill="1" visible="no" active="no"/>
+<layer number="16" name="Bottom" color="1" fill="1" visible="no" active="no"/>
+<layer number="17" name="Pads" color="2" fill="1" visible="no" active="no"/>
+<layer number="18" name="Vias" color="2" fill="1" visible="no" active="no"/>
+<layer number="19" name="Unrouted" color="6" fill="1" visible="no" active="no"/>
+<layer number="20" name="Dimension" color="15" fill="1" visible="no" active="no"/>
+<layer number="21" name="tPlace" color="7" fill="1" visible="no" active="no"/>
+<layer number="22" name="bPlace" color="7" fill="1" visible="no" active="no"/>
+<layer number="23" name="tOrigins" color="15" fill="1" visible="no" active="no"/>
+<layer number="24" name="bOrigins" color="15" fill="1" visible="no" active="no"/>
+<layer number="25" name="tNames" color="7" fill="1" visible="no" active="no"/>
+<layer number="26" name="bNames" color="7" fill="1" visible="no" active="no"/>
+<layer number="27" name="tValues" color="7" fill="1" visible="no" active="no"/>
+<layer number="28" name="bValues" color="7" fill="1" visible="no" active="no"/>
 <layer number="29" name="tStop" color="7" fill="3" visible="no" active="no"/>
 <layer number="30" name="bStop" color="7" fill="6" visible="no" active="no"/>
@@
 <layer number="35" name="tGlue" color="7" fill="4" visible="no" active="no"/>
 <layer number="36" name="bGlue" color="7" fill="5" visible="no" active="no"/>
-<layer number="37" name="tTest" color="7" fill="1" visible="yes" active="no"/>
-<layer number="38" name="bTest" color="7" fill="1" visible="yes" active="no"/>
+<layer number="37" name="tTest" color="7" fill="1" visible="no" active="no"/>
+<layer number="38" name="bTest" color="7" fill="1" visible="no" active="no"/>
 <layer number="39" name="tKeepout" color="4" fill="11" visible="no" active="no"/>
 <layer number="40" name="bKeepout" color="1" fill="11" visible="no" active="no"/>
@@
 <layer number="44" name="Drills" color="7" fill="1" visible="no" active="no"/>
 <layer number="45" name="Holes" color="7" fill="1" visible="no" active="no"/>
-<layer number="46" name="Milling" color="3" fill="1" visible="yes" active="no"/>
-<layer number="47" name="Measures" color="7" fill="1" visible="yes" active="no"/>
-<layer number="48" name="Document" color="7" fill="1" visible="yes" active="no"/>
-<layer number="49" name="Reference" color="7" fill="1" visible="yes" active="no"/>
-<layer number="50" name="dxf" color="7" fill="1" visible="yes" active="no"/>
-<layer number="51" name="tDocu" color="7" fill="1" visible="yes" active="no"/>
-<layer number="52" name="bDocu" color="7" fill="1" visible="yes" active="no"/>
-<layer number="53" name="tGND_GNDA" color="7" fill="1" visible="yes" active="no"/>
-<layer number="54" name="bGND_GNDA" color="7" fill="1" visible="yes" active="no"/>
-<layer number="56" name="wert" color="7" fill="1" visible="yes" active="no"/>
+<layer number="46" name="Milling" color="3" fill="1" visible="no" active="no"/>
+<layer number="47" name="Measures" color="7" fill="1" visible="no" active="no"/>
+<layer number="48" name="Document" color="7" fill="1" visible="no" active="no"/>
+<layer number="49" name="Reference" color="7" fill="1" visible="no" active="no"/>
+<layer number="50" name="dxf" color="7" fill="1" visible="no" active="no"/>
+<layer number="51" name="tDocu" color="7" fill="1" visible="no" active="no"/>
+<layer number="52" name="bDocu" color="7" fill="1" visible="no" active="no"/>
+<layer number="53" name="tGND_GNDA" color="7" fill="1" visible="no" active="no"/>
+<layer number="54" name="bGND_GNDA" color="7" fill="1" visible="no" active="no"/>
+<layer number="56" name="wert" color="7" fill="1" visible="no" active="no"/>
 <layer number="91" name="Nets" color="2" fill="1" visible="yes" active="yes"/>
 <layer number="92" name="Busses" color="1" fill="1" visible="yes" active="yes"/>
@@
 <part name="GND131" library="supply1" deviceset="GND" device=""/>
 <part name="R149" library="rcl_custom" deviceset="R-US_" device="0402-B-NOSILK" value="51"/>
-<part name="R151" library="rcl_custom" deviceset="R-US_" device="0402-B-NOSILK" value="1n"/>
+<part name="R151" library="rcl_custom" deviceset="R-US_" device="0402-B-NOSILK" value="51"/>
 <part name="R152" library="rcl_custom" deviceset="R-US_" device="0402-B-NOSILK" value="51"/>
 <part name="R153" library="rcl_custom" deviceset="R-US_" device="0402-B-NOSILK" value="51"/>

Commit message: Replaced 2 ohm resistor; updated bom
Parts:
- R11: device rcl_custom:R-US_1206-B -> rcl_custom:R-US_R2512
Changed lines of the file:
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@@
 <part name="U2" library="RNH_BQ24725" deviceset="BQ24725" device="QFN-20"/>
 <part name="C60" library="rcl_custom" deviceset="C-EU" device="0805-B-NOSILK" value="2.2uF/40V"/>
-<part name="R11" library="rcl_custom" deviceset="R-US_" device="1206-B" value="2"/>
+<part name="R11" library="rcl_custom" deviceset="R-US_" device="R2512" value="2"/>
 <part name="Q2" library="RNH_FDS6680A" deviceset="FDS6680A" device="SOIC8"/>
 <part name="Q3" library="RNH_FDS6680A" deviceset="FDS6680A" device="SOIC8"/>

Commit message: Added D1,D2,D3 part number in schematic and bom
Parts:
- D1: value DIODE-0603 -> CDBU0520
- D2, D3: value DIODE-0603 -> CDBU0130L
Changed lines of the file:
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@@
 <part name="R46" library="rcl_custom" deviceset="R-US_" device="0402-B-NOSILK" value="750"/>
 <part name="+3V7" library="supply1" deviceset="+3V3" device=""/>
-<part name="D2" library="diode-0603" deviceset="DIODE-0603" device=""/>
+<part name="D2" library="diode-0603" deviceset="DIODE-0603" device="" value="CDBU0130L"/>
 <part name="R47" library="rcl_custom" deviceset="R-US_" device="0402-B-NOSILK" value="10k"/>
 <part name="C83" library="rcl_custom" deviceset="C-EU" device="0402-B-NOSILK" value="0.1u"/>
@@
 <part name="TP34" library="testpad" deviceset="TP" device="TP06R"/>
 <part name="TP35" library="testpad" deviceset="TP" device="TP06R"/>
-<part name="D3" library="diode-0603" deviceset="DIODE-0603" device=""/>
+<part name="D3" library="diode-0603" deviceset="DIODE-0603" device="" value="CDBU0130L"/>
 <part name="TP37" library="testpad" deviceset="TP" device="TP06R"/>
 <part name="LED22" library="led" deviceset="LED" device="CHIPLED_0603" value="GREEN"/>
@@
 <part name="GND130" library="supply1" deviceset="GND" device=""/>
 <part name="+3V39" library="supply1" deviceset="+3V3" device=""/>
-<part name="D1" library="diode-0603" deviceset="DIODE-0603" device=""/>
+<part name="D1" library="diode-0603" deviceset="DIODE-0603" device="" value="CDBU0520"/>
 <part name="GND138" library="supply1" deviceset="GND" device=""/>
 <part name="R130" library="rcl_custom" deviceset="R-US_" device="0402-B-NOSILK" value="10k"/>
