File: av3/rocketnet-hub/eagle/mcu_page_combined_routed.sch (EAGLE design)
At the start: 441 parts, among them J1 ROCKETNET-CONNECTOR-16M, J10 UART Header, J11 I2C Header, J12 BOOT1 Jumper, J13 PGOOD Jumper, J14 ROCKETNET-UMBILICAL-18, J15 Auxiliary Header, J16 Auxiliary Header, J17 Auxiliary Header, J18 Auxiliary Header, J19 Auxiliary Header, J2 ROCKETNET-CONNECTOR-16M, J20 Auxiliary Header, J21 Auxiliary Header, J22 Debug Header, J3 ROCKETNET-CONNECTOR-16M, J4 ROCKETNET-CONNECTOR-16M, J5 BOOT0 Jumper, J6 ROCKETNET-CONNECTOR-16M, J7 ROCKETNET-CONNECTOR-16M, J8 ROCKETNET-CONNECTOR-16M, J9 ROCKETNET-BATTERY-14, Q2 FDS6680ASOIC8, Q3 FDS6680ASOIC8, Q4 FDS6680ASOIC8, Q5 SIS412DNSOP-8, Q6 BSS138W-7-F, Q7 SIS412DNSOP-8, T1 BSS84, T10 ALT4532, T11 ALT4532, T12 ALT4532, T13 ALT4532, T14 ALT4532, T15 ALT4532, T16 ALT4532, T17 ALT4532, T18 ALT4532, T19 BSS84, T2 NDS335N, T20 NDS335N, T3 ALT4532, T4 ALT4532, T5 ALT4532, T6 ALT4532, T7 ALT4532, T8 ALT4532, T9 ALT4532, U1 STM32F407V100-PIN_QFP, U10 TPS2420QFN-16, U11 TPS2420QFN-16, U12 TPS2420QFN-16, U13 TPS2420QFN-16, U14 MAX4734ETC+, U15 MAX4734ETC+, U2 BQ24725QFN-20, U3 SN65220DBV, U4 KS8999, U5 LTM8023, U6 MIC37101-2.1YM, U7 TPS2420QFN-16, U8 TPS2420QFN-16, U9 TPS2420QFN-16

Commit message: Added R25 in 25 MHz clock line.
Parts:
- added R25: 200, rcl_custom:R-US_0402-B-NOSILK
Connections:
- removed net 25MHZ_REF_CLK: U1.PC9, U4.X1
- new net 25MHZ_REF_CLK_KSZ: R25.1, U4.X1
- new net 25MHZ_REF_CLK_STM: R25.2, U1.PC9
Changed lines of the file:
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@@
 <part name="R18" library="rcl_custom" deviceset="R-US_" device="0402-B-NOSILK" value="10k"/>
 <part name="GND9" library="supply1" deviceset="GND" device=""/>
+<part name="R25" library="rcl_custom" deviceset="R-US_" device="0402-B-NOSILK" value="200"/>
 </parts>
 <sheets>
@@
 <instance part="J11" gate="J" x="-12.7" y="358.14" rot="MR0"/>
 <instance part="GND8" gate="1" x="-5.08" y="350.52"/>
+<instance part="R25" gate="R" x="182.88" y="414.02" rot="R180"/>
 </instances>
 <busses>
@@
 </segment>
 </net>
-<net name="25MHZ_REF_CLK" class="0">
-<segment>
-<pinref part="U1" gate="U1" pin="PC9"/>
-<wire x1="154.94" y1="398.78" x2="152.4" y2="398.78" width="0.1524" layer="91"/>
-<label x="154.94" y="398.78" size="1.016" layer="95" xref="yes"/>
-</segment>
-</net>
 <net name="NODE7_!FLT" class="0">
 <segment>
@@
 </segment>
 </net>
+<net name="25MHZ_REF_CLK_KSZ" class="0">
+<segment>
+<wire x1="190.5" y1="414.02" x2="187.96" y2="414.02" width="0.1524" layer="91"/>
+<pinref part="R25" gate="R" pin="1"/>
+<label x="190.5" y="414.02" size="1.016" layer="95" xref="yes"/>
+</segment>
+</net>
+<net name="25MHZ_REF_CLK_STM" class="0">
+<segment>
+<pinref part="U1" gate="U1" pin="PC9"/>
+<wire x1="177.8" y1="414.02" x2="170.18" y2="414.02" width="0.1524" layer="91"/>
+<wire x1="170.18" y1="414.02" x2="170.18" y2="398.78" width="0.1524" layer="91"/>
+<wire x1="170.18" y1="398.78" x2="152.4" y2="398.78" width="0.1524" layer="91"/>
+<pinref part="R25" gate="R" pin="2"/>
+</segment>
+</net>
 </nets>
 </sheet>
@@
 </segment>
 </net>
-<net name="25MHZ_REF_CLK" class="0">
-<segment>
-<label x="-27.94" y="149.86" size="1.016" layer="95" rot="R180" xref="yes"/>
-<pinref part="U4" gate="U" pin="X1"/>
-<wire x1="-27.94" y1="149.86" x2="78.74" y2="149.86" width="0.1524" layer="91"/>
-</segment>
-</net>
 <net name="RX1_N" class="0">
 <segment>
@@
 </segment>
 </net>
+<net name="25MHZ_REF_CLK_KSZ" class="0">
+<segment>
+<pinref part="U4" gate="U" pin="X1"/>
+<wire x1="78.74" y1="149.86" x2="-5.08" y2="149.86" width="0.1524" layer="91"/>
+<wire x1="-5.08" y1="149.86" x2="-5.08" y2="144.78" width="0.1524" layer="91"/>
+<wire x1="-5.08" y1="144.78" x2="-12.7" y2="144.78" width="0.1524" layer="91"/>
+<label x="-12.7" y="144.78" size="1.778" layer="95" rot="R180" xref="yes"/>
+</segment>
+</net>

Commit message: Added diodes to power supply of BQ24725 so it's always on, even without shore power (duh!). Also cleaned up rocket ready circuitry.
Parts:
- added D6: BAT54C, diode:BAT54C
Connections:
- new net N$13: C105.1, C113.1, D6.CC, U2.VCC
- net +18V: now also D6.A1; no longer C105.1, C113.1, U2.VCC
- net VIN: now also D6.A2
Changed lines of the file:
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@@
 <layer number="2" name="Route2" color="9" fill="1" visible="no" active="no"/>
 <layer number="3" name="Route3" color="12" fill="1" visible="no" active="no"/>
+<layer number="4" name="Route4" color="1" fill="4" visible="no" active="no"/>
+<layer number="5" name="Route5" color="4" fill="4" visible="no" active="no"/>
+<layer number="6" name="Route6" color="1" fill="8" visible="no" active="no"/>
+<layer number="7" name="Route7" color="4" fill="8" visible="no" active="no"/>
+<layer number="8" name="Route8" color="1" fill="2" visible="no" active="no"/>
+<layer number="9" name="Route9" color="4" fill="2" visible="no" active="no"/>
+<layer number="10" name="Route10" color="1" fill="7" visible="no" active="no"/>
+<layer number="11" name="Route11" color="4" fill="7" visible="no" active="no"/>
+<layer number="12" name="Route12" color="1" fill="5" visible="no" active="no"/>
+<layer number="13" name="Route13" color="4" fill="5" visible="no" active="no"/>
 <layer number="14" name="Route14" color="11" fill="3" visible="no" active="no"/>
 <layer number="15" name="Route15" color="6" fill="1" visible="no" active="no"/>
@@
 <part name="GND9" library="supply1" deviceset="GND" device=""/>
 <part name="R25" library="rcl_custom" deviceset="R-US_" device="0402-B-NOSILK" value="200"/>
+<part name="D6" library="diode" deviceset="BAT54C" device=""/>
 </parts>
 <sheets>
@@
 <attribute name="VALUE" x="-17.78" y="12.7" size="1.778" layer="96" rot="R180"/>
 </instance>
+<instance part="D6" gate="G$1" x="48.26" y="60.96" rot="R180"/>
 </instances>
 <busses>
@@
 <pinref part="D5" gate="G$1" pin="C"/>
 <wire x1="-96.52" y1="58.42" x2="-96.52" y2="71.12" width="0.1524" layer="91"/>
-<wire x1="-96.52" y1="71.12" x2="-76.2" y2="71.12" width="0.1524" layer="91"/>
+<wire x1="-96.52" y1="71.12" x2="-86.36" y2="71.12" width="0.1524" layer="91"/>
 <pinref part="R137" gate="R" pin="2"/>
+<wire x1="-86.36" y1="71.12" x2="-76.2" y2="71.12" width="0.1524" layer="91"/>
 <wire x1="-76.2" y1="45.72" x2="-76.2" y2="71.12" width="0.1524" layer="91"/>
 <junction x="-76.2" y="71.12"/>
@@
 <wire x1="-50.8" y1="71.12" x2="-68.58" y2="71.12" width="0.1524" layer="91"/>
 <junction x="-68.58" y="71.12"/>
+<pinref part="D6" gate="G$1" pin="A2"/>
+<wire x1="43.18" y1="60.96" x2="40.64" y2="60.96" width="0.1524" layer="91"/>
+<wire x1="40.64" y1="60.96" x2="40.64" y2="106.68" width="0.1524" layer="91"/>
+<wire x1="40.64" y1="106.68" x2="-86.36" y2="106.68" width="0.1524" layer="91"/>
+<wire x1="-86.36" y1="106.68" x2="-86.36" y2="71.12" width="0.1524" layer="91"/>
+<junction x="-86.36" y="71.12"/>
 </segment>
 </net>
@@
 <wire x1="7.62" y1="71.12" x2="7.62" y2="48.26" width="0.1524" layer="91"/>
 <junction x="7.62" y="71.12"/>
-<wire x1="7.62" y1="71.12" x2="48.26" y2="71.12" width="0.1524" layer="91"/>
-<wire x1="48.26" y1="71.12" x2="48.26" y2="68.58" width="0.1524" layer="91"/>
-<junction x="48.26" y="71.12"/>
+<wire x1="7.62" y1="71.12" x2="58.42" y2="71.12" width="0.1524" layer="91"/>
 <label x="172.72" y="71.12" size="1.778" layer="95" xref="yes"/>
-<wire x1="48.26" y1="71.12" x2="86.36" y2="71.12" width="0.1524" layer="91"/>
 <pinref part="Q5" gate="&gt;NAME" pin="D"/>
+<wire x1="58.42" y1="71.12" x2="86.36" y2="71.12" width="0.1524" layer="91"/>
 <wire x1="86.36" y1="71.12" x2="91.44" y2="71.12" width="0.1524" layer="91"/>
 <wire x1="91.44" y1="71.12" x2="106.68" y2="71.12" width="0.1524" layer="91"/>
@@
 <wire x1="160.02" y1="45.72" x2="160.02" y2="71.12" width="0.1524" layer="91"/>
 <junction x="160.02" y="71.12"/>
-<pinref part="U2" gate="U" pin="VCC"/>
-<wire x1="45.72" y1="45.72" x2="48.26" y2="45.72" width="0.1524" layer="91"/>
-<wire x1="48.26" y1="45.72" x2="48.26" y2="55.88" width="0.1524" layer="91"/>
-<pinref part="C113" gate="CE" pin="1"/>
-<wire x1="48.26" y1="55.88" x2="48.26" y2="58.42" width="0.1524" layer="91"/>
-<junction x="48.26" y="55.88"/>
-<wire x1="48.26" y1="55.88" x2="48.26" y2="71.12" width="0.1524" layer="91"/>
 <pinref part="C124" gate="CE" pin="1"/>
 <wire x1="152.4" y1="68.58" x2="152.4" y2="71.12" width="0.1524" layer="91"/>
@@
 <wire x1="91.44" y1="68.58" x2="91.44" y2="71.12" width="0.1524" layer="91"/>
 <junction x="91.44" y="71.12"/>
-<pinref part="C105" gate="CE" pin="1"/>
 <pinref part="P+2" gate="1" pin="+18V"/>
 <wire x1="170.18" y1="81.28" x2="170.18" y2="71.12" width="0.1524" layer="91"/>
 <junction x="170.18" y="71.12"/>
-<junction x="58.42" y="55.88"/>
-<wire x1="58.42" y1="55.88" x2="73.66" y2="55.88" width="0.1524" layer="91"/>
-<wire x1="58.42" y1="55.88" x2="48.26" y2="55.88" width="0.1524" layer="91"/>
+<pinref part="D6" gate="G$1" pin="A1"/>
+<wire x1="53.34" y1="60.96" x2="58.42" y2="60.96" width="0.1524" layer="91"/>
+<wire x1="58.42" y1="60.96" x2="58.42" y2="71.12" width="0.1524" layer="91"/>
+<junction x="58.42" y="71.12"/>
 </segment>
 </net>
@@
 </segment>
 </net>
+<net name="N$13" class="1">
+<segment>
+<pinref part="C105" gate="CE" pin="1"/>
+<pinref part="C113" gate="CE" pin="1"/>
+<junction x="58.42" y="55.88"/>
+<wire x1="58.42" y1="55.88" x2="73.66" y2="55.88" width="0.1524" layer="91"/>
+<wire x1="58.42" y1="55.88" x2="48.26" y2="55.88" width="0.1524" layer="91"/>
+<wire x1="48.26" y1="45.72" x2="48.26" y2="55.88" width="0.1524" layer="91"/>
+<pinref part="U2" gate="U" pin="VCC"/>
+<wire x1="45.72" y1="45.72" x2="48.26" y2="45.72" width="0.1524" layer="91"/>
+<pinref part="D6" gate="G$1" pin="CC"/>
+<wire x1="48.26" y1="58.42" x2="48.26" y2="55.88" width="0.1524" layer="91"/>
+<junction x="48.26" y="55.88"/>
+</segment>
+</net>

Commit message: Cleaned up current sense resistor circuitry.
Parts:
- R143, R144: device rcl_custom:R-US_0603-B-NOSILK -> rcl_custom:R-US_0402-B-NOSILK
Other:
- moved on the sheet: C112
Changed lines of the file:
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@@
 <part name="GND86" library="supply1" deviceset="GND" device=""/>
 <part name="+3V33" library="supply1" deviceset="+3V3" device=""/>
-<part name="R143" library="rcl_custom" deviceset="R-US_" device="0603-B-NOSILK" value="7.5"/>
-<part name="R144" library="rcl_custom" deviceset="R-US_" device="0603-B-NOSILK" value="10"/>
+<part name="R143" library="rcl_custom" deviceset="R-US_" device="0402-B-NOSILK" value="7.5"/>
+<part name="R144" library="rcl_custom" deviceset="R-US_" device="0402-B-NOSILK" value="10"/>
 <part name="C111" library="rcl_custom" deviceset="C-EU" device="0402-B-NOSILK" value="0.1uF"/>
 <part name="C112" library="rcl_custom" deviceset="C-EU" device="0402-B-NOSILK" value="0.1uF"/>
@@
 <attribute name="VALUE" x="138.684" y="-19.939" size="1.778" layer="96"/>
 </instance>
-<instance part="C112" gate="CE" x="162.56" y="-25.4" smashed="yes">
-<attribute name="NAME" x="164.084" y="-25.019" size="1.778" layer="95"/>
-<attribute name="VALUE" x="164.084" y="-30.099" size="1.778" layer="96"/>
+<instance part="C112" gate="CE" x="137.16" y="-22.86" smashed="yes">
+<attribute name="NAME" x="138.684" y="-22.479" size="1.778" layer="95"/>
+<attribute name="VALUE" x="138.684" y="-27.559" size="1.778" layer="96"/>
 </instance>
 <instance part="C113" gate="CE" x="58.42" y="53.34" smashed="yes">
@@
 <attribute name="VALUE" x="83.82" y="-12.7" size="1.778" layer="96"/>
 </instance>
-<instance part="GND90" gate="1" x="162.56" y="-35.56" smashed="yes">
-<attribute name="VALUE" x="160.02" y="-38.1" size="1.778" layer="96"/>
+<instance part="GND90" gate="1" x="137.16" y="-33.02" smashed="yes">
+<attribute name="VALUE" x="134.62" y="-35.56" size="1.778" layer="96"/>
 </instance>
 <instance part="R146" gate="R" x="149.86" y="7.62" smashed="yes">
@@
 <pinref part="C112" gate="CE" pin="2"/>
 <pinref part="GND90" gate="1" pin="GND"/>
-<wire x1="162.56" y1="-33.02" x2="162.56" y2="-30.48" width="0.1524" layer="91"/>
+<wire x1="137.16" y1="-30.48" x2="137.16" y2="-27.94" width="0.1524" layer="91"/>
 </segment>
 <segment>
@@
 <wire x1="154.94" y1="7.62" x2="160.02" y2="7.62" width="0.1524" layer="91"/>
 <pinref part="C120" gate="CE" pin="1"/>
-<wire x1="160.02" y1="7.62" x2="162.56" y2="7.62" width="0.1524" layer="91"/>
-<wire x1="162.56" y1="7.62" x2="172.72" y2="7.62" width="0.1524" layer="91"/>
+<wire x1="160.02" y1="7.62" x2="172.72" y2="7.62" width="0.1524" layer="91"/>
 <wire x1="172.72" y1="7.62" x2="185.42" y2="7.62" width="0.1524" layer="91"/>
 <junction x="172.72" y="7.62"/>
@@
 <junction x="185.42" y="7.62"/>
 <pinref part="C112" gate="CE" pin="1"/>
-<wire x1="162.56" y1="-22.86" x2="162.56" y2="-20.32" width="0.1524" layer="91"/>
-<junction x="162.56" y="7.62"/>
-<wire x1="162.56" y1="-20.32" x2="162.56" y2="7.62" width="0.1524" layer="91"/>
 <pinref part="C111" gate="CE" pin="2"/>
 <pinref part="R143" gate="R" pin="2"/>
 <wire x1="132.08" y1="-20.32" x2="137.16" y2="-20.32" width="0.1524" layer="91"/>
-<wire x1="137.16" y1="-20.32" x2="162.56" y2="-20.32" width="0.1524" layer="91"/>
 <junction x="137.16" y="-20.32"/>
-<junction x="162.56" y="-20.32"/>
 <pinref part="Q4" gate="&gt;NAME" pin="S"/>
 <wire x1="160.02" y1="22.86" x2="160.02" y2="33.02" width="0.1524" layer="91"/>
@@
 <junction x="160.02" y="22.86"/>
 <junction x="160.02" y="7.62"/>
+<wire x1="154.94" y1="7.62" x2="154.94" y2="-20.32" width="0.1524" layer="91"/>
+<junction x="154.94" y="7.62"/>
+<wire x1="137.16" y1="-20.32" x2="154.94" y2="-20.32" width="0.1524" layer="91"/>
 </segment>
 </net>
@@
 <wire x1="132.08" y1="-12.7" x2="137.16" y2="-12.7" width="0.1524" layer="91"/>
 <pinref part="R146" gate="R" pin="1"/>
-<wire x1="132.08" y1="7.62" x2="137.16" y2="7.62" width="0.1524" layer="91"/>
 <pinref part="L1" gate="L" pin="P$1"/>
-<wire x1="137.16" y1="7.62" x2="144.78" y2="7.62" width="0.1524" layer="91"/>
-<wire x1="137.16" y1="-12.7" x2="137.16" y2="7.62" width="0.1524" layer="91"/>
+<wire x1="132.08" y1="7.62" x2="144.78" y2="7.62" width="0.1524" layer="91"/>
 <junction x="137.16" y="-12.7"/>
-<junction x="137.16" y="7.62"/>
+<wire x1="144.78" y1="7.62" x2="144.78" y2="-12.7" width="0.1524" layer="91"/>
+<wire x1="144.78" y1="-12.7" x2="137.16" y2="-12.7" width="0.1524" layer="91"/>
+<junction x="144.78" y="7.62"/>
 </segment>
 </net>

Commit message: Huge cleanup of power planes and vias. Removed secondary ground planes around KSZ, which was causing DRC errors.
Changed lines of the file:
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@@
 <segment>
 <pinref part="U5" gate="U" pin="SYNC"/>
-<wire x1="-20.32" y1="-20.32" x2="-20.32" y2="-25.4" width="0.1524" layer="91"/>
-<label x="-20.32" y="-25.4" size="1.27" layer="95" rot="R180" xref="yes"/>
+<wire x1="-20.32" y1="-20.32" x2="-20.32" y2="-22.86" width="0.1524" layer="91"/>
 <pinref part="R131" gate="R" pin="1"/>
+<wire x1="-20.32" y1="-22.86" x2="-20.32" y2="-25.4" width="0.1524" layer="91"/>
+<wire x1="-20.32" y1="-22.86" x2="-27.94" y2="-22.86" width="0.1524" layer="91"/>
+<junction x="-20.32" y="-22.86"/>
+<label x="-27.94" y="-22.86" size="1.778" layer="95" rot="R180" xref="yes"/>
 </segment>
 </net>

Commit message: more power plane cleanup, now of the 2.1V area around the KSZ.
Other:
- moved on the sheet: C12, C13, C14, C15, C77, D1, R42, R43, T1, T2
