File: av3/rocketnet-hub/eagle/mcu_page_combined_routed.sch (EAGLE design)
At the start: 443 parts, among them J1 ROCKETNET-CONNECTOR-16M, J10 UART Header, J11 I2C Header, J12 BOOT1 Jumper, J13 PGOOD Jumper, J14 ROCKETNET-UMBILICAL-18, J15 Auxiliary Header, J16 Auxiliary Header, J17 Auxiliary Header, J18 Auxiliary Header, J19 Auxiliary Header, J2 ROCKETNET-CONNECTOR-16M, J20 Auxiliary Header, J21 Auxiliary Header, J22 Debug Header, J3 ROCKETNET-CONNECTOR-16M, J4 ROCKETNET-CONNECTOR-16M, J5 BOOT0 Jumper, J6 ROCKETNET-CONNECTOR-16M, J7 ROCKETNET-CONNECTOR-16M, J8 ROCKETNET-CONNECTOR-16M, J9 ROCKETNET-BATTERY-14, Q2 FDS6680ASOIC8, Q3 FDS6680ASOIC8, Q4 FDS6680ASOIC8, Q5 SIS412DNSOP-8, Q6 BSS138W-7-F, Q7 SIS412DNSOP-8, T1 BSS84, T10 ALT4532, T11 ALT4532, T12 ALT4532, T13 ALT4532, T14 ALT4532, T15 ALT4532, T16 ALT4532, T17 ALT4532, T18 ALT4532, T19 BSS84, T2 NDS335N, T20 NDS335N, T3 ALT4532, T4 ALT4532, T5 ALT4532, T6 ALT4532, T7 ALT4532, T8 ALT4532, T9 ALT4532, U1 STM32F407V100-PIN_QFP, U10 TPS2420QFN-16, U11 TPS2420QFN-16, U12 TPS2420QFN-16, U13 TPS2420QFN-16, U14 MAX4734ETC+, U15 MAX4734ETC+, U2 BQ24725QFN-20, U3 SN65220DBV, U4 KS8999, U5 LTM8023, U6 MIC37101-2.1YM, U7 TPS2420QFN-16, U8 TPS2420QFN-16, U9 TPS2420QFN-16

Commit message: More tweaking around KSZ, distributed capacitors, simplified some runs.
Other:
- moved on the sheet: C78, C79, C80, C81, C82
Changed lines of the file:
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@@
 <instance part="C76" gate="CE" x="172.72" y="259.08"/>
 <instance part="C77" gate="CE" x="68.58" y="248.92" rot="R180"/>
-<instance part="C78" gate="CE" x="101.6" y="274.32"/>
-<instance part="C79" gate="CE" x="121.92" y="274.32"/>
-<instance part="C80" gate="CE" x="142.24" y="274.32"/>
-<instance part="C81" gate="CE" x="162.56" y="274.32"/>
-<instance part="C82" gate="CE" x="172.72" y="274.32"/>
+<instance part="C78" gate="CE" x="101.6" y="274.32" rot="MR180"/>
+<instance part="C79" gate="CE" x="121.92" y="274.32" rot="MR180"/>
+<instance part="C80" gate="CE" x="142.24" y="274.32" rot="MR180"/>
+<instance part="C81" gate="CE" x="162.56" y="274.32" rot="MR180"/>
+<instance part="C82" gate="CE" x="172.72" y="274.32" rot="MR180"/>
 <instance part="GND13" gate="1" x="73.66" y="236.22"/>
 <instance part="T1" gate="A" x="35.56" y="274.32" rot="MR180"/>
@@
 <instance part="ETHERNET_SWITCH" gate="G$2" x="342.9" y="-60.96"/>
 <instance part="D1" gate="G$1" x="-2.54" y="279.4"/>
-<instance part="+2V1" gate="G$1" x="185.42" y="276.86"/>
+<instance part="+2V1" gate="G$1" x="185.42" y="284.48"/>
 <instance part="+2V11" gate="G$1" x="2.54" y="198.12"/>
 <instance part="+2V12" gate="G$1" x="60.96" y="238.76"/>
@@
 <instance part="T20" gate="A" x="198.12" y="266.7"/>
 <instance part="+3V41" gate="G$1" x="198.12" y="299.72"/>
-<instance part="GND43" gate="1" x="91.44" y="274.32"/>
+<instance part="GND43" gate="1" x="142.24" y="266.7" rot="MR0"/>
 <instance part="GND149" gate="1" x="93.98" y="259.08"/>
 <instance part="GND150" gate="1" x="68.58" y="243.84"/>
@@
 <pinref part="C82" gate="CE" pin="1"/>
 <pinref part="C81" gate="CE" pin="1"/>
-<wire x1="162.56" y1="276.86" x2="172.72" y2="276.86" width="0.1524" layer="91"/>
-<junction x="162.56" y="276.86"/>
+<wire x1="162.56" y1="271.78" x2="172.72" y2="271.78" width="0.1524" layer="91"/>
+<junction x="162.56" y="271.78"/>
 <pinref part="C80" gate="CE" pin="1"/>
-<wire x1="142.24" y1="276.86" x2="162.56" y2="276.86" width="0.1524" layer="91"/>
-<junction x="142.24" y="276.86"/>
+<wire x1="142.24" y1="271.78" x2="162.56" y2="271.78" width="0.1524" layer="91"/>
+<junction x="142.24" y="271.78"/>
 <pinref part="C79" gate="CE" pin="1"/>
-<wire x1="121.92" y1="276.86" x2="142.24" y2="276.86" width="0.1524" layer="91"/>
-<junction x="121.92" y="276.86"/>
+<wire x1="121.92" y1="271.78" x2="142.24" y2="271.78" width="0.1524" layer="91"/>
+<junction x="121.92" y="271.78"/>
 <pinref part="C78" gate="CE" pin="1"/>
-<wire x1="101.6" y1="276.86" x2="121.92" y2="276.86" width="0.1524" layer="91"/>
-<junction x="101.6" y="276.86"/>
+<wire x1="101.6" y1="271.78" x2="121.92" y2="271.78" width="0.1524" layer="91"/>
 <pinref part="GND43" gate="1" pin="GND"/>
-<wire x1="91.44" y1="276.86" x2="101.6" y2="276.86" width="0.1524" layer="91"/>
+<wire x1="142.24" y1="269.24" x2="142.24" y2="271.78" width="0.1524" layer="91"/>
 </segment>
 <segment>
@@
 <segment>
 <pinref part="+2V1" gate="G$1" pin="+2V1"/>
-<wire x1="185.42" y1="274.32" x2="185.42" y2="269.24" width="0.1524" layer="91"/>
+<wire x1="185.42" y1="281.94" x2="185.42" y2="279.4" width="0.1524" layer="91"/>
 <pinref part="C71" gate="CE" pin="2"/>
 <pinref part="U4" gate="U" pin="VDD_RCV"/>
@@
 <junction x="142.24" y="243.84"/>
 <wire x1="142.24" y1="254" x2="139.7" y2="254" width="0.1524" layer="91"/>
-<wire x1="139.7" y1="254" x2="139.7" y2="266.7" width="0.1524" layer="91"/>
+<wire x1="139.7" y1="254" x2="139.7" y2="279.4" width="0.1524" layer="91"/>
 <junction x="142.24" y="254"/>
 <pinref part="C80" gate="CE" pin="2"/>
-<wire x1="139.7" y1="266.7" x2="142.24" y2="266.7" width="0.1524" layer="91"/>
-<wire x1="142.24" y1="266.7" x2="142.24" y2="269.24" width="0.1524" layer="91"/>
-<junction x="142.24" y="269.24"/>
+<wire x1="139.7" y1="279.4" x2="142.24" y2="279.4" width="0.1524" layer="91"/>
+<junction x="142.24" y="279.4"/>
 <pinref part="C24" gate="CE" pin="2"/>
 <pinref part="U4" gate="U" pin="VDD_RX7"/>
@@
 <pinref part="C79" gate="CE" pin="2"/>
 <wire x1="121.92" y1="243.84" x2="121.92" y2="238.76" width="0.1524" layer="91"/>
-<wire x1="121.92" y1="269.24" x2="121.92" y2="266.7" width="0.1524" layer="91"/>
-<wire x1="121.92" y1="266.7" x2="119.38" y2="266.7" width="0.1524" layer="91"/>
-<wire x1="119.38" y1="266.7" x2="119.38" y2="254" width="0.1524" layer="91"/>
+<wire x1="121.92" y1="279.4" x2="119.38" y2="279.4" width="0.1524" layer="91"/>
+<wire x1="119.38" y1="279.4" x2="119.38" y2="254" width="0.1524" layer="91"/>
 <wire x1="119.38" y1="254" x2="121.92" y2="254" width="0.1524" layer="91"/>
 <junction x="121.92" y="254"/>
@@
 <wire x1="137.16" y1="243.84" x2="139.7" y2="243.84" width="0.1524" layer="91"/>
 <junction x="139.7" y="243.84"/>
-<wire x1="142.24" y1="269.24" x2="121.92" y2="269.24" width="0.1524" layer="91"/>
-<junction x="121.92" y="269.24"/>
+<wire x1="142.24" y1="279.4" x2="139.7" y2="279.4" width="0.1524" layer="91"/>
+<junction x="121.92" y="279.4"/>
 <pinref part="C78" gate="CE" pin="2"/>
-<wire x1="101.6" y1="269.24" x2="101.6" y2="266.7" width="0.1524" layer="91"/>
-<wire x1="101.6" y1="266.7" x2="99.06" y2="266.7" width="0.1524" layer="91"/>
+<wire x1="139.7" y1="279.4" x2="121.92" y2="279.4" width="0.1524" layer="91"/>
+<wire x1="101.6" y1="279.4" x2="99.06" y2="279.4" width="0.1524" layer="91"/>
 <pinref part="C16" gate="CE" pin="2"/>
-<wire x1="99.06" y1="266.7" x2="99.06" y2="254" width="0.1524" layer="91"/>
+<wire x1="99.06" y1="279.4" x2="99.06" y2="254" width="0.1524" layer="91"/>
 <wire x1="99.06" y1="254" x2="101.6" y2="254" width="0.1524" layer="91"/>
 <pinref part="U4" gate="U" pin="VDD_TX7"/>
@@
 <wire x1="116.84" y1="243.84" x2="119.38" y2="243.84" width="0.1524" layer="91"/>
 <junction x="119.38" y="243.84"/>
-<wire x1="121.92" y1="269.24" x2="101.6" y2="269.24" width="0.1524" layer="91"/>
-<junction x="101.6" y="269.24"/>
+<wire x1="121.92" y1="279.4" x2="119.38" y2="279.4" width="0.1524" layer="91"/>
+<junction x="101.6" y="279.4"/>
 <pinref part="C18" gate="CE" pin="2"/>
-<wire x1="172.72" y1="269.24" x2="162.56" y2="269.24" width="0.1524" layer="91"/>
-<wire x1="162.56" y1="269.24" x2="142.24" y2="269.24" width="0.1524" layer="91"/>
+<wire x1="119.38" y1="279.4" x2="101.6" y2="279.4" width="0.1524" layer="91"/>
+<wire x1="172.72" y1="279.4" x2="170.18" y2="279.4" width="0.1524" layer="91"/>
+<wire x1="170.18" y1="279.4" x2="162.56" y2="279.4" width="0.1524" layer="91"/>
+<wire x1="162.56" y1="279.4" x2="160.02" y2="279.4" width="0.1524" layer="91"/>
+<wire x1="160.02" y1="279.4" x2="142.24" y2="279.4" width="0.1524" layer="91"/>
 <wire x1="101.6" y1="254" x2="106.68" y2="254" width="0.1524" layer="91"/>
 <pinref part="C20" gate="CE" pin="2"/>
@@
 <pinref part="U4" gate="U" pin="VDD"/>
 <pinref part="C82" gate="CE" pin="2"/>
-<wire x1="172.72" y1="266.7" x2="172.72" y2="269.24" width="0.1524" layer="91"/>
-<wire x1="170.18" y1="266.7" x2="172.72" y2="266.7" width="0.1524" layer="91"/>
-<wire x1="170.18" y1="254" x2="170.18" y2="266.7" width="0.1524" layer="91"/>
+<wire x1="170.18" y1="279.4" x2="172.72" y2="279.4" width="0.1524" layer="91"/>
+<wire x1="170.18" y1="254" x2="170.18" y2="279.4" width="0.1524" layer="91"/>
 <pinref part="C76" gate="CE" pin="2"/>
 <wire x1="172.72" y1="254" x2="170.18" y2="254" width="0.1524" layer="91"/>
@@
 <pinref part="C72" gate="CE" pin="2"/>
 <pinref part="C81" gate="CE" pin="2"/>
-<wire x1="162.56" y1="269.24" x2="162.56" y2="266.7" width="0.1524" layer="91"/>
-<wire x1="160.02" y1="266.7" x2="162.56" y2="266.7" width="0.1524" layer="91"/>
-<wire x1="160.02" y1="266.7" x2="160.02" y2="254" width="0.1524" layer="91"/>
+<wire x1="160.02" y1="279.4" x2="162.56" y2="279.4" width="0.1524" layer="91"/>
+<wire x1="160.02" y1="279.4" x2="160.02" y2="254" width="0.1524" layer="91"/>
 <wire x1="160.02" y1="254" x2="162.56" y2="254" width="0.1524" layer="91"/>
 <junction x="162.56" y="254"/>
 <wire x1="162.56" y1="254" x2="162.56" y2="243.84" width="0.1524" layer="91"/>
-<junction x="162.56" y="269.24"/>
-<junction x="172.72" y="269.24"/>
+<junction x="162.56" y="279.4"/>
+<junction x="172.72" y="279.4"/>
 <wire x1="162.56" y1="243.84" x2="162.56" y2="238.76" width="0.1524" layer="91"/>
 <wire x1="119.38" y1="243.84" x2="121.92" y2="243.84" width="0.1524" layer="91"/>
@@
 <junction x="162.56" y="243.84"/>
 <wire x1="165.1" y1="243.84" x2="162.56" y2="243.84" width="0.1524" layer="91"/>
-<wire x1="185.42" y1="269.24" x2="172.72" y2="269.24" width="0.1524" layer="91"/>
-<wire x1="185.42" y1="269.24" x2="185.42" y2="264.16" width="0.1524" layer="91"/>
-<junction x="185.42" y="269.24"/>
+<wire x1="185.42" y1="279.4" x2="172.72" y2="279.4" width="0.1524" layer="91"/>
+<wire x1="185.42" y1="279.4" x2="185.42" y2="264.16" width="0.1524" layer="91"/>
+<junction x="185.42" y="279.4"/>
 <pinref part="T20" gate="A" pin="G"/>
 <wire x1="185.42" y1="264.16" x2="193.04" y2="264.16" width="0.1524" layer="91"/>
-</segment>
-</net>
+<junction x="170.18" y="279.4"/>
+<junction x="160.02" y="279.4"/>
+<junction x="139.7" y="279.4"/>
+<junction x="119.38" y="279.4"/>
+</segment>
+</net>

Commit message: Cleanup around STM32 - JTAG, UART. Replaced small signal N and P channel MOSFETs with known parts.
Parts:
- removed T1, T19: BSS84, zetex:PMOSSOT23
- removed T2: NDS335N, zetex:NMOSSOT23
- added Q1: NTR401P, Tova:NTR4101P
- added Q8: PMV45EN, Tova:PMV45EN
- added Q9: NTR4101P, Tova:NTR4101P
Connections:
- net +3V3: now also Q1.S, Q9.S; no longer T1.S, T19.S
- net GND: now also Q8.S; no longer T2.S
- net N$16: now also Q8.D, Q9.G; no longer T1.G, T2.D
- net N$28: now also Q8.G; no longer T2.G
- net N$31: now also Q1.D; no longer T19.D
- net ROCKET_RDY_MCU: now also Q1.G; no longer T19.G
- net VDDIO_IN: now also Q9.D; no longer T1.D
Changed lines of the file:
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@@
 <part name="C82" library="rcl_custom" deviceset="C-EU" device="0603-A-NOSILK" value="10u"/>
 <part name="GND13" library="supply1" deviceset="GND" device=""/>
-<part name="T1" library="zetex" deviceset="PMOSSOT23" device="" value="BSS84"/>
+<part name="Q9" library="Tova" deviceset="NTR4101P" device="" value="NTR4101P"/>
 <part name="R42" library="rcl_custom" deviceset="R-US_" device="0402-B-NOSILK" value="10k"/>
 <part name="+3V5" library="supply1" deviceset="+3V3" device=""/>
-<part name="T2" library="zetex" deviceset="NMOSSOT23" device="" value="NDS335N"/>
+<part name="Q8" library="Tova" deviceset="PMV45EN" device="" value="PMV45EN"/>
 <part name="C12" library="rcl_custom" deviceset="C-EU" device="0402-B-NOSILK" value="10n"/>
 <part name="GND11" library="supply1" deviceset="GND" device=""/>
@@
 <part name="L17" library="magnetics" deviceset="ACM2012" device=""/>
 <part name="GND100" library="supply1" deviceset="GND" device=""/>
-<part name="T19" library="zetex" deviceset="PMOSSOT23" device="" value="BSS84"/>
+<part name="Q1" library="Tova" deviceset="NTR4101P" device="" value="NTR401P"/>
 <part name="R147" library="rcl_custom" deviceset="R-US_" device="0402-B-NOSILK" value="1k"/>
 <part name="+3V37" library="supply1" deviceset="+3V3" device=""/>
@@
 <instance part="TP36" gate="G$1" x="43.18" y="370.84"/>
 <instance part="GND100" gate="1" x="40.64" y="386.08"/>
-<instance part="T19" gate="A" x="246.38" y="370.84" rot="MR180"/>
+<instance part="Q1" gate="G$1" x="246.38" y="370.84"/>
 <instance part="R147" gate="R" x="233.68" y="381" rot="R90"/>
 <instance part="+3V37" gate="G$1" x="246.38" y="388.62"/>
@@
 <segment>
 <pinref part="+3V37" gate="G$1" pin="+3V3"/>
-<pinref part="T19" gate="A" pin="S"/>
+<pinref part="Q1" gate="G$1" pin="S"/>
 <wire x1="246.38" y1="386.08" x2="246.38" y2="375.92" width="0.1524" layer="91"/>
 </segment>
@@
 <pinref part="R147" gate="R" pin="1"/>
 <wire x1="233.68" y1="375.92" x2="233.68" y2="373.38" width="0.1524" layer="91"/>
-<pinref part="T19" gate="A" pin="G"/>
+<pinref part="Q1" gate="G$1" pin="G"/>
 <wire x1="241.3" y1="373.38" x2="233.68" y2="373.38" width="0.1524" layer="91"/>
 <junction x="233.68" y="373.38"/>
@@
 <segment>
 <pinref part="R148" gate="R" pin="2"/>
-<pinref part="T19" gate="A" pin="D"/>
+<pinref part="Q1" gate="G$1" pin="D"/>
 <wire x1="246.38" y1="353.06" x2="246.38" y2="358.14" width="0.1524" layer="91"/>
 <wire x1="246.38" y1="358.14" x2="246.38" y2="365.76" width="0.1524" layer="91"/>
@@
 <description>Ethernet Switch</description>
 <plain>
-<wire x1="-43.18" y1="304.8" x2="50.8" y2="304.8" width="0.1524" layer="97" style="shortdash"/>
-<wire x1="50.8" y1="304.8" x2="50.8" y2="246.38" width="0.1524" layer="97" style="shortdash"/>
-<wire x1="50.8" y1="246.38" x2="-43.18" y2="246.38" width="0.1524" layer="97" style="shortdash"/>
+<wire x1="-43.18" y1="304.8" x2="53.34" y2="304.8" width="0.1524" layer="97" style="shortdash"/>
+<wire x1="53.34" y1="304.8" x2="53.34" y2="246.38" width="0.1524" layer="97" style="shortdash"/>
+<wire x1="53.34" y1="246.38" x2="-43.18" y2="246.38" width="0.1524" layer="97" style="shortdash"/>
 <wire x1="-43.18" y1="246.38" x2="-43.18" y2="304.8" width="0.1524" layer="97" style="shortdash"/>
 <text x="-12.7" y="299.72" size="1.778" layer="97">Ethernet Start-Up</text>
@@
 <instance part="C82" gate="CE" x="172.72" y="274.32" rot="MR180"/>
 <instance part="GND13" gate="1" x="73.66" y="236.22"/>
-<instance part="T1" gate="A" x="35.56" y="274.32" rot="MR180"/>
+<instance part="Q9" gate="G$1" x="35.56" y="274.32"/>
 <instance part="R42" gate="R" x="17.78" y="284.48" rot="R270"/>
 <instance part="+3V5" gate="G$1" x="35.56" y="299.72"/>
-<instance part="T2" gate="A" x="17.78" y="271.78"/>
+<instance part="Q8" gate="G$1" x="17.78" y="271.78"/>
 <instance part="C12" gate="CE" x="5.08" y="264.16"/>
 <instance part="GND11" gate="1" x="5.08" y="251.46"/>
@@
 <segment>
 <pinref part="GND14" gate="1" pin="GND"/>
-<pinref part="T2" gate="A" pin="S"/>
+<pinref part="Q8" gate="G$1" pin="S"/>
 <wire x1="17.78" y1="254" x2="17.78" y2="266.7" width="0.1524" layer="91"/>
 </segment>
@@
 </segment>
 <segment>
-<pinref part="T1" gate="A" pin="S"/>
+<pinref part="Q9" gate="G$1" pin="S"/>
 <pinref part="R42" gate="R" pin="1"/>
 <wire x1="35.56" y1="289.56" x2="35.56" y2="279.4" width="0.1524" layer="91"/>
@@
 <pinref part="R42" gate="R" pin="2"/>
 <wire x1="17.78" y1="276.86" x2="17.78" y2="279.4" width="0.1524" layer="91"/>
-<pinref part="T1" gate="A" pin="G"/>
+<pinref part="Q9" gate="G$1" pin="G"/>
 <wire x1="30.48" y1="276.86" x2="17.78" y2="276.86" width="0.1524" layer="91"/>
-<pinref part="T2" gate="A" pin="D"/>
+<pinref part="Q8" gate="G$1" pin="D"/>
 <junction x="17.78" y="276.86"/>
 </segment>
@@
 <wire x1="81.28" y1="241.3" x2="93.98" y2="241.3" width="0.1524" layer="91"/>
 <wire x1="93.98" y1="241.3" x2="93.98" y2="238.76" width="0.1524" layer="91"/>
-<pinref part="T1" gate="A" pin="D"/>
+<pinref part="Q9" gate="G$1" pin="D"/>
 <wire x1="35.56" y1="269.24" x2="35.56" y2="254" width="0.1524" layer="91"/>
 <wire x1="35.56" y1="254" x2="68.58" y2="254" width="0.1524" layer="91"/>
@@
 <net name="N$28" class="0">
 <segment>
-<pinref part="T2" gate="A" pin="G"/>
+<pinref part="Q8" gate="G$1" pin="G"/>
 <pinref part="R43" gate="R" pin="1"/>
 <wire x1="12.7" y1="269.24" x2="7.62" y2="269.24" width="0.1524" layer="91"/>
