File: av3/imu-adapter/imu-adapter-e407.brd (EAGLE design)
At the start: 63.5 x 35.6 mm, 22 parts, among them J1 CLM-112-02, P1 TSM-106-DV, P2 TSM-106-DV, P3 TSM-106-DV

Commit message: Final cleanup on imu adapter board before production tomorrow. Moved from 3x 6x2 connector to 1x 8x2. Added libraries locally.
Parts:
- removed P1, P2, P3: TSM-106-DV, con-samtec:TSM-106-DV
- added J2: TSM-116-DV, con-samtec:TSM-116-DV
Connections:
- removed net LPC-!EINT0: P2.1
- removed net LPC-!EINT1: P2.3
- removed net LPC-!RST: P2.2
- removed net LPC-DIO4: P1.2
- removed net LPC-MOSI: P1.5
- removed net LPC-SCLK: P1.3
- removed net LPC-SSEL: P1.6
- removed net PD14: P1.1
- net +3V3: now also J2.13, J2.14; no longer P3.1, P3.2
- net +5V: now also J2.11, J2.12; no longer P2.5, P2.6
- net E407-D10: now also J2.6
- net E407-D11: now also J2.5
- net E407-D12: now also J2.4; no longer P1.4
- net E407-D13: now also J2.3
- net E407-PD11: now also J2.8
- net E407-PD12: now also J2.7
- net E407-PD13: now also J2.9
- net E407-PD14: now also J2.1
- net E407-PD15: now also J2.2
- net GND: now also J2.10, J2.15, J2.16; no longer P2.4, P3.3, P3.4
Routing:
- net E407-PD11: track 0.00 -> 37.5 mm
- net E407-D10: track 0.00 -> 29.8 mm
- net LPC-!RST: track 28.6 -> 0.00 mm
- net LPC-SSEL: track 24.3 -> 0.00 mm
- net E407-PD15: track 0.00 -> 14.3 mm
- net E407-PD14: track 0.00 -> 12.8 mm
- net E407-D11: track 0.00 -> 11.2 mm
- net LPC-MOSI: track 11.2 -> 0.00 mm
- net E407-PD13: track 0.00 -> 11.2 mm
- net E407-D13: track 0.00 -> 8.54 mm
- net PD14: track 7.99 -> 0.00 mm
- net E407-PD12: track 0.00 -> 7.61 mm
- net LPC-DIO4: track 5.98 -> 0.00 mm
- net LPC-SCLK: track 5.79 -> 0.00 mm
- net LPC-!EINT1: track 5.35 -> 0.00 mm
Other:
- board text added: "ADIS IMU BREAKOUT"
- board text added: "FOR E407"
- board text removed: "ADIS IMU"
- board text removed: "BREAKOUT FOR E407"
