File: av3/imu-adapter/imu-adapter-e407.sch (EAGLE design)
At the start: 22 parts, among them J1 CLM-112-02, P1 TSM-106-DV, P2 TSM-106-DV, P3 TSM-106-DV

Commit message: Final cleanup on imu adapter board before production tomorrow. Moved from 3x 6x2 connector to 1x 8x2. Added libraries locally.
Parts:
- removed P1, P2, P3: TSM-106-DV, con-samtec:TSM-106-DV
- added J2: TSM-116-DV, con-samtec:TSM-116-DV
Connections:
- removed net LPC-!EINT0: P2.1
- removed net LPC-!EINT1: P2.3
- removed net LPC-!RST: P2.2
- removed net LPC-DIO4: P1.2
- removed net LPC-MOSI: P1.5
- removed net LPC-SCLK: P1.3
- removed net LPC-SSEL: P1.6
- removed net PD14: P1.1
- net +3V3: now also J2.13, J2.14; no longer P3.1, P3.2
- net +5V: now also J2.11, J2.12; no longer P2.5, P2.6
- net E407-D10: now also J2.6
- net E407-D11: now also J2.5
- net E407-D12: now also J2.4; no longer P1.4
- net E407-D13: now also J2.3
- net E407-PD11: now also J2.8
- net E407-PD12: now also J2.7
- net E407-PD13: now also J2.9
- net E407-PD14: now also J2.1
- net E407-PD15: now also J2.2
- net GND: now also J2.10, J2.15, J2.16; no longer P2.4, P3.3, P3.4
Other:
- moved on the sheet: TP5

Commit message: Added stupid EAGLE temporary files to the gitignore. Updated IMU adapter with sane net names so we could easily trace nets. And updated the e407 shield to add a RGB LED, correct some schematic mistakes found out while double checking connections, and updated to being routable on a PCB router.
Connections:
- net E407-D10 renamed ADIS-!CS!-!SS
- net E407-D11 renamed ADIS-DIN-MOSI
- net E407-D12 renamed ADIS-DOUT-MISO
- net E407-D13 renamed ADIS-SCLK
- net E407-PD11 renamed ADIS-!RST
- net E407-PD12 renamed ADIS-DIO1-INT
- net E407-PD13 renamed ADIS-DIO2-NC
- net E407-PD14 renamed ADIS-DIO3-NC
- net E407-PD15 renamed ADIS-DIO4-NC
Other:
- moved on the sheet: C1, J1, J2, R1, R10, R11, R12, R2, R3, R4, R5, R6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
