File: av3/rocketnet-connector/eagle/rocketnet-test.brd (EAGLE design)
At the start: 30 x 20 mm, 2 parts, among them J1 ROCKETNET-CONNECTOR-16M

Commit message: Updated rocketnet connectors and boards to match new rocketnet stackup.
Parts:
- J1: device rocketnet-connector:ROCKNET-CONNECTOR-M-16 -> rocketnet-connector:ROCKETNET-M-16
Connections:
- removed net N$1: J1.T+@11, J1.T+@9, JP2.5
- new net N$11: J1.T+@13, J1.T+@14, JP2.4
- net N$2: now also J1.R+@5, J1.R+@7; no longer J1.R-@5, J1.R-@7
- net N$3: now also J1.R-@3, J1.R-@4; no longer J1.R+@1, J1.R+@3
- net N$4: now also J1.T-@11, J1.T-@9, JP2.5; no longer J1.T-@13, J1.T-@15, JP2.4
- net N$5: now also J1.B+@15, J1.B+@16, JP2.1; no longer J1.B+@2, J1.B+@4, JP2.10
- net N$6: now also J1.B-@1, J1.B-@2, JP2.10; no longer J1.B-@14, J1.B-@16, JP2.1
Routing:
- net N$11: track 0.00 -> 12.0 mm
- net N$1: track 11.9 -> 0.00 mm
- net N$5: track 24.6 -> 16.0 mm
- net N$6: track 24.2 -> 16.1 mm
- net N$3: track 11.9 -> 12.4 mm
Changed lines of the file:
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@@
 </autorouter>
 <elements>
-<element name="J1" library="rocketnet-connector" package="ROCKNET-CONNECTOR-M-16" value="ROCKETNET-CONNECTOR-16M" x="15.1" y="14.32"/>
+<element name="J1" library="rocketnet-connector" package="ROCKETNET-M-16" value="ROCKETNET-CONNECTOR-16M" x="15.1" y="14.32"/>
 <element name="JP2" library="pinhead" package="1X10" value="" x="15.2" y="3.3" rot="R180"/>
 </elements>
 <signals>
-<signal name="N$1">
-<contactref element="J1" pad="T+@9"/>
-<contactref element="J1" pad="T+@11"/>
-<contactref element="JP2" pad="5"/>
-<wire x1="16.47" y1="3.3" x2="16.47" y2="10.67" width="0.5" layer="16"/>
-<wire x1="16.47" y1="10.67" x2="17" y2="11.2" width="0.5" layer="16"/>
-<wire x1="17" y1="11.2" x2="17" y2="13.68" width="0.5" layer="16"/>
-<wire x1="17" y1="13.68" x2="17.005" y2="13.685" width="0.5" layer="16"/>
-<wire x1="17.005" y1="13.685" x2="15.735" y2="13.685" width="0.5" layer="16"/>
-</signal>
 <signal name="N$2">
-<contactref element="J1" pad="R-@7"/>
-<contactref element="J1" pad="R-@5"/>
 <contactref element="JP2" pad="6"/>
-<wire x1="13.195" y1="13.685" x2="14.465" y2="13.685" width="0.5" layer="16"/>
-<wire x1="13.93" y1="3.3" x2="13.93" y2="11.07" width="0.5" layer="16"/>
-<wire x1="13.93" y1="11.07" x2="13.2" y2="11.8" width="0.5" layer="16"/>
-<wire x1="13.2" y1="11.8" x2="13.2" y2="13.68" width="0.5" layer="16"/>
-<wire x1="13.2" y1="13.68" x2="13.195" y2="13.685" width="0.5" layer="16"/>
+<contactref element="J1" pad="R+@5"/>
+<contactref element="J1" pad="R+@7"/>
+<wire x1="14.465" y1="13.685" x2="13.195" y2="13.685" width="0.4064" layer="16"/>
+<wire x1="13.195" y1="13.685" x2="13.195" y2="8.905" width="0.4064" layer="16"/>
+<wire x1="13.195" y1="8.905" x2="13.9" y2="8.2" width="0.4064" layer="16"/>
+<wire x1="13.9" y1="8.2" x2="13.9" y2="3.33" width="0.4064" layer="16"/>
+<wire x1="13.9" y1="3.33" x2="13.93" y2="3.3" width="0.4064" layer="16"/>
 </signal>
 <signal name="N$3">
-<contactref element="J1" pad="R+@1"/>
-<contactref element="J1" pad="R+@3"/>
 <contactref element="JP2" pad="7"/>
-<wire x1="11.39" y1="3.3" x2="11.4" y2="3.3" width="0.5" layer="16"/>
-<wire x1="11.4" y1="3.3" x2="11.4" y2="11.4" width="0.5" layer="16"/>
-<wire x1="11.4" y1="11.4" x2="11.9" y2="11.9" width="0.5" layer="16"/>
-<wire x1="11.9" y1="11.9" x2="11.9" y2="13.66" width="0.5" layer="16"/>
-<wire x1="11.9" y1="13.66" x2="11.925" y2="13.685" width="0.5" layer="16"/>
-<wire x1="11.925" y1="13.685" x2="10.655" y2="13.685" width="0.5" layer="16"/>
+<contactref element="J1" pad="R-@4"/>
+<contactref element="J1" pad="R-@3"/>
+<wire x1="11.925" y1="14.955" x2="11.925" y2="14.2" width="0.4064" layer="16"/>
+<wire x1="11.925" y1="14.2" x2="11.925" y2="13.685" width="0.4064" layer="16"/>
+<wire x1="11.39" y1="3.3" x2="11.39" y2="9.69" width="0.4064" layer="16"/>
+<wire x1="11.39" y1="9.69" x2="11.9" y2="10.2" width="0.4064" layer="16"/>
+<wire x1="11.9" y1="10.2" x2="11.9" y2="14.175" width="0.4064" layer="16"/>
+<wire x1="11.9" y1="14.175" x2="11.925" y2="14.2" width="0.4064" layer="16"/>
 </signal>
 <signal name="N$4">
-<contactref element="J1" pad="T-@13"/>
-<contactref element="J1" pad="T-@15"/>
-<contactref element="JP2" pad="4"/>
-<wire x1="19.01" y1="3.3" x2="19.01" y2="10.79" width="0.5" layer="16"/>
-<wire x1="19.01" y1="10.79" x2="18.3" y2="11.5" width="0.5" layer="16"/>
-<wire x1="18.3" y1="11.5" x2="18.3" y2="13.66" width="0.5" layer="16"/>
-<wire x1="18.3" y1="13.66" x2="18.275" y2="13.685" width="0.5" layer="16"/>
-<wire x1="18.275" y1="13.685" x2="19.545" y2="13.685" width="0.5" layer="16"/>
+<contactref element="J1" pad="T-@9"/>
+<contactref element="J1" pad="T-@11"/>
+<contactref element="JP2" pad="5"/>
+<wire x1="16.47" y1="3.3" x2="16.47" y2="8.47" width="0.4064" layer="16"/>
+<wire x1="16.47" y1="8.47" x2="17" y2="9" width="0.4064" layer="16"/>
+<wire x1="17" y1="9" x2="17" y2="13.68" width="0.4064" layer="16"/>
+<wire x1="17" y1="13.68" x2="17.005" y2="13.685" width="0.4064" layer="16"/>
+<wire x1="17.005" y1="13.685" x2="15.735" y2="13.685" width="0.4064" layer="16"/>
 </signal>
 <signal name="N$5">
-<contactref element="J1" pad="B+@2"/>
-<contactref element="J1" pad="B+@4"/>
-<contactref element="JP2" pad="10"/>
-<wire x1="11.925" y1="14.955" x2="10.655" y2="14.955" width="0.5" layer="16"/>
-<wire x1="10.655" y1="14.955" x2="10.655" y2="17.345" width="0.5" layer="16"/>
-<wire x1="10.655" y1="17.345" x2="10.3" y2="17.7" width="0.5" layer="16"/>
-<wire x1="10.3" y1="17.7" x2="4.6" y2="17.7" width="0.5" layer="16"/>
-<wire x1="4.6" y1="17.7" x2="3.8" y2="16.9" width="0.5" layer="16"/>
-<wire x1="3.8" y1="16.9" x2="3.8" y2="3.33" width="0.5" layer="16"/>
-<wire x1="3.8" y1="3.33" x2="3.77" y2="3.3" width="0.5" layer="16"/>
+<contactref element="J1" pad="B+@15"/>
+<contactref element="J1" pad="B+@16"/>
+<contactref element="JP2" pad="1"/>
+<wire x1="19.545" y1="14.955" x2="19.545" y2="13.685" width="0.4064" layer="16"/>
+<wire x1="19.545" y1="13.685" x2="19.545" y2="10.955" width="0.4064" layer="16"/>
+<wire x1="19.545" y1="10.955" x2="21.4" y2="9.1" width="0.4064" layer="16"/>
+<wire x1="21.4" y1="9.1" x2="23.7" y2="9.1" width="0.4064" layer="16"/>
+<wire x1="23.7" y1="9.1" x2="26.7" y2="6.1" width="0.4064" layer="16"/>
+<wire x1="26.7" y1="6.1" x2="26.7" y2="3.37" width="0.4064" layer="16"/>
+<wire x1="26.7" y1="3.37" x2="26.63" y2="3.3" width="0.4064" layer="16"/>
 </signal>
 <signal name="N$6">
-<contactref element="J1" pad="B-@16"/>
-<contactref element="J1" pad="B-@14"/>
-<contactref element="JP2" pad="1"/>
-<wire x1="18.275" y1="14.955" x2="19.545" y2="14.955" width="0.5" layer="16"/>
-<wire x1="19.545" y1="14.955" x2="19.545" y2="17.345" width="0.5" layer="16"/>
-<wire x1="19.545" y1="17.345" x2="19.9" y2="17.7" width="0.5" layer="16"/>
-<wire x1="19.9" y1="17.7" x2="24.8" y2="17.7" width="0.5" layer="16"/>
-<wire x1="24.8" y1="17.7" x2="26.6" y2="15.9" width="0.5" layer="16"/>
-<wire x1="26.6" y1="15.9" x2="26.6" y2="3.33" width="0.5" layer="16"/>
-<wire x1="26.6" y1="3.33" x2="26.63" y2="3.3" width="0.5" layer="16"/>
+<contactref element="J1" pad="B-@2"/>
+<contactref element="J1" pad="B-@1"/>
+<contactref element="JP2" pad="10"/>
+<wire x1="3.77" y1="3.3" x2="3.77" y2="6.67" width="0.4064" layer="16"/>
+<wire x1="3.77" y1="6.67" x2="6.6" y2="9.5" width="0.4064" layer="16"/>
+<wire x1="6.6" y1="9.5" x2="9.4" y2="9.5" width="0.4064" layer="16"/>
+<wire x1="9.4" y1="9.5" x2="10.655" y2="10.755" width="0.4064" layer="16"/>
+<wire x1="10.655" y1="14.955" x2="10.655" y2="13.685" width="0.4064" layer="16"/>
+<wire x1="10.655" y1="13.685" x2="10.655" y2="10.755" width="0.4064" layer="16"/>
 </signal>
 <signal name="N$7">
@@
 <wire x1="21.5" y1="3.35" x2="21.55" y2="3.3" width="0.5" layer="1"/>
 </signal>
+<signal name="N$11">
+<contactref element="J1" pad="T+@13"/>
+<contactref element="J1" pad="T+@14"/>
+<contactref element="JP2" pad="4"/>
+<wire x1="18.275" y1="14.955" x2="18.275" y2="13.685" width="0.4064" layer="16"/>
+<wire x1="18.275" y1="13.685" x2="18.275" y2="10.325" width="0.4064" layer="16"/>
+<wire x1="18.275" y1="10.325" x2="19" y2="9.6" width="0.4064" layer="16"/>
+<wire x1="19" y1="9.6" x2="19" y2="3.31" width="0.4064" layer="16"/>
+<wire x1="19" y1="3.31" x2="19.01" y2="3.3" width="0.4064" layer="16"/>
+</signal>
 </signals>
