File: av3/rocketnet-connector/eagle/rocketnet-test.sch (EAGLE design)
At the start: 2 parts, among them J1 ROCKETNET-CONNECTOR-16M

Commit message: Updated rocketnet connectors and boards to match new rocketnet stackup.
Connections:
- removed net N$1: J1.TX+@1, J1.TX+@2, JP2.5
- new net N$11: J1.TX+@1, J1.TX+@2, JP2.4
- net N$2: now also J1.RX+@1, J1.RX+@2; no longer J1.RX-@1, J1.RX-@2
- net N$3: now also J1.RX-@1, J1.RX-@2; no longer J1.RX+@1, J1.RX+@2
- net N$4: now also JP2.5; no longer JP2.4
- net N$5: now also JP2.1; no longer JP2.10
- net N$6: now also JP2.10; no longer JP2.1
Changed lines of the file:
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@@
 </busses>
 <nets>
-<net name="N$1" class="0">
-<segment>
-<pinref part="J1" gate="G$1" pin="TX+@1"/>
-<pinref part="J1" gate="G$1" pin="TX+@2"/>
-<wire x1="63.5" y1="63.5" x2="63.5" y2="60.96" width="0.1524" layer="91"/>
-<junction x="63.5" y="60.96"/>
-<wire x1="63.5" y1="60.96" x2="78.74" y2="60.96" width="0.1524" layer="91"/>
-<wire x1="78.74" y1="60.96" x2="78.74" y2="53.34" width="0.1524" layer="91"/>
-<pinref part="JP2" gate="A" pin="5"/>
-<wire x1="78.74" y1="53.34" x2="116.84" y2="53.34" width="0.1524" layer="91"/>
-</segment>
-</net>
 <net name="N$2" class="0">
 <segment>
-<pinref part="J1" gate="G$1" pin="RX-@2"/>
-<pinref part="J1" gate="G$1" pin="RX-@1"/>
-<wire x1="63.5" y1="45.72" x2="63.5" y2="48.26" width="0.1524" layer="91"/>
-<wire x1="63.5" y1="48.26" x2="78.74" y2="48.26" width="0.1524" layer="91"/>
-<wire x1="78.74" y1="48.26" x2="78.74" y2="50.8" width="0.1524" layer="91"/>
-<junction x="63.5" y="48.26"/>
 <pinref part="JP2" gate="A" pin="6"/>
-<wire x1="78.74" y1="50.8" x2="116.84" y2="50.8" width="0.1524" layer="91"/>
+<wire x1="63.5" y1="50.8" x2="116.84" y2="50.8" width="0.1524" layer="91"/>
+<pinref part="J1" gate="G$1" pin="RX+@2"/>
+<pinref part="J1" gate="G$1" pin="RX+@1"/>
+<wire x1="63.5" y1="53.34" x2="63.5" y2="50.8" width="0.1524" layer="91"/>
+<junction x="63.5" y="50.8"/>
 </segment>
 </net>
 <net name="N$3" class="0">
 <segment>
-<pinref part="J1" gate="G$1" pin="RX+@1"/>
-<pinref part="J1" gate="G$1" pin="RX+@2"/>
-<wire x1="63.5" y1="53.34" x2="63.5" y2="50.8" width="0.1524" layer="91"/>
-<wire x1="63.5" y1="50.8" x2="73.66" y2="50.8" width="0.1524" layer="91"/>
-<junction x="63.5" y="50.8"/>
-<wire x1="73.66" y1="50.8" x2="73.66" y2="45.72" width="0.1524" layer="91"/>
-<wire x1="73.66" y1="45.72" x2="81.28" y2="45.72" width="0.1524" layer="91"/>
-<wire x1="81.28" y1="45.72" x2="81.28" y2="48.26" width="0.1524" layer="91"/>
 <pinref part="JP2" gate="A" pin="7"/>
-<wire x1="81.28" y1="48.26" x2="116.84" y2="48.26" width="0.1524" layer="91"/>
+<wire x1="63.5" y1="48.26" x2="116.84" y2="48.26" width="0.1524" layer="91"/>
+<pinref part="J1" gate="G$1" pin="RX-@1"/>
+<pinref part="J1" gate="G$1" pin="RX-@2"/>
+<wire x1="63.5" y1="45.72" x2="63.5" y2="48.26" width="0.1524" layer="91"/>
+<junction x="63.5" y="48.26"/>
 </segment>
 </net>
@@
 <pinref part="J1" gate="G$1" pin="TX-@2"/>
 <wire x1="63.5" y1="58.42" x2="63.5" y2="55.88" width="0.1524" layer="91"/>
-<pinref part="JP2" gate="A" pin="4"/>
-<wire x1="63.5" y1="55.88" x2="116.84" y2="55.88" width="0.1524" layer="91"/>
+<pinref part="JP2" gate="A" pin="5"/>
+<wire x1="78.74" y1="53.34" x2="116.84" y2="53.34" width="0.1524" layer="91"/>
+<wire x1="63.5" y1="55.88" x2="78.74" y2="55.88" width="0.1524" layer="91"/>
+<wire x1="78.74" y1="55.88" x2="78.74" y2="53.34" width="0.1524" layer="91"/>
 <junction x="63.5" y="55.88"/>
 </segment>
@@
 <junction x="63.5" y="66.04"/>
 <wire x1="81.28" y1="66.04" x2="81.28" y2="68.58" width="0.1524" layer="91"/>
-<wire x1="81.28" y1="68.58" x2="134.62" y2="68.58" width="0.1524" layer="91"/>
-<wire x1="134.62" y1="68.58" x2="134.62" y2="40.64" width="0.1524" layer="91"/>
-<pinref part="JP2" gate="A" pin="10"/>
-<wire x1="134.62" y1="40.64" x2="116.84" y2="40.64" width="0.1524" layer="91"/>
+<wire x1="81.28" y1="68.58" x2="116.84" y2="68.58" width="0.1524" layer="91"/>
+<pinref part="JP2" gate="A" pin="1"/>
+<wire x1="116.84" y1="63.5" x2="116.84" y2="68.58" width="0.1524" layer="91"/>
 </segment>
 </net>
@@
 <pinref part="J1" gate="G$1" pin="B-@1"/>
 <wire x1="63.5" y1="30.48" x2="63.5" y2="33.02" width="0.1524" layer="91"/>
-<wire x1="63.5" y1="33.02" x2="129.54" y2="33.02" width="0.1524" layer="91"/>
+<wire x1="63.5" y1="33.02" x2="116.84" y2="33.02" width="0.1524" layer="91"/>
 <junction x="63.5" y="33.02"/>
-<wire x1="129.54" y1="33.02" x2="129.54" y2="63.5" width="0.1524" layer="91"/>
-<wire x1="129.54" y1="63.5" x2="116.84" y2="63.5" width="0.1524" layer="91"/>
-<pinref part="JP2" gate="A" pin="1"/>
+<pinref part="JP2" gate="A" pin="10"/>
+<wire x1="116.84" y1="40.64" x2="116.84" y2="33.02" width="0.1524" layer="91"/>
 </segment>
 </net>
@@
 </segment>
 </net>
+<net name="N$11" class="0">
+<segment>
+<pinref part="J1" gate="G$1" pin="TX+@2"/>
+<pinref part="J1" gate="G$1" pin="TX+@1"/>
+<wire x1="63.5" y1="63.5" x2="63.5" y2="60.96" width="0.1524" layer="91"/>
+<pinref part="JP2" gate="A" pin="4"/>
+<wire x1="116.84" y1="55.88" x2="81.28" y2="55.88" width="0.1524" layer="91"/>
+<wire x1="81.28" y1="55.88" x2="81.28" y2="60.96" width="0.1524" layer="91"/>
+<wire x1="81.28" y1="60.96" x2="63.5" y2="60.96" width="0.1524" layer="91"/>
+<junction x="63.5" y="60.96"/>
+</segment>
+</net>
