File: av3/e407-sensor-shield/e407-sensor-shield.brd (EAGLE design)
At the start: 101.6 x 85.6 mm, 9 parts, among them CON1 CON1, CON4 CON4

Commit message: Changes to e407 sensor shield with Bob. Double checked connector and sensor placement, added rocketbus connector, stapled board, made the board outline slidely bigger given the e407 layout.
Parts:
- added C1, R1: (no value), rcl_custom:0603-B-NOSILK
- added CON2: CON1, SparkFun-Connectors:1X06
- added J1: ROCKETBUS, rocketbus:ROCKETBUS-PKG
- added TP1, TP2, TP3, TP4, TP5, TP6: TEST-POINT, apdm:2MM-TEST-POINT
- moved MPL 0.30 mm to (37.3, 38.4)
- moved CON4 0.20 mm to (60.3, 64.4)
- moved MPU 0.13 mm to (55.9, 33.3)
- moved PG 0.10 mm to (69.2, 4.70)
Connections:
- new net N$10: J1.AUX_2@1, J1.AUX_2@2, TP6.1
- new net N$3: J1.CAN_H@1, J1.CAN_H@2, TP1.1
- new net N$4: CON1.1, CON2.1
- new net N$5: C1.1, J1.CHASSIS@1, J1.CHASSIS@2, R1.2
- new net N$6: J1.CAN_L@1, J1.CAN_L@2, TP2.1
- new net N$7: J1.USB_H@1, J1.USB_H@2, TP3.1
- new net N$8: J1.USB_L@1, J1.USB_L@2, TP4.1
- new net N$9: J1.AUX_1@1, J1.AUX_1@2, TP5.1
- new net TRIPLE_UP_ARROW: CON1.6, CON2.6, J1.B+@1, J1.B+@2
- net DOUBLE_UP_ARROW: now also CON2.3
- net TRIPLE_BAR_GND: now also C1.2, CON2.4, CON2.5, J1.B-@1, J1.B-@2, R1.1
- net UP_ARROW: now also CON2.2
Routing:
- net TRIPLE_UP_ARROW: track 0.00 -> 77.4 mm
- net N$5: track 0.00 -> 14.3 mm
- net N$7: track 0.00 -> 8.30 mm
- net N$3: track 0.00 -> 8.29 mm
- net N$9: track 0.00 -> 8.25 mm
- net N$8: track 0.00 -> 6.03 mm
- net N$6: track 0.00 -> 6.01 mm
- net N$10: track 0.00 -> 5.19 mm
- net N$4: track 0.00 -> 5.08 mm
- net DOUBLE_UP_ARROW: track 46.2 -> 51.3 mm
- net PFP04: track 73.2 -> 68.3 mm
- net PFP03: track 73.6 -> 68.8 mm
- net PFP06: track 44.3 -> 39.5 mm
- net PFP07: track 42.7 -> 38.3 mm
- net UP_ARROW: track 83.7 -> 87.0 mm
Other:
- outline, holes or cut-outs redrawn
- board text added: "!RST"
- board text added: "3.3V"
- board text added: "5V"
- board text added: "ADIS ribbon cable"
- board text added: "AUX1"
- board text added: "AUX2"
- board text added: "MPL3115A2 Breakout"
- board text added: "MPU-9150 Breakout"
- board text added: "Vin"

Commit message: Brought ethernet up to e407 daughter board and connected via caps to rocketnet connector. Made cutout in board an internal cutout just for TH caps on e407 to gain stability in daugher board. Misc cleanup.
Parts:
- added C2, C3, C4, C5: 200n, rcl_custom:0603-B-NOSILK
- added LAN: RJLBC-060TC1, OLIMEX_CONNECTORS:RJLBC-060TC1
- C1: value (none) -> 100n
- R1: value (none) -> 10M
- moved C1 11.8 mm to (2.92, 25.0), flipped to the top, turned to 270 degrees
- moved R1 9.34 mm to (4.95, 25.0), flipped to the top, turned to 90 degrees
Connections:
- new net N$11: C2.1, LAN.1
- new net N$12: C3.1, LAN.2
- new net N$13: C4.1, LAN.7
- new net N$14: C5.1, LAN.8
- net N$3: now also C2.2
- net N$6: now also C3.2
- net N$7: now also C4.2
- net N$8: now also C5.2
Routing:
- net N$12: track 0.00 -> 22.6 mm
- net N$11: track 0.00 -> 16.8 mm
- net N$8: track 6.03 -> 20.6 mm
- net N$13: track 0.00 -> 9.55 mm
- net N$7: track 8.30 -> 17.6 mm
- net N$14: track 0.00 -> 8.02 mm
- net N$6: track 6.01 -> 12.9 mm
- net N$3: track 8.29 -> 13.4 mm
- net N$5: track 14.3 -> 18.9 mm
Other:
- outline, holes or cut-outs redrawn
- board text removed: "Connector"
- board text removed: "Enet"

Commit message: Added LEDs for ethernet status, cleaned up silkscreen.
Parts:
- added LED1: YEL, led:CHIPLED_0603
- added LED2: GRN, led:CHIPLED_0603
Connections:
- new net N$15: LAN.KY, LED1.C
- new net N$16: LAN.AY, LED1.A
- new net N$17: LAN.KG, LED2.C
- new net N$18: LAN.AG, LED2.A
Routing:
- net N$17: track 0.00 -> 3.22 mm
- net N$15: track 0.00 -> 3.21 mm
- net N$16: track 0.00 -> 3.19 mm
- net N$18: track 0.00 -> 3.19 mm

Commit message: Added stupid EAGLE temporary files to the gitignore. Updated IMU adapter with sane net names so we could easily trace nets. And updated the e407 shield to add a RGB LED, correct some schematic mistakes found out while double checking connections, and updated to being routable on a PCB router.
Parts:
- removed C3, C4, C5: 200n, rcl_custom:0603-B-NOSILK
- removed TP6: TEST-POINT, apdm:2MM-TEST-POINT
- added L1, L2: ACM2012, magnetics:TDK-ACM2012
- added LED3: (no value), Tova:PLCC-6
- added R2, R3, R4, R5: 50, rcl_custom:0603-B-NOSILK
- added T1, T2: ALT4532, magnetics:TDK-ALT4532
- C1: value 100n -> 100nF
- C2: value 200n -> 10u; device rcl_custom:0603-B-NOSILK -> rcl_custom:0805-B-NOSILK
- J1: value ROCKETBUS -> ROCKETNET-CONNECTOR-16M; device rocketbus:ROCKETBUS-PKG -> rocketnet-connector:ROCKETNET-M-16
- R1: value 10M -> 50
- TP5: value TEST-POINT -> TPPAD1-13; device apdm:2MM-TEST-POINT -> testpad:P1-13
- moved C2 39.5 mm to (52.9, 57.9), flipped to the bottom, turned to 90 degrees
- moved TP5 24.5 mm to (37.4, 33.8)
- moved C1 15.7 mm to (17.6, 30.7), turned to 180 degrees
- moved R1 14.5 mm to (17.6, 32.2), turned to 180 degrees
- moved TP1 14.3 mm to (1.20, 32.5)
- moved TP3 12.9 mm to (1.20, 36.1)
- moved TP4 11.1 mm to (1.20, 37.9)
- moved TP2 11.0 mm to (1.20, 34.3)
- moved J1 1.33 mm to (4.57, 35.2), turned to 90 degrees
Connections:
- net C4D11 renamed ADIS-DIN-MOSI
- net C4D12 renamed ADIS-DOUT-MISO
- net PDP11 renamed ADIS-!RST
- net PDP12 renamed ADIS-DIO1-INT
- net PDP13 renamed ADIS-DIO2-NC
- net PDP14 renamed ADIS-DIO3-NC
- net PDP15 renamed ADIS-DIO4-NC
- net PFP06 renamed MPL-INT1
- removed net C4D10: ADIS.3, CON4.3
- removed net C4D13: ADIS.6, CON4.6
- new net ADIS-!CS!-!SS: ADIS.6, CON4.3
- new net ADIS-SCLK: ADIS.3, CON4.6
- new net B: PF.17, R5.1
- new net G: PF.16, R4.1
- new net N$19: J1.R-@3, J1.R-@4, L2.2
- new net N$20: J1.A4, TP4.1
- new net N$21: J1.A3, TP3.1
- new net N$22: J1.A2, TP2.1
- new net N$23: J1.A1, TP1.1
- new net N$24: LAN.3, T1.6, T2.6
- new net N$25: C1.1, R1.1, R2.1
- new net N$26: R1.2, T2.3
- new net N$27: R2.2, T1.3
- new net N$28: LED3.1, R3.2
- new net N$29: LED3.3, R4.2
- new net N$30: LED3.4, R5.2
- new net R: PF.15, R3.1
- net N$10: now also J1.R+@5, J1.R+@7, L2.1; no longer J1.AUX_2@1, J1.AUX_2@2, TP6.1
- net N$11: now also T1.1; no longer C2.1
- net N$12: now also T1.2; no longer C3.1
- net N$13: now also T2.1; no longer C4.1
- net N$14: now also T2.2; no longer C5.1
- net N$3: now also L1.4, T1.5; no longer C2.2, J1.CAN_H@1, J1.CAN_H@2, TP1.1
- net N$5: now also L1.3, T1.4; no longer C1.1, J1.CHASSIS@1, J1.CHASSIS@2, R1.2
- net N$6: now also L2.4, T2.5; no longer C3.2, J1.CAN_L@1, J1.CAN_L@2, TP2.1
- net N$7: now also L2.3, T2.4; no longer C4.2, J1.USB_H@1, J1.USB_H@2, TP3.1
- net N$8: now also J1.T+@13, J1.T+@14, L1.1; no longer C5.2, J1.USB_L@1, J1.USB_L@2, TP4.1
- net N$9: now also J1.T-@11, J1.T-@9, L1.2; no longer J1.AUX_1@1, J1.AUX_1@2, TP5.1
- net PFP07: now also TP5.TP; no longer PF.7
- net TRIPLE_BAR_GND: now also C2.2, LED3.2, LED3.5, LED3.6, PD.2, PD.20, PE.2, PE.20, PF.2, PF.20, PG.2, PG.20; no longer R1.1
- net TRIPLE_UP_ARROW: now also J1.B+@15, J1.B+@16; no longer J1.B+@1, J1.B+@2
- net UP_ARROW: now also C2.1
Routing:
- net C4D13: track 55.2 -> 0.00 mm, vias 1 -> 0
- net ADIS-SCLK: track 0.00 -> 55.0 mm, vias 0 -> 1
- net N$24: track 0.00 -> 46.2 mm
- net C4D10: track 45.2 -> 0.00 mm
- net ADIS-!CS!-!SS: track 0.00 -> 42.5 mm, vias 0 -> 1
- net PFP07: track 38.3 -> 4.58 mm
- net N$5: track 18.9 -> 1.49 mm
- net N$7: track 17.6 -> 1.49 mm
- net N$8: track 20.6 -> 4.96 mm, vias 0 -> 1
- net N$3: track 13.4 -> 1.51 mm
- net N$27: track 0.00 -> 11.7 mm
- net B: track 0.00 -> 11.6 mm
- net N$6: track 12.9 -> 1.51 mm
- net R: track 0.00 -> 11.0 mm
- net N$14: track 8.02 -> 18.8 mm
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Other:
- outline, holes or cut-outs redrawn
- board text added: "TOP"
