File: av3/e407-sensor-shield/e407-sensor-shield.brd (EAGLE design)
At the start: 101.6 x 85.6 mm, 31 parts, among them CON1 CON1, CON2 CON1, CON4 CON4, J1 ROCKETNET-CONNECTOR-16M, T1 ALT4532, T2 ALT4532

Commit message: Updates to the sensor board, these files were made on the LPKF. Includes BOM in xls.
Parts:
- R3: value 50 -> 900
- R4: value 50 -> 400
- R5: value 50 -> 110
Changed lines of the file:
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@@
 </element>
 <element name="LED3" library="Tova" package="PLCC-6" value="" x="47.4" y="11.3"/>
-<element name="R3" library="rcl_custom" package="0603-B-NOSILK" value="50" x="43" y="12.4"/>
-<element name="R4" library="rcl_custom" package="0603-B-NOSILK" value="50" x="43" y="10.2"/>
-<element name="R5" library="rcl_custom" package="0603-B-NOSILK" value="50" x="51.6" y="10.2" rot="R180"/>
+<element name="R3" library="rcl_custom" package="0603-B-NOSILK" value="900" x="43" y="12.4"/>
+<element name="R4" library="rcl_custom" package="0603-B-NOSILK" value="400" x="43" y="10.2"/>
+<element name="R5" library="rcl_custom" package="0603-B-NOSILK" value="110" x="51.6" y="10.2" rot="R180"/>
 <element name="C2" library="rcl_custom" package="0805-B-NOSILK" value="10u" x="52.9" y="57.9" rot="MR90"/>
 </elements>
