File: av3/e407-sensor-shield/e407-sensor-shield.sch (EAGLE design)
At the start: 9 parts, among them CON1 CON1, CON4 CON4

Commit message: Changes to e407 sensor shield with Bob. Double checked connector and sensor placement, added rocketbus connector, stapled board, made the board outline slidely bigger given the e407 layout.
Parts:
- added C1: (no value), rcl_custom:C-EU0603-B-NOSILK
- added CON2: CON1, SparkFun-Connectors:M06SIP
- added J1: ROCKETBUS, rocketbus:ROCKETBUS
- added R1: (no value), rcl_custom:R-US_0603-B-NOSILK
- added TP1, TP2, TP3, TP4, TP5, TP6: TEST-POINT, apdm:TEST-POINT
Connections:
- new net N$10: J1.AUX_2@1, J1.AUX_2@2, TP6.1
- new net N$3: J1.CAN_H@1, J1.CAN_H@2, TP1.1
- new net N$4: CON1.1, CON2.1
- new net N$5: C1.1, J1.CHASSIS@1, J1.CHASSIS@2, R1.2
- new net N$6: J1.CAN_L@1, J1.CAN_L@2, TP2.1
- new net N$7: J1.USB_H@1, J1.USB_H@2, TP3.1
- new net N$8: J1.USB_L@1, J1.USB_L@2, TP4.1
- new net N$9: J1.AUX_1@1, J1.AUX_1@2, TP5.1
- new net TRIPLE_UP_ARROW: CON1.6, CON2.6, J1.B+@1, J1.B+@2
- net DOUBLE_UP_ARROW: now also CON2.3
- net TRIPLE_BAR_GND: now also C1.2, CON2.4, CON2.5, J1.B-@1, J1.B-@2, R1.1
- net UP_ARROW: now also CON2.2

Commit message: Brought ethernet up to e407 daughter board and connected via caps to rocketnet connector. Made cutout in board an internal cutout just for TH caps on e407 to gain stability in daugher board. Misc cleanup.
Parts:
- added C2, C3, C4, C5: 200n, rcl_custom:C-EU0603-B-NOSILK
- added LAN: RJLBC-060TC1, OLIMEX_CONNECTORS:RJLBC-060TC1
- C1: value (none) -> 100n
- R1: value (none) -> 10M
Connections:
- new net N$11: C2.1, LAN.TD+
- new net N$12: C3.1, LAN.TD-
- new net N$13: C4.1, LAN.RD+
- new net N$14: C5.1, LAN.RD-
- net N$3: now also C2.2
- net N$6: now also C3.2
- net N$7: now also C4.2
- net N$8: now also C5.2
Other:
- moved on the sheet: ADIS, C1, CON1, CON2, CON4, J1, MPL, MPU, PD, PE, PF, PG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

Commit message: Added LEDs for ethernet status, cleaned up silkscreen.
Parts:
- added LED1: YEL, led:LEDCHIPLED_0603
- added LED2: GRN, led:LEDCHIPLED_0603
Connections:
- new net N$15: LAN.KY, LED1.C
- new net N$16: LAN.AY, LED1.A
- new net N$17: LAN.KG, LED2.C
- new net N$18: LAN.AG, LED2.A
Other:
- moved on the sheet: LAN
Changed lines of the file:
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@@
 <setting verticaltext="up"/>
 </settings>
-<grid distance="0.05" unitdist="inch" unit="inch" style="lines" multiple="2" display="yes" altdistance="0.01" altunitdist="inch" altunit="inch"/>
+<grid distance="0.1" unitdist="inch" unit="inch" style="lines" multiple="1" display="yes" altdistance="0.01" altunitdist="inch" altunit="inch"/>
 <layers>
 <layer number="1" name="Top" color="4" fill="1" visible="no" active="no"/>
@@
 <part name="C5" library="rcl_custom" deviceset="C-EU" device="0603-B-NOSILK" value="200n"/>
 <part name="FRAME1" library="frames" deviceset="FRAME_A_L" device=""/>
+<part name="LED1" library="led" deviceset="LED" device="CHIPLED_0603" value="YEL"/>
+<part name="LED2" library="led" deviceset="LED" device="CHIPLED_0603" value="GRN"/>
 </parts>
 <sheets>
@@
 <instance part="TP5" gate="G$1" x="134.62" y="165.1" rot="MR0"/>
 <instance part="TP6" gate="G$1" x="134.62" y="160.02" rot="MR0"/>
-<instance part="LAN" gate="G$1" x="55.88" y="172.72" smashed="yes" rot="MR0">
-<attribute name="NAME" x="61.595" y="188.595" size="1.778" layer="95" rot="MR0"/>
-<attribute name="VALUE" x="69.215" y="157.48" size="1.778" layer="96" rot="MR0"/>
+<instance part="LAN" gate="G$1" x="30.48" y="172.72" smashed="yes" rot="MR0">
+<attribute name="NAME" x="36.195" y="188.595" size="1.778" layer="95" rot="MR0"/>
+<attribute name="VALUE" x="43.815" y="157.48" size="1.778" layer="96" rot="MR0"/>
 </instance>
 <instance part="C2" gate="CE" x="91.44" y="185.42" rot="R90"/>
@@
 <instance part="FRAME1" gate="G$1" x="0" y="0"/>
 <instance part="FRAME1" gate="G$2" x="173.99" y="0"/>
+<instance part="LED1" gate="G$1" x="66.04" y="152.4"/>
+<instance part="LED2" gate="G$1" x="81.28" y="152.4"/>
 </instances>
 <busses>
@@
 <pinref part="LAN" gate="G$1" pin="TD+"/>
 <pinref part="C2" gate="CE" pin="1"/>
-<wire x1="83.82" y1="185.42" x2="88.9" y2="185.42" width="0.1524" layer="91"/>
+<wire x1="58.42" y1="185.42" x2="88.9" y2="185.42" width="0.1524" layer="91"/>
 </segment>
 </net>
@@
 <pinref part="C3" gate="CE" pin="1"/>
 <pinref part="LAN" gate="G$1" pin="TD-"/>
-<wire x1="96.52" y1="180.34" x2="83.82" y2="180.34" width="0.1524" layer="91"/>
+<wire x1="96.52" y1="180.34" x2="58.42" y2="180.34" width="0.1524" layer="91"/>
 </segment>
 </net>
@@
 <pinref part="LAN" gate="G$1" pin="RD+"/>
 <pinref part="C4" gate="CE" pin="1"/>
-<wire x1="83.82" y1="167.64" x2="88.9" y2="167.64" width="0.1524" layer="91"/>
+<wire x1="58.42" y1="167.64" x2="88.9" y2="167.64" width="0.1524" layer="91"/>
 </segment>
 </net>
@@
 <pinref part="LAN" gate="G$1" pin="RD-"/>
 <pinref part="C5" gate="CE" pin="1"/>
-<wire x1="83.82" y1="162.56" x2="96.52" y2="162.56" width="0.1524" layer="91"/>
-</segment>
-</net>
+<wire x1="58.42" y1="162.56" x2="96.52" y2="162.56" width="0.1524" layer="91"/>
+</segment>
+</net>
+<net name="N$15" class="0">
+<segment>
+<pinref part="LAN" gate="G$1" pin="KY"/>
+<wire x1="58.42" y1="170.18" x2="60.96" y2="170.18" width="0.1524" layer="91"/>
+<wire x1="60.96" y1="170.18" x2="60.96" y2="144.78" width="0.1524" layer="91"/>
+<pinref part="LED1" gate="G$1" pin="C"/>
+<wire x1="60.96" y1="144.78" x2="66.04" y2="144.78" width="0.1524" layer="91"/>
+<wire x1="66.04" y1="144.78" x2="66.04" y2="147.32" width="0.1524" layer="91"/>
+</segment>
+</net>
+<net name="N$16" class="0">
+<segment>
+<pinref part="LED1" gate="G$1" pin="A"/>
+<wire x1="66.04" y1="154.94" x2="66.04" y2="172.72" width="0.1524" layer="91"/>
+<pinref part="LAN" gate="G$1" pin="AY"/>
+<wire x1="58.42" y1="172.72" x2="66.04" y2="172.72" width="0.1524" layer="91"/>
+</segment>
+</net>
+<net name="N$17" class="0">
+<segment>
+<pinref part="LAN" gate="G$1" pin="KG"/>
+<wire x1="58.42" y1="175.26" x2="76.2" y2="175.26" width="0.1524" layer="91"/>
+<wire x1="76.2" y1="175.26" x2="76.2" y2="144.78" width="0.1524" layer="91"/>
+<pinref part="LED2" gate="G$1" pin="C"/>
+<wire x1="76.2" y1="144.78" x2="81.28" y2="144.78" width="0.1524" layer="91"/>
+<wire x1="81.28" y1="144.78" x2="81.28" y2="147.32" width="0.1524" layer="91"/>
+</segment>
+</net>
+<net name="N$18" class="0">
+<segment>
+<pinref part="LED2" gate="G$1" pin="A"/>
+<wire x1="81.28" y1="154.94" x2="81.28" y2="177.8" width="0.1524" layer="91"/>
+<pinref part="LAN" gate="G$1" pin="AG"/>
+<wire x1="81.28" y1="177.8" x2="58.42" y2="177.8" width="0.1524" layer="91"/>
+</segment>
+</net>

Commit message: Added stupid EAGLE temporary files to the gitignore. Updated IMU adapter with sane net names so we could easily trace nets. And updated the e407 shield to add a RGB LED, correct some schematic mistakes found out while double checking connections, and updated to being routable on a PCB router.
Parts:
- removed C3, C4, C5: 200n, rcl_custom:C-EU0603-B-NOSILK
- removed TP6: TEST-POINT, apdm:TEST-POINT
- added L1, L2: ACM2012, magnetics:ACM2012
- added LED3: (no value), Tova:LED_RGB_PLCC-6
- added R2, R3, R4, R5: 50, rcl_custom:R-US_0603-B-NOSILK
- added T1, T2: ALT4532, magnetics:ALT4532
- C1: value 100n -> 100nF
- C2: value 200n -> 10u; device rcl_custom:C-EU0603-B-NOSILK -> rcl_custom:C-EU0805-B-NOSILK
- J1: value ROCKETBUS -> ROCKETNET-CONNECTOR-16M; device rocketbus:ROCKETBUS -> rocketnet-connector:ROCKETNET-CONNECTOR-16M
- R1: value 10M -> 50
- TP5: value TEST-POINT -> TPPAD1-13; device apdm:TEST-POINT -> testpad:TPPAD1-13
Connections:
- net C4D11 renamed ADIS-DIN-MOSI
- net C4D12 renamed ADIS-DOUT-MISO
- net PDP11 renamed ADIS-!RST
- net PDP12 renamed ADIS-DIO1-INT
- net PDP13 renamed ADIS-DIO2-NC
- net PDP14 renamed ADIS-DIO3-NC
- net PDP15 renamed ADIS-DIO4-NC
- net PFP06 renamed MPL-INT1
- removed net C4D10: ADIS.3, CON4.3
- removed net C4D13: ADIS.6, CON4.6
- new net ADIS-!CS!-!SS: ADIS.6, CON4.3
- new net ADIS-SCLK: ADIS.3, CON4.6
- new net B: PF.17, R5.1
- new net G: PF.16, R4.1
- new net N$19: J1.RX-@1, J1.RX-@2, L2.2
- new net N$20: J1.AUX4, TP4.1
- new net N$21: J1.AUX3, TP3.1
- new net N$22: J1.AUX2, TP2.1
- new net N$23: J1.AUX1, TP1.1
- new net N$24: LAN.COM, T1.6, T2.6
- new net N$25: C1.1, R1.1, R2.1
- new net N$26: R1.2, T2.3
- new net N$27: R2.2, T1.3
- new net N$28: LED3R.A, R3.2
- new net N$29: LED3G.A, R4.2
- new net N$30: LED3B.A, R5.2
- new net R: PF.15, R3.1
- net N$10: now also J1.RX+@1, J1.RX+@2, L2.1; no longer J1.AUX_2@1, J1.AUX_2@2, TP6.1
- net N$11: now also T1.1; no longer C2.1
- net N$12: now also T1.2; no longer C3.1
- net N$13: now also T2.1; no longer C4.1
- net N$14: now also T2.2; no longer C5.1
- net N$3: now also L1.4, T1.5; no longer C2.2, J1.CAN_H@1, J1.CAN_H@2, TP1.1
- net N$5: now also L1.3, T1.4; no longer C1.1, J1.CHASSIS@1, J1.CHASSIS@2, R1.2
- net N$6: now also L2.4, T2.5; no longer C3.2, J1.CAN_L@1, J1.CAN_L@2, TP2.1
- net N$7: now also L2.3, T2.4; no longer C4.2, J1.USB_H@1, J1.USB_H@2, TP3.1
- net N$8: now also J1.TX+@1, J1.TX+@2, L1.1; no longer C5.2, J1.USB_L@1, J1.USB_L@2, TP4.1
- net N$9: now also J1.TX-@1, J1.TX-@2, L1.2; no longer J1.AUX_1@1, J1.AUX_1@2, TP5.1
- net PFP07: now also TP5.TP; no longer PF.7
- net TRIPLE_BAR_GND: now also C2.2, LED3B.K, LED3G.K, LED3R.K, PD.2, PD.20, PE.2, PE.20, PF.2, PF.20, PG.2, PG.20; no longer R1.1
- net UP_ARROW: now also C2.1
Other:
- note added: "!RST"
- note added: "!SS"
- note added: "3.3V"
- note added: "5V"
- note added: "AD0"
- note added: "ADIS16405 Breakout"
- note added: "AGND"
- note added: "AREF"
- note added: "CLKIN"
- note added: "CLKOUT"
- note added: "ESC"
- note added: "ESD"
- note added: "FSYNC"
- note added: "GND"
- note added: "INT"
- note added: "INT2"
- note added: "MISO"
- note added: "MOSI"
- note added: "MPL??? Pressure breakout board"
- note added: "MPU-9150 single-IC IMU breakout board"
- note added: "NOTE: I2C resistors removed"
- note added: "PA4"
- note added: "PA5"
- note added: "PA6"
- note added: "PB5"
- note added: "PD0"
- note added: "PD1"
- note added: "PD10"
- note added: "PD11"
- note added: "PD12"
- note added: "PD13"
- note added: "PD14"
- note added: "PD15"
- note added: "PD3"
- note added: "PD4"
- note added: "PD5"
- note added: "PD6"
- note added: "PD7"
- note added: "PD8"
- note added: "PD9"
- note added: "PF0"
- note added: "PF1"
- note added: "PF12"
- note added: "PF13"
- note added: "PF14"
- note added: "PF15"
- note added: "PF2"
- note added: "PF3"
- note added: "PF4"
- note added: "PF5"
- note added: "PG12"
- note added: "PG15"
- note added: "SCK"
- note added: "SCL"
- note added: "SDA"
- note added: "SPI1"
- note removed: "C4D10"
- note removed: "C4D11"
- note removed: "C4D12"
- note removed: "C4D13"
- note removed: "PDP11"
- note removed: "PDP12"
- note removed: "PDP13"
- note removed: "PDP14"
- note removed: "PDP15"
- note removed: "PFP07"
- moved on the sheet: ADIS, C1, C2, CON1, CON2, CON4, LAN, LED1, LED2, MPL, MPU, PD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

Commit message: Updates to the sensor board, these files were made on the LPKF. Includes BOM in xls.
Parts:
- R3: value 50 -> 900
- R4: value 50 -> 400
- R5: value 50 -> 110
Changed lines of the file:
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@@
 <setting verticaltext="up"/>
 </settings>
-<grid distance="0.05" unitdist="inch" unit="inch" style="lines" multiple="2" display="yes" altdistance="0.01" altunitdist="inch" altunit="inch"/>
+<grid distance="0.1" unitdist="inch" unit="inch" style="lines" multiple="1" display="no" altdistance="0.01" altunitdist="inch" altunit="inch"/>
 <layers>
 <layer number="1" name="Top" color="4" fill="1" visible="no" active="no"/>
@@
 <part name="LED3" library="Tova" deviceset="LED_RGB_*" device="PLCC-6"/>
 <part name="TRIPLE_BAR_GND4" library="psas_eagle_library-2" deviceset="SUP_GND_BAR_TRIPLE" device="" value="GND"/>
-<part name="R3" library="rcl_custom" deviceset="R-US_" device="0603-B-NOSILK" value="50"/>
-<part name="R4" library="rcl_custom" deviceset="R-US_" device="0603-B-NOSILK" value="50"/>
-<part name="R5" library="rcl_custom" deviceset="R-US_" device="0603-B-NOSILK" value="50"/>
+<part name="R3" library="rcl_custom" deviceset="R-US_" device="0603-B-NOSILK" value="900"/>
+<part name="R4" library="rcl_custom" deviceset="R-US_" device="0603-B-NOSILK" value="400"/>
+<part name="R5" library="rcl_custom" deviceset="R-US_" device="0603-B-NOSILK" value="110"/>
 <part name="C2" library="rcl_custom" deviceset="C-EU" device="0805-B-NOSILK" value="10u"/>
 </parts>
@@
 <instance part="R3" gate="R" x="154.94" y="111.76" smashed="yes" rot="MR0">
 <attribute name="NAME" x="153.67" y="114.3" size="1.778" layer="95" rot="MR0"/>
-<attribute name="VALUE" x="158.75" y="114.3" size="1.778" layer="96" rot="MR0"/>
+<attribute name="VALUE" x="161.29" y="114.3" size="1.778" layer="96" rot="MR0"/>
 </instance>
 <instance part="R4" gate="R" x="154.94" y="104.14" smashed="yes" rot="MR0">
 <attribute name="NAME" x="153.67" y="106.68" size="1.778" layer="95" rot="MR0"/>
-<attribute name="VALUE" x="158.75" y="106.68" size="1.778" layer="96" rot="MR0"/>
+<attribute name="VALUE" x="161.29" y="106.68" size="1.778" layer="96" rot="MR0"/>
 </instance>
 <instance part="R5" gate="R" x="154.94" y="96.52" smashed="yes" rot="MR0">
 <attribute name="NAME" x="153.67" y="99.06" size="1.778" layer="95" rot="MR0"/>
-<attribute name="VALUE" x="158.75" y="99.06" size="1.778" layer="96" rot="MR0"/>
+<attribute name="VALUE" x="161.29" y="99.06" size="1.778" layer="96" rot="MR0"/>
 </instance>
 <instance part="C2" gate="CE" x="50.8" y="33.02"/>
