File: av3/e407-roll-control/e407-roll-control.brd (EAGLE design)
At the start: 101.6 x 85.6 mm, 26 parts, among them CON1 CON1, CON2 CON1, CON4 CON4, J1 ROCKETNET-CONNECTOR-16M, T1 ALT4532, T2 ALT4532

Commit message: STM32-E407 -based roll control module, with onboard SPS.
Parts:
- added C2: 100nF, rcl_custom:0603-B-NOSILK
- added C3: NP, rcl_custom:0603-B-NOSILK
- added JP1, JP3: (no value), pinhead:1X02
- added JP2, JP5: (no value), pinhead:1X03
- added R6, R8: 100, rcl_custom:0603-B-NOSILK
- added R7, R9: 4.7k, rcl_custom:0603-B-NOSILK
- added TP5: TPPAD1-13, testpad:P1-13
- added U1, U2: SN65220DBV, sn65220:SOT23-6L
Connections:
- new net LAUNCHDETECT: C2.2, PD.14, R6.1, R7.2, U1.4
- new net N$31: JP1.1, R6.2
- new net N$32: JP5.1, TP5.TP
- new net N$33: JP2.1, R8.1
- new net N$34: JP2.2, JP5.2, U2.4
- new net PWM: C3.2, PD.18, R8.2, R9.2, U2.6
- net TRIPLE_BAR_GND: now also C2.1, C3.1, JP1.2, JP2.3, JP3.1, JP5.3, U1.2, U1.5, U2.2, U2.5
- net TRIPLE_UP_ARROW: now also JP3.2
- net UP_ARROW: now also R7.1, R9.1
Routing:
- net PWM: track 0.00 -> 61.3 mm, vias 0 -> 2
- net LAUNCHDETECT: track 0.00 -> 56.7 mm
- net UP_ARROW: track 5.08 -> 37.5 mm
- net N$34: track 0.00 -> 19.7 mm, vias 0 -> 2
- net N$32: track 0.00 -> 7.68 mm
- net N$33: track 0.00 -> 6.82 mm, vias 0 -> 1
- net N$31: track 0.00 -> 6.82 mm, vias 0 -> 1
- net TRIPLE_UP_ARROW: track 85.2 -> 89.0 mm

Commit message: Various changes to daughterboards, including updating libraries, etc. ISSUE: Connectors still flipped on "bottom" of boards.
Parts:
- R3: value 50 -> 900
- R4: value 50 -> 400
- R5: value 50 -> 110
Changed lines of the file:
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@@
 <layer number="14" name="Route14" color="1" fill="6" visible="no" active="no"/>
 <layer number="15" name="Route15" color="4" fill="6" visible="no" active="no"/>
-<layer number="16" name="Bottom" color="1" fill="1" visible="yes" active="yes"/>
+<layer number="16" name="Bottom" color="1" fill="1" visible="no" active="yes"/>
 <layer number="17" name="Pads" color="2" fill="1" visible="yes" active="yes"/>
 <layer number="18" name="Vias" color="2" fill="1" visible="yes" active="yes"/>
@@
 <layer number="20" name="Dimension" color="15" fill="1" visible="yes" active="yes"/>
 <layer number="21" name="tPlace" color="7" fill="1" visible="yes" active="yes"/>
-<layer number="22" name="bPlace" color="7" fill="1" visible="yes" active="yes"/>
+<layer number="22" name="bPlace" color="7" fill="1" visible="no" active="yes"/>
 <layer number="23" name="tOrigins" color="15" fill="1" visible="yes" active="yes"/>
-<layer number="24" name="bOrigins" color="15" fill="1" visible="yes" active="yes"/>
+<layer number="24" name="bOrigins" color="15" fill="1" visible="no" active="yes"/>
 <layer number="25" name="tNames" color="7" fill="1" visible="no" active="yes"/>
 <layer number="26" name="bNames" color="7" fill="1" visible="no" active="yes"/>
@@
 <layer number="50" name="dxf" color="7" fill="1" visible="no" active="no"/>
 <layer number="51" name="tDocu" color="7" fill="1" visible="yes" active="yes"/>
-<layer number="52" name="bDocu" color="7" fill="1" visible="yes" active="yes"/>
+<layer number="52" name="bDocu" color="7" fill="1" visible="no" active="yes"/>
 <layer number="53" name="tGND_GNDA" color="7" fill="9" visible="no" active="no"/>
 <layer number="54" name="bGND_GNDA" color="1" fill="9" visible="no" active="no"/>
@@
 <param name="mvStopFrame" value="1"/>
 <param name="mvCreamFrame" value="0"/>
-<param name="mlMinStopFrame" value="3mil"/>
-<param name="mlMaxStopFrame" value="3mil"/>
+<param name="mlMinStopFrame" value="1mil"/>
+<param name="mlMaxStopFrame" value="1mil"/>
 <param name="mlMinCreamFrame" value="0mil"/>
 <param name="mlMaxCreamFrame" value="0mil"/>
@@
 <element name="R2" library="rcl_custom" package="0603-B-NOSILK" value="50" x="17.626" y="29.202" rot="R180"/>
 <element name="LED3" library="Tova" package="PLCC-6" value="" x="47.4" y="11.3"/>
-<element name="R3" library="rcl_custom" package="0603-B-NOSILK" value="50" x="43" y="12.4"/>
-<element name="R4" library="rcl_custom" package="0603-B-NOSILK" value="50" x="43" y="10.2"/>
-<element name="R5" library="rcl_custom" package="0603-B-NOSILK" value="50" x="51.6" y="10.2" rot="R180"/>
+<element name="R3" library="rcl_custom" package="0603-B-NOSILK" value="900" x="43" y="12.4"/>
+<element name="R4" library="rcl_custom" package="0603-B-NOSILK" value="400" x="43" y="10.2"/>
+<element name="R5" library="rcl_custom" package="0603-B-NOSILK" value="110" x="51.6" y="10.2" rot="R180"/>
 <element name="U1" library="sn65220" package="SOT23-6L" value="SN65220DBV" x="49.53" y="51.054" rot="R180"/>
 <element name="C2" library="rcl_custom" package="0603-B-NOSILK" value="100nF" x="46.228" y="48.514"/>
