File: av3/e407-roll-control/e407-roll-control.sch (EAGLE design)
At the start: 26 parts, among them CON1 CON1, CON2 CON1, CON4 CON4, J1 ROCKETNET-CONNECTOR-16M, T1 ALT4532, T2 ALT4532

Commit message: STM32-E407 -based roll control module, with onboard SPS.
Parts:
- added C2: 100nF, rcl_custom:C-EU0603-B-NOSILK
- added C3: NP, rcl_custom:C-EU0603-B-NOSILK
- added JP1, JP3: (no value), pinhead:PINHD-1X2
- added JP2, JP5: (no value), pinhead:PINHD-1X3
- added R6, R8: 100, rcl_custom:R-US_0603-B-NOSILK
- added R7, R9: 4.7k, rcl_custom:R-US_0603-B-NOSILK
- added TP5: TPPAD1-13, testpad:TPPAD1-13
- added U1, U2: SN65220DBV, sn65220:SN65220DBV
Connections:
- new net LAUNCHDETECT: C2.2, PD.14, R6.1, R7.2, U1.B
- new net N$31: JP1.1, R6.2
- new net N$32: JP5.1, TP5.TP
- new net N$33: JP2.1, R8.1
- new net N$34: JP2.2, JP5.2, U2.B
- new net PWM: C3.2, PD.18, R8.2, R9.2, U2.A
- net TRIPLE_BAR_GND: now also C2.1, C3.1, JP1.2, JP2.3, JP3.1, JP5.3, U1.GND, U1.GND2, U2.GND, U2.GND2
- net TRIPLE_UP_ARROW: now also JP3.2
- net UP_ARROW: now also R7.1, R9.1
Other:
- note added: "6V out SPS"
- note added: "Launch Detect Tether"
- note added: "Roll Control Servo"

Commit message: Various changes to daughterboards, including updating libraries, etc. ISSUE: Connectors still flipped on "bottom" of boards.
Parts:
- R3: value 50 -> 900
- R4: value 50 -> 400
- R5: value 50 -> 110
Changed lines of the file:
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@@
 <setting verticaltext="up"/>
 </settings>
-<grid distance="0.05" unitdist="inch" unit="inch" style="lines" multiple="2" display="yes" altdistance="0.01" altunitdist="inch" altunit="inch"/>
+<grid distance="0.1" unitdist="inch" unit="inch" style="lines" multiple="1" display="no" altdistance="0.01" altunitdist="inch" altunit="inch"/>
 <layers>
 <layer number="1" name="Top" color="4" fill="1" visible="no" active="no"/>
@@
 <part name="LED3" library="Tova" deviceset="LED_RGB_*" device="PLCC-6"/>
 <part name="TRIPLE_BAR_GND4" library="psas_eagle_library-2" deviceset="SUP_GND_BAR_TRIPLE" device="" value="GND"/>
-<part name="R3" library="rcl_custom" deviceset="R-US_" device="0603-B-NOSILK" value="50"/>
-<part name="R4" library="rcl_custom" deviceset="R-US_" device="0603-B-NOSILK" value="50"/>
-<part name="R5" library="rcl_custom" deviceset="R-US_" device="0603-B-NOSILK" value="50"/>
+<part name="R3" library="rcl_custom" deviceset="R-US_" device="0603-B-NOSILK" value="900"/>
+<part name="R4" library="rcl_custom" deviceset="R-US_" device="0603-B-NOSILK" value="400"/>
+<part name="R5" library="rcl_custom" deviceset="R-US_" device="0603-B-NOSILK" value="110"/>
 <part name="U1" library="sn65220" deviceset="SN65220" device="DBV"/>
 <part name="TRIPLE_BAR_GND2" library="psas_eagle_library-2" deviceset="SUP_GND_BAR_TRIPLE" device="" value="GND"/>
