File: av4/rocketnet-connector/eagle/rocketnet-daughter-18.brd (EAGLE design)
At the start: 20 x 6.6 mm, 8 parts

Commit message: 18 pin rocketnet connector specifically for RNH umbilical cable.
Parts:
- moved E$12 1.60 mm to (-4.40, -1.90)
- moved E$9 1.60 mm to (4.40, -1.90)
Changed lines of the file:
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@@
 <layer number="47" name="Measures" color="7" fill="1" visible="no" active="yes"/>
 <layer number="48" name="Document" color="7" fill="1" visible="yes" active="yes"/>
-<layer number="49" name="Reference" color="7" fill="1" visible="no" active="yes"/>
+<layer number="49" name="Reference" color="7" fill="1" visible="yes" active="yes"/>
 <layer number="50" name="dxf" color="7" fill="1" visible="no" active="yes"/>
 <layer number="51" name="tDocu" color="7" fill="1" visible="yes" active="yes"/>
@@
 <rectangle x1="-0.4" y1="-2.8" x2="0.4" y2="2.8" layer="16"/>
 <rectangle x1="0.8" y1="0.3" x2="6" y2="2.8" layer="16"/>
-<rectangle x1="-6.7" y1="-2.8" x2="-3.4" y2="-1.1" layer="16"/>
+<rectangle x1="-5.9" y1="-2.8" x2="-3.4" y2="-1.1" layer="16"/>
 <text x="0.5" y="3.7" size="0.762" layer="48" rot="R90">RKTRDY</text>
 <rectangle x1="-2.9" y1="-2.8" x2="-0.8" y2="-1.1" layer="16"/>
 <rectangle x1="0.8" y1="-2.8" x2="2.9" y2="-1.1" layer="16"/>
-<rectangle x1="3.4" y1="-2.8" x2="6.7" y2="-1.1" layer="16"/>
+<rectangle x1="3.4" y1="-2.8" x2="5.9" y2="-1.1" layer="16"/>
 <rectangle x1="-2.1" y1="-1.1" x2="-0.9" y2="0" layer="16"/>
 <rectangle x1="0.9" y1="-1.1" x2="2.1" y2="0" layer="16"/>
@@
 <rectangle x1="-4" y1="-0.5" x2="-2.4" y2="2.8" layer="1"/>
 <rectangle x1="2.4" y1="-0.6" x2="4" y2="2.8" layer="1"/>
-<rectangle x1="3.4" y1="-2.8" x2="6.7" y2="-1.1" layer="1"/>
-<rectangle x1="-6.7" y1="-2.8" x2="-3.4" y2="-1.1" layer="1"/>
+<rectangle x1="3.4" y1="-2.8" x2="5.9" y2="-1.1" layer="1"/>
+<rectangle x1="-5.9" y1="-2.8" x2="-3.4" y2="-1.1" layer="1"/>
 <rectangle x1="-2.1" y1="-2.8" x2="-0.9" y2="0" layer="1"/>
 <rectangle x1="0.9" y1="-2.8" x2="2.1" y2="0" layer="1"/>
@@
 <element name="E$4" library="rocketnet-connector" package="22AWG-WIRE" value="" x="3.2" y="0.3" rot="R90"/>
 <element name="E$8" library="rocketnet-connector" package="26AWG-WIRE" value="" x="1.5" y="-0.5" rot="R90"/>
-<element name="E$9" library="rocketnet-connector" package="26AWG-WIRE" value="" x="6" y="-1.9" rot="R90"/>
+<element name="E$9" library="rocketnet-connector" package="26AWG-WIRE" value="" x="4.4" y="-1.9" rot="R90"/>
 <element name="E$10" library="rocketnet-connector" package="26AWG-WIRE" value="" x="0" y="0" rot="R90"/>
-<element name="E$12" library="rocketnet-connector" package="26AWG-WIRE" value="" x="-6" y="-1.9" rot="R90"/>
+<element name="E$12" library="rocketnet-connector" package="26AWG-WIRE" value="" x="-4.4" y="-1.9" rot="R90"/>
 <element name="E$13" library="rocketnet-connector" package="26AWG-WIRE" value="" x="-1.5" y="-0.5" rot="R90"/>
 </elements>
