File: av4/rocketnet-connector/eagle/rocketnet-daughter-16-RA.brd (EAGLE design)
At the start: 19.9 x 7.7 mm, 7 parts

Commit message: Another try on the rocketnet connector: expanded drills (0.9 mm), added second 45 degree for fun.
Parts:
- removed B+, E$4: (no value), rocketnet-connector:22AWG-WIRE
- removed E$12, E$13, E$14, E$15: (no value), rocketnet-connector:26AWG-WIRE
Connections:
- removed net B+: B+.P$1
- removed net B-: E$4.P$1
- removed net RX+: E$14.P$1
- removed net RX-: E$15.P$1
- removed net TX+: E$12.P$1
- removed net TX-: E$13.P$1
Routing:
- net RX-: track 14.5 -> 13.3 mm, vias 2 -> 3
- net TX+: track 13.1 -> 11.9 mm, vias 2 -> 3
- net B-: track 13.7 -> 13.0 mm, vias 2 -> 3
- net B+: track 9.91 -> 10.5 mm, vias 2 -> 3
- net TX-: track 14.2 -> 14.4 mm, vias 2 -> 3
- net RX+: track 14.3 -> 14.6 mm, vias 2 -> 3
Other:
- outline, holes or cut-outs redrawn
