File: av4/rocketnet-connector/eagle/rocketnet-daughter-18-RA-down.brd (EAGLE design)
At the start: 21.2 x 7.7 mm, 1 part

Commit message: Received boards from OSH Park: made minor changes to board for future runs: moved silk screen and moved edge of board away from wire holes, which are clipped in the first run.
Other:
- board size 21.2 x 7.7 mm -> 21.2 x 8.3 mm
Changed lines of the file:
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@@
 <layer number="27" name="tValues" color="7" fill="1" visible="no" active="yes"/>
 <layer number="28" name="bValues" color="7" fill="1" visible="no" active="yes"/>
-<layer number="29" name="tStop" color="7" fill="3" visible="no" active="yes"/>
+<layer number="29" name="tStop" color="7" fill="3" visible="yes" active="yes"/>
 <layer number="30" name="bStop" color="7" fill="6" visible="no" active="yes"/>
 <layer number="31" name="tCream" color="7" fill="4" visible="no" active="yes"/>
@@
 <plain>
 <wire x1="10.287" y1="-3.175" x2="10.287" y2="1.27" width="0.02" layer="20"/>
-<wire x1="10.287" y1="1.27" x2="6.985" y2="4.572" width="0.02" layer="20"/>
+<wire x1="10.287" y1="1.27" x2="6.477" y2="5.08" width="0.02" layer="20"/>
 <wire x1="10.287" y1="-3.175" x2="-10.922" y2="-3.175" width="0.02" layer="20"/>
-<wire x1="6.985" y1="4.572" x2="-7.6454" y2="4.572" width="0.02" layer="20"/>
-<wire x1="-7.6454" y1="4.572" x2="-10.922" y2="1.27" width="0.02" layer="20"/>
+<wire x1="6.477" y1="5.08" x2="-7.112" y2="5.08" width="0.02" layer="20"/>
+<wire x1="-7.112" y1="5.08" x2="-10.922" y2="1.27" width="0.02" layer="20"/>
 <wire x1="-10.922" y1="1.27" x2="-10.922" y2="-3.175" width="0.02" layer="20"/>
 <circle x="8.135" y="-0.0762" radius="2.159" width="0.0254" layer="51"/>

Commit message: Updated RNC for Umbilical with new "!umb_detect" signal. Also added old LPKF 16 pin RNC that should have been committed long ago.
Routing:
- net RR: track 5.71 -> 2.03 mm
- net !UD: track 0.00 -> 2.03 mm, vias 0 -> 1
Other:
- board size 21.2 x 8.3 mm -> 21.2 x 12.8 mm
- board text added: "!UMB"
- board text removed: "RKTRDY"
