File: av4/node6/node6_pcb/node6-gfe.brd (EAGLE design)
At the start: 100 x 80 mm, 17 parts, among them J1 MICROSDMOL500873, J15 Auxiliary Header, J2 ROCKETNET-CONNECTOR-16M, U1 DP83630/LLP

Commit message: node6: added generic stm32 to pcb for reference (will move to customized symbol). Added datasheets for several parts.
Parts:
- added U$1: STM32F407V100-PIN_QFP, stm32:LQFP-100
Changed lines of the file:
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@@
 <element name="C4" library="rcl_custom" package="0402-B-NOSILK" value="100n" x="31" y="13"/>
 <element name="C5" library="rcl_custom" package="0402-B-NOSILK" value="100n" x="31" y="15"/>
+<element name="U$1" library="stm32" package="LQFP-100" value="STM32F407V100-PIN_QFP" x="30" y="33"/>
 </elements>
 <signals>

Commit message: node6: removed eagle project file from source control. Added node6 specific stm32 symbol, connected rmii
Parts:
- removed U$1: STM32F407V100-PIN_QFP, stm32:LQFP-100
- added U2: STM32F407V_NODE6/LQFP100, stm32:QFP50P1600X1600X160-100N
- moved J1 9.22 mm to (59.0, 30.0), turned to 270 degrees
Connections:
- new net N$13: U1.2, U2.48
- new net N$14: U1.3, U2.51
- new net N$15: U1.4, U2.52
- new net N$16: U1.46, U2.33
- new net N$17: U1.45, U2.34
- new net N$18: U1.34, U2.67
- new net N$19: U1.30, U2.25
- new net N$20: U1.31, U2.16
- new net N$3: U1.1, U2.24
Changed lines of the file:
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@@
 <layer number="25" name="tNames" color="7" fill="1" visible="yes" active="yes"/>
 <layer number="26" name="bNames" color="7" fill="1" visible="yes" active="yes"/>
-<layer number="27" name="tValues" color="7" fill="1" visible="yes" active="yes"/>
-<layer number="28" name="bValues" color="7" fill="1" visible="yes" active="yes"/>
+<layer number="27" name="tValues" color="7" fill="1" visible="no" active="yes"/>
+<layer number="28" name="bValues" color="7" fill="1" visible="no" active="yes"/>
 <layer number="29" name="tStop" color="7" fill="3" visible="no" active="yes"/>
 <layer number="30" name="bStop" color="7" fill="6" visible="no" active="yes"/>
@@
 </autorouter>
 <elements>
-<element name="J1" library="connector" package="MOLEX-MICROSD-500873" value="MICROSDMOL500873" x="68" y="32"/>
+<element name="J1" library="connector" package="MOLEX-MICROSD-500873" value="MICROSDMOL500873" x="59" y="30" rot="R270"/>
 <element name="U1" library="DP83630" package="QFN50P700X700X80-49N" value="DP83630/LLP" x="43" y="13" rot="R270"/>
 <element name="LED1" library="LED_RGB_PLCC6" package="PLCC-6" value="" x="43" y="21"/>
@@
 <element name="C4" library="rcl_custom" package="0402-B-NOSILK" value="100n" x="31" y="13"/>
 <element name="C5" library="rcl_custom" package="0402-B-NOSILK" value="100n" x="31" y="15"/>
-<element name="U$1" library="stm32" package="LQFP-100" value="STM32F407V100-PIN_QFP" x="30" y="33"/>
+<element name="U2" library="stm32" package="QFP50P1600X1600X160-100N" value="STM32F407V_NODE6/LQFP100" x="61" y="12" rot="R180"/>
 </elements>
 <signals>
@@
 <wire x1="30.52" y1="15" x2="28.15" y2="16.905" width="0" layer="19" extent="1-1"/>
 </signal>
+<signal name="N$3">
+<contactref element="U2" pad="24"/>
+<contactref element="U1" pad="1"/>
+<wire x1="68.7" y1="17.5" x2="45.75" y2="16.5" width="0" layer="19" extent="1-1"/>
+</signal>
+<signal name="N$13">
+<contactref element="U2" pad="48"/>
+<contactref element="U1" pad="2"/>
+<wire x1="56" y1="19.7" x2="45.25" y2="16.5" width="0" layer="19" extent="1-1"/>
+</signal>
+<signal name="N$14">
+<contactref element="U2" pad="51"/>
+<contactref element="U1" pad="3"/>
+<wire x1="53.3" y1="18" x2="44.75" y2="16.5" width="0" layer="19" extent="1-1"/>
+</signal>
+<signal name="N$15">
+<contactref element="U2" pad="52"/>
+<contactref element="U1" pad="4"/>
+<wire x1="53.3" y1="17.5" x2="44.25" y2="16.5" width="0" layer="19" extent="1-1"/>
+</signal>
+<signal name="N$16">
+<contactref element="U2" pad="33"/>
+<contactref element="U1" pad="46"/>
+<wire x1="63.5" y1="19.7" x2="46.5" y2="14.75" width="0" layer="19" extent="1-1"/>
+</signal>
+<signal name="N$17">
+<contactref element="U2" pad="34"/>
+<contactref element="U1" pad="45"/>
+<wire x1="63" y1="19.7" x2="46.5" y2="14.25" width="0" layer="19" extent="1-1"/>
+</signal>
+<signal name="N$18">
+<contactref element="U2" pad="67"/>
+<contactref element="U1" pad="34"/>
+<wire x1="53.3" y1="10" x2="44.75" y2="9.5" width="0" layer="19" extent="1-1"/>
+</signal>
+<signal name="N$19">
+<contactref element="U2" pad="25"/>
+<contactref element="U1" pad="30"/>
+<wire x1="68.7" y1="18" x2="42.75" y2="9.5" width="0" layer="19" extent="1-1"/>
+</signal>
+<signal name="N$20">
+<contactref element="U2" pad="16"/>
+<contactref element="U1" pad="31"/>
+<wire x1="68.7" y1="13.5" x2="43.25" y2="9.5" width="0" layer="19" extent="1-1"/>
+</signal>
 </signals>
