File: av4/node6/node6_pcb/node6-gfe.sch (EAGLE design)
At the start: 2 parts, among them J1 MICROSDMOL500873, U1 STM32F407V100-PIN_QFP

Commit message: removed backup files, new node6-specific symbol and package for stm32
Parts:
- removed U1: STM32F407V100-PIN_QFP, STM32:STM32F407V100-PIN_QFP
Changed lines of the file:
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@@
 <parts>
 <part name="FRAME1" library="frames" deviceset="TABL_L" device=""/>
-<part name="U1" library="STM32" deviceset="STM32F407V" device="100-PIN_QFP"/>
 <part name="J1" library="connector" deviceset="MICROSD" device="MOL500873"/>
 </parts>
@@
 <instance part="FRAME1" gate="G$1" x="0" y="0"/>
 <instance part="FRAME1" gate="G$2" x="299.72" y="0"/>
-<instance part="U1" gate="U1" x="241.3" y="139.7"/>
 <instance part="J1" gate="G$1" x="327.66" y="195.58"/>
 </instances>

Commit message: enet phy for node6
Parts:
- added U1: DP83630/LLP, DP83630:DP83630/LLP
Changed lines of the file:
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@@
 <part name="FRAME1" library="frames" deviceset="TABL_L" device=""/>
 <part name="J1" library="connector" deviceset="MICROSD" device="MOL500873"/>
+<part name="U1" library="DP83630" deviceset="DP83630" device="/LLP"/>
 </parts>
 <sheets>
@@
 <instance part="FRAME1" gate="G$2" x="299.72" y="0"/>
 <instance part="J1" gate="G$1" x="327.66" y="195.58"/>
+<instance part="U1" gate="A" x="327.66" y="109.22"/>
 </instances>
 <busses>

Commit message: new ethernet transformer, enet connection and termination
Parts:
- added C1, C2, C4, C5: 100n, rcl_custom:C-EU0402-B-NOSILK
- added C3: 1n, rcl_custom:C-EU0402-B-NOSILK
- added J15: Auxiliary Header, headers:1.27MM_HDR_1X4
- added J2: ROCKETNET-CONNECTOR-16M, rocketnet-connector:ROCKETNET-CONNECTOR-16M
- added L1: PULSE-H0068ANL/SO, magnetics:PULSE-H0068ANL/SO
- added LED1: (no value), LED_RGB_PLCC6:LED_RGB_PLCC-6
- added R1, R2, R3, R4: 49.9, rcl_custom:R-US_0402-B-NOSILK
- added R5, R6: 75.0, rcl_custom:R-US_0402-B-NOSILK
Connections:
- new net ENET_RD+: L1.TD+, R3.2, U1.RD+
- new net ENET_RD-: L1.TD-, R4.2, U1.RD-
- new net ENET_TD+: L1.RD+, R1.2, U1.TD+
- new net ENET_TD-: L1.RD-, R2.2, U1.TD-
- new net GND: C1.2, C2.2, C3.2, C4.2, C5.2
- new net N$1: J2.TX-@1, J2.TX-@2, L1.RX-
- new net N$10: C3.1, R5.1, R6.1
- new net N$11: C4.1, L1.RDCT
- new net N$12: C5.1, L1.TDCT
- new net N$2: J2.RX+@1, J2.RX+@2, L1.TX+
- new net N$4: J2.RX-@1, J2.RX-@2, L1.TX-
- new net N$5: C1.1, R1.1, R2.1
- new net N$6: J2.TX+@1, J2.TX+@2, L1.RX+
- new net N$7: L1.TXCT, R5.2
- new net N$8: C2.1, R3.1, R4.1
- new net N$9: L1.RXCT, R6.2
Other:
- moved on the sheet: U1

Commit message: node6: added generic stm32 to pcb for reference (will move to customized symbol). Added datasheets for several parts.
Parts:
- added U$1: STM32F407V100-PIN_QFP, stm32:STM32F407V100-PIN_QFP
Changed lines of the file:
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@@
 <part name="GND3" library="supply1" deviceset="GND" device=""/>
 <part name="GND4" library="supply1" deviceset="GND" device=""/>
+<part name="U$1" library="stm32" deviceset="STM32F407V" device="100-PIN_QFP"/>
 </parts>
 <sheets>
@@
 <instance part="GND3" gate="1" x="289.56" y="99.06"/>
 <instance part="GND4" gate="1" x="299.72" y="99.06"/>
+<instance part="U$1" gate="G$1" x="119.38" y="93.98"/>
 </instances>
 <busses>

Commit message: node6: removed eagle project file from source control. Added node6 specific stm32 symbol, connected rmii
Parts:
- removed U$1: STM32F407V100-PIN_QFP, stm32:STM32F407V100-PIN_QFP
- added U2: STM32F407V_NODE6/LQFP100, stm32:STM32F407V_NODE6/LQFP100
Connections:
- new net N$13: U1.TX_EN, U2.PB11ETH_RMII_TX_EN
- new net N$14: U1.TXD_0, U2.PB12/ETH_RMII_TXD0
- new net N$15: U1.TXD_1, U2.PB13/ETH_RMII_TXD1
- new net N$16: U1.RXD_0, U2.PC4/ETH_RMII_RX_D0
- new net N$17: U1.RXD_1, U2.PC5/ETH_RMII_RX_D1
- new net N$18: U1.X1, U2.PA8/MCO1
- new net N$19: U1.MDIO, U2.PA2/ETH_MDIO
- new net N$20: U1.MDC, U2.PC1/ETH_MDC
- new net N$3: U1.TX_CLK, U2.PA1/ETH_RMII_REF_CLK
Other:
- moved on the sheet: C1, C2, C3, C4, C5, J1, J15, J2, L1, R1, R2, R3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
