File: av4/node6/eagle/node6-gfe.brd (EAGLE design)
At the start: 100 x 80 mm, 18 parts, among them J1 MICROSDMOL500873, J15 Auxiliary Header, J2 ROCKETNET-CONNECTOR-16M, U1 DP83630/LLP, U2 STM32F407V_NODE6/LQFP100

Commit message: node6: hooked up aux connector to rocketnet
Parts:
- moved J2 2.00 mm to (3.00, 15.0), turned to 90 degrees
Connections:
- new net N$21: J15.1, J2.A1
- new net N$22: J15.2, J2.A2
- new net N$23: J15.3, J2.A3
- new net N$24: J15.4, J2.A4
Changed lines of the file:
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@@
 <attribute name="TOLERANCE" value="1%" x="34" y="9" size="1.778" layer="27" display="off"/>
 </element>
-<element name="J2" library="rocketnet-connector" package="ROCKETNET-M-16" value="ROCKETNET-CONNECTOR-16M" x="5" y="15" rot="R270"/>
+<element name="J2" library="rocketnet-connector" package="ROCKETNET-M-16" value="ROCKETNET-CONNECTOR-16M" x="3" y="15" rot="R90"/>
 <element name="J15" library="headers" package="INLINE" value="Auxiliary Header" x="15.63" y="3.95" rot="R90"/>
 <element name="C1" library="rcl_custom" package="0402-B-NOSILK" value="100n" x="32" y="10"/>
@@
 <contactref element="J2" pad="B-@1"/>
 <contactref element="J2" pad="B-@2"/>
-<wire x1="4.365" y1="19.445" x2="5.635" y2="19.445" width="0" layer="19" extent="1-1"/>
+<wire x1="3.635" y1="10.555" x2="2.365" y2="10.555" width="0" layer="19" extent="1-1"/>
 </signal>
 <signal name="B+">
 <contactref element="J2" pad="B+@16"/>
 <contactref element="J2" pad="B+@15"/>
-<wire x1="4.365" y1="10.555" x2="5.635" y2="10.555" width="0" layer="19" extent="1-1"/>
+<wire x1="3.635" y1="19.445" x2="2.365" y2="19.445" width="0" layer="19" extent="1-1"/>
 </signal>
 <signal name="ENET_TD+">
@@
 <contactref element="J2" pad="T-@9"/>
 <contactref element="J2" pad="T-@11"/>
-<wire x1="4.365" y1="13.095" x2="19.85" y2="11.825" width="0" layer="19" extent="1-1"/>
-<wire x1="4.365" y1="14.365" x2="4.365" y2="13.095" width="0" layer="19" extent="1-1"/>
+<wire x1="3.635" y1="16.905" x2="19.85" y2="11.825" width="0" layer="19" extent="1-1"/>
+<wire x1="3.635" y1="15.635" x2="3.635" y2="16.905" width="0" layer="19" extent="1-1"/>
 </signal>
 <signal name="N$2">
@@
 <contactref element="J2" pad="R+@7"/>
 <contactref element="J2" pad="R+@5"/>
-<wire x1="4.365" y1="16.905" x2="19.85" y2="18.175" width="0" layer="19" extent="1-1"/>
-<wire x1="4.365" y1="15.635" x2="4.365" y2="16.905" width="0" layer="19" extent="1-1"/>
+<wire x1="3.635" y1="13.095" x2="19.85" y2="18.175" width="0" layer="19" extent="1-1"/>
+<wire x1="3.635" y1="14.365" x2="3.635" y2="13.095" width="0" layer="19" extent="1-1"/>
 </signal>
 <signal name="N$4">
@@
 <contactref element="J2" pad="R-@4"/>
 <contactref element="J2" pad="R-@3"/>
-<wire x1="5.635" y1="18.175" x2="19.85" y2="19.445" width="0" layer="19" extent="1-1"/>
-<wire x1="4.365" y1="18.175" x2="5.635" y2="18.175" width="0" layer="19" extent="1-1"/>
+<wire x1="2.365" y1="11.825" x2="19.85" y2="19.445" width="0" layer="19" extent="1-1"/>
+<wire x1="3.635" y1="11.825" x2="2.365" y2="11.825" width="0" layer="19" extent="1-1"/>
 </signal>
 <signal name="N$6">
@@
 <contactref element="J2" pad="T+@13"/>
 <contactref element="J2" pad="T+@14"/>
-<wire x1="5.635" y1="11.825" x2="19.85" y2="10.555" width="0" layer="19" extent="1-1"/>
-<wire x1="4.365" y1="11.825" x2="5.635" y2="11.825" width="0" layer="19" extent="1-1"/>
+<wire x1="2.365" y1="18.175" x2="19.85" y2="10.555" width="0" layer="19" extent="1-1"/>
+<wire x1="3.635" y1="18.175" x2="2.365" y2="18.175" width="0" layer="19" extent="1-1"/>
 </signal>
 <signal name="N$9">
@@
 <wire x1="68.7" y1="13.5" x2="43.25" y2="9.5" width="0" layer="19" extent="1-1"/>
 </signal>
+<signal name="N$21">
+<contactref element="J2" pad="A1"/>
+<contactref element="J15" pad="1"/>
+<wire x1="2.365" y1="13.095" x2="13.725" y2="3.95" width="0" layer="19" extent="1-1"/>
+</signal>
+<signal name="N$22">
+<contactref element="J15" pad="2"/>
+<contactref element="J2" pad="A2"/>
+<wire x1="2.365" y1="14.365" x2="14.995" y2="3.95" width="0" layer="19" extent="1-1"/>
+</signal>
+<signal name="N$23">
+<contactref element="J15" pad="3"/>
+<contactref element="J2" pad="A3"/>
+<wire x1="2.365" y1="15.635" x2="16.265" y2="3.95" width="0" layer="19" extent="1-1"/>
+</signal>
+<signal name="N$24">
+<contactref element="J15" pad="4"/>
+<contactref element="J2" pad="A4"/>
+<wire x1="2.365" y1="16.905" x2="17.535" y2="3.95" width="0" layer="19" extent="1-1"/>
+</signal>
 </signals>

Commit message: node6: finished sd card symbol. added sd and power supply front end to schematic
Parts:
- removed J1: MICROSDMOL500873, connector:MOLEX-MICROSD-500873
- added C2000: 100n 50V, rcl_custom:0603-B-NOSILK
- added C2001: 22u 50V, rcl:D/7343-31R
- added C2002: 330n 50V, rcl_custom:0603-B-NOSILK
- added C2003: 2.7u, rcl_custom:0603-B-NOSILK
- added C2004: 15n, rcl_custom:0603-B-NOSILK
- added C2011: 10n 50V, rcl_custom:0603-B-NOSILK
- added D2001: CDSU101A, psas_eagle_library:0603-DIODE
- added F2000: 2.0A Fast, custom:1206
- added J3: MICROSD-7T-DET504077, sd_card:MOLEX_504077-1891
- added L2000: CMS1, choke:CMS1
- added Q2000, Q2002: PMV45EN, Tova:SOT23
- added Q2001: Si7309DN, 0kaz:1212-8_POWERPAK
- added R2000: 100k, rcl_custom:0603-B-NOSILK
- added R2001: 61.9k, rcl_custom:0603-B-NOSILK
- added R2002, R2012: 10k, rcl_custom:0603-B-NOSILK
- added R2003: .033, rcl_custom:0805-B-NOSILK
- added R2004: 1k, rcl_custom:0603-B-NOSILK
- added R2005: 34.0k 1%, rcl_custom:0603-B-NOSILK
- added R2006: 10k 1%, rcl_custom:0603-B-NOSILK
- added TVS2000: TVS_SMB, 0kaz:DO-214AA/SMB
- added U2000: MAX5902AAEUT, node4:SOT23-6
- added U2001: TLV3012AIDBVT, node4:SOT23-6
- turned U2 to 270 degrees
Connections:
- net N$1 renamed RNET_TX-
- net N$2 renamed RNET_RX+
- net N$21 renamed RNET_AUX1
- net N$22 renamed RNET_AUX2
- net N$23 renamed RNET_AUX3
- net N$24 renamed RNET_AUX4
- net N$4 renamed RNET_RX-
- net N$6 renamed RNET_TX+
- removed net ANAVSS: U1.18
- removed net B+: J2.B+@15, J2.B+@16
- removed net B-: J2.B-@1, J2.B-@2
- removed net CD_VSS: U1.15
- removed net IO_CORE_VSS: U1.35
- removed net IO_VSS: U1.47
- new net BIN: F2000.1, L2000.3
- new net CHASSIS: C2000.1, R2000.1
- new net IN+: C2004.1, R2005.1, R2006.2, U2001.3
- new net MAX_UVLO: Q2000.3, R2001.1, R2002.2, U2000.6
- new net N$334: Q2001.5-6-7-8, R2003.1
- new net N_DRAIN: Q2002.3, R2004.1, U2000.2
- new net N_GATE: C2004.2, Q2002.1, U2001.1
- new net PORT1.0/GPIO_SPS_DISABLE: Q2000.1, R2012.2
- new net PORT1.1/GPIO_SPS_V-IN_GOOD: U2000.5
- new net P_GATE: Q2001.4, U2000.3
- new net REF: U2001.4, U2001.5
- new net RNET_B+: J2.B+@15, J2.B+@16, L2000.4
- new net RNET_B-: J2.B-@1, J2.B-@2, L2000.1
- new net SPS_OUT: D2001.A, R2005.2
- new net V+1: C2003.2, D2001.K, U2001.6
- new net VIN: R2003.2, R2004.2
- new net V_FUSED: C2001.+, C2002.2, C2011.2, F2000.2, Q2001.1-2-3, R2001.2, TVS2000.CATHODE, U2000.1
- net GND: now also C2000.2, C2001.-, C2002.1, C2003.1, C2011.1, J3.T1, J3.T2, J3.T3, J3.T4, J3.T5, J3.T6, J3.T7, L2000.2, Q2000.2, Q2002.2, R2000.2, R2002.1, R2006.1, R2012.1, TVS2000.ANODE, U1.15, U1.18, U1.35, U1.47, U1.49, U2000.4, U2001.2
- net SD_CLK: now also J3.5, U2.80; no longer J1.5
- net SD_CMD: now also J3.3, U2.83; no longer J1.3
- net SD_DAT0: now also J3.7, U2.65; no longer J1.7
- net SD_DAT1: now also J3.8, U2.66; no longer J1.8
- net SD_DAT2: now also J3.1, U2.78; no longer J1.1
- net SD_DAT3: now also J3.2, U2.79; no longer J1.2
- net VDD: now also J3.4; no longer J1.4
- net VSS: now also J3.6; no longer J1.6

Commit message: node6: added ltm8023 power supply
Parts:
- added C103: 2.2u/40V, rcl_custom:0603-B-NOSILK
- added C104: 2.2u, rcl_custom:0603-B-NOSILK
- added J13: PGOOD Jumper, headers:1.27MM_2X1
- added LED22: GREEN, led:CHIPLED_0603
- added R128: 750, rcl_custom:0402-B-NOSILK
- added R131: 10k, rcl_custom:0402-B-NOSILK
- added R73: 154k, rcl_custom:0402-B-NOSILK
- added R74: 49.9k, rcl_custom:0402-B-NOSILK
- added U5: LTM8023, RNH_LTM8023:LGA-50
Connections:
- removed net VIN: R2003.2, R2004.2
- new net +18V: C103.1, R2003.2, R2004.2, U5.RUN/SS, U5.VIN@1, U5.VIN@2, U5.VIN@3, U5.VIN@4, U5.VIN@5, U5.VIN@6
- new net +3V3: C104.1, R128.1, U5.VOUT@1, U5.VOUT@10, U5.VOUT@11, U5.VOUT@12, U5.VOUT@2, U5.VOUT@3, U5.VOUT@4, U5.VOUT@5, U5.VOUT@6, U5.VOUT@7, U5.VOUT@8, U5.VOUT@9
- new net N$116: R73.2, U5.ADJ
- new net N$117: R74.2, U5.RT
- new net N$29: J13.2, LED22.A, U5.PGOOD
- new net N$30: J13.1, R128.2
- new net N$37: U5.AUX, U5.BIAS
- new net SD_DETECT: J3.DET
- new net SYNC: R131.1, U5.SYNC
- net GND: now also C103.2, C104.2, LED22.C, R131.2, R73.1, R74.1, U5.GND@1, U5.GND@10, U5.GND@11, U5.GND@12, U5.GND@13, U5.GND@14, U5.GND@15, U5.GND@16, U5.GND@17, U5.GND@18, U5.GND@19, U5.GND@2, U5.GND@20, U5.GND@21, U5.GND@22, U5.GND@23, U5.GND@24, U5.GND@3, U5.GND@4, U5.GND@5, U5.GND@6, U5.GND@7, U5.GND@8, U5.GND@9

Commit message: node6: new regulator library, added ltc3586, primary switcher output +5
moving toward ltc3586 as main switching chip to generate 3.3 and 5, buck
regulators available to generate other supplies if needed in other
projects.
Parts:
- removed J13: PGOOD Jumper, headers:1.27MM_2X1
- removed R128: 750, rcl_custom:0402-B-NOSILK
- added U3: LTC3586, regulator:QFN40P600X400X75-39N
- R73: value 154k -> 93.1k
- moved U5 84.9 mm to (17.0, 31.0)
Connections:
- removed net +3V3: C104.1, R128.1, U5.VOUT@1, U5.VOUT@10, U5.VOUT@11, U5.VOUT@12, U5.VOUT@2, U5.VOUT@3, U5.VOUT@4, U5.VOUT@5, U5.VOUT@6, U5.VOUT@7, U5.VOUT@8, U5.VOUT@9
- removed net N$29: J13.2, LED22.A, U5.PGOOD
- removed net N$30: J13.1, R128.2
- new net +5V_RAW: C104.1, U3.35, U3.36, U5.VOUT@1, U5.VOUT@10, U5.VOUT@11, U5.VOUT@12, U5.VOUT@2, U5.VOUT@3, U5.VOUT@4, U5.VOUT@5, U5.VOUT@6, U5.VOUT@7, U5.VOUT@8, U5.VOUT@9
- new net PGOOD_5V: LED22.A, U5.PGOOD
- net GND: now also U3.39
