File: av4/battery-board/eagle/battery-board.brd (EAGLE design)
At the start: 71.2 x 35.3 mm, 71 parts, among them J1 ROCKETNET-BATTERY-14, J100 87758-0216, J101 87758-0216, Q100 SI4435DDY, Q101 SI4435DDY, Q102 SI4435DDY, Q103 SI1023X, Q104 SI1023X, U100 BQ3060PW

Commit message: Updated battery board after reviewing EVM and messing around the BQ3060 with Kenny on the RNH tonight.
Parts:
- removed C100: 100n, rcl_custom:0603-B-NOSILK
- removed D103, D104: >5V TVS, tvs-0603:0603-B-NOSILK-DIODE
- removed D105: > 5V TVS, tvs-0603:0603-B-NOSILK-DIODE
- removed J1: ROCKETNET-BATTERY-14, rocketnet-connector:ROCKETNET-CONNECTOR-M-14
- added J102: 87758-0216, con-molex:87758-0216
- C115: value 100n -> 100n/100V
- D100: value > 20 V TVS -> TVS-0603
- F100: value 20A -> 10A slow blow
- J100: value 87758-0216 -> ROCKETNET-BATTERY-14; device con-molex:87758-0216 -> rocketnet-connector:ROCKETNET-M-14
- moved J100 28.1 mm to (23.0, 32.3), turned to 0 degrees
- moved F100 19.2 mm to (25.1, 8.12), turned to 0 degrees
- moved R102 5.01 mm to (26.0, 11.1)
- moved J101 2.29 mm to (47.8, 19.1)
- moved D100 2.20 mm to (22.0, 28.3)
- moved C115 1.98 mm to (22.0, 26.7)
- moved C107 1.13 mm to (52.3, 32.5), turned to 180 degrees
- moved C106 1.13 mm to (56.6, 32.5), turned to 180 degrees
- moved C108 1.13 mm to (48.0, 32.5), turned to 180 degrees
- moved R100 0.80 mm to (11.2, 14.9)
- moved R104 0.32 mm to (12.2, 25.9)
Connections:
- removed net N$37: C100.2, C115.1
- removed net N$43: C100.1, C117.2, D100.ANODE, D102.ANODE, F100.1, Q100.1, Q100.2, Q100.3, Q102.1, Q102.2, Q102.3, R101.1, R104.1
- new net B+FUSED: C116.1, D101.ANODE, F100.1, Q101.1, Q101.2, Q101.3, R103.1
- net B+: now also F100.2; no longer C116.1, D101.ANODE, Q101.1, Q101.2, Q101.3, R103.1
- net B+PACKOUT: now also C115.1, C117.2, D100.ANODE, D102.ANODE, J100.B+@1, J100.B+@2, J100.B+@3, J100.B+@4, Q100.1, Q100.2, Q100.3, Q102.1, Q102.2, Q102.3, R101.1, R104.1; no longer F100.2, J1.B+@1, J1.B+@2, J1.B+@3, J1.B+@4
- net BAR_GND: now also J102.2; no longer J100.2
- net N$1: now also J101.1; no longer J100.1
- net N$2: now also J102.1; no longer J101.1
- net N$22: now also J100.SMDAT@7, J100.SMDAT@8; no longer D103.ANODE, J1.SMDAT@7, J1.SMDAT@8
- net N$25: now also J100.SMCLK@3, J100.SMCLK@4; no longer D104.ANODE, J1.SMCLK@3, J1.SMCLK@4
- net N$35: now also J100.!PRSNT@10, J100.!PRSNT@9; no longer D105.ANODE, J1.!PRSNT@10, J1.!PRSNT@9
- net TRIANGLE_GND: now also J100.B-@11, J100.B-@12, J100.B-@13, J100.B-@14; no longer D103.CATHODE, D104.CATHODE, D105.CATHODE, J1.B-@11, J1.B-@12, J1.B-@13, J1.B-@14
Routing:
- net B+PACKOUT: track 0.00 -> 51.4 mm, vias 0 -> 2
- net N$43: track 51.1 -> 0.00 mm, vias 2 -> 0
- net B+FUSED: track 0.00 -> 45.0 mm, vias 0 -> 2
- net B+: track 46.3 -> 6.26 mm, vias 1 -> 0
- net TRIANGLE_GND: track 47.7 -> 53.2 mm
- net N$19: track 43.2 -> 48.0 mm
- net N$25: track 37.5 -> 35.3 mm
- net N$22: track 39.8 -> 38.2 mm
- net N$37: track 1.50 -> 0.00 mm
- net N$24: track 26.4 -> 27.0 mm
- net N$17: track 24.9 -> 25.5 mm
- net N$33: track 26.6 -> 27.2 mm
- added copper zone on layer 1, net B+FUSED
- removed copper zone on layer 1, net N$43

Commit message: Interim step in the battery board. Commit early, commit often.
Parts:
- removed TP104, TP105: TEST-POINT, Tova:2MM-TEST-POINT
- added C118: 100n/50V, rcl_custom:0603-B-NOSILK
- C103, C104: value 1u -> 1u 40V
- C115: value 100n/100V -> 100n/50V
- C116, C117: value 100n -> 100n/50V
- D100: value TVS-0603 -> SMBJ20A; device tvs-0603:0603-B-NOSILK-DIODE -> diode:SMBJ
- F100: value 10A slow blow -> 0501010.WR
- Q100: value SI4435DDY -> Si2343DS-T1; device si4435ddy:SO-8 -> Tova:SOT23
- R100: value 301 1W -> 249 0.5W
- R101, R102, R103, R104, R106, R107, R108, R109, R111, R119, R120, R121: device rcl_custom:0402-B-NOSILK -> rcl_custom:0603-B-NOSILK
- moved TP102 51.5 mm to (6.40, 13.5)
- moved TP101 51.3 mm to (5.90, 25.4)
- moved TP100 32.6 mm to (22.5, 9.60)
- moved F100 21.7 mm to (16.0, 27.8)
- moved C117 12.4 mm to (17.7, 20.0)
- moved C116 6.37 mm to (17.7, 11.9), turned to 90 degrees
- moved R108 4.55 mm to (5.30, 16.0)
- moved R107 3.11 mm to (8.50, 24.3)
- moved R101 2.93 mm to (7.50, 21.8)
- moved R100 2.46 mm to (9.00, 16.0)
- moved C115 2.19 mm to (23.5, 25.1)
- moved Q101 2.10 mm to (14.2, 12.1)
- moved Q102 2.10 mm to (14.2, 20.1)
- moved R103 1.92 mm to (17.7, 8.80)
- moved Q100 1.75 mm to (7.50, 19.2), turned to 0 degrees
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Connections:
- net N$15 renamed SMBD
- net N$16 renamed SMBC
- net N$22 renamed RNC-SDAT
- net N$25 renamed RNC-SCLK
- net N$3 renamed BAT
- net N$31 renamed PACK
- net N$35 renamed RNC-!PRSNT
- net N$45 renamed !PRES
- removed net B+FUSED: C116.1, D101.ANODE, F100.1, Q101.1, Q101.2, Q101.3, R103.1
- removed net B+PACKOUT: C115.1, C117.2, D100.ANODE, D102.ANODE, J100.B+@1, J100.B+@2, J100.B+@3, J100.B+@4, Q100.1, Q100.2, Q100.3, Q102.1, Q102.2, Q102.3, R101.1, R104.1
- new net N$15: C115.1, C118.2
- new net PACK+: F100.1, J100.B+@1, J100.B+@2, J100.B+@3, J100.B+@4
- new net PACK+PREFUSE: C117.2, C118.1, D100.C, D102.ANODE, F100.2, Q100.2, Q102.1, Q102.2, Q102.3, R101.1, R104.1
- net B+: now also C116.1, D101.ANODE, Q101.1, Q101.2, Q101.3, R103.1; no longer F100.2
- net N$39: now also Q100.1; no longer Q100.4
- net N$5: no longer TP104.1
- net N$6: no longer TP105.1
- net PRE-CHARGE: now also Q100.3; no longer Q100.5, Q100.6, Q100.7, Q100.8
- net TRIANGLE_GND: now also D100.A; no longer D100.CATHODE
Routing:
- net B+PACKOUT: track 51.4 -> 0.00 mm, vias 2 -> 0
- net PACK+PREFUSE: track 0.00 -> 50.4 mm, vias 0 -> 2
- net B+FUSED: track 45.0 -> 0.00 mm, vias 2 -> 0
- net B+: track 6.26 -> 41.2 mm, vias 0 -> 1
- net N$7: track 25.8 -> 16.1 mm
- net N$40: track 14.5 -> 6.50 mm
- net N$12: track 40.7 -> 33.3 mm
- net N$36: track 10.7 -> 4.43 mm
- net N$29: track 80.3 -> 75.9 mm
- net PRE-CHARGE: track 0.00 -> 4.34 mm
- net N$5: track 15.2 -> 11.0 mm
- net N$6: track 13.9 -> 10.5 mm
- net BAR_GND: track 26.2 -> 23.2 mm
- net N$11: track 40.3 -> 37.7 mm
- net TRIANGLE_GND: track 53.2 -> 51.1 mm
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- added copper zone on layer 1, net PACK+
- added copper zone on layer 1, net PACK+PREFUSE
- removed copper zone on layer 1, net B+FUSED
- removed copper zone on layer 1, net B+PACKOUT
- removed copper zone on layer 1, net PRE-CHARGE
Other:
- board text added: "PSAS Battery Board v1 - http://psas.pdx.edu/"
- board text removed: "PSAS Battery Board v1"

Commit message: Latest battery boards notes, handing off to Michael for final polishing.
Parts:
- C101, C102, C105, C109, C111, C112, C113, C114: device rcl_custom:0402-B-NOSILK -> rcl_custom:0603-B-NOSILK
Routing:
- net N$6: track 10.5 -> 11.1 mm
Changed lines of the file:
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@@
 <element name="R120" library="rcl_custom" package="0603-B-NOSILK" value="100" x="46" y="24.9"/>
 <element name="R121" library="rcl_custom" package="0603-B-NOSILK" value="100" x="46" y="23.8"/>
-<element name="C111" library="rcl_custom" package="0402-B-NOSILK" value="100n" x="48.9" y="25.3" rot="R270"/>
-<element name="C113" library="rcl_custom" package="0402-B-NOSILK" value="100n" x="48.9" y="23.3" rot="R270"/>
-<element name="C112" library="rcl_custom" package="0402-B-NOSILK" value="100n" x="47.7" y="24.3" rot="R270"/>
+<element name="C111" library="rcl_custom" package="0603-B-NOSILK" value="100n" x="48.9" y="25.3" rot="R270"/>
+<element name="C113" library="rcl_custom" package="0603-B-NOSILK" value="100n" x="48.9" y="23.3" rot="R270"/>
+<element name="C112" library="rcl_custom" package="0603-B-NOSILK" value="100n" x="47.7" y="24.3" rot="R270"/>
 <element name="R102" library="rcl_custom" package="0603-B-NOSILK" value="1K" x="26" y="11.1" rot="R90"/>
 <element name="R109" library="rcl_custom" package="0603-B-NOSILK" value="1K" x="22.1" y="16.8" rot="R270"/>
 <element name="R111" library="rcl_custom" package="0603-B-NOSILK" value="1K" x="25.2" y="21.5"/>
 <element name="R119" library="rcl_custom" package="0603-B-NOSILK" value="1K" x="23.7" y="22.9"/>
-<element name="C101" library="rcl_custom" package="0402-B-NOSILK" value="100n" x="47.8" y="10.6"/>
-<element name="C102" library="rcl_custom" package="0402-B-NOSILK" value="100n" x="47.8" y="12.4"/>
-<element name="C105" library="rcl_custom" package="0402-B-NOSILK" value="100n" x="47.8" y="13.4"/>
-<element name="C114" library="rcl_custom" package="0402-B-NOSILK" value="100n" x="47.8" y="15.2"/>
-<element name="C109" library="rcl_custom" package="0402-B-NOSILK" value="100n" x="63.2" y="20.2"/>
+<element name="C101" library="rcl_custom" package="0603-B-NOSILK" value="100n" x="47.8" y="10.6"/>
+<element name="C102" library="rcl_custom" package="0603-B-NOSILK" value="100n" x="47.8" y="12.4"/>
+<element name="C105" library="rcl_custom" package="0603-B-NOSILK" value="100n" x="47.8" y="13.4"/>
+<element name="C114" library="rcl_custom" package="0603-B-NOSILK" value="100n" x="47.8" y="15.2"/>
+<element name="C109" library="rcl_custom" package="0603-B-NOSILK" value="100n" x="63.2" y="20.2"/>
 <element name="C110" library="rcl_custom" package="0603-B-NOSILK" value="1u" x="63.2" y="21.9"/>
 <element name="D101" library="diode-0603" package="0603-B-NOSILK-DIODE" value="DIODE-0603" x="53.2" y="26.6"/>
@@
 <contactref element="C112" pad="1"/>
 <wire x1="46.8" y1="24.9" x2="47.58" y2="24.9" width="0.2" layer="1"/>
-<wire x1="47.58" y1="24.9" x2="47.7" y2="24.78" width="0.2" layer="1"/>
-<wire x1="47.7" y1="24.78" x2="48.78" y2="24.78" width="0.2" layer="1"/>
+<wire x1="47.58" y1="24.9" x2="47.7" y2="25.1" width="0.2" layer="1"/>
+<wire x1="47.7" y1="25.1" x2="48.78" y2="24.78" width="0.2" layer="1"/>
 <wire x1="48.78" y1="24.78" x2="48.8" y2="24.8" width="0.2" layer="1"/>
 <wire x1="48.8" y1="24.8" x2="48.88" y2="24.8" width="0.2" layer="1"/>
-<wire x1="48.88" y1="24.8" x2="48.9" y2="24.82" width="0.2" layer="1"/>
-<wire x1="48.9" y1="24.82" x2="49.78" y2="24.82" width="0.2" layer="1"/>
+<wire x1="48.88" y1="24.8" x2="48.9" y2="24.5" width="0.2" layer="1"/>
+<wire x1="48.9" y1="24.5" x2="49.78" y2="24.82" width="0.2" layer="1"/>
 <wire x1="49.78" y1="24.82" x2="50.7" y2="23.9" width="0.2" layer="1"/>
 <wire x1="50.7" y1="23.9" x2="50.7" y2="21" width="0.2" layer="1"/>
@@
 <contactref element="C112" pad="2"/>
 <wire x1="46.8" y1="23.8" x2="47.68" y2="23.8" width="0.2" layer="1"/>
-<wire x1="47.68" y1="23.8" x2="47.7" y2="23.82" width="0.2" layer="1"/>
-<wire x1="47.7" y1="23.82" x2="48.86" y2="23.82" width="0.2" layer="1"/>
-<wire x1="48.86" y1="23.82" x2="48.9" y2="23.78" width="0.2" layer="1"/>
-<wire x1="48.9" y1="23.78" x2="49.52" y2="23.78" width="0.2" layer="1"/>
+<wire x1="47.68" y1="23.8" x2="47.7" y2="23.5" width="0.2" layer="1"/>
+<wire x1="47.7" y1="23.5" x2="48.86" y2="23.82" width="0.2" layer="1"/>
+<wire x1="48.86" y1="23.82" x2="48.9" y2="24.1" width="0.2" layer="1"/>
+<wire x1="48.9" y1="24.1" x2="49.52" y2="23.78" width="0.2" layer="1"/>
 <wire x1="49.52" y1="23.78" x2="50.2" y2="23.1" width="0.2" layer="1"/>
 <wire x1="50.2" y1="23.1" x2="50.2" y2="20.8" width="0.2" layer="1"/>
@@
 <wire x1="52.4" y1="15.2" x2="48.9" y2="11.7" width="0.2" layer="1"/>
 <wire x1="48.9" y1="11.7" x2="48.3" y2="11.7" width="0.2" layer="1"/>
-<wire x1="48.28" y1="12.4" x2="48.3" y2="12.38" width="0.2" layer="1"/>
+<wire x1="48.6" y1="12.4" x2="48.3" y2="12.38" width="0.2" layer="1"/>
 <wire x1="48.3" y1="12.38" x2="48.3" y2="11.7" width="0.2" layer="1"/>
 <wire x1="48.3" y1="11.7" x2="40.8" y2="11.7" width="0.2" layer="1"/>
@@
 <wire x1="49.9" y1="14.1" x2="48.3" y2="14.1" width="0.2" layer="1"/>
 <wire x1="48.3" y1="14.1" x2="45.9" y2="14.1" width="0.2" layer="1"/>
-<wire x1="48.28" y1="13.4" x2="48.28" y2="14.08" width="0.2" layer="1"/>
+<wire x1="48.6" y1="13.4" x2="48.28" y2="14.08" width="0.2" layer="1"/>
 <wire x1="48.28" y1="14.08" x2="48.3" y2="14.1" width="0.2" layer="1"/>
 <wire x1="45.9" y1="14.1" x2="42.45" y2="17.55" width="0.2" layer="1"/>
@@
 <via x="51.8" y="17.1" extent="1-16" drill="0.2032"/>
 <wire x1="51.8" y1="17.1" x2="49.2" y2="14.5" width="0.2" layer="1"/>
-<wire x1="48.28" y1="15.2" x2="48.28" y2="14.58" width="0.2" layer="1"/>
+<wire x1="48.6" y1="15.2" x2="48.28" y2="14.58" width="0.2" layer="1"/>
 <wire x1="49.2" y1="14.5" x2="48.2" y2="14.5" width="0.2" layer="1"/>
 <wire x1="48.2" y1="14.5" x2="46" y2="14.5" width="0.2" layer="1"/>
@@
 <wire x1="59.8" y1="19.875" x2="61.175" y2="19.875" width="0.3" layer="1"/>
 <wire x1="61.175" y1="19.875" x2="61.5" y2="20.2" width="0.3" layer="1"/>
-<wire x1="61.5" y1="20.2" x2="62.72" y2="20.2" width="0.3" layer="1"/>
+<wire x1="61.5" y1="20.2" x2="62.4" y2="20.2" width="0.3" layer="1"/>
 </signal>
 <signal name="N$14">
@@
 <wire x1="49.1" y1="11.3" x2="48.28" y2="11.3" width="0.2" layer="1"/>
 <wire x1="48.28" y1="11.3" x2="40.7" y2="11.3" width="0.2" layer="1"/>
-<wire x1="48.28" y1="10.6" x2="48.28" y2="11.3" width="0.2" layer="1"/>
+<wire x1="48.6" y1="10.6" x2="48.28" y2="11.3" width="0.2" layer="1"/>
 <wire x1="40.7" y1="11.3" x2="31.8" y2="16.6" width="0.2" layer="1"/>
 <wire x1="26" y1="11.9" x2="26" y2="16.3" width="0.2" layer="1"/>
@@
 <contactref element="C117" pad="1"/>
 <contactref element="C116" pad="2"/>
-<wire x1="17.7" y1="19.2" x2="17.7" y2="12.7" width="0.4" layer="1"/>
+<wire x1="17.7" y1="19.2" x2="17.7" y2="12.7" width="0.7" layer="1"/>
 </signal>
 <signal name="N$1">
@@
 <contactref element="C115" pad="1"/>
 <contactref element="C118" pad="2"/>
-<wire x1="21.2" y1="25.1" x2="22" y2="25.1" width="0.4" layer="1"/>
-<wire x1="22" y1="25.1" x2="22.5" y2="25.1" width="0.4" layer="1"/>
-<wire x1="22.5" y1="25.1" x2="22.6" y2="25" width="0.4" layer="1"/>
-<wire x1="22.7" y1="25.1" x2="22.5" y2="25.1" width="0.4" layer="1"/>
+<wire x1="21.2" y1="25.1" x2="22.7" y2="25.1" width="0.7" layer="1"/>
 </signal>
 <signal name="PACK+">

Commit message: updated routing
Parts:
- moved R109 3.13 mm to (22.5, 13.7)
- moved Q103 2.40 mm to (24.5, 14.0)
- moved R105 1.88 mm to (20.8, 13.7), turned to 270 degrees
Routing:
- net N$19: track 47.8 -> 31.7 mm
- net N$10: track 47.0 -> 60.3 mm, vias 2 -> 3
- net N$12: track 33.4 -> 20.5 mm
- net N$11: track 37.8 -> 27.2 mm
- net N$8: track 31.0 -> 24.3 mm, vias 1 -> 0
- net N$21: track 1.36 -> 5.65 mm
- net B+: track 41.2 -> 39.1 mm
- net N$20: track 1.70 -> 0.00 mm
- net RNC-!PRSNT: track 28.9 -> 30.1 mm
- net RNC-SDAT: track 38.4 -> 39.4 mm
- net N$4: track 22.8 -> 23.6 mm
- removed copper zone on layer 16, net BAR_GND

Commit message: finished laout
Parts:
- moved R111 3.18 mm to (23.9, 18.6), turned to 90 degrees
- moved R122 3.08 mm to (24.1, 23.1), turned to 0 degrees
- moved R119 2.72 mm to (22.1, 20.7), turned to 270 degrees
- moved C102 2.00 mm to (47.8, 10.4)
- moved R116 1.97 mm to (20.2, 20.7)
- moved C101 1.80 mm to (47.8, 8.80)
- moved R110 1.25 mm to (25.8, 18.6)
- moved R120 1.21 mm to (44.9, 25.4)
- moved R121 1.10 mm to (44.9, 23.8)
- moved C105 1.00 mm to (47.8, 12.4)
- moved C111 0.90 mm to (48.9, 26.2)
- moved Q104 0.81 mm to (24.2, 21.0)
- moved C114 0.80 mm to (47.8, 14.4)
- moved R114 0.70 mm to (65.5, 16.5)
- moved R117 0.70 mm to (65.5, 14.5)
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Routing:
- net N$12: track 20.5 -> 48.6 mm
- net N$11: track 27.2 -> 47.3 mm, vias 2 -> 0
- net N$19: track 31.7 -> 49.6 mm
- net N$7: track 16.5 -> 29.7 mm
- net N$10: track 60.3 -> 51.0 mm, vias 3 -> 2
- net N$9: track 0.00 -> 5.63 mm
- net N$20: track 0.00 -> 3.30 mm
- net N$18: track 0.00 -> 1.65 mm
- net N$33: track 27.2 -> 28.7 mm
- net TRIANGLE_GND: track 51.1 -> 49.6 mm
- net N$4: track 23.6 -> 25.0 mm
- net BAR_GND: track 23.2 -> 22.0 mm, vias 15 -> 16
- net N$6: track 11.1 -> 12.0 mm
- net N$5: track 11.5 -> 12.2 mm
- net SMBD: track 5.88 -> 6.58 mm
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
Commit message: moved some routing to top layer, needs drc work
Parts:
- removed C106, C107, C108: 100p, rcl_custom:0603-B-NOSILK
- removed R112, R114, R117: 200, rcl_custom:0603-B-NOSILK
- removed R113, R115, R118: 100, rcl_custom:0603-B-NOSILK
- moved TP100 15.6 mm to (7.30, 5.90)
- moved R106 11.9 mm to (8.10, 8.60), turned to 180 degrees
- moved R103 8.12 mm to (9.70, 10.2), turned to 180 degrees
- moved R110 2.91 mm to (24.5, 16.0), turned to 0 degrees
- moved TP102 1.14 mm to (5.30, 13.2)
- moved R111 1.08 mm to (24.8, 19.2), turned to 180 degrees
Connections:
- removed net N$17: C106.1, R117.1, R118.2
- removed net N$24: C107.1, R114.1, R115.2
- removed net N$33: C108.1, R112.1, R113.2
- removed net RNC-!PRSNT: J100.!PRSNT@10, J100.!PRSNT@9, R113.1
- removed net RNC-SDAT: J100.SMDAT@7, J100.SMDAT@8, R118.1
- removed net SMBC: R114.2, TP107.1, U100.16
- net !PRES: now also J100.!PRSNT@10, J100.!PRSNT@9; no longer R112.2
- net RNC-SCLK: now also TP107.1, U100.16; no longer R115.1
- net SMBD: now also J100.SMDAT@7, J100.SMDAT@8; no longer R117.2
- net TRIANGLE_GND: no longer C106.2, C107.2, C108.2
Routing:
- net SMBD: track 6.58 -> 60.7 mm, vias 0 -> 1
- net !PRES: track 5.10 -> 56.3 mm
- net RNC-SDAT: track 39.4 -> 0.00 mm, vias 1 -> 0
- net TRIANGLE_GND: track 49.6 -> 15.0 mm, vias 1 -> 0
- net RNC-!PRSNT: track 30.1 -> 0.00 mm, vias 1 -> 0
- net N$33: track 28.7 -> 0.00 mm
- net N$24: track 27.4 -> 0.00 mm
- net N$17: track 25.6 -> 0.00 mm
- net RNC-SCLK: track 36.2 -> 60.2 mm, vias 1 -> 0
- net N$27: track 46.9 -> 67.1 mm, vias 1 -> 0
- net B+: track 39.1 -> 48.7 mm
- net N$8: track 24.6 -> 33.7 mm
- net PACK+PREFUSE: track 50.4 -> 59.3 mm, vias 2 -> 0
- net N$34: track 3.10 -> 11.6 mm
- net N$4: track 25.0 -> 31.2 mm
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
Commit message: final routing of battery board. DRC passed. Ready for post-processing and artwork generation.
Parts:
- moved F100 1.98 mm to (14.7, 26.3), turned to 270 degrees
- moved R119 1.93 mm to (22.2, 18.8)
- moved R116 1.91 mm to (20.0, 18.8)
- moved R122 1.72 mm to (25.1, 21.7), turned to 180 degrees
- moved R111 1.41 mm to (26.2, 19.0), turned to 90 degrees
- moved Q104 1.20 mm to (24.2, 19.8)
- moved R110 1.14 mm to (25.4, 16.7), turned to 180 degrees
- moved Q103 1.12 mm to (24.0, 15.0)
- moved R105 1.12 mm to (20.0, 14.7)
- moved R109 1.00 mm to (22.1, 14.7)
- moved R102 0.14 mm to (26.1, 11.2)
Routing:
- net N$7: track 29.7 -> 82.3 mm
- net N$8: track 33.7 -> 82.8 mm
- net N$4: track 31.2 -> 78.1 mm
- net RNC-SCLK: track 60.2 -> 104.6 mm, vias 0 -> 1
- net !PRES: track 56.3 -> 100.7 mm, vias 0 -> 1
- net SMBD: track 60.7 -> 102.3 mm
- net B+: track 48.7 -> 53.8 mm, vias 1 -> 15
- net N$11: track 47.5 -> 46.1 mm
- net PACK+PREFUSE: track 59.3 -> 60.4 mm, vias 0 -> 12
- net N$10: track 51.0 -> 50.0 mm
- net BAR_GND: track 16.8 -> 17.6 mm, vias 14 -> 76
- net N$19: track 49.6 -> 50.2 mm
- net N$27: track 67.1 -> 66.6 mm
- net TRIANGLE_GND: vias 0 -> 14
- added copper zone on layer 16, net B+
- added copper zone on layer 2, net B+
- added copper zone on layer 3, net B+
- added copper zone on layer 16, net BAR_GND
- added copper zone on layer 3, net BAR_GND
- added copper zone on layer 16, net N$28
- added copper zone on layer 2, net N$28
- added copper zone on layer 3, net N$28
- added copper zone on layer 16, net PACK+
- added copper zone on layer 2, net PACK+
- added copper zone on layer 3, net PACK+
- added copper zone on layer 16, net PACK+PREFUSE
- added copper zone on layer 2, net PACK+PREFUSE
- added copper zone on layer 3, net PACK+PREFUSE
- added copper zone on layer 16, net TRIANGLE_GND
- added copper zone on layer 2, net TRIANGLE_GND
- added copper zone on layer 3, net TRIANGLE_GND

Commit message: Final cleanup on battery board. Made stitching more focused on power rather than RF, redid shunt library part to be a real kelvin connection (see Analog Devices cute write up on Kelvin sense shunt resistors), changes all polygons to be consistenly 0.2 mm wid and 0.2 mm isolate.
Parts:
- moved TP101 1.10 mm to (5.90, 24.3)
- moved C112 0.60 mm to (47.3, 24.0)
- moved C113 0.60 mm to (48.9, 22.4)
- moved R105 0.60 mm to (20.6, 14.7)
- moved R116 0.60 mm to (20.6, 18.8)
- moved R121 0.60 mm to (44.9, 23.2)
- moved C111 0.60 mm to (48.9, 25.6)
- moved R120 0.60 mm to (44.9, 24.8)
- moved Q101 0.10 mm to (14.2, 12.0)
- moved R119 0.07 mm to (22.1, 18.8)
- turned R123 to 180 degrees
Connections:
- new net N$16: R121.1, R123.K2
- new net N$3: R120.1, R123.K1
- net BAR_GND: now also R123.1@1, R123.1@2; no longer R120.1, R123.P$1
- net TRIANGLE_GND: now also R123.2@1, R123.2@2; no longer R121.1, R123.P$2
Routing:
- net N$16: track 0.00 -> 20.3 mm, vias 0 -> 2
- net N$3: track 0.00 -> 18.7 mm, vias 0 -> 2
- net BAR_GND: track 17.6 -> 1.93 mm, vias 76 -> 88
- net TRIANGLE_GND: track 15.0 -> 0.04 mm, vias 14 -> 12
- net N$8: track 82.8 -> 74.9 mm
- net N$4: track 78.1 -> 71.0 mm
- net N$7: track 82.3 -> 76.4 mm
- net B+: track 53.8 -> 49.7 mm, vias 15 -> 16
- net N$30: track 90.4 -> 89.3 mm
- net N$19: track 50.2 -> 49.4 mm
- net N$12: track 48.9 -> 48.1 mm
- net N$10: track 50.0 -> 49.3 mm
- net N$11: track 46.1 -> 45.4 mm
- net N$9: track 6.12 -> 5.52 mm
- net N$6: track 12.0 -> 11.4 mm
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Other:
- board text added: "2014/01/07"
- board text added: "Battery Board v1"
- board text added: "PSAS - http://psas.pdx.edu/"
- board text removed: "2013/05/01"
- board text removed: "PSAS Battery Board v1 - http://psas.pdx.edu/"
