File: av4/battery-board/eagle/battery-board.sch (EAGLE design)
At the start: 57 parts, among them J100 ROCKETNET-BATTERY-14, J101 87758-0216, J102 87758-0216, Q100 Si2343DS-T1, Q101 SI4435DDY, Q102 SI4435DDY, Q103 SI1023X, Q104 SI1023X, U100 BQ3060PW

Commit message: Final cleanup on battery board after design review today. Caught lots of polygon weirdness with ranks, redistributed the power vias, cleaned up transistor package, added ground test points.
Parts:
- added TP109, TP110: TEST-POINT, Tova:TEST-POINT
Connections:
- net N$1 renamed T1
- net N$2 renamed T2
- net N$38 renamed FUSE
- net N$4 renamed B23
- net N$7 renamed B12
- net N$8 renamed B34
- net BAR_GND: now also TP110.P$1
- net TRIANGLE_GND: now also TP109.P$1
Other:
- moved on the sheet: TP106, TP107
Changed lines of the file:
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@@
 <setting verticaltext="up"/>
 </settings>
-<grid distance="0.05" unitdist="inch" unit="inch" style="lines" multiple="2" display="no" altdistance="0.01" altunitdist="inch" altunit="inch"/>
+<grid distance="0.1" unitdist="inch" unit="inch" style="lines" multiple="1" display="no" altdistance="0.01" altunitdist="inch" altunit="inch"/>
 <layers>
 <layer number="1" name="Top" color="4" fill="1" visible="no" active="no"/>
@@
 <part name="Q100" library="Tova" deviceset="NTR4101P" device="" value="Si2343DS-T1"/>
 <part name="R123" library="shunt" deviceset="R-US-2818" device="" value="0.01 5W 1% 75ppm"/>
+<part name="TP109" library="Tova" deviceset="TEST-POINT" device=""/>
+<part name="TP110" library="Tova" deviceset="TEST-POINT" device=""/>
 </parts>
 <sheets>
@@
 <instance part="TP102" gate="G$1" x="223.52" y="160.02"/>
 <instance part="TP103" gate="G$1" x="229.87" y="139.7"/>
-<instance part="TP106" gate="G$1" x="229.87" y="129.54"/>
-<instance part="TP107" gate="G$1" x="223.52" y="127"/>
+<instance part="TP106" gate="G$1" x="238.76" y="129.54"/>
+<instance part="TP107" gate="G$1" x="229.87" y="127"/>
 <instance part="TP108" gate="G$1" x="229.87" y="121.92"/>
 <instance part="Q101" gate="G$1" x="175.26" y="200.66" smashed="yes" rot="R90">
@@
 <attribute name="VALUE" x="156.21" y="83.312" size="1.778" layer="96" rot="MR180"/>
 </instance>
+<instance part="TP109" gate="G$1" x="189.23" y="88.9"/>
+<instance part="TP110" gate="G$1" x="229.87" y="114.3"/>
 </instances>
 <busses>
@@
 <segment>
 <wire x1="78.74" y1="83.82" x2="78.74" y2="88.9" width="1.27" layer="91"/>
-<wire x1="101.6" y1="88.9" x2="78.74" y2="88.9" width="1.27" layer="91"/>
+<wire x1="100.33" y1="88.9" x2="78.74" y2="88.9" width="1.27" layer="91"/>
 <wire x1="101.6" y1="91.44" x2="101.6" y2="88.9" width="0.1524" layer="91"/>
-<wire x1="160.02" y1="88.9" x2="101.6" y2="88.9" width="1.27" layer="91"/>
+<wire x1="160.02" y1="88.9" x2="160.02" y2="77.47" width="0.1524" layer="91"/>
+<wire x1="160.02" y1="77.47" x2="229.87" y2="77.47" width="0.1524" layer="91"/>
+<wire x1="229.87" y1="77.47" x2="229.87" y2="114.3" width="0.1524" layer="91"/>
 <wire x1="78.74" y1="88.9" x2="78.74" y2="96.52" width="1.27" layer="91"/>
-<junction x="101.6" y="88.9"/>
 <junction x="78.74" y="88.9"/>
 <pinref part="BAR_GND7" gate="1" pin="BAR_GND"/>
@@
 <pinref part="R123" gate="G$1" pin="1@2"/>
 <wire x1="160.02" y1="88.9" x2="160.02" y2="91.44" width="1.27" layer="91"/>
+<pinref part="TP110" gate="G$1" pin="P$1"/>
+<wire x1="100.33" y1="88.9" x2="101.6" y2="88.9" width="1.27" layer="91"/>
+<junction x="100.33" y="88.9"/>
+<wire x1="101.6" y1="88.9" x2="160.02" y2="88.9" width="1.27" layer="91"/>
 </segment>
 <segment>
@@
 </segment>
 </net>
-<net name="N$2" class="0">
+<net name="T2" class="0">
 <segment>
 <wire x1="185.42" y1="124.46" x2="147.32" y2="124.46" width="0.1524" layer="91"/>
@@
 <net name="TRIANGLE_GND" class="0">
 <segment>
-<wire x1="175.26" y1="88.9" x2="309.88" y2="88.9" width="1.27" layer="91"/>
+<wire x1="175.26" y1="88.9" x2="189.23" y2="88.9" width="1.27" layer="91"/>
+<wire x1="189.23" y1="88.9" x2="309.88" y2="88.9" width="1.27" layer="91"/>
 <wire x1="309.88" y1="111.76" x2="309.88" y2="88.9" width="1.27" layer="91"/>
 <junction x="309.88" y="88.9"/>
@@
 <pinref part="R123" gate="G$1" pin="2@2"/>
 <wire x1="175.26" y1="91.44" x2="175.26" y2="88.9" width="1.27" layer="91"/>
+<pinref part="TP109" gate="G$1" pin="P$1"/>
+<junction x="189.23" y="88.9"/>
 </segment>
 <segment>
@@
 <pinref part="J100" gate="G$1" pin="SMCLK@1"/>
 <junction x="325.12" y="127"/>
-<wire x1="210.82" y1="127" x2="223.52" y2="127" width="0.1524" layer="91"/>
-<junction x="223.52" y="127"/>
+<wire x1="210.82" y1="127" x2="229.87" y2="127" width="0.1524" layer="91"/>
+<junction x="229.87" y="127"/>
 <pinref part="U100" gate="G$1" pin="SMBC"/>
 <pinref part="TP107" gate="G$1" pin="P$1"/>
-<wire x1="325.12" y1="127" x2="223.52" y2="127" width="0.1524" layer="91"/>
+<wire x1="325.12" y1="127" x2="229.87" y2="127" width="0.1524" layer="91"/>
+<label x="300.99" y="127" size="1.778" layer="95"/>
 </segment>
 </net>
@@
 <net name="!PRES" class="0">
 <segment>
-<wire x1="210.82" y1="129.54" x2="229.87" y2="129.54" width="0.1524" layer="91"/>
-<wire x1="229.87" y1="129.54" x2="238.76" y2="129.54" width="0.1524" layer="91"/>
+<wire x1="210.82" y1="129.54" x2="238.76" y2="129.54" width="0.1524" layer="91"/>
 <wire x1="238.76" y1="129.54" x2="238.76" y2="132.08" width="0.1524" layer="91"/>
-<wire x1="238.76" y1="132.08" x2="251.46" y2="132.08" width="0.1524" layer="91"/>
-<junction x="229.87" y="129.54"/>
+<junction x="238.76" y="129.54"/>
 <pinref part="U100" gate="G$1" pin="!PRES"/>
 <pinref part="TP106" gate="G$1" pin="P$1"/>
-<wire x1="251.46" y1="132.08" x2="255.27" y2="132.08" width="0.1524" layer="91"/>
-<wire x1="299.72" y1="132.08" x2="302.26" y2="132.08" width="0.1524" layer="91"/>
-<wire x1="302.26" y1="132.08" x2="320.04" y2="132.08" width="0.1524" layer="91"/>
 <wire x1="320.04" y1="132.08" x2="320.04" y2="116.84" width="0.1524" layer="91"/>
 <pinref part="J100" gate="G$1" pin="!PRSNT@1"/>
@@
 <wire x1="320.04" y1="114.3" x2="320.04" y2="116.84" width="0.1524" layer="91"/>
 <junction x="320.04" y="116.84"/>
-<wire x1="255.27" y1="132.08" x2="299.72" y2="132.08" width="0.1524" layer="91"/>
-</segment>
-</net>
-<net name="N$38" class="0">
+<wire x1="238.76" y1="132.08" x2="320.04" y2="132.08" width="0.1524" layer="91"/>
+<label x="300.99" y="132.08" size="1.778" layer="95"/>
+</segment>
+</net>
+<net name="FUSE" class="0">
 <segment>
 <wire x1="210.82" y1="139.7" x2="229.87" y2="139.7" width="0.1524" layer="91"/>
@@
 </segment>
 </net>
-<net name="N$7" class="0">
+<net name="B12" class="0">
 <segment>
 <wire x1="77.47" y1="104.14" x2="78.74" y2="104.14" width="1.27" layer="91"/>
@@
 </segment>
 </net>
-<net name="N$4" class="0">
+<net name="B23" class="0">
 <segment>
 <wire x1="77.47" y1="129.54" x2="78.74" y2="129.54" width="1.27" layer="91"/>
@@
 </segment>
 </net>
-<net name="N$8" class="0">
+<net name="B34" class="0">
 <segment>
 <wire x1="77.47" y1="154.94" x2="78.74" y2="154.94" width="1.27" layer="91"/>
@@
 </segment>
 </net>
-<net name="N$1" class="0">
+<net name="T1" class="0">
 <segment>
 <pinref part="U100" gate="G$1" pin="TS1"/>
@@
 <wire x1="231.14" y1="121.92" x2="232.41" y2="121.92" width="0.1524" layer="91"/>
 <wire x1="233.68" y1="121.92" x2="232.41" y2="121.92" width="0.1524" layer="91"/>
-</segment>
-</net>
+<label x="300.99" y="121.92" size="1.778" layer="95"/>
+</segment>
+</net>

Commit message: Generated BOM and made a Digi-Key order. Found an ERC error that popped up, double checked part values in writeup.
Parts:
- Q101, Q102: value SI4435DDY -> SI4413ADY-T1-E3
Changed lines of the file:
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@@
 <part name="TP107" library="Tova" deviceset="TEST-POINT" device=""/>
 <part name="TP108" library="Tova" deviceset="TEST-POINT" device=""/>
-<part name="Q101" library="si4435ddy" deviceset="SI4435DDY" device=""/>
-<part name="Q102" library="si4435ddy" deviceset="SI4435DDY" device=""/>
+<part name="Q101" library="si4435ddy" deviceset="SI4435DDY" device="" value="SI4413ADY-T1-E3"/>
+<part name="Q102" library="si4435ddy" deviceset="SI4435DDY" device="" value="SI4413ADY-T1-E3"/>
 <part name="R103" library="rcl_custom" deviceset="R-US_" device="0603-B-NOSILK" value="1M"/>
 <part name="R104" library="rcl_custom" deviceset="R-US_" device="0603-B-NOSILK" value="1M"/>
@@
 <junction x="100.33" y="88.9"/>
 <wire x1="101.6" y1="88.9" x2="160.02" y2="88.9" width="1.27" layer="91"/>
-</segment>
-<segment>
+<junction x="101.6" y="88.9"/>
+</segment>
+<segment>
