File: av4/stm32f4-dev-board/v1-psas-dev-board.sch (EAGLE design)
At the start: 88 parts, among them J1 1.27MM-SWD-CONNECTOR, J3 ROCKETNET-CONNECTOR-16M, Q1 NTR4101P, T1 ALT4532, T2 ALT4532, U10 LMZ12001, U3 LAN8710A-EZC, U8 STM32F4V, X1 25 MHz

Commit message: Updated LED connections
Connections:
- removed net N$1: U8.PA4
- removed net N$11: LED2.C, R40.2
- removed net N$12: LED3.C, R38.2
- removed net N$18: LED4.C, R39.2
- new net N$2: LED4.A, R39.2
- new net N$3: LED3.A, R38.2
- new net N$4: LED2.A, R40.2
- net LED2: now also LED2.C; no longer LED2.A
- net LED3: now also LED3.C; no longer LED3.A
- net LED4: now also LED4.C; no longer LED4.A
Other:
- note added: "MAYBE: RGB LED package instead?"
- moved on the sheet: LED2, LED3, LED4
