File: av4/raspi-camera/eagle/raspi-rnc.brd (EAGLE design)
At the start: 85 x 56 mm, 3 parts, among them J1 ROCKETNET-CONNECTOR-16M

Commit message: Moved daughterboard to behind RP (duh). Added parts form olimex DBs and olf PPC FC carrier: RNC, magnetics,  5/3.3 LTM supply, LED.
Parts:
- removed J1: ROCKETNET-CONNECTOR-16M, rocketnet-connector:ROCKETNET-M-16
- removed U$2: LT4619_REDUCED, LT4619:LT4619
- added C1: 100nF, rcl_custom:0603-B-NOSILK
- added C1000, C1007: 22p, rcl_custom:0603-B-NOSILK
- added C1001, C1008: 100u, rcl:D/7343-31R
- added C1002, C1009: 200p, rcl_custom:0603-B-NOSILK
- added C1003, C1004, C1043, C1044: 10u, rcl_custom:0805-B-NOSILK
- added C1045, C1046: 15n, rcl_custom:0603-B-NOSILK
- added J2: ROCKETNET-CONNECTOR-16M, rocketnet-connector:ROCKETNET-M-16
- added L1, L2: ACM2012, magnetics:TDK-ACM2012
- added LAN: RJLBC-060TC1, OLIMEX_CONNECTORS:RJLBC-060TC1
- added LED3: (no value), Tova:PLCC-6
- added R1, R2: 50, rcl_custom:0603-B-NOSILK
- added R1000: 11.5k, rcl_custom:0603-B-NOSILK
- added R1001: 19.1k, rcl_custom:0603-B-NOSILK
- added R1069: 0, rcl_custom:0603-B-NOSILK
- added R3: 900, rcl_custom:0603-B-NOSILK
- added R4: 400, rcl_custom:0603-B-NOSILK
- added R5: 110, rcl_custom:0603-B-NOSILK
- added T1, T2: ALT4532, magnetics:TDK-ALT4532
- added TP1, TP2, TP3, TP4: TEST-POINT, apdm:2MM-TEST-POINT
- added TP1000, TP1001, TP1002, TP1003, TP1004, TP1005, TP1007, TP1009, TP1010, TP1011, TP1234, TP1235: TEST, tqm:TEST
- added U1000: LT4619, LT4619:LT4619
Connections:
- removed net INTVCC: U$2.F6
- removed net N$1: J1.B+@15, J1.B+@16, U$2.J1, U$2.J10, U$2.J11, U$2.J12, U$2.J2, U$2.J3, U$2.K1, U$2.K10, U$2.K11, U$2.K12, U$2.K2, U$2.K3, U$2.K4, U$2.K9, U$2.L1, U$2.L10, U$2.L11, U$2.L12, U$2.L2, U$2.L3, U$2.L4, U$2.L5, U$2.L8, U$2.L9, U$2.M1, U$2.M10, U$2.M11, U$2.M12, U$2.M2, U$2.M3, U$2.M4, U$2.M5, U$2.M6, U$2.M7, U$2.M8, U$2.M9
- removed net VOUT1: U$2.A10, U$2.A11, U$2.A12, U$2.B10, U$2.B11, U$2.B12, U$2.C10, U$2.C11, U$2.C12, U$2.D10, U$2.D11, U$2.D12
- removed net VOUT2: U$2.A1, U$2.A2, U$2.A3, U$2.B1, U$2.B2, U$2.B3, U$2.C1, U$2.C2, U$2.C3, U$2.D1, U$2.D2, U$2.D3
- new net AGND: C1002.2, C1009.2, R1000.1, R1001.1, R1069.2, U1000.H6, U1000.H7, U1000.J6, U1000.J7
- new net COMP1: TP1003.P$1, U1000.L7
- new net COMP2: TP1005.P$1, U1000.L6
- new net EXTVCC: TP1001.P$1, U1000.J4
- new net FREQ: TP1000.P$1, U1000.J8
- new net INTVCC1: TP1002.P$1, U1000.F6
- new net N$10: J2.R+@5, J2.R+@7, L2.1
- new net N$11: LAN.1, T1.1
- new net N$12: LAN.2, T1.2
- new net N$13: LAN.7, T2.1
- new net N$14: LAN.8, T2.2
- new net N$15: LED3.5
- new net N$19: J2.R-@3, J2.R-@4, L2.2
- new net N$2: LED3.6
- new net N$20: J2.A4, TP4.1
- new net N$21: J2.A3, TP3.1
- new net N$22: J2.A2, TP2.1
- new net N$23: J2.A1, TP1.1
- new net N$24: LAN.3, T1.6, T2.6
- new net N$25: C1.1, R1.1, R2.1
- new net N$26: R1.2, T2.3
- new net N$27: R2.2, T1.3
- new net N$28: LED3.1, R3.2
- new net N$29: LED3.3, R4.2
- new net N$3: L1.4, T1.5
- new net N$30: LED3.4, R5.2
- new net N$4: LED3.2
- new net N$5: L1.3, T1.4
- new net N$6: L2.4, T2.5
- new net N$7: L2.3, T2.4
- new net N$8: J2.T+@13, J2.T+@14, L1.1
- new net N$9: J2.T-@11, J2.T-@9, L1.2
- new net PGOOD: TP1009.P$1, U1000.H5
- new net RUN1: TP1004.P$1, U1000.J9
- new net RUN2: TP1007.P$1, U1000.J5
- new net SPS-500KHZ: U1000.H8
- new net SW1: TP1011.P$1, U1000.H10
- new net SW2: TP1010.P$1, U1000.H3
- new net TK-SS1: C1002.1, U1000.K8
- new net TK-SS2: C1009.1, U1000.K5
- new net TRIPLE_UP_ARROW: C1003.1, C1004.1, J2.B+@15, J2.B+@16, U1000.J1, U1000.J10, U1000.J11, U1000.J12, U1000.J2, U1000.J3, U1000.K1, U1000.K10, U1000.K11, U1000.K12, U1000.K2, U1000.K3, U1000.K4, U1000.K9, U1000.L1, U1000.L10, U1000.L11, U1000.L12, U1000.L2, U1000.L3, U1000.L4, U1000.L5, U1000.L8, U1000.L9, U1000.M1, U1000.M10, U1000.M11, U1000.M12, U1000.M2, U1000.M3, U1000.M4, U1000.M5, U1000.M6, U1000.M7, U1000.M8, U1000.M9
- new net VFB1: C1000.1, R1000.2, U1000.K7
- new net VFB2: C1007.2, R1001.2, U1000.K6
- net +3V3: now also C1007.1, C1008.+, C1044.1, C1046.1, R3.1, R4.1, R5.1, TP1235.P$1, U1000.A1, U1000.A2, U1000.A3, U1000.B1, U1000.B2, U1000.B3, U1000.C1, U1000.C2, U1000.C3, U1000.D1, U1000.D2, U1000.D3
- net +5V: now also C1000.2, C1001.+, C1043.1, C1045.1, TP1234.P$1, U1000.A10, U1000.A11, U1000.A12, U1000.B10, U1000.B11, U1000.B12, U1000.C10, U1000.C11, U1000.C12, U1000.D10, U1000.D11, U1000.D12
- net GND: now also C1.2, C1001.-, C1003.2, C1004.2, C1008.-, C1043.2, C1044.2, C1045.2, C1046.2, J2.B-@1, J2.B-@2, R1069.1, U1000.A4, U1000.A5, U1000.A6, U1000.A7, U1000.A8, U1000.A9, U1000.B4, U1000.B5, U1000.B6, U1000.B7, U1000.B8, U1000.B9, U1000.C4, U1000.C5, U1000.C6, U1000.C7, U1000.C8, U1000.C9, U1000.D4, U1000.D5, U1000.D6, U1000.D7, U1000.D8, U1000.D9, U1000.E1, U1000.E10, U1000.E11, U1000.E12, U1000.E2, U1000.E3, U1000.E4, U1000.E5, U1000.E6, U1000.E7, U1000.E8, U1000.E9, U1000.F1, U1000.F10, U1000.F11, U1000.F12, U1000.F2, U1000.F3, U1000.F4, U1000.F5, U1000.F7, U1000.F8, U1000.F9, U1000.G1, U1000.G10, U1000.G11, U1000.G12, U1000.G2, U1000.G3, U1000.G4, U1000.G5, U1000.G6, U1000.G7, U1000.G8, U1000.G9, U1000.H1, U1000.H11, U1000.H12, U1000.H2, U1000.H4, U1000.H9; no longer J1.B-@1, J1.B-@2, U$2.A4, U$2.A5, U$2.A6, U$2.A7, U$2.A8, U$2.A9, U$2.B4, U$2.B5, U$2.B6, U$2.B7, U$2.B8, U$2.B9, U$2.C4, U$2.C5, U$2.C6, U$2.C7, U$2.C8, U$2.C9, U$2.D4, U$2.D5, U$2.D6, U$2.D7, U$2.D8, U$2.D9, U$2.E1, U$2.E10, U$2.E11, U$2.E12, U$2.E2, U$2.E3, U$2.E4, U$2.E5, U$2.E6, U$2.E7, U$2.E8, U$2.E9, U$2.F1, U$2.F10, U$2.F11, U$2.F12, U$2.F2, U$2.F3, U$2.F4, U$2.F5, U$2.F7, U$2.F8, U$2.F9, U$2.G1, U$2.G10, U$2.G11, U$2.G12, U$2.G2, U$2.G3, U$2.G4, U$2.G5, U$2.G6, U$2.G7, U$2.G8, U$2.G9, U$2.H1, U$2.H11, U$2.H12, U$2.H2, U$2.H4, U$2.H6, U$2.H7, U$2.H9, U$2.J6, U$2.J7
Other:
- board text added: "- Board fits UNDER RP rev 2"
- board text added: "- Remove P1 header and move to BOTTOM of RP."
- board text added: "- Remove P4 (Ethernet jack)."
- board text added: "- Remove RCA, audio, USB as necessary."
- board text added: "- Remove RG2 (NCP1117-3v3)"
- board text removed: "Ethernet here"

Commit message: Added scan of RP bottom side at 2400 dpi (sorry, it's 50 MB!). Used that to verify P5 and P4 placement. Updated EAGLE library schematic and footprint to be better.
Parts:
- removed U$1: RASPBERRY-PI_REV2, RaspberryPi:RASPBERRY-PI_REV2
- added J1: RP-REV2-MOAR, RaspberryPi:RP_REV2_MOAR
- moved LED3 103.0 mm to (91.4, 49.4), turned to 270 degrees
- moved R3 98.0 mm to (91.0, 53.7), turned to 0 degrees
- moved R4 90.6 mm to (88.3, 49.8)
- moved TP1000 89.4 mm to (60.9, 54.8), turned to 180 degrees
- moved TP1001 87.6 mm to (58.8, 54.8), turned to 180 degrees
- moved TP1002 85.8 mm to (56.7, 54.8), turned to 180 degrees
- moved R5 85.0 mm to (90.3, 43.6)
- moved R1069 85.0 mm to (60.4, 51.2), turned to 180 degrees
- moved TP1003 84.2 mm to (54.6, 54.8), turned to 180 degrees
- moved TP1 83.6 mm to (97.3, 33.0), turned to 270 degrees
- moved TP1004 82.6 mm to (52.5, 54.8), turned to 180 degrees
- moved TP1005 81.1 mm to (50.4, 54.8), turned to 180 degrees
- moved C1003 80.1 mm to (54.8, 51.2), turned to 180 degrees
- moved C1009 79.8 mm to (60.4, 46.3), turned to 180 degrees
- moved TP1007 79.6 mm to (48.3, 54.8), turned to 180 degrees
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Connections:
- new net 3V3: J1.P5_2
- net +3V3: now also J1.P1_1, J1.P1_17, J1.P5_1; no longer U$1.P1_1, U$1.P1_17, U$1.P5_2
- net +5V: now also J1.P1_2, J1.P1_4; no longer U$1.P1_2, U$1.P1_4, U$1.P5_1
- net GND: now also J1.P1_14, J1.P1_20, J1.P1_25, J1.P1_6, J1.P1_9, J1.P5_7, J1.P5_8; no longer U$1.P1_14, U$1.P1_20, U$1.P1_25, U$1.P1_6, U$1.P1_9, U$1.P5_7, U$1.P5_8
- net N$11: now also J1.P4_1
- net N$12: now also J1.P4_2
- net N$13: now also J1.P4_4
- net N$14: now also J1.P4_5
- net N$24: now also J1.P4_3
Other:
- board text removed: "ARM HEATSINK?!"

Commit message: More on the RP carrier: added the ethernet connector wiring, and LED randomly, and first pass of the power switchers using TI's simple switchers because we're lazy and they're relatively cheap for a one off.
Parts:
- removed C1000, C1007: 22p, rcl_custom:0603-B-NOSILK
- removed C1002, C1009: 200p, rcl_custom:0603-B-NOSILK
- removed LAN: RJLBC-060TC1, OLIMEX_CONNECTORS:RJLBC-060TC1
- removed R1000: 11.5k, rcl_custom:0603-B-NOSILK
- removed R1001: 19.1k, rcl_custom:0603-B-NOSILK
- removed R1069: 0, rcl_custom:0603-B-NOSILK
- removed TP1000, TP1001, TP1002, TP1003, TP1004, TP1005, TP1007, TP1009, TP1010, TP1011: TEST, tqm:TEST
- removed U1000: LT4619, LT4619:LT4619
- added C2, C3, C4, C5: TBD, rcl_custom:0603-B-NOSILK
- added R10, R11, R6, R7, R8, R9: 11.5k, rcl_custom:0603-B-NOSILK
- added TP5, TP6: TEST, tqm:TEST
- added U1, U2: LMZ14203, SparkFun-PowerIC:TO-PMOD-7
- moved TP1234 33.6 mm to (41.5, 21.2)
- moved C1043 33.4 mm to (45.8, 17.9), turned to 270 degrees
- moved C1045 29.2 mm to (47.4, 18.1), turned to 270 degrees
- moved C1003 29.1 mm to (59.3, 22.4), turned to 270 degrees
- moved C1 23.0 mm to (78.3, 36.2)
- moved R2 14.9 mm to (79.2, 33.1), turned to 270 degrees
- moved C1004 14.5 mm to (60.2, 41.8), turned to 270 degrees
- moved R1 11.4 mm to (77.6, 33.1), turned to 270 degrees
- moved C1008 10.6 mm to (38.9, 39.9), turned to 90 degrees
- moved C1044 9.86 mm to (43.0, 42.7), turned to 270 degrees
- moved TP1235 9.28 mm to (39.0, 45.6)
- moved L2 8.41 mm to (84.4, 30.5), turned to 180 degrees
- moved C1001 8.21 mm to (41.4, 15.2), turned to 90 degrees
- moved T2 7.99 mm to (79.5, 29.5), turned to 0 degrees
- moved L1 6.08 mm to (84.4, 25.4), turned to 180 degrees
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Connections:
- removed net 3V3: J1.P5_2
- removed net AGND: C1002.2, C1009.2, R1000.1, R1001.1, R1069.2, U1000.H6, U1000.H7, U1000.J6, U1000.J7
- removed net COMP1: TP1003.P$1, U1000.L7
- removed net COMP2: TP1005.P$1, U1000.L6
- removed net EXTVCC: TP1001.P$1, U1000.J4
- removed net FREQ: TP1000.P$1, U1000.J8
- removed net INTVCC1: TP1002.P$1, U1000.F6
- removed net PGOOD: TP1009.P$1, U1000.H5
- removed net RUN1: TP1004.P$1, U1000.J9
- removed net RUN2: TP1007.P$1, U1000.J5
- removed net SPS-500KHZ: U1000.H8
- removed net SW1: TP1011.P$1, U1000.H10
- removed net SW2: TP1010.P$1, U1000.H3
- removed net TK-SS1: C1002.1, U1000.K8
- removed net TK-SS2: C1009.1, U1000.K5
- removed net VFB1: C1000.1, R1000.2, U1000.K7
- removed net VFB2: C1007.2, R1001.2, U1000.K6
- new net N$1: J1.P4_2, T1.6
- new net N$16: J1.P4_5, T2.6
- new net N$17: C3.1, U2.5
- new net N$18: C2.1, U1.5
- new net N$31: R7.2, U2.2
- new net N$32: TP6.P$1, U1.3
- new net N$33: TP5.P$1, U2.3
- new net N$34: C4.2, R8.2, R9.1, U2.6
- new net N$35: C5.2, R10.2, R11.1, U1.6
- net +3V3: now also C4.1, R8.1, U2.7; no longer C1007.1, U1000.A1, U1000.A2, U1000.A3, U1000.B1, U1000.B2, U1000.B3, U1000.C1, U1000.C2, U1000.C3, U1000.D1, U1000.D2, U1000.D3
- net +5V: now also C5.1, J1.P5_2, R10.1, U1.7; no longer C1000.2, U1000.A10, U1000.A11, U1000.A12, U1000.B10, U1000.B11, U1000.B12, U1000.C10, U1000.C11, U1000.C12, U1000.D10, U1000.D11, U1000.D12
- net GND: now also C2.2, C3.2, R11.2, R9.2, U1.4, U2.4; no longer R1069.1, U1000.A4, U1000.A5, U1000.A6, U1000.A7, U1000.A8, U1000.A9, U1000.B4, U1000.B5, U1000.B6, U1000.B7, U1000.B8, U1000.B9, U1000.C4, U1000.C5, U1000.C6, U1000.C7, U1000.C8, U1000.C9, U1000.D4, U1000.D5, U1000.D6, U1000.D7, U1000.D8, U1000.D9, U1000.E1, U1000.E10, U1000.E11, U1000.E12, U1000.E2, U1000.E3, U1000.E4, U1000.E5, U1000.E6, U1000.E7, U1000.E8, U1000.E9, U1000.F1, U1000.F10, U1000.F11, U1000.F12, U1000.F2, U1000.F3, U1000.F4, U1000.F5, U1000.F7, U1000.F8, U1000.F9, U1000.G1, U1000.G10, U1000.G11, U1000.G12, U1000.G2, U1000.G3, U1000.G4, U1000.G5, U1000.G6, U1000.G7, U1000.G8, U1000.G9, U1000.H1, U1000.H11, U1000.H12, U1000.H2, U1000.H4, U1000.H9
- net N$11: no longer LAN.1
- net N$12: now also J1.P4_3; no longer J1.P4_2, LAN.2
- net N$13: no longer LAN.7
- net N$14: now also J1.P4_6; no longer J1.P4_5, LAN.8
- net N$15: now also J1.P5_6
- net N$2: now also J1.P5_4
- net N$24: now also R6.2, U1.2; no longer J1.P4_3, LAN.3, T1.6, T2.6
- net N$4: now also J1.P5_5
- net TRIPLE_UP_ARROW: now also R6.1, R7.1, U1.1, U2.1; no longer U1000.J1, U1000.J10, U1000.J11, U1000.J12, U1000.J2, U1000.J3, U1000.K1, U1000.K10, U1000.K11, U1000.K12, U1000.K2, U1000.K3, U1000.K4, U1000.K9, U1000.L1, U1000.L10, U1000.L11, U1000.L12, U1000.L2, U1000.L3, U1000.L4, U1000.L5, U1000.L8, U1000.L9, U1000.M1, U1000.M10, U1000.M11, U1000.M12, U1000.M2, U1000.M3, U1000.M4, U1000.M5, U1000.M6, U1000.M7, U1000.M8, U1000.M9
Routing:
- net TRIPLE_UP_ARROW: track 0.00 -> 36.5 mm
- net +3V3: track 0.00 -> 35.8 mm, vias 0 -> 3
- net N$2: track 0.00 -> 32.7 mm
- net N$15: track 0.00 -> 30.8 mm
- net N$1: track 0.00 -> 30.5 mm
- net N$4: track 0.00 -> 29.7 mm
- net N$16: track 0.00 -> 26.1 mm
- net N$13: track 0.00 -> 23.8 mm
- net N$14: track 0.00 -> 23.6 mm
- net N$11: track 0.00 -> 20.9 mm
- net N$12: track 0.00 -> 20.6 mm
- net N$27: track 0.00 -> 7.16 mm
- net N$9: track 0.00 -> 4.98 mm
- net N$19: track 0.00 -> 4.92 mm
- net N$8: track 0.00 -> 4.92 mm
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- added copper zone on layer 1, net GND
- added copper zone on layer 16, net GND

Commit message: Added FTDI breakout, cleaned up schematic a bit, design review with Paul.
Parts:
- added JP1: (no value), pinhead:1X06/90
- U1, U2: value LMZ14203 -> LMZ12001
Connections:
- new net N$36: J1.P1_10, JP1.4
- new net N$37: J1.P1_8, JP1.5
- net GND: now also JP1.1
Changed lines of the file:
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@@
 <layer number="14" name="Route14" color="1" fill="6" visible="no" active="no"/>
 <layer number="15" name="Route15" color="4" fill="6" visible="no" active="no"/>
-<layer number="16" name="Bottom" color="1" fill="1" visible="yes" active="yes"/>
+<layer number="16" name="Bottom" color="1" fill="1" visible="no" active="yes"/>
 <layer number="17" name="Pads" color="2" fill="1" visible="yes" active="yes"/>
 <layer number="18" name="Vias" color="2" fill="1" visible="yes" active="yes"/>
@@
 <layer number="20" name="Dimension" color="15" fill="1" visible="yes" active="yes"/>
 <layer number="21" name="tPlace" color="7" fill="1" visible="yes" active="yes"/>
-<layer number="22" name="bPlace" color="7" fill="1" visible="yes" active="yes"/>
+<layer number="22" name="bPlace" color="7" fill="1" visible="no" active="yes"/>
 <layer number="23" name="tOrigins" color="15" fill="1" visible="yes" active="yes"/>
-<layer number="24" name="bOrigins" color="15" fill="1" visible="yes" active="yes"/>
+<layer number="24" name="bOrigins" color="15" fill="1" visible="no" active="yes"/>
 <layer number="25" name="tNames" color="7" fill="1" visible="no" active="yes"/>
 <layer number="26" name="bNames" color="7" fill="1" visible="no" active="yes"/>
@@
 <layer number="50" name="dxf" color="7" fill="1" visible="no" active="no"/>
 <layer number="51" name="tDocu" color="7" fill="1" visible="yes" active="yes"/>
-<layer number="52" name="bDocu" color="7" fill="1" visible="yes" active="yes"/>
+<layer number="52" name="bDocu" color="7" fill="1" visible="no" active="yes"/>
 <layer number="53" name="tGND_GNDA" color="7" fill="9" visible="no" active="no"/>
 <layer number="54" name="bGND_GNDA" color="1" fill="9" visible="no" active="no"/>
@@
 <layer number="97" name="Info" color="7" fill="1" visible="no" active="no"/>
 <layer number="98" name="Guide" color="6" fill="1" visible="no" active="no"/>
-<layer number="100" name="Top" color="12" fill="1" visible="no" active="yes"/>
-<layer number="101" name="Bottom" color="1" fill="1" visible="no" active="yes"/>
-<layer number="102" name="Vscore" color="7" fill="1" visible="no" active="yes"/>
-<layer number="103" name="tMap" color="7" fill="1" visible="no" active="yes"/>
-<layer number="104" name="Name" color="16" fill="1" visible="no" active="yes"/>
-<layer number="105" name="tPlate" color="7" fill="1" visible="no" active="yes"/>
-<layer number="106" name="bPlate" color="7" fill="1" visible="no" active="yes"/>
-<layer number="107" name="Crop" color="7" fill="1" visible="no" active="yes"/>
-<layer number="108" name="tplace-old" color="10" fill="1" visible="no" active="yes"/>
-<layer number="109" name="ref-old" color="11" fill="1" visible="no" active="yes"/>
-<layer number="116" name="Patch_BOT" color="9" fill="4" visible="no" active="yes"/>
-<layer number="121" name="_tsilk" color="7" fill="1" visible="no" active="yes"/>
-<layer number="122" name="_bsilk" color="7" fill="1" visible="no" active="yes"/>
-<layer number="125" name="_tNames" color="7" fill="1" visible="no" active="yes"/>
-<layer number="144" name="Drill_legend" color="7" fill="1" visible="no" active="yes"/>
-<layer number="151" name="HeatSink" color="7" fill="1" visible="no" active="yes"/>
-<layer number="199" name="Contour" color="7" fill="1" visible="no" active="yes"/>
-<layer number="200" name="200bmp" color="1" fill="10" visible="no" active="yes"/>
-<layer number="201" name="201bmp" color="2" fill="10" visible="no" active="yes"/>
-<layer number="202" name="202bmp" color="3" fill="10" visible="no" active="yes"/>
-<layer number="203" name="203bmp" color="4" fill="10" visible="no" active="yes"/>
-<layer number="204" name="204bmp" color="5" fill="10" visible="no" active="yes"/>
-<layer number="205" name="205bmp" color="6" fill="10" visible="no" active="yes"/>
-<layer number="206" name="206bmp" color="7" fill="10" visible="no" active="yes"/>
-<layer number="207" name="207bmp" color="8" fill="10" visible="no" active="yes"/>
-<layer number="208" name="208bmp" color="9" fill="10" visible="no" active="yes"/>
-<layer number="209" name="209bmp" color="7" fill="1" visible="no" active="yes"/>
-<layer number="210" name="210bmp" color="7" fill="1" visible="no" active="yes"/>
-<layer number="211" name="211bmp" color="7" fill="1" visible="no" active="yes"/>
-<layer number="212" name="212bmp" color="7" fill="1" visible="no" active="yes"/>
-<layer number="213" name="213bmp" color="7" fill="1" visible="no" active="yes"/>
-<layer number="214" name="214bmp" color="7" fill="1" visible="no" active="yes"/>
-<layer number="215" name="215bmp" color="7" fill="1" visible="no" active="yes"/>
-<layer number="216" name="216bmp" color="7" fill="1" visible="no" active="yes"/>
 <layer number="217" name="217bmp" color="18" fill="1" visible="no" active="no"/>
 <layer number="218" name="218bmp" color="19" fill="1" visible="no" active="no"/>
@@
 <layer number="250" name="Descript" color="3" fill="1" visible="no" active="no"/>
 <layer number="251" name="SMDround" color="12" fill="11" visible="no" active="no"/>
-<layer number="254" name="cooling" color="7" fill="1" visible="no" active="yes"/>
 </layers>
 <board>
@@
 <element name="TP1235" library="tqm" package="TEST" value="TEST" x="39" y="45.6" rot="R180"/>
 <element name="J1" library="RaspberryPi" package="RP_REV2_MOAR" value="RP-REV2-MOAR" x="0" y="0"/>
-<element name="U1" library="SparkFun-PowerIC" package="TO-PMOD-7" value="LMZ14203" x="53.1" y="10.8" rot="R180"/>
-<element name="U2" library="SparkFun-PowerIC" package="TO-PMOD-7" value="LMZ14203" x="53.3" y="34.4" rot="R180"/>
+<element name="U1" library="SparkFun-PowerIC" package="TO-PMOD-7" value="LMZ12001" x="53.1" y="10.8" rot="R180"/>
+<element name="U2" library="SparkFun-PowerIC" package="TO-PMOD-7" value="LMZ12001" x="53.3" y="34.4" rot="R180"/>
 <element name="C2" library="rcl_custom" package="0603-B-NOSILK" value="TBD" x="52.7" y="20.9"/>
 <element name="R6" library="rcl_custom" package="0603-B-NOSILK" value="11.5k" x="55.8" y="22" rot="R270"/>
@@
 <element name="C4" library="rcl_custom" package="0603-B-NOSILK" value="TBD" x="49.9" y="46.7"/>
 <element name="C5" library="rcl_custom" package="0603-B-NOSILK" value="TBD" x="49.8" y="21.4"/>
+<element name="JP1" library="pinhead" package="1X06/90" value="" x="31" y="4.9" rot="R180"/>
 </elements>
 <signals>
@@
 <contactref element="R9" pad="2"/>
 <contactref element="R11" pad="2"/>
+<contactref element="JP1" pad="1"/>
+<via x="1.7" y="1.6" extent="1-16" drill="0.3302"/>
+<via x="91.8" y="3.1" extent="1-16" drill="0.3302"/>
+<via x="92.8" y="54.8" extent="1-16" drill="0.3302"/>
+<via x="50.1" y="54.9" extent="1-16" drill="0.3302"/>
+<via x="1" y="26.8" extent="1-16" drill="0.3302"/>
+<via x="1.2" y="39.2" extent="1-16" drill="0.3302"/>
+<via x="1.2" y="14.4" extent="1-16" drill="0.3302"/>
 </signal>
 <signal name="+5V">
@@
 <wire x1="50.53" y1="18.43" x2="50.6" y2="21.4" width="0" layer="19" extent="1-1"/>
 </signal>
+<signal name="N$36">
+<contactref element="JP1" pad="4"/>
+<contactref element="J1" pad="P1_10"/>
+<wire x1="29.73" y1="8.71" x2="12.56" y2="53.265" width="0" layer="19" extent="1-1"/>
+</signal>
+<signal name="N$37">
+<contactref element="J1" pad="P1_8"/>
+<contactref element="JP1" pad="5"/>
+<wire x1="27.19" y1="8.71" x2="10.02" y2="53.265" width="0" layer="19" extent="1-1"/>
+</signal>
 </signals>

Commit message: Draft 1 of RNC to RasPi daughterboard layout
Parts:
- removed JP1: (no value), pinhead:1X06/90
- moved R7 15.2 mm to (59.5, 40.0), turned to 180 degrees
- moved C1 8.61 mm to (73.0, 29.5), turned to 0 degrees
- moved R2 7.97 mm to (73.0, 28.0), turned to 0 degrees
- moved R6 6.63 mm to (59.5, 16.5), turned to 180 degrees
- moved R3 5.78 mm to (86.5, 50.5)
- moved R1 5.01 mm to (73.0, 31.0), turned to 0 degrees
- moved C1046 4.95 mm to (44.0, 38.1)
- moved C1043 4.78 mm to (42.0, 15.0)
- moved C1044 4.73 mm to (41.9, 38.1)
- moved C1045 4.60 mm to (44.0, 15.0)
- moved C1003 4.48 mm to (61.5, 18.5), turned to 0 degrees
- moved R11 3.89 mm to (49.5, 24.0), turned to 180 degrees
- moved R9 3.61 mm to (49.5, 47.5), turned to 180 degrees
- moved TP1234 3.36 mm to (38.1, 21.4)
- moved C1001 3.27 mm to (38.1, 15.0)
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Connections:
- removed net N$36: J1.P1_10, JP1.4
- removed net N$37: J1.P1_8, JP1.5
- net GND: no longer JP1.1
Routing:
- net +5V: track 0.00 -> 89.0 mm
- net +3V3: track 35.8 -> 112.2 mm, vias 3 -> 2
- net N$2: track 32.7 -> 97.4 mm
- net N$15: track 30.8 -> 92.9 mm
- net N$4: track 29.7 -> 85.8 mm
- net TRIPLE_UP_ARROW: track 36.5 -> 64.4 mm, vias 0 -> 2
- net N$28: track 2.44 -> 9.82 mm, vias 0 -> 2
- net N$14: track 23.6 -> 30.2 mm, vias 0 -> 2
- net N$35: track 0.00 -> 5.42 mm
- net N$34: track 0.00 -> 5.42 mm
- net N$24: track 0.00 -> 5.05 mm
- net N$31: track 0.00 -> 5.02 mm
- net N$1: track 30.5 -> 34.9 mm
- net N$11: track 20.9 -> 25.2 mm
- net N$13: track 23.8 -> 27.7 mm, vias 0 -> 2
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
Commit message: Completed RPi daughterboard layout.
Parts:
- removed TP1234, TP1235: TEST, tqm:TEST
- added JP1: (no value), pinhead:1X06
- added JP2: (no value), pinhead:1X02
- added Q1: NTR4101P, Tova:SOT23
- added R12: 50, rcl_custom:0603-B-NOSILK
- added TP7, TP8: TEST-POINT, apdm:2MM-TEST-POINT
- TP5, TP6: value TEST -> TEST-POINT; device tqm:TEST -> apdm:2MM-TEST-POINT
- moved TP6 24.0 mm to (54.3, 46.0), flipped to the bottom, turned to 0 degrees
- moved TP5 23.5 mm to (54.3, 22.0), turned to 0 degrees
- moved C1008 3.85 mm to (41.5, 39.9)
- moved C1001 3.74 mm to (41.7, 16.0)
- moved C1044 3.33 mm to (44.7, 39.9)
- moved C1046 3.16 mm to (46.5, 39.9)
- moved C1043 3.07 mm to (44.9, 16.0)
- moved C1045 3.07 mm to (46.9, 16.0)
- moved C1003 3.01 mm to (58.7, 19.6), turned to 90 degrees
- moved C1004 2.88 mm to (58.8, 43.0), turned to 90 degrees
- moved R11 1.61 mm to (51.1, 24.2), turned to 0 degrees
- moved R9 1.60 mm to (51.1, 47.6), turned to 0 degrees
- moved R7 1.50 mm to (58.0, 40.0)
- moved C3 0.73 mm to (51.8, 45.3)
Connections:
- new net N$36: J1.P1_10, JP1.4
- new net N$37: J1.P1_8, JP1.5
- new net N$38: J1.P1_26, Q1.1
- new net N$39: JP2.1, Q1.3
- new net N$40: Q1.2, R12.1
- net +3V3: now also TP8.1; no longer TP1235.P$1
- net +5V: now also R12.2, TP7.1; no longer TP1234.P$1
- net GND: now also JP1.1, JP2.2, U1.EP, U2.EP
- net N$32: now also TP5.1; no longer TP6.P$1
- net N$33: now also TP6.1; no longer TP5.P$1
Routing:
- net N$36: track 0.00 -> 134.9 mm, vias 0 -> 2
- net N$37: track 0.00 -> 134.0 mm, vias 0 -> 2
- net N$38: track 0.00 -> 64.4 mm, vias 0 -> 1
- net +5V: track 89.0 -> 121.6 mm
- net +3V3: track 112.2 -> 103.1 mm, vias 2 -> 5
- net TRIPLE_UP_ARROW: track 64.4 -> 71.7 mm, vias 2 -> 6
- net N$2: track 97.4 -> 100.3 mm
- net N$40: track 0.00 -> 2.46 mm
- net N$39: track 0.00 -> 2.45 mm
- net N$31: track 5.02 -> 3.52 mm
- net N$17: track 3.18 -> 2.40 mm
- added copper zone on layer 1, net +3V3
- added copper zone on layer 1, net +5V

Commit message: Fixed gearcam transistor (no 5V to the RP!!11!), made power wires bigger, fixed tname.
Parts:
- Q1: value NTR4101P -> PMV45EN
- R12: value 50 -> 10k
- moved R2 5.53 mm to (74.2, 33.4)
- moved C1 3.64 mm to (71.1, 32.6), turned to 180 degrees
- moved Q1 2.19 mm to (86.5, 42.6), turned to 0 degrees
- moved R1 1.44 mm to (74.2, 31.8)
- moved R12 0.82 mm to (84.7, 39.8), turned to 0 degrees
- moved C2 0.36 mm to (51.7, 21.8)
- moved C5 0.10 mm to (49.4, 21.0)
- moved R10 0.10 mm to (49.4, 22.5)
- moved R11 0.10 mm to (51.0, 24.2)
- moved C1046 0.05 mm to (46.6, 39.9)
Connections:
- removed net N$39: JP2.1, Q1.3
- net +5V: now also JP2.1; no longer R12.2
- net GND: now also Q1.2, R12.1; no longer JP2.2
- net N$38: now also R12.2
- net N$40: now also JP2.2, Q1.3; no longer Q1.2, R12.1
Routing:
- net +5V: track 121.6 -> 129.8 mm
- net N$27: track 3.57 -> 9.62 mm
- net N$38: track 64.4 -> 67.2 mm
- net N$40: track 2.46 -> 5.01 mm
- net N$39: track 2.45 -> 0.00 mm
- net N$14: track 30.2 -> 28.5 mm, vias 2 -> 0
- net N$26: track 3.28 -> 1.75 mm
- net TRIPLE_UP_ARROW: track 71.7 -> 70.8 mm
- net N$13: vias 2 -> 0
- net N$37: vias 2 -> 1
- net N$36: vias 2 -> 1
Other:
- board text added: "PSAS RASPI to RNC Adapter v1"
- board text removed: "PSAS RNC to RASPI Adapter v1"
