File: av4/raspi-camera/eagle/raspi-rnc.brd (EAGLE design)
At the start: 45 parts, among them J1 RP-REV2-MOAR, J2 ROCKETNET-CONNECTOR-16M, Q1 PMV45EN, T1 ALT4532, T2 ALT4532, U1 LMZ12001, U2 LMZ12001

Commit message: Set values on RP carriers, also BOM.
Parts:
- C1: value 100nF -> 1n 2kv
- C1003, C1004: value 10u -> 10u 40V
- C2, C3, C4, C5: value TBD -> 22n
- R1, R2: value 50 -> 75
- R10: value 11.5k -> 5.62k
- R11, R9: value 11.5k -> 1.07k
- R8: value 11.5k -> 3.32k
Changed lines of the file:
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@@
 <attribute name="NAME" x="84.72" y="29.38" size="0.762" layer="25" font="vector" ratio="20" rot="R180"/>
 </element>
-<element name="C1" library="rcl_custom" package="0603-B-NOSILK" value="100nF" x="71.1" y="32.6" smashed="yes" rot="R180">
+<element name="C1" library="rcl_custom" package="0603-B-NOSILK" value="1n 2kv" x="71.1" y="32.6" smashed="yes" rot="R180">
 <attribute name="NAME" x="71.8" y="31.7" size="0.762" layer="25" font="vector" ratio="20" rot="R180"/>
 <attribute name="VALUE" x="71.9" y="34.65" size="1" layer="27" ratio="10" rot="R180"/>
 </element>
-<element name="R1" library="rcl_custom" package="0603-B-NOSILK" value="50" x="74.2" y="31.8" smashed="yes">
+<element name="R1" library="rcl_custom" package="0603-B-NOSILK" value="75" x="74.2" y="31.8" smashed="yes">
 <attribute name="NAME" x="73.6" y="30.2" size="0.762" layer="25" font="vector" ratio="20"/>
 <attribute name="VALUE" x="73.4" y="29.75" size="1" layer="27" ratio="10"/>
 </element>
-<element name="R2" library="rcl_custom" package="0603-B-NOSILK" value="50" x="74.2" y="33.4" smashed="yes">
+<element name="R2" library="rcl_custom" package="0603-B-NOSILK" value="75" x="74.2" y="33.4" smashed="yes">
 <attribute name="NAME" x="73.4" y="34.4" size="0.762" layer="25" font="vector" ratio="20"/>
 <attribute name="VALUE" x="73.4" y="31.35" size="1" layer="27" ratio="10"/>
@@
 <attribute name="VALUE" x="85.7" y="46.95" size="1" layer="27" ratio="10"/>
 </element>
-<element name="C1003" library="rcl_custom" package="0805-B-NOSILK" value="10u" x="58.7" y="19.6" smashed="yes" rot="R90">
+<element name="C1003" library="rcl_custom" package="0805-B-NOSILK" value="10u 40V" x="58.7" y="19.6" smashed="yes" rot="R90">
 <attribute name="NAME" x="56.9" y="22.4" size="0.762" layer="25" font="vector" ratio="20"/>
 <attribute name="VALUE" x="60.7" y="18.8" size="1" layer="27" ratio="10" rot="R90"/>
 </element>
-<element name="C3" library="rcl_custom" package="0603-B-NOSILK" value="TBD" x="51.8" y="45.3" smashed="yes" rot="R90">
+<element name="C3" library="rcl_custom" package="0603-B-NOSILK" value="22n" x="51.8" y="45.3" smashed="yes" rot="R90">
 <attribute name="NAME" x="53.4" y="45.8" size="0.762" layer="25" font="vector" ratio="20" rot="R90"/>
 <attribute name="VALUE" x="53.85" y="44.5" size="1" layer="27" ratio="10" rot="R90"/>
 </element>
-<element name="C1004" library="rcl_custom" package="0805-B-NOSILK" value="10u" x="58.8" y="43" smashed="yes" rot="R90">
+<element name="C1004" library="rcl_custom" package="0805-B-NOSILK" value="10u 40V" x="58.8" y="43" smashed="yes" rot="R90">
 <attribute name="NAME" x="60.7" y="43.2" size="0.762" layer="25" font="vector" ratio="20" rot="R90"/>
 <attribute name="VALUE" x="60.8" y="42.2" size="1" layer="27" ratio="10" rot="R90"/>
@@
 <attribute name="NAME" x="58.5" y="29.4" size="0.762" layer="25" font="vector" ratio="20"/>
 </element>
-<element name="C2" library="rcl_custom" package="0603-B-NOSILK" value="TBD" x="51.7" y="21.8" smashed="yes" rot="R90">
+<element name="C2" library="rcl_custom" package="0603-B-NOSILK" value="22n" x="51.7" y="21.8" smashed="yes" rot="R90">
 <attribute name="NAME" x="52.5" y="22.5" size="0.762" layer="25" font="vector" ratio="20"/>
 <attribute name="VALUE" x="53.75" y="21" size="1" layer="27" ratio="10" rot="R90"/>
@@
 <attribute name="VALUE" x="58.8" y="42.05" size="1" layer="27" ratio="10" rot="R180"/>
 </element>
-<element name="R8" library="rcl_custom" package="0603-B-NOSILK" value="11.5k" x="49.5" y="44.5" smashed="yes">
+<element name="R8" library="rcl_custom" package="0603-B-NOSILK" value="3.32k" x="49.5" y="44.5" smashed="yes">
 <attribute name="NAME" x="46.8" y="44.2" size="0.762" layer="25" font="vector" ratio="20"/>
 <attribute name="VALUE" x="48.7" y="42.45" size="1" layer="27" ratio="10"/>
 </element>
-<element name="R9" library="rcl_custom" package="0603-B-NOSILK" value="11.5k" x="51.1" y="47.6" smashed="yes">
+<element name="R9" library="rcl_custom" package="0603-B-NOSILK" value="1.07k" x="51.1" y="47.6" smashed="yes">
 <attribute name="NAME" x="50.7" y="48.3" size="0.762" layer="25" font="vector" ratio="20"/>
 <attribute name="VALUE" x="50.3" y="45.55" size="1" layer="27" ratio="10"/>
 </element>
-<element name="R10" library="rcl_custom" package="0603-B-NOSILK" value="11.5k" x="49.4" y="22.5" smashed="yes">
+<element name="R10" library="rcl_custom" package="0603-B-NOSILK" value="5.62k" x="49.4" y="22.5" smashed="yes">
 <attribute name="NAME" x="46.9" y="23.3" size="0.762" layer="25" font="vector" ratio="20"/>
 <attribute name="VALUE" x="48.6" y="20.45" size="1" layer="27" ratio="10"/>
 </element>
-<element name="R11" library="rcl_custom" package="0603-B-NOSILK" value="11.5k" x="51" y="24.2" smashed="yes">
+<element name="R11" library="rcl_custom" package="0603-B-NOSILK" value="1.07k" x="51" y="24.2" smashed="yes">
 <attribute name="NAME" x="50.2" y="25.2" size="0.762" layer="25" font="vector" ratio="20"/>
 <attribute name="VALUE" x="50.2" y="22.15" size="1" layer="27" ratio="10"/>
 </element>
-<element name="C4" library="rcl_custom" package="0603-B-NOSILK" value="TBD" x="49.5" y="46" smashed="yes">
+<element name="C4" library="rcl_custom" package="0603-B-NOSILK" value="22n" x="49.5" y="46" smashed="yes">
 <attribute name="NAME" x="46.8" y="45.7" size="0.762" layer="25" font="vector" ratio="20"/>
 <attribute name="VALUE" x="48.7" y="43.95" size="1" layer="27" ratio="10"/>
 </element>
-<element name="C5" library="rcl_custom" package="0603-B-NOSILK" value="TBD" x="49.4" y="21" smashed="yes">
+<element name="C5" library="rcl_custom" package="0603-B-NOSILK" value="22n" x="49.4" y="21" smashed="yes">
 <attribute name="NAME" x="46.9" y="19.5" size="0.762" layer="25" font="vector" ratio="20"/>
 <attribute name="VALUE" x="48.6" y="18.95" size="1" layer="27" ratio="10"/>
