File: av4/raspi-camera/eagle/raspi-rnc.brd (EAGLE design)
At the start: 45 parts, among them J1 RP-REV2-MOAR, J2 ROCKETNET-CONNECTOR-16M, Q1 PMV45EN, T1 ALT4532, T2 ALT4532, U1 LMZ12001, U2 LMZ12001

Commit message: Updated RasPi 0.1" header position and hole placement, as well as added a new 3rd hole. Extended board to have more room for RNC, moved resistor, version is now 2!
Parts:
- removed TP1, TP2, TP3, TP4: TEST-POINT, apdm:2MM-TEST-POINT
- moved J2 10.0 mm to (98.9, 27.9)
- moved L1 10.0 mm to (93.8, 25.4)
- moved L2 10.0 mm to (93.8, 30.5)
- moved C1 9.80 mm to (80.9, 32.6)
- moved T1 9.80 mm to (88.5, 25.4)
- moved T2 9.80 mm to (88.5, 30.5)
- moved R1 9.80 mm to (84.0, 31.8)
- moved R2 9.80 mm to (84.0, 33.4)
- moved JP1 8.00 mm to (99.5, 8.50)
- moved JP2 8.00 mm to (99.5, 42.5)
- moved LED3 8.00 mm to (99.5, 50.5)
- moved Q1 8.00 mm to (94.5, 42.6)
- moved R3 8.00 mm to (94.5, 50.5)
- moved R4 8.00 mm to (94.5, 52.0)
- moved R5 8.00 mm to (94.5, 49.0)
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Connections:
- removed net N$20: J2.A4, TP4.1
- removed net N$21: J2.A3, TP3.1
- removed net N$22: J2.A2, TP2.1
- removed net N$23: J2.A1, TP1.1
Routing:
- net N$14: track 28.5 -> 38.1 mm
- net TRIPLE_UP_ARROW: track 70.8 -> 80.2 mm
- net N$13: track 27.7 -> 36.9 mm
- net N$16: track 27.8 -> 36.6 mm
- net N$12: track 23.4 -> 31.8 mm
- net N$4: track 85.8 -> 93.8 mm
- net N$2: track 100.3 -> 108.3 mm
- net N$15: track 92.9 -> 100.9 mm
- net +5V: track 129.8 -> 137.8 mm
- net +3V3: track 103.1 -> 111.1 mm
- net N$1: track 35.1 -> 42.9 mm
- net N$11: track 25.3 -> 32.4 mm
- net N$37: track 134.0 -> 140.9 mm
- net N$36: track 134.9 -> 139.8 mm
- net N$23: track 3.79 -> 0.00 mm
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Other:
- board text added: "3.3V"
- board text added: "5V"
- board text added: "PSAS RASPI to RNC Adapter v2"
- board text removed: "PSAS RASPI to RNC Adapter v1"

Commit message: Note to remove RG2 *and* F3. Fixed TP6 that was mirrored (weird) and and a tname collision. Otherwise, schematically the same as what was sent to OSHPark today.
Parts:
- flipped TP6 to the top
Other:
- board text added: "- Remove RG2 (NCP1117-3v3) and F3."
- board text removed: "- Remove RG2 (NCP1117-3v3)"
Changed lines of the file:
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@@
 <layer number="23" name="tOrigins" color="15" fill="1" visible="yes" active="yes"/>
 <layer number="24" name="bOrigins" color="15" fill="1" visible="yes" active="yes"/>
-<layer number="25" name="tNames" color="7" fill="1" visible="no" active="yes"/>
+<layer number="25" name="tNames" color="7" fill="1" visible="yes" active="yes"/>
 <layer number="26" name="bNames" color="7" fill="1" visible="no" active="yes"/>
 <layer number="27" name="tValues" color="7" fill="1" visible="no" active="yes"/>
@@
 <text x="1" y="76" size="1.778" layer="51">- Board fits UNDER RP rev 2</text>
 <text x="1" y="73" size="1.778" layer="51">- Remove P1 header and move to BOTTOM of RP.</text>
-<text x="1" y="70" size="1.778" layer="51">- Remove RG2 (NCP1117-3v3)</text>
+<text x="1" y="70" size="1.778" layer="51">- Remove RG2 (NCP1117-3v3) and F3.</text>
 <text x="1" y="67" size="1.778" layer="51">- Remove P4 (Ethernet jack).</text>
 <text x="1" y="64" size="1.778" layer="51">- Remove RCA, audio, USB as necessary.</text>
@@
 </element>
 <element name="C1008" library="rcl" package="D/7343-31R" value="100u" x="41.5" y="39.9" smashed="yes" rot="R90">
-<attribute name="NAME" x="39" y="38.45" size="0.762" layer="25" font="vector" ratio="20" rot="R90"/>
+<attribute name="NAME" x="38.8" y="36.05" size="0.762" layer="25" font="vector" ratio="20" rot="R90"/>
 <attribute name="VALUE" x="45.075" y="36.25" size="1.27" layer="27" rot="R90"/>
 </element>
@@
 <attribute name="NAME" x="52.7" y="23.5" size="0.762" layer="25" font="vector" ratio="20"/>
 </element>
-<element name="TP6" library="apdm" package="2MM-TEST-POINT" value="TEST-POINT" x="54.3" y="46" rot="MR0"/>
+<element name="TP6" library="apdm" package="2MM-TEST-POINT" value="TEST-POINT" x="54.3" y="46" smashed="yes">
+<attribute name="NAME" x="55.4" y="45.6" size="0.8" layer="25" font="vector" ratio="20"/>
+</element>
 <element name="TP7" library="apdm" package="2MM-TEST-POINT" value="TEST-POINT" x="46.1" y="21.7" smashed="yes">
 <attribute name="NAME" x="44.9" y="21" size="0.762" layer="25" font="vector" ratio="20" rot="R90"/>

Commit message: how is it that this wasn't committed a bzillion years ago? This new schematic has the mods for the optoisolator on it.
Parts:
- added JP3: (no value), pinhead:1X02
- added OK1: 4N28SM, optocoupler:DIL6-SMD
- added R13: ??k, rcl_custom:0603-B-NOSILK
Connections:
- new net N$20: J1.P5_3, R13.2
- new net N$21: OK1.1, R13.1
- new net N$23: JP3.2, OK1.5
- new net N$39: JP3.1, OK1.4
- net GND: now also OK1.2
Changed lines of the file:
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@@
 <layer number="14" name="Route14" color="1" fill="6" visible="no" active="no"/>
 <layer number="15" name="Route15" color="4" fill="6" visible="no" active="no"/>
-<layer number="16" name="Bottom" color="1" fill="1" visible="yes" active="yes"/>
+<layer number="16" name="Bottom" color="1" fill="1" visible="no" active="yes"/>
 <layer number="17" name="Pads" color="2" fill="1" visible="yes" active="yes"/>
 <layer number="18" name="Vias" color="2" fill="1" visible="yes" active="yes"/>
@@
 <layer number="20" name="Dimension" color="15" fill="1" visible="yes" active="yes"/>
 <layer number="21" name="tPlace" color="16" fill="1" visible="yes" active="yes"/>
-<layer number="22" name="bPlace" color="14" fill="1" visible="yes" active="yes"/>
+<layer number="22" name="bPlace" color="14" fill="1" visible="no" active="yes"/>
 <layer number="23" name="tOrigins" color="15" fill="1" visible="yes" active="yes"/>
-<layer number="24" name="bOrigins" color="15" fill="1" visible="yes" active="yes"/>
-<layer number="25" name="tNames" color="7" fill="1" visible="yes" active="yes"/>
+<layer number="24" name="bOrigins" color="15" fill="1" visible="no" active="yes"/>
+<layer number="25" name="tNames" color="7" fill="1" visible="no" active="yes"/>
 <layer number="26" name="bNames" color="7" fill="1" visible="no" active="yes"/>
 <layer number="27" name="tValues" color="7" fill="1" visible="no" active="yes"/>
@@
 <layer number="29" name="tStop" color="7" fill="3" visible="no" active="yes"/>
 <layer number="30" name="bStop" color="7" fill="6" visible="no" active="yes"/>
-<layer number="31" name="tCream" color="7" fill="4" visible="no" active="yes"/>
+<layer number="31" name="tCream" color="7" fill="4" visible="yes" active="yes"/>
 <layer number="32" name="bCream" color="7" fill="5" visible="no" active="yes"/>
 <layer number="33" name="tFinish" color="6" fill="3" visible="no" active="yes"/>
@@
 <layer number="47" name="Measures" color="7" fill="1" visible="no" active="yes"/>
 <layer number="48" name="Document" color="7" fill="1" visible="no" active="yes"/>
-<layer number="49" name="Reference" color="7" fill="1" visible="yes" active="yes"/>
+<layer number="49" name="Reference" color="7" fill="1" visible="no" active="yes"/>
 <layer number="50" name="dxf" color="7" fill="1" visible="no" active="no"/>
 <layer number="51" name="tDocu" color="6" fill="1" visible="yes" active="yes"/>
-<layer number="52" name="bDocu" color="7" fill="1" visible="yes" active="yes"/>
+<layer number="52" name="bDocu" color="7" fill="1" visible="no" active="yes"/>
 <layer number="53" name="tGND_GNDA" color="7" fill="9" visible="no" active="no"/>
 <layer number="54" name="bGND_GNDA" color="1" fill="9" visible="no" active="no"/>
@@
 <param name="mlMinStopFrame" value="3mil"/>
 <param name="mlMaxStopFrame" value="3mil"/>
-<param name="mlMinCreamFrame" value="0mil"/>
-<param name="mlMaxCreamFrame" value="0mil"/>
+<param name="mlMinCreamFrame" value="3mil"/>
+<param name="mlMaxCreamFrame" value="3mil"/>
 <param name="mlViaStopLimit" value="20mil"/>
 <param name="srRoundness" value="0"/>
@@
 <attribute name="VALUE" x="92.5" y="39.6" size="1" layer="27"/>
 </element>
+<element name="OK1" library="optocoupler" package="DIL6-SMD" value="4N28SM" x="-8.2" y="-6.8">
+<attribute name="OC_NEWARK" value="05C3314" x="-8.2" y="-6.8" size="1.778" layer="27" display="off"/>
+<attribute name="MPN" value="4N28S-M" x="-8.2" y="-6.8" size="1.778" layer="27" display="off"/>
+<attribute name="MF" value="FAIRCHILD SEMICONDUCTOR" x="-8.2" y="-6.8" size="1.778" layer="27" display="off"/>
+<attribute name="OC_FARNELL" value="unknown" x="-8.2" y="-6.8" size="1.778" layer="27" display="off"/>
+</element>
+<element name="R13" library="rcl_custom" package="0603-B-NOSILK" value="??k" x="-13.4" y="-14.7"/>
+<element name="JP3" library="pinhead" package="1X02" value="" x="-11.9" y="-20.8"/>
 </elements>
 <signals>
@@
 <via x="88.5" y="25.4" extent="1-16" drill="0.3302"/>
 <via x="88.5" y="30.5" extent="1-16" drill="0.3302"/>
+<contactref element="OK1" pad="2"/>
+<wire x1="1" y1="1" x2="-8.2" y2="-11.445" width="0" layer="19" extent="1-1"/>
 </signal>
 <signal name="+5V">
@@
 <wire x1="99.473" y1="43.743" x2="99.5" y2="43.77" width="0.6096" layer="1"/>
 </signal>
+<signal name="N$20">
+<contactref element="J1" pad="P5_3"/>
+<contactref element="R13" pad="2"/>
+<wire x1="-12.6" y1="-14.7" x2="10.02" y2="48.185" width="0" layer="19" extent="1-1"/>
+</signal>
+<signal name="N$21">
+<contactref element="R13" pad="1"/>
+<contactref element="OK1" pad="1"/>
+<wire x1="-10.74" y1="-11.445" x2="-14.2" y2="-14.7" width="0" layer="19" extent="1-1"/>
+</signal>
+<signal name="N$23">
+<contactref element="OK1" pad="5"/>
+<contactref element="JP3" pad="2"/>
+<wire x1="-8.2" y1="-2.155" x2="-10.63" y2="-20.8" width="0" layer="19" extent="1-1"/>
+</signal>
+<signal name="N$39">
+<contactref element="OK1" pad="4"/>
+<contactref element="JP3" pad="1"/>
+<wire x1="-5.66" y1="-2.155" x2="-13.17" y2="-20.8" width="0" layer="19" extent="1-1"/>
+</signal>
 </signals>
