File: av4/raspi-camera/eagle/raspi-rnc.sch (EAGLE design)
At the start: 1 part

Commit message: The beginnings of a Raspberry Pi to rocketnet connector adapter. Man, what a terrible board the RPI is.. no CAD, no drawings... how do people even use it?!
Parts:
- added J1: ROCKETNET-CONNECTOR-16M, rocketnet-connector:ROCKETNET-CONNECTOR-16M
- added U$2: LT4619_REDUCED, LT4619:LT4619_REDUCED
Connections:
- new net +3V3: U$1.3V3@1, U$1.3V3@17, U$1.3V3@P5_2
- new net +5V: U$1.5V@2, U$1.5V@4, U$1.5V@P5_1
- new net GND: J1.B-@1, J1.B-@2, U$1.GND@14, U$1.GND@20, U$1.GND@25, U$1.GND@6, U$1.GND@9, U$1.GND@P5_7, U$1.GND@P5_8, U$2.PGND, U$2.SGND
- new net N$1: J1.B+@1, J1.B+@2, U$2.VIN
Other:
- moved on the sheet: U$1
Changed lines of the file:
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@@
 <setting verticaltext="up"/>
 </settings>
-<grid distance="0.1" unitdist="inch" unit="inch" style="lines" multiple="1" display="no" altdistance="0.01" altunitdist="inch" altunit="inch"/>
+<grid distance="0.05" unitdist="inch" unit="inch" style="lines" multiple="2" display="yes" altdistance="0.01" altunitdist="inch" altunit="inch"/>
 <layers>
 <layer number="1" name="Top" color="4" fill="1" visible="no" active="no"/>
@@
 <parts>
 <part name="U$1" library="RaspberryPi" deviceset="RASPBERRY-PI_REV2" device=""/>
+<part name="J1" library="rocketnet-connector" deviceset="ROCKETNET-CONNECTOR-16" device="M"/>
+<part name="GND1" library="supply1" deviceset="GND" device=""/>
+<part name="GND2" library="supply1" deviceset="GND" device=""/>
+<part name="GND3" library="supply1" deviceset="GND" device=""/>
+<part name="FRAME1" library="frames" deviceset="FRAME_B_L" device=""/>
+<part name="U$2" library="LT4619" deviceset="LT4619_REDUCED" device=""/>
+<part name="GND4" library="supply1" deviceset="GND" device=""/>
+<part name="+3V1" library="supply1" deviceset="+3V3" device=""/>
+<part name="P+1" library="supply1" deviceset="+5V" device=""/>
+<part name="P+2" library="supply1" deviceset="+5V" device=""/>
+<part name="+3V2" library="supply1" deviceset="+3V3" device=""/>
 </parts>
 <sheets>
@@
 </plain>
 <instances>
-<instance part="U$1" gate="G$1" x="27.94" y="38.1"/>
+<instance part="U$1" gate="G$1" x="157.48" y="139.7"/>
+<instance part="J1" gate="G$1" x="309.88" y="132.08" rot="MR0"/>
+<instance part="GND1" gate="1" x="302.26" y="104.14"/>
+<instance part="GND2" gate="1" x="190.5" y="106.68"/>
+<instance part="GND3" gate="1" x="121.92" y="106.68"/>
+<instance part="FRAME1" gate="G$1" x="0" y="0"/>
+<instance part="FRAME1" gate="G$2" x="325.12" y="0"/>
+<instance part="U$2" gate="G$1" x="259.08" y="113.03"/>
+<instance part="GND4" gate="1" x="223.52" y="106.68"/>
+<instance part="+3V1" gate="G$1" x="200.66" y="165.1"/>
+<instance part="P+1" gate="1" x="119.38" y="162.56"/>
+<instance part="P+2" gate="1" x="193.04" y="165.1"/>
+<instance part="+3V2" gate="G$1" x="111.76" y="162.56"/>
 </instances>
 <busses>
 </busses>
 <nets>
+<net name="GND" class="0">
+<segment>
+<pinref part="GND1" gate="1" pin="GND"/>
+<pinref part="J1" gate="G$1" pin="B-@1"/>
+<wire x1="302.26" y1="106.68" x2="302.26" y2="111.76" width="0.1524" layer="91"/>
+<wire x1="302.26" y1="111.76" x2="302.26" y2="114.3" width="0.1524" layer="91"/>
+<wire x1="302.26" y1="114.3" x2="304.8" y2="114.3" width="0.1524" layer="91"/>
+<pinref part="J1" gate="G$1" pin="B-@2"/>
+<wire x1="304.8" y1="111.76" x2="302.26" y2="111.76" width="0.1524" layer="91"/>
+<junction x="302.26" y="111.76"/>
+</segment>
+<segment>
+<pinref part="U$1" gate="G$1" pin="GND@6"/>
+<pinref part="GND2" gate="1" pin="GND"/>
+<wire x1="185.42" y1="149.86" x2="190.5" y2="149.86" width="0.1524" layer="91"/>
+<wire x1="190.5" y1="149.86" x2="190.5" y2="139.7" width="0.1524" layer="91"/>
+<pinref part="U$1" gate="G$1" pin="GND@14"/>
+<wire x1="190.5" y1="139.7" x2="190.5" y2="132.08" width="0.1524" layer="91"/>
+<wire x1="190.5" y1="132.08" x2="190.5" y2="111.76" width="0.1524" layer="91"/>
+<wire x1="190.5" y1="111.76" x2="190.5" y2="109.22" width="0.1524" layer="91"/>
+<wire x1="185.42" y1="139.7" x2="190.5" y2="139.7" width="0.1524" layer="91"/>
+<junction x="190.5" y="139.7"/>
+<pinref part="U$1" gate="G$1" pin="GND@20"/>
+<wire x1="185.42" y1="132.08" x2="190.5" y2="132.08" width="0.1524" layer="91"/>
+<junction x="190.5" y="132.08"/>
+<pinref part="U$1" gate="G$1" pin="GND@P5_8"/>
+<wire x1="185.42" y1="111.76" x2="190.5" y2="111.76" width="0.1524" layer="91"/>
+<junction x="190.5" y="111.76"/>
+</segment>
+<segment>
+<pinref part="GND3" gate="1" pin="GND"/>
+<pinref part="U$1" gate="G$1" pin="GND@9"/>
+<wire x1="121.92" y1="109.22" x2="121.92" y2="111.76" width="0.1524" layer="91"/>
+<wire x1="121.92" y1="111.76" x2="121.92" y2="124.46" width="0.1524" layer="91"/>
+<wire x1="121.92" y1="124.46" x2="121.92" y2="144.78" width="0.1524" layer="91"/>
+<wire x1="121.92" y1="144.78" x2="129.54" y2="144.78" width="0.1524" layer="91"/>
+<pinref part="U$1" gate="G$1" pin="GND@25"/>
+<wire x1="129.54" y1="124.46" x2="121.92" y2="124.46" width="0.1524" layer="91"/>
+<junction x="121.92" y="124.46"/>
+<pinref part="U$1" gate="G$1" pin="GND@P5_7"/>
+<wire x1="129.54" y1="111.76" x2="121.92" y2="111.76" width="0.1524" layer="91"/>
+<junction x="121.92" y="111.76"/>
+</segment>
+<segment>
+<pinref part="GND4" gate="1" pin="GND"/>
+<wire x1="223.52" y1="109.22" x2="223.52" y2="121.92" width="0.1524" layer="91"/>
+<pinref part="U$2" gate="G$1" pin="PGND"/>
+<wire x1="223.52" y1="121.92" x2="223.52" y2="124.46" width="0.1524" layer="91"/>
+<wire x1="228.6" y1="124.46" x2="223.52" y2="124.46" width="0.1524" layer="91"/>
+<pinref part="U$2" gate="G$1" pin="SGND"/>
+<wire x1="228.6" y1="121.92" x2="223.52" y2="121.92" width="0.1524" layer="91"/>
+<junction x="223.52" y="121.92"/>
+</segment>
+</net>
+<net name="N$1" class="0">
+<segment>
+<pinref part="U$2" gate="G$1" pin="VIN"/>
+<wire x1="228.6" y1="128.27" x2="220.98" y2="128.27" width="0.1524" layer="91"/>
+<wire x1="220.98" y1="128.27" x2="220.98" y2="149.86" width="0.1524" layer="91"/>
+<wire x1="220.98" y1="149.86" x2="304.8" y2="149.86" width="0.1524" layer="91"/>
+<pinref part="J1" gate="G$1" pin="B+@1"/>
+<pinref part="J1" gate="G$1" pin="B+@2"/>
+<wire x1="304.8" y1="147.32" x2="304.8" y2="149.86" width="0.1524" layer="91"/>
+<junction x="304.8" y="149.86"/>
+</segment>
+</net>
+<net name="+5V" class="0">
+<segment>
+<pinref part="U$1" gate="G$1" pin="5V@4"/>
+<pinref part="P+2" gate="1" pin="+5V"/>
+<wire x1="185.42" y1="152.4" x2="193.04" y2="152.4" width="0.1524" layer="91"/>
+<wire x1="193.04" y1="152.4" x2="193.04" y2="154.94" width="0.1524" layer="91"/>
+<pinref part="U$1" gate="G$1" pin="5V@2"/>
+<wire x1="193.04" y1="154.94" x2="193.04" y2="162.56" width="0.1524" layer="91"/>
+<wire x1="185.42" y1="154.94" x2="193.04" y2="154.94" width="0.1524" layer="91"/>
+<junction x="193.04" y="154.94"/>
+</segment>
+<segment>
+<pinref part="P+1" gate="1" pin="+5V"/>
+<pinref part="U$1" gate="G$1" pin="5V@P5_1"/>
+<wire x1="119.38" y1="160.02" x2="119.38" y2="119.38" width="0.1524" layer="91"/>
+<wire x1="119.38" y1="119.38" x2="129.54" y2="119.38" width="0.1524" layer="91"/>
+</segment>
+</net>
+<net name="+3V3" class="0">
+<segment>
+<pinref part="+3V1" gate="G$1" pin="+3V3"/>
+<pinref part="U$1" gate="G$1" pin="3V3@P5_2"/>
+<wire x1="200.66" y1="162.56" x2="200.66" y2="119.38" width="0.1524" layer="91"/>
+<wire x1="200.66" y1="119.38" x2="185.42" y2="119.38" width="0.1524" layer="91"/>
+</segment>
+<segment>
+<pinref part="+3V2" gate="G$1" pin="+3V3"/>
+<pinref part="U$1" gate="G$1" pin="3V3@1"/>
+<wire x1="111.76" y1="160.02" x2="111.76" y2="154.94" width="0.1524" layer="91"/>
+<wire x1="111.76" y1="154.94" x2="129.54" y2="154.94" width="0.1524" layer="91"/>
+<pinref part="U$1" gate="G$1" pin="3V3@17"/>
+<wire x1="129.54" y1="134.62" x2="111.76" y2="134.62" width="0.1524" layer="91"/>
+<wire x1="111.76" y1="134.62" x2="111.76" y2="154.94" width="0.1524" layer="91"/>
+<junction x="111.76" y="154.94"/>
+</segment>
+</net>
 </nets>
 </sheet>

Commit message: Moved daughterboard to behind RP (duh). Added parts form olimex DBs and olf PPC FC carrier: RNC, magnetics,  5/3.3 LTM supply, LED.
Parts:
- removed J1: ROCKETNET-CONNECTOR-16M, rocketnet-connector:ROCKETNET-CONNECTOR-16M
- removed U$2: LT4619_REDUCED, LT4619:LT4619_REDUCED
- added C1: 100nF, rcl_custom:C-EU0603-B-NOSILK
- added C1000, C1007: 22p, rcl_custom:C-EU0603-B-NOSILK
- added C1001, C1008: 100u, rcl:CPOL-EUD/7343-31R
- added C1002, C1009: 200p, rcl_custom:C-EU0603-B-NOSILK
- added C1003, C1004, C1043, C1044: 10u, rcl_custom:C-EU0805-B-NOSILK
- added C1045, C1046: 15n, rcl_custom:C-EU0603-B-NOSILK
- added J2: ROCKETNET-CONNECTOR-16M, rocketnet-connector:ROCKETNET-CONNECTOR-16M
- added L1, L2: ACM2012, magnetics:ACM2012
- added LAN: RJLBC-060TC1, OLIMEX_CONNECTORS:RJLBC-060TC1
- added LED3: (no value), Tova:LED_RGB_PLCC-6
- added R1, R2: 50, rcl_custom:R-US_0603-B-NOSILK
- added R1000: 11.5k, rcl_custom:R-US_0603-B-NOSILK
- added R1001: 19.1k, rcl_custom:R-US_0603-B-NOSILK
- added R1069: 0, rcl_custom:R-US_0603-B-NOSILK
- added R3: 900, rcl_custom:R-US_0603-B-NOSILK
- added R4: 400, rcl_custom:R-US_0603-B-NOSILK
- added R5: 110, rcl_custom:R-US_0603-B-NOSILK
- added T1, T2: ALT4532, magnetics:ALT4532
- added TP1, TP2, TP3, TP4: TEST-POINT, apdm:TEST-POINT
- added TP1000, TP1001, TP1002, TP1003, TP1004, TP1005, TP1007, TP1009, TP1010, TP1011, TP1234, TP1235: TEST, tqm:TEST
- added U1000: LT4619, LT4619:LT4619
Connections:
- removed net N$1: J1.B+@1, J1.B+@2, U$2.VIN
- new net AGND: C1002.2, C1009.2, R1000.1, R1001.1, R1069.2, U1000.SGND@1, U1000.SGND@2, U1000.SGND@3, U1000.SGND@4
- new net COMP1: TP1003.P$1, U1000.COMP1
- new net COMP2: TP1005.P$1, U1000.COMP2
- new net EXTVCC: TP1001.P$1, U1000.EXTVCC
- new net FREQ: TP1000.P$1, U1000.FREQ/PLLFLTR
- new net INTVCC1: TP1002.P$1, U1000.INTVCC
- new net N$10: J2.RX+@1, J2.RX+@2, L2.1
- new net N$11: LAN.TD+, T1.1
- new net N$12: LAN.TD-, T1.2
- new net N$13: LAN.RD+, T2.1
- new net N$14: LAN.RD-, T2.2
- new net N$15: LED3B.K
- new net N$19: J2.RX-@1, J2.RX-@2, L2.2
- new net N$2: LED3R.K
- new net N$20: J2.AUX4, TP4.1
- new net N$21: J2.AUX3, TP3.1
- new net N$22: J2.AUX2, TP2.1
- new net N$23: J2.AUX1, TP1.1
- new net N$24: LAN.COM, T1.6, T2.6
- new net N$25: C1.1, R1.1, R2.1
- new net N$26: R1.2, T2.3
- new net N$27: R2.2, T1.3
- new net N$28: LED3R.A, R3.2
- new net N$29: LED3G.A, R4.2
- new net N$3: L1.4, T1.5
- new net N$30: LED3B.A, R5.2
- new net N$4: LED3G.K
- new net N$5: L1.3, T1.4
- new net N$6: L2.4, T2.5
- new net N$7: L2.3, T2.4
- new net N$8: J2.TX+@1, J2.TX+@2, L1.1
- new net N$9: J2.TX-@1, J2.TX-@2, L1.2
- new net PGOOD: TP1009.P$1, U1000.PGOOD
- new net RUN1: TP1004.P$1, U1000.RUN1
- new net RUN2: TP1007.P$1, U1000.RUN2
- new net SPS-500KHZ: U1000.MODE/PLLIN
- new net SW1: TP1011.P$1, U1000.SW1
- new net SW2: TP1010.P$1, U1000.SW2
- new net TK-SS1: C1002.1, U1000.TK/SS1
- new net TK-SS2: C1009.1, U1000.TK/SS2
- new net TRIPLE_UP_ARROW: C1003.1, C1004.1, J2.B+@1, J2.B+@2, U1000.VIN@1, U1000.VIN@10, U1000.VIN@11, U1000.VIN@12, U1000.VIN@13, U1000.VIN@14, U1000.VIN@15, U1000.VIN@16, U1000.VIN@17, U1000.VIN@18, U1000.VIN@19, U1000.VIN@2, U1000.VIN@20, U1000.VIN@21, U1000.VIN@22, U1000.VIN@23, U1000.VIN@24, U1000.VIN@25, U1000.VIN@26, U1000.VIN@27, U1000.VIN@28, U1000.VIN@29, U1000.VIN@3, U1000.VIN@30, U1000.VIN@31, U1000.VIN@32, U1000.VIN@33, U1000.VIN@34, U1000.VIN@35, U1000.VIN@36, U1000.VIN@4, U1000.VIN@5, U1000.VIN@6, U1000.VIN@7, U1000.VIN@8, U1000.VIN@9
- new net VFB1: C1000.1, R1000.2, U1000.VFB1
- new net VFB2: C1007.2, R1001.2, U1000.VFB2
- net +3V3: now also C1007.1, C1008.+, C1044.1, C1046.1, R3.1, R4.1, R5.1, TP1235.P$1, U1000.VOUT2@1, U1000.VOUT2@10, U1000.VOUT2@11, U1000.VOUT2@12, U1000.VOUT2@2, U1000.VOUT2@3, U1000.VOUT2@4, U1000.VOUT2@5, U1000.VOUT2@6, U1000.VOUT2@7, U1000.VOUT2@8, U1000.VOUT2@9
- net +5V: now also C1000.2, C1001.+, C1043.1, C1045.1, TP1234.P$1, U1000.VOUT1@1, U1000.VOUT1@10, U1000.VOUT1@11, U1000.VOUT1@12, U1000.VOUT1@2, U1000.VOUT1@3, U1000.VOUT1@4, U1000.VOUT1@5, U1000.VOUT1@6, U1000.VOUT1@7, U1000.VOUT1@8, U1000.VOUT1@9
- net GND: now also C1.2, C1001.-, C1003.2, C1004.2, C1008.-, C1043.2, C1044.2, C1045.2, C1046.2, J2.B-@1, J2.B-@2, R1069.1, U1000.PGND@1, U1000.PGND@10, U1000.PGND@11, U1000.PGND@12, U1000.PGND@13, U1000.PGND@14, U1000.PGND@15, U1000.PGND@16, U1000.PGND@17, U1000.PGND@18, U1000.PGND@19, U1000.PGND@2, U1000.PGND@20, U1000.PGND@21, U1000.PGND@22, U1000.PGND@23, U1000.PGND@24, U1000.PGND@25, U1000.PGND@26, U1000.PGND@27, U1000.PGND@28, U1000.PGND@29, U1000.PGND@3, U1000.PGND@30, U1000.PGND@31, U1000.PGND@32, U1000.PGND@33, U1000.PGND@34, U1000.PGND@35, U1000.PGND@36, U1000.PGND@37, U1000.PGND@38, U1000.PGND@39, U1000.PGND@4, U1000.PGND@40, U1000.PGND@41, U1000.PGND@42, U1000.PGND@43, U1000.PGND@44, U1000.PGND@45, U1000.PGND@46, U1000.PGND@47, U1000.PGND@48, U1000.PGND@49, U1000.PGND@5, U1000.PGND@50, U1000.PGND@51, U1000.PGND@52, U1000.PGND@53, U1000.PGND@54, U1000.PGND@55, U1000.PGND@56, U1000.PGND@57, U1000.PGND@58, U1000.PGND@59, U1000.PGND@6, U1000.PGND@60, U1000.PGND@61, U1000.PGND@62, U1000.PGND@63, U1000.PGND@64, U1000.PGND@65, U1000.PGND@7, U1000.PGND@8, U1000.PGND@9; no longer J1.B-@1, J1.B-@2, U$2.PGND, U$2.SGND
Other:
- note added: "1%"
- note added: "FIXME: WHICH GPIO?"
- note added: "FIXME: WRONG ETH CONNECTOR FOR RP"
- moved on the sheet: U$1

Commit message: Added scan of RP bottom side at 2400 dpi (sorry, it's 50 MB!). Used that to verify P5 and P4 placement. Updated EAGLE library schematic and footprint to be better.
Parts:
- removed U$1: RASPBERRY-PI_REV2, RaspberryPi:RASPBERRY-PI_REV2
- added J1: RP-REV2-MOAR, RaspberryPi:RP-REV2-MOAR
Connections:
- net +3V3: now also J1G$1.3V3@1, J1G$1.3V3@17, J1G$3.5V@P5_1; no longer U$1.3V3@1, U$1.3V3@17, U$1.3V3@P5_2
- net +5V: now also J1G$1.5V@2, J1G$1.5V@4; no longer U$1.5V@2, U$1.5V@4, U$1.5V@P5_1
- net GND: now also J1G$1.GND@14, J1G$1.GND@20, J1G$1.GND@25, J1G$1.GND@6, J1G$1.GND@9, J1G$3.GND@P5_7, J1G$3.GND@P5_8; no longer U$1.GND@14, U$1.GND@20, U$1.GND@25, U$1.GND@6, U$1.GND@9, U$1.GND@P5_7, U$1.GND@P5_8
- net N$11: now also J1G$2.P4_1
- net N$12: now also J1G$2.P4_2
- net N$13: now also J1G$2.P4_4
- net N$14: now also J1G$2.P4_5
- net N$24: now also J1G$2.P4_3
Other:
- note added: "FIXME: NOT CORRECT"

Commit message: More on the RP carrier: added the ethernet connector wiring, and LED randomly, and first pass of the power switchers using TI's simple switchers because we're lazy and they're relatively cheap for a one off.
Parts:
- removed C1000, C1007: 22p, rcl_custom:C-EU0603-B-NOSILK
- removed C1002, C1009: 200p, rcl_custom:C-EU0603-B-NOSILK
- removed LAN: RJLBC-060TC1, OLIMEX_CONNECTORS:RJLBC-060TC1
- removed R1000: 11.5k, rcl_custom:R-US_0603-B-NOSILK
- removed R1001: 19.1k, rcl_custom:R-US_0603-B-NOSILK
- removed R1069: 0, rcl_custom:R-US_0603-B-NOSILK
- removed TP1000, TP1001, TP1002, TP1003, TP1004, TP1005, TP1007, TP1009, TP1010, TP1011: TEST, tqm:TEST
- removed U1000: LT4619, LT4619:LT4619
- added C2, C3, C4, C5: TBD, rcl_custom:C-EU0603-B-NOSILK
- added R10, R11, R6, R7, R8, R9: 11.5k, rcl_custom:R-US_0603-B-NOSILK
- added TP5, TP6: TEST, tqm:TEST
- added U1, U2: LMZ14203, SparkFun-PowerIC:LMZ14203
Connections:
- removed net AGND: C1002.2, C1009.2, R1000.1, R1001.1, R1069.2, U1000.SGND@1, U1000.SGND@2, U1000.SGND@3, U1000.SGND@4
- removed net COMP1: TP1003.P$1, U1000.COMP1
- removed net COMP2: TP1005.P$1, U1000.COMP2
- removed net EXTVCC: TP1001.P$1, U1000.EXTVCC
- removed net FREQ: TP1000.P$1, U1000.FREQ/PLLFLTR
- removed net INTVCC1: TP1002.P$1, U1000.INTVCC
- removed net PGOOD: TP1009.P$1, U1000.PGOOD
- removed net RUN1: TP1004.P$1, U1000.RUN1
- removed net RUN2: TP1007.P$1, U1000.RUN2
- removed net SPS-500KHZ: U1000.MODE/PLLIN
- removed net SW1: TP1011.P$1, U1000.SW1
- removed net SW2: TP1010.P$1, U1000.SW2
- removed net TK-SS1: C1002.1, U1000.TK/SS1
- removed net TK-SS2: C1009.1, U1000.TK/SS2
- removed net VFB1: C1000.1, R1000.2, U1000.VFB1
- removed net VFB2: C1007.2, R1001.2, U1000.VFB2
- new net N$1: J1G$2.P4_2, T1.6
- new net N$16: J1G$2.P4_5, T2.6
- new net N$17: C3.1, U2.SS
- new net N$18: C2.1, U1.SS
- new net N$31: R7.2, U2.RON
- new net N$32: TP6.P$1, U1.EN
- new net N$33: TP5.P$1, U2.EN
- new net N$34: C4.2, R8.2, R9.1, U2.FB
- new net N$35: C5.2, R10.2, R11.1, U1.FB
- net +3V3: now also C4.1, R8.1, U2.VOUT; no longer C1007.1, U1000.VOUT2@1, U1000.VOUT2@10, U1000.VOUT2@11, U1000.VOUT2@12, U1000.VOUT2@2, U1000.VOUT2@3, U1000.VOUT2@4, U1000.VOUT2@5, U1000.VOUT2@6, U1000.VOUT2@7, U1000.VOUT2@8, U1000.VOUT2@9
- net +5V: now also C5.1, J1G$3.3V3@P5_2, R10.1, U1.VOUT; no longer C1000.2, U1000.VOUT1@1, U1000.VOUT1@10, U1000.VOUT1@11, U1000.VOUT1@12, U1000.VOUT1@2, U1000.VOUT1@3, U1000.VOUT1@4, U1000.VOUT1@5, U1000.VOUT1@6, U1000.VOUT1@7, U1000.VOUT1@8, U1000.VOUT1@9
- net GND: now also C2.2, C3.2, R11.2, R9.2, U1.GND, U2.GND; no longer R1069.1, U1000.PGND@1, U1000.PGND@10, U1000.PGND@11, U1000.PGND@12, U1000.PGND@13, U1000.PGND@14, U1000.PGND@15, U1000.PGND@16, U1000.PGND@17, U1000.PGND@18, U1000.PGND@19, U1000.PGND@2, U1000.PGND@20, U1000.PGND@21, U1000.PGND@22, U1000.PGND@23, U1000.PGND@24, U1000.PGND@25, U1000.PGND@26, U1000.PGND@27, U1000.PGND@28, U1000.PGND@29, U1000.PGND@3, U1000.PGND@30, U1000.PGND@31, U1000.PGND@32, U1000.PGND@33, U1000.PGND@34, U1000.PGND@35, U1000.PGND@36, U1000.PGND@37, U1000.PGND@38, U1000.PGND@39, U1000.PGND@4, U1000.PGND@40, U1000.PGND@41, U1000.PGND@42, U1000.PGND@43, U1000.PGND@44, U1000.PGND@45, U1000.PGND@46, U1000.PGND@47, U1000.PGND@48, U1000.PGND@49, U1000.PGND@5, U1000.PGND@50, U1000.PGND@51, U1000.PGND@52, U1000.PGND@53, U1000.PGND@54, U1000.PGND@55, U1000.PGND@56, U1000.PGND@57, U1000.PGND@58, U1000.PGND@59, U1000.PGND@6, U1000.PGND@60, U1000.PGND@61, U1000.PGND@62, U1000.PGND@63, U1000.PGND@64, U1000.PGND@65, U1000.PGND@7, U1000.PGND@8, U1000.PGND@9
- net N$11: no longer LAN.TD+
- net N$12: now also J1G$2.P4_3; no longer J1G$2.P4_2, LAN.TD-
- net N$13: no longer LAN.RD+
- net N$14: now also J1G$2.P4_6; no longer J1G$2.P4_5, LAN.RD-
- net N$15: now also J1G$3.GPIO31
- net N$2: now also J1G$3.GPIO29
- net N$24: now also R6.2, U1.RON; no longer J1G$2.P4_3, LAN.COM, T1.6, T2.6
- net N$4: now also J1G$3.GPIO30
- net TRIPLE_UP_ARROW: now also R6.1, R7.1, U1.VIN, U2.VIN; no longer U1000.VIN@1, U1000.VIN@10, U1000.VIN@11, U1000.VIN@12, U1000.VIN@13, U1000.VIN@14, U1000.VIN@15, U1000.VIN@16, U1000.VIN@17, U1000.VIN@18, U1000.VIN@19, U1000.VIN@2, U1000.VIN@20, U1000.VIN@21, U1000.VIN@22, U1000.VIN@23, U1000.VIN@24, U1000.VIN@25, U1000.VIN@26, U1000.VIN@27, U1000.VIN@28, U1000.VIN@29, U1000.VIN@3, U1000.VIN@30, U1000.VIN@31, U1000.VIN@32, U1000.VIN@33, U1000.VIN@34, U1000.VIN@35, U1000.VIN@36, U1000.VIN@4, U1000.VIN@5, U1000.VIN@6, U1000.VIN@7, U1000.VIN@8, U1000.VIN@9
Other:
- note added: "RX+"
- note added: "RX-"
- note added: "TX+"
- note added: "TX-"
- note removed: "FIXME: NOT CORRECT"
- note removed: "FIXME: WHICH GPIO?"
- note removed: "FIXME: WRONG ETH CONNECTOR FOR RP"
- moved on the sheet: C1, C1001, C1003, C1004, C1008, C1043, C1044, C1045, C1046, J1G$1, J2, L1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

Commit message: Added FTDI breakout, cleaned up schematic a bit, design review with Paul.
Parts:
- added JP1: (no value), pinhead:PINHD-1X6/90
- U1, U2: value LMZ14203 -> LMZ12001
Connections:
- new net N$36: J1G$1.GPIO15,UART0_RXD, JP1.4
- new net N$37: J1G$1.GPIO14,UART0_TXD, JP1.5
- net GND: now also JP1.1
Changed lines of the file:
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@@
 <setting verticaltext="up"/>
 </settings>
-<grid distance="0.05" unitdist="inch" unit="inch" style="lines" multiple="2" display="yes" altdistance="0.01" altunitdist="inch" altunit="inch"/>
+<grid distance="0.1" unitdist="inch" unit="inch" style="lines" multiple="1" display="no" altdistance="0.01" altunitdist="inch" altunit="inch"/>
 <layers>
 <layer number="1" name="Top" color="4" fill="1" visible="no" active="no"/>
@@
 <part name="P+2" library="supply1" deviceset="+5V" device=""/>
 <part name="+3V1" library="supply1" deviceset="+3V3" device=""/>
-<part name="U1" library="SparkFun-PowerIC" deviceset="LMZ14203" device=""/>
-<part name="U2" library="SparkFun-PowerIC" deviceset="LMZ14203" device=""/>
+<part name="U1" library="SparkFun-PowerIC" deviceset="LMZ14203" device="" value="LMZ12001"/>
+<part name="U2" library="SparkFun-PowerIC" deviceset="LMZ14203" device="" value="LMZ12001"/>
 <part name="GND2" library="supply1" deviceset="GND" device=""/>
 <part name="GND4" library="supply1" deviceset="GND" device=""/>
@@
 <part name="C4" library="rcl_custom" deviceset="C-EU" device="0603-B-NOSILK" value="TBD"/>
 <part name="C5" library="rcl_custom" deviceset="C-EU" device="0603-B-NOSILK" value="TBD"/>
+<part name="JP1" library="pinhead" deviceset="PINHD-1X6" device="/90"/>
+<part name="GND19" library="supply1" deviceset="GND" device=""/>
 </parts>
 <sheets>
@@
 <instance part="C4" gate="CE" x="195.58" y="109.22" rot="MR0"/>
 <instance part="C5" gate="CE" x="195.58" y="144.78" rot="MR0"/>
+<instance part="JP1" gate="A" x="256.54" y="152.4" rot="MR0"/>
+<instance part="GND19" gate="1" x="266.7" y="142.24"/>
 </instances>
 <busses>
@@
 <pinref part="R11" gate="R" pin="2"/>
 <pinref part="GND18" gate="1" pin="GND"/>
+</segment>
+<segment>
+<pinref part="JP1" gate="A" pin="1"/>
+<pinref part="GND19" gate="1" pin="GND"/>
+<wire x1="259.08" y1="160.02" x2="266.7" y2="160.02" width="0.1524" layer="91"/>
+<wire x1="266.7" y1="160.02" x2="266.7" y2="144.78" width="0.1524" layer="91"/>
 </segment>
 </net>
@@
 </segment>
 </net>
+<net name="N$36" class="0">
+<segment>
+<pinref part="JP1" gate="A" pin="4"/>
+<wire x1="259.08" y1="152.4" x2="274.32" y2="152.4" width="0.1524" layer="91"/>
+<wire x1="274.32" y1="152.4" x2="274.32" y2="142.24" width="0.1524" layer="91"/>
+<pinref part="J1" gate="G$1" pin="GPIO15,UART0_RXD"/>
+<wire x1="274.32" y1="142.24" x2="284.48" y2="142.24" width="0.1524" layer="91"/>
+</segment>
+</net>
+<net name="N$37" class="0">
+<segment>
+<pinref part="J1" gate="G$1" pin="GPIO14,UART0_TXD"/>
+<wire x1="284.48" y1="144.78" x2="276.86" y2="144.78" width="0.1524" layer="91"/>
+<wire x1="276.86" y1="144.78" x2="276.86" y2="149.86" width="0.1524" layer="91"/>
+<pinref part="JP1" gate="A" pin="5"/>
+<wire x1="276.86" y1="149.86" x2="259.08" y2="149.86" width="0.1524" layer="91"/>
+</segment>
+</net>

Commit message: Completed RPi daughterboard layout.
Parts:
- removed TP1234, TP1235: TEST, tqm:TEST
- added JP2: (no value), pinhead:PINHD-1X2
- added Q1: NTR4101P, Tova:NTR4101P
- added R12: 50, rcl_custom:R-US_0603-B-NOSILK
- added TP7, TP8: TEST-POINT, apdm:TEST-POINT
- JP1: device pinhead:PINHD-1X6/90 -> pinhead:PINHD-1X6
- TP5, TP6: value TEST -> TEST-POINT; device tqm:TEST -> apdm:TEST-POINT
Connections:
- new net N$38: J1G$1.GPIO17, Q1.G
- new net N$39: JP2.1, Q1.D
- new net N$40: Q1.S, R12.1
- net +3V3: now also TP8.1; no longer TP1235.P$1
- net +5V: now also R12.2, TP7.1; no longer TP1234.P$1
- net GND: now also JP2.2, U1.EP, U2.EP
- net N$32: now also TP5.1; no longer TP6.P$1
- net N$33: now also TP6.1; no longer TP5.P$1
Other:
- moved on the sheet: C1001, C1003, C1004, C1008, C1043, C1044, C1045, C1046, C2, C3, C4, C5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
