File: av4/raspi-camera/eagle/raspi-rnc.sch (EAGLE design)
At the start: 45 parts, among them J1 RP-REV2-MOAR, J2 ROCKETNET-CONNECTOR-16M, Q1 NTR4101P, T1 ALT4532, T2 ALT4532, U1 LMZ12001, U2 LMZ12001

Commit message: Fixed gearcam transistor (no 5V to the RP!!11!), made power wires bigger, fixed tname.
Parts:
- Q1: value NTR4101P -> PMV45EN; device Tova:NTR4101P -> Tova:PMV45EN
- R12: value 50 -> 10k
Connections:
- removed net N$39: JP2.1, Q1.D
- net +5V: now also JP2.1; no longer R12.2
- net GND: now also Q1.S, R12.1; no longer JP2.2
- net N$38: now also R12.2
- net N$40: now also JP2.2, Q1.D; no longer Q1.S, R12.1
Other:
- note added: "Camera Power"
- note added: "FTDI 3.3V cable"
- moved on the sheet: Q1, R12
Changed lines of the file:
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@@
 <part name="P+3" library="supply1" deviceset="+5V" device=""/>
 <part name="GND20" library="supply1" deviceset="GND" device=""/>
-<part name="Q1" library="Tova" deviceset="NTR4101P" device=""/>
-<part name="R12" library="rcl_custom" deviceset="R-US_" device="0603-B-NOSILK" value="50"/>
+<part name="R12" library="rcl_custom" deviceset="R-US_" device="0603-B-NOSILK" value="10k"/>
 <part name="TP5" library="apdm" deviceset="TEST-POINT" device=""/>
 <part name="TP6" library="apdm" deviceset="TEST-POINT" device=""/>
 <part name="TP7" library="apdm" deviceset="TEST-POINT" device=""/>
 <part name="TP8" library="apdm" deviceset="TEST-POINT" device=""/>
+<part name="Q1" library="Tova" deviceset="PMV45EN" device=""/>
 </parts>
 <sheets>
@@
 <text x="194.31" y="220.98" size="1.778" layer="97">RX+</text>
 <text x="194.31" y="208.28" size="1.778" layer="97">RX-</text>
+<text x="238.76" y="162.56" size="1.778" layer="97">FTDI 3.3V cable</text>
+<text x="208.28" y="121.92" size="1.778" layer="97">Camera Power</text>
 </plain>
 <instances>
@@
 <instance part="GND17" gate="1" x="130.81" y="91.44"/>
 <instance part="GND18" gate="1" x="130.81" y="127"/>
-<instance part="C4" gate="CE" x="138.43" y="111.76" rot="MR0"/>
+<instance part="C4" gate="CE" x="138.43" y="111.76" smashed="yes" rot="MR0">
+<attribute name="NAME" x="143.51" y="111.76" size="1.778" layer="95" rot="MR0"/>
+<attribute name="VALUE" x="143.51" y="106.68" size="1.778" layer="96" rot="MR0"/>
+</instance>
 <instance part="C5" gate="CE" x="138.43" y="147.32" smashed="yes" rot="MR0">
 <attribute name="NAME" x="143.51" y="147.32" size="1.778" layer="95" rot="MR0"/>
@@
 </instance>
 <instance part="JP1" gate="A" x="261.62" y="162.56" rot="MR0"/>
-<instance part="GND19" gate="1" x="271.78" y="149.86"/>
+<instance part="GND19" gate="1" x="271.78" y="165.1"/>
 <instance part="JP2" gate="G$1" x="228.6" y="121.92" rot="MR0"/>
-<instance part="P+3" gate="1" x="238.76" y="160.02"/>
-<instance part="GND20" gate="1" x="238.76" y="115.57" rot="MR0"/>
-<instance part="Q1" gate="G$1" x="238.76" y="134.62" rot="MR0"/>
-<instance part="R12" gate="R" x="238.76" y="147.32" smashed="yes" rot="R90">
-<attribute name="NAME" x="232.41" y="147.32" size="1.778" layer="95"/>
-<attribute name="VALUE" x="232.41" y="145.288" size="1.778" layer="96"/>
+<instance part="P+3" gate="1" x="238.76" y="134.62"/>
+<instance part="GND20" gate="1" x="238.76" y="101.6" rot="MR0"/>
+<instance part="R12" gate="R" x="246.38" y="109.22" smashed="yes" rot="R90">
+<attribute name="NAME" x="240.03" y="109.22" size="1.778" layer="95"/>
+<attribute name="VALUE" x="240.03" y="107.188" size="1.778" layer="96"/>
 </instance>
 <instance part="TP5" gate="G$1" x="95.25" y="144.78" rot="MR0"/>
@@
 <instance part="TP7" gate="G$1" x="158.75" y="149.86" rot="MR0"/>
 <instance part="TP8" gate="G$1" x="158.75" y="114.3" rot="MR0"/>
+<instance part="Q1" gate="G$1" x="238.76" y="116.84" rot="MR0"/>
 </instances>
 <busses>
@@
 <pinref part="GND19" gate="1" pin="GND"/>
 <wire x1="264.16" y1="170.18" x2="271.78" y2="170.18" width="0.1524" layer="91"/>
-<wire x1="271.78" y1="170.18" x2="271.78" y2="152.4" width="0.1524" layer="91"/>
-</segment>
-<segment>
-<pinref part="JP2" gate="G$1" pin="2"/>
+<wire x1="271.78" y1="170.18" x2="271.78" y2="167.64" width="0.1524" layer="91"/>
+</segment>
+<segment>
 <pinref part="GND20" gate="1" pin="GND"/>
-<wire x1="231.14" y1="121.92" x2="238.76" y2="121.92" width="0.1524" layer="91"/>
-<wire x1="238.76" y1="121.92" x2="238.76" y2="118.11" width="0.1524" layer="91"/>
+<pinref part="Q1" gate="G$1" pin="S"/>
+<wire x1="238.76" y1="104.14" x2="238.76" y2="111.76" width="0.1524" layer="91"/>
+<pinref part="R12" gate="R" pin="1"/>
+<wire x1="238.76" y1="104.14" x2="246.38" y2="104.14" width="0.1524" layer="91"/>
+<junction x="238.76" y="104.14"/>
 </segment>
 </net>
@@
 </segment>
 <segment>
+<pinref part="JP2" gate="G$1" pin="1"/>
+<wire x1="238.76" y1="124.46" x2="231.14" y2="124.46" width="0.1524" layer="91"/>
 <pinref part="P+3" gate="1" pin="+5V"/>
-<pinref part="R12" gate="R" pin="2"/>
-<wire x1="238.76" y1="157.48" x2="238.76" y2="152.4" width="0.1524" layer="91"/>
+<wire x1="238.76" y1="132.08" x2="238.76" y2="124.46" width="0.1524" layer="91"/>
 </segment>
 </net>
@@
 <segment>
 <pinref part="JP1" gate="A" pin="4"/>
-<wire x1="264.16" y1="162.56" x2="279.4" y2="162.56" width="0.1524" layer="91"/>
-<wire x1="279.4" y1="162.56" x2="279.4" y2="142.24" width="0.1524" layer="91"/>
+<wire x1="264.16" y1="162.56" x2="276.86" y2="162.56" width="0.1524" layer="91"/>
+<wire x1="276.86" y1="162.56" x2="276.86" y2="142.24" width="0.1524" layer="91"/>
 <pinref part="J1" gate="G$1" pin="GPIO15,UART0_RXD"/>
-<wire x1="279.4" y1="142.24" x2="284.48" y2="142.24" width="0.1524" layer="91"/>
+<wire x1="276.86" y1="142.24" x2="284.48" y2="142.24" width="0.1524" layer="91"/>
 </segment>
 </net>
@@
 <segment>
 <pinref part="JP1" gate="A" pin="5"/>
-<wire x1="264.16" y1="160.02" x2="280.67" y2="160.02" width="0.1524" layer="91"/>
-<wire x1="280.67" y1="160.02" x2="280.67" y2="144.78" width="0.1524" layer="91"/>
+<wire x1="264.16" y1="160.02" x2="279.4" y2="160.02" width="0.1524" layer="91"/>
+<wire x1="279.4" y1="160.02" x2="279.4" y2="144.78" width="0.1524" layer="91"/>
 <pinref part="J1" gate="G$1" pin="GPIO14,UART0_TXD"/>
-<wire x1="280.67" y1="144.78" x2="284.48" y2="144.78" width="0.1524" layer="91"/>
+<wire x1="279.4" y1="144.78" x2="284.48" y2="144.78" width="0.1524" layer="91"/>
 </segment>
 </net>
 <net name="N$38" class="0">
 <segment>
+<pinref part="J1" gate="G$1" pin="GPIO17"/>
+<wire x1="246.38" y1="137.16" x2="284.48" y2="137.16" width="0.1524" layer="91"/>
 <pinref part="Q1" gate="G$1" pin="G"/>
-<pinref part="J1" gate="G$1" pin="GPIO17"/>
-<wire x1="243.84" y1="137.16" x2="284.48" y2="137.16" width="0.1524" layer="91"/>
-</segment>
-</net>
-<net name="N$39" class="0">
-<segment>
+<wire x1="243.84" y1="114.3" x2="246.38" y2="114.3" width="0.1524" layer="91"/>
+<wire x1="246.38" y1="114.3" x2="246.38" y2="137.16" width="0.1524" layer="91"/>
+<pinref part="R12" gate="R" pin="2"/>
+<junction x="246.38" y="114.3"/>
+</segment>
+</net>
+<net name="N$40" class="0">
+<segment>
+<pinref part="JP2" gate="G$1" pin="2"/>
+<wire x1="231.14" y1="121.92" x2="238.76" y2="121.92" width="0.1524" layer="91"/>
 <pinref part="Q1" gate="G$1" pin="D"/>
-<wire x1="238.76" y1="129.54" x2="238.76" y2="124.46" width="0.1524" layer="91"/>
-<pinref part="JP2" gate="G$1" pin="1"/>
-<wire x1="238.76" y1="124.46" x2="231.14" y2="124.46" width="0.1524" layer="91"/>
-</segment>
-</net>
-<net name="N$40" class="0">
-<segment>
-<pinref part="R12" gate="R" pin="1"/>
-<pinref part="Q1" gate="G$1" pin="S"/>
-<wire x1="238.76" y1="142.24" x2="238.76" y2="139.7" width="0.1524" layer="91"/>
-</segment>
-</net>
+</segment>
+</net>

Commit message: Set values on RP carriers, also BOM.
Parts:
- C1: value 100nF -> 1n 2kv
- C1003, C1004: value 10u -> 10u 40V
- C2, C3, C4, C5: value TBD -> 22n
- R1, R2: value 50 -> 75
- R10: value 11.5k -> 5.62k
- R11, R9: value 11.5k -> 1.07k
- R8: value 11.5k -> 3.32k
Changed lines of the file:
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@@
 <setting verticaltext="up"/>
 </settings>
-<grid distance="0.05" unitdist="inch" unit="inch" style="lines" multiple="2" display="yes" altdistance="0.01" altunitdist="inch" altunit="inch"/>
+<grid distance="0.1" unitdist="inch" unit="inch" style="lines" multiple="1" display="no" altdistance="0.01" altunitdist="inch" altunit="inch"/>
 <layers>
 <layer number="1" name="Top" color="4" fill="1" visible="no" active="no"/>
@@
 <part name="L1" library="magnetics" deviceset="ACM2012" device=""/>
 <part name="L2" library="magnetics" deviceset="ACM2012" device=""/>
-<part name="C1" library="rcl_custom" deviceset="C-EU" device="0603-B-NOSILK" value="100nF"/>
-<part name="R1" library="rcl_custom" deviceset="R-US_" device="0603-B-NOSILK" value="50"/>
-<part name="R2" library="rcl_custom" deviceset="R-US_" device="0603-B-NOSILK" value="50"/>
+<part name="C1" library="rcl_custom" deviceset="C-EU" device="0603-B-NOSILK" value="1n 2kv"/>
+<part name="R1" library="rcl_custom" deviceset="R-US_" device="0603-B-NOSILK" value="75"/>
+<part name="R2" library="rcl_custom" deviceset="R-US_" device="0603-B-NOSILK" value="75"/>
 <part name="LED3" library="Tova" deviceset="LED_RGB_*" device="PLCC-6"/>
 <part name="R3" library="rcl_custom" deviceset="R-US_" device="0603-B-NOSILK" value="900"/>
@@
 <part name="GND6" library="supply1" deviceset="GND" device=""/>
 <part name="+3V3" library="supply1" deviceset="+3V3" device=""/>
-<part name="C1003" library="rcl_custom" deviceset="C-EU" device="0805-B-NOSILK" value="10u"/>
-<part name="C3" library="rcl_custom" deviceset="C-EU" device="0603-B-NOSILK" value="TBD"/>
-<part name="C1004" library="rcl_custom" deviceset="C-EU" device="0805-B-NOSILK" value="10u"/>
+<part name="C1003" library="rcl_custom" deviceset="C-EU" device="0805-B-NOSILK" value="10u 40V"/>
+<part name="C3" library="rcl_custom" deviceset="C-EU" device="0603-B-NOSILK" value="22n"/>
+<part name="C1004" library="rcl_custom" deviceset="C-EU" device="0805-B-NOSILK" value="10u 40V"/>
 <part name="+3V4" library="supply1" deviceset="+3V3" device=""/>
 <part name="P+4" library="supply1" deviceset="+5V" device=""/>
@@
 <part name="GND13" library="supply1" deviceset="GND" device=""/>
 <part name="GND14" library="supply1" deviceset="GND" device=""/>
-<part name="C2" library="rcl_custom" deviceset="C-EU" device="0603-B-NOSILK" value="TBD"/>
+<part name="C2" library="rcl_custom" deviceset="C-EU" device="0603-B-NOSILK" value="22n"/>
 <part name="GND15" library="supply1" deviceset="GND" device=""/>
 <part name="GND16" library="supply1" deviceset="GND" device=""/>
 <part name="R6" library="rcl_custom" deviceset="R-US_" device="0603-B-NOSILK" value="11.5k"/>
 <part name="R7" library="rcl_custom" deviceset="R-US_" device="0603-B-NOSILK" value="11.5k"/>
-<part name="R8" library="rcl_custom" deviceset="R-US_" device="0603-B-NOSILK" value="11.5k"/>
-<part name="R9" library="rcl_custom" deviceset="R-US_" device="0603-B-NOSILK" value="11.5k"/>
-<part name="R10" library="rcl_custom" deviceset="R-US_" device="0603-B-NOSILK" value="11.5k"/>
-<part name="R11" library="rcl_custom" deviceset="R-US_" device="0603-B-NOSILK" value="11.5k"/>
+<part name="R8" library="rcl_custom" deviceset="R-US_" device="0603-B-NOSILK" value="3.32k"/>
+<part name="R9" library="rcl_custom" deviceset="R-US_" device="0603-B-NOSILK" value="1.07k"/>
+<part name="R10" library="rcl_custom" deviceset="R-US_" device="0603-B-NOSILK" value="5.62k"/>
+<part name="R11" library="rcl_custom" deviceset="R-US_" device="0603-B-NOSILK" value="1.07k"/>
 <part name="GND17" library="supply1" deviceset="GND" device=""/>
 <part name="GND18" library="supply1" deviceset="GND" device=""/>
-<part name="C4" library="rcl_custom" deviceset="C-EU" device="0603-B-NOSILK" value="TBD"/>
-<part name="C5" library="rcl_custom" deviceset="C-EU" device="0603-B-NOSILK" value="TBD"/>
+<part name="C4" library="rcl_custom" deviceset="C-EU" device="0603-B-NOSILK" value="22n"/>
+<part name="C5" library="rcl_custom" deviceset="C-EU" device="0603-B-NOSILK" value="22n"/>
 <part name="JP1" library="pinhead" deviceset="PINHD-1X6" device=""/>
 <part name="GND19" library="supply1" deviceset="GND" device=""/>
