File: av4/raspi-camera/eagle/raspi-rnc.sch (EAGLE design)
At the start: 45 parts, among them J1 RP-REV2-MOAR, J2 ROCKETNET-CONNECTOR-16M, Q1 PMV45EN, T1 ALT4532, T2 ALT4532, U1 LMZ12001, U2 LMZ12001

Commit message: Updated RasPi 0.1" header position and hole placement, as well as added a new 3rd hole. Extended board to have more room for RNC, moved resistor, version is now 2!
Parts:
- removed TP1, TP2, TP3, TP4: TEST-POINT, apdm:TEST-POINT
Connections:
- removed net N$20: J2.AUX4, TP4.1
- removed net N$21: J2.AUX3, TP3.1
- removed net N$22: J2.AUX2, TP2.1
- removed net N$23: J2.AUX1, TP1.1
Changed lines of the file:
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@@
 <?xml version="1.0" encoding="utf-8"?>
 <!DOCTYPE eagle SYSTEM "eagle.dtd">
-<eagle version="6.5.0">
+<eagle version="6.6.0">
 <drawing>
 <settings>
@@
 <part name="+3V2" library="supply1" deviceset="+3V3" device=""/>
 <part name="TRIPLE_UP_ARROW2" library="supply" deviceset="POS_ARROW_TRIPLE" device="" value="Vin"/>
-<part name="TP1" library="apdm" deviceset="TEST-POINT" device=""/>
-<part name="TP2" library="apdm" deviceset="TEST-POINT" device=""/>
-<part name="TP3" library="apdm" deviceset="TEST-POINT" device=""/>
-<part name="TP4" library="apdm" deviceset="TEST-POINT" device=""/>
 <part name="J2" library="rocketnet-connector" deviceset="ROCKETNET-CONNECTOR-16" device="M"/>
 <part name="T1" library="magnetics" deviceset="ALT4532" device=""/>
@@
 <instance part="+3V2" gate="G$1" x="309.88" y="185.42"/>
 <instance part="TRIPLE_UP_ARROW2" gate="1" x="248.92" y="248.92" rot="MR0"/>
-<instance part="TP1" gate="G$1" x="243.84" y="218.44" rot="MR0"/>
-<instance part="TP2" gate="G$1" x="243.84" y="215.9" rot="MR0"/>
-<instance part="TP3" gate="G$1" x="243.84" y="213.36" rot="MR0"/>
-<instance part="TP4" gate="G$1" x="243.84" y="210.82" rot="MR0"/>
 <instance part="J2" gate="G$1" x="256.54" y="226.06" rot="MR0"/>
 <instance part="T1" gate="G$1" x="208.28" y="236.22"/>
@@
 </segment>
 </net>
-<net name="N$20" class="0">
-<segment>
-<pinref part="TP4" gate="G$1" pin="1"/>
-<pinref part="J2" gate="G$1" pin="AUX4"/>
-<wire x1="243.84" y1="210.82" x2="251.46" y2="210.82" width="0.1524" layer="91"/>
-</segment>
-</net>
-<net name="N$21" class="0">
-<segment>
-<pinref part="J2" gate="G$1" pin="AUX3"/>
-<pinref part="TP3" gate="G$1" pin="1"/>
-<wire x1="251.46" y1="213.36" x2="243.84" y2="213.36" width="0.1524" layer="91"/>
-</segment>
-</net>
-<net name="N$22" class="0">
-<segment>
-<pinref part="TP2" gate="G$1" pin="1"/>
-<pinref part="J2" gate="G$1" pin="AUX2"/>
-<wire x1="243.84" y1="215.9" x2="251.46" y2="215.9" width="0.1524" layer="91"/>
-</segment>
-</net>
-<net name="N$23" class="0">
-<segment>
-<pinref part="J2" gate="G$1" pin="AUX1"/>
-<pinref part="TP1" gate="G$1" pin="1"/>
-<wire x1="251.46" y1="218.44" x2="243.84" y2="218.44" width="0.1524" layer="91"/>
-</segment>
-</net>

Commit message: how is it that this wasn't committed a bzillion years ago? This new schematic has the mods for the optoisolator on it.
Parts:
- added JP3: (no value), pinhead:PINHD-1X2
- added OK1: 4N28SM, optocoupler:4N28SM
- added R13: ??k, rcl_custom:R-US_0603-B-NOSILK
Connections:
- new net N$20: J1G$3.GPIO28, R13.2
- new net N$21: OK1.A, R13.1
- new net N$23: JP3.2, OK1.COL
- new net N$39: JP3.1, OK1.EMI
- net GND: now also OK1.C
Other:
- note added: "GoPro "Start" (not stop!) signal"
Changed lines of the file:
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@@
 <setting verticaltext="up"/>
 </settings>
-<grid distance="0.1" unitdist="inch" unit="inch" style="lines" multiple="1" display="no" altdistance="0.01" altunitdist="inch" altunit="inch"/>
+<grid distance="0.05" unitdist="inch" unit="inch" style="lines" multiple="2" display="no" altdistance="0.01" altunitdist="inch" altunit="inch"/>
 <layers>
 <layer number="1" name="Top" color="4" fill="1" visible="no" active="no"/>
@@
 <part name="TP8" library="apdm" deviceset="TEST-POINT" device=""/>
 <part name="Q1" library="Tova" deviceset="PMV45EN" device=""/>
+<part name="OK1" library="optocoupler" deviceset="4N*?M" device="S" technology="28"/>
+<part name="R13" library="rcl_custom" deviceset="R-US_" device="0603-B-NOSILK" value="??k"/>
+<part name="GND21" library="supply1" deviceset="GND" device=""/>
+<part name="JP3" library="pinhead" deviceset="PINHD-1X2" device=""/>
 </parts>
 <sheets>
@@
 <text x="238.76" y="162.56" size="1.778" layer="97">FTDI 3.3V cable</text>
 <text x="208.28" y="121.92" size="1.778" layer="97">Camera Power</text>
+<wire x1="175.26" y1="91.44" x2="248.92" y2="91.44" width="0.1524" layer="97" style="shortdash"/>
+<wire x1="248.92" y1="91.44" x2="248.92" y2="52.07" width="0.1524" layer="97" style="shortdash"/>
+<wire x1="248.92" y1="52.07" x2="175.26" y2="52.07" width="0.1524" layer="97" style="shortdash"/>
+<wire x1="175.26" y1="52.07" x2="175.26" y2="91.44" width="0.1524" layer="97" style="shortdash"/>
+<text x="194.31" y="54.61" size="1.778" layer="97">GoPro "Start" (not stop!) signal</text>
 </plain>
 <instances>
@@
 <instance part="TP8" gate="G$1" x="158.75" y="114.3" rot="MR0"/>
 <instance part="Q1" gate="G$1" x="238.76" y="116.84" rot="MR0"/>
+<instance part="OK1" gate="G$1" x="210.82" y="73.66" rot="MR0"/>
+<instance part="R13" gate="R" x="233.68" y="76.2" rot="MR180"/>
+<instance part="GND21" gate="1" x="226.06" y="66.04"/>
+<instance part="JP3" gate="G$1" x="182.88" y="72.39" rot="R180"/>
 </instances>
 <busses>
@@
 <wire x1="238.76" y1="104.14" x2="246.38" y2="104.14" width="0.1524" layer="91"/>
 <junction x="238.76" y="104.14"/>
+</segment>
+<segment>
+<pinref part="OK1" gate="G$1" pin="C"/>
+<wire x1="220.98" y1="68.58" x2="226.06" y2="68.58" width="0.1524" layer="91" style="shortdash"/>
+<pinref part="GND21" gate="1" pin="GND"/>
 </segment>
 </net>
@@
 </segment>
 </net>
+<net name="N$20" class="0">
+<segment>
+<pinref part="J1" gate="G$3" pin="GPIO28"/>
+<wire x1="299.72" y1="76.2" x2="238.76" y2="76.2" width="0.1524" layer="91" style="shortdash"/>
+<pinref part="R13" gate="R" pin="2"/>
+</segment>
+</net>
+<net name="N$21" class="0">
+<segment>
+<pinref part="R13" gate="R" pin="1"/>
+<pinref part="OK1" gate="G$1" pin="A"/>
+<wire x1="228.6" y1="76.2" x2="220.98" y2="76.2" width="0.1524" layer="91" style="shortdash"/>
+</segment>
+</net>
+<net name="N$23" class="0">
+<segment>
+<pinref part="OK1" gate="G$1" pin="COL"/>
+<wire x1="203.2" y1="73.66" x2="187.96" y2="73.66" width="0.1524" layer="91" style="shortdash"/>
+<wire x1="187.96" y1="73.66" x2="187.96" y2="72.39" width="0.1524" layer="91" style="shortdash"/>
+<pinref part="JP3" gate="G$1" pin="2"/>
+<wire x1="187.96" y1="72.39" x2="185.42" y2="72.39" width="0.1524" layer="91" style="shortdash"/>
+</segment>
+</net>
+<net name="N$39" class="0">
+<segment>
+<pinref part="OK1" gate="G$1" pin="EMI"/>
+<wire x1="203.2" y1="68.58" x2="187.96" y2="68.58" width="0.1524" layer="91" style="shortdash"/>
+<pinref part="JP3" gate="G$1" pin="1"/>
+<wire x1="185.42" y1="69.85" x2="187.96" y2="69.85" width="0.1524" layer="91" style="shortdash"/>
+<wire x1="187.96" y1="69.85" x2="187.96" y2="68.58" width="0.1524" layer="91" style="shortdash"/>
+</segment>
+</net>
