File: av4/wifi-carrier/wifi-carrier.brd (EAGLE design)
At the start: 100 x 80 mm, 13 parts, among them J1 ROCKETNET-CONNECTOR-16M, U1 UEI15

Commit message: adding caps to wifi carrier
Parts:
- removed X2: (no value), con-wago-500:W237-102
- added C1, C2: 100n, rcl:C0603
- added C3: 1u, rcl:C0805
- added C4: 33u, rcl:C1206
- added X1: 5V, con-phoenix-254:2POL254
- R1, R2: device rcl:R0805 -> rcl:R0603
Connections:
- net GND: now also C1.2, C2.2, C3.2, C4.2, X1.2; no longer X2.2
- net VCC: now also C1.1
- net VOUT: now also C2.1, C3.1, C4.1, X1.1; no longer X2.1
Changed lines of the file:
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@@
 <element name="BOLT3" library="mount-2" package="_4/.325-BARE+SMALL_TOOL_CLEARANCE" value="_4-BARE_MOUNTING_HOLE/.325" x="-45.72" y="92.71"/>
 <element name="U1" library="wifi-carrier" package="UEI15_PIN" value="UEI15" x="-27.94" y="12.7"/>
-<element name="R1" library="rcl" package="R0805" value="NP" x="-53.34" y="91.44"/>
-<element name="R2" library="rcl" package="R0805" value="NP" x="-58.42" y="91.44"/>
+<element name="R1" library="rcl" package="R0603" value="NP" x="-53.34" y="91.44"/>
+<element name="R2" library="rcl" package="R0603" value="NP" x="-58.42" y="91.44"/>
 <element name="CTRL" library="testpad" package="P1-13" value="PTR1PAD1-13" x="-17.78" y="99.06">
 <attribute name="TP_SIGNAL_NAME" value="" x="0" y="0" size="1.778" layer="27" display="off"/>
@@
 <attribute name="TP_SIGNAL_NAME" value="" x="0" y="0" size="1.778" layer="27" display="off"/>
 </element>
-<element name="X2" library="con-wago-500" package="W237-102" value="" x="-39.37" y="54.61">
-<attribute name="OC_NEWARK" value="70K9898" x="0" y="0" size="1.778" layer="27" display="off"/>
-<attribute name="MPN" value="237-102" x="0" y="0" size="1.778" layer="27" display="off"/>
-<attribute name="MF" value="" x="0" y="0" size="1.778" layer="27" display="off"/>
-<attribute name="OC_FARNELL" value="unknown" x="0" y="0" size="1.778" layer="27" display="off"/>
+<element name="C1" library="rcl" package="C0603" value="100n" x="-77.47" y="-2.54"/>
+<element name="C2" library="rcl" package="C0603" value="100n" x="-77.47" y="-6.35"/>
+<element name="C3" library="rcl" package="C0805" value="1u" x="-77.47" y="-12.7"/>
+<element name="C4" library="rcl" package="C1206" value="33u" x="-76.2" y="-19.05"/>
+<element name="X1" library="con-phoenix-254" package="2POL254" value="5V" x="-76.2" y="-26.67">
+<attribute name="OC_NEWARK" value="unknown" x="-76.2" y="-26.67" size="1.778" layer="27" display="off"/>
+<attribute name="MPN" value="" x="-76.2" y="-26.67" size="1.778" layer="27" display="off"/>
+<attribute name="MF" value="" x="-76.2" y="-26.67" size="1.778" layer="27" display="off"/>
+<attribute name="OC_FARNELL" value="unknown" x="-76.2" y="-26.67" size="1.778" layer="27" display="off"/>
 </element>
 </elements>
@@
 <contactref element="R2" pad="1"/>
 <contactref element="U1" pad="5"/>
-<contactref element="X2" pad="2"/>
-<wire x1="-36.87" y1="53.34" x2="-59.37" y2="91.44" width="0" layer="19" extent="1-1"/>
-<wire x1="-27.305" y1="56.515" x2="-36.87" y2="53.34" width="0" layer="19" extent="1-1"/>
+<contactref element="C1" pad="2"/>
+<contactref element="C2" pad="2"/>
+<contactref element="C3" pad="2"/>
+<contactref element="C4" pad="2"/>
+<contactref element="X1" pad="2"/>
+<wire x1="-74.8" y1="-19.05" x2="-74.93" y2="-26.67" width="0" layer="19" extent="1-1"/>
+<wire x1="-76.52" y1="-12.7" x2="-74.8" y2="-19.05" width="0" layer="19" extent="1-1"/>
+<wire x1="-76.62" y1="-6.35" x2="-76.52" y2="-12.7" width="0" layer="19" extent="1-1"/>
+<wire x1="-76.62" y1="-2.54" x2="-76.62" y2="-6.35" width="0" layer="19" extent="1-1"/>
+<wire x1="-38.1" y1="15.24" x2="-76.62" y2="-2.54" width="0" layer="19" extent="1-1"/>
+<wire x1="-17.78" y1="22.86" x2="-38.1" y2="15.24" width="0" layer="19" extent="1-1"/>
+<wire x1="-27.305" y1="56.515" x2="-17.78" y2="22.86" width="0" layer="19" extent="1-1"/>
 <wire x1="-27.305" y1="57.785" x2="-27.305" y2="56.515" width="0" layer="19" extent="1-1"/>
-<wire x1="-17.78" y1="22.86" x2="-27.305" y2="56.515" width="0" layer="19" extent="1-1"/>
-<wire x1="-38.1" y1="15.24" x2="-17.78" y2="22.86" width="0" layer="19" extent="1-1"/>
+<wire x1="-59.27" y1="91.44" x2="-27.305" y2="57.785" width="0" layer="19" extent="1-1"/>
 </signal>
 <signal name="VCC">
 <contactref element="J1" pad="B+@15"/>
 <contactref element="J1" pad="B+@16"/>
+<contactref element="VBATT" pad="TP"/>
 <contactref element="U1" pad="1"/>
-<contactref element="VBATT" pad="TP"/>
+<contactref element="C1" pad="1"/>
+<wire x1="-38.1" y1="10.16" x2="-78.32" y2="-2.54" width="0" layer="19" extent="1-1"/>
+<wire x1="-18.415" y1="56.515" x2="-38.1" y2="10.16" width="0" layer="19" extent="1-1"/>
 <wire x1="-18.415" y1="57.785" x2="-18.415" y2="56.515" width="0" layer="19" extent="1-1"/>
-<wire x1="-38.1" y1="10.16" x2="-18.415" y2="56.515" width="0" layer="19" extent="1-1"/>
 <wire x1="-66.04" y1="90.17" x2="-18.415" y2="57.785" width="0" layer="19" extent="1-1"/>
 </signal>
@@
 <contactref element="R1" pad="1"/>
 <contactref element="U1" pad="4"/>
-<wire x1="-57.47" y1="91.44" x2="-54.29" y2="91.44" width="0" layer="19" extent="1-1"/>
-<wire x1="-17.78" y1="12.7" x2="-54.29" y2="91.44" width="0" layer="19" extent="1-1"/>
+<wire x1="-57.57" y1="91.44" x2="-54.19" y2="91.44" width="0" layer="19" extent="1-1"/>
+<wire x1="-17.78" y1="12.7" x2="-54.19" y2="91.44" width="0" layer="19" extent="1-1"/>
 </signal>
 <signal name="VOUT">
 <contactref element="R1" pad="2"/>
 <contactref element="U1" pad="3"/>
-<contactref element="X2" pad="1"/>
-<wire x1="-41.87" y1="53.34" x2="-52.39" y2="91.44" width="0" layer="19" extent="1-1"/>
-<wire x1="-17.78" y1="2.54" x2="-41.87" y2="53.34" width="0" layer="19" extent="1-1"/>
+<contactref element="C2" pad="1"/>
+<contactref element="C3" pad="1"/>
+<contactref element="C4" pad="1"/>
+<contactref element="X1" pad="1"/>
+<wire x1="-77.6" y1="-19.05" x2="-77.47" y2="-26.67" width="0" layer="19" extent="1-1"/>
+<wire x1="-78.42" y1="-12.7" x2="-77.6" y2="-19.05" width="0" layer="19" extent="1-1"/>
+<wire x1="-78.32" y1="-6.35" x2="-78.42" y2="-12.7" width="0" layer="19" extent="1-1"/>
+<wire x1="-17.78" y1="2.54" x2="-78.32" y2="-6.35" width="0" layer="19" extent="1-1"/>
+<wire x1="-52.49" y1="91.44" x2="-17.78" y2="2.54" width="0" layer="19" extent="1-1"/>
 </signal>
 <signal name="CTRL">

Commit message: New cap for wifi-carrier, added it to its own library file and to the board.
Parts:
- added C5: 100u, cap-3024-7660:7660
Connections:
- net GND: now also C5.-
- net VCC: now also C5.+
Changed lines of the file:
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@@
 <?xml version="1.0" encoding="utf-8"?>
 <!DOCTYPE eagle SYSTEM "eagle.dtd">
-<eagle version="6.4">
+<eagle version="6.5.0">
 <drawing>
 <settings>
@@
 <layers>
 <layer number="1" name="Top" color="4" fill="1" visible="yes" active="yes"/>
+<layer number="2" name="Route2" color="1" fill="3" visible="yes" active="yes"/>
+<layer number="3" name="Route3" color="4" fill="3" visible="yes" active="yes"/>
+<layer number="4" name="Route4" color="1" fill="4" visible="yes" active="yes"/>
+<layer number="5" name="Route5" color="4" fill="4" visible="yes" active="yes"/>
+<layer number="6" name="Route6" color="1" fill="8" visible="yes" active="yes"/>
+<layer number="7" name="Route7" color="4" fill="8" visible="yes" active="yes"/>
+<layer number="8" name="Route8" color="1" fill="2" visible="yes" active="yes"/>
+<layer number="9" name="Route9" color="4" fill="2" visible="yes" active="yes"/>
+<layer number="10" name="Route10" color="1" fill="7" visible="yes" active="yes"/>
+<layer number="11" name="Route11" color="4" fill="7" visible="yes" active="yes"/>
+<layer number="12" name="Route12" color="1" fill="5" visible="yes" active="yes"/>
+<layer number="13" name="Route13" color="4" fill="5" visible="yes" active="yes"/>
+<layer number="14" name="Route14" color="1" fill="6" visible="yes" active="yes"/>
+<layer number="15" name="Route15" color="4" fill="6" visible="yes" active="yes"/>
 <layer number="16" name="Bottom" color="1" fill="1" visible="yes" active="yes"/>
 <layer number="17" name="Pads" color="2" fill="1" visible="yes" active="yes"/>
@@
 <attribute name="OC_FARNELL" value="unknown" x="-76.2" y="-26.67" size="1.778" layer="27" display="off"/>
 </element>
+<element name="C5" library="cap-3024-7660" package="7660" value="100u" x="-76.2" y="-35.56"/>
 </elements>
 <signals>
@@
 <contactref element="C4" pad="2"/>
 <contactref element="X1" pad="2"/>
+<contactref element="C5" pad="-"/>
+<wire x1="-74.93" y1="-26.67" x2="-76.2" y2="-38.51" width="0" layer="19" extent="1-1"/>
 <wire x1="-74.8" y1="-19.05" x2="-74.93" y2="-26.67" width="0" layer="19" extent="1-1"/>
 <wire x1="-76.52" y1="-12.7" x2="-74.8" y2="-19.05" width="0" layer="19" extent="1-1"/>
@@
 <contactref element="U1" pad="1"/>
 <contactref element="C1" pad="1"/>
+<contactref element="C5" pad="+"/>
+<wire x1="-78.32" y1="-2.54" x2="-76.2" y2="-32.61" width="0" layer="19" extent="1-1"/>
 <wire x1="-38.1" y1="10.16" x2="-78.32" y2="-2.54" width="0" layer="19" extent="1-1"/>
 <wire x1="-18.415" y1="56.515" x2="-38.1" y2="10.16" width="0" layer="19" extent="1-1"/>

Commit message: first shot at wifi carrier board
Parts:
- moved X1 157.5 mm to (52.1, 64.8), turned to 180 degrees
- moved C4 151.4 mm to (64.0, 38.1)
- moved C3 151.1 mm to (63.5, 41.7)
- moved C2 150.1 mm to (63.5, 45.2)
- moved R2 124.9 mm to (59.7, 50.8), turned to 90 degrees
- moved C5 122.4 mm to (20.3, 39.8)
- moved BOLT 119.5 mm to (56.6, 4.32)
- moved R1 118.9 mm to (59.7, 54.6), turned to 90 degrees
- moved BOLT2 111.7 mm to (64.3, 64.3)
- moved C1 102.1 mm to (14.5, 41.9), turned to 270 degrees
- moved VUSB 93.5 mm to (3.56, 35.6)
- moved BOLT1 91.2 mm to (11.9, 4.32)
- moved VBATT 89.1 mm to (14.5, 52.1)
- moved UWIFI 83.2 mm to (36.8, 20.3)
- moved U1 78.2 mm to (43.2, 45.2)
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Routing:
- net USB+: track 0.00 -> 57.8 mm
- net D+: track 0.00 -> 56.2 mm
- net D-: track 0.00 -> 55.4 mm, vias 0 -> 1
- net USB-: track 0.00 -> 51.4 mm
- net VOUT: track 0.00 -> 44.4 mm
- net VCC: track 0.00 -> 41.7 mm
- net TRIM: track 0.00 -> 13.2 mm
- net CTRL: track 0.00 -> 12.7 mm
- added copper zone on layer 1, net GND
- added copper zone on layer 16, net GND
Other:
- board size 100 x 80 mm -> 68.6 x 68.6 mm

Commit message: wifi board outline to avoid bolts
Parts:
- moved BOLT3 2.84 mm to (6.86, 63.0)
- moved BOLT2 2.84 mm to (61.7, 63.0)
- moved BOLT 2.54 mm to (54.1, 4.32)
- moved BOLT1 2.54 mm to (14.5, 4.32)
- moved X1 1.27 mm to (52.1, 63.5)
Routing:
- net VOUT: track 44.4 -> 42.4 mm
Other:
- board size 68.6 x 68.6 mm -> 68.6 x 67.3 mm
Changed lines of the file:
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@@
 <setting verticaltext="up"/>
 </settings>
-<grid distance="0.1" unitdist="inch" unit="inch" style="lines" multiple="1" display="yes" altdistance="0.025" altunitdist="inch" altunit="inch"/>
+<grid distance="0.05" unitdist="inch" unit="inch" style="lines" multiple="1" display="yes" altdistance="0.025" altunitdist="inch" altunit="inch"/>
 <layers>
 <layer number="1" name="Top" color="4" fill="1" visible="yes" active="yes"/>
@@
 <board>
 <plain>
-<wire x1="0" y1="0" x2="68.58" y2="0" width="0" layer="20"/>
-<wire x1="68.58" y1="0" x2="68.58" y2="68.58" width="0" layer="20"/>
-<wire x1="68.58" y1="68.58" x2="0" y2="68.58" width="0" layer="20"/>
-<wire x1="0" y1="68.58" x2="0" y2="0" width="0" layer="20"/>
+<wire x1="7.62" y1="0" x2="60.96" y2="0" width="0" layer="20"/>
+<wire x1="60.96" y1="0" x2="60.96" y2="7.62" width="0" layer="20"/>
+<wire x1="60.96" y1="7.62" x2="68.58" y2="7.62" width="0" layer="20"/>
+<wire x1="68.58" y1="7.62" x2="68.58" y2="58.42" width="0" layer="20"/>
+<wire x1="68.58" y1="58.42" x2="66.04" y2="58.42" width="0" layer="20"/>
+<wire x1="66.04" y1="58.42" x2="66.04" y2="67.31" width="0" layer="20"/>
+<wire x1="66.04" y1="67.31" x2="2.54" y2="67.31" width="0" layer="20"/>
+<wire x1="2.54" y1="67.31" x2="2.54" y2="55.88" width="0" layer="20"/>
+<wire x1="2.54" y1="55.88" x2="0" y2="55.88" width="0" layer="20"/>
+<wire x1="0" y1="55.88" x2="0" y2="7.62" width="0" layer="20"/>
+<wire x1="0" y1="7.62" x2="7.62" y2="7.62" width="0" layer="20"/>
+<wire x1="7.62" y1="7.62" x2="7.62" y2="0" width="0" layer="20"/>
 </plain>
 <attributes>
@@
 <element name="UWIFI" library="wifi-carrier" package="ZCN-722M" value="ZCN-722M" x="36.83" y="20.32"/>
 <element name="J1" library="rocketnet-connector" package="ROCKETNET-M-16" value="ROCKETNET-CONNECTOR-16M" x="22.86" y="63.5" rot="R180"/>
-<element name="BOLT" library="mount-2" package="_4/.325-BARE+SMALL_TOOL_CLEARANCE" value="_4-BARE_MOUNTING_HOLE/.325" x="56.642" y="4.318" smashed="yes"/>
-<element name="BOLT1" library="mount-2" package="_4/.325-BARE+SMALL_TOOL_CLEARANCE" value="_4-BARE_MOUNTING_HOLE/.325" x="11.938" y="4.318" smashed="yes"/>
-<element name="BOLT2" library="mount-2" package="_4/.325-BARE+SMALL_TOOL_CLEARANCE" value="_4-BARE_MOUNTING_HOLE/.325" x="64.262" y="64.262" smashed="yes"/>
-<element name="BOLT3" library="mount-2" package="_4/.325-BARE+SMALL_TOOL_CLEARANCE" value="_4-BARE_MOUNTING_HOLE/.325" x="4.318" y="64.262" smashed="yes"/>
+<element name="BOLT" library="mount-2" package="_4/.325-BARE+SMALL_TOOL_CLEARANCE" value="_4-BARE_MOUNTING_HOLE/.325" x="54.102" y="4.318" smashed="yes"/>
+<element name="BOLT1" library="mount-2" package="_4/.325-BARE+SMALL_TOOL_CLEARANCE" value="_4-BARE_MOUNTING_HOLE/.325" x="14.478" y="4.318" smashed="yes"/>
+<element name="BOLT2" library="mount-2" package="_4/.325-BARE+SMALL_TOOL_CLEARANCE" value="_4-BARE_MOUNTING_HOLE/.325" x="61.722" y="62.992" smashed="yes"/>
+<element name="BOLT3" library="mount-2" package="_4/.325-BARE+SMALL_TOOL_CLEARANCE" value="_4-BARE_MOUNTING_HOLE/.325" x="6.858" y="62.992" smashed="yes"/>
 <element name="U1" library="wifi-carrier" package="UEI15_PIN" value="UEI15" x="43.18" y="45.212"/>
 <element name="R1" library="rcl" package="R0603" value="NP" x="59.69" y="54.61" rot="R90"/>
@@
 <element name="C3" library="rcl" package="C0805" value="1u" x="63.5" y="41.656"/>
 <element name="C4" library="rcl" package="C1206" value="33u" x="64.008" y="38.1"/>
-<element name="X1" library="con-phoenix-254" package="2POL254" value="5V" x="52.07" y="64.77" rot="R180">
-<attribute name="OC_NEWARK" value="unknown" x="52.07" y="64.77" size="1.778" layer="27" rot="R180" display="off"/>
-<attribute name="MPN" value="" x="52.07" y="64.77" size="1.778" layer="27" rot="R180" display="off"/>
-<attribute name="MF" value="" x="52.07" y="64.77" size="1.778" layer="27" rot="R180" display="off"/>
-<attribute name="OC_FARNELL" value="unknown" x="52.07" y="64.77" size="1.778" layer="27" rot="R180" display="off"/>
+<element name="X1" library="con-phoenix-254" package="2POL254" value="5V" x="52.07" y="63.5" rot="R180">
+<attribute name="OC_NEWARK" value="unknown" x="52.07" y="63.5" size="1.778" layer="27" rot="R180" display="off"/>
+<attribute name="MPN" value="" x="52.07" y="63.5" size="1.778" layer="27" rot="R180" display="off"/>
+<attribute name="MF" value="" x="52.07" y="63.5" size="1.778" layer="27" rot="R180" display="off"/>
+<attribute name="OC_FARNELL" value="unknown" x="52.07" y="63.5" size="1.778" layer="27" rot="R180" display="off"/>
 </element>
 <element name="C5" library="cap-3024-7660" package="7660" value="100u" x="20.32" y="39.751"/>
@@
 <wire x1="61.468" y1="55.372" x2="59.778" y2="55.372" width="1.016" layer="1"/>
 <wire x1="59.778" y1="55.372" x2="59.69" y2="55.46" width="1.016" layer="1"/>
-<wire x1="59.69" y1="55.46" x2="59.69" y2="58.166" width="1.016" layer="1"/>
-<wire x1="59.69" y1="58.166" x2="57.15" y2="60.706" width="1.016" layer="1"/>
-<wire x1="57.15" y1="60.706" x2="54.864" y2="60.706" width="1.016" layer="1"/>
+<wire x1="59.69" y1="55.46" x2="59.69" y2="56.896" width="1.016" layer="1"/>
+<wire x1="59.69" y1="56.896" x2="55.88" y2="60.706" width="1.016" layer="1"/>
+<wire x1="55.88" y1="60.706" x2="54.864" y2="60.706" width="1.016" layer="1"/>
 <wire x1="54.864" y1="60.706" x2="53.34" y2="62.23" width="1.016" layer="1"/>
-<wire x1="53.34" y1="62.23" x2="53.34" y2="64.77" width="1.016" layer="1"/>
+<wire x1="53.34" y1="62.23" x2="53.34" y2="63.5" width="1.016" layer="1"/>
 </signal>
 <signal name="CTRL">

Commit message: rearrange caps and minor bolt adjustment on wifi carrier
Parts:
- moved C2 10.9 mm to (59.4, 35.1)
- moved VUSB 10.8 mm to (14.0, 38.4)
- moved VBATT 7.41 mm to (20.8, 48.3)
- moved C1 6.35 mm to (20.8, 41.9)
- moved C3 5.57 mm to (59.7, 37.6)
- moved C5 5.08 mm to (25.4, 39.8)
- moved C4 4.44 mm to (60.2, 40.4)
- moved BOLT 2.54 mm to (56.6, 4.32)
- moved BOLT1 2.54 mm to (11.9, 4.32)
- moved J1 1.02 mm to (22.9, 62.5)
Routing:
- net D-: track 55.4 -> 73.0 mm, vias 1 -> 0
- net VCC: track 41.7 -> 35.7 mm
- net USB+: track 57.8 -> 52.1 mm
- net D+: track 56.2 -> 59.2 mm
- net VOUT: track 42.4 -> 41.0 mm
- net USB-: track 51.4 -> 50.4 mm
Other:
- outline, holes or cut-outs redrawn
