File: av4/wifi-carrier/wifi-carrier.sch (EAGLE design)
At the start: 1 part

Commit message: repurposed rocketnet hub connector as USB
Parts:
- added BOLT, BOLT1, BOLT2, BOLT3: _4-BARE_MOUNTING_HOLE/.325, mount-2:_4-BARE_MOUNTING_HOLE/.325
- added J1: ROCKETNET-CONNECTOR-16M, rocketnet-connector:ROCKETNET-CONNECTOR-16M
Connections:
- new net D+: J1.TX+@1, J1.TX+@2, UWIFI.D+
- new net D-: J1.TX-@1, J1.TX-@2, UWIFI.D-
- new net GND: J1.B-@1, J1.B-@2
- new net USB+: J1.RX+@1, J1.RX+@2, UWIFI.VCC
- new net USB-: J1.RX-@1, J1.RX-@2, UWIFI.GND
Other:
- moved on the sheet: UWIFI
Changed lines of the file:
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@@
 <layer number="48" name="Document" color="7" fill="1" visible="no" active="no"/>
 <layer number="49" name="Reference" color="7" fill="1" visible="no" active="no"/>
+<layer number="50" name="dxf" color="7" fill="1" visible="no" active="no"/>
 <layer number="51" name="tDocu" color="7" fill="1" visible="no" active="no"/>
 <layer number="52" name="bDocu" color="7" fill="1" visible="no" active="no"/>
+<layer number="53" name="tGND_GNDA" color="7" fill="1" visible="no" active="no"/>
+<layer number="54" name="bGND_GNDA" color="7" fill="1" visible="no" active="no"/>
+<layer number="56" name="wert" color="7" fill="1" visible="no" active="no"/>
 <layer number="91" name="Nets" color="2" fill="1" visible="yes" active="yes"/>
 <layer number="92" name="Busses" color="1" fill="1" visible="yes" active="yes"/>
@@
 <layer number="97" name="Info" color="7" fill="1" visible="yes" active="yes"/>
 <layer number="98" name="Guide" color="6" fill="1" visible="yes" active="yes"/>
+<layer number="100" name="Hidden_Layer" color="7" fill="1" visible="yes" active="yes"/>
+<layer number="101" name="Patch_Top" color="7" fill="1" visible="yes" active="yes"/>
+<layer number="102" name="Vscore" color="7" fill="1" visible="yes" active="yes"/>
+<layer number="103" name="tMap" color="7" fill="1" visible="yes" active="yes"/>
+<layer number="104" name="Name" color="7" fill="1" visible="yes" active="yes"/>
+<layer number="105" name="tPlate" color="7" fill="1" visible="yes" active="yes"/>
+<layer number="106" name="bPlate" color="7" fill="1" visible="yes" active="yes"/>
+<layer number="107" name="Crop" color="7" fill="1" visible="yes" active="yes"/>
+<layer number="116" name="Patch_BOT" color="7" fill="1" visible="yes" active="yes"/>
+<layer number="121" name="_tsilk" color="7" fill="1" visible="yes" active="yes"/>
+<layer number="122" name="_bsilk" color="7" fill="1" visible="yes" active="yes"/>
+<layer number="151" name="HeatSink" color="7" fill="1" visible="yes" active="yes"/>
+<layer number="200" name="200bmp" color="7" fill="1" visible="yes" active="yes"/>
+<layer number="201" name="201bmp" color="7" fill="1" visible="yes" active="yes"/>
+<layer number="202" name="202bmp" color="7" fill="1" visible="yes" active="yes"/>
+<layer number="203" name="203bmp" color="7" fill="1" visible="yes" active="yes"/>
+<layer number="204" name="204bmp" color="7" fill="1" visible="yes" active="yes"/>
+<layer number="205" name="205bmp" color="7" fill="1" visible="yes" active="yes"/>
+<layer number="206" name="206bmp" color="7" fill="1" visible="yes" active="yes"/>
+<layer number="207" name="207bmp" color="7" fill="1" visible="yes" active="yes"/>
+<layer number="208" name="208bmp" color="7" fill="1" visible="yes" active="yes"/>
+<layer number="215" name="ResistanceBottom" color="7" fill="1" visible="yes" active="yes"/>
+<layer number="250" name="Descript" color="7" fill="1" visible="yes" active="yes"/>
+<layer number="251" name="SMDround" color="7" fill="1" visible="yes" active="yes"/>
+<layer number="254" name="cooling" color="7" fill="1" visible="yes" active="yes"/>
 </layers>
 <schematic xreflabel="%F%N/%S.%C%R" xrefpart="/%S.%C%R">
@@
 <parts>
 <part name="UWIFI" library="wifi-carrier" deviceset="ZCN-722M" device=""/>
+<part name="J1" library="rocketnet-connector" deviceset="ROCKETNET-CONNECTOR-16" device="M"/>
+<part name="SUPPLY1" library="supply2" deviceset="GND" device=""/>
+<part name="BOLT" library="mount-2" deviceset="_4-BARE_MOUNTING_HOLE" device="/.325"/>
+<part name="BOLT1" library="mount-2" deviceset="_4-BARE_MOUNTING_HOLE" device="/.325"/>
+<part name="BOLT2" library="mount-2" deviceset="_4-BARE_MOUNTING_HOLE" device="/.325"/>
+<part name="BOLT3" library="mount-2" deviceset="_4-BARE_MOUNTING_HOLE" device="/.325"/>
 </parts>
 <sheets>
@@
 </plain>
 <instances>
-<instance part="UWIFI" gate="G$1" x="30.48" y="22.86"/>
+<instance part="UWIFI" gate="G$1" x="127" y="68.58"/>
+<instance part="J1" gate="G$1" x="25.4" y="66.04"/>
+<instance part="SUPPLY1" gate="GND" x="30.48" y="30.48"/>
+<instance part="BOLT" gate="MT" x="137.16" y="48.26"/>
+<instance part="BOLT1" gate="MT" x="137.16" y="40.64"/>
+<instance part="BOLT2" gate="MT" x="137.16" y="33.02"/>
+<instance part="BOLT3" gate="MT" x="137.16" y="25.4"/>
 </instances>
 <busses>
+<bus name="USB-,USB+,D+,D-">
+<segment>
+<wire x1="45.72" y1="73.66" x2="45.72" y2="58.42" width="0.762" layer="92"/>
+<wire x1="45.72" y1="58.42" x2="48.26" y2="55.88" width="0.762" layer="92"/>
+<wire x1="48.26" y1="55.88" x2="111.76" y2="55.88" width="0.762" layer="92"/>
+<wire x1="111.76" y1="55.88" x2="114.3" y2="58.42" width="0.762" layer="92"/>
+<wire x1="114.3" y1="58.42" x2="114.3" y2="68.58" width="0.762" layer="92"/>
+</segment>
+</bus>
 </busses>
 <nets>
+<net name="D+" class="0">
+<segment>
+<pinref part="J1" gate="G$1" pin="TX+@1"/>
+<pinref part="J1" gate="G$1" pin="TX+@2"/>
+<wire x1="30.48" y1="78.74" x2="30.48" y2="76.2" width="0.1524" layer="91"/>
+<wire x1="43.18" y1="76.2" x2="30.48" y2="76.2" width="0.1524" layer="91"/>
+<junction x="30.48" y="76.2"/>
+<wire x1="43.18" y1="76.2" x2="45.72" y2="73.66" width="0.1524" layer="91"/>
+<label x="33.02" y="76.2" size="1.778" layer="95"/>
+</segment>
+<segment>
+<wire x1="114.3" y1="63.5" x2="116.84" y2="66.04" width="0.1524" layer="91"/>
+<pinref part="UWIFI" gate="G$1" pin="D+"/>
+<wire x1="116.84" y1="66.04" x2="119.38" y2="66.04" width="0.1524" layer="91"/>
+</segment>
+</net>
+<net name="D-" class="0">
+<segment>
+<wire x1="45.72" y1="68.58" x2="43.18" y2="71.12" width="0.1524" layer="91"/>
+<pinref part="J1" gate="G$1" pin="TX-@2"/>
+<wire x1="43.18" y1="71.12" x2="30.48" y2="71.12" width="0.1524" layer="91"/>
+<pinref part="J1" gate="G$1" pin="TX-@1"/>
+<wire x1="30.48" y1="71.12" x2="30.48" y2="73.66" width="0.1524" layer="91"/>
+<junction x="30.48" y="71.12"/>
+<label x="33.02" y="71.12" size="1.778" layer="95"/>
+</segment>
+<segment>
+<wire x1="114.3" y1="66.04" x2="116.84" y2="68.58" width="0.1524" layer="91"/>
+<pinref part="UWIFI" gate="G$1" pin="D-"/>
+<wire x1="116.84" y1="68.58" x2="119.38" y2="68.58" width="0.1524" layer="91"/>
+</segment>
+</net>
+<net name="USB+" class="0">
+<segment>
+<wire x1="45.72" y1="63.5" x2="43.18" y2="66.04" width="0.1524" layer="91"/>
+<pinref part="J1" gate="G$1" pin="RX+@2"/>
+<wire x1="43.18" y1="66.04" x2="30.48" y2="66.04" width="0.1524" layer="91"/>
+<pinref part="J1" gate="G$1" pin="RX+@1"/>
+<wire x1="30.48" y1="66.04" x2="30.48" y2="68.58" width="0.1524" layer="91"/>
+<junction x="30.48" y="66.04"/>
+<label x="33.02" y="66.04" size="1.778" layer="95"/>
+</segment>
+<segment>
+<wire x1="114.3" y1="68.58" x2="116.84" y2="71.12" width="0.1524" layer="91"/>
+<pinref part="UWIFI" gate="G$1" pin="VCC"/>
+<wire x1="116.84" y1="71.12" x2="119.38" y2="71.12" width="0.1524" layer="91"/>
+</segment>
+</net>
+<net name="USB-" class="0">
+<segment>
+<wire x1="45.72" y1="58.42" x2="43.18" y2="60.96" width="0.1524" layer="91"/>
+<pinref part="J1" gate="G$1" pin="RX-@2"/>
+<wire x1="43.18" y1="60.96" x2="30.48" y2="60.96" width="0.1524" layer="91"/>
+<pinref part="J1" gate="G$1" pin="RX-@1"/>
+<wire x1="30.48" y1="60.96" x2="30.48" y2="63.5" width="0.1524" layer="91"/>
+<junction x="30.48" y="60.96"/>
+<label x="33.02" y="60.96" size="1.778" layer="95"/>
+</segment>
+<segment>
+<wire x1="114.3" y1="60.96" x2="116.84" y2="63.5" width="0.1524" layer="91"/>
+<pinref part="UWIFI" gate="G$1" pin="GND"/>
+<wire x1="116.84" y1="63.5" x2="119.38" y2="63.5" width="0.1524" layer="91"/>
+</segment>
+</net>
+<net name="GND" class="0">
+<segment>
+<pinref part="J1" gate="G$1" pin="B-@1"/>
+<pinref part="J1" gate="G$1" pin="B-@2"/>
+<wire x1="30.48" y1="48.26" x2="30.48" y2="45.72" width="0.1524" layer="91"/>
+<pinref part="SUPPLY1" gate="GND" pin="GND"/>
+<wire x1="30.48" y1="45.72" x2="30.48" y2="33.02" width="0.1524" layer="91"/>
+<junction x="30.48" y="45.72"/>
+</segment>
+</net>
 </nets>
 </sheet>

Commit message: switcher layout
Parts:
- added CTRL, VBATT, VUSB: PTR1PAD1-13, testpad:PTR1PAD1-13
- added R1, R2: NP, rcl:R-US_R0805
- added U1: UEI15, wifi-carrier:UEI15
Connections:
- new net CTRL: CTRL.TP, U1.CTRL
- new net TRIM: R1.1, R2.2, U1.TRIM
- new net VCC: J1.B+@1, J1.B+@2, U1.VIN, VBATT.TP
- new net VOUT: R1.2, U1.VOUT
- net GND: now also R2.1, U1.INGND, U1.OUTGND
- net USB+: now also VUSB.TP
Other:
- moved on the sheet: BOLT, BOLT1, BOLT2, BOLT3, UWIFI
Changed lines of the file:
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@@
 <part name="BOLT2" library="mount-2" deviceset="_4-BARE_MOUNTING_HOLE" device="/.325"/>
 <part name="BOLT3" library="mount-2" deviceset="_4-BARE_MOUNTING_HOLE" device="/.325"/>
+<part name="U1" library="wifi-carrier" deviceset="UEI15" device=""/>
+<part name="P+1" library="supply1" deviceset="VCC" device=""/>
+<part name="R1" library="rcl" deviceset="R-US_" device="R0805" value="NP"/>
+<part name="R2" library="rcl" deviceset="R-US_" device="R0805" value="NP"/>
+<part name="SUPPLY2" library="supply2" deviceset="GND" device=""/>
+<part name="SUPPLY3" library="supply2" deviceset="GND" device=""/>
+<part name="SUPPLY4" library="supply2" deviceset="GND" device=""/>
+<part name="CTRL" library="testpad" deviceset="PTR1" device="PAD1-13"/>
+<part name="VBATT" library="testpad" deviceset="PTR1" device="PAD1-13"/>
+<part name="VUSB" library="testpad" deviceset="PTR1" device="PAD1-13"/>
 </parts>
 <sheets>
@@
 </plain>
 <instances>
-<instance part="UWIFI" gate="G$1" x="127" y="68.58"/>
+<instance part="UWIFI" gate="G$1" x="88.9" y="63.5"/>
 <instance part="J1" gate="G$1" x="25.4" y="66.04"/>
 <instance part="SUPPLY1" gate="GND" x="30.48" y="30.48"/>
-<instance part="BOLT" gate="MT" x="137.16" y="48.26"/>
-<instance part="BOLT1" gate="MT" x="137.16" y="40.64"/>
-<instance part="BOLT2" gate="MT" x="137.16" y="33.02"/>
-<instance part="BOLT3" gate="MT" x="137.16" y="25.4"/>
+<instance part="BOLT" gate="MT" x="144.78" y="68.58"/>
+<instance part="BOLT1" gate="MT" x="144.78" y="60.96"/>
+<instance part="BOLT2" gate="MT" x="144.78" y="53.34"/>
+<instance part="BOLT3" gate="MT" x="144.78" y="45.72"/>
+<instance part="U1" gate="G$1" x="88.9" y="109.22"/>
+<instance part="P+1" gate="VCC" x="30.48" y="127"/>
+<instance part="R1" gate="G$1" x="119.38" y="109.22" rot="R90"/>
+<instance part="R2" gate="G$1" x="119.38" y="99.06" rot="R90"/>
+<instance part="SUPPLY2" gate="GND" x="55.88" y="86.36"/>
+<instance part="SUPPLY3" gate="GND" x="119.38" y="86.36"/>
+<instance part="SUPPLY4" gate="GND" x="109.22" y="86.36"/>
+<instance part="CTRL" gate="G$1" x="71.12" y="99.06"/>
+<instance part="VBATT" gate="G$1" x="43.18" y="109.22"/>
+<instance part="VUSB" gate="G$1" x="66.04" y="45.72"/>
 </instances>
 <busses>
 <bus name="USB-,USB+,D+,D-">
 <segment>
-<wire x1="45.72" y1="73.66" x2="45.72" y2="58.42" width="0.762" layer="92"/>
-<wire x1="45.72" y1="58.42" x2="48.26" y2="55.88" width="0.762" layer="92"/>
-<wire x1="48.26" y1="55.88" x2="111.76" y2="55.88" width="0.762" layer="92"/>
-<wire x1="111.76" y1="55.88" x2="114.3" y2="58.42" width="0.762" layer="92"/>
-<wire x1="114.3" y1="58.42" x2="114.3" y2="68.58" width="0.762" layer="92"/>
+<wire x1="45.72" y1="73.66" x2="45.72" y2="53.34" width="0.762" layer="92"/>
+<wire x1="45.72" y1="53.34" x2="48.26" y2="50.8" width="0.762" layer="92"/>
+<wire x1="48.26" y1="50.8" x2="73.66" y2="50.8" width="0.762" layer="92"/>
+<wire x1="73.66" y1="50.8" x2="76.2" y2="53.34" width="0.762" layer="92"/>
+<wire x1="76.2" y1="53.34" x2="76.2" y2="63.5" width="0.762" layer="92"/>
 </segment>
 </bus>
@@
 </segment>
 <segment>
-<wire x1="114.3" y1="63.5" x2="116.84" y2="66.04" width="0.1524" layer="91"/>
+<wire x1="76.2" y1="58.42" x2="78.74" y2="60.96" width="0.1524" layer="91"/>
 <pinref part="UWIFI" gate="G$1" pin="D+"/>
-<wire x1="116.84" y1="66.04" x2="119.38" y2="66.04" width="0.1524" layer="91"/>
+<wire x1="78.74" y1="60.96" x2="81.28" y2="60.96" width="0.1524" layer="91"/>
 </segment>
 </net>
@@
 </segment>
 <segment>
-<wire x1="114.3" y1="66.04" x2="116.84" y2="68.58" width="0.1524" layer="91"/>
+<wire x1="76.2" y1="60.96" x2="78.74" y2="63.5" width="0.1524" layer="91"/>
 <pinref part="UWIFI" gate="G$1" pin="D-"/>
-<wire x1="116.84" y1="68.58" x2="119.38" y2="68.58" width="0.1524" layer="91"/>
+<wire x1="78.74" y1="63.5" x2="81.28" y2="63.5" width="0.1524" layer="91"/>
 </segment>
 </net>
@@
 </segment>
 <segment>
-<wire x1="114.3" y1="68.58" x2="116.84" y2="71.12" width="0.1524" layer="91"/>
+<wire x1="76.2" y1="63.5" x2="78.74" y2="66.04" width="0.1524" layer="91"/>
 <pinref part="UWIFI" gate="G$1" pin="VCC"/>
-<wire x1="116.84" y1="71.12" x2="119.38" y2="71.12" width="0.1524" layer="91"/>
+<wire x1="78.74" y1="66.04" x2="81.28" y2="66.04" width="0.1524" layer="91"/>
+</segment>
+<segment>
+<pinref part="VUSB" gate="G$1" pin="TP"/>
+<wire x1="63.5" y1="50.8" x2="66.04" y2="48.26" width="0.1524" layer="91"/>
 </segment>
 </net>
@@
 </segment>
 <segment>
-<wire x1="114.3" y1="60.96" x2="116.84" y2="63.5" width="0.1524" layer="91"/>
+<wire x1="76.2" y1="55.88" x2="78.74" y2="58.42" width="0.1524" layer="91"/>
 <pinref part="UWIFI" gate="G$1" pin="GND"/>
-<wire x1="116.84" y1="63.5" x2="119.38" y2="63.5" width="0.1524" layer="91"/>
+<wire x1="78.74" y1="58.42" x2="81.28" y2="58.42" width="0.1524" layer="91"/>
 </segment>
 </net>
@@
 <junction x="30.48" y="45.72"/>
 </segment>
+<segment>
+<pinref part="U1" gate="G$1" pin="INGND"/>
+<pinref part="SUPPLY2" gate="GND" pin="GND"/>
+<wire x1="71.12" y1="109.22" x2="55.88" y2="109.22" width="0.1524" layer="91"/>
+<wire x1="55.88" y1="109.22" x2="55.88" y2="88.9" width="0.1524" layer="91"/>
+</segment>
+<segment>
+<pinref part="R2" gate="G$1" pin="1"/>
+<pinref part="SUPPLY3" gate="GND" pin="GND"/>
+<wire x1="119.38" y1="88.9" x2="119.38" y2="93.98" width="0.1524" layer="91"/>
+</segment>
+<segment>
+<pinref part="U1" gate="G$1" pin="OUTGND"/>
+<pinref part="SUPPLY4" gate="GND" pin="GND"/>
+<wire x1="106.68" y1="109.22" x2="109.22" y2="109.22" width="0.1524" layer="91"/>
+<wire x1="109.22" y1="109.22" x2="109.22" y2="88.9" width="0.1524" layer="91"/>
+</segment>
 </net>
+<net name="VCC" class="0">
+<segment>
+<pinref part="P+1" gate="VCC" pin="VCC"/>
+<pinref part="J1" gate="G$1" pin="B+@1"/>
+<wire x1="30.48" y1="124.46" x2="30.48" y2="111.76" width="0.1524" layer="91"/>
+<pinref part="J1" gate="G$1" pin="B+@2"/>
+<wire x1="30.48" y1="111.76" x2="30.48" y2="83.82" width="0.1524" layer="91"/>
+<wire x1="30.48" y1="83.82" x2="30.48" y2="81.28" width="0.1524" layer="91"/>
+<junction x="30.48" y="83.82"/>
+<pinref part="U1" gate="G$1" pin="VIN"/>
+<junction x="30.48" y="111.76"/>
+<wire x1="71.12" y1="111.76" x2="43.18" y2="111.76" width="0.1524" layer="91"/>
+<pinref part="VBATT" gate="G$1" pin="TP"/>
+<wire x1="43.18" y1="111.76" x2="30.48" y2="111.76" width="0.1524" layer="91"/>
+<junction x="43.18" y="111.76"/>
+</segment>
+</net>
+<net name="TRIM" class="0">
+<segment>
+<pinref part="R2" gate="G$1" pin="2"/>
+<pinref part="R1" gate="G$1" pin="1"/>
+<pinref part="U1" gate="G$1" pin="TRIM"/>
+<wire x1="119.38" y1="104.14" x2="106.68" y2="104.14" width="0.1524" layer="91"/>
+<junction x="119.38" y="104.14"/>
+</segment>
+</net>
+<net name="VOUT" class="0">
+<segment>
+<pinref part="R1" gate="G$1" pin="2"/>
+<pinref part="U1" gate="G$1" pin="VOUT"/>
+<wire x1="106.68" y1="114.3" x2="119.38" y2="114.3" width="0.1524" layer="91"/>
+</segment>
+</net>
+<net name="CTRL" class="0">
+<segment>
+<pinref part="U1" gate="G$1" pin="CTRL"/>
+<pinref part="CTRL" gate="G$1" pin="TP"/>
+<wire x1="71.12" y1="101.6" x2="71.12" y2="104.14" width="0.1524" layer="91"/>
+</segment>
+</net>

Commit message: screw terminal vout
Parts:
- added X2: (no value), con-wago-500:W237-102
Connections:
- net GND: now also X2-2.KL
- net VOUT: now also X2-1.KL
Other:
- note added: "TO PA"
- moved on the sheet: BOLT, BOLT1, BOLT2, BOLT3, CTRL, J1, R1, R2, U1, UWIFI, VBATT, VUSB

Commit message: change usb binout on wificarrer
Connections:
- net D+: now also J1.TX-@1, J1.TX-@2; no longer J1.TX+@1, J1.TX+@2
- net D-: now also J1.RX+@1, J1.RX+@2; no longer J1.TX-@1, J1.TX-@2
- net USB+: now also J1.TX+@1, J1.TX+@2; no longer J1.RX+@1, J1.RX+@2
Changed lines of the file:
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@@
 <net name="D+" class="0">
-<segment>
-<pinref part="J1" gate="G$1" pin="TX+@1"/>
-<pinref part="J1" gate="G$1" pin="TX+@2"/>
-<wire x1="58.42" y1="106.68" x2="58.42" y2="104.14" width="0.1524" layer="91"/>
-<wire x1="71.12" y1="104.14" x2="58.42" y2="104.14" width="0.1524" layer="91"/>
-<junction x="58.42" y="104.14"/>
-<wire x1="71.12" y1="104.14" x2="73.66" y2="101.6" width="0.1524" layer="91"/>
-<label x="60.96" y="104.14" size="1.778" layer="95"/>
-</segment>
 <segment>
 <wire x1="124.46" y1="86.36" x2="127" y2="88.9" width="0.1524" layer="91"/>
@@
 <wire x1="127" y1="88.9" x2="129.54" y2="88.9" width="0.1524" layer="91"/>
 </segment>
-</net>
-<net name="D-" class="0">
 <segment>
 <wire x1="73.66" y1="96.52" x2="71.12" y2="99.06" width="0.1524" layer="91"/>
@@
 <label x="60.96" y="99.06" size="1.778" layer="95"/>
 </segment>
+</net>
+<net name="D-" class="0">
 <segment>
 <wire x1="124.46" y1="88.9" x2="127" y2="91.44" width="0.1524" layer="91"/>
@@
 <wire x1="127" y1="91.44" x2="129.54" y2="91.44" width="0.1524" layer="91"/>
 </segment>
-</net>
-<net name="USB+" class="0">
 <segment>
 <wire x1="73.66" y1="91.44" x2="71.12" y2="93.98" width="0.1524" layer="91"/>
@@
 <wire x1="71.12" y1="93.98" x2="58.42" y2="93.98" width="0.1524" layer="91"/>
 <pinref part="J1" gate="G$1" pin="RX+@1"/>
-<wire x1="58.42" y1="93.98" x2="58.42" y2="96.52" width="0.1524" layer="91"/>
+<wire x1="58.42" y1="96.52" x2="58.42" y2="93.98" width="0.1524" layer="91"/>
 <junction x="58.42" y="93.98"/>
 <label x="60.96" y="93.98" size="1.778" layer="95"/>
 </segment>
+</net>
+<net name="USB+" class="0">
 <segment>
 <wire x1="124.46" y1="91.44" x2="127" y2="93.98" width="0.1524" layer="91"/>
@@
 <wire x1="111.76" y1="78.74" x2="114.3" y2="76.2" width="0.1524" layer="91"/>
 </segment>
+<segment>
+<wire x1="73.66" y1="101.6" x2="71.12" y2="104.14" width="0.1524" layer="91"/>
+<pinref part="J1" gate="G$1" pin="TX+@2"/>
+<wire x1="71.12" y1="104.14" x2="58.42" y2="104.14" width="0.1524" layer="91"/>
+<pinref part="J1" gate="G$1" pin="TX+@1"/>
+<wire x1="58.42" y1="104.14" x2="58.42" y2="106.68" width="0.1524" layer="91"/>
+<junction x="58.42" y="104.14"/>
+<label x="60.96" y="104.14" size="1.778" layer="95"/>
+</segment>
 </net>
 <net name="USB-" class="0">
+<segment>
+<wire x1="124.46" y1="83.82" x2="127" y2="86.36" width="0.1524" layer="91"/>
+<pinref part="UWIFI" gate="G$1" pin="GND"/>
+<wire x1="127" y1="86.36" x2="129.54" y2="86.36" width="0.1524" layer="91"/>
+</segment>
 <segment>
 <wire x1="73.66" y1="86.36" x2="71.12" y2="88.9" width="0.1524" layer="91"/>
@@
 <wire x1="71.12" y1="88.9" x2="58.42" y2="88.9" width="0.1524" layer="91"/>
 <pinref part="J1" gate="G$1" pin="RX-@1"/>
-<wire x1="58.42" y1="88.9" x2="58.42" y2="91.44" width="0.1524" layer="91"/>
+<wire x1="58.42" y1="91.44" x2="58.42" y2="88.9" width="0.1524" layer="91"/>
 <junction x="58.42" y="88.9"/>
 <label x="60.96" y="88.9" size="1.778" layer="95"/>
 </segment>
-<segment>
-<wire x1="124.46" y1="83.82" x2="127" y2="86.36" width="0.1524" layer="91"/>
-<pinref part="UWIFI" gate="G$1" pin="GND"/>
-<wire x1="127" y1="86.36" x2="129.54" y2="86.36" width="0.1524" layer="91"/>
-</segment>
 </net>

Commit message: adding caps to wifi carrier
Parts:
- removed X2: (no value), con-wago-500:W237-102
- added C1, C2: 100n, rcl:C-EUC0603
- added C3: 1u, rcl:C-EUC0805
- added C4: 33u, rcl:C-EUC1206
- added X1: 5V, con-phoenix-254:MPT2
- R1, R2: device rcl:R-US_R0805 -> rcl:R-US_R0603
Connections:
- net GND: now also C1.2, C2.2, C3.2, C4.2, X1-2.1; no longer X2-2.KL
- net VCC: now also C1.1
- net VOUT: now also C2.1, C3.1, C4.1, X1-1.1; no longer X2-1.KL
Other:
- moved on the sheet: BOLT, BOLT1, BOLT2, BOLT3, CTRL, J1, R1, R2, U1, UWIFI, VBATT, VUSB
