File: av4/wifi-carrier/wifi-carrier.sch (EAGLE design)
At the start: 17 parts, among them J1 ROCKETNET-CONNECTOR-16M, U1 UEI15, X1 5V

Commit message: New cap for wifi-carrier, added it to its own library file and to the board.
Parts:
- added C5: 100u, cap-3024-7660:C-POL-7660
Connections:
- net GND: now also C5.-
- net VCC: now also C5.+
Changed lines of the file:
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@@
 <?xml version="1.0" encoding="utf-8"?>
 <!DOCTYPE eagle SYSTEM "eagle.dtd">
-<eagle version="6.4">
+<eagle version="6.5.0">
 <drawing>
 <settings>
@@
 <layers>
 <layer number="1" name="Top" color="4" fill="1" visible="no" active="no"/>
+<layer number="2" name="Route2" color="1" fill="3" visible="no" active="no"/>
+<layer number="3" name="Route3" color="4" fill="3" visible="no" active="no"/>
+<layer number="4" name="Route4" color="1" fill="4" visible="no" active="no"/>
+<layer number="5" name="Route5" color="4" fill="4" visible="no" active="no"/>
+<layer number="6" name="Route6" color="1" fill="8" visible="no" active="no"/>
+<layer number="7" name="Route7" color="4" fill="8" visible="no" active="no"/>
+<layer number="8" name="Route8" color="1" fill="2" visible="no" active="no"/>
+<layer number="9" name="Route9" color="4" fill="2" visible="no" active="no"/>
+<layer number="10" name="Route10" color="1" fill="7" visible="no" active="no"/>
+<layer number="11" name="Route11" color="4" fill="7" visible="no" active="no"/>
+<layer number="12" name="Route12" color="1" fill="5" visible="no" active="no"/>
+<layer number="13" name="Route13" color="4" fill="5" visible="no" active="no"/>
+<layer number="14" name="Route14" color="1" fill="6" visible="no" active="no"/>
+<layer number="15" name="Route15" color="4" fill="6" visible="no" active="no"/>
 <layer number="16" name="Bottom" color="1" fill="1" visible="no" active="no"/>
 <layer number="17" name="Pads" color="2" fill="1" visible="no" active="no"/>
@@
 <part name="C4" library="rcl" deviceset="C-EU" device="C1206" value="33u"/>
 <part name="X1" library="con-phoenix-254" deviceset="MPT2" device="" value="5V"/>
+<part name="C5" library="cap-3024-7660" deviceset="C-POL-7660" device="" value="100u"/>
 </parts>
 <sheets>
@@
 <instance part="X1" gate="-1" x="238.76" y="160.02"/>
 <instance part="X1" gate="-2" x="238.76" y="154.94"/>
+<instance part="C5" gate="G$1" x="66.04" y="154.94"/>
 </instances>
 <busses>
@@
 <wire x1="86.36" y1="137.16" x2="99.06" y2="137.16" width="0.1524" layer="91"/>
 <junction x="99.06" y="137.16"/>
+<pinref part="C5" gate="G$1" pin="-"/>
+<wire x1="66.04" y1="149.86" x2="66.04" y2="137.16" width="0.1524" layer="91"/>
+<wire x1="66.04" y1="137.16" x2="86.36" y2="137.16" width="0.1524" layer="91"/>
+<junction x="86.36" y="137.16"/>
 </segment>
 <segment>
@@
 <junction x="43.18" y="157.48"/>
 <pinref part="C1" gate="G$1" pin="1"/>
-<wire x1="86.36" y1="157.48" x2="43.18" y2="157.48" width="0.1524" layer="91"/>
+<wire x1="86.36" y1="157.48" x2="66.04" y2="157.48" width="0.1524" layer="91"/>
 <junction x="86.36" y="157.48"/>
-</segment>
-</net>
+<pinref part="C5" gate="G$1" pin="+"/>
+<wire x1="66.04" y1="157.48" x2="43.18" y2="157.48" width="0.1524" layer="91"/>
+<junction x="66.04" y="157.48"/>
+</segment>
+</net>

Commit message: More isolation on fasteners, better tplace/tname.
Parts:
- renumbered X1 to J2
Changed lines of the file:
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@@
 <?xml version="1.0" encoding="utf-8"?>
 <!DOCTYPE eagle SYSTEM "eagle.dtd">
-<eagle version="6.4">
+<eagle version="6.5.0">
 <drawing>
 <settings>
@@
 <part name="C3" library="rcl" deviceset="C-EU" device="C0805" value="1u"/>
 <part name="C4" library="rcl" deviceset="C-EU" device="C1206" value="33u"/>
-<part name="X1" library="con-phoenix-254" deviceset="MPT2" device="" value="5V"/>
+<part name="J2" library="con-phoenix-254" deviceset="MPT2" device="" value="5V"/>
 <part name="C5" library="cap-3024-7660" deviceset="C-POL-7660" device="" value="100u"/>
 </parts>
@@
 <instance part="C3" gate="G$1" x="182.88" y="157.48"/>
 <instance part="C4" gate="G$1" x="193.04" y="157.48"/>
-<instance part="X1" gate="-1" x="238.76" y="160.02"/>
-<instance part="X1" gate="-2" x="238.76" y="154.94"/>
+<instance part="J2" gate="-1" x="238.76" y="160.02"/>
+<instance part="J2" gate="-2" x="238.76" y="154.94"/>
 <instance part="C5" gate="G$1" x="66.04" y="154.94"/>
 </instances>
@@
 <pinref part="SUPPLY5" gate="GND" pin="GND"/>
 <wire x1="231.14" y1="154.94" x2="231.14" y2="134.62" width="0.1524" layer="91"/>
-<pinref part="X1" gate="-2" pin="1"/>
+<pinref part="J2" gate="-2" pin="1"/>
 <wire x1="236.22" y1="154.94" x2="231.14" y2="154.94" width="0.1524" layer="91"/>
 </segment>
@@
 <pinref part="C4" gate="G$1" pin="1"/>
 <junction x="193.04" y="160.02"/>
-<pinref part="X1" gate="-1" pin="1"/>
-</segment>
-</net>
+<pinref part="J2" gate="-1" pin="1"/>
+</segment>
+</net>
