File: av4/rocketnet-hub/eagle/mcu_page_combined_routed.brd (EAGLE design)
At the start: 112.7 x 76.2 mm, 449 parts, among them J1 ROCKETNET-CONNECTOR-16M, J10 UART Header, J11 I2C Header, J12 BOOT1 Jumper, J13 PGOOD Jumper, J14 ROCKETNET-UMBILICAL-18, J15 Auxiliary Header, J16 Auxiliary Header, J17 Auxiliary Header, J18 Auxiliary Header, J19 Auxiliary Header, J2 ROCKETNET-CONNECTOR-16M, J20 Auxiliary Header, J21 Auxiliary Header, J22 Debug Header, J3 ROCKETNET-CONNECTOR-16M, J4 ROCKETNET-CONNECTOR-16M, J5 BOOT0 Jumper, J6 ROCKETNET-CONNECTOR-16M, J7 ROCKETNET-CONNECTOR-16M, J8 ROCKETNET-CONNECTOR-16M, J9 ROCKETNET-BATTERY-14, Q1 NTR4101P, Q10 PMV45EN, Q2 FDS6680ASOIC8, Q3 FDS6680ASOIC8, Q4 FDS6680ASOIC8, Q5 SIS412DNSOP-8, Q6 BSS138W-7-F, Q7 SIS412DNSOP-8, Q8 PMV45EN, Q9 NTR4101P, T10 ALT4532, T11 ALT4532, T12 ALT4532, T13 ALT4532, T14 ALT4532, T15 ALT4532, T16 ALT4532, T17 ALT4532, T18 ALT4532, T3 ALT4532, T4 ALT4532, T5 ALT4532, T6 ALT4532, T7 ALT4532, T8 ALT4532, T9 ALT4532, U1 STM32F407V100-PIN_QFP, U10 TPS2420QFN-16, U11 TPS2420QFN-16, U12 TPS2420QFN-16, U13 TPS2420QFN-16, U14 MAX4734ETC+, U15 MAX4734ETC+, U2 BQ24725QFN-20, U3 SN65220DBV, U4 KS8999, U5 LTM8023, U6 MIC37101-2.1YM, U7 TPS2420QFN-16, U8 TPS2420QFN-16, U9 TPS2420QFN-16, X1 25 MHz

Commit message: Added "mods" to schematic: TP39 to GND, removed R10 and R14.
Parts:
- R10: value 0 -> NP
- R14: value 1k -> NP
Changed lines of the file:
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@@
 <?xml version="1.0" encoding="utf-8"?>
 <!DOCTYPE eagle SYSTEM "eagle.dtd">
-<eagle version="6.4">
+<eagle version="6.5.0">
 <drawing>
 <settings>
@@
 <grid distance="5" unitdist="mil" unit="mil" style="lines" multiple="1" display="yes" altdistance="0.1" altunitdist="mil" altunit="mil"/>
 <layers>
-<layer number="1" name="Top" color="4" fill="1" visible="yes" active="yes"/>
+<layer number="1" name="Top" color="4" fill="1" visible="no" active="yes"/>
 <layer number="2" name="GND" color="9" fill="1" visible="no" active="yes"/>
 <layer number="3" name="Power" color="12" fill="1" visible="no" active="yes"/>
@@
 <layer number="14" name="NS" color="15" fill="1" visible="no" active="yes"/>
 <layer number="15" name="EW" color="6" fill="1" visible="no" active="yes"/>
-<layer number="16" name="Bottom" color="1" fill="1" visible="no" active="yes"/>
+<layer number="16" name="Bottom" color="1" fill="1" visible="yes" active="yes"/>
 <layer number="17" name="Pads" color="2" fill="1" visible="yes" active="yes"/>
 <layer number="18" name="Vias" color="2" fill="1" visible="yes" active="yes"/>
 <layer number="19" name="Unrouted" color="6" fill="1" visible="yes" active="yes"/>
 <layer number="20" name="Dimension" color="15" fill="1" visible="yes" active="yes"/>
-<layer number="21" name="tPlace" color="7" fill="1" visible="yes" active="yes"/>
-<layer number="22" name="bPlace" color="7" fill="1" visible="no" active="yes"/>
-<layer number="23" name="tOrigins" color="15" fill="1" visible="yes" active="yes"/>
-<layer number="24" name="bOrigins" color="15" fill="1" visible="no" active="yes"/>
+<layer number="21" name="tPlace" color="7" fill="1" visible="no" active="yes"/>
+<layer number="22" name="bPlace" color="7" fill="1" visible="yes" active="yes"/>
+<layer number="23" name="tOrigins" color="15" fill="1" visible="no" active="yes"/>
+<layer number="24" name="bOrigins" color="15" fill="1" visible="yes" active="yes"/>
 <layer number="25" name="tNames" color="7" fill="1" visible="no" active="yes"/>
-<layer number="26" name="bNames" color="7" fill="1" visible="no" active="yes"/>
+<layer number="26" name="bNames" color="7" fill="1" visible="yes" active="yes"/>
 <layer number="27" name="tValues" color="7" fill="1" visible="no" active="yes"/>
 <layer number="28" name="bValues" color="7" fill="1" visible="no" active="yes"/>
@@
 <layer number="49" name="Reference" color="7" fill="1" visible="no" active="yes"/>
 <layer number="50" name="dxf" color="7" fill="1" visible="no" active="no"/>
-<layer number="51" name="tDocu" color="7" fill="1" visible="yes" active="yes"/>
-<layer number="52" name="bDocu" color="7" fill="1" visible="no" active="yes"/>
+<layer number="51" name="tDocu" color="7" fill="1" visible="no" active="yes"/>
+<layer number="52" name="bDocu" color="7" fill="1" visible="yes" active="yes"/>
 <layer number="53" name="tGND_GNDA" color="7" fill="1" visible="no" active="no"/>
 <layer number="54" name="bGND_GNDA" color="7" fill="1" visible="no" active="no"/>
@@
 <attribute name="VALUE" x="96.724" y="57.025" size="1" layer="27" ratio="10" rot="R180"/>
 </element>
-<element name="R10" library="rcl_custom" package="0402-B-NOSILK" value="0" x="95.219" y="57" smashed="yes" rot="MR90">
+<element name="R10" library="rcl_custom" package="0402-B-NOSILK" value="NP" x="95.219" y="57" smashed="yes" rot="MR90">
 <attribute name="NAME" x="95.8342" y="55.88" size="0.762" layer="26" ratio="20" rot="MR270"/>
 <attribute name="VALUE" x="93.369" y="56.2" size="1" layer="28" ratio="10" rot="MR90"/>
 </element>
-<element name="R14" library="rcl_custom" package="0402-B-NOSILK" value="1k" x="99.441" y="14.605" smashed="yes" rot="R180">
+<element name="R14" library="rcl_custom" package="0402-B-NOSILK" value="NP" x="99.441" y="14.605" smashed="yes" rot="R180">
 <attribute name="NAME" x="98.4812" y="15.196" size="0.762" layer="25" ratio="20"/>
 <attribute name="VALUE" x="100.241" y="16.455" size="1" layer="27" ratio="10" rot="R180"/>

Commit message: Added proposed patches to the RNH, including for the NODE8 bug and for the new LED Ethernet link detect.
Connections:
- removed net MRXER: TP39.TP, U1.47
- net GND: now also TP39.TP, U1.47
- net LED5-3: now also U1.43
- net NODE8_!EN: now also U1.38
- net NODE8_!FLT: now also U1.46
Routing:
- net GND: track 36.3 -> 37.4 mm
- net MRXER: track 1.16 -> 0.00 mm
Changed lines of the file:
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@@
 <grid distance="5" unitdist="mil" unit="mil" style="lines" multiple="1" display="yes" altdistance="0.1" altunitdist="mil" altunit="mil"/>
 <layers>
-<layer number="1" name="Top" color="4" fill="1" visible="no" active="yes"/>
+<layer number="1" name="Top" color="4" fill="1" visible="yes" active="yes"/>
 <layer number="2" name="GND" color="9" fill="1" visible="no" active="yes"/>
 <layer number="3" name="Power" color="12" fill="1" visible="no" active="yes"/>
@@
 <layer number="19" name="Unrouted" color="6" fill="1" visible="yes" active="yes"/>
 <layer number="20" name="Dimension" color="15" fill="1" visible="yes" active="yes"/>
-<layer number="21" name="tPlace" color="7" fill="1" visible="no" active="yes"/>
+<layer number="21" name="tPlace" color="7" fill="1" visible="yes" active="yes"/>
 <layer number="22" name="bPlace" color="7" fill="1" visible="yes" active="yes"/>
-<layer number="23" name="tOrigins" color="15" fill="1" visible="no" active="yes"/>
+<layer number="23" name="tOrigins" color="15" fill="1" visible="yes" active="yes"/>
 <layer number="24" name="bOrigins" color="15" fill="1" visible="yes" active="yes"/>
 <layer number="25" name="tNames" color="7" fill="1" visible="no" active="yes"/>
-<layer number="26" name="bNames" color="7" fill="1" visible="yes" active="yes"/>
+<layer number="26" name="bNames" color="7" fill="1" visible="no" active="yes"/>
 <layer number="27" name="tValues" color="7" fill="1" visible="no" active="yes"/>
 <layer number="28" name="bValues" color="7" fill="1" visible="no" active="yes"/>
@@
 <layer number="49" name="Reference" color="7" fill="1" visible="no" active="yes"/>
 <layer number="50" name="dxf" color="7" fill="1" visible="no" active="no"/>
-<layer number="51" name="tDocu" color="7" fill="1" visible="no" active="yes"/>
+<layer number="51" name="tDocu" color="7" fill="1" visible="yes" active="yes"/>
 <layer number="52" name="bDocu" color="7" fill="1" visible="yes" active="yes"/>
 <layer number="53" name="tGND_GNDA" color="7" fill="1" visible="no" active="no"/>
@@
 <layer number="98" name="Guide" color="6" fill="1" visible="no" active="no"/>
 <layer number="100" name="Muster" color="7" fill="1" visible="no" active="no"/>
-<layer number="101" name="Patch_Top" color="7" fill="1" visible="no" active="yes"/>
-<layer number="102" name="Vscore" color="7" fill="1" visible="no" active="yes"/>
-<layer number="103" name="tMap" color="7" fill="1" visible="no" active="yes"/>
-<layer number="104" name="Name" color="7" fill="1" visible="no" active="yes"/>
-<layer number="105" name="tPlate" color="7" fill="1" visible="no" active="yes"/>
-<layer number="106" name="bPlate" color="7" fill="1" visible="no" active="yes"/>
-<layer number="107" name="Crop" color="7" fill="1" visible="no" active="yes"/>
+<layer number="101" name="Patch_Top" color="11" fill="1" visible="yes" active="yes"/>
 <layer number="116" name="Patch_BOT" color="7" fill="1" visible="no" active="yes"/>
-<layer number="121" name="_tsilk" color="7" fill="1" visible="no" active="yes"/>
-<layer number="122" name="_bsilk" color="7" fill="1" visible="no" active="yes"/>
-<layer number="151" name="HeatSink" color="7" fill="1" visible="no" active="yes"/>
 <layer number="200" name="200bmp" color="1" fill="10" visible="no" active="no"/>
-<layer number="201" name="201bmp" color="7" fill="1" visible="no" active="yes"/>
-<layer number="202" name="202bmp" color="7" fill="1" visible="no" active="yes"/>
-<layer number="203" name="203bmp" color="7" fill="1" visible="no" active="yes"/>
-<layer number="204" name="204bmp" color="7" fill="1" visible="no" active="yes"/>
-<layer number="205" name="205bmp" color="7" fill="1" visible="no" active="yes"/>
-<layer number="206" name="206bmp" color="7" fill="1" visible="no" active="yes"/>
-<layer number="207" name="207bmp" color="7" fill="1" visible="no" active="yes"/>
-<layer number="208" name="208bmp" color="7" fill="1" visible="no" active="yes"/>
-<layer number="209" name="209bmp" color="8" fill="1" visible="no" active="yes"/>
-<layer number="210" name="210bmp" color="9" fill="1" visible="no" active="yes"/>
-<layer number="211" name="211bmp" color="12" fill="1" visible="no" active="yes"/>
-<layer number="212" name="212bmp" color="11" fill="1" visible="no" active="yes"/>
-<layer number="213" name="213bmp" color="12" fill="1" visible="no" active="yes"/>
-<layer number="214" name="214bmp" color="13" fill="1" visible="no" active="yes"/>
-<layer number="215" name="ResistanceBottom" color="7" fill="1" visible="no" active="yes"/>
-<layer number="216" name="216bmp" color="15" fill="1" visible="no" active="yes"/>
-<layer number="217" name="217bmp" color="16" fill="1" visible="no" active="yes"/>
-<layer number="218" name="218bmp" color="17" fill="1" visible="no" active="yes"/>
 <layer number="250" name="Descript" color="3" fill="1" visible="no" active="no"/>
 <layer number="251" name="SMDround" color="12" fill="11" visible="no" active="no"/>
-<layer number="254" name="cooling" color="7" fill="1" visible="no" active="yes"/>
 </layers>
 <board>
@@
 <text x="30.353" y="48.133" size="1.27" layer="21" ratio="18">JTAG</text>
 <text x="56.515" y="18.161" size="1.27" layer="21" ratio="18">v1.0 2013/06/17</text>
+<wire x1="52.959" y1="14.732" x2="52.959" y2="26.035" width="0.254" layer="101"/>
+<wire x1="52.959" y1="26.035" x2="59.309" y2="32.385" width="0.254" layer="101"/>
+<wire x1="59.309" y1="32.385" x2="57.658" y2="34.036" width="0.254" layer="101"/>
+<wire x1="80.772" y1="7.747" x2="77.343" y2="7.747" width="0.254" layer="101"/>
+<wire x1="77.343" y1="7.747" x2="76.2" y2="8.89" width="0.254" layer="101"/>
+<wire x1="76.2" y1="8.89" x2="76.2" y2="19.812" width="0.254" layer="101"/>
+<wire x1="76.2" y1="19.812" x2="61.341" y2="34.671" width="0.254" layer="101"/>
+<wire x1="61.341" y1="34.671" x2="60.198" y2="33.528" width="0.254" layer="101"/>
+<wire x1="60.198" y1="33.528" x2="58.547" y2="35.179" width="0.254" layer="101"/>
+<wire x1="78.867" y1="7.493" x2="79.502" y2="7.493" width="0.254" layer="101"/>
+<wire x1="79.502" y1="7.493" x2="79.502" y2="-0.254" width="0.254" layer="101"/>
+<wire x1="79.502" y1="-0.254" x2="78.105" y2="-0.254" width="0.254" layer="101"/>
+<wire x1="78.105" y1="-0.254" x2="78.105" y2="6.35" width="0.254" layer="101"/>
+<wire x1="78.105" y1="6.35" x2="75.819" y2="8.636" width="0.254" layer="101"/>
+<wire x1="75.819" y1="8.636" x2="75.819" y2="19.685" width="0.254" layer="101"/>
+<wire x1="75.819" y1="19.685" x2="66.675" y2="28.829" width="0.254" layer="101"/>
+<wire x1="66.675" y1="28.829" x2="59.309" y2="28.829" width="0.254" layer="101"/>
+<wire x1="59.309" y1="28.829" x2="55.753" y2="32.385" width="0.254" layer="101"/>
 </plain>
 <attributes>
@@
 <via x="19.558" y="57.658" extent="1-16" drill="0.2032" diameter="0.4572"/>
 <via x="12.954" y="17.907" extent="1-16" drill="0.2032" diameter="0.4572"/>
+<contactref element="U1" pad="47"/>
+<contactref element="TP39" pad="TP"/>
+<wire x1="58.67884375" y1="35.823115625" x2="59.309" y2="35.192959375" width="0.1778" layer="1"/>
+<wire x1="59.309" y1="35.192959375" x2="59.309" y2="34.925" width="0.1778" layer="1"/>
 </signal>
 <signal name="+3V3" class="1">
@@
 <wire x1="57.912" y1="15.24" x2="68.199" y2="25.527" width="0.1778" layer="14"/>
 <wire x1="28.321" y1="8.89" x2="27.293" y2="8.89" width="0.1778" layer="1"/>
+<contactref element="U1" pad="43"/>
+<wire x1="68.199" y1="25.527" x2="57.26463125" y2="34.4089" width="0" layer="19" extent="1-14"/>
 </signal>
 <signal name="LED6-3">
@@
 <wire x1="80.701" y1="8.693" x2="80.701" y2="7.818" width="0.1778" layer="16"/>
 <wire x1="80.701" y1="7.818" x2="80.772" y2="7.747" width="0.1778" layer="16"/>
+<contactref element="U1" pad="46"/>
+<wire x1="80.701" y1="8.693" x2="58.325290625" y2="35.4695625" width="0" layer="19" extent="1-16"/>
 </signal>
 <signal name="NODE8_!EN">
@@
 <wire x1="79.502" y1="7.62" x2="78.895" y2="7.62" width="0.1778" layer="16"/>
 <wire x1="78.895" y1="7.62" x2="78.867" y2="7.592" width="0.1778" layer="16"/>
+<contactref element="U1" pad="38"/>
+<wire x1="55.4968625" y1="32.641134375" x2="78.895" y2="7.62" width="0" layer="19" extent="1-16"/>
 </signal>
 <signal name="N$139">
@@
 <wire x1="47.879" y1="45.915853125" x2="47.879" y2="45.339" width="0.1778" layer="1"/>
 </signal>
-<signal name="MRXER">
-<contactref element="U1" pad="47"/>
-<contactref element="TP39" pad="TP"/>
-<wire x1="58.67884375" y1="35.823115625" x2="59.309" y2="35.192959375" width="0.1778" layer="1"/>
-<wire x1="59.309" y1="35.192959375" x2="59.309" y2="34.925" width="0.1778" layer="1"/>
-</signal>
 <signal name="N$254" class="1">
