File: av4/rocketnet-hub/eagle/mcu_page_combined_routed.sch (EAGLE design)
At the start: 444 parts, among them J1 ROCKETNET-CONNECTOR-16M, J10 UART Header, J11 I2C Header, J12 BOOT1 Jumper, J13 PGOOD Jumper, J14 ROCKETNET-UMBILICAL-18, J15 Auxiliary Header, J16 Auxiliary Header, J17 Auxiliary Header, J18 Auxiliary Header, J19 Auxiliary Header, J2 ROCKETNET-CONNECTOR-16M, J20 Auxiliary Header, J21 Auxiliary Header, J22 Debug Header, J3 ROCKETNET-CONNECTOR-16M, J4 ROCKETNET-CONNECTOR-16M, J5 BOOT0 Jumper, J6 ROCKETNET-CONNECTOR-16M, J7 ROCKETNET-CONNECTOR-16M, J8 ROCKETNET-CONNECTOR-16M, J9 ROCKETNET-BATTERY-14, Q1 NTR4101P, Q10 PMV45EN, Q2 FDS6680ASOIC8, Q3 FDS6680ASOIC8, Q4 FDS6680ASOIC8, Q5 SIS412DNSOP-8, Q6 BSS138W-7-F, Q7 SIS412DNSOP-8, Q8 PMV45EN, Q9 NTR4101P, T10 ALT4532, T11 ALT4532, T12 ALT4532, T13 ALT4532, T14 ALT4532, T15 ALT4532, T16 ALT4532, T17 ALT4532, T18 ALT4532, T3 ALT4532, T4 ALT4532, T5 ALT4532, T6 ALT4532, T7 ALT4532, T8 ALT4532, T9 ALT4532, U1 STM32F407V100-PIN_QFP, U10 TPS2420QFN-16, U11 TPS2420QFN-16, U12 TPS2420QFN-16, U13 TPS2420QFN-16, U14 MAX4734ETC+, U15 MAX4734ETC+, U2 BQ24725QFN-20, U3 SN65220DBV, U4 KS8999, U5 LTM8023, U6 MIC37101-2.1YM, U7 TPS2420QFN-16, U8 TPS2420QFN-16, U9 TPS2420QFN-16, X1 25 MHz

Commit message: Added "mods" to schematic: TP39 to GND, removed R10 and R14.
Other:
- note added: "CHANGE: NP"
- note added: "MODWIRE"
- note removed: "ETH_MII_RX_ER is being disabled (assumed Active High)"
Changed lines of the file:
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@@
 <?xml version="1.0" encoding="utf-8"?>
 <!DOCTYPE eagle SYSTEM "eagle.dtd">
-<eagle version="6.4">
+<eagle version="6.5.0">
 <drawing>
 <settings>
@@
 <setting verticaltext="up"/>
 </settings>
-<grid distance="0.05" unitdist="inch" unit="inch" style="lines" multiple="2" display="no" altdistance="0.01" altunitdist="inch" altunit="inch"/>
+<grid distance="0.05" unitdist="inch" unit="inch" style="lines" multiple="2" display="yes" altdistance="0.01" altunitdist="inch" altunit="inch"/>
 <layers>
 <layer number="1" name="Top" color="4" fill="1" visible="no" active="no"/>
@@
 <layer number="101" name="Patch_Top" color="12" fill="4" visible="yes" active="yes"/>
 <layer number="102" name="Vscore" color="7" fill="1" visible="yes" active="yes"/>
-<layer number="103" name="tMap" color="7" fill="1" visible="yes" active="yes"/>
 <layer number="104" name="Name" color="7" fill="1" visible="yes" active="yes"/>
-<layer number="105" name="tPlate" color="7" fill="1" visible="yes" active="yes"/>
-<layer number="106" name="bPlate" color="7" fill="1" visible="yes" active="yes"/>
 <layer number="107" name="Crop" color="7" fill="1" visible="yes" active="yes"/>
 <layer number="116" name="Patch_BOT" color="9" fill="4" visible="yes" active="yes"/>
-<layer number="121" name="_tsilk" color="7" fill="1" visible="yes" active="yes"/>
-<layer number="122" name="_bsilk" color="7" fill="1" visible="yes" active="yes"/>
-<layer number="151" name="HeatSink" color="7" fill="1" visible="yes" active="yes"/>
 <layer number="200" name="200bmp" color="1" fill="10" visible="no" active="no"/>
-<layer number="201" name="201bmp" color="7" fill="1" visible="yes" active="yes"/>
-<layer number="202" name="202bmp" color="7" fill="1" visible="yes" active="yes"/>
-<layer number="203" name="203bmp" color="7" fill="1" visible="yes" active="yes"/>
-<layer number="204" name="204bmp" color="7" fill="1" visible="yes" active="yes"/>
-<layer number="205" name="205bmp" color="7" fill="1" visible="yes" active="yes"/>
-<layer number="206" name="206bmp" color="7" fill="1" visible="yes" active="yes"/>
-<layer number="207" name="207bmp" color="7" fill="1" visible="yes" active="yes"/>
-<layer number="208" name="208bmp" color="7" fill="1" visible="yes" active="yes"/>
-<layer number="209" name="209bmp" color="8" fill="1" visible="yes" active="yes"/>
-<layer number="210" name="210bmp" color="9" fill="1" visible="yes" active="yes"/>
-<layer number="211" name="211bmp" color="12" fill="1" visible="yes" active="yes"/>
-<layer number="212" name="212bmp" color="11" fill="1" visible="yes" active="yes"/>
-<layer number="213" name="213bmp" color="12" fill="1" visible="yes" active="yes"/>
-<layer number="214" name="214bmp" color="13" fill="1" visible="yes" active="yes"/>
-<layer number="215" name="ResistanceBottom" color="7" fill="1" visible="yes" active="yes"/>
-<layer number="216" name="216bmp" color="15" fill="1" visible="no" active="yes"/>
-<layer number="217" name="217bmp" color="16" fill="1" visible="no" active="yes"/>
-<layer number="218" name="218bmp" color="17" fill="1" visible="no" active="yes"/>
 <layer number="250" name="Descript" color="3" fill="1" visible="no" active="no"/>
 <layer number="251" name="SMDround" color="12" fill="11" visible="no" active="no"/>
-<layer number="254" name="cooling" color="7" fill="1" visible="yes" active="yes"/>
 </layers>
 <schematic xreflabel="%F%N/%S.%C%R" xrefpart="/%S.%C%R">
@@
 <part name="R72" library="rcl_custom" deviceset="R-US_" device="0402-B-NOSILK" value="0"/>
 <part name="GND147" library="supply1" deviceset="GND" device=""/>
-<part name="GND148" library="supply1" deviceset="GND" device=""/>
 <part name="Q10" library="zetex" deviceset="NMOSSOT23" device="" value="PMV45EN"/>
 <part name="+3V41" library="supply1" deviceset="+3V3" device=""/>
@@
 <part name="GND151" library="supply1" deviceset="GND" device=""/>
 <part name="GND153" library="supply1" deviceset="GND" device=""/>
+<part name="GND17" library="supply1" deviceset="GND" device=""/>
 </parts>
 <sheets>
@@
 <wire x1="15.24" y1="378.46" x2="15.24" y2="414.02" width="0.1524" layer="95" style="shortdash"/>
 <text x="17.78" y="408.94" size="2.54" layer="95">UART Interface</text>
-<text x="-5.08" y="327.66" size="1.016" layer="95">ETH_MII_RX_ER is being disabled (assumed Active High)</text>
 <text x="38.1" y="322.58" size="1.016" layer="95">Ferrite bead position before/after capacitors</text>
+<wire x1="17.78" y1="342.9" x2="17.78" y2="353.06" width="0.1524" layer="101"/>
+<text x="16.51" y="342.9" size="1.778" layer="101" rot="R90">MODWIRE</text>
 </plain>
 <instances>
@@
 <instance part="R65" gate="R" x="198.12" y="388.62" rot="R90"/>
 <instance part="GND146" gate="1" x="198.12" y="381"/>
-<instance part="GND148" gate="1" x="17.78" y="332.74"/>
 <instance part="+3V42" gate="G$1" x="233.68" y="388.62"/>
 <instance part="TP39" gate="G$1" x="17.78" y="355.6"/>
@@
 <instance part="GND151" gate="1" x="137.16" y="307.34"/>
 <instance part="GND153" gate="1" x="124.46" y="307.34"/>
+<instance part="GND17" gate="1" x="17.78" y="340.36"/>
 </instances>
 <busses>
@@
 </segment>
 <segment>
-<pinref part="GND148" gate="1" pin="GND"/>
-<wire x1="17.78" y1="340.36" x2="17.78" y2="335.28" width="0.1524" layer="91"/>
-</segment>
-<segment>
 <pinref part="J11" gate="J" pin="GND"/>
 <wire x1="-5.08" y1="358.14" x2="-5.08" y2="353.06" width="0.1524" layer="91"/>
@@
 <wire x1="55.88" y1="170.18" x2="17.78" y2="170.18" width="0.1524" layer="97" style="shortdash"/>
 <text x="27.94" y="165.1" size="1.778" layer="97">Mode Select</text>
+<text x="201.93" y="20.32" size="1.778" layer="101" rot="R90">CHANGE: NP</text>
+<text x="49.53" y="72.39" size="1.778" layer="101" rot="R90">CHANGE: NP</text>
 </plain>
 <instances>
@@
 <instance part="GND71" gate="1" x="27.94" y="127"/>
 <instance part="R3" gate="R" x="66.04" y="78.74" rot="R180"/>
-<instance part="R10" gate="R" x="48.26" y="91.44" rot="R180"/>
+<instance part="R10" gate="R" x="48.26" y="91.44" smashed="yes" rot="R180">
+<attribute name="NAME" x="52.07" y="89.9414" size="1.778" layer="95" rot="R180"/>
+<attribute name="VALUE" x="52.07" y="87.122" size="1.778" layer="96" rot="R180"/>
+</instance>
 <instance part="GND72" gate="1" x="38.1" y="20.32"/>
 <instance part="R14" gate="R" x="195.58" y="30.48" rot="R90"/>

Commit message: Added proposed patches to the RNH, including for the NODE8 bug and for the new LED Ethernet link detect.
Parts:
- R10: value 0 -> NP
- R14: value 1k -> NP
Connections:
- removed net MRXER: TP39.TP, U1.PB10
- net GND: now also TP39.TP, U1.PB10
- net LED5-3: now also U1.PE12
- net NODE8_!EN: now also U1.PE7
- net NODE8_!FLT: now also U1.PE15
Other:
- note added: "Launch Detect"
- note added: "MODWIRE for Launch Detect"
Changed lines of the file:
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@@
 <setting verticaltext="up"/>
 </settings>
-<grid distance="0.05" unitdist="inch" unit="inch" style="lines" multiple="2" display="yes" altdistance="0.01" altunitdist="inch" altunit="inch"/>
+<grid distance="0.05" unitdist="inch" unit="inch" style="lines" multiple="2" display="no" altdistance="0.01" altunitdist="inch" altunit="inch"/>
 <layers>
 <layer number="1" name="Top" color="4" fill="1" visible="no" active="no"/>
@@
 <part name="GND71" library="supply1" deviceset="GND" device=""/>
 <part name="R3" library="rcl_custom" deviceset="R-US_" device="0402-B-NOSILK" value="0"/>
-<part name="R10" library="rcl_custom" deviceset="R-US_" device="0402-B-NOSILK" value="0"/>
+<part name="R10" library="rcl_custom" deviceset="R-US_" device="0402-B-NOSILK" value="NP"/>
 <part name="GND72" library="supply1" deviceset="GND" device=""/>
-<part name="R14" library="rcl_custom" deviceset="R-US_" device="0402-B-NOSILK" value="1k"/>
+<part name="R14" library="rcl_custom" deviceset="R-US_" device="0402-B-NOSILK" value="NP"/>
 <part name="+3V2" library="supply1" deviceset="+3V3" device=""/>
 <part name="TP28" library="testpad" deviceset="TP" device="TP06R"/>
@@
 <text x="17.78" y="408.94" size="2.54" layer="95">UART Interface</text>
 <text x="38.1" y="322.58" size="1.016" layer="95">Ferrite bead position before/after capacitors</text>
-<wire x1="17.78" y1="342.9" x2="17.78" y2="353.06" width="0.1524" layer="101"/>
-<text x="16.51" y="342.9" size="1.778" layer="101" rot="R90">MODWIRE</text>
+<text x="16.51" y="341.63" size="1.778" layer="101" rot="R90">MODWIRE</text>
+<text x="170.18" y="440.69" size="1.778" layer="101">MODWIRE for Launch Detect</text>
+<text x="170.18" y="453.39" size="1.778" layer="101">MODWIRE</text>
+<text x="170.18" y="433.07" size="1.778" layer="101">MODWIRE</text>
 </plain>
 <instances>
@@
 <junction x="137.16" y="312.42"/>
 </segment>
+<segment>
+<pinref part="U1" gate="U1" pin="PB10"/>
+<wire x1="63.5" y1="353.06" x2="17.78" y2="353.06" width="0.1524" layer="91"/>
+<pinref part="TP39" gate="G$1" pin="TP"/>
+<pinref part="GND17" gate="1" pin="GND"/>
+<wire x1="17.78" y1="342.9" x2="17.78" y2="353.06" width="0.1524" layer="91"/>
+<junction x="17.78" y="353.06"/>
+</segment>
 </net>
 <net name="+3V3" class="1">
@@
 </segment>
 </net>
-<net name="MRXER" class="0">
-<segment>
-<pinref part="U1" gate="U1" pin="PB10"/>
-<wire x1="63.5" y1="353.06" x2="17.78" y2="353.06" width="0.1524" layer="91"/>
-<pinref part="TP39" gate="G$1" pin="TP"/>
-</segment>
-</net>
 <net name="25MHZ_REF_CLK_KSZ" class="0">
 <segment>
@@
 </segment>
 </net>
+<net name="LED5-3" class="0">
+<segment>
+<wire x1="127" y1="444.5" x2="167.64" y2="444.5" width="0.1524" layer="91"/>
+<label x="167.64" y="444.5" size="1.778" layer="95" xref="yes"/>
+<pinref part="U1" gate="U1" pin="PE12"/>
+<wire x1="127" y1="444.5" x2="127" y2="434.34" width="0.1524" layer="91"/>
+</segment>
+</net>
+<net name="NODE8_!EN" class="0">
+<segment>
+<pinref part="U1" gate="U1" pin="PE7"/>
+<wire x1="114.3" y1="434.34" x2="114.3" y2="457.2" width="0.1524" layer="91"/>
+<wire x1="114.3" y1="457.2" x2="167.64" y2="457.2" width="0.1524" layer="91"/>
+<label x="167.64" y="457.2" size="1.778" layer="95" xref="yes"/>
+</segment>
+</net>
+<net name="NODE8_!FLT" class="0">
+<segment>
+<pinref part="U1" gate="U1" pin="PE15"/>
+<wire x1="134.62" y1="434.34" x2="134.62" y2="436.88" width="0.1524" layer="91"/>
+<wire x1="134.62" y1="436.88" x2="167.64" y2="436.88" width="0.1524" layer="91"/>
+<label x="167.64" y="436.88" size="1.778" layer="95" xref="yes"/>
+</segment>
+</net>
 </nets>
 </sheet>
@@
 <text x="201.93" y="20.32" size="1.778" layer="101" rot="R90">CHANGE: NP</text>
 <text x="49.53" y="72.39" size="1.778" layer="101" rot="R90">CHANGE: NP</text>
+<text x="278.13" y="133.35" size="1.778" layer="101">Launch Detect</text>
 </plain>
 <instances>
@@
 <pinref part="LED17" gate="G$1" pin="C"/>
 <wire x1="187.96" y1="134.62" x2="193.04" y2="134.62" width="0.1524" layer="91"/>
+<wire x1="193.04" y1="134.62" x2="193.04" y2="137.16" width="0.1524" layer="91"/>
+<junction x="193.04" y="134.62"/>
+<wire x1="193.04" y1="137.16" x2="279.4" y2="137.16" width="0.1524" layer="91"/>
+<label x="279.4" y="137.16" size="1.778" layer="95" xref="yes"/>
 </segment>
 </net>

Commit message: Latest patches on the RNH: added connections for port 8, added proposed umbilical disconect patch. Still to do: vbat, and a checklist to make sure we have both RNHs up to the same patch level.
Parts:
- added C58: 100n, rcl_custom:C-EU0402-B-NOSILK
- added R31: 100, rcl_custom:R-US_0402-B-NOSILK
- LED37: value RGB -> (none)
- R44: value 750 -> 110
- R45: value 750 -> 400
- R49, R52, R54, R56, R58, R60, R62: value TBD -> 69.8k
Connections:
- new net N$3: C58.1, R31.2, U1.PC13
- new net UMB-DETECT: J14.RR@10, R31.1
- net GND: now also C58.2
- net LED5-3: no longer U1.PE12
- net ROCKET_RDY: no longer J14.RR@10
Other:
- note added: "CUT + MODWIRE"
- note added: "PATCH"
- note added: "REPLACED BY SPS ON DAUGHTERBOARD"
- note added: "Umbilical Detect"
- note removed: "Launch Detect"
- note removed: "MODWIRE for Launch Detect"
- moved on the sheet: C1, C10, C100, C101, C102, C103, C104, C105, C106, C107, C108, C109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

Commit message: Connected Vbat to VDD, changed umb-detect to 1k from 100 ohms.
Parts:
- R31: value 100 -> 1k
Connections:
- net +3V3: now also U1.VBAT
Changed lines of the file:
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@@
 <?xml version="1.0" encoding="utf-8"?>
 <!DOCTYPE eagle SYSTEM "eagle.dtd">
-<eagle version="6.5.0">
+<eagle version="6.6.0">
 <drawing>
 <settings>
@@
 <part name="GND153" library="supply1" deviceset="GND" device=""/>
 <part name="GND17" library="supply1" deviceset="GND" device=""/>
-<part name="R31" library="rcl_custom" deviceset="R-US_" device="0402-B-NOSILK" value="100"/>
+<part name="R31" library="rcl_custom" deviceset="R-US_" device="0402-B-NOSILK" value="1k"/>
 <part name="GND94" library="supply1" deviceset="GND" device=""/>
 <part name="C58" library="rcl_custom" deviceset="C-EU" device="0402-B-NOSILK" value="100n"/>
@@
 <wire x1="106.68" y1="121.92" x2="106.68" y2="157.48" width="0.1524" layer="95" style="shortdash"/>
 <text x="109.22" y="152.4" size="2.54" layer="95">UART Interface</text>
-<text x="129.54" y="66.04" size="1.016" layer="95">Ferrite bead position before/after capacitors</text>
+<text x="142.24" y="60.96" size="1.016" layer="95">Ferrite bead position before/after capacitors</text>
 <text x="107.95" y="85.09" size="1.778" layer="101" rot="R90">MODWIRE</text>
 <text x="261.62" y="196.85" size="1.778" layer="101">MODWIRE</text>
@@
 <text x="337.82" y="50.8" size="1.778" layer="101">PATCH</text>
 <text x="360.68" y="60.96" size="1.778" layer="101">PATCH</text>
+<text x="156.21" y="64.77" size="1.778" layer="101" rot="R90">MODWIRE</text>
 </plain>
 <instances>
@@
 <pinref part="+3V1" gate="G$1" pin="+3V3"/>
 <wire x1="167.64" y1="71.12" x2="167.64" y2="68.58" width="0.1524" layer="91"/>
-<wire x1="167.64" y1="68.58" x2="167.64" y2="63.5" width="0.1524" layer="91"/>
 <pinref part="E5" gate="E" pin="1"/>
 <wire x1="167.64" y1="68.58" x2="170.18" y2="68.58" width="0.1524" layer="91"/>
@@
 <pinref part="C46" gate="CE" pin="1"/>
 <wire x1="175.26" y1="63.5" x2="167.64" y2="63.5" width="0.1524" layer="91"/>
+<wire x1="167.64" y1="63.5" x2="157.48" y2="63.5" width="0.1524" layer="91"/>
 <wire x1="175.26" y1="60.96" x2="175.26" y2="63.5" width="0.1524" layer="91"/>
 <junction x="175.26" y="63.5"/>
-</segment>
-<segment>
+<pinref part="U1" gate="U1" pin="VBAT"/>
+<wire x1="175.26" y1="71.12" x2="170.18" y2="71.12" width="0.1524" layer="91"/>
+<wire x1="170.18" y1="71.12" x2="170.18" y2="78.74" width="0.1524" layer="91"/>
+<wire x1="170.18" y1="78.74" x2="157.48" y2="78.74" width="0.1524" layer="91"/>
+<wire x1="157.48" y1="78.74" x2="157.48" y2="63.5" width="0.1524" layer="91"/>
+<wire x1="167.64" y1="68.58" x2="167.64" y2="63.5" width="0.1524" layer="91"/>
+<junction x="167.64" y="63.5"/>
+</segment>
+<segment>

Commit message: Changed name of umbilical patch to be active low.
Connections:
- net N$3 renamed !UMB_DETECT_MCU
- net UMB-DETECT renamed !UMB-DETECT
Changed lines of the file:
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@@
 <setting verticaltext="up"/>
 </settings>
-<grid distance="0.1" unitdist="inch" unit="inch" style="lines" multiple="1" display="no" altdistance="0.01" altunitdist="inch" altunit="inch"/>
+<grid distance="0.05" unitdist="inch" unit="inch" style="lines" multiple="2" display="no" altdistance="0.01" altunitdist="inch" altunit="inch"/>
 <layers>
 <layer number="1" name="Top" color="4" fill="1" visible="no" active="no"/>
@@
 </segment>
 </net>
-<net name="UMB-DETECT" class="0">
+<net name="!UMB-DETECT" class="0">
 <segment>
 <label x="388.62" y="55.88" size="1.778" layer="95" xref="yes"/>
@@
 </segment>
 </net>
-<net name="N$3" class="0">
+<net name="!UMB_DETECT_MCU" class="0">
 <segment>
 <pinref part="C58" gate="CE" pin="1"/>
@@
 </segment>
 </net>
-<net name="UMB-DETECT" class="0">
+<net name="!UMB-DETECT" class="0">
 <segment>
 <pinref part="J14" gate="G$1" pin="RR@10"/>
