File: av4/gps-carrier/gps-carrier.brd (EAGLE design)
At the start: 100 x 80 mm, 8 parts

Commit message: supercap for RAM backup
Parts:
- added C1: 10u, rcl:C0805
- added C2: 100p, rcl:C0603
- added D1: PMLL4150, diode:SOD80C
- added R1: 300, rcl:R0603
- added SUPERCAP: 220 mF, gps-carrier:DSK-HL
- renumbered GPS1 to COTSLNA, GPS2 to COTSGPS
Connections:
- new net BACKUPRAM: COTSGPS.4, D1.C, SUPERCAP.A
- new net N$1: D1.A, R1.2
- net GND: now also C1.2, C2.2, SUPERCAP.C
- net VCC: now also C1.1, C2.1, R1.1
Changed lines of the file:
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@@
 </autorouter>
 <elements>
-<element name="GPS1" library="GPS_Hemisphere" package="GPS_LNA" value="GPS_LNA" x="-53.34" y="52.07"/>
-<element name="GPS2" library="GPS_Hemisphere" package="GPS_CRECENT_OUTLINE" value="HEMISPHERE_GPS_MOUNT" x="-49.53" y="21.59"/>
+<element name="COTSLNA" library="GPS_Hemisphere" package="GPS_LNA" value="GPS_LNA" x="-53.34" y="52.07"/>
+<element name="COTSGPS" library="GPS_Hemisphere" package="GPS_CRECENT_OUTLINE" value="HEMISPHERE_GPS_MOUNT" x="-49.53" y="21.59"/>
 <element name="SV1" library="con-lstb" package="MA04-1" value="pow+uart" x="-59.69" y="85.09">
 <attribute name="OC_NEWARK" value="unknown" x="0" y="0" size="1.778" layer="27" display="off"/>
@@
 <element name="U$3" library="mount-2" package="_4/.325-BARE+SMALL_TOOL_CLEARANCE" value="_4-BARE_MOUNTING_HOLE/.325" x="-82.55" y="77.47"/>
 <element name="U$4" library="mount-2" package="_4/.325-BARE+SMALL_TOOL_CLEARANCE" value="_4-BARE_MOUNTING_HOLE/.325" x="-45.72" y="86.36"/>
+<element name="C1" library="rcl" package="C0805" value="10u" x="-91.44" y="-3.81"/>
+<element name="C2" library="rcl" package="C0603" value="100p" x="-91.44" y="-11.43"/>
+<element name="SUPERCAP" library="gps-carrier" package="DSK-HL" value="220 mF" x="-100.33" y="-5.08"/>
+<element name="D1" library="diode" package="SOD80C" value="PMLL4150" x="-101.6" y="-17.78"/>
+<element name="R1" library="rcl" package="R0603" value="300" x="-102.87" y="-24.13"/>
 </elements>
 <signals>
 <signal name="VCC">
-<contactref element="GPS2" pad="1"/>
-<contactref element="GPS2" pad="2"/>
-<contactref element="GPS2" pad="3"/>
+<contactref element="COTSGPS" pad="1"/>
+<contactref element="COTSGPS" pad="2"/>
+<contactref element="COTSGPS" pad="3"/>
 <contactref element="SV1" pad="4"/>
 <contactref element="SV2" pad="1"/>
+<contactref element="C2" pad="1"/>
+<contactref element="C1" pad="1"/>
+<contactref element="R1" pad="1"/>
+<wire x1="-92.29" y1="-11.43" x2="-103.72" y2="-24.13" width="0" layer="19" extent="1-1"/>
+<wire x1="-92.39" y1="-3.81" x2="-92.29" y2="-11.43" width="0" layer="19" extent="1-1"/>
+<wire x1="-82.296" y1="11.43" x2="-92.39" y2="-3.81" width="0" layer="19" extent="1-1"/>
 <wire x1="-82.296" y1="12.7" x2="-82.296" y2="11.43" width="0" layer="19" extent="1-1"/>
 <wire x1="-78.994" y1="11.43" x2="-82.296" y2="11.43" width="0" layer="19" extent="1-1"/>
@@
 </signal>
 <signal name="GND">
-<contactref element="GPS2" pad="28"/>
-<contactref element="GPS2" pad="27"/>
-<contactref element="GPS2" pad="7"/>
-<contactref element="GPS2" pad="8"/>
+<contactref element="COTSGPS" pad="28"/>
+<contactref element="COTSGPS" pad="27"/>
+<contactref element="COTSGPS" pad="7"/>
+<contactref element="COTSGPS" pad="8"/>
 <contactref element="SV1" pad="1"/>
 <contactref element="SV2" pad="8"/>
+<contactref element="C2" pad="2"/>
+<contactref element="C1" pad="2"/>
+<contactref element="SUPERCAP" pad="C"/>
+<wire x1="-90.59" y1="-11.43" x2="-100.33" y2="-10.08" width="0" layer="19" extent="1-1"/>
+<wire x1="-90.49" y1="-3.81" x2="-90.59" y2="-11.43" width="0" layer="19" extent="1-1"/>
+<wire x1="-82.296" y1="15.24" x2="-90.49" y2="-3.81" width="0" layer="19" extent="1-1"/>
 <wire x1="-78.994" y1="15.24" x2="-82.296" y2="15.24" width="0" layer="19" extent="1-1"/>
 <wire x1="-82.296" y1="27.94" x2="-82.296" y2="15.24" width="0" layer="19" extent="1-1"/>
@@
 </signal>
 <signal name="PORTA_TX">
-<contactref element="GPS2" pad="9"/>
+<contactref element="COTSGPS" pad="9"/>
 <contactref element="SV1" pad="3"/>
 <wire x1="-58.42" y1="85.09" x2="-82.296" y2="16.51" width="0" layer="19" extent="1-1"/>
 </signal>
 <signal name="PORTA_RX">
-<contactref element="GPS2" pad="10"/>
+<contactref element="COTSGPS" pad="10"/>
 <contactref element="SV1" pad="2"/>
 <wire x1="-60.96" y1="85.09" x2="-78.994" y2="16.51" width="0" layer="19" extent="1-1"/>
@@
 <signal name="PPS">
 <contactref element="SV2" pad="7"/>
-<contactref element="GPS2" pad="15"/>
+<contactref element="COTSGPS" pad="15"/>
 <wire x1="-15.24" y1="66.04" x2="-82.296" y2="20.32" width="0" layer="19" extent="1-1"/>
 </signal>
 <signal name="LOCK">
 <contactref element="SV2" pad="5"/>
-<contactref element="GPS2" pad="17"/>
+<contactref element="COTSGPS" pad="17"/>
 <wire x1="-17.78" y1="66.04" x2="-82.296" y2="21.59" width="0" layer="19" extent="1-1"/>
 </signal>
 <signal name="DIFF_LOCK">
-<contactref element="GPS2" pad="18"/>
+<contactref element="COTSGPS" pad="18"/>
 <contactref element="SV2" pad="3"/>
 <wire x1="-20.32" y1="66.04" x2="-78.994" y2="21.59" width="0" layer="19" extent="1-1"/>
 </signal>
 <signal name="DGPS">
-<contactref element="GPS2" pad="19"/>
+<contactref element="COTSGPS" pad="19"/>
 <contactref element="SV2" pad="2"/>
 <wire x1="-22.86" y1="68.58" x2="-82.296" y2="22.86" width="0" layer="19" extent="1-1"/>
 </signal>
 <signal name="ALARM">
-<contactref element="GPS2" pad="30"/>
+<contactref element="COTSGPS" pad="30"/>
 <contactref element="SV2" pad="6"/>
 <wire x1="-17.78" y1="68.58" x2="-78.994" y2="29.21" width="0" layer="19" extent="1-1"/>
 </signal>
+<signal name="BACKUPRAM">
+<contactref element="SUPERCAP" pad="A"/>
+<contactref element="COTSGPS" pad="4"/>
+<contactref element="D1" pad="C"/>
+<wire x1="-100.33" y1="-0.08" x2="-103.3" y2="-17.78" width="0" layer="19" extent="1-1"/>
+<wire x1="-78.994" y1="12.7" x2="-100.33" y2="-0.08" width="0" layer="19" extent="1-1"/>
+</signal>
+<signal name="N$1">
+<contactref element="R1" pad="2"/>
+<contactref element="D1" pad="A"/>
+<wire x1="-99.9" y1="-17.78" x2="-102.02" y2="-24.13" width="0" layer="19" extent="1-1"/>
+</signal>
 </signals>

Commit message: New GPS board layout, trying it in the real world.
Parts:
- moved R1 150.4 mm to (18.7, 64.5), turned to 180 degrees
- moved D1 144.5 mm to (14.0, 69.0)
- moved C1 135.3 mm to (22.8, 68.8)
- moved C2 135.3 mm to (22.8, 61.2)
- moved SUPERCAP 129.5 mm to (12.5, 58.4), turned to 90 degrees
- moved U$2 125.7 mm to (57.0, 5.00)
- moved U$1 116.0 mm to (57.0, 88.0)
- moved COTSLNA 103.5 mm to (50.0, 46.0), turned to 90 degrees
- moved U$4 95.9 mm to (5.00, 5.00)
- moved U$3 88.2 mm to (5.00, 88.0)
- moved COTSGPS 76.5 mm to (23.0, 46.0), turned to 270 degrees
- moved SV1 76.4 mm to (16.7, 87.6), turned to 180 degrees
- moved SV2 64.5 mm to (42.3, 87.3), turned to 90 degrees
Other:
- board size 100 x 80 mm -> 62 x 93 mm

Commit message: GPS carrier board for AV4. Should be ready for fab.
Parts:
- U$1, U$2, U$3, U$4: value _4-BARE_MOUNTING_HOLE/.325 -> #4-BARE_MOUNTING_HOLE/.300; device mount-2:_4/.325-BARE+SMALL_TOOL_CLEARANCE -> mount:#4/.300-BARE+STD_NUT_OR_STAR_WASHER
- moved C2 22.5 mm to (13.8, 81.8)
- moved C1 11.1 mm to (11.8, 70.8), turned to 180 degrees
- moved SUPERCAP 8.99 mm to (20.6, 62.3)
- moved R1 6.92 mm to (12.8, 68.2), turned to 270 degrees
- moved D1 5.14 mm to (12.8, 64.0), turned to 90 degrees
- moved SV2 0.61 mm to (42.9, 87.4), turned to 270 degrees
- moved U$1 0.50 mm to (56.5, 88.0)
- moved U$2 0.50 mm to (56.5, 5.00)
- moved U$3 0.50 mm to (5.50, 88.0)
- moved U$4 0.50 mm to (5.50, 5.00)
- moved SV1 0.14 mm to (16.6, 87.5)
Connections:
- net PORTA_TX renamed PARTA_TX
- new net N$2: COTSGPS.34, SV2.5
- net DGPS: now also SV2.4; no longer SV2.2
- net DIFF_LOCK: now also SV2.7; no longer SV2.3
- net LOCK: now also SV2.3; no longer SV2.5
- net PPS: now also SV2.2; no longer SV2.7
Routing:
- net VCC: track 0.00 -> 65.2 mm
- net DIFF_LOCK: track 0.00 -> 32.5 mm, vias 0 -> 1
- net PPS: track 0.00 -> 32.4 mm
- net DGPS: track 0.00 -> 27.6 mm
- net ALARM: track 0.00 -> 27.0 mm, vias 0 -> 1
- net LOCK: track 0.00 -> 26.9 mm
- net PORTA_RX: track 0.00 -> 22.7 mm, vias 0 -> 1
- net N$2: track 0.00 -> 18.3 mm, vias 0 -> 1
- net BACKUPRAM: track 0.00 -> 16.6 mm
- net PARTA_TX: track 0.00 -> 9.81 mm
- net N$1: track 0.00 -> 1.73 mm
- added copper zone on layer 1, net GND
- added copper zone on layer 16, net GND
Other:
- outline, holes or cut-outs redrawn
- board text added: "3.3V"
- board text added: "GND"
- board text added: "RX"
- board text added: "TX"
